Commit message: Add zed cameras and additional params for sensors

File: cetc_sat_urdf/urdf/cetc_sat.urdf (robot description, URDF)
Before this commit: robot cetc_sat, 125 links, 124 joints
Links:
- removed link D435_front1_accel_frame
- removed link D435_front1_accel_optical_frame
- removed link D435_front1_bottom_screw_frame
- removed link D435_front1_color_frame
- removed link D435_front1_color_optical_frame
- removed link D435_front1_depth_frame
- removed link D435_front1_depth_optical_frame
- removed link D435_front1_gyro_frame
- removed link D435_front1_gyro_optical_frame
- removed link D435_front1_left_ir_frame
- removed link D435_front1_left_ir_optical_frame
- removed link D435_front1_link
- removed link D435_front1_right_ir_frame
- removed link D435_front1_right_ir_optical_frame
- removed link D435_front2_accel_frame
- removed link D435_front2_accel_optical_frame
- removed link D435_front2_bottom_screw_frame
- removed link D435_front2_color_frame
- removed link D435_front2_color_optical_frame
- removed link D435_front2_depth_frame
- removed link D435_front2_depth_optical_frame
- removed link D435_front2_gyro_frame
- removed link D435_front2_gyro_optical_frame
- removed link D435_front2_left_ir_frame
- removed link D435_front2_left_ir_optical_frame
- removed link D435_front2_link
- removed link D435_front2_right_ir_frame
- removed link D435_front2_right_ir_optical_frame
- removed link D435_left_accel_frame
- removed link D435_left_accel_optical_frame
- removed link D435_left_bottom_screw_frame
- removed link D435_left_color_frame
- removed link D435_left_color_optical_frame
- removed link D435_left_depth_frame
- removed link D435_left_depth_optical_frame
- removed link D435_left_gyro_frame
- removed link D435_left_gyro_optical_frame
- removed link D435_left_left_ir_frame
- removed link D435_left_left_ir_optical_frame
- removed link D435_left_link
- removed link D435_left_right_ir_frame
- removed link D435_left_right_ir_optical_frame
- removed link D435_right_accel_frame
- removed link D435_right_accel_optical_frame
- removed link D435_right_bottom_screw_frame
- removed link D435_right_color_frame
- removed link D435_right_color_optical_frame
- removed link D435_right_depth_frame
- removed link D435_right_depth_optical_frame
- removed link D435_right_gyro_frame
- removed link D435_right_gyro_optical_frame
- removed link D435_right_left_ir_frame
- removed link D435_right_left_ir_optical_frame
- removed link D435_right_link
- removed link D435_right_right_ir_frame
- removed link D435_right_right_ir_optical_frame
- removed link velodyne
- removed link velodyne_base_link
- added link zedx_front1_baro_link
- added link zedx_front1_camera_center, mass 0.16140; collision box size=0.094 0.030 0.037; visual box size=0.030 0.094 0.037
- added link zedx_front1_left_camera_frame
- added link zedx_front1_left_camera_optical_frame
- added link zedx_front1_mag_link
- added link zedx_front1_right_camera_frame
- added link zedx_front1_right_camera_optical_frame
- added link zedx_front1_temp_left_link
- added link zedx_front1_temp_right_link
- added link zedx_front2_baro_link
- added link zedx_front2_camera_center, mass 0.16140; collision box size=0.094 0.030 0.037; visual box size=0.030 0.094 0.037
- added link zedx_front2_left_camera_frame
- added link zedx_front2_left_camera_optical_frame
- added link zedx_front2_mag_link
- added link zedx_front2_right_camera_frame
- added link zedx_front2_right_camera_optical_frame
- added link zedx_front2_temp_left_link
- added link zedx_front2_temp_right_link
- added link zedx_left_baro_link
- added link zedx_left_camera_center, mass 0.16140; collision box size=0.094 0.030 0.037; visual box size=0.030 0.094 0.037
- added link zedx_left_left_camera_frame
- added link zedx_left_left_camera_optical_frame
- added link zedx_left_mag_link
- added link zedx_left_right_camera_frame
- added link zedx_left_right_camera_optical_frame
- added link zedx_left_temp_left_link
- added link zedx_left_temp_right_link
- added link zedx_right_baro_link
- added link zedx_right_camera_center, mass 0.16140; collision box size=0.094 0.030 0.037; visual box size=0.030 0.094 0.037
- added link zedx_right_left_camera_frame
- added link zedx_right_left_camera_optical_frame
- added link zedx_right_mag_link
- added link zedx_right_right_camera_frame
- added link zedx_right_right_camera_optical_frame
- added link zedx_right_temp_left_link
- added link zedx_right_temp_right_link
Joints:
- removed joint D435_front1_accel_joint
- removed joint D435_front1_accel_optical_joint
- removed joint D435_front1_color_joint
- removed joint D435_front1_color_optical_joint
- removed joint D435_front1_depth_joint
- removed joint D435_front1_depth_optical_joint
- removed joint D435_front1_gyro_joint
- removed joint D435_front1_gyro_optical_joint
- removed joint D435_front1_joint
- removed joint D435_front1_left_ir_joint
- removed joint D435_front1_left_ir_optical_joint
- removed joint D435_front1_link_joint
- removed joint D435_front1_right_ir_joint
- removed joint D435_front1_right_ir_optical_joint
- removed joint D435_front2_accel_joint
- removed joint D435_front2_accel_optical_joint
- removed joint D435_front2_color_joint
- removed joint D435_front2_color_optical_joint
- removed joint D435_front2_depth_joint
- removed joint D435_front2_depth_optical_joint
- removed joint D435_front2_gyro_joint
- removed joint D435_front2_gyro_optical_joint
- removed joint D435_front2_joint
- removed joint D435_front2_left_ir_joint
- removed joint D435_front2_left_ir_optical_joint
- removed joint D435_front2_link_joint
- removed joint D435_front2_right_ir_joint
- removed joint D435_front2_right_ir_optical_joint
- removed joint D435_left_accel_joint
- removed joint D435_left_accel_optical_joint
- removed joint D435_left_color_joint
- removed joint D435_left_color_optical_joint
- removed joint D435_left_depth_joint
- removed joint D435_left_depth_optical_joint
- removed joint D435_left_gyro_joint
- removed joint D435_left_gyro_optical_joint
- removed joint D435_left_joint
- removed joint D435_left_left_ir_joint
- removed joint D435_left_left_ir_optical_joint
- removed joint D435_left_link_joint
- removed joint D435_left_right_ir_joint
- removed joint D435_left_right_ir_optical_joint
- removed joint D435_right_accel_joint
- removed joint D435_right_accel_optical_joint
- removed joint D435_right_color_joint
- removed joint D435_right_color_optical_joint
- removed joint D435_right_depth_joint
- removed joint D435_right_depth_optical_joint
- removed joint D435_right_gyro_joint
- removed joint D435_right_gyro_optical_joint
- removed joint D435_right_joint
- removed joint D435_right_left_ir_joint
- removed joint D435_right_left_ir_optical_joint
- removed joint D435_right_link_joint
- removed joint D435_right_right_ir_joint
- removed joint D435_right_right_ir_optical_joint
- removed joint velodyne_base_mount_joint
- removed joint velodyne_base_scan_joint
- added joint zedx_front1_baro_joint: type fixed, parent zedx_front1_camera_center, child zedx_front1_baro_link, origin xyz=0 0 0 rpy=0 0 0
- added joint zedx_front1_base_joint: type fixed, parent pelvis, child zedx_front1_camera_center, origin xyz=0.40 0.065 0 rpy=-1.57 0 0.5
- added joint zedx_front1_left_camera_joint: type fixed, parent zedx_front1_camera_center, child zedx_front1_left_camera_frame, origin xyz=0 0.025 0 rpy=0 0 0
- added joint zedx_front1_left_camera_optical_joint: type fixed, parent zedx_front1_left_camera_frame, child zedx_front1_left_camera_optical_frame, origin xyz=0 0 0 rpy=-1.5707963267948966 0.0 -1.5707963267948966
- added joint zedx_front1_mag_joint: type fixed, parent zedx_front1_camera_center, child zedx_front1_mag_link, origin xyz=0 0 0 rpy=0 0 0
- added joint zedx_front1_right_camera_joint: type fixed, parent zedx_front1_camera_center, child zedx_front1_right_camera_frame, origin xyz=0 -0.025 0 rpy=0 0 0
- added joint zedx_front1_right_camera_optical_joint: type fixed, parent zedx_front1_right_camera_frame, child zedx_front1_right_camera_optical_frame, origin xyz=0 0 0 rpy=-1.5707963267948966 0.0 -1.5707963267948966
- added joint zedx_front1_temp_left_joint: type fixed, parent zedx_front1_left_camera_frame, child zedx_front1_temp_left_link, origin xyz=0 0 0 rpy=0 0 0
- added joint zedx_front1_temp_right_joint: type fixed, parent zedx_front1_right_camera_frame, child zedx_front1_temp_right_link, origin xyz=0 0 0 rpy=0 0 0
- added joint zedx_front2_baro_joint: type fixed, parent zedx_front2_camera_center, child zedx_front2_baro_link, origin xyz=0 0 0 rpy=0 0 0
- added joint zedx_front2_base_joint: type fixed, parent pelvis, child zedx_front2_camera_center, origin xyz=0.40 -0.065 0 rpy=-1.57 0 -0.5
- added joint zedx_front2_left_camera_joint: type fixed, parent zedx_front2_camera_center, child zedx_front2_left_camera_frame, origin xyz=0 0.025 0 rpy=0 0 0
- added joint zedx_front2_left_camera_optical_joint: type fixed, parent zedx_front2_left_camera_frame, child zedx_front2_left_camera_optical_frame, origin xyz=0 0 0 rpy=-1.5707963267948966 0.0 -1.5707963267948966
- added joint zedx_front2_mag_joint: type fixed, parent zedx_front2_camera_center, child zedx_front2_mag_link, origin xyz=0 0 0 rpy=0 0 0
- added joint zedx_front2_right_camera_joint: type fixed, parent zedx_front2_camera_center, child zedx_front2_right_camera_frame, origin xyz=0 -0.025 0 rpy=0 0 0
- added joint zedx_front2_right_camera_optical_joint: type fixed, parent zedx_front2_right_camera_frame, child zedx_front2_right_camera_optical_frame, origin xyz=0 0 0 rpy=-1.5707963267948966 0.0 -1.5707963267948966
- added joint zedx_front2_temp_left_joint: type fixed, parent zedx_front2_left_camera_frame, child zedx_front2_temp_left_link, origin xyz=0 0 0 rpy=0 0 0
- added joint zedx_front2_temp_right_joint: type fixed, parent zedx_front2_right_camera_frame, child zedx_front2_temp_right_link, origin xyz=0 0 0 rpy=0 0 0
- added joint zedx_left_baro_joint: type fixed, parent zedx_left_camera_center, child zedx_left_baro_link, origin xyz=0 0 0 rpy=0 0 0
- added joint zedx_left_base_joint: type fixed, parent pelvis, child zedx_left_camera_center, origin xyz=-0.175 0.22 0 rpy=0 0.35 1.57
- added joint zedx_left_left_camera_joint: type fixed, parent zedx_left_camera_center, child zedx_left_left_camera_frame, origin xyz=0 0.025 0 rpy=0 0 0
- added joint zedx_left_left_camera_optical_joint: type fixed, parent zedx_left_left_camera_frame, child zedx_left_left_camera_optical_frame, origin xyz=0 0 0 rpy=-1.5707963267948966 0.0 -1.5707963267948966
- added joint zedx_left_mag_joint: type fixed, parent zedx_left_camera_center, child zedx_left_mag_link, origin xyz=0 0 0 rpy=0 0 0
- added joint zedx_left_right_camera_joint: type fixed, parent zedx_left_camera_center, child zedx_left_right_camera_frame, origin xyz=0 -0.025 0 rpy=0 0 0
- added joint zedx_left_right_camera_optical_joint: type fixed, parent zedx_left_right_camera_frame, child zedx_left_right_camera_optical_frame, origin xyz=0 0 0 rpy=-1.5707963267948966 0.0 -1.5707963267948966
- added joint zedx_left_temp_left_joint: type fixed, parent zedx_left_left_camera_frame, child zedx_left_temp_left_link, origin xyz=0 0 0 rpy=0 0 0
- added joint zedx_left_temp_right_joint: type fixed, parent zedx_left_right_camera_frame, child zedx_left_temp_right_link, origin xyz=0 0 0 rpy=0 0 0
- added joint zedx_right_baro_joint: type fixed, parent zedx_right_camera_center, child zedx_right_baro_link, origin xyz=0 0 0 rpy=0 0 0
- added joint zedx_right_base_joint: type fixed, parent pelvis, child zedx_right_camera_center, origin xyz=-0.175 -0.22 0 rpy=0 0.35 -1.57
- added joint zedx_right_left_camera_joint: type fixed, parent zedx_right_camera_center, child zedx_right_left_camera_frame, origin xyz=0 0.025 0 rpy=0 0 0
- added joint zedx_right_left_camera_optical_joint: type fixed, parent zedx_right_left_camera_frame, child zedx_right_left_camera_optical_frame, origin xyz=0 0 0 rpy=-1.5707963267948966 0.0 -1.5707963267948966
- added joint zedx_right_mag_joint: type fixed, parent zedx_right_camera_center, child zedx_right_mag_link, origin xyz=0 0 0 rpy=0 0 0
- added joint zedx_right_right_camera_joint: type fixed, parent zedx_right_camera_center, child zedx_right_right_camera_frame, origin xyz=0 -0.025 0 rpy=0 0 0
- added joint zedx_right_right_camera_optical_joint: type fixed, parent zedx_right_right_camera_frame, child zedx_right_right_camera_optical_frame, origin xyz=0 0 0 rpy=-1.5707963267948966 0.0 -1.5707963267948966
- added joint zedx_right_temp_left_joint: type fixed, parent zedx_right_left_camera_frame, child zedx_right_temp_left_link, origin xyz=0 0 0 rpy=0 0 0
- added joint zedx_right_temp_right_joint: type fixed, parent zedx_right_right_camera_frame, child zedx_right_temp_right_link, origin xyz=0 0 0 rpy=0 0 0
- joint hip_pitch_1: origin xyz=0.0 0.0 0.0 rpy=0.0 0.0 0.0 -> xyz=0.0 -0.0 0.0 rpy=0.0 0.0 0.0
- joint hip_pitch_2: origin xyz=0.0 -0.0 0.0 rpy=0.0 0.0 0.0 -> xyz=0.0 0.0 0.0 rpy=0.0 0.0 0.0
- joint hip_pitch_3: origin xyz=0.0 0.0 0.0 rpy=0.0 0.0 0.0 -> xyz=0.0 -0.0 0.0 rpy=0.0 0.0 0.0
- joint hip_pitch_4: origin xyz=0.0 -0.0 0.0 rpy=0.0 0.0 0.0 -> xyz=0.0 0.0 0.0 rpy=0.0 0.0 0.0

File: cetc_sat_urdf/urdf/cetc_sat_base.urdf.xacro (robot description, xacro)
@@ -36,48 +36,68 @@
     <origin xyz="0 0 0" rpy="0 0 0" />
 </joint>
-<xacro:if value="${ADD_SENSORS}">
+<xacro:if value="${ADD_REALSENSES}">
     <xacro:include filename="$(find realsense_gazebo_description)/urdf/_d435i.urdf.xacro" />
-    <!-- LEFT D435 CAMERA -->
-    <xacro:sensor_d435i parent="pelvis"
-        name="D435_left"
-        topics_ns="D435_left"
-        enable_pointCloud="true"
-        align_depth="true"
-        unite_imu_method="false"
-        visualize="true"
-        accel_fps="300"
-        gyro_fps="300"
-        depth_width="1280"
-        depth_height="720"
-        depth_fps="90"
-        infra_width="1280"
-        infra_height="720"
-        infra_fps="90"
-        color_width="1280"
-        color_height="720"
-        color_fps="30">
-        <origin xyz="-0.175 0.22 0" rpy="0 0.35 1.57"/>
-    </xacro:sensor_d435i>
-    <!-- RIGHT D435 CAMERA -->
-    <xacro:sensor_d435i parent="pelvis"
-        name="D435_right"
-        topics_ns="D435_right"
-        enable_pointCloud="true"
-        align_depth="true"
-        unite_imu_method="false"
-        visualize="true"
-        accel_fps="300"
-        gyro_fps="300"
-        depth_width="1280"
-        depth_height="720"
-        depth_fps="90"
-        infra_width="1280"
-        infra_height="720"
-        infra_fps="90"
-        color_width="1280"
-        color_height="720"
-        color_fps="30">
-        <origin xyz="-0.175 -0.22 0" rpy="0 0.35 -1.57"/>
-    </xacro:sensor_d435i>
+    <xacro:include filename="$(find realsense_gazebo_description)/urdf/_d455.urdf.xacro" />
+    <xacro:include filename="$(find cetc_sat_urdf)/urdf/parts/zed.urdf.xacro" />
+    <xacro:if value="${ADD_LATERAL_REALSENSE}">
+        <!-- LEFT D435 CAMERA -->
+        <xacro:sensor_d435i parent="pelvis"
+            name="D435_left"
+            topics_ns="D435_left"
+            enable_pointCloud="true"
+            align_depth="true"
+            unite_imu_method="false"
+            visualize="true"
+            accel_fps="300"
+            gyro_fps="300"
+            depth_width="1280"
+            depth_height="720"
+            depth_fps="90"
+            infra_width="1280"
+            infra_height="720"
+            infra_fps="90"
+            color_width="1280"
+            color_height="720"
+            color_fps="30">
+            <origin xyz="-0.175 0.22 0" rpy="0 0.35 1.57"/>
+        </xacro:sensor_d435i>
+        <!-- RIGHT D435 CAMERA -->
+        <xacro:sensor_d435i parent="pelvis"
+            name="D435_right"
+            topics_ns="D435_right"
+            enable_pointCloud="true"
+            align_depth="true"
+            unite_imu_method="false"
+            visualize="true"
+            accel_fps="300"
+            gyro_fps="300"
+            depth_width="1280"
+            depth_height="720"
+            depth_fps="90"
+            infra_width="1280"
+            infra_height="720"
+            infra_fps="90"
+            color_width="1280"
+            color_height="720"
+            color_fps="30">
+            <origin xyz="-0.175 -0.22 0" rpy="0 0.35 -1.57"/>
+        </xacro:sensor_d435i>
+    </xacro:if>
+    <xacro:if value="${ADD_LATERAL_ZED}">
+        <xacro:zed_x
+                name="zedx_left"
+                parent="pelvis">
+            <origin xyz="-0.175 0.22 0" rpy="0 0.35 1.57"/>
+        </xacro:zed_x>
+        <xacro:zed_x_gazebo
+                name="zedx_left"/>
+        <xacro:zed_x
+                name="zedx_right"
+                parent="pelvis">
+            <origin xyz="-0.175 -0.22 0" rpy="0 0.35 -1.57"/>
+        </xacro:zed_x>
+        <xacro:zed_x_gazebo
+                name="zedx_right"/>
+    </xacro:if>
     <!-- REAR D435 CAMERA -->
     <xacro:sensor_d435i parent="pelvis"
@@ -101,46 +121,106 @@
         <origin xyz="-0.39 0 0" rpy="0 0.35 3.14"/>
     </xacro:sensor_d435i>
-    <!-- FRONT1 D435 CAMERA -->
-    <xacro:sensor_d435i parent="pelvis"
-        name="D435_front1"
-        topics_ns="D435_front1"
-        enable_pointCloud="true"
-        align_depth="true"
-        unite_imu_method="false"
-        visualize="true"
-        accel_fps="300"
-        gyro_fps="300"
-        depth_width="1280"
-        depth_height="720"
-        depth_fps="90"
-        infra_width="1280"
-        infra_height="720"
-        infra_fps="90"
-        color_width="1280"
-        color_height="720"
-        color_fps="30">
-        <origin xyz="0.40 -0.08 0" rpy="-1.57 0 0.34"/>
-    </xacro:sensor_d435i>
-    <!-- FRONT2 D435 CAMERA -->
-    <xacro:sensor_d435i parent="pelvis"
-        name="D435_front2"
-        topics_ns="D435_front2"
-        enable_pointCloud="true"
-        align_depth="true"
-        unite_imu_method="false"
-        visualize="true"
-        accel_fps="300"
-        gyro_fps="300"
-        depth_width="1280"
-        depth_height="720"
-        depth_fps="90"
-        infra_width="1280"
-        infra_height="720"
-        infra_fps="90"
-        color_width="1280"
-        color_height="720"
-        color_fps="30">
-        <origin xyz="0.40 0.08 0" rpy="-1.57 0 -0.34"/>
-    </xacro:sensor_d435i>
+    <xacro:if value="${ADD_FRONT_D435}">
+        <!-- FRONT1 D435 CAMERA -->
+        <xacro:sensor_d435i parent="pelvis"
+            name="D435_front1"
+            topics_ns="D435_front1"
+            enable_pointCloud="true"
+            align_depth="true"
+            unite_imu_method="false"
+            visualize="true"
+            accel_fps="300"
+            gyro_fps="300"
+            depth_width="1280"
+            depth_height="720"
+            depth_fps="90"
+            infra_width="1280"
+            infra_height="720"
+            infra_fps="90"
+            color_width="1280"
+            color_height="720"
+            color_fps="30">
+            <origin xyz="0.40 -0.065 0" rpy="-1.57 0 0.5"/>
+        </xacro:sensor_d435i>
+        <!-- FRONT2 D435 CAMERA -->
+        <xacro:sensor_d435i parent="pelvis"
+            name="D435_front2"
+            topics_ns="D435_front2"
+            enable_pointCloud="true"
+            align_depth="true"
+            unite_imu_method="false"
+            visualize="true"
+            accel_fps="300"
+            gyro_fps="300"
+            depth_width="1280"
+            depth_height="720"
+            depth_fps="90"
+            infra_width="1280"
+            infra_height="720"
+            infra_fps="90"
+            color_width="1280"
+            color_height="720"
+            color_fps="30">
+            <origin xyz="0.40 0.065 -0.01" rpy="-1.57 0 -0.5"/>
+        </xacro:sensor_d435i>
+    </xacro:if>
+    <xacro:if value="${ADD_FRONT_D455}">
+        <xacro:sensor_d455 parent="pelvis"
+            name="D455_front1"
+            topics_ns="D455_front1"
+            enable_pointCloud="true"
+            align_depth="true"
+            unite_imu_method="false"
+            visualize="true"
+            accel_fps="300"
+            gyro_fps="300"
+            depth_width="1280"
+            depth_height="720"
+            depth_fps="90"
+            infra_width="1280"
+            infra_height="720"
+            infra_fps="90"
+            color_width="1280"
+            color_height="720"
+            color_fps="30">
+            <origin xyz="0.40 0.065 0" rpy="-1.57 0 0.4"/>
+        </xacro:sensor_d455>
+        <xacro:sensor_d455 parent="pelvis"
+            name="D455_front2"
+            topics_ns="D455_front2"
+            enable_pointCloud="true"
+            align_depth="true"
+            unite_imu_method="false"
+            visualize="true"
+            accel_fps="300"
+            gyro_fps="300"
+            depth_width="1280"
+            depth_height="720"
+            depth_fps="90"
+            infra_width="1280"
+            infra_height="720"
+            infra_fps="90"
+            color_width="1280"
+            color_height="720"
+            color_fps="30">
+            <origin xyz="0.40 0.06 0" rpy="-1.57 0 -0.4"/>
+        </xacro:sensor_d455>
+    </xacro:if>
+    <xacro:if value="${ADD_FRONT_ZED}">
+        <xacro:zed_x
+        name="zedx_front1"
+        parent="pelvis">
+            <origin xyz="0.40 0.065 0" rpy="-1.57 0 0.5"/>
+        </xacro:zed_x>
+        <xacro:zed_x_gazebo
+                name="zedx_front1"/>
+        <xacro:zed_x
+        name="zedx_front2"
+        parent="pelvis">
+            <origin xyz="0.40 -0.065 0" rpy="-1.57 0 -0.5"/>
+        </xacro:zed_x>
+        <xacro:zed_x_gazebo
+                name="zedx_front2"/>
+    </xacro:if>
     <!-- FRONT3 (down) D435 CAMERA -->
     <xacro:sensor_d435i parent="pelvis"
@@ -164,5 +244,7 @@
         <origin xyz="0.37 0 -0.11" rpy="0 0.75 0"/>
     </xacro:sensor_d435i>
-    <!-- Velodyne -->
+</xacro:if>
+<xacro:if value="${ADD_VELODYNE}">
+<!-- Velodyne -->
     <xacro:include filename="$(find velodyne_description)/urdf/VLP-16.urdf.xacro"/>
     <xacro:VLP-16 parent="pelvis" name="velodyne" topic="/velodyne_points" hz="10" samples="440">
