Commit message: Add zed cameras and additional params for sensors

File: cetc_sat_urdf/urdf/config/cetc_sat.urdf.xacro (robot description, xacro)
@@ -7,10 +7,22 @@
 <xacro:arg name="upper_body" default="true"/>
 <xacro:arg name="floating_joint" default="true"/>
-<xacro:arg name="sensors" default="true"/>
+<xacro:arg name="velodyne" default="false"/>
+<xacro:arg name="realsenses" default="true"/>
+<xacro:arg name="front_d435" default="false"/>
+<xacro:arg name="front_d455" default="false"/>
+<xacro:arg name="front_zed" default="true"/>
+<xacro:arg name="lateral_realsense" default="false"/>
+<xacro:arg name="lateral_zed" default="true"/>
 <!-- ************SELECT PARTS*************-->
 <!-- *************************************-->
 <xacro:property name="ADD_LEGS" value="$(arg legs)" />
 <xacro:property name="ADD_UPPER_BODY" value="$(arg upper_body)" />
-<xacro:property name="ADD_SENSORS" value="$(arg sensors)" />
+<xacro:property name="ADD_VELODYNE" value="$(arg velodyne)" />
+<xacro:property name="ADD_REALSENSES" value="$(arg realsenses)" />
+<xacro:property name="ADD_FRONT_D435" value="$(arg front_d435)" />
+<xacro:property name="ADD_FRONT_D455" value="$(arg front_d455)" />
+<xacro:property name="ADD_FRONT_ZED" value="$(arg front_zed)" />
+<xacro:property name="ADD_LATERAL_REALSENSE" value="$(arg lateral_realsense)" />
+<xacro:property name="ADD_LATERAL_ZED" value="$(arg lateral_zed)" />
 <xacro:property name="ADD_FLOATING_BASE" value="$(arg floating_joint)" />
 <xacro:property name="ADD_VIRTUAL_FRAME" value="false" />

Commit message: Update zed depth cutoff and rotation

File: cetc_sat_urdf/urdf/cetc_sat.urdf (robot description, URDF)
Before this commit: robot cetc_sat, 103 links, 102 joints
Joints:
- joint zedx_front1_base_joint: origin xyz=0.40 0.065 0 rpy=-1.57 0 0.5 -> xyz=0.40 0.065 0 rpy=-1.57 0 -0.5
- joint zedx_front2_base_joint: origin xyz=0.40 -0.065 0 rpy=-1.57 0 -0.5 -> xyz=0.40 -0.065 0 rpy=-1.57 0 0.5

File: cetc_sat_urdf/urdf/cetc_sat_base.urdf.xacro (robot description, xacro)
@@ -211,5 +211,5 @@
         name="zedx_front1"
         parent="pelvis">
-            <origin xyz="0.40 0.065 0" rpy="-1.57 0 0.5"/>
+            <origin xyz="0.40 0.065 0" rpy="-1.57 0 -0.5"/>
         </xacro:zed_x>
         <xacro:zed_x_gazebo
@@ -218,5 +218,5 @@
         name="zedx_front2"
         parent="pelvis">
-            <origin xyz="0.40 -0.065 0" rpy="-1.57 0 -0.5"/>
+            <origin xyz="0.40 -0.065 0" rpy="-1.57 0 0.5"/>
         </xacro:zed_x>
         <xacro:zed_x_gazebo

File: cetc_sat_urdf/urdf/parts/zed.urdf.xacro (robot description, xacro)
@@ -135,5 +135,5 @@
           <Cx>648.5</Cx>
           <Cy>366.8340148925781</Cy>
-          <hackBaseline>0.0</hackBaseline>
+          <hackBaseline>0.05</hackBaseline>
         </plugin>
       </sensor>
@@ -151,5 +151,5 @@
           </image>
           <clip>
-            <near>0.1</near>
+            <near>0.10</near>
             <far>10</far>
           </clip>
@@ -167,6 +167,6 @@
           <depthImageInfoTopicName>depth/camera_info</depthImageInfoTopicName>
           <pointCloudTopicName>point_cloud/cloud_registered</pointCloudTopicName>
-          <pointCloudCutoff>0.3</pointCloudCutoff>
-          <pointCloudCutoffMax>20.0</pointCloudCutoffMax>
+          <pointCloudCutoff>0.1</pointCloudCutoff>
+          <pointCloudCutoffMax>10.0</pointCloudCutoffMax>
           <frameName>${name}_left_camera_optical_frame</frameName>
           <baseline>0.05</baseline>
@@ -174,5 +174,5 @@
           <Cx>658.8206787109375</Cx>
           <Cy>372.25787353515625</Cy>
-          <hackBaseline>0.0</hackBaseline>
+          <hackBaseline>0.05</hackBaseline>
         </plugin>
       </sensor>
@@ -193,5 +193,5 @@
           </image>
           <clip>
-            <near>0.1</near>
+            <near>0.10</near>
             <far>10</far>
           </clip>
@@ -239,5 +239,5 @@
           </image>
           <clip>
-            <near>0.1</near>
+            <near>0.10</near>
             <far>10</far>
           </clip>

Commit message: changed masses. moved legs' pitch motors in the same position

File: cetc_sat_urdf/urdf/cetc_sat.urdf (robot description, URDF)
Before this commit: robot cetc_sat, 125 links, 124 joints
Links:
- removed link D435_front1_accel_frame
- removed link D435_front1_accel_optical_frame
- removed link D435_front1_bottom_screw_frame
- removed link D435_front1_color_frame
- removed link D435_front1_color_optical_frame
- removed link D435_front1_depth_frame
- removed link D435_front1_depth_optical_frame
- removed link D435_front1_gyro_frame
- removed link D435_front1_gyro_optical_frame
- removed link D435_front1_left_ir_frame
- removed link D435_front1_left_ir_optical_frame
- removed link D435_front1_link
- removed link D435_front1_right_ir_frame
- removed link D435_front1_right_ir_optical_frame
- removed link D435_front2_accel_frame
- removed link D435_front2_accel_optical_frame
- removed link D435_front2_bottom_screw_frame
- removed link D435_front2_color_frame
- removed link D435_front2_color_optical_frame
- removed link D435_front2_depth_frame
- removed link D435_front2_depth_optical_frame
- removed link D435_front2_gyro_frame
- removed link D435_front2_gyro_optical_frame
- removed link D435_front2_left_ir_frame
- removed link D435_front2_left_ir_optical_frame
- removed link D435_front2_link
- removed link D435_front2_right_ir_frame
- removed link D435_front2_right_ir_optical_frame
- removed link D435_front3_accel_frame
- removed link D435_front3_accel_optical_frame
- removed link D435_front3_bottom_screw_frame
- removed link D435_front3_color_frame
- removed link D435_front3_color_optical_frame
- removed link D435_front3_depth_frame
- removed link D435_front3_depth_optical_frame
- removed link D435_front3_gyro_frame
- removed link D435_front3_gyro_optical_frame
- removed link D435_front3_left_ir_frame
- removed link D435_front3_left_ir_optical_frame
- removed link D435_front3_link
- removed link D435_front3_right_ir_frame
- removed link D435_front3_right_ir_optical_frame
- removed link D435_left_accel_frame
- removed link D435_left_accel_optical_frame
- removed link D435_left_bottom_screw_frame
- removed link D435_left_color_frame
- removed link D435_left_color_optical_frame
- removed link D435_left_depth_frame
- removed link D435_left_depth_optical_frame
- removed link D435_left_gyro_frame
- removed link D435_left_gyro_optical_frame
- removed link D435_left_left_ir_frame
- removed link D435_left_left_ir_optical_frame
- removed link D435_left_link
- removed link D435_left_right_ir_frame
- removed link D435_left_right_ir_optical_frame
- removed link D435_rear_accel_frame
- removed link D435_rear_accel_optical_frame
- removed link D435_rear_bottom_screw_frame
- removed link D435_rear_color_frame
- removed link D435_rear_color_optical_frame
- removed link D435_rear_depth_frame
- removed link D435_rear_depth_optical_frame
- removed link D435_rear_gyro_frame
- removed link D435_rear_gyro_optical_frame
- removed link D435_rear_left_ir_frame
- removed link D435_rear_left_ir_optical_frame
- removed link D435_rear_link
- removed link D435_rear_right_ir_frame
- removed link D435_rear_right_ir_optical_frame
- removed link D435_right_accel_frame
- removed link D435_right_accel_optical_frame
- removed link D435_right_bottom_screw_frame
- removed link D435_right_color_frame
- removed link D435_right_color_optical_frame
- removed link D435_right_depth_frame
- removed link D435_right_depth_optical_frame
- removed link D435_right_gyro_frame
- removed link D435_right_gyro_optical_frame
- removed link D435_right_left_ir_frame
- removed link D435_right_left_ir_optical_frame
- removed link D435_right_link
- removed link D435_right_right_ir_frame
- removed link D435_right_right_ir_optical_frame
- removed link velodyne
- removed link velodyne_base_link
- link ball_1: mass 3 -> 0.1
- link ball_2: mass 3 -> 0.1
- link ball_3: mass 3 -> 0.1
- link ball_4: mass 3 -> 0.1
- link ball_arm_1: mass 3 -> 0.1
- link ball_arm_2: mass 3 -> 0.1
- link elbow_pitch_motor_1: mass 5 -> 1.8
- link elbow_pitch_motor_2: mass 5 -> 1.8
- link hip_pitch_motor_1: mass 5 -> 1.8
- link hip_pitch_motor_2: mass 5 -> 1.8
- link hip_pitch_motor_3: mass 5 -> 1.8
- link hip_pitch_motor_4: mass 5 -> 1.8
- link hip_roll_motor_1: mass 5 -> 1.8
- link hip_roll_motor_2: mass 5 -> 1.8
- link hip_roll_motor_3: mass 5 -> 1.8
- link hip_roll_motor_4: mass 5 -> 1.8
- link knee_pitch_motor_1: mass 5 -> 1.8
- link knee_pitch_motor_2: mass 5 -> 1.8
- link knee_pitch_motor_3: mass 5 -> 1.8
- link knee_pitch_motor_4: mass 5 -> 1.8
- link lower_arm_1: mass 5 -> 2.0
- link lower_arm_2: mass 5 -> 2.0
- link lower_leg_1: mass 3 -> 1.0
- link lower_leg_2: mass 3 -> 1.0
- link lower_leg_3: mass 3 -> 1.0
- link lower_leg_4: mass 3 -> 1.0
- link pelvis: mass 10 -> 14
- link shoulder_pitch_motor_1: mass 5 -> 1.8
- link shoulder_pitch_motor_2: mass 5 -> 1.8
- link shoulder_yaw_motor_1: mass 5 -> 1.8
- link shoulder_yaw_motor_2: mass 5 -> 1.8
- link upper_arm_1: mass 3 -> 1.0
- link upper_arm_2: mass 3 -> 1.0
- link upper_leg_1: mass 5 -> 2.0
- link upper_leg_2: mass 5 -> 2.0
- link upper_leg_3: mass 5 -> 2.0
- link upper_leg_4: mass 5 -> 2.0
Joints:
- removed joint D435_front1_accel_joint
- removed joint D435_front1_accel_optical_joint
- removed joint D435_front1_color_joint
- removed joint D435_front1_color_optical_joint
- removed joint D435_front1_depth_joint
- removed joint D435_front1_depth_optical_joint
- removed joint D435_front1_gyro_joint
- removed joint D435_front1_gyro_optical_joint
- removed joint D435_front1_joint
- removed joint D435_front1_left_ir_joint
- removed joint D435_front1_left_ir_optical_joint
- removed joint D435_front1_link_joint
- removed joint D435_front1_right_ir_joint
- removed joint D435_front1_right_ir_optical_joint
- removed joint D435_front2_accel_joint
- removed joint D435_front2_accel_optical_joint
- removed joint D435_front2_color_joint
- removed joint D435_front2_color_optical_joint
- removed joint D435_front2_depth_joint
- removed joint D435_front2_depth_optical_joint
- removed joint D435_front2_gyro_joint
- removed joint D435_front2_gyro_optical_joint
- removed joint D435_front2_joint
- removed joint D435_front2_left_ir_joint
- removed joint D435_front2_left_ir_optical_joint
- removed joint D435_front2_link_joint
- removed joint D435_front2_right_ir_joint
- removed joint D435_front2_right_ir_optical_joint
- removed joint D435_front3_accel_joint
- removed joint D435_front3_accel_optical_joint
- removed joint D435_front3_color_joint
- removed joint D435_front3_color_optical_joint
- removed joint D435_front3_depth_joint
- removed joint D435_front3_depth_optical_joint
- removed joint D435_front3_gyro_joint
- removed joint D435_front3_gyro_optical_joint
- removed joint D435_front3_joint
- removed joint D435_front3_left_ir_joint
- removed joint D435_front3_left_ir_optical_joint
- removed joint D435_front3_link_joint
- removed joint D435_front3_right_ir_joint
- removed joint D435_front3_right_ir_optical_joint
- removed joint D435_left_accel_joint
- removed joint D435_left_accel_optical_joint
- removed joint D435_left_color_joint
- removed joint D435_left_color_optical_joint
- removed joint D435_left_depth_joint
- removed joint D435_left_depth_optical_joint
- removed joint D435_left_gyro_joint
- removed joint D435_left_gyro_optical_joint
- removed joint D435_left_joint
- removed joint D435_left_left_ir_joint
- removed joint D435_left_left_ir_optical_joint
- removed joint D435_left_link_joint
- removed joint D435_left_right_ir_joint
- removed joint D435_left_right_ir_optical_joint
- removed joint D435_rear_accel_joint
- removed joint D435_rear_accel_optical_joint
- removed joint D435_rear_color_joint
- removed joint D435_rear_color_optical_joint
- removed joint D435_rear_depth_joint
- removed joint D435_rear_depth_optical_joint
- removed joint D435_rear_gyro_joint
- removed joint D435_rear_gyro_optical_joint
- removed joint D435_rear_joint
- removed joint D435_rear_left_ir_joint
- removed joint D435_rear_left_ir_optical_joint
- removed joint D435_rear_link_joint
- removed joint D435_rear_right_ir_joint
- removed joint D435_rear_right_ir_optical_joint
- removed joint D435_right_accel_joint
- removed joint D435_right_accel_optical_joint
- removed joint D435_right_color_joint
- removed joint D435_right_color_optical_joint
- removed joint D435_right_depth_joint
- removed joint D435_right_depth_optical_joint
- removed joint D435_right_gyro_joint
- removed joint D435_right_gyro_optical_joint
- removed joint D435_right_joint
- removed joint D435_right_left_ir_joint
- removed joint D435_right_left_ir_optical_joint
- removed joint D435_right_link_joint
- removed joint D435_right_right_ir_joint
- removed joint D435_right_right_ir_optical_joint
- removed joint velodyne_base_mount_joint
- removed joint velodyne_base_scan_joint
- joint hip_pitch_1: origin xyz=0.0 0.0 0.0 rpy=0.0 0.0 0.0 -> xyz=0.0 -0.0 0.0 rpy=0.0 0.0 0.0
- joint hip_pitch_2: origin xyz=0.0 -0.0 0.0 rpy=0.0 0.0 0.0 -> xyz=0.0 0.0 0.0 rpy=0.0 0.0 0.0
- joint hip_pitch_3: origin xyz=0.0 0.0 0.0 rpy=0.0 0.0 0.0 -> xyz=0.0 -0.0 0.0 rpy=0.0 0.0 0.0
- joint hip_pitch_4: origin xyz=0.0 -0.0 0.0 rpy=0.0 0.0 0.0 -> xyz=0.0 0.0 0.0 rpy=0.0 0.0 0.0

File: cetc_sat_urdf/urdf/parts/cetc_sat_leg.urdf.xacro (robot description, xacro)
@@ -44,4 +44,24 @@
 	</collision>
 </link>
+<link name="knee_pitch_motor_${leg_num}">
+	<inertial>
+		<origin xyz="0.0 0.0 0.0"/>
+		<mass value="${props_inertial['motorA_mass']}"/>
+		<inertia ixx="${MotorA_xx}" ixy="${MotorA_xy}" ixz="${MotorA_xz}" iyy="${MotorA_yy}" iyz="${MotorA_yz}" izz="${MotorA_zz}"/>
+	</inertial>
+	<visual>
+		<origin xyz="0.0 0.0 0.0"  rpy="0.0 0.0 0.0"/>
+	  	<geometry>
+	 		<cylinder radius="${props['cylinder_radius']}" length="${props['cylinder_length']}"/>
+	  	</geometry>
+  		<material name="dark_grey"/>
+	</visual>
+	<collision>
+		<origin xyz="0.0 0.0 0.0"  rpy="0.0 0.0 0.0"/>
+		<geometry>
+			<cylinder radius="${props['cylinder_radius']}" length="${props['cylinder_length']}"/>
+		</geometry>
+	</collision>
+</link>
 <link name="upper_leg_${leg_num}">
 	<inertial>
@@ -62,24 +82,4 @@
 		<geometry>
 			<box size="${props['big_box_length']} ${props['big_box_width']} ${props['big_box_height']}"/>
-		</geometry>
-	</collision>
-</link>
-<link name="knee_pitch_motor_${leg_num}">
-	<inertial>
-		<origin xyz="0.0 0.0 0.0"/>
-		<mass value="${props_inertial['motorA_mass']}"/>
-		<inertia ixx="${MotorA_xx}" ixy="${MotorA_xy}" ixz="${MotorA_xz}" iyy="${MotorA_yy}" iyz="${MotorA_yz}" izz="${MotorA_zz}"/>
-	</inertial>
-	<visual>
-		<origin xyz="0.0 0.0 0.0"  rpy="0.0 0.0 0.0"/>
-	  	<geometry>
-	 		<cylinder radius="${props['cylinder_radius']}" length="${props['cylinder_length']}"/>
-	  	</geometry>
-  		<material name="dark_grey"/>
-	</visual>
-	<collision>
-		<origin xyz="0.0 0.0 0.0"  rpy="0.0 0.0 0.0"/>
-		<geometry>
-			<cylinder radius="${props['cylinder_radius']}" length="${props['cylinder_length']}"/>
 		</geometry>
 	</collision>
@@ -137,4 +137,9 @@
 	<origin xyz="${HipPitch_Ox} ${mirror * (HipPitch_Oy)} ${HipPitch_Oz}" rpy="${HipPitch_roll} ${HipPitch_pitch} ${HipPitch_yaw}"/>
 </joint>
+<joint name="knee_pitch_stator_${leg_num}" type="fixed">
+	<parent link="hip_pitch_motor_${leg_num}"/>
+	<child link="knee_pitch_motor_${leg_num}"/>
+	<origin xyz="${KneePitch_Ox} ${KneePitch_Oy} ${KneePitch_Oz}" rpy="${KneePitch_roll} ${KneePitch_pitch} ${KneePitch_yaw}"/>
+</joint>
 <joint name="hip_pitch_${leg_num}" type="revolute">
 	<parent link="hip_pitch_motor_${leg_num}"/>
@@ -144,11 +149,6 @@
    <limit lower="${hip_pitch_lower[leg_num-1]}" upper="${hip_pitch_upper[leg_num-1]}" effort="${motor_A_effort}" velocity="${motor_A_velocity}"/> <!-- 200 Nm, 1 rad/s-->
 </joint>
-<joint name="knee_pitch_stator_${leg_num}" type="fixed">
+<joint name="knee_pitch_${leg_num}" type="revolute">
 	<parent link="upper_leg_${leg_num}"/>
-	<child link="knee_pitch_motor_${leg_num}"/>
-	<origin xyz="${KneePitch_Ox} ${KneePitch_Oy} ${KneePitch_Oz}" rpy="${KneePitch_roll} ${KneePitch_pitch} ${KneePitch_yaw}"/>
-</joint>
-<joint name="knee_pitch_${leg_num}" type="revolute">
-	<parent link="knee_pitch_motor_${leg_num}"/>
 	<child link="lower_leg_${leg_num}"/>
 	<origin xyz="${LowerLeg_Ox} ${LowerLeg_Oy} ${LowerLeg_Oz}" rpy="${LowerLeg_roll} ${LowerLeg_pitch} ${LowerLeg_yaw}"/>

File: cetc_sat_urdf/urdf/parts/kinematics_properties.urdf.xacro (robot description, xacro)
@@ -26,5 +26,5 @@
 <xacro:property name="UpperLeg_yaw" value="0.0"/>
 <!-- Origin -->
-<xacro:property name="KneePitch_Ox" value="${props['big_box_length']}"/>
+<xacro:property name="KneePitch_Ox" value="0.0"/>
 <xacro:property name="KneePitch_Oy" value="0.0"/>
 <xacro:property name="KneePitch_Oz" value="0.0"/>
@@ -32,5 +32,5 @@
 <xacro:property name="KneePitch_pitch" value="0.0"/>
 <xacro:property name="KneePitch_yaw" value="0.0"/>
-<xacro:property name="LowerLeg_Ox" value="0.0"/>
+<xacro:property name="LowerLeg_Ox" value="${props['big_box_length']}"/>
 <xacro:property name="LowerLeg_Oy" value="0.0"/>
 <xacro:property name="LowerLeg_Oz" value="0.0"/>
