Commit message: gear ratio for motor torque and velocity limits

File: cetc_sat_urdf/urdf/cetc_sat.urdf (robot description, URDF)
Before this commit: robot cetc_sat, 39 links, 38 joints
Links:
- added link D435_front1_accel_frame
- added link D435_front1_accel_optical_frame
- added link D435_front1_bottom_screw_frame
- added link D435_front1_color_frame
- added link D435_front1_color_optical_frame
- added link D435_front1_depth_frame
- added link D435_front1_depth_optical_frame
- added link D435_front1_gyro_frame
- added link D435_front1_gyro_optical_frame
- added link D435_front1_left_ir_frame
- added link D435_front1_left_ir_optical_frame
- added link D435_front1_link, mass 0.564; collision box size=0.02505 0.09 0.025; visual mesh filename=package://realsense2_description/meshes/d435.dae
- added link D435_front1_right_ir_frame
- added link D435_front1_right_ir_optical_frame
- added link D435_front2_accel_frame
- added link D435_front2_accel_optical_frame
- added link D435_front2_bottom_screw_frame
- added link D435_front2_color_frame
- added link D435_front2_color_optical_frame
- added link D435_front2_depth_frame
- added link D435_front2_depth_optical_frame
- added link D435_front2_gyro_frame
- added link D435_front2_gyro_optical_frame
- added link D435_front2_left_ir_frame
- added link D435_front2_left_ir_optical_frame
- added link D435_front2_link, mass 0.564; collision box size=0.02505 0.09 0.025; visual mesh filename=package://realsense2_description/meshes/d435.dae
- added link D435_front2_right_ir_frame
- added link D435_front2_right_ir_optical_frame
- added link D435_front3_accel_frame
- added link D435_front3_accel_optical_frame
- added link D435_front3_bottom_screw_frame
- added link D435_front3_color_frame
- added link D435_front3_color_optical_frame
- added link D435_front3_depth_frame
- added link D435_front3_depth_optical_frame
- added link D435_front3_gyro_frame
- added link D435_front3_gyro_optical_frame
- added link D435_front3_left_ir_frame
- added link D435_front3_left_ir_optical_frame
- added link D435_front3_link, mass 0.564; collision box size=0.02505 0.09 0.025; visual mesh filename=package://realsense2_description/meshes/d435.dae
- added link D435_front3_right_ir_frame
- added link D435_front3_right_ir_optical_frame
- added link D435_left_accel_frame
- added link D435_left_accel_optical_frame
- added link D435_left_bottom_screw_frame
- added link D435_left_color_frame
- added link D435_left_color_optical_frame
- added link D435_left_depth_frame
- added link D435_left_depth_optical_frame
- added link D435_left_gyro_frame
- added link D435_left_gyro_optical_frame
- added link D435_left_left_ir_frame
- added link D435_left_left_ir_optical_frame
- added link D435_left_link, mass 0.564; collision box size=0.02505 0.09 0.025; visual mesh filename=package://realsense2_description/meshes/d435.dae
- added link D435_left_right_ir_frame
- added link D435_left_right_ir_optical_frame
- added link D435_rear_accel_frame
- added link D435_rear_accel_optical_frame
- added link D435_rear_bottom_screw_frame
- added link D435_rear_color_frame
- added link D435_rear_color_optical_frame
- added link D435_rear_depth_frame
- added link D435_rear_depth_optical_frame
- added link D435_rear_gyro_frame
- added link D435_rear_gyro_optical_frame
- added link D435_rear_left_ir_frame
- added link D435_rear_left_ir_optical_frame
- added link D435_rear_link, mass 0.564; collision box size=0.02505 0.09 0.025; visual mesh filename=package://realsense2_description/meshes/d435.dae
- added link D435_rear_right_ir_frame
- added link D435_rear_right_ir_optical_frame
- added link D435_right_accel_frame
- added link D435_right_accel_optical_frame
- added link D435_right_bottom_screw_frame
- added link D435_right_color_frame
- added link D435_right_color_optical_frame
- added link D435_right_depth_frame
- added link D435_right_depth_optical_frame
- added link D435_right_gyro_frame
- added link D435_right_gyro_optical_frame
- added link D435_right_left_ir_frame
- added link D435_right_left_ir_optical_frame
- added link D435_right_link, mass 0.564; collision box size=0.02505 0.09 0.025; visual mesh filename=package://realsense2_description/meshes/d435.dae
- added link D435_right_right_ir_frame
- added link D435_right_right_ir_optical_frame
- added link velodyne, mass 0.01; collision sphere radius=0; visual mesh filename=package://velodyne_description/meshes/VLP16_scan.dae
- added link velodyne_base_link, mass 0.83; collision cylinder length=0.0717 radius=0.0516; visual mesh filename=package://velodyne_description/meshes/VLP16_base_1.dae
Joints:
- added joint D435_front1_accel_joint: type fixed, parent D435_front1_link, child D435_front1_accel_frame, origin xyz=-0.00174 0.00552 0.0176 rpy=0 0 0
- added joint D435_front1_accel_optical_joint: type fixed, parent D435_front1_accel_frame, child D435_front1_accel_optical_frame, origin xyz=0 0 0 rpy=-1.5707963267948966 0 -1.5707963267948966
- added joint D435_front1_color_joint: type fixed, parent D435_front1_depth_frame, child D435_front1_color_frame, origin xyz=0 0.015 0 rpy=0 0 0
- added joint D435_front1_color_optical_joint: type fixed, parent D435_front1_color_frame, child D435_front1_color_optical_frame, origin xyz=0 0 0 rpy=-1.5707963267948966 0 -1.5707963267948966
- added joint D435_front1_depth_joint: type fixed, parent D435_front1_link, child D435_front1_depth_frame, origin xyz=0 0 0 rpy=0 0 0
- added joint D435_front1_depth_optical_joint: type fixed, parent D435_front1_depth_frame, child D435_front1_depth_optical_frame, origin xyz=0 0 0 rpy=-1.5707963267948966 0 -1.5707963267948966
- added joint D435_front1_gyro_joint: type fixed, parent D435_front1_link, child D435_front1_gyro_frame, origin xyz=-0.00174 0.00552 0.0176 rpy=0 0 0
- added joint D435_front1_gyro_optical_joint: type fixed, parent D435_front1_gyro_frame, child D435_front1_gyro_optical_frame, origin xyz=0 0 0 rpy=-1.5707963267948966 0 -1.5707963267948966
- added joint D435_front1_joint: type fixed, parent pelvis, child D435_front1_bottom_screw_frame, origin xyz=0.40 -0.08 0 rpy=-1.57 0 0.34
- added joint D435_front1_left_ir_joint: type fixed, parent D435_front1_depth_frame, child D435_front1_left_ir_frame, origin xyz=0 0.0 0 rpy=0 0 0
- added joint D435_front1_left_ir_optical_joint: type fixed, parent D435_front1_left_ir_frame, child D435_front1_left_ir_optical_frame, origin xyz=0 0 0 rpy=-1.5707963267948966 0 -1.5707963267948966
- added joint D435_front1_link_joint: type fixed, parent D435_front1_bottom_screw_frame, child D435_front1_link, origin xyz=0 0.0175 0.0125 rpy=0 0 0
- added joint D435_front1_right_ir_joint: type fixed, parent D435_front1_depth_frame, child D435_front1_right_ir_frame, origin xyz=0 -0.05 0 rpy=0 0 0
- added joint D435_front1_right_ir_optical_joint: type fixed, parent D435_front1_right_ir_frame, child D435_front1_right_ir_optical_frame, origin xyz=0 0 0 rpy=-1.5707963267948966 0 -1.5707963267948966
- added joint D435_front2_accel_joint: type fixed, parent D435_front2_link, child D435_front2_accel_frame, origin xyz=-0.00174 0.00552 0.0176 rpy=0 0 0
- added joint D435_front2_accel_optical_joint: type fixed, parent D435_front2_accel_frame, child D435_front2_accel_optical_frame, origin xyz=0 0 0 rpy=-1.5707963267948966 0 -1.5707963267948966
- added joint D435_front2_color_joint: type fixed, parent D435_front2_depth_frame, child D435_front2_color_frame, origin xyz=0 0.015 0 rpy=0 0 0
- added joint D435_front2_color_optical_joint: type fixed, parent D435_front2_color_frame, child D435_front2_color_optical_frame, origin xyz=0 0 0 rpy=-1.5707963267948966 0 -1.5707963267948966
- added joint D435_front2_depth_joint: type fixed, parent D435_front2_link, child D435_front2_depth_frame, origin xyz=0 0 0 rpy=0 0 0
- added joint D435_front2_depth_optical_joint: type fixed, parent D435_front2_depth_frame, child D435_front2_depth_optical_frame, origin xyz=0 0 0 rpy=-1.5707963267948966 0 -1.5707963267948966
- added joint D435_front2_gyro_joint: type fixed, parent D435_front2_link, child D435_front2_gyro_frame, origin xyz=-0.00174 0.00552 0.0176 rpy=0 0 0
- added joint D435_front2_gyro_optical_joint: type fixed, parent D435_front2_gyro_frame, child D435_front2_gyro_optical_frame, origin xyz=0 0 0 rpy=-1.5707963267948966 0 -1.5707963267948966
- added joint D435_front2_joint: type fixed, parent pelvis, child D435_front2_bottom_screw_frame, origin xyz=0.40 0.08 0 rpy=-1.57 0 -0.34
- added joint D435_front2_left_ir_joint: type fixed, parent D435_front2_depth_frame, child D435_front2_left_ir_frame, origin xyz=0 0.0 0 rpy=0 0 0
- added joint D435_front2_left_ir_optical_joint: type fixed, parent D435_front2_left_ir_frame, child D435_front2_left_ir_optical_frame, origin xyz=0 0 0 rpy=-1.5707963267948966 0 -1.5707963267948966
- added joint D435_front2_link_joint: type fixed, parent D435_front2_bottom_screw_frame, child D435_front2_link, origin xyz=0 0.0175 0.0125 rpy=0 0 0
- added joint D435_front2_right_ir_joint: type fixed, parent D435_front2_depth_frame, child D435_front2_right_ir_frame, origin xyz=0 -0.05 0 rpy=0 0 0
- added joint D435_front2_right_ir_optical_joint: type fixed, parent D435_front2_right_ir_frame, child D435_front2_right_ir_optical_frame, origin xyz=0 0 0 rpy=-1.5707963267948966 0 -1.5707963267948966
- added joint D435_front3_accel_joint: type fixed, parent D435_front3_link, child D435_front3_accel_frame, origin xyz=-0.00174 0.00552 0.0176 rpy=0 0 0
- added joint D435_front3_accel_optical_joint: type fixed, parent D435_front3_accel_frame, child D435_front3_accel_optical_frame, origin xyz=0 0 0 rpy=-1.5707963267948966 0 -1.5707963267948966
- added joint D435_front3_color_joint: type fixed, parent D435_front3_depth_frame, child D435_front3_color_frame, origin xyz=0 0.015 0 rpy=0 0 0
- added joint D435_front3_color_optical_joint: type fixed, parent D435_front3_color_frame, child D435_front3_color_optical_frame, origin xyz=0 0 0 rpy=-1.5707963267948966 0 -1.5707963267948966
- added joint D435_front3_depth_joint: type fixed, parent D435_front3_link, child D435_front3_depth_frame, origin xyz=0 0 0 rpy=0 0 0
- added joint D435_front3_depth_optical_joint: type fixed, parent D435_front3_depth_frame, child D435_front3_depth_optical_frame, origin xyz=0 0 0 rpy=-1.5707963267948966 0 -1.5707963267948966
- added joint D435_front3_gyro_joint: type fixed, parent D435_front3_link, child D435_front3_gyro_frame, origin xyz=-0.00174 0.00552 0.0176 rpy=0 0 0
- added joint D435_front3_gyro_optical_joint: type fixed, parent D435_front3_gyro_frame, child D435_front3_gyro_optical_frame, origin xyz=0 0 0 rpy=-1.5707963267948966 0 -1.5707963267948966
- added joint D435_front3_joint: type fixed, parent pelvis, child D435_front3_bottom_screw_frame, origin xyz=0.37 0 -0.11 rpy=0 0.75 0
- added joint D435_front3_left_ir_joint: type fixed, parent D435_front3_depth_frame, child D435_front3_left_ir_frame, origin xyz=0 0.0 0 rpy=0 0 0
- added joint D435_front3_left_ir_optical_joint: type fixed, parent D435_front3_left_ir_frame, child D435_front3_left_ir_optical_frame, origin xyz=0 0 0 rpy=-1.5707963267948966 0 -1.5707963267948966
- added joint D435_front3_link_joint: type fixed, parent D435_front3_bottom_screw_frame, child D435_front3_link, origin xyz=0 0.0175 0.0125 rpy=0 0 0
- added joint D435_front3_right_ir_joint: type fixed, parent D435_front3_depth_frame, child D435_front3_right_ir_frame, origin xyz=0 -0.05 0 rpy=0 0 0
- added joint D435_front3_right_ir_optical_joint: type fixed, parent D435_front3_right_ir_frame, child D435_front3_right_ir_optical_frame, origin xyz=0 0 0 rpy=-1.5707963267948966 0 -1.5707963267948966
- added joint D435_left_accel_joint: type fixed, parent D435_left_link, child D435_left_accel_frame, origin xyz=-0.00174 0.00552 0.0176 rpy=0 0 0
- added joint D435_left_accel_optical_joint: type fixed, parent D435_left_accel_frame, child D435_left_accel_optical_frame, origin xyz=0 0 0 rpy=-1.5707963267948966 0 -1.5707963267948966
- added joint D435_left_color_joint: type fixed, parent D435_left_depth_frame, child D435_left_color_frame, origin xyz=0 0.015 0 rpy=0 0 0
- added joint D435_left_color_optical_joint: type fixed, parent D435_left_color_frame, child D435_left_color_optical_frame, origin xyz=0 0 0 rpy=-1.5707963267948966 0 -1.5707963267948966
- added joint D435_left_depth_joint: type fixed, parent D435_left_link, child D435_left_depth_frame, origin xyz=0 0 0 rpy=0 0 0
- added joint D435_left_depth_optical_joint: type fixed, parent D435_left_depth_frame, child D435_left_depth_optical_frame, origin xyz=0 0 0 rpy=-1.5707963267948966 0 -1.5707963267948966
- added joint D435_left_gyro_joint: type fixed, parent D435_left_link, child D435_left_gyro_frame, origin xyz=-0.00174 0.00552 0.0176 rpy=0 0 0
- added joint D435_left_gyro_optical_joint: type fixed, parent D435_left_gyro_frame, child D435_left_gyro_optical_frame, origin xyz=0 0 0 rpy=-1.5707963267948966 0 -1.5707963267948966
- added joint D435_left_joint: type fixed, parent pelvis, child D435_left_bottom_screw_frame, origin xyz=-0.175 0.22 0 rpy=0 0.35 1.57
- added joint D435_left_left_ir_joint: type fixed, parent D435_left_depth_frame, child D435_left_left_ir_frame, origin xyz=0 0.0 0 rpy=0 0 0
- added joint D435_left_left_ir_optical_joint: type fixed, parent D435_left_left_ir_frame, child D435_left_left_ir_optical_frame, origin xyz=0 0 0 rpy=-1.5707963267948966 0 -1.5707963267948966
- added joint D435_left_link_joint: type fixed, parent D435_left_bottom_screw_frame, child D435_left_link, origin xyz=0 0.0175 0.0125 rpy=0 0 0
- added joint D435_left_right_ir_joint: type fixed, parent D435_left_depth_frame, child D435_left_right_ir_frame, origin xyz=0 -0.05 0 rpy=0 0 0
- added joint D435_left_right_ir_optical_joint: type fixed, parent D435_left_right_ir_frame, child D435_left_right_ir_optical_frame, origin xyz=0 0 0 rpy=-1.5707963267948966 0 -1.5707963267948966
- added joint D435_rear_accel_joint: type fixed, parent D435_rear_link, child D435_rear_accel_frame, origin xyz=-0.00174 0.00552 0.0176 rpy=0 0 0
- added joint D435_rear_accel_optical_joint: type fixed, parent D435_rear_accel_frame, child D435_rear_accel_optical_frame, origin xyz=0 0 0 rpy=-1.5707963267948966 0 -1.5707963267948966
- added joint D435_rear_color_joint: type fixed, parent D435_rear_depth_frame, child D435_rear_color_frame, origin xyz=0 0.015 0 rpy=0 0 0
- added joint D435_rear_color_optical_joint: type fixed, parent D435_rear_color_frame, child D435_rear_color_optical_frame, origin xyz=0 0 0 rpy=-1.5707963267948966 0 -1.5707963267948966
- added joint D435_rear_depth_joint: type fixed, parent D435_rear_link, child D435_rear_depth_frame, origin xyz=0 0 0 rpy=0 0 0
- added joint D435_rear_depth_optical_joint: type fixed, parent D435_rear_depth_frame, child D435_rear_depth_optical_frame, origin xyz=0 0 0 rpy=-1.5707963267948966 0 -1.5707963267948966
- added joint D435_rear_gyro_joint: type fixed, parent D435_rear_link, child D435_rear_gyro_frame, origin xyz=-0.00174 0.00552 0.0176 rpy=0 0 0
- added joint D435_rear_gyro_optical_joint: type fixed, parent D435_rear_gyro_frame, child D435_rear_gyro_optical_frame, origin xyz=0 0 0 rpy=-1.5707963267948966 0 -1.5707963267948966
- added joint D435_rear_joint: type fixed, parent pelvis, child D435_rear_bottom_screw_frame, origin xyz=-0.39 0 0 rpy=0 0.35 3.14
- added joint D435_rear_left_ir_joint: type fixed, parent D435_rear_depth_frame, child D435_rear_left_ir_frame, origin xyz=0 0.0 0 rpy=0 0 0
- added joint D435_rear_left_ir_optical_joint: type fixed, parent D435_rear_left_ir_frame, child D435_rear_left_ir_optical_frame, origin xyz=0 0 0 rpy=-1.5707963267948966 0 -1.5707963267948966
- added joint D435_rear_link_joint: type fixed, parent D435_rear_bottom_screw_frame, child D435_rear_link, origin xyz=0 0.0175 0.0125 rpy=0 0 0
- added joint D435_rear_right_ir_joint: type fixed, parent D435_rear_depth_frame, child D435_rear_right_ir_frame, origin xyz=0 -0.05 0 rpy=0 0 0
- added joint D435_rear_right_ir_optical_joint: type fixed, parent D435_rear_right_ir_frame, child D435_rear_right_ir_optical_frame, origin xyz=0 0 0 rpy=-1.5707963267948966 0 -1.5707963267948966
- added joint D435_right_accel_joint: type fixed, parent D435_right_link, child D435_right_accel_frame, origin xyz=-0.00174 0.00552 0.0176 rpy=0 0 0
- added joint D435_right_accel_optical_joint: type fixed, parent D435_right_accel_frame, child D435_right_accel_optical_frame, origin xyz=0 0 0 rpy=-1.5707963267948966 0 -1.5707963267948966
- added joint D435_right_color_joint: type fixed, parent D435_right_depth_frame, child D435_right_color_frame, origin xyz=0 0.015 0 rpy=0 0 0
- added joint D435_right_color_optical_joint: type fixed, parent D435_right_color_frame, child D435_right_color_optical_frame, origin xyz=0 0 0 rpy=-1.5707963267948966 0 -1.5707963267948966
- added joint D435_right_depth_joint: type fixed, parent D435_right_link, child D435_right_depth_frame, origin xyz=0 0 0 rpy=0 0 0
- added joint D435_right_depth_optical_joint: type fixed, parent D435_right_depth_frame, child D435_right_depth_optical_frame, origin xyz=0 0 0 rpy=-1.5707963267948966 0 -1.5707963267948966
- added joint D435_right_gyro_joint: type fixed, parent D435_right_link, child D435_right_gyro_frame, origin xyz=-0.00174 0.00552 0.0176 rpy=0 0 0
- added joint D435_right_gyro_optical_joint: type fixed, parent D435_right_gyro_frame, child D435_right_gyro_optical_frame, origin xyz=0 0 0 rpy=-1.5707963267948966 0 -1.5707963267948966
- added joint D435_right_joint: type fixed, parent pelvis, child D435_right_bottom_screw_frame, origin xyz=-0.175 -0.22 0 rpy=0 0.35 -1.57
- added joint D435_right_left_ir_joint: type fixed, parent D435_right_depth_frame, child D435_right_left_ir_frame, origin xyz=0 0.0 0 rpy=0 0 0
- added joint D435_right_left_ir_optical_joint: type fixed, parent D435_right_left_ir_frame, child D435_right_left_ir_optical_frame, origin xyz=0 0 0 rpy=-1.5707963267948966 0 -1.5707963267948966
- added joint D435_right_link_joint: type fixed, parent D435_right_bottom_screw_frame, child D435_right_link, origin xyz=0 0.0175 0.0125 rpy=0 0 0
- added joint D435_right_right_ir_joint: type fixed, parent D435_right_depth_frame, child D435_right_right_ir_frame, origin xyz=0 -0.05 0 rpy=0 0 0
- added joint D435_right_right_ir_optical_joint: type fixed, parent D435_right_right_ir_frame, child D435_right_right_ir_optical_frame, origin xyz=0 0 0 rpy=-1.5707963267948966 0 -1.5707963267948966
- added joint velodyne_base_mount_joint: type fixed, parent pelvis, child velodyne_base_link, origin xyz=0.36 0 0.11 rpy=0 0 0
- added joint velodyne_base_scan_joint: type fixed, parent velodyne_base_link, child velodyne, origin xyz=0 0 0.0377 rpy=0 0 0
- joint elbow_pitch_1: limit lower=-2.4056 upper=2.4056 effort=147.0 velocity=3.86 -> lower=-2.4056 upper=2.4056 effort=220 velocity=9.3
- joint elbow_pitch_2: limit lower=-2.3266 upper=2.3266 effort=147.0 velocity=3.86 -> lower=-2.3266 upper=2.3266 effort=220 velocity=9.3
- joint hip_pitch_1: limit lower=-2.4056 upper=2.4056 effort=304 velocity=8.8 -> lower=-2.4056 upper=2.4056 effort=220 velocity=9.3
- joint hip_pitch_2: limit lower=-2.3266 upper=2.3266 effort=304 velocity=8.8 -> lower=-2.3266 upper=2.3266 effort=220 velocity=9.3
- joint hip_pitch_3: limit lower=-2.4696 upper=2.4696 effort=304 velocity=8.8 -> lower=-2.4696 upper=2.4696 effort=220 velocity=9.3
- joint hip_pitch_4: limit lower=-2.3426 upper=2.3426 effort=304 velocity=8.8 -> lower=-2.3426 upper=2.3426 effort=220 velocity=9.3
- joint hip_roll_1: limit lower=-2.03 upper=2.51 effort=304 velocity=8.8 -> lower=-2.03 upper=2.51 effort=220 velocity=9.3
- joint hip_roll_2: limit lower=-2.51 upper=2.03 effort=304 velocity=8.8 -> lower=-2.51 upper=2.03 effort=220 velocity=9.3
- joint hip_roll_3: limit lower=-2.51 upper=2.03 effort=304 velocity=8.8 -> lower=-2.51 upper=2.03 effort=220 velocity=9.3
- joint hip_roll_4: limit lower=-2.03 upper=2.51 effort=304 velocity=8.8 -> lower=-2.03 upper=2.51 effort=220 velocity=9.3
- joint knee_pitch_1: limit lower=-2.4056 upper=2.4056 effort=304 velocity=8.8 -> lower=-2.4056 upper=2.4056 effort=220 velocity=9.3; origin xyz=0.0 0.0 0.0 rpy=0.0 0.0 0.0 -> xyz=0.4 0.0 0.0 rpy=0.0 0.0 0.0; parent knee_pitch_motor_1 -> upper_leg_1
- joint knee_pitch_2: limit lower=-2.3266 upper=2.3266 effort=304 velocity=8.8 -> lower=-2.3266 upper=2.3266 effort=220 velocity=9.3; origin xyz=0.0 0.0 0.0 rpy=0.0 0.0 0.0 -> xyz=0.4 0.0 0.0 rpy=0.0 0.0 0.0; parent knee_pitch_motor_2 -> upper_leg_2
- joint knee_pitch_3: limit lower=-2.4696 upper=2.4696 effort=304 velocity=8.8 -> lower=-2.4696 upper=2.4696 effort=220 velocity=9.3; origin xyz=0.0 0.0 0.0 rpy=0.0 0.0 0.0 -> xyz=0.4 0.0 0.0 rpy=0.0 0.0 0.0; parent knee_pitch_motor_3 -> upper_leg_3
- joint knee_pitch_4: limit lower=-2.3426 upper=2.3426 effort=304 velocity=8.8 -> lower=-2.3426 upper=2.3426 effort=220 velocity=9.3; origin xyz=0.0 0.0 0.0 rpy=0.0 0.0 0.0 -> xyz=0.4 0.0 0.0 rpy=0.0 0.0 0.0; parent knee_pitch_motor_4 -> upper_leg_4
- joint knee_pitch_stator_1: origin xyz=0.4 0.0 0.0 rpy=0.0 0.0 0.0 -> xyz=0.0 0.0 0.0 rpy=0.0 0.0 0.0; parent upper_leg_1 -> hip_pitch_motor_1
- joint knee_pitch_stator_2: origin xyz=0.4 0.0 0.0 rpy=0.0 0.0 0.0 -> xyz=0.0 0.0 0.0 rpy=0.0 0.0 0.0; parent upper_leg_2 -> hip_pitch_motor_2
- joint knee_pitch_stator_3: origin xyz=0.4 0.0 0.0 rpy=0.0 0.0 0.0 -> xyz=0.0 0.0 0.0 rpy=0.0 0.0 0.0; parent upper_leg_3 -> hip_pitch_motor_3
- joint knee_pitch_stator_4: origin xyz=0.4 0.0 0.0 rpy=0.0 0.0 0.0 -> xyz=0.0 0.0 0.0 rpy=0.0 0.0 0.0; parent upper_leg_4 -> hip_pitch_motor_4
- joint shoulder_pitch_1: limit lower=-2.4056 upper=2.4056 effort=147.0 velocity=3.86 -> lower=-2.4056 upper=2.4056 effort=220 velocity=9.3
- joint shoulder_pitch_2: limit lower=-2.3266 upper=2.3266 effort=147.0 velocity=3.86 -> lower=-2.3266 upper=2.3266 effort=220 velocity=9.3
- joint shoulder_yaw_1: limit lower=-3.312 upper=3.312 effort=147.0 velocity=3.86 -> lower=-3.312 upper=3.312 effort=220 velocity=9.3
- joint shoulder_yaw_2: limit lower=-3.3458 upper=3.3458 effort=147.0 velocity=3.86 -> lower=-3.3458 upper=3.3458 effort=220 velocity=9.3
