Commit message: gear ratio for motor torque and velocity limits

File: cetc_sat_urdf/urdf/parts/cetc_sat_arm.urdf.xacro (robot description, xacro)
@@ -132,5 +132,5 @@
 	<origin xyz="${ShoulderYaw_Ox - ShoulderYaw_OffsetX} ${rot * ShoulderYaw_Oy - rot * ShoulderYaw_OffsetY} ${ShoulderYaw_Oz - ShoulderYaw_OffsetZ}" rpy="${ShoulderYaw_roll} ${ShoulderYaw_pitch} ${ShoulderYaw_yaw}"/>
 	<axis xyz="0 0 1"/>
-	<limit lower="${j_shoulder_yaw_lower[arm_num-1]}" upper="${j_shoulder_yaw_upper[arm_num-1]}" effort="${j_shoulder_torque[arm_num-1]}" velocity="${j_shoulder_velocity[arm_num-1]}"/>
+	<limit lower="${j_shoulder_yaw_lower[arm_num-1]}" upper="${j_shoulder_yaw_upper[arm_num-1]}" effort="${motor_effort}" velocity="${motor_velocity}"/>
 </joint>
 <joint name="shoulder_pitch_stator_${arm_num}" type="fixed">
@@ -145,5 +145,5 @@
 	<origin xyz="${LowerArm_Ox} ${LowerArm_Oy} ${LowerArm_Oz}" rpy="${LowerArm_roll} ${LowerArm_pitch} ${LowerArm_yaw}"/>
 	<axis xyz="0 0 1"/>
-	<limit lower="${j_pitch_1_lower[arm_num-1]}" upper="${j_pitch_1_upper[arm_num-1]}" effort="${j_pitch_1_torque[arm_num-1]}" velocity="${j_pitch_1_velocity[arm_num-1]}"/>
+	<limit lower="${j_pitch_1_lower[arm_num-1]}" upper="${j_pitch_1_upper[arm_num-1]}" effort="${motor_effort}" velocity="${motor_velocity}"/>
 </joint>
 <joint name="elbow_pitch_stator_${arm_num}" type="fixed">
@@ -158,5 +158,5 @@
 	<origin xyz="${UpperArm_Ox} ${UpperArm_Oy} ${UpperArm_Oz}" rpy="${UpperArm_roll} ${UpperArm_pitch} ${UpperArm_yaw}"/>
 	<axis xyz="0 0 1"/>
-	<limit lower="${j_pitch_2_lower[arm_num-1]}" upper="${j_pitch_2_upper[arm_num-1]}" effort="${j_pitch_2_torque[arm_num-1]}" velocity="${j_pitch_2_velocity[arm_num-1]}"/>
+	<limit lower="${j_pitch_2_lower[arm_num-1]}" upper="${j_pitch_2_upper[arm_num-1]}" effort="${motor_effort}" velocity="${motor_velocity}"/>
 </joint>
 <!-- end effector  -->

File: cetc_sat_urdf/urdf/parts/cetc_sat_leg.urdf.xacro (robot description, xacro)
@@ -130,5 +130,5 @@
 	<origin xyz="${origin_x * HipRoll_Ox} ${origin_y * HipRoll_Oy} ${HipRoll_Oz}" rpy="${HipRoll_roll} ${HipRoll_pitch} ${HipRoll_yaw}"/>
 	<axis xyz="0 0 1"/>
-    <limit lower="${hip_roll_lower[leg_num-1]}" upper="${hip_roll_upper[leg_num-1]}" effort="${motor_A_effort}" velocity="${motor_A_velocity}"/> <!-- 200 Nm, 1 rad/s-->
+    <limit lower="${hip_roll_lower[leg_num-1]}" upper="${hip_roll_upper[leg_num-1]}" effort="${motor_effort}" velocity="${motor_velocity}"/> <!-- 200 Nm, 1 rad/s-->
 </joint>
 <joint name="hip_pitch_stator_${leg_num}" type="fixed">
@@ -147,5 +147,5 @@
 	<origin xyz="${UpperLeg_Ox} ${mirror*(UpperLeg_Oy)} ${UpperLeg_Oz}" rpy="${UpperLeg_roll} ${UpperLeg_pitch} ${UpperLeg_yaw}"/>
 	<axis xyz="0 0 1"/>
-   <limit lower="${hip_pitch_lower[leg_num-1]}" upper="${hip_pitch_upper[leg_num-1]}" effort="${motor_A_effort}" velocity="${motor_A_velocity}"/> <!-- 200 Nm, 1 rad/s-->
+   <limit lower="${hip_pitch_lower[leg_num-1]}" upper="${hip_pitch_upper[leg_num-1]}" effort="${motor_effort}" velocity="${motor_velocity}"/> <!-- 200 Nm, 1 rad/s-->
 </joint>
 <joint name="knee_pitch_${leg_num}" type="revolute">
@@ -154,5 +154,5 @@
 	<origin xyz="${LowerLeg_Ox} ${LowerLeg_Oy} ${LowerLeg_Oz}" rpy="${LowerLeg_roll} ${LowerLeg_pitch} ${LowerLeg_yaw}"/>
 	<axis xyz="0 0 1"/>
-   <limit lower="${knee_pitch_lower[leg_num-1]}" upper="${knee_pitch_upper[leg_num-1]}" effort="${motor_A_effort}" velocity="${motor_A_velocity}"/> <!-- 200 Nm, 1 rad/s-->
+   <limit lower="${knee_pitch_lower[leg_num-1]}" upper="${knee_pitch_upper[leg_num-1]}" effort="${motor_effort}" velocity="${motor_velocity}"/> <!-- 200 Nm, 1 rad/s-->
 </joint>
 <joint name="ball_joint_${leg_num}" type="fixed">

File: cetc_sat_urdf/urdf/parts/limits.urdf.xacro (robot description, xacro)
@@ -22,10 +22,16 @@
 <xacro:property name="j_pitch_2_torque" value="${[147.00, 147.00 ]}"/>
 <!-- Motor velocities -->
-<xacro:property name="motor_A_velocity" value="8.8"/>
-<xacro:property name="motor_B_velocity" value="8.1"/>
-<xacro:property name="motor_C_velocity" value="20.0"/>
+<xacro:if value="${inertial_props['gear_ratio'] == 30}">
+	<xacro:property name="motor_velocity" value="15.5"/>
+</xacro:if>
+<xacro:if value="${inertial_props['gear_ratio'] == 50}">
+	<xacro:property name="motor_velocity" value="9.3"/>
+</xacro:if>
 <!-- Motor effort -->
-<xacro:property name="motor_A_effort" value="304"/>
-<xacro:property name="motor_B_effort" value="147"/>
-<xacro:property name="motor_C_effort" value="35"/>
+<xacro:if value="${inertial_props['gear_ratio'] == 30}">
+	<xacro:property name="motor_effort" value="132"/>
+</xacro:if>
+<xacro:if value="${inertial_props['gear_ratio'] == 50}">
+	<xacro:property name="motor_effort" value="220"/>
+</xacro:if>
 </robot>
