Commit message: added gear ratios, renamed arms and legs links

File: cetc_sat_urdf/urdf/cetc_sat.urdf (robot description, URDF)
Before this commit: robot cetc_sat, 125 links, 124 joints
Links:
- removed link D435_front1_accel_frame
- removed link D435_front1_accel_optical_frame
- removed link D435_front1_bottom_screw_frame
- removed link D435_front1_color_frame
- removed link D435_front1_color_optical_frame
- removed link D435_front1_depth_frame
- removed link D435_front1_depth_optical_frame
- removed link D435_front1_gyro_frame
- removed link D435_front1_gyro_optical_frame
- removed link D435_front1_left_ir_frame
- removed link D435_front1_left_ir_optical_frame
- removed link D435_front1_link
- removed link D435_front1_right_ir_frame
- removed link D435_front1_right_ir_optical_frame
- removed link D435_front2_accel_frame
- removed link D435_front2_accel_optical_frame
- removed link D435_front2_bottom_screw_frame
- removed link D435_front2_color_frame
- removed link D435_front2_color_optical_frame
- removed link D435_front2_depth_frame
- removed link D435_front2_depth_optical_frame
- removed link D435_front2_gyro_frame
- removed link D435_front2_gyro_optical_frame
- removed link D435_front2_left_ir_frame
- removed link D435_front2_left_ir_optical_frame
- removed link D435_front2_link
- removed link D435_front2_right_ir_frame
- removed link D435_front2_right_ir_optical_frame
- removed link D435_front3_accel_frame
- removed link D435_front3_accel_optical_frame
- removed link D435_front3_bottom_screw_frame
- removed link D435_front3_color_frame
- removed link D435_front3_color_optical_frame
- removed link D435_front3_depth_frame
- removed link D435_front3_depth_optical_frame
- removed link D435_front3_gyro_frame
- removed link D435_front3_gyro_optical_frame
- removed link D435_front3_left_ir_frame
- removed link D435_front3_left_ir_optical_frame
- removed link D435_front3_link
- removed link D435_front3_right_ir_frame
- removed link D435_front3_right_ir_optical_frame
- removed link D435_left_accel_frame
- removed link D435_left_accel_optical_frame
- removed link D435_left_bottom_screw_frame
- removed link D435_left_color_frame
- removed link D435_left_color_optical_frame
- removed link D435_left_depth_frame
- removed link D435_left_depth_optical_frame
- removed link D435_left_gyro_frame
- removed link D435_left_gyro_optical_frame
- removed link D435_left_left_ir_frame
- removed link D435_left_left_ir_optical_frame
- removed link D435_left_link
- removed link D435_left_right_ir_frame
- removed link D435_left_right_ir_optical_frame
- removed link D435_rear_accel_frame
- removed link D435_rear_accel_optical_frame
- removed link D435_rear_bottom_screw_frame
- removed link D435_rear_color_frame
- removed link D435_rear_color_optical_frame
- removed link D435_rear_depth_frame
- removed link D435_rear_depth_optical_frame
- removed link D435_rear_gyro_frame
- removed link D435_rear_gyro_optical_frame
- removed link D435_rear_left_ir_frame
- removed link D435_rear_left_ir_optical_frame
- removed link D435_rear_link
- removed link D435_rear_right_ir_frame
- removed link D435_rear_right_ir_optical_frame
- removed link D435_right_accel_frame
- removed link D435_right_accel_optical_frame
- removed link D435_right_bottom_screw_frame
- removed link D435_right_color_frame
- removed link D435_right_color_optical_frame
- removed link D435_right_depth_frame
- removed link D435_right_depth_optical_frame
- removed link D435_right_gyro_frame
- removed link D435_right_gyro_optical_frame
- removed link D435_right_left_ir_frame
- removed link D435_right_left_ir_optical_frame
- removed link D435_right_link
- removed link D435_right_right_ir_frame
- removed link D435_right_right_ir_optical_frame
- removed link velodyne
- removed link velodyne_base_link
- link lower_arm_1: mass 2.0 -> 1.0; geometry collision box size=0.6 0.1 0.1; visual box size=0.6 0.1 0.1
- link lower_arm_2: mass 2.0 -> 1.0; geometry collision box size=0.6 0.1 0.1; visual box size=0.6 0.1 0.1
- link lower_leg_1: geometry collision box size=0.6 0.1 0.1; visual box size=0.6 0.1 0.1
- link lower_leg_2: geometry collision box size=0.6 0.1 0.1; visual box size=0.6 0.1 0.1
- link lower_leg_3: geometry collision box size=0.6 0.1 0.1; visual box size=0.6 0.1 0.1
- link lower_leg_4: geometry collision box size=0.6 0.1 0.1; visual box size=0.6 0.1 0.1
- link upper_arm_1: mass 1.0 -> 2.0; geometry collision box size=0.6 0.1 0.1; visual box size=0.6 0.1 0.1
- link upper_arm_2: mass 1.0 -> 2.0; geometry collision box size=0.6 0.1 0.1; visual box size=0.6 0.1 0.1
- link upper_leg_1: geometry collision box size=0.6 0.1 0.1; visual box size=0.6 0.1 0.1
- link upper_leg_2: geometry collision box size=0.6 0.1 0.1; visual box size=0.6 0.1 0.1
- link upper_leg_3: geometry collision box size=0.6 0.1 0.1; visual box size=0.6 0.1 0.1
- link upper_leg_4: geometry collision box size=0.6 0.1 0.1; visual box size=0.6 0.1 0.1
Joints:
- removed joint D435_front1_accel_joint
- removed joint D435_front1_accel_optical_joint
- removed joint D435_front1_color_joint
- removed joint D435_front1_color_optical_joint
- removed joint D435_front1_depth_joint
- removed joint D435_front1_depth_optical_joint
- removed joint D435_front1_gyro_joint
- removed joint D435_front1_gyro_optical_joint
- removed joint D435_front1_joint
- removed joint D435_front1_left_ir_joint
- removed joint D435_front1_left_ir_optical_joint
- removed joint D435_front1_link_joint
- removed joint D435_front1_right_ir_joint
- removed joint D435_front1_right_ir_optical_joint
- removed joint D435_front2_accel_joint
- removed joint D435_front2_accel_optical_joint
- removed joint D435_front2_color_joint
- removed joint D435_front2_color_optical_joint
- removed joint D435_front2_depth_joint
- removed joint D435_front2_depth_optical_joint
- removed joint D435_front2_gyro_joint
- removed joint D435_front2_gyro_optical_joint
- removed joint D435_front2_joint
- removed joint D435_front2_left_ir_joint
- removed joint D435_front2_left_ir_optical_joint
- removed joint D435_front2_link_joint
- removed joint D435_front2_right_ir_joint
- removed joint D435_front2_right_ir_optical_joint
- removed joint D435_front3_accel_joint
- removed joint D435_front3_accel_optical_joint
- removed joint D435_front3_color_joint
- removed joint D435_front3_color_optical_joint
- removed joint D435_front3_depth_joint
- removed joint D435_front3_depth_optical_joint
- removed joint D435_front3_gyro_joint
- removed joint D435_front3_gyro_optical_joint
- removed joint D435_front3_joint
- removed joint D435_front3_left_ir_joint
- removed joint D435_front3_left_ir_optical_joint
- removed joint D435_front3_link_joint
- removed joint D435_front3_right_ir_joint
- removed joint D435_front3_right_ir_optical_joint
- removed joint D435_left_accel_joint
- removed joint D435_left_accel_optical_joint
- removed joint D435_left_color_joint
- removed joint D435_left_color_optical_joint
- removed joint D435_left_depth_joint
- removed joint D435_left_depth_optical_joint
- removed joint D435_left_gyro_joint
- removed joint D435_left_gyro_optical_joint
- removed joint D435_left_joint
- removed joint D435_left_left_ir_joint
- removed joint D435_left_left_ir_optical_joint
- removed joint D435_left_link_joint
- removed joint D435_left_right_ir_joint
- removed joint D435_left_right_ir_optical_joint
- removed joint D435_rear_accel_joint
- removed joint D435_rear_accel_optical_joint
- removed joint D435_rear_color_joint
- removed joint D435_rear_color_optical_joint
- removed joint D435_rear_depth_joint
- removed joint D435_rear_depth_optical_joint
- removed joint D435_rear_gyro_joint
- removed joint D435_rear_gyro_optical_joint
- removed joint D435_rear_joint
- removed joint D435_rear_left_ir_joint
- removed joint D435_rear_left_ir_optical_joint
- removed joint D435_rear_link_joint
- removed joint D435_rear_right_ir_joint
- removed joint D435_rear_right_ir_optical_joint
- removed joint D435_right_accel_joint
- removed joint D435_right_accel_optical_joint
- removed joint D435_right_color_joint
- removed joint D435_right_color_optical_joint
- removed joint D435_right_depth_joint
- removed joint D435_right_depth_optical_joint
- removed joint D435_right_gyro_joint
- removed joint D435_right_gyro_optical_joint
- removed joint D435_right_joint
- removed joint D435_right_left_ir_joint
- removed joint D435_right_left_ir_optical_joint
- removed joint D435_right_link_joint
- removed joint D435_right_right_ir_joint
- removed joint D435_right_right_ir_optical_joint
- removed joint velodyne_base_mount_joint
- removed joint velodyne_base_scan_joint
- joint ball_joint_1: origin xyz=0.4 0.0 0.0 rpy=0.0 0.0 0.0 -> xyz=0.6 0.0 0.0 rpy=0.0 0.0 0.0
- joint ball_joint_2: origin xyz=0.4 0.0 0.0 rpy=0.0 0.0 0.0 -> xyz=0.6 0.0 0.0 rpy=0.0 0.0 0.0
- joint ball_joint_3: origin xyz=0.4 0.0 0.0 rpy=0.0 0.0 0.0 -> xyz=0.6 0.0 0.0 rpy=0.0 0.0 0.0
- joint ball_joint_4: origin xyz=0.4 0.0 0.0 rpy=0.0 0.0 0.0 -> xyz=0.6 0.0 0.0 rpy=0.0 0.0 0.0
- joint elbow_pitch_1: limit lower=-2.4056 upper=2.4056 effort=220 velocity=9.3 -> lower=-2.4056 upper=2.4056 effort=132 velocity=15.5
- joint elbow_pitch_2: limit lower=-2.3266 upper=2.3266 effort=220 velocity=9.3 -> lower=-2.3266 upper=2.3266 effort=132 velocity=15.5
- joint elbow_pitch_stator_1: origin xyz=0.4 0.0 0.0 rpy=0.0 0.0 0.0 -> xyz=0.6 0.0 0.0 rpy=0.0 0.0 0.0
- joint elbow_pitch_stator_2: origin xyz=0.4 0.0 0.0 rpy=0.0 0.0 0.0 -> xyz=0.6 0.0 0.0 rpy=0.0 0.0 0.0
- joint hand_joint_1: origin xyz=0.4 0.0 0.0 rpy=0.0 0.0 0.0 -> xyz=0.6 0.0 0.0 rpy=0.0 0.0 0.0
- joint hand_joint_2: origin xyz=0.4 0.0 0.0 rpy=0.0 0.0 0.0 -> xyz=0.6 0.0 0.0 rpy=0.0 0.0 0.0
- joint hip_pitch_1: limit lower=-2.4056 upper=2.4056 effort=220 velocity=9.3 -> lower=-2.4056 upper=2.4056 effort=132 velocity=15.5
- joint hip_pitch_2: limit lower=-2.3266 upper=2.3266 effort=220 velocity=9.3 -> lower=-2.3266 upper=2.3266 effort=132 velocity=15.5
- joint hip_pitch_3: limit lower=-2.4696 upper=2.4696 effort=220 velocity=9.3 -> lower=-2.4696 upper=2.4696 effort=132 velocity=15.5
- joint hip_pitch_4: limit lower=-2.3426 upper=2.3426 effort=220 velocity=9.3 -> lower=-2.3426 upper=2.3426 effort=132 velocity=15.5
- joint hip_roll_1: limit lower=-2.03 upper=2.51 effort=220 velocity=9.3 -> lower=-2.03 upper=2.51 effort=132 velocity=15.5
- joint hip_roll_2: limit lower=-2.51 upper=2.03 effort=220 velocity=9.3 -> lower=-2.51 upper=2.03 effort=132 velocity=15.5
- joint hip_roll_3: limit lower=-2.51 upper=2.03 effort=220 velocity=9.3 -> lower=-2.51 upper=2.03 effort=132 velocity=15.5
- joint hip_roll_4: limit lower=-2.03 upper=2.51 effort=220 velocity=9.3 -> lower=-2.03 upper=2.51 effort=132 velocity=15.5
- joint knee_pitch_1: limit lower=-2.4056 upper=2.4056 effort=220 velocity=9.3 -> lower=-2.4056 upper=2.4056 effort=132 velocity=15.5; origin xyz=0.4 0.0 0.0 rpy=0.0 0.0 0.0 -> xyz=0.6 0.0 0.0 rpy=0.0 0.0 0.0
- joint knee_pitch_2: limit lower=-2.3266 upper=2.3266 effort=220 velocity=9.3 -> lower=-2.3266 upper=2.3266 effort=132 velocity=15.5; origin xyz=0.4 0.0 0.0 rpy=0.0 0.0 0.0 -> xyz=0.6 0.0 0.0 rpy=0.0 0.0 0.0
- joint knee_pitch_3: limit lower=-2.4696 upper=2.4696 effort=220 velocity=9.3 -> lower=-2.4696 upper=2.4696 effort=132 velocity=15.5; origin xyz=0.4 0.0 0.0 rpy=0.0 0.0 0.0 -> xyz=0.6 0.0 0.0 rpy=0.0 0.0 0.0
- joint knee_pitch_4: limit lower=-2.3426 upper=2.3426 effort=220 velocity=9.3 -> lower=-2.3426 upper=2.3426 effort=132 velocity=15.5; origin xyz=0.4 0.0 0.0 rpy=0.0 0.0 0.0 -> xyz=0.6 0.0 0.0 rpy=0.0 0.0 0.0
- joint shoulder_pitch_1: limit lower=-2.4056 upper=2.4056 effort=220 velocity=9.3 -> lower=-2.4056 upper=2.4056 effort=132 velocity=15.5
- joint shoulder_pitch_2: limit lower=-2.3266 upper=2.3266 effort=220 velocity=9.3 -> lower=-2.3266 upper=2.3266 effort=132 velocity=15.5
- joint shoulder_yaw_1: limit lower=-3.312 upper=3.312 effort=220 velocity=9.3 -> lower=-3.312 upper=3.312 effort=132 velocity=15.5
- joint shoulder_yaw_2: limit lower=-3.3458 upper=3.3458 effort=220 velocity=9.3 -> lower=-3.3458 upper=3.3458 effort=132 velocity=15.5

File: cetc_sat_urdf/urdf/parts/cetc_sat_arm.urdf.xacro (robot description, xacro)
@@ -48,17 +48,17 @@
 	<inertial>
 		<origin xyz="0.0 0.0 0.0"/>
-		<mass value="${big_box_mass}"/>
-		<inertia ixx="${BigBox_xx}" ixy="${BigBox_xy}" ixz="${BigBox_xz}" iyy="${BigBox_xx}" iyz="${BigBox_yz}" izz="${BigBox_zz}"/>
+		<mass value="${upper_arm_mass}"/>
+		<inertia ixx="${LowerArm_xx}" ixy="${LowerArm_xy}" ixz="${LowerArm_xz}" iyy="${LowerArm_xx}" iyz="${LowerArm_yz}" izz="${LowerArm_zz}"/>
 	</inertial>
 	<visual>
-		<origin xyz="${big_box_length / 2} 0.0 0.0"  rpy="0.0 0.0 0.0"/>
+		<origin xyz="${lower_arm_length / 2} 0.0 0.0"  rpy="0.0 0.0 0.0"/>
 		<geometry>
-			<box size="${big_box_length} ${big_box_width} ${big_box_height}"/>
+			<box size="${lower_arm_length} ${lower_arm_width} ${lower_arm_height}"/>
 		</geometry>
 	</visual>
 	<collision>
-		<origin xyz="${big_box_length / 2} 0.0 0.0"  rpy="0.0 0.0 0.0"/>
+		<origin xyz="${lower_arm_length / 2} 0.0 0.0"  rpy="0.0 0.0 0.0"/>
 		<geometry>
-			<box size="${big_box_length} ${big_box_width} ${big_box_height}"/>
+			<box size="${lower_arm_length} ${lower_arm_width} ${lower_arm_height}"/>
 		</geometry>
 	</collision>
@@ -87,18 +87,18 @@
 	<inertial>
 		<origin xyz="0.0 0.0 0.0"/>
-		<mass value="${small_box_mass}"/>
-		<inertia ixx="${SmallBox_xx}" ixy="${SmallBox_xy}" ixz="${SmallBox_xz}" iyy="${SmallBox_xx}" iyz="${SmallBox_yz}" izz="${SmallBox_zz}"/>
+		<mass value="${lower_arm_mass}"/>
+		<inertia ixx="${UpperArm_xx}" ixy="${UpperArm_xy}" ixz="${UpperArm_xz}" iyy="${UpperArm_xx}" iyz="${UpperArm_yz}" izz="${UpperArm_zz}"/>
 	</inertial>
 	<visual>
-		<origin xyz="${small_box_length / 2} 0.0 0.0"  rpy="0.0 0.0 0.0"/>
+		<origin xyz="${upper_arm_length / 2} 0.0 0.0"  rpy="0.0 0.0 0.0"/>
 		<geometry>
-			<box size="${small_box_length} ${small_box_width} ${small_box_height}"/>
+			<box size="${upper_arm_length} ${upper_arm_width} ${upper_arm_height}"/>
 		</geometry>
 		<material name="dark_grey"/>
 	</visual>
 	<collision>
-		<origin xyz="${small_box_length / 2} 0.0 0.0"  rpy="0.0 0.0 0.0"/>
+		<origin xyz="${lower_arm_length / 2} 0.0 0.0"  rpy="0.0 0.0 0.0"/>
 		<geometry>
-			<box size="${small_box_length} ${small_box_width} ${small_box_height}"/>
+			<box size="${upper_arm_length} ${upper_arm_width} ${upper_arm_height}"/>
 		</geometry>
 	</collision>

File: cetc_sat_urdf/urdf/parts/cetc_sat_leg.urdf.xacro (robot description, xacro)
@@ -67,19 +67,19 @@
 	<inertial>
 		<origin xyz="0.0 0.0 0.0"/>
-		<mass value="${big_box_mass}"/>
-		<inertia ixx="${BigBox_xx}" ixy="${BigBox_xy}" ixz="${BigBox_xz}" iyy="${BigBox_xx}" iyz="${BigBox_yz}" izz="${BigBox_zz}"/>
+		<mass value="${upper_leg_mass}"/>
+		<inertia ixx="${UpperLeg_xx}" ixy="${UpperLeg_xy}" ixz="${UpperLeg_xz}" iyy="${UpperLeg_xx}" iyz="${UpperLeg_yz}" izz="${UpperLeg_zz}"/>
 	</inertial>
 	<origin xyz="0.0 0.0 0.0" rpy="0.0 0.0 0.0"/>
 	<visual>
-		<origin xyz="${big_box_length / 2} 0.0 0.0"  rpy="0.0 0.0 0.0"/>
+		<origin xyz="${upper_leg_length / 2} 0.0 0.0"  rpy="0.0 0.0 0.0"/>
 	  	<geometry>
-	 		<box size="${big_box_length} ${big_box_width} ${big_box_height}"/>
+	 		<box size="${upper_leg_length} ${upper_leg_width} ${upper_leg_height}"/>
 	  	</geometry>
   		<material name="dark_grey"/>
 	</visual>
 	<collision>
-		<origin xyz="${big_box_length / 2} 0.0 0.0"  rpy="0.0 0.0 0.0"/>
+		<origin xyz="${upper_leg_length / 2} 0.0 0.0"  rpy="0.0 0.0 0.0"/>
 		<geometry>
-			<box size="${big_box_length} ${big_box_width} ${big_box_height}"/>
+			<box size="${upper_leg_length} ${upper_leg_width} ${upper_leg_height}"/>
 		</geometry>
 	</collision>
@@ -88,18 +88,18 @@
 	<inertial>
 		<origin xyz="0.0 0.0 0.0"/>
-		<mass value="${small_box_mass}"/>
-		<inertia ixx="${SmallBox_xx}" ixy="${SmallBox_xy}" ixz="${SmallBox_xz}" iyy="${SmallBox_xx}" iyz="${SmallBox_yz}" izz="${SmallBox_zz}"/>
+		<mass value="${lower_leg_mass}"/>
+		<inertia ixx="${LowerLeg_xx}" ixy="${LowerLeg_xy}" ixz="${LowerLeg_xz}" iyy="${LowerLeg_xx}" iyz="${LowerLeg_yz}" izz="${LowerLeg_zz}"/>
 	</inertial>
 	<visual>
-		<origin xyz="${small_box_length / 2} 0.0 0.0"  rpy="0.0 0.0 0.0"/>
+		<origin xyz="${lower_leg_length / 2} 0.0 0.0"  rpy="0.0 0.0 0.0"/>
 	  	<geometry>
-	 		<box size="${small_box_length} ${small_box_width} ${small_box_height}"/>
+	 		<box size="${lower_leg_length} ${lower_leg_width} ${lower_leg_height}"/>
 	  	</geometry>
   		<material name="dark_grey"/>
 	</visual>
 	<collision>
-		<origin xyz="${small_box_length / 2} 0.0 0.0"  rpy="0.0 0.0 0.0"/>
+		<origin xyz="${lower_leg_length / 2} 0.0 0.0"  rpy="0.0 0.0 0.0"/>
 		<geometry>
-	 		<box size="${small_box_length} ${small_box_width} ${small_box_height}"/>
+	 		<box size="${lower_leg_length} ${lower_leg_width} ${lower_leg_height}"/>
 		</geometry>
 	</collision>

File: cetc_sat_urdf/urdf/parts/inertial_properties.urdf.xacro (robot description, xacro)
@@ -7,6 +7,8 @@
         <xacro:property name="inertial_props" value="${xacro.load_yaml(inertial_yaml_file)}"/>
         <xacro:property name="pelvis_mass" value="${inertial_props['pelvis_mass'][id]}"/>
-        <xacro:property name="big_box_mass" value="${inertial_props['big_box_mass'][id]}"/>
-        <xacro:property name="small_box_mass" value="${inertial_props['small_box_mass'][id]}"/>
+        <xacro:property name="upper_leg_mass" value="${inertial_props['upper_leg_mass'][id]}"/>
+        <xacro:property name="lower_leg_mass" value="${inertial_props['lower_leg_mass'][id]}"/>
+        <xacro:property name="upper_arm_mass" value="${inertial_props['upper_arm_mass'][id]}"/>
+        <xacro:property name="lower_arm_mass" value="${inertial_props['lower_arm_mass'][id]}"/>
         <xacro:property name="ball_mass" value="${inertial_props['ball_mass'][id]}"/>
         <xacro:property name="motorA_mass" value="${inertial_props['motorA_mass'][id]}"/>
@@ -17,6 +19,8 @@
         <xacro:property name="inertial_props" value="${xacro.load_yaml(inertial_yaml_file)}"/>
         <xacro:property name="pelvis_mass" value="${inertial_props['pelvis_mass']}"/>
-        <xacro:property name="big_box_mass" value="${inertial_props['big_box_mass']}"/>
-        <xacro:property name="small_box_mass" value="${inertial_props['small_box_mass']}"/>
+        <xacro:property name="upper_leg_mass" value="${inertial_props['upper_leg_mass']}"/>
+        <xacro:property name="lower_leg_mass" value="${inertial_props['lower_leg_mass']}"/>
+        <xacro:property name="upper_arm_mass" value="${inertial_props['upper_arm_mass']}"/>
+        <xacro:property name="lower_arm_mass" value="${inertial_props['lower_arm_mass']}"/>
         <xacro:property name="ball_mass" value="${inertial_props['ball_mass']}"/>
         <xacro:property name="motorA_mass" value="${inertial_props['motorA_mass']}"/>
@@ -45,17 +49,31 @@
     <xacro:property name="Pelvis_zz" value="${1/12 * pelvis_mass * (pelvis_width * pelvis_width + pelvis_length * pelvis_length)}"/>
     <!-- Upper Leg -->
-    <xacro:property name="BigBox_xx" value="${1/3 * big_box_mass * (big_box_width * big_box_width + big_box_height * big_box_height)}"/>
-    <xacro:property name="BigBox_xy" value="0.0"/>
-    <xacro:property name="BigBox_xz" value="0.0"/>
-    <xacro:property name="BigBox_yy" value="${1/3 * big_box_mass * (big_box_length * big_box_length + big_box_height * big_box_height)}"/>
-    <xacro:property name="BigBox_yz" value="0.0"/>
-    <xacro:property name="BigBox_zz" value="${1/3 * big_box_mass * (big_box_width * big_box_width + big_box_length * big_box_length)}"/>
+    <xacro:property name="UpperLeg_xx" value="${1/3 * upper_leg_mass * (upper_leg_width * upper_leg_width + upper_leg_height * upper_leg_height)}"/>
+    <xacro:property name="UpperLeg_xy" value="0.0"/>
+    <xacro:property name="UpperLeg_xz" value="0.0"/>
+    <xacro:property name="UpperLeg_yy" value="${1/3 * upper_leg_mass * (upper_leg_length * upper_leg_length + upper_leg_height * upper_leg_height)}"/>
+    <xacro:property name="UpperLeg_yz" value="0.0"/>
+    <xacro:property name="UpperLeg_zz" value="${1/3 * upper_leg_mass * (upper_leg_width * upper_leg_width + upper_leg_length * upper_leg_length)}"/>
     <!-- Lower Leg -->
-    <xacro:property name="SmallBox_xx" value="${1/3 * small_box_mass * (small_box_width * small_box_width + small_box_height * small_box_height)}"/>
-    <xacro:property name="SmallBox_xy" value="0.0"/>
-    <xacro:property name="SmallBox_xz" value="0.0"/>
-    <xacro:property name="SmallBox_yy" value="${1/3 * small_box_mass * (small_box_length * small_box_length + small_box_height * small_box_height)}"/>
-    <xacro:property name="SmallBox_yz" value="0.0"/>
-    <xacro:property name="SmallBox_zz" value="${1/3 * small_box_mass * (small_box_width * small_box_width + small_box_length * small_box_length)}"/>
+    <xacro:property name="LowerLeg_xx" value="${1/3 * lower_leg_mass * (lower_leg_width * lower_leg_width + lower_leg_height * lower_leg_height)}"/>
+    <xacro:property name="LowerLeg_xy" value="0.0"/>
+    <xacro:property name="LowerLeg_xz" value="0.0"/>
+    <xacro:property name="LowerLeg_yy" value="${1/3 * lower_leg_mass * (lower_leg_length * lower_leg_length + lower_leg_height * lower_leg_height)}"/>
+    <xacro:property name="LowerLeg_yz" value="0.0"/>
+    <xacro:property name="LowerLeg_zz" value="${1/3 * lower_leg_mass * (lower_leg_width * lower_leg_width + lower_leg_length * lower_leg_length)}"/>
+    <!-- Upper Arm -->
+    <xacro:property name="UpperArm_xx" value="${1/3 * upper_arm_mass * (upper_arm_width * upper_arm_width + upper_arm_height * upper_arm_height)}"/>
+    <xacro:property name="UpperArm_xy" value="0.0"/>
+    <xacro:property name="UpperArm_xz" value="0.0"/>
+    <xacro:property name="UpperArm_yy" value="${1/3 * upper_arm_mass * (upper_arm_length * upper_arm_length + upper_arm_height * upper_arm_height)}"/>
+    <xacro:property name="UpperArm_yz" value="0.0"/>
+    <xacro:property name="UpperArm_zz" value="${1/3 * upper_arm_mass * (upper_arm_width * upper_arm_width + upper_arm_length * upper_arm_length)}"/>
+    <!-- Lower Arm -->
+    <xacro:property name="LowerArm_xx" value="${1/3 * lower_arm_mass * (lower_arm_width * lower_arm_width + lower_arm_height * lower_arm_height)}"/>
+    <xacro:property name="LowerArm_xy" value="0.0"/>
+    <xacro:property name="LowerArm_xz" value="0.0"/>
+    <xacro:property name="LowerArm_yy" value="${1/3 * lower_arm_mass * (lower_arm_length * lower_arm_length + lower_arm_height * lower_arm_height)}"/>
+    <xacro:property name="LowerArm_yz" value="0.0"/>
+    <xacro:property name="LowerArm_zz" value="${1/3 * lower_arm_mass * (lower_arm_width * lower_arm_width + lower_arm_length * lower_arm_length)}"/>
     <!-- Ball (hollow sphere) -->
     <xacro:property name="Ball_xx" value="${2/3 * ball_mass * ball_radius * ball_radius}"/>
