Commit message: added gear ratios, renamed arms and legs links

File: cetc_sat_urdf/urdf/parts/kinematics_properties.urdf.xacro (robot description, xacro)
@@ -8,10 +8,16 @@
         <xacro:property name="cylinder_radius" value="${kin_props['cylinder_radius'][id]}"/>
         <xacro:property name="cylinder_length" value="${kin_props['cylinder_length'][id]}"/>
-        <xacro:property name="big_box_length" value="${kin_props['big_box_length'][id]}"/>
-        <xacro:property name="big_box_width" value="${kin_props['big_box_width'][id]}"/>
-        <xacro:property name="big_box_height" value="${kin_props['big_box_height'][id]}"/>
-        <xacro:property name="small_box_length" value="${kin_props['small_box_length'][id]}"/>
-        <xacro:property name="small_box_width" value="${kin_props['small_box_width'][id]}"/>
-        <xacro:property name="small_box_height" value="${kin_props['small_box_height'][id]}"/>
+        <xacro:property name="upper_leg_length" value="${kin_props['upper_leg_length'][id]}"/>
+        <xacro:property name="upper_leg_width" value="${kin_props['upper_leg_width'][id]}"/>
+        <xacro:property name="upper_leg_height" value="${kin_props['upper_leg_height'][id]}"/>
+        <xacro:property name="lower_upper_leg_length" value="${kin_props['lower_leg_length'][id]}"/>
+        <xacro:property name="lower_upper_leg_width" value="${kin_props['lower_leg_width'][id]}"/>
+        <xacro:property name="lower_upper_leg_height" value="${kin_props['lower_leg_height'][id]}"/>
+        <xacro:property name="upper_arm_length" value="${kin_props['upper_arm_length'][id]}"/>
+        <xacro:property name="upper_arm_width" value="${kin_props['upper_arm_width'][id]}"/>
+        <xacro:property name="upper_arm_height" value="${kin_props['upper_arm_height'][id]}"/>
+        <xacro:property name="lower_arm_length" value="${kin_props['lower_arm_length'][id]}"/>
+        <xacro:property name="lower_arm_width" value="${kin_props['lower_arm_width'][id]}"/>
+        <xacro:property name="lower_arm_height" value="${kin_props['lower_arm_height'][id]}"/>
         <xacro:property name="ball_radius" value="${kin_props['ball_radius'][id]}"/>
         <xacro:property name="pelvis_length" value="${kin_props['pelvis_length'][id]}"/>
@@ -24,10 +30,16 @@
         <xacro:property name="cylinder_radius" value="${kin_props['cylinder_radius']}"/>
         <xacro:property name="cylinder_length" value="${kin_props['cylinder_length']}"/>
-        <xacro:property name="big_box_length" value="${kin_props['big_box_length']}"/>
-        <xacro:property name="big_box_width" value="${kin_props['big_box_width']}"/>
-        <xacro:property name="big_box_height" value="${kin_props['big_box_height']}"/>
-        <xacro:property name="small_box_length" value="${kin_props['small_box_length']}"/>
-        <xacro:property name="small_box_width" value="${kin_props['small_box_width']}"/>
-        <xacro:property name="small_box_height" value="${kin_props['small_box_height']}"/>
+        <xacro:property name="upper_leg_length" value="${kin_props['upper_leg_length']}"/>
+        <xacro:property name="upper_leg_width" value="${kin_props['upper_leg_width']}"/>
+        <xacro:property name="upper_leg_height" value="${kin_props['upper_leg_height']}"/>
+        <xacro:property name="lower_leg_length" value="${kin_props['lower_leg_length']}"/>
+        <xacro:property name="lower_leg_width" value="${kin_props['lower_leg_width']}"/>
+        <xacro:property name="lower_leg_height" value="${kin_props['lower_leg_height']}"/>
+        <xacro:property name="upper_arm_length" value="${kin_props['upper_arm_length']}"/>
+        <xacro:property name="upper_arm_width" value="${kin_props['upper_arm_width']}"/>
+        <xacro:property name="upper_arm_height" value="${kin_props['upper_arm_height']}"/>
+        <xacro:property name="lower_arm_length" value="${kin_props['lower_arm_length']}"/>
+        <xacro:property name="lower_arm_width" value="${kin_props['lower_arm_width']}"/>
+        <xacro:property name="lower_arm_height" value="${kin_props['lower_arm_height']}"/>
         <xacro:property name="ball_radius" value="${kin_props['ball_radius']}"/>
         <xacro:property name="pelvis_length" value="${kin_props['pelvis_length']}"/>
@@ -63,5 +75,5 @@
     <xacro:property name="KneePitch_pitch" value="0.0"/>
     <xacro:property name="KneePitch_yaw" value="0.0"/>
-    <xacro:property name="LowerLeg_Ox" value="${big_box_length}"/>
+    <xacro:property name="LowerLeg_Ox" value="${upper_leg_length}"/>
     <xacro:property name="LowerLeg_Oy" value="0.0"/>
     <xacro:property name="LowerLeg_Oz" value="0.0"/>
@@ -70,5 +82,5 @@
     <xacro:property name="LowerLeg_yaw" value="0.0"/>
     <!-- Origin -->
-    <xacro:property name="Ankle_Ox" value="${big_box_length}"/>
+    <xacro:property name="Ankle_Ox" value="${lower_leg_length}"/>
     <xacro:property name="Ankle_Oy" value="0.0"/>
     <xacro:property name="Ankle_Oz" value="0.0"/>
@@ -98,5 +110,5 @@
     <xacro:property name="LowerArm_pitch" value="0.0"/>
     <xacro:property name="LowerArm_yaw" value="${-PI_2}"/>
-    <xacro:property name="ElbowPitch_Ox" value="${big_box_length}"/>
+    <xacro:property name="ElbowPitch_Ox" value="${lower_arm_length}"/>
     <xacro:property name="ElbowPitch_Oy" value="0.0"/>
     <xacro:property name="ElbowPitch_Oz" value="0.0"/>
@@ -110,5 +122,5 @@
     <xacro:property name="UpperArm_pitch" value="0.0"/>
     <xacro:property name="UpperArm_yaw" value="0.0"/>
-    <xacro:property name="EndEffector_Ox" value="${big_box_length}"/>
+    <xacro:property name="EndEffector_Ox" value="${upper_arm_length}"/>
     <xacro:property name="EndEffector_Oy" value="0.0"/>
     <xacro:property name="EndEffector_Oz" value="0.0"/>

Commit message: added payload

File: cetc_sat_urdf/urdf/cetc_sat.urdf (robot description, URDF)
Before this commit: robot cetc_sat, 39 links, 38 joints
Links:
- added link payload_1, mass 4; visual box size=0.2 0.2 0.2
- added link payload_2, mass 4; visual box size=0.2 0.2 0.2
- added link payload_pelvis, mass 4; visual box size=0.2 0.2 0.2
- link lower_arm_1: geometry collision box size=0.3 0.1 0.1; visual box size=0.3 0.1 0.1
- link lower_arm_2: geometry collision box size=0.3 0.1 0.1; visual box size=0.3 0.1 0.1
- link lower_leg_1: geometry collision box size=0.3 0.05 0.05; visual box size=0.3 0.05 0.05
- link lower_leg_2: geometry collision box size=0.3 0.05 0.05; visual box size=0.3 0.05 0.05
- link lower_leg_3: geometry collision box size=0.3 0.05 0.05; visual box size=0.3 0.05 0.05
- link lower_leg_4: geometry collision box size=0.3 0.05 0.05; visual box size=0.3 0.05 0.05
- link pelvis: mass 14 -> 34
- link upper_arm_1: geometry collision box size=0.3 0.05 0.05; visual box size=0.3 0.05 0.05
- link upper_arm_2: geometry collision box size=0.3 0.05 0.05; visual box size=0.3 0.05 0.05
- link upper_leg_1: geometry collision box size=0.35 0.1 0.1; visual box size=0.35 0.1 0.1
- link upper_leg_2: geometry collision box size=0.35 0.1 0.1; visual box size=0.35 0.1 0.1
- link upper_leg_3: geometry collision box size=0.35 0.1 0.1; visual box size=0.35 0.1 0.1
- link upper_leg_4: geometry collision box size=0.35 0.1 0.1; visual box size=0.35 0.1 0.1
Joints:
- added joint hand_to_payload_1: type fixed, parent ball_arm_1, child payload_1
- added joint hand_to_payload_2: type fixed, parent ball_arm_2, child payload_2
- added joint pelvis_to_payload: type fixed, parent pelvis, child payload_pelvis, origin xyz=-0.3 0.0 0.225
- joint ball_joint_1: origin xyz=0.6 0.0 0.0 rpy=0.0 0.0 0.0 -> xyz=0.3 0.0 0.0 rpy=0.0 0.0 0.0
- joint ball_joint_2: origin xyz=0.6 0.0 0.0 rpy=0.0 0.0 0.0 -> xyz=0.3 0.0 0.0 rpy=0.0 0.0 0.0
- joint ball_joint_3: origin xyz=0.6 0.0 0.0 rpy=0.0 0.0 0.0 -> xyz=0.3 0.0 0.0 rpy=0.0 0.0 0.0
- joint ball_joint_4: origin xyz=0.6 0.0 0.0 rpy=0.0 0.0 0.0 -> xyz=0.3 0.0 0.0 rpy=0.0 0.0 0.0
- joint elbow_pitch_stator_1: origin xyz=0.6 0.0 0.0 rpy=0.0 0.0 0.0 -> xyz=0.3 0.0 0.0 rpy=0.0 0.0 0.0
- joint elbow_pitch_stator_2: origin xyz=0.6 0.0 0.0 rpy=0.0 0.0 0.0 -> xyz=0.3 0.0 0.0 rpy=0.0 0.0 0.0
- joint hand_joint_1: origin xyz=0.6 0.0 0.0 rpy=0.0 0.0 0.0 -> xyz=0.3 0.0 0.0 rpy=0.0 0.0 0.0
- joint hand_joint_2: origin xyz=0.6 0.0 0.0 rpy=0.0 0.0 0.0 -> xyz=0.3 0.0 0.0 rpy=0.0 0.0 0.0
- joint knee_pitch_1: origin xyz=0.6 0.0 0.0 rpy=0.0 0.0 0.0 -> xyz=0.35 0.0 0.0 rpy=0.0 0.0 0.0
- joint knee_pitch_2: origin xyz=0.6 0.0 0.0 rpy=0.0 0.0 0.0 -> xyz=0.35 0.0 0.0 rpy=0.0 0.0 0.0
- joint knee_pitch_3: origin xyz=0.6 0.0 0.0 rpy=0.0 0.0 0.0 -> xyz=0.35 0.0 0.0 rpy=0.0 0.0 0.0
- joint knee_pitch_4: origin xyz=0.6 0.0 0.0 rpy=0.0 0.0 0.0 -> xyz=0.35 0.0 0.0 rpy=0.0 0.0 0.0

File: cetc_sat_urdf/urdf/cetc_sat_base.urdf.xacro (robot description, xacro)
@@ -175,3 +175,24 @@
 	<xacro:include filename="$(find cetc_sat_urdf)/urdf/parts/legs.urdf.xacro" />
 </xacro:if>
+<xacro:if value="${PAYLOAD}">
+	<link name="payload_pelvis">
+		<inertial>
+		    <origin xyz="0.0 0.0 0.0"/>
+			<mass value="20"/>
+			<inertia ixx="0.13" iyy="0.13" izz="0.13" ixy="0" ixz="0" iyz="0"/>
+		</inertial>
+		<visual>
+			<origin xyz="0.0 0.0 0.0"  rpy="0.0 0.0 0.0"/>
+			<geometry>
+				<box size="0.2 0.2 0.2"/>
+			</geometry>
+			<material name="dark_grey"/>
+		</visual>
+	</link>
+	<joint name="pelvis_to_payload" type="fixed">
+		<origin xyz="-0.2 0.0 ${pelvis_height / 2 + 0.1}"/>
+		<parent link="pelvis"/>
+		<child link="payload_pelvis"/>
+	</joint>
+</xacro:if>
 </robot>

File: cetc_sat_urdf/urdf/config/cetc_sat.urdf.xacro (robot description, xacro)
@@ -8,4 +8,5 @@
 <xacro:arg name="floating_joint" default="true"/>
 <xacro:arg name="sensors" default="true"/>
+<xacro:arg name="payload" default="false"/>
 <!-- ************SELECT PARTS*************-->
 <!-- *************************************-->
@@ -15,3 +16,4 @@
 <xacro:property name="ADD_FLOATING_BASE" value="$(arg floating_joint)" />
 <xacro:property name="ADD_VIRTUAL_FRAME" value="false" />
+<xacro:property name="PAYLOAD" value="$(arg payload)"/>
 </robot>
