Commit message: fixed inertias

File: cetc_sat_urdf/urdf/cetc_sat.urdf (robot description, URDF)
Before this commit: robot cetc_sat, 42 links, 41 joints
Links:
- removed link ball_arm_1
- removed link ball_arm_2
- removed link payload_1
- removed link payload_2
- removed link payload_pelvis
- removed link upper_arm_1
- removed link upper_arm_2
- added link dagana_1_bottom_link, mass 4.6117745e-01; collision mesh filename=package://dagana_urdf/meshes/dg0002-ch.stl scale=0.001 0.001 0.001; visual mesh filename=package://dagana_urdf/meshes/dg0002.stl scale=0.001 0.001 0.001
- added link dagana_1_palm_frame
- added link dagana_1_top_link, mass 1.7432400; collision mesh filename=package://dagana_urdf/meshes/dg0001-ch.stl scale=0.001 0.001 0.001; visual mesh filename=package://dagana_urdf/meshes/dg0001-simplified.stl scale=0.001 0.001 0.001
- added link dagana_2_bottom_link, mass 4.6117745e-01; collision mesh filename=package://dagana_urdf/meshes/dg0002-ch.stl scale=0.001 0.001 0.001; visual mesh filename=package://dagana_urdf/meshes/dg0002.stl scale=0.001 0.001 0.001
- added link dagana_2_palm_frame
- added link dagana_2_top_link, mass 1.7432400; collision mesh filename=package://dagana_urdf/meshes/dg0001-ch.stl scale=0.001 0.001 0.001; visual mesh filename=package://dagana_urdf/meshes/dg0001-simplified.stl scale=0.001 0.001 0.001
- added link upper_arm1_1, mass 0.7; collision box size=0.2 0.05 0.05; visual box size=0.2 0.05 0.05
- added link upper_arm1_2, mass 0.7; collision box size=0.2 0.05 0.05; visual box size=0.2 0.05 0.05
- added link upper_arm2_1, mass 0.3; collision box size=0.1 0.05 0.05; visual box size=0.1 0.05 0.05
- added link upper_arm2_2, mass 0.3; collision box size=0.1 0.05 0.05; visual box size=0.1 0.05 0.05
- added link wrist_1, mass 1.8; collision cylinder length=0.05 radius=0.035; visual cylinder length=0.016666666666666666 radius=0.07
- added link wrist_2, mass 1.8; collision cylinder length=0.05 radius=0.035; visual cylinder length=0.016666666666666666 radius=0.07
- added link wrist_pitch_motor_1, mass 1.8; collision cylinder length=0.1 radius=0.07; visual cylinder length=0.05 radius=0.035
- added link wrist_pitch_motor_2, mass 1.8; collision cylinder length=0.1 radius=0.07; visual cylinder length=0.05 radius=0.035
- link lower_arm_1: mass 1.0 -> 2.0
- link lower_arm_2: mass 1.0 -> 2.0
- link pelvis: mass 34 -> 14
Joints:
- removed joint hand_joint_1
- removed joint hand_joint_2
- removed joint hand_to_payload_1
- removed joint hand_to_payload_2
- removed joint pelvis_to_payload
- added joint dagana_1_claw_joint: type fixed, parent dagana_1_top_link, child dagana_1_bottom_link, origin xyz=0.0 -0.028 0.05025 rpy=1.57079632679 0 3.14159265359, axis 0 0 1
- added joint dagana_1_mount_joint: type fixed, parent wrist_1, child dagana_1_top_link, origin xyz=0 0 0 rpy=0 0 0
- added joint dagana_1_pal_joint: type fixed, parent dagana_1_top_link, child dagana_1_palm_frame, origin xyz=0. 0. 0. rpy=1.57079632679 0 3.14159265359
- added joint dagana_2_claw_joint: type fixed, parent dagana_2_top_link, child dagana_2_bottom_link, origin xyz=0.0 -0.028 0.05025 rpy=1.57079632679 0 3.14159265359, axis 0 0 1
- added joint dagana_2_mount_joint: type fixed, parent wrist_2, child dagana_2_top_link, origin xyz=0 0 0 rpy=0 0 0
- added joint dagana_2_pal_joint: type fixed, parent dagana_2_top_link, child dagana_2_palm_frame, origin xyz=0. 0. 0. rpy=1.57079632679 0 3.14159265359
- added joint wrist_pitch_1: type revolute, parent wrist_pitch_motor_1, child upper_arm2_1, origin xyz=0.0 0.0 0.0 rpy=0.0 0.0 0.0, axis 0 0 1, limit lower=-2.4056 upper=2.4056 effort=132 velocity=15.5
- added joint wrist_pitch_2: type revolute, parent wrist_pitch_motor_2, child upper_arm2_2, origin xyz=0.0 0.0 0.0 rpy=0.0 0.0 0.0, axis 0 0 1, limit lower=-2.3266 upper=2.3266 effort=132 velocity=15.5
- added joint wrist_pitch_stator_1: type fixed, parent upper_arm1_1, child wrist_pitch_motor_1, origin xyz=0.2 0.0 0.0 rpy=0.0 0.0 0.0
- added joint wrist_pitch_stator_2: type fixed, parent upper_arm1_2, child wrist_pitch_motor_2, origin xyz=0.2 0.0 0.0 rpy=0.0 0.0 0.0
- added joint wrist_yaw_1: type revolute, parent upper_arm2_1, child wrist_1, origin xyz=0.1 0.0 0.0 rpy=0.0 1.57079632679 0.0, axis 0 0 1, limit lower=-2.4056 upper=2.4056 effort=132 velocity=15.5
- added joint wrist_yaw_2: type revolute, parent upper_arm2_2, child wrist_2, origin xyz=0.1 0.0 0.0 rpy=0.0 1.57079632679 0.0, axis 0 0 1, limit lower=-2.3266 upper=2.3266 effort=132 velocity=15.5
- joint elbow_pitch_1: child upper_arm_1 -> upper_arm1_1
- joint elbow_pitch_2: child upper_arm_2 -> upper_arm1_2
- joint shoulder_yaw_1: origin xyz=0.30000000000000004 0.175 0.1 rpy=0.0 0.0 0.0 -> xyz=0.30000000000000004 0.175 0.1 rpy=-0.0 0.0 0.0

File: cetc_sat_urdf/urdf/parts/cetc_sat_arm.urdf.xacro (robot description, xacro)
@@ -48,7 +48,7 @@
 <link name="lower_arm_${arm_num}">
 	<inertial>
-		<origin xyz="0.0 0.0 0.0"/>
+		<origin xyz="${lower_arm_length / 2} 0.0 0.0"/>
 		<mass value="${lower_arm_mass}"/>
-		<inertia ixx="${LowerArm_xx}" ixy="${LowerArm_xy}" ixz="${LowerArm_xz}" iyy="${LowerArm_xx}" iyz="${LowerArm_yz}" izz="${LowerArm_zz}"/>
+		<inertia ixx="${LowerArm_xx}" ixy="${LowerArm_xy}" ixz="${LowerArm_xz}" iyy="${LowerArm_yy}" iyz="${LowerArm_yz}" izz="${LowerArm_zz}"/>
 	</inertial>
 	<visual>
@@ -87,7 +87,7 @@
 <link name="upper_arm1_${arm_num}">
 	<inertial>
-		<origin xyz="0.0 0.0 0.0"/>
+		<origin xyz="${upper_arm1_length / 2} 0.0 0.0"/>
 		<mass value="${upper_arm1_mass}"/>
-		<inertia ixx="${UpperArm1_xx}" ixy="${UpperArm1_xy}" ixz="${UpperArm1_xz}" iyy="${UpperArm1_xx}" iyz="${UpperArm1_yz}" izz="${UpperArm1_zz}"/>
+		<inertia ixx="${UpperArm1_xx}" ixy="${UpperArm1_xy}" ixz="${UpperArm1_xz}" iyy="${UpperArm1_yy}" iyz="${UpperArm1_yz}" izz="${UpperArm1_zz}"/>
 	</inertial>
 	<visual>
@@ -126,7 +126,7 @@
 <link name="upper_arm2_${arm_num}">
 	<inertial>
-		<origin xyz="0.0 0.0 0.0"/>
+		<origin xyz="${upper_arm2_length / 2} 0.0 0.0"/>
 		<mass value="${upper_arm2_mass}"/>
-		<inertia ixx="${UpperArm2_xx}" ixy="${UpperArm2_xy}" ixz="${UpperArm2_xz}" iyy="${UpperArm2_xx}" iyz="${UpperArm2_yz}" izz="${UpperArm2_zz}"/>
+		<inertia ixx="${UpperArm2_xx}" ixy="${UpperArm2_xy}" ixz="${UpperArm2_xz}" iyy="${UpperArm2_yy}" iyz="${UpperArm2_yz}" izz="${UpperArm2_zz}"/>
 	</inertial>
 	<visual>
@@ -142,5 +142,5 @@
 		</geometry>
 	</collision>
-</link>
+</link>>
 <!-- /shoulder-elbow -->
 <link name="wrist_${arm_num}">
@@ -164,4 +164,23 @@
 	</collision>
 </link>
+<!--link name="ball_arm_${arm_num}">
+	<inertial>
+		<origin xyz="0.0 0.0 0.0"/>
+		<mass value="${ball_mass}"/>
+		<inertia ixx="${Ball_xx}" ixy="${Ball_xy}" ixz="${Ball_xz}" iyy="${Ball_yy}" iyz="${Ball_yz}" izz="${Ball_zz}"/>
+	</inertial>
+	<visual>
+		<origin xyz="0.0 0.0 0.0" rpy="0.0 0.0 0.0"/>
+		<geometry>
+			<sphere radius="${ball_radius}"/>
+		</geometry>
+	</visual>
+	<collision>
+		<origin xyz="0.0 0.0 0.0" rpy="0.0 0.0 0.0"/>
+		<geometry>
+			<sphere radius="${ball_radius}"/>
+		</geometry>
+	</collision>
+</link-->
 <xacro:dagana_gripper name="dagana_${arm_num}" parent_link="wrist_${arm_num}" joint_type="fixed">
 	<origin xyz="0 0 0" rpy="0 0 0"/>
@@ -203,10 +222,10 @@
 	<limit lower="${j_pitch_2_lower[arm_num-1]}" upper="${j_pitch_2_upper[arm_num-1]}" effort="${motor_effort}" velocity="${motor_velocity}"/>
 </joint>
-<joint name="wrist_pitch_motor_${arm_num}" type="fixed">
+<joint name="wrist_pitch_stator_${arm_num}" type="fixed">
 	<parent link="upper_arm1_${arm_num}"/>
 	<child link="wrist_pitch_motor_${arm_num}"/>
 	<origin xyz="${WristPitch_Ox} ${WristPitch_Oy} ${WristPitch_Oz}" rpy="${WristPitch_roll} ${WristPitch_pitch} ${WristPitch_yaw}"/>
 </joint>
-<joint name="wrist_pitch_joint_${arm_num}" type="revolute">
+<joint name="wrist_pitch_${arm_num}" type="revolute">
 	<parent link="wrist_pitch_motor_${arm_num}"/>
 	<child link="upper_arm2_${arm_num}"/>
@@ -216,5 +235,5 @@
 </joint>
 <!-- end effector  -->
-<joint name="wrist_yaw_joint_${arm_num}" type="revolute">
+<joint name="wrist_yaw_${arm_num}" type="revolute">
 	<parent link="upper_arm2_${arm_num}"/>
 	<child link="wrist_${arm_num}"/>
@@ -223,5 +242,10 @@
 	<limit lower="${j_pitch_2_lower[arm_num-1]}" upper="${j_pitch_2_upper[arm_num-1]}" effort="${motor_effort}" velocity="${motor_velocity}"/>
 </joint>
-<xacro:if value="${PAYLOAD}">
+<!--joint name="hand_joint_${arm_num}" type="fixed">
+	<parent link="wrist_${arm_num}"/>
+	<child link="ball_arm_${arm_num}"/>
+	<origin xyz="0 0 ${ball_radius}" rpy="0 0 0"/>
+</joint-->
+<!--xacro:if value="${PAYLOAD}">
 	<link name="payload_${arm_num}">
 		<inertial>
@@ -242,5 +266,5 @@
 		<child link="payload_${arm_num}"/>
 	</joint>
-</xacro:if>
+</xacro:if-->
 </xacro:macro>
 <!-- /macro arms -->

File: cetc_sat_urdf/urdf/parts/cetc_sat_leg.urdf.xacro (robot description, xacro)
@@ -66,7 +66,7 @@
 <link name="upper_leg_${leg_num}">
 	<inertial>
-		<origin xyz="0.0 0.0 0.0"/>
+		<origin xyz="${upper_leg_length / 2} 0.0 0.0"/>
 		<mass value="${upper_leg_mass}"/>
-		<inertia ixx="${UpperLeg_xx}" ixy="${UpperLeg_xy}" ixz="${UpperLeg_xz}" iyy="${UpperLeg_xx}" iyz="${UpperLeg_yz}" izz="${UpperLeg_zz}"/>
+		<inertia ixx="${UpperLeg_xx}" ixy="${UpperLeg_xy}" ixz="${UpperLeg_xz}" iyy="${UpperLeg_yy}" iyz="${UpperLeg_yz}" izz="${UpperLeg_zz}"/>
 	</inertial>
 	<origin xyz="0.0 0.0 0.0" rpy="0.0 0.0 0.0"/>
@@ -87,7 +87,7 @@
 <link name="lower_leg_${leg_num}">
 	<inertial>
-		<origin xyz="0.0 0.0 0.0"/>
+		<origin xyz="${lower_leg_length / 2} 0.0 0.0"/>
 		<mass value="${lower_leg_mass}"/>
-		<inertia ixx="${LowerLeg_xx}" ixy="${LowerLeg_xy}" ixz="${LowerLeg_xz}" iyy="${LowerLeg_xx}" iyz="${LowerLeg_yz}" izz="${LowerLeg_zz}"/>
+		<inertia ixx="${LowerLeg_xx}" ixy="${LowerLeg_xy}" ixz="${LowerLeg_xz}" iyy="${LowerLeg_yy}" iyz="${LowerLeg_yz}" izz="${LowerLeg_zz}"/>
 	</inertial>
 	<visual>

File: cetc_sat_urdf/urdf/parts/inertial_properties.urdf.xacro (robot description, xacro)
@@ -51,37 +51,37 @@
     <xacro:property name="Pelvis_zz" value="${1/12 * pelvis_mass * (pelvis_width * pelvis_width + pelvis_length * pelvis_length)}"/>
     <!-- Upper Leg -->
-    <xacro:property name="UpperLeg_xx" value="${1/3 * upper_leg_mass * (upper_leg_width * upper_leg_width + upper_leg_height * upper_leg_height)}"/>
+    <xacro:property name="UpperLeg_xx" value="${1/12 * upper_leg_mass * (upper_leg_width * upper_leg_width + upper_leg_height * upper_leg_height)}"/>
     <xacro:property name="UpperLeg_xy" value="0.0"/>
     <xacro:property name="UpperLeg_xz" value="0.0"/>
-    <xacro:property name="UpperLeg_yy" value="${1/3 * upper_leg_mass * (upper_leg_length * upper_leg_length + upper_leg_height * upper_leg_height)}"/>
+    <xacro:property name="UpperLeg_yy" value="${1/12 * upper_leg_mass * (upper_leg_length * upper_leg_length + upper_leg_height * upper_leg_height)}"/>
     <xacro:property name="UpperLeg_yz" value="0.0"/>
-    <xacro:property name="UpperLeg_zz" value="${1/3 * upper_leg_mass * (upper_leg_width * upper_leg_width + upper_leg_length * upper_leg_length)}"/>
+    <xacro:property name="UpperLeg_zz" value="${1/12 * upper_leg_mass * (upper_leg_width * upper_leg_width + upper_leg_length * upper_leg_length)}"/>
     <!-- Lower Leg -->
-    <xacro:property name="LowerLeg_xx" value="${1/3 * lower_leg_mass * (lower_leg_width * lower_leg_width + lower_leg_height * lower_leg_height)}"/>
+    <xacro:property name="LowerLeg_xx" value="${1/12 * lower_leg_mass * (lower_leg_width * lower_leg_width + lower_leg_height * lower_leg_height)}"/>
     <xacro:property name="LowerLeg_xy" value="0.0"/>
     <xacro:property name="LowerLeg_xz" value="0.0"/>
-    <xacro:property name="LowerLeg_yy" value="${1/3 * lower_leg_mass * (lower_leg_length * lower_leg_length + lower_leg_height * lower_leg_height)}"/>
+    <xacro:property name="LowerLeg_yy" value="${1/12 * lower_leg_mass * (lower_leg_length * lower_leg_length + lower_leg_height * lower_leg_height)}"/>
     <xacro:property name="LowerLeg_yz" value="0.0"/>
-    <xacro:property name="LowerLeg_zz" value="${1/3 * lower_leg_mass * (lower_leg_width * lower_leg_width + lower_leg_length * lower_leg_length)}"/>
+    <xacro:property name="LowerLeg_zz" value="${1/12 * lower_leg_mass * (lower_leg_width * lower_leg_width + lower_leg_length * lower_leg_length)}"/>
     <!-- Upper Arm -->
-    <xacro:property name="UpperArm1_xx" value="${1/3 * upper_arm1_mass * (upper_arm1_width * upper_arm1_width + upper_arm1_height * upper_arm1_height)}"/>
+    <xacro:property name="UpperArm1_xx" value="${1/12 * upper_arm1_mass * (upper_arm1_width * upper_arm1_width + upper_arm1_height * upper_arm1_height)}"/>
     <xacro:property name="UpperArm1_xy" value="0.0"/>
     <xacro:property name="UpperArm1_xz" value="0.0"/>
-    <xacro:property name="UpperArm1_yy" value="${1/3 * upper_arm1_mass * (upper_arm1_length * upper_arm1_length + upper_arm1_height * upper_arm1_height)}"/>
+    <xacro:property name="UpperArm1_yy" value="${1/12 * upper_arm1_mass * (upper_arm1_length * upper_arm1_length + upper_arm1_height * upper_arm1_height)}"/>
     <xacro:property name="UpperArm1_yz" value="0.0"/>
-    <xacro:property name="UpperArm1_zz" value="${1/3 * upper_arm1_mass * (upper_arm1_width * upper_arm1_width + upper_arm1_length * upper_arm1_length)}"/>
-    <xacro:property name="UpperArm2_xx" value="${1/3 * upper_arm2_mass * (upper_arm2_width * upper_arm2_width + upper_arm2_height * upper_arm2_height)}"/>
+    <xacro:property name="UpperArm1_zz" value="${1/12 * upper_arm1_mass * (upper_arm1_width * upper_arm1_width + upper_arm1_length * upper_arm1_length)}"/>
+    <xacro:property name="UpperArm2_xx" value="${1/12 * upper_arm2_mass * (upper_arm2_width * upper_arm2_width + upper_arm2_height * upper_arm2_height)}"/>
     <xacro:property name="UpperArm2_xy" value="0.0"/>
     <xacro:property name="UpperArm2_xz" value="0.0"/>
-    <xacro:property name="UpperArm2_yy" value="${1/3 * upper_arm2_mass * (upper_arm2_length * upper_arm2_length + upper_arm2_height * upper_arm2_height)}"/>
+    <xacro:property name="UpperArm2_yy" value="${1/12 * upper_arm2_mass * (upper_arm2_length * upper_arm2_length + upper_arm2_height * upper_arm2_height)}"/>
     <xacro:property name="UpperArm2_yz" value="0.0"/>
-    <xacro:property name="UpperArm2_zz" value="${1/3 * upper_arm2_mass * (upper_arm2_width * upper_arm2_width + upper_arm2_length * upper_arm2_length)}"/>
+    <xacro:property name="UpperArm2_zz" value="${1/12 * upper_arm2_mass * (upper_arm2_width * upper_arm2_width + upper_arm2_length * upper_arm2_length)}"/>
     <!-- Lower Arm -->
-    <xacro:property name="LowerArm_xx" value="${1/3 * lower_arm_mass * (lower_arm_width * lower_arm_width + lower_arm_height * lower_arm_height)}"/>
+    <xacro:property name="LowerArm_xx" value="${1/12 * lower_arm_mass * (lower_arm_width * lower_arm_width + lower_arm_height * lower_arm_height)}"/>
     <xacro:property name="LowerArm_xy" value="0.0"/>
     <xacro:property name="LowerArm_xz" value="0.0"/>
-    <xacro:property name="LowerArm_yy" value="${1/3 * lower_arm_mass * (lower_arm_length * lower_arm_length + lower_arm_height * lower_arm_height)}"/>
+    <xacro:property name="LowerArm_yy" value="${1/12 * lower_arm_mass * (lower_arm_length * lower_arm_length + lower_arm_height * lower_arm_height)}"/>
     <xacro:property name="LowerArm_yz" value="0.0"/>
-    <xacro:property name="LowerArm_zz" value="${1/3 * lower_arm_mass * (lower_arm_width * lower_arm_width + lower_arm_length * lower_arm_length)}"/>
+    <xacro:property name="LowerArm_zz" value="${1/12 * lower_arm_mass * (lower_arm_width * lower_arm_width + lower_arm_length * lower_arm_length)}"/>
     <!-- Ball (hollow sphere) -->
     <xacro:property name="Ball_xx" value="${2/3 * ball_mass * ball_radius * ball_radius}"/>
