Commit message: parameters passed thorugh yaml file

File: cetc_sat_urdf/urdf/cetc_sat_base.urdf.xacro (robot description, xacro)
@@ -9,4 +9,6 @@
 <!--xacro:include filename="$(find cetc_sat_urdf)/urdf/parts/inertial_properties.urdf.xacro" /-->
 <xacro:include filename="$(find cetc_sat_urdf)/urdf/parts/limits.urdf.xacro" />
+<xacro:property name="yaml_file" value="$(find cetc_sat_urdf)/urdf/config/kinematics_properties.yaml" />
+<xacro:property name="props" value="${load_yaml(yaml_file)}"/>
 <link name="base_link"/>
 <link name="pelvis">

File: cetc_sat_urdf/urdf/parts/cetc_sat_arm.urdf.xacro (robot description, xacro)
@@ -9,5 +9,5 @@
 		<origin xyz="0.0 0.0 0.0"  rpy="0.0 0.0 0.0"/>
 		<geometry>
-			<cylinder radius="${cylinder_radius}" length="${cylinder_length}"/>
+			<cylinder radius="${props['cylinder_radius']}" length="${props['cylinder_length']}"/>
 		</geometry>
 		<material name="dark_grey"/>
@@ -16,5 +16,5 @@
 		<origin xyz="0.0 0.0 0.0"  rpy="0.0 0.0 0.0"/>
 		<geometry>
-			<cylinder radius="${cylinder_radius}" length="${cylinder_length}"/>
+			<cylinder radius="${props['cylinder_radius']}" length="${props['cylinder_length']}"/>
 		</geometry>
 	</collision>
@@ -23,13 +23,13 @@
 <link name="arm${arm_num}_1">
 	<visual>
-		<origin xyz="${Pitch_2_Ox / 2} 0.0 0.0"  rpy="0.0 0.0 0.0"/>
+		<origin xyz="${props['Pitch_2_Ox'] / 2} 0.0 0.0"  rpy="0.0 0.0 0.0"/>
 		<geometry>
-			<box size="${big_box_length} ${big_box_width} ${big_box_height}"/>
+			<box size="${props['big_box_length']} ${props['big_box_width']} ${props['big_box_height']}"/>
 		</geometry>
 	</visual>
 	<collision>
-		<origin xyz="${Pitch_2_Ox / 2} 0.0 0.0"  rpy="0.0 0.0 0.0"/>
+		<origin xyz="${props['Pitch_2_Ox'] / 2} 0.0 0.0"  rpy="0.0 0.0 0.0"/>
 		<geometry>
-			<box size="${big_box_length} ${big_box_width} ${big_box_height}"/>
+			<box size="${props['big_box_length']} ${props['big_box_width']} ${props['big_box_height']}"/>
 		</geometry>
 	</collision>
@@ -39,14 +39,14 @@
 <link name="arm${arm_num}_2">
 	<visual>
-		<origin xyz="${EndEffector_Ox / 2} 0.0 0.0"  rpy="0.0 0.0 0.0"/>
+		<origin xyz="${props['EndEffector_Ox'] / 2} 0.0 0.0"  rpy="0.0 0.0 0.0"/>
 		<geometry>
-			<box size="${small_box_length} ${small_box_width} ${small_box_height}"/>
+			<box size="${props['small_box_length']} ${props['small_box_width']} ${props['small_box_height']}"/>
 		</geometry>
 		<material name="dark_grey"/>
 	</visual>
 	<collision>
-		<origin xyz="${EndEffector_Ox / 2} 0.0 0.0"  rpy="0.0 0.0 0.0"/>
+		<origin xyz="${props['EndEffector_Ox'] / 2} 0.0 0.0"  rpy="0.0 0.0 0.0"/>
 		<geometry>
-			<box size="${small_box_length} ${small_box_width} ${small_box_height}"/>
+			<box size="${props['small_box_length']} ${props['small_box_width']} ${props['small_box_height']}"/>
 		</geometry>
 	</collision>
@@ -57,5 +57,5 @@
 		<origin xyz="0.0 0.0 0.0" rpy="0.0 0.0 0.0"/>
 		<geometry>
-			<sphere radius="${ball_radius}"/>
+			<sphere radius="${props['ball_radius']}"/>
 		</geometry>
 	</visual>
@@ -63,5 +63,5 @@
 		<origin xyz="0.0 0.0 0.0" rpy="0.0 0.0 0.0"/>
 		<geometry>
-			<sphere radius="${ball_radius}"/>
+			<sphere radius="${props['ball_radius']}"/>
 		</geometry>
 	</collision>
@@ -73,5 +73,5 @@
 	<parent link="${parent}"/>
 	<child link="shoulder_${arm_num}"/>
-	<origin xyz="${Shoulder_Ox} ${rot*Shoulder_Oy} ${Shoulder_Oz}" rpy="${Shoulder_roll} ${Shoulder_pitch} ${Shoulder_roll}"/>
+	<origin xyz="${props['Shoulder_Ox'] / 2 -0.1} ${rot*props['Shoulder_Oy'] / 2 - 0.05} ${props['Shoulder_Oz'] / 2}" rpy="${props['Shoulder_roll']} ${props['Shoulder_pitch']} ${props['Shoulder_yaw']}"/>
 	<axis xyz="0 0 1"/>
 	<limit lower="${j_shoulder_yaw_lower[arm_num-1]}" upper="${j_shoulder_yaw_upper[arm_num-1]}" effort="${j_shoulder_torque[arm_num-1]}" velocity="${j_shoulder_velocity[arm_num-1]}"/>
@@ -81,5 +81,5 @@
 	<parent link="shoulder_${arm_num}"/>
 	<child link="arm${arm_num}_1"/>
-	<origin xyz="${Pitch_1_Ox} ${Pitch_1_Oy} ${Pitch_1_Oz}" rpy="${Pitch_1_roll} ${Pitch_1_pitch} ${Pitch_1_yaw}"/>
+	<origin xyz="${props['Pitch_1_Ox']} ${props['Pitch_1_Oy']} ${props['Pitch_1_Oz'] / 2}" rpy="${props['Pitch_1_roll']} ${-props['Pitch_1_pitch']} ${props['Pitch_1_yaw']}"/>
 	<axis xyz="0 1 0"/>
 	<limit lower="${j_pitch_1_lower[arm_num-1]}" upper="${j_pitch_1_upper[arm_num-1]}" effort="${j_pitch_1_torque[arm_num-1]}" velocity="${j_pitch_1_velocity[arm_num-1]}"/>
@@ -89,5 +89,5 @@
 	<parent link="arm${arm_num}_1"/>
 	<child link="arm${arm_num}_2"/>
-	<origin xyz="${Pitch_2_Ox} ${Pitch_2_Oy} ${Pitch_2_Oz}" rpy="${Pitch_2_roll} ${Pitch_2_pitch} ${Pitch_2_yaw}"/>
+	<origin xyz="${props['Pitch_2_Ox']} ${props['Pitch_2_Oy']} ${props['Pitch_2_Oz']}" rpy="${props['Pitch_2_roll']} ${props['Pitch_2_pitch']} ${props['Pitch_2_yaw']}"/>
 	<axis xyz="0 1 0"/>
 	<limit lower="${j_pitch_2_lower[arm_num-1]}" upper="${j_pitch_2_upper[arm_num-1]}" effort="${j_pitch_2_torque[arm_num-1]}" velocity="${j_pitch_2_velocity[arm_num-1]}"/>
@@ -97,5 +97,5 @@
 	<parent link="arm${arm_num}_2"/>
 	<child link="ball_arm_${arm_num}"/>
-	<origin xyz="${EndEffector_Ox} ${EndEffector_Oy} ${EndEffector_Oz}" rpy="${EndEffector_roll} ${EndEffector_pitch} ${EndEffector_yaw}"/>
+	<origin xyz="${props['EndEffector_Ox']} ${props['EndEffector_Oy']} ${props['EndEffector_Oz']}" rpy="${props['EndEffector_roll']} ${props['EndEffector_pitch']} ${props['EndEffector_yaw']}"/>
 </joint>
 </xacro:macro>

File: cetc_sat_urdf/urdf/parts/cetc_sat_leg.urdf.xacro (robot description, xacro)
@@ -9,5 +9,5 @@
 		<origin xyz="0.0 0.0 0.0"  rpy="0.0 0.0 0.0"/>
 	  	<geometry>
-	 		<cylinder radius="${cylinder_radius}" length="${cylinder_length}"/>
+	 		<cylinder radius="${props['cylinder_radius']}" length="${props['cylinder_length']}"/>
 	  	</geometry>
   		<material name="dark_grey"/>
@@ -16,5 +16,5 @@
 		<origin xyz="0.0 0.0 0.0"  rpy="0.0 0.0 0.0"/>
 		<geometry>
-			<cylinder radius="${cylinder_radius}" length="${cylinder_length}"/>
+			<cylinder radius="${props['cylinder_radius']}" length="${props['cylinder_length']}"/>
 		</geometry>
 	</collision>
@@ -23,14 +23,14 @@
 	<origin xyz="0.0 0.0 0.0" rpy="0.0 0.0 0.0"/>
 	<visual>
-		<origin xyz="${Leg_3_Ox / 2} 0.0 0.0"  rpy="0.0 0.0 0.0"/>
+		<origin xyz="${props['Leg_3_Ox'] / 2} 0.0 0.0"  rpy="0.0 0.0 0.0"/>
 	  	<geometry>
-	 		<box size="${big_box_length} ${big_box_width} ${big_box_height}"/>
+	 		<box size="${props['big_box_length']} ${props['big_box_width']} ${props['big_box_height']}"/>
 	  	</geometry>
   		<material name="dark_grey"/>
 	</visual>
 	<collision>
-		<origin xyz="${Leg_3_Ox / 2} 0.0 0.0"  rpy="0.0 0.0 0.0"/>
+		<origin xyz="${props['Leg_3_Ox'] / 2} 0.0 0.0"  rpy="0.0 0.0 0.0"/>
 		<geometry>
-			<box size="${big_box_length} ${big_box_width} ${big_box_height}"/>
+			<box size="${props['big_box_length']} ${props['big_box_width']} ${props['big_box_height']}"/>
 		</geometry>
 	</collision>
@@ -38,14 +38,14 @@
 <link name="lower_leg_${leg_num}">
 <visual>
-		<origin xyz="${Ankle_Ox / 2} 0.0 0.0"  rpy="0.0 0.0 0.0"/>
+		<origin xyz="${props['Ankle_Ox'] / 2} 0.0 0.0"  rpy="0.0 0.0 0.0"/>
 	  	<geometry>
-	 		<box size="${small_box_length} ${small_box_width} ${small_box_height}"/>
+	 		<box size="${props['small_box_length']} ${props['small_box_width']} ${props['small_box_height']}"/>
 	  	</geometry>
   		<material name="dark_grey"/>
 	</visual>
 	<collision>
-		<origin xyz="${Ankle_Ox / 2} 0.0 0.0"  rpy="0.0 0.0 0.0"/>
+		<origin xyz="${props['Ankle_Ox'] / 2} 0.0 0.0"  rpy="0.0 0.0 0.0"/>
 		<geometry>
-	 		<box size="${small_box_length} ${small_box_width} ${small_box_height}"/>
+	 		<box size="${props['small_box_length']} ${props['small_box_width']} ${props['small_box_height']}"/>
 		</geometry>
 	</collision>
@@ -55,5 +55,5 @@
 		<origin xyz="0.0 0.0 0.0" rpy="0.0 0.0 0.0"/>
 		<geometry>
-			<sphere radius="${ball_radius}"/>
+			<sphere radius="${props['ball_radius']}"/>
 		</geometry>
 	</visual>
@@ -61,5 +61,5 @@
 		<origin xyz="0.0 0.0 0.0" rpy="0.0 0.0 0.0"/>
 		<geometry>
-			<sphere radius="${ball_radius}"/>
+			<sphere radius="${props['ball_radius']}"/>
 		</geometry>
 	</collision>
@@ -69,5 +69,5 @@
 	<parent link="pelvis"/>
 	<child link="hip_${leg_num}"/>
-	<origin xyz="${origin_x*Leg_1_Ox} ${origin_y*Leg_1_Oy} ${Leg_1_Oz}" rpy="${Leg_1_roll} ${Leg_1_pitch} ${Leg_1_yaw}"/>
+	<origin xyz="${origin_x*props['Leg_1_Ox'] / 2} ${origin_y*(-props['Leg_1_Oy'] / 2)} ${props['Leg_1_Oz']}" rpy="${props['Leg_1_roll']} ${props['Leg_1_pitch']} ${props['Leg_1_yaw']}"/>
 	<axis xyz="0 0 1"/>
    <limit lower="${hip_roll_lower[leg_num-1]}" upper="${hip_roll_upper[leg_num-1]}" effort="${motor_A_effort}" velocity="${motor_A_velocity}"/> <!-- 200 Nm, 1 rad/s-->
@@ -76,5 +76,5 @@
 	<parent link="hip_${leg_num}"/>
 	<child link="upper_leg_${leg_num}"/>
-	<origin xyz="${Leg_2_Ox} ${mirror*Leg_2_Oy} ${Leg_2_Oz}" rpy="${Leg_2_roll} ${Leg_2_pitch} ${Leg_2_yaw}"/>
+	<origin xyz="${props['Leg_2_Ox']} ${mirror*(-props['Leg_2_Oy']/2)} ${props['Leg_2_Oz']}" rpy="${props['Leg_2_roll']} ${props['Leg_2_pitch']} ${props['Leg_2_yaw']}"/>
 	<axis xyz="0 1 0"/>
    <limit lower="${hip_pitch_lower[leg_num-1]}" upper="${hip_pitch_upper[leg_num-1]}" effort="${motor_A_effort}" velocity="${motor_A_velocity}"/> <!-- 200 Nm, 1 rad/s-->
@@ -83,5 +83,5 @@
 	<parent link="upper_leg_${leg_num}"/>
 	<child link="lower_leg_${leg_num}"/>
-	<origin xyz="${Leg_3_Ox} ${Leg_3_Oy} ${Leg_3_Oz}" rpy="${Leg_3_roll} ${Leg_3_pitch} ${Leg_3_yaw}"/>
+	<origin xyz="${props['Leg_3_Ox']} ${props['Leg_3_Oy']} ${props['Leg_3_Oz']}" rpy="${props['Leg_3_roll']} ${props['Leg_3_pitch']} ${props['Leg_3_yaw']}"/>
 	<axis xyz="0 1 0"/>
    <limit lower="${knee_pitch_lower[leg_num-1]}" upper="${knee_pitch_upper[leg_num-1]}" effort="${motor_A_effort}" velocity="${motor_A_velocity}"/> <!-- 200 Nm, 1 rad/s-->
@@ -90,5 +90,5 @@
 	<parent link="lower_leg_${leg_num}"/>
 	<child link="ball_${leg_num}"/>
-	<origin xyz="${Ankle_Ox} ${Ankle_Oy} ${Ankle_Oz}" rpy="${Ankle_roll} ${Ankle_pitch} ${Ankle_yaw}"/>
+	<origin xyz="${props['Ankle_Ox']} ${props['Ankle_Oy']} ${props['Ankle_Oz']}" rpy="${props['Ankle_roll']} ${props['Ankle_pitch']} ${props['Ankle_yaw']}"/>
 </joint>
 </xacro:macro>

File: cetc_sat_urdf/urdf/parts/kinematics_properties.urdf.xacro (robot description, xacro)
@@ -2,5 +2,5 @@
 <robot  xmlns:xacro="http://ros.org/wiki/xacro">
 <!-- link dimensions -->
-<xacro:property name="cylinder_radius" value="0.07"/>
+<!--xacro:property name="cylinder_radius" value="0.07"/>
 <xacro:property name="cylinder_length" value="0.1"/>
 <xacro:property name="big_box_length" value="0.4"/>
@@ -10,5 +10,5 @@
 <xacro:property name="small_box_width" value="0.05"/>
 <xacro:property name="small_box_height" value="0.05"/>
-<xacro:property name="ball_radius" value="0.05"/>
+<xacro:property name="ball_radius" value="0.05"/-->
 <!--pelvis dimensions: length: 0.80-1.1m, width: 0.45-0.60m-->
 <xacro:property name="pelvis_length" value="0.80"/>
@@ -24,5 +24,5 @@
 <!-- Origin -->
 <xacro:property name="Leg_2_Ox" value="0.0"/>
-<xacro:property name="Leg_2_Oy" value="-${cylinder_radius / 2}"/>
+<xacro:property name="Leg_2_Oy" value="-${props['cylinder_radius'] / 2}"/>
 <xacro:property name="Leg_2_Oz" value="0.0"/>
 <xacro:property name="Leg_2_roll" value="0.0"/>
@@ -30,5 +30,5 @@
 <xacro:property name="Leg_2_yaw" value="0.0"/>
 <!-- Origin -->
-<xacro:property name="Leg_3_Ox" value="${big_box_length}"/>
+<xacro:property name="Leg_3_Ox" value="${props['big_box_length']}"/>
 <xacro:property name="Leg_3_Oy" value="0.0"/>
 <xacro:property name="Leg_3_Oz" value="0.0"/>
@@ -37,5 +37,5 @@
 <xacro:property name="Leg_3_yaw" value="0.0"/>
 <!-- Origin -->
-<xacro:property name="Ankle_Ox" value="${big_box_length}"/>
+<xacro:property name="Ankle_Ox" value="${props['big_box_length']}"/>
 <xacro:property name="Ankle_Oy" value="0.0"/>
 <xacro:property name="Ankle_Oz" value="0.0"/>
@@ -52,9 +52,9 @@
 <xacro:property name="Pitch_1_Ox" value="0.0"/>
 <xacro:property name="Pitch_1_Oy" value="0.0"/>
-<xacro:property name="Pitch_1_Oz" value="${cylinder_length / 2}"/>
+<xacro:property name="Pitch_1_Oz" value="${props['cylinder_length'] / 2}"/>
 <xacro:property name="Pitch_1_roll" value="0.0"/>
 <xacro:property name="Pitch_1_pitch" value="${-PI_2}"/>
 <xacro:property name="Pitch_1_yaw" value="0.0"/>
-<xacro:property name="Pitch_2_Ox" value="${big_box_length}"/>
+<xacro:property name="Pitch_2_Ox" value="${props['big_box_length']}"/>
 <xacro:property name="Pitch_2_Oy" value="0.0"/>
 <xacro:property name="Pitch_2_Oz" value="0.0"/>
@@ -62,5 +62,5 @@
 <xacro:property name="Pitch_2_pitch" value="0.0"/>
 <xacro:property name="Pitch_2_yaw" value="0.0"/>
-<xacro:property name="EndEffector_Ox" value="${big_box_length}"/>
+<xacro:property name="EndEffector_Ox" value="${props['big_box_length']}"/>
 <xacro:property name="EndEffector_Oy" value="0.0"/>
 <xacro:property name="EndEffector_Oz" value="0.0"/>

Commit message: First perception draft

File: cetc_sat_urdf/urdf/cetc_sat_base.urdf.xacro (robot description, xacro)
@@ -38,4 +38,117 @@
     <origin xyz="0 0 0" rpy="0 0 0" />
 </joint>
+<xacro:if value="${ADD_SENSORS}">
+    <xacro:include filename="$(find realsense_gazebo_description)/urdf/_d435i.urdf.xacro" />
+    <!-- LEFT D435 CAMERA -->
+    <xacro:sensor_d435i parent="pelvis"
+        name="D435_left"
+        topics_ns="D435_left"
+        enable_pointCloud="true"
+        align_depth="true"
+        unite_imu_method="false"
+        visualize="true"
+        accel_fps="300"
+        gyro_fps="300"
+        depth_width="1280"
+        depth_height="720"
+        depth_fps="90"
+        infra_width="1280"
+        infra_height="720"
+        infra_fps="90"
+        color_width="1280"
+        color_height="720"
+        color_fps="30">
+        <origin xyz="-0.1 0.22 0" rpy="0 0.25 1.57"/>
+    </xacro:sensor_d435i>
+    <!-- RIGHT D435 CAMERA -->
+    <xacro:sensor_d435i parent="pelvis"
+        name="D435_right"
+        topics_ns="D435_right"
+        enable_pointCloud="true"
+        align_depth="true"
+        unite_imu_method="false"
+        visualize="true"
+        accel_fps="300"
+        gyro_fps="300"
+        depth_width="1280"
+        depth_height="720"
+        depth_fps="90"
+        infra_width="1280"
+        infra_height="720"
+        infra_fps="90"
+        color_width="1280"
+        color_height="720"
+        color_fps="30">
+        <origin xyz="-0.1 -0.22 0" rpy="0 0.25 -1.57"/>
+    </xacro:sensor_d435i>
+    <!-- REAR D435 CAMERA -->
+    <xacro:sensor_d435i parent="pelvis"
+        name="D435_rear"
+        topics_ns="D435_rear"
+        enable_pointCloud="true"
+        align_depth="true"
+        unite_imu_method="false"
+        visualize="true"
+        accel_fps="300"
+        gyro_fps="300"
+        depth_width="1280"
+        depth_height="720"
+        depth_fps="90"
+        infra_width="1280"
+        infra_height="720"
+        infra_fps="90"
+        color_width="1280"
+        color_height="720"
+        color_fps="30">
+        <origin xyz="-0.39 0 0" rpy="0 0.25 3.14"/>
+    </xacro:sensor_d435i>
+    <!-- FRONT1 D435 CAMERA -->
+    <xacro:sensor_d435i parent="pelvis"
+        name="D435_front1"
+        topics_ns="D435_front1"
+        enable_pointCloud="true"
+        align_depth="true"
+        unite_imu_method="false"
+        visualize="true"
+        accel_fps="300"
+        gyro_fps="300"
+        depth_width="1280"
+        depth_height="720"
+        depth_fps="90"
+        infra_width="1280"
+        infra_height="720"
+        infra_fps="90"
+        color_width="1280"
+        color_height="720"
+        color_fps="30">
+        <origin xyz="0.40 -0.075 0" rpy="1.57 0 0.21"/>
+    </xacro:sensor_d435i>
+    <!-- FRONT2 D435 CAMERA -->
+    <xacro:sensor_d435i parent="pelvis"
+        name="D435_front2"
+        topics_ns="D435_front2"
+        enable_pointCloud="true"
+        align_depth="true"
+        unite_imu_method="false"
+        visualize="true"
+        accel_fps="300"
+        gyro_fps="300"
+        depth_width="1280"
+        depth_height="720"
+        depth_fps="90"
+        infra_width="1280"
+        infra_height="720"
+        infra_fps="90"
+        color_width="1280"
+        color_height="720"
+        color_fps="30">
+        <origin xyz="0.40 0.075 0" rpy="1.57 0 -0.21"/>
+    </xacro:sensor_d435i>
+    <!-- Velodyne -->
+    <xacro:include filename="$(find velodyne_description)/urdf/VLP-16.urdf.xacro"/>
+    <xacro:VLP-16 parent="pelvis" name="velodyne" topic="/velodyne_points" hz="10" samples="440">
+        <origin xyz="0.36 0 0.11" rpy="0 0 0" />
+    </xacro:VLP-16>
+</xacro:if>
 <xacro:if value="${ADD_UPPER_BODY}">
     <xacro:include filename="$(find cetc_sat_urdf)/urdf/parts/arms.urdf.xacro" />

File: cetc_sat_urdf/urdf/config/cetc_sat.urdf.xacro (robot description, xacro)
@@ -7,8 +7,10 @@
 <xacro:arg name="upper_body" default="true"/>
 <xacro:arg name="floating_joint" default="true"/>
+<xacro:arg name="sensors" default="true"/>
 <!-- ************SELECT PARTS*************-->
 <!-- *************************************-->
 <xacro:property name="ADD_LEGS" value="$(arg legs)" />
 <xacro:property name="ADD_UPPER_BODY" value="$(arg upper_body)" />
+<xacro:property name="ADD_SENSORS" value="$(arg sensors)" />
 <xacro:property name="ADD_FLOATING_BASE" value="$(arg floating_joint)" />
 <xacro:property name="ADD_VIRTUAL_FRAME" value="false" />

Commit message: removed deprecation warning for load_yaml() call by using xacro.load_yaml()

File: cetc_sat_urdf/urdf/cetc_sat_base.urdf.xacro (robot description, xacro)
@@ -6,7 +6,7 @@
 <xacro:include filename="$(find cetc_sat_urdf)/urdf/parts/limits.urdf.xacro" />
 <xacro:property name="yaml_file" value="$(find cetc_sat_urdf)/urdf/config/kinematics_properties.yaml" />
-<xacro:property name="props" value="${load_yaml(yaml_file)}"/>
+<xacro:property name="props" value="${xacro.load_yaml(yaml_file)}"/>
 <xacro:property name="yaml_file_inertial" value="$(find cetc_sat_urdf)/urdf/config/inertial_properties.yaml" />
-<xacro:property name="props_inertial" value="${load_yaml(yaml_file_inertial)}"/>
+<xacro:property name="props_inertial" value="${xacro.load_yaml(yaml_file_inertial)}"/>
 <link name="base_link"/>
 <link name="pelvis">

Commit message: added optional argument to specify from where to load codesign variables

File: cetc_sat_urdf/urdf/cetc_sat_base.urdf.xacro (robot description, xacro)
@@ -5,8 +5,11 @@
 <xacro:include filename="$(find cetc_sat_urdf)/urdf/parts/inertial_properties.urdf.xacro" />
 <xacro:include filename="$(find cetc_sat_urdf)/urdf/parts/limits.urdf.xacro" />
-<xacro:property name="yaml_file" value="$(find cetc_sat_urdf)/urdf/config/kinematics_properties.yaml" />
+<xacro:arg name="bilevel_codes" default="false" /> <!-- if true, load codes vars from externally provided files-->
+<xacro:arg name="inertial_props_path" default="$(find cetc_sat_urdf)/urdf/config/kinematics_properties.yaml" />
+<xacro:arg name="kinematic_props_path" default="$(find cetc_sat_urdf)/urdf/config/inertial_properties.yaml" />
+<xacro:property name="yaml_file_inertial" value="$(arg inertial_props_path)" />
+<xacro:property name="yaml_file" value="$(arg kinematic_props_path)" />
+<xacro:property name="props_inertial" value="${xacro.load_yaml(yaml_file_inertial)}"/>
 <xacro:property name="props" value="${xacro.load_yaml(yaml_file)}"/>
-<xacro:property name="yaml_file_inertial" value="$(find cetc_sat_urdf)/urdf/config/inertial_properties.yaml" />
-<xacro:property name="props_inertial" value="${xacro.load_yaml(yaml_file_inertial)}"/>
 <link name="base_link"/>
 <link name="pelvis">
