Commit message: added optional argument to load yaml for bilevel codes

File: cetc_sat_urdf/urdf/cetc_sat_base.urdf.xacro (robot description, xacro)
@@ -1,20 +1,16 @@
 <?xml version="1.0"?>
 <robot xmlns:xacro="http://ros.org/wiki/xacro" name="cetc_sat">
+<xacro:arg name="bilevel_codes" default="false" /> <!-- if true, load codes vars from externally provided files-->
+<xacro:arg name="sample_idx" default = "0"/>
 <xacro:include filename="$(find cetc_sat_urdf)/urdf/utils.urdf.xacro" />
 <xacro:include filename="$(find cetc_sat_urdf)/urdf/parts/kinematics_properties.urdf.xacro" />
+<!-- NOTE: here we need to include "kinematics_properties" first because "inertial_properties" depends on it-->
 <xacro:include filename="$(find cetc_sat_urdf)/urdf/parts/inertial_properties.urdf.xacro" />
 <xacro:include filename="$(find cetc_sat_urdf)/urdf/parts/limits.urdf.xacro" />
-<xacro:arg name="bilevel_codes" default="false" /> <!-- if true, load codes vars from externally provided files-->
-<xacro:arg name="inertial_props_path" default="$(find cetc_sat_urdf)/urdf/config/kinematics_properties.yaml" />
-<xacro:arg name="kinematic_props_path" default="$(find cetc_sat_urdf)/urdf/config/inertial_properties.yaml" />
-<xacro:property name="yaml_file_inertial" value="$(arg inertial_props_path)" />
-<xacro:property name="yaml_file" value="$(arg kinematic_props_path)" />
-<xacro:property name="props_inertial" value="${xacro.load_yaml(yaml_file_inertial)}"/>
-<xacro:property name="props" value="${xacro.load_yaml(yaml_file)}"/>
 <link name="base_link"/>
 <link name="pelvis">
 	<inertial>
 		<origin xyz="0.0 0.0 0.0"/>
-		<mass value="${props_inertial['pelvis_mass']}"/>
+		<mass value="${pelvis_mass}"/>
 		<inertia ixx="${Pelvis_xx}" ixy="${Pelvis_xy}" ixz="${Pelvis_xz}" iyy="${Pelvis_yy}" iyz="${Pelvis_yz}" izz="${Pelvis_zz}"/>
 	</inertial>

File: cetc_sat_urdf/urdf/parts/cetc_sat_arm.urdf.xacro (robot description, xacro)
@@ -8,5 +8,5 @@
 	<inertial>
 		<origin xyz="0.0 0.0 0.0"/>
-		<mass value="${props_inertial['motorA_mass']}"/>
+		<mass value="${motorA_mass}"/>
 		<inertia ixx="${MotorA_xx}" ixy="${MotorA_xy}" ixz="${MotorA_xz}" iyy="${MotorA_yy}" iyz="${MotorA_yz}" izz="${MotorA_zz}"/>
 	</inertial>
@@ -14,5 +14,5 @@
 		<origin xyz="0.0 0.0 0.0"  rpy="0.0 0.0 0.0"/>
 		<geometry>
-			<cylinder radius="${props['cylinder_radius']}" length="${props['cylinder_length']}"/>
+			<cylinder radius="${cylinder_radius}" length="${cylinder_length}"/>
 		</geometry>
 		<material name="dark_grey"/>
@@ -21,5 +21,5 @@
 		<origin xyz="0.0 0.0 0.0"  rpy="0.0 0.0 0.0"/>
 		<geometry>
-			<cylinder radius="${props['cylinder_radius']}" length="${props['cylinder_length']}"/>
+			<cylinder radius="${cylinder_radius}" length="${cylinder_length}"/>
 		</geometry>
 	</collision>
@@ -28,5 +28,5 @@
 	<inertial>
 		<origin xyz="0.0 0.0 0.0"/>
-		<mass value="${props_inertial['motorA_mass']}"/>
+		<mass value="${motorA_mass}"/>
 		<inertia ixx="${MotorA_xx}" ixy="${MotorA_xy}" ixz="${MotorA_xz}" iyy="${MotorA_yy}" iyz="${MotorA_yz}" izz="${MotorA_zz}"/>
 	</inertial>
@@ -34,5 +34,5 @@
 		<origin xyz="0.0 0.0 0.0"  rpy="0.0 0.0 0.0"/>
 	  	<geometry>
-	 		<cylinder radius="${props['cylinder_radius']}" length="${props['cylinder_length']}"/>
+	 		<cylinder radius="${cylinder_radius}" length="${cylinder_length}"/>
 	  	</geometry>
   		<material name="dark_grey"/>
@@ -41,5 +41,5 @@
 		<origin xyz="0.0 0.0 0.0"  rpy="0.0 0.0 0.0"/>
 		<geometry>
-			<cylinder radius="${props['cylinder_radius']}" length="${props['cylinder_length']}"/>
+			<cylinder radius="${cylinder_radius}" length="${cylinder_length}"/>
 		</geometry>
 	</collision>
@@ -48,17 +48,17 @@
 	<inertial>
 		<origin xyz="0.0 0.0 0.0"/>
-		<mass value="${props_inertial['big_box_mass']}"/>
+		<mass value="${big_box_mass}"/>
 		<inertia ixx="${BigBox_xx}" ixy="${BigBox_xy}" ixz="${BigBox_xz}" iyy="${BigBox_xx}" iyz="${BigBox_yz}" izz="${BigBox_zz}"/>
 	</inertial>
 	<visual>
-		<origin xyz="${props['big_box_length'] / 2} 0.0 0.0"  rpy="0.0 0.0 0.0"/>
+		<origin xyz="${big_box_length / 2} 0.0 0.0"  rpy="0.0 0.0 0.0"/>
 		<geometry>
-			<box size="${props['big_box_length']} ${props['big_box_width']} ${props['big_box_height']}"/>
+			<box size="${big_box_length} ${big_box_width} ${big_box_height}"/>
 		</geometry>
 	</visual>
 	<collision>
-		<origin xyz="${props['big_box_length'] / 2} 0.0 0.0"  rpy="0.0 0.0 0.0"/>
+		<origin xyz="${big_box_length / 2} 0.0 0.0"  rpy="0.0 0.0 0.0"/>
 		<geometry>
-			<box size="${props['big_box_length']} ${props['big_box_width']} ${props['big_box_height']}"/>
+			<box size="${big_box_length} ${big_box_width} ${big_box_height}"/>
 		</geometry>
 	</collision>
@@ -67,5 +67,5 @@
 	<inertial>
 		<origin xyz="0.0 0.0 0.0"/>
-		<mass value="${props_inertial['motorA_mass']}"/>
+		<mass value="${motorA_mass}"/>
 		<inertia ixx="${MotorA_xx}" ixy="${MotorA_xy}" ixz="${MotorA_xz}" iyy="${MotorA_yy}" iyz="${MotorA_yz}" izz="${MotorA_zz}"/>
 	</inertial>
@@ -73,5 +73,5 @@
 		<origin xyz="0.0 0.0 0.0"  rpy="0.0 0.0 0.0"/>
 	  	<geometry>
-	 		<cylinder radius="${props['cylinder_radius']}" length="${props['cylinder_length']}"/>
+	 		<cylinder radius="${cylinder_radius}" length="${cylinder_length}"/>
 	  	</geometry>
   		<material name="dark_grey"/>
@@ -80,5 +80,5 @@
 		<origin xyz="0.0 0.0 0.0"  rpy="0.0 0.0 0.0"/>
 		<geometry>
-			<cylinder radius="${props['cylinder_radius']}" length="${props['cylinder_length']}"/>
+			<cylinder radius="${cylinder_radius}" length="${cylinder_length}"/>
 		</geometry>
 	</collision>
@@ -87,18 +87,18 @@
 	<inertial>
 		<origin xyz="0.0 0.0 0.0"/>
-		<mass value="${props_inertial['small_box_mass']}"/>
+		<mass value="${small_box_mass}"/>
 		<inertia ixx="${SmallBox_xx}" ixy="${SmallBox_xy}" ixz="${SmallBox_xz}" iyy="${SmallBox_xx}" iyz="${SmallBox_yz}" izz="${SmallBox_zz}"/>
 	</inertial>
 	<visual>
-		<origin xyz="${props['small_box_length'] / 2} 0.0 0.0"  rpy="0.0 0.0 0.0"/>
+		<origin xyz="${small_box_length / 2} 0.0 0.0"  rpy="0.0 0.0 0.0"/>
 		<geometry>
-			<box size="${props['small_box_length']} ${props['small_box_width']} ${props['small_box_height']}"/>
+			<box size="${small_box_length} ${small_box_width} ${small_box_height}"/>
 		</geometry>
 		<material name="dark_grey"/>
 	</visual>
 	<collision>
-		<origin xyz="${props['small_box_length'] / 2} 0.0 0.0"  rpy="0.0 0.0 0.0"/>
+		<origin xyz="${small_box_length / 2} 0.0 0.0"  rpy="0.0 0.0 0.0"/>
 		<geometry>
-			<box size="${props['small_box_length']} ${props['small_box_width']} ${props['small_box_height']}"/>
+			<box size="${small_box_length} ${small_box_width} ${small_box_height}"/>
 		</geometry>
 	</collision>
@@ -108,5 +108,5 @@
     <inertial>
 		<origin xyz="0.0 0.0 0.0"/>
-		<mass value="${props_inertial['ball_mass']}"/>
+		<mass value="${ball_mass}"/>
 		<inertia ixx="${Ball_xx}" ixy="${Ball_xy}" ixz="${Ball_xz}" iyy="${Ball_yy}" iyz="${Ball_yz}" izz="${Ball_zz}"/>
 	</inertial>
@@ -114,5 +114,5 @@
 		<origin xyz="0.0 0.0 0.0" rpy="0.0 0.0 0.0"/>
 		<geometry>
-			<sphere radius="${props['ball_radius']}"/>
+			<sphere radius="${ball_radius}"/>
 		</geometry>
 	</visual>
@@ -120,5 +120,5 @@
 		<origin xyz="0.0 0.0 0.0" rpy="0.0 0.0 0.0"/>
 		<geometry>
-			<sphere radius="${props['ball_radius']}"/>
+			<sphere radius="${ball_radius}"/>
 		</geometry>
 	</collision>

File: cetc_sat_urdf/urdf/parts/cetc_sat_leg.urdf.xacro (robot description, xacro)
@@ -7,5 +7,5 @@
 	<inertial>
 		<origin xyz="0.0 0.0 0.0"/>
-		<mass value="${props_inertial['motorA_mass']}"/>
+		<mass value="${motorA_mass}"/>
 		<inertia ixx="${MotorA_xx}" ixy="${MotorA_xy}" ixz="${MotorA_xz}" iyy="${MotorA_yy}" iyz="${MotorA_yz}" izz="${MotorA_zz}"/>
 	</inertial>
@@ -13,5 +13,5 @@
 		<origin xyz="0.0 0.0 0.0"  rpy="0.0 0.0 0.0"/>
 	  	<geometry>
-	 		<cylinder radius="${props['cylinder_radius']}" length="${props['cylinder_length']}"/>
+	 		<cylinder radius="${cylinder_radius}" length="${cylinder_length}"/>
 	  	</geometry>
   		<material name="dark_grey"/>
@@ -20,5 +20,5 @@
 		<origin xyz="0.0 0.0 0.0"  rpy="0.0 0.0 0.0"/>
 		<geometry>
-			<cylinder radius="${props['cylinder_radius']}" length="${props['cylinder_length']}"/>
+			<cylinder radius="${cylinder_radius}" length="${cylinder_length}"/>
 		</geometry>
 	</collision>
@@ -27,5 +27,5 @@
 	<inertial>
 		<origin xyz="0.0 0.0 0.0"/>
-		<mass value="${props_inertial['motorA_mass']}"/>
+		<mass value="${motorA_mass}"/>
 		<inertia ixx="${MotorA_xx}" ixy="${MotorA_xy}" ixz="${MotorA_xz}" iyy="${MotorA_yy}" iyz="${MotorA_yz}" izz="${MotorA_zz}"/>
 	</inertial>
@@ -33,5 +33,5 @@
 		<origin xyz="0.0 0.0 0.0"  rpy="0.0 0.0 0.0"/>
 	  	<geometry>
-	 		<cylinder radius="${props['cylinder_radius']}" length="${props['cylinder_length']}"/>
+	 		<cylinder radius="${cylinder_radius}" length="${cylinder_length}"/>
 	  	</geometry>
   		<material name="dark_grey"/>
@@ -40,5 +40,5 @@
 		<origin xyz="0.0 0.0 0.0"  rpy="0.0 0.0 0.0"/>
 		<geometry>
-			<cylinder radius="${props['cylinder_radius']}" length="${props['cylinder_length']}"/>
+			<cylinder radius="${cylinder_radius}" length="${cylinder_length}"/>
 		</geometry>
 	</collision>
@@ -47,5 +47,5 @@
 	<inertial>
 		<origin xyz="0.0 0.0 0.0"/>
-		<mass value="${props_inertial['motorA_mass']}"/>
+		<mass value="${motorA_mass}"/>
 		<inertia ixx="${MotorA_xx}" ixy="${MotorA_xy}" ixz="${MotorA_xz}" iyy="${MotorA_yy}" iyz="${MotorA_yz}" izz="${MotorA_zz}"/>
 	</inertial>
@@ -53,5 +53,5 @@
 		<origin xyz="0.0 0.0 0.0"  rpy="0.0 0.0 0.0"/>
 	  	<geometry>
-	 		<cylinder radius="${props['cylinder_radius']}" length="${props['cylinder_length']}"/>
+	 		<cylinder radius="${cylinder_radius}" length="${cylinder_length}"/>
 	  	</geometry>
   		<material name="dark_grey"/>
@@ -60,5 +60,5 @@
 		<origin xyz="0.0 0.0 0.0"  rpy="0.0 0.0 0.0"/>
 		<geometry>
-			<cylinder radius="${props['cylinder_radius']}" length="${props['cylinder_length']}"/>
+			<cylinder radius="${cylinder_radius}" length="${cylinder_length}"/>
 		</geometry>
 	</collision>
@@ -67,19 +67,19 @@
 	<inertial>
 		<origin xyz="0.0 0.0 0.0"/>
-		<mass value="${props_inertial['big_box_mass']}"/>
+		<mass value="${big_box_mass}"/>
 		<inertia ixx="${BigBox_xx}" ixy="${BigBox_xy}" ixz="${BigBox_xz}" iyy="${BigBox_xx}" iyz="${BigBox_yz}" izz="${BigBox_zz}"/>
 	</inertial>
 	<origin xyz="0.0 0.0 0.0" rpy="0.0 0.0 0.0"/>
 	<visual>
-		<origin xyz="${props['big_box_length'] / 2} 0.0 0.0"  rpy="0.0 0.0 0.0"/>
+		<origin xyz="${big_box_length / 2} 0.0 0.0"  rpy="0.0 0.0 0.0"/>
 	  	<geometry>
-	 		<box size="${props['big_box_length']} ${props['big_box_width']} ${props['big_box_height']}"/>
+	 		<box size="${big_box_length} ${big_box_width} ${big_box_height}"/>
 	  	</geometry>
   		<material name="dark_grey"/>
 	</visual>
 	<collision>
-		<origin xyz="${props['big_box_length'] / 2} 0.0 0.0"  rpy="0.0 0.0 0.0"/>
+		<origin xyz="${big_box_length / 2} 0.0 0.0"  rpy="0.0 0.0 0.0"/>
 		<geometry>
-			<box size="${props['big_box_length']} ${props['big_box_width']} ${props['big_box_height']}"/>
+			<box size="${big_box_length} ${big_box_width} ${big_box_height}"/>
 		</geometry>
 	</collision>
@@ -88,18 +88,18 @@
 	<inertial>
 		<origin xyz="0.0 0.0 0.0"/>
-		<mass value="${props_inertial['small_box_mass']}"/>
+		<mass value="${small_box_mass}"/>
 		<inertia ixx="${SmallBox_xx}" ixy="${SmallBox_xy}" ixz="${SmallBox_xz}" iyy="${SmallBox_xx}" iyz="${SmallBox_yz}" izz="${SmallBox_zz}"/>
 	</inertial>
 	<visual>
-		<origin xyz="${props['small_box_length'] / 2} 0.0 0.0"  rpy="0.0 0.0 0.0"/>
+		<origin xyz="${small_box_length / 2} 0.0 0.0"  rpy="0.0 0.0 0.0"/>
 	  	<geometry>
-	 		<box size="${props['small_box_length']} ${props['small_box_width']} ${props['small_box_height']}"/>
+	 		<box size="${small_box_length} ${small_box_width} ${small_box_height}"/>
 	  	</geometry>
   		<material name="dark_grey"/>
 	</visual>
 	<collision>
-		<origin xyz="${props['small_box_length'] / 2} 0.0 0.0"  rpy="0.0 0.0 0.0"/>
+		<origin xyz="${small_box_length / 2} 0.0 0.0"  rpy="0.0 0.0 0.0"/>
 		<geometry>
-	 		<box size="${props['small_box_length']} ${props['small_box_width']} ${props['small_box_height']}"/>
+	 		<box size="${small_box_length} ${small_box_width} ${small_box_height}"/>
 		</geometry>
 	</collision>
@@ -108,5 +108,5 @@
 	<inertial>
 		<origin xyz="0.0 0.0 0.0"/>
-		<mass value="${props_inertial['ball_mass']}"/>
+		<mass value="${ball_mass}"/>
 		<inertia ixx="${Ball_xx}" ixy="${Ball_xy}" ixz="${Ball_xz}" iyy="${Ball_yy}" iyz="${Ball_yz}" izz="${Ball_zz}"/>
 	</inertial>
@@ -114,5 +114,5 @@
 		<origin xyz="0.0 0.0 0.0" rpy="0.0 0.0 0.0"/>
 		<geometry>
-			<sphere radius="${props['ball_radius']}"/>
+			<sphere radius="${ball_radius}"/>
 		</geometry>
 	</visual>
@@ -120,5 +120,5 @@
 		<origin xyz="0.0 0.0 0.0" rpy="0.0 0.0 0.0"/>
 		<geometry>
-			<sphere radius="${props['ball_radius']}"/>
+			<sphere radius="${ball_radius}"/>
 		</geometry>
 	</collision>

File: cetc_sat_urdf/urdf/parts/inertial_properties.urdf.xacro (robot description, xacro)
@@ -1,44 +1,68 @@
-<!--<?xml version="1.0"?>-->
+<?xml version="1.0"?>
 <robot  xmlns:xacro="http://ros.org/wiki/xacro">
-<!-- Motor -->
-<xacro:property name="MotorA_xx" value="${1/12 * props_inertial['motorA_mass'] * (3 * props['cylinder_radius'] * props['cylinder_radius'] + props['cylinder_length'] * props['cylinder_length'])}"/>
-<xacro:property name="MotorA_xy" value="0.0"/>
-<xacro:property name="MotorA_xz" value="0.0"/>
-<xacro:property name="MotorA_yy" value="${1/12 * props_inertial['motorA_mass'] * (3 * props['cylinder_radius'] * props['cylinder_radius'] + props['cylinder_length'] * props['cylinder_length'])}"/>
-<xacro:property name="MotorA_yz" value="0.0"/>
-<xacro:property name="MotorA_zz" value="${1/2 * props_inertial['motorA_mass'] * props['cylinder_radius'] * props['cylinder_radius']}"/>
-<xacro:property name="MotorB_xx" value="${1/12 * props_inertial['motorB_mass'] * (3 * props['cylinder_radius'] * props['cylinder_radius'] + props['cylinder_length'] * props['cylinder_length'])}"/>
-<xacro:property name="MotorB_xy" value="0.0"/>
-<xacro:property name="MotorB_xz" value="0.0"/>
-<xacro:property name="MotorB_yy" value="${1/12 * props_inertial['motorB_mass'] * (3 * props['cylinder_radius'] * props['cylinder_radius'] + props['cylinder_length'] * props['cylinder_length'])}"/>
-<xacro:property name="MotorB_yz" value="0.0"/>
-<xacro:property name="MotorB_zz" value="${1/2 * props_inertial['motorB_mass'] * props['cylinder_radius'] * props['cylinder_radius']}"/>
-<!-- Pelvis -->
-<xacro:property name="Pelvis_xx" value="${1/12 * props_inertial['pelvis_mass'] * (props['pelvis_width'] * props['pelvis_width'] + props['pelvis_height'] * props['pelvis_height'])}"/>
-<xacro:property name="Pelvis_xy" value="0.0"/>
-<xacro:property name="Pelvis_xz" value="0.0"/>
-<xacro:property name="Pelvis_yy" value="${1/12 * props_inertial['pelvis_mass'] * (props['pelvis_length'] * props['pelvis_length'] + props['pelvis_height'] * props['pelvis_height'])}"/>
-<xacro:property name="Pelvis_yz" value="0.0"/>
-<xacro:property name="Pelvis_zz" value="${1/12 * props_inertial['pelvis_mass'] * (props['pelvis_width'] * props['pelvis_width'] + props['pelvis_length'] * props['pelvis_length'])}"/>
-<!-- Upper Leg -->
-<xacro:property name="BigBox_xx" value="${1/3 * props_inertial['big_box_mass'] * (props['big_box_width'] * props['big_box_width'] + props['big_box_height'] * props['big_box_height'])}"/>
-<xacro:property name="BigBox_xy" value="0.0"/>
-<xacro:property name="BigBox_xz" value="0.0"/>
-<xacro:property name="BigBox_yy" value="${1/3 * props_inertial['big_box_mass'] * (props['big_box_length'] * props['big_box_length'] + props['big_box_height'] * props['big_box_height'])}"/>
-<xacro:property name="BigBox_yz" value="0.0"/>
-<xacro:property name="BigBox_zz" value="${1/3 * props_inertial['big_box_mass'] * (props['big_box_width'] * props['big_box_width'] + props['big_box_length'] * props['big_box_length'])}"/>
-<!-- Lower Leg -->
-<xacro:property name="SmallBox_xx" value="${1/3 * props_inertial['small_box_mass'] * (props['small_box_width'] * props['small_box_width'] + props['small_box_height'] * props['small_box_height'])}"/>
-<xacro:property name="SmallBox_xy" value="0.0"/>
-<xacro:property name="SmallBox_xz" value="0.0"/>
-<xacro:property name="SmallBox_yy" value="${1/3 * props_inertial['small_box_mass'] * (props['small_box_length'] * props['small_box_length'] + props['small_box_height'] * props['small_box_height'])}"/>
-<xacro:property name="SmallBox_yz" value="0.0"/>
-<xacro:property name="SmallBox_zz" value="${1/3 * props_inertial['small_box_mass'] * (props['small_box_width'] * props['small_box_width'] + props['small_box_length'] * props['small_box_length'])}"/>
-<!-- Ball (hollow sphere) -->
-<xacro:property name="Ball_xx" value="${2/3 * props_inertial['ball_mass'] * props['ball_radius'] * props['ball_radius']}"/>
-<xacro:property name="Ball_xy" value="0.0"/>
-<xacro:property name="Ball_xz" value="0.0"/>
-<xacro:property name="Ball_yy" value="${2/3 * props_inertial['ball_mass'] * props['ball_radius'] * props['ball_radius']}"/>
-<xacro:property name="Ball_yz" value="0.0"/>
-<xacro:property name="Ball_zz" value="${2/3 * props_inertial['ball_mass'] * props['ball_radius'] * props['ball_radius']}"/>
+    <xacro:if value="$(arg bilevel_codes)">
+        <!-- no default, so that if bilevel_codes is true the user is forced to specify the paths-->
+        <xacro:arg name="inertial_props_path" default="$(find cetc_sat_urdf)/urdf/config/inertial_properties.yaml" />
+        <xacro:property name="id" value="$(arg sample_idx)" />
+        <xacro:property name="inertial_yaml_file" value="$(arg inertial_props_path)" />
+        <xacro:property name="inertial_props" value="${xacro.load_yaml(inertial_yaml_file)}"/>
+        <xacro:property name="pelvis_mass" value="${inertial_props['pelvis_mass'][id]}"/>
+        <xacro:property name="big_box_mass" value="${inertial_props['big_box_mass'][id]}"/>
+        <xacro:property name="small_box_mass" value="${inertial_props['small_box_mass'][id]}"/>
+        <xacro:property name="ball_mass" value="${inertial_props['ball_mass'][id]}"/>
+        <xacro:property name="motorA_mass" value="${inertial_props['motorA_mass'][id]}"/>
+        <xacro:property name="motorB_mass" value="${inertial_props['motorB_mass'][id]}"/>
+    </xacro:if>
+    <xacro:unless value="$(arg bilevel_codes)">
+        <xacro:property name="inertial_yaml_file" value="$(find cetc_sat_urdf)/urdf/config/inertial_properties.yaml" />
+        <xacro:property name="inertial_props" value="${xacro.load_yaml(inertial_yaml_file)}"/>
+        <xacro:property name="pelvis_mass" value="${inertial_props['pelvis_mass']}"/>
+        <xacro:property name="big_box_mass" value="${inertial_props['big_box_mass']}"/>
+        <xacro:property name="small_box_mass" value="${inertial_props['small_box_mass']}"/>
+        <xacro:property name="ball_mass" value="${inertial_props['ball_mass']}"/>
+        <xacro:property name="motorA_mass" value="${inertial_props['motorA_mass']}"/>
+        <xacro:property name="motorB_mass" value="${inertial_props['motorB_mass']}"/>
+    </xacro:unless>
+    <!-- Compound properties (i.e. based on the props parsed from the yaml) -->
+    <!-- Motor -->
+    <xacro:property name="MotorA_xx" value="${1/12 * motorA_mass * (3 * cylinder_radius * cylinder_radius + cylinder_length * cylinder_length)}"/>
+    <xacro:property name="MotorA_xy" value="0.0"/>
+    <xacro:property name="MotorA_xz" value="0.0"/>
+    <xacro:property name="MotorA_yy" value="${1/12 * motorA_mass * (3 * cylinder_radius * cylinder_radius + cylinder_length * cylinder_length)}"/>
+    <xacro:property name="MotorA_yz" value="0.0"/>
+    <xacro:property name="MotorA_zz" value="${1/2 * motorA_mass * cylinder_radius * cylinder_radius}"/>
+    <xacro:property name="MotorB_xx" value="${1/12 * motorB_mass * (3 * cylinder_radius * cylinder_radius + cylinder_length * cylinder_length)}"/>
+    <xacro:property name="MotorB_xy" value="0.0"/>
+    <xacro:property name="MotorB_xz" value="0.0"/>
+    <xacro:property name="MotorB_yy" value="${1/12 * motorB_mass * (3 * cylinder_radius * cylinder_radius + cylinder_length * cylinder_length)}"/>
+    <xacro:property name="MotorB_yz" value="0.0"/>
+    <xacro:property name="MotorB_zz" value="${1/2 * motorB_mass * cylinder_radius * cylinder_radius}"/>
+    <!-- Pelvis -->
+    <xacro:property name="Pelvis_xx" value="${1/12 * pelvis_mass * (pelvis_width * pelvis_width + pelvis_height * pelvis_height)}"/>
+    <xacro:property name="Pelvis_xy" value="0.0"/>
+    <xacro:property name="Pelvis_xz" value="0.0"/>
+    <xacro:property name="Pelvis_yy" value="${1/12 * pelvis_mass * (pelvis_length * pelvis_length + pelvis_height * pelvis_height)}"/>
+    <xacro:property name="Pelvis_yz" value="0.0"/>
+    <xacro:property name="Pelvis_zz" value="${1/12 * pelvis_mass * (pelvis_width * pelvis_width + pelvis_length * pelvis_length)}"/>
+    <!-- Upper Leg -->
+    <xacro:property name="BigBox_xx" value="${1/3 * big_box_mass * (big_box_width * big_box_width + big_box_height * big_box_height)}"/>
+    <xacro:property name="BigBox_xy" value="0.0"/>
+    <xacro:property name="BigBox_xz" value="0.0"/>
+    <xacro:property name="BigBox_yy" value="${1/3 * big_box_mass * (big_box_length * big_box_length + big_box_height * big_box_height)}"/>
+    <xacro:property name="BigBox_yz" value="0.0"/>
+    <xacro:property name="BigBox_zz" value="${1/3 * big_box_mass * (big_box_width * big_box_width + big_box_length * big_box_length)}"/>
+    <!-- Lower Leg -->
+    <xacro:property name="SmallBox_xx" value="${1/3 * small_box_mass * (small_box_width * small_box_width + small_box_height * small_box_height)}"/>
+    <xacro:property name="SmallBox_xy" value="0.0"/>
+    <xacro:property name="SmallBox_xz" value="0.0"/>
+    <xacro:property name="SmallBox_yy" value="${1/3 * small_box_mass * (small_box_length * small_box_length + small_box_height * small_box_height)}"/>
+    <xacro:property name="SmallBox_yz" value="0.0"/>
+    <xacro:property name="SmallBox_zz" value="${1/3 * small_box_mass * (small_box_width * small_box_width + small_box_length * small_box_length)}"/>
+    <!-- Ball (hollow sphere) -->
+    <xacro:property name="Ball_xx" value="${2/3 * ball_mass * ball_radius * ball_radius}"/>
+    <xacro:property name="Ball_xy" value="0.0"/>
+    <xacro:property name="Ball_xz" value="0.0"/>
+    <xacro:property name="Ball_yy" value="${2/3 * ball_mass * ball_radius * ball_radius}"/>
+    <xacro:property name="Ball_yz" value="0.0"/>
+    <xacro:property name="Ball_zz" value="${2/3 * ball_mass * ball_radius * ball_radius}"/>
 </robot>
