Commit message: added package.xml to urdf and srdf folder

File: cetc_sat_srdf/srdf/cetc_sat.srdf.xacro (robot description, xacro)
@@ -6,5 +6,5 @@
 <robot xmlns:xacro="http://ros.org/wiki/xacro" name="cetc_sat">
     <!-- ************ MODEL CONFIGURATION ************ -->
-    <xacro:arg name="config" default="$(find CETC_SAT_description)/cetc_sat_urdf/urdf/config/cetc_sat.urdf.xacro"/>
+    <xacro:arg name="config" default="$(find cetc_sat_urdf)/urdf/config/cetc_sat.urdf.xacro"/>
     <xacro:include filename="$(arg config)"/>
     <group name="base">

File: cetc_sat_urdf/urdf/cetc_sat.urdf.xacro (robot description, xacro)
@@ -1,9 +1,9 @@
 <?xml version="1.0"?>
 <robot xmlns:xacro="http://ros.org/wiki/xacro" name="cetc_sat">
-<xacro:arg name="config" default="$(find CETC_SAT_description)/cetc_sat_urdf/urdf/config/cetc_sat.urdf.xacro"/>
+<xacro:arg name="config" default="$(find cetc_sat_urdf)/urdf/config/cetc_sat.urdf.xacro"/>
 <!-- ************ MODEL CONFIGURATION ************ -->
 <xacro:include filename="$(arg config)"/>
 <!-- ************ CETC-SAT plain model ************ -->
-<xacro:include filename="$(find CETC_SAT_description)/cetc_sat_urdf/urdf/cetc_sat_base.urdf.xacro"/>
+<xacro:include filename="$(find cetc_sat_urdf)/urdf/cetc_sat_base.urdf.xacro"/>
 <!-- ************ Control frames ************ -->
 <!--xacro:include filename="$(find pholus_urdf)/urdf/control_frames.urdf.xacro"/-->

File: cetc_sat_urdf/urdf/cetc_sat_base.urdf.xacro (robot description, xacro)
@@ -5,8 +5,8 @@
   Author: Luca Rossini
 -->
-<xacro:include filename="$(find CETC_SAT_description)/cetc_sat_urdf/urdf/utils.urdf.xacro" />
-<xacro:include filename="$(find CETC_SAT_description)/cetc_sat_urdf/urdf/parts/kinematics_properties.urdf.xacro" />
+<xacro:include filename="$(find cetc_sat_urdf)/urdf/utils.urdf.xacro" />
+<xacro:include filename="$(find cetc_sat_urdf)/urdf/parts/kinematics_properties.urdf.xacro" />
 <!--xacro:include filename="$(find cetc_sat_urdf)/urdf/parts/inertial_properties.urdf.xacro" /-->
-<xacro:include filename="$(find CETC_SAT_description)/cetc_sat_urdf/urdf/parts/limits.urdf.xacro" />
+<xacro:include filename="$(find cetc_sat_urdf)/urdf/parts/limits.urdf.xacro" />
 <link name="base_link"/>
 <link name="pelvis">
@@ -30,8 +30,8 @@
 </joint>
 <xacro:if value="${ADD_UPPER_BODY}">
-    <xacro:include filename="$(find CETC_SAT_description)/cetc_sat_urdf/urdf/parts/arms.urdf.xacro" />
+    <xacro:include filename="$(find cetc_sat_urdf)/urdf/parts/arms.urdf.xacro" />
 </xacro:if>
 <xacro:if value="${ADD_LEGS}">
-	<xacro:include filename="$(find CETC_SAT_description)/cetc_sat_urdf/urdf/parts/legs.urdf.xacro" />
+	<xacro:include filename="$(find cetc_sat_urdf)/urdf/parts/legs.urdf.xacro" />
 </xacro:if>
 </robot>

File: cetc_sat_urdf/urdf/parts/arms.urdf.xacro (robot description, xacro)
@@ -1,5 +1,5 @@
 <?xml version="1.0"?>
 <robot xmlns:xacro="http://ros.org/wiki/xacro">
-<xacro:include filename="$(find CETC_SAT_description)/cetc_sat_urdf/urdf/parts/cetc_sat_arm.urdf.xacro" />
+<xacro:include filename="$(find cetc_sat_urdf)/urdf/parts/cetc_sat_arm.urdf.xacro" />
 <!-- arms -->
 <xacro:cetc_sat_arm arm_num="1"  rot="1"  parent="pelvis">

File: cetc_sat_urdf/urdf/parts/cetc_sat_arm.urdf.xacro (robot description, xacro)
@@ -41,5 +41,5 @@
 		<origin xyz="${EndEffector_Ox / 2} 0.0 0.0"  rpy="0.0 0.0 0.0"/>
 		<geometry>
-			<box size="${big_box_length} ${big_box_width} ${big_box_height}"/>
+			<box size="${small_box_length} ${small_box_width} ${small_box_height}"/>
 		</geometry>
 		<material name="dark_grey"/>
@@ -48,5 +48,5 @@
 		<origin xyz="${EndEffector_Ox / 2} 0.0 0.0"  rpy="0.0 0.0 0.0"/>
 		<geometry>
-			<box size="${big_box_length} ${big_box_width} ${big_box_height}"/>
+			<box size="${small_box_length} ${small_box_width} ${small_box_height}"/>
 		</geometry>
 	</collision>

File: cetc_sat_urdf/urdf/parts/legs.urdf.xacro (robot description, xacro)
@@ -1,5 +1,5 @@
 <?xml version="1.0"?>
 <robot xmlns:xacro="http://ros.org/wiki/xacro">
-<xacro:include filename="$(find CETC_SAT_description)/cetc_sat_urdf/urdf/parts/cetc_sat_leg.urdf.xacro" />
+<xacro:include filename="$(find cetc_sat_urdf)/urdf/parts/cetc_sat_leg.urdf.xacro" />
 <xacro:cetc_sat_leg leg_num="1" origin_x="1" origin_y="-1" mirror="-1">
 </xacro:cetc_sat_leg>

Commit message: added inertial parameters and motors as cylinders

File: cetc_sat_srdf/srdf/cetc_sat.srdf.xacro (robot description, xacro)
@@ -60,10 +60,10 @@
 		    <joint name="hip_pitch_4" value="0.7"/>
 		    <joint name="knee_pitch_4" value="-1.4"/>
-		    <joint name="j_shoulder_yaw_1" value="0.0"/>
-		    <joint name="j_pitch_1_1" value="0.7"/>
-		    <joint name="j_pitch_2_1" value="1.4"/>
-		    <joint name="j_shoulder_yaw_2" value="0.0"/>
-		    <joint name="j_pitch_1_2" value="0.7"/>
-		    <joint name="j_pitch_2_2" value="1.4"/>
+		    <joint name="shoulder_yaw_1" value="0.0"/>
+		    <joint name="shoulder_pitch_1" value="0.7"/>
+		    <joint name="elbow_pitch_1" value="1.4"/>
+		    <joint name="shoulder_yaw_2" value="0.0"/>
+		    <joint name="shoulder_pitch_2" value="0.7"/>
+		    <joint name="elbow_pitch_2" value="1.4"/>
 		</xacro:if>
     </group_state>

File: cetc_sat_urdf/urdf/cetc_sat_base.urdf.xacro (robot description, xacro)
@@ -7,10 +7,17 @@
 <xacro:include filename="$(find cetc_sat_urdf)/urdf/utils.urdf.xacro" />
 <xacro:include filename="$(find cetc_sat_urdf)/urdf/parts/kinematics_properties.urdf.xacro" />
-<!--xacro:include filename="$(find cetc_sat_urdf)/urdf/parts/inertial_properties.urdf.xacro" /-->
+<xacro:include filename="$(find cetc_sat_urdf)/urdf/parts/inertial_properties.urdf.xacro" />
 <xacro:include filename="$(find cetc_sat_urdf)/urdf/parts/limits.urdf.xacro" />
 <xacro:property name="yaml_file" value="$(find cetc_sat_urdf)/urdf/config/kinematics_properties.yaml" />
 <xacro:property name="props" value="${load_yaml(yaml_file)}"/>
+<xacro:property name="yaml_file_inertial" value="$(find cetc_sat_urdf)/urdf/config/inertial_properties.yaml" />
+<xacro:property name="props_inertial" value="${load_yaml(yaml_file_inertial)}"/>
 <link name="base_link"/>
 <link name="pelvis">
+	<inertial>
+		<origin xyz="0.0 0.0 0.0"/>
+		<mass value="${props_inertial['pelvis_mass']}"/>
+		<inertia ixx="${Pelvis_xx}" ixy="${Pelvis_xy}" ixz="${Pelvis_xz}" iyy="${Pelvis_yy}" iyz="${Pelvis_yz}" izz="${Pelvis_zz}"/>
+	</inertial>
 	<visual>
 		<origin xyz="0.0 0 0.0"  rpy="0.0 0.0 0.0"/>

File: cetc_sat_urdf/urdf/parts/cetc_sat_arm.urdf.xacro (robot description, xacro)
@@ -5,5 +5,10 @@
 <!-- LINKS -->
 <!-- shoulder yaw -->
-<link name="shoulder_${arm_num}">
+<link name="shoulder_yaw_motor_${arm_num}">
+	<inertial>
+		<origin xyz="0.0 0.0 0.0"/>
+		<mass value="${props_inertial['motorA_mass']}"/>
+		<inertia ixx="${MotorA_xx}" ixy="${MotorA_xy}" ixz="${MotorA_xz}" iyy="${MotorA_yy}" iyz="${MotorA_yz}" izz="${MotorA_zz}"/>
+	</inertial>
 	<visual>
 		<origin xyz="0.0 0.0 0.0"  rpy="0.0 0.0 0.0"/>
@@ -20,8 +25,32 @@
 	</collision>
 </link>
-<!-- base arm-->
-<link name="arm${arm_num}_1">
+<link name="shoulder_pitch_motor_${arm_num}">
+	<inertial>
+		<origin xyz="0.0 0.0 0.0"/>
+		<mass value="${props_inertial['motorA_mass']}"/>
+		<inertia ixx="${MotorA_xx}" ixy="${MotorA_xy}" ixz="${MotorA_xz}" iyy="${MotorA_yy}" iyz="${MotorA_yz}" izz="${MotorA_zz}"/>
+	</inertial>
 	<visual>
-		<origin xyz="${props['Pitch_2_Ox'] / 2} 0.0 0.0"  rpy="0.0 0.0 0.0"/>
+		<origin xyz="0.0 0.0 0.0"  rpy="0.0 0.0 0.0"/>
+	  	<geometry>
+	 		<cylinder radius="${props['cylinder_radius']}" length="${props['cylinder_length']}"/>
+	  	</geometry>
+  		<material name="dark_grey"/>
+	</visual>
+	<collision>
+		<origin xyz="0.0 0.0 0.0"  rpy="0.0 0.0 0.0"/>
+		<geometry>
+			<cylinder radius="${props['cylinder_radius']}" length="${props['cylinder_length']}"/>
+		</geometry>
+	</collision>
+</link>
+<link name="lower_arm_${arm_num}">
+	<inertial>
+		<origin xyz="0.0 0.0 0.0"/>
+		<mass value="${props_inertial['big_box_mass']}"/>
+		<inertia ixx="${BigBox_xx}" ixy="${BigBox_xy}" ixz="${BigBox_xz}" iyy="${BigBox_xx}" iyz="${BigBox_yz}" izz="${BigBox_zz}"/>
+	</inertial>
+	<visual>
+		<origin xyz="${props['big_box_length'] / 2} 0.0 0.0"  rpy="0.0 0.0 0.0"/>
 		<geometry>
 			<box size="${props['big_box_length']} ${props['big_box_width']} ${props['big_box_height']}"/>
@@ -29,5 +58,5 @@
 	</visual>
 	<collision>
-		<origin xyz="${props['Pitch_2_Ox'] / 2} 0.0 0.0"  rpy="0.0 0.0 0.0"/>
+		<origin xyz="${props['big_box_length'] / 2} 0.0 0.0"  rpy="0.0 0.0 0.0"/>
 		<geometry>
 			<box size="${props['big_box_length']} ${props['big_box_width']} ${props['big_box_height']}"/>
@@ -35,9 +64,32 @@
 	</collision>
 </link>
-<!-- shoulder roll-pitch-->
-<!-- shoulder-elbow -->
-<link name="arm${arm_num}_2">
+<link name="elbow_pitch_motor_${arm_num}">
+	<inertial>
+		<origin xyz="0.0 0.0 0.0"/>
+		<mass value="${props_inertial['motorA_mass']}"/>
+		<inertia ixx="${MotorA_xx}" ixy="${MotorA_xy}" ixz="${MotorA_xz}" iyy="${MotorA_yy}" iyz="${MotorA_yz}" izz="${MotorA_zz}"/>
+	</inertial>
 	<visual>
-		<origin xyz="${props['EndEffector_Ox'] / 2} 0.0 0.0"  rpy="0.0 0.0 0.0"/>
+		<origin xyz="0.0 0.0 0.0"  rpy="0.0 0.0 0.0"/>
+	  	<geometry>
+	 		<cylinder radius="${props['cylinder_radius']}" length="${props['cylinder_length']}"/>
+	  	</geometry>
+  		<material name="dark_grey"/>
+	</visual>
+	<collision>
+		<origin xyz="0.0 0.0 0.0"  rpy="0.0 0.0 0.0"/>
+		<geometry>
+			<cylinder radius="${props['cylinder_radius']}" length="${props['cylinder_length']}"/>
+		</geometry>
+	</collision>
+</link>
+<link name="upper_arm_${arm_num}">
+	<inertial>
+		<origin xyz="0.0 0.0 0.0"/>
+		<mass value="${props_inertial['small_box_mass']}"/>
+		<inertia ixx="${SmallBox_xx}" ixy="${SmallBox_xy}" ixz="${SmallBox_xz}" iyy="${SmallBox_xx}" iyz="${SmallBox_yz}" izz="${SmallBox_zz}"/>
+	</inertial>
+	<visual>
+		<origin xyz="${props['small_box_length'] / 2} 0.0 0.0"  rpy="0.0 0.0 0.0"/>
 		<geometry>
 			<box size="${props['small_box_length']} ${props['small_box_width']} ${props['small_box_height']}"/>
@@ -46,5 +98,5 @@
 	</visual>
 	<collision>
-		<origin xyz="${props['EndEffector_Ox'] / 2} 0.0 0.0"  rpy="0.0 0.0 0.0"/>
+		<origin xyz="${props['small_box_length'] / 2} 0.0 0.0"  rpy="0.0 0.0 0.0"/>
 		<geometry>
 			<box size="${props['small_box_length']} ${props['small_box_width']} ${props['small_box_height']}"/>
@@ -54,4 +106,9 @@
 <!-- /shoulder-elbow -->
 <link name="ball_arm_${arm_num}">
+    <inertial>
+		<origin xyz="0.0 0.0 0.0"/>
+		<mass value="${props_inertial['ball_mass']}"/>
+		<inertia ixx="${Ball_xx}" ixy="${Ball_xy}" ixz="${Ball_xz}" iyy="${Ball_yy}" iyz="${Ball_yz}" izz="${Ball_zz}"/>
+	</inertial>
 	<visual>
 		<origin xyz="0.0 0.0 0.0" rpy="0.0 0.0 0.0"/>
@@ -70,30 +127,40 @@
 <!-- JOINTS -->
 <!-- shoulder yaw -->
-<joint name="j_shoulder_yaw_${arm_num}" type="revolute">
+<joint name="shoulder_yaw_${arm_num}" type="revolute">
 	<parent link="${parent}"/>
-	<child link="shoulder_${arm_num}"/>
-	<origin xyz="${props['Shoulder_Ox'] / 2 -0.1} ${rot*props['Shoulder_Oy'] / 2 - 0.05} ${props['Shoulder_Oz'] / 2}" rpy="${props['Shoulder_roll']} ${props['Shoulder_pitch']} ${props['Shoulder_yaw']}"/>
+	<child link="shoulder_yaw_motor_${arm_num}"/>
+	<origin xyz="${props['ShoulderYaw_Ox'] / 2 -0.1} ${rot*props['ShoulderYaw_Oy'] / 2 - rot*0.05} ${props['ShoulderYaw_Oz'] / 2}" rpy="${props['ShoulderYaw_roll']} ${props['ShoulderYaw_pitch']} ${props['ShoulderYaw_yaw']}"/>
 	<axis xyz="0 0 1"/>
 	<limit lower="${j_shoulder_yaw_lower[arm_num-1]}" upper="${j_shoulder_yaw_upper[arm_num-1]}" effort="${j_shoulder_torque[arm_num-1]}" velocity="${j_shoulder_velocity[arm_num-1]}"/>
 </joint>
+<joint name="shoulder_pitch_stator_${arm_num}" type="fixed">
+	<parent link="shoulder_yaw_motor_${arm_num}"/>
+	<child link="shoulder_pitch_motor_${arm_num}"/>
+	<origin xyz="${props['ShoulderPitch_Ox']} ${props['ShoulderPitch_Oy']} ${props['ShoulderPitch_Oz'] / 2}" rpy="${-props['ShoulderPitch_roll']} ${props['ShoulderPitch_pitch']} ${props['ShoulderPitch_yaw']}"/>
+</joint>
 <!-- arm pitch 1 -->
-<joint name="j_pitch_1_${arm_num}" type="revolute">
-	<parent link="shoulder_${arm_num}"/>
-	<child link="arm${arm_num}_1"/>
-	<origin xyz="${props['Pitch_1_Ox']} ${props['Pitch_1_Oy']} ${props['Pitch_1_Oz'] / 2}" rpy="${props['Pitch_1_roll']} ${-props['Pitch_1_pitch']} ${props['Pitch_1_yaw']}"/>
-	<axis xyz="0 1 0"/>
+<joint name="shoulder_pitch_${arm_num}" type="revolute">
+	<parent link="shoulder_pitch_motor_${arm_num}"/>
+	<child link="lower_arm_${arm_num}"/>
+	<origin xyz="${props['LowerArm_Ox']} ${props['LowerArm_Oy']} ${props['LowerArm_Oz'] / 2}" rpy="${props['LowerArm_roll']} ${props['LowerArm_pitch']} ${-props['LowerArm_yaw']}"/>
+	<axis xyz="0 0 1"/>
 	<limit lower="${j_pitch_1_lower[arm_num-1]}" upper="${j_pitch_1_upper[arm_num-1]}" effort="${j_pitch_1_torque[arm_num-1]}" velocity="${j_pitch_1_velocity[arm_num-1]}"/>
 </joint>
+<joint name="elbow_pitch_stator_${arm_num}" type="fixed">
+	<parent link="lower_arm_${arm_num}"/>
+	<child link="elbow_pitch_motor_${arm_num}"/>
+	<origin xyz="${props['ElbowPitch_Ox']} ${props['ElbowPitch_Oy']} ${props['ElbowPitch_Oz']}" rpy="${props['ElbowPitch_roll']} ${props['ElbowPitch_pitch']} ${props['ElbowPitch_yaw']}"/>
+</joint>
 <!-- arm pitch 2 -->
-<joint name="j_pitch_2_${arm_num}" type="revolute">
-	<parent link="arm${arm_num}_1"/>
-	<child link="arm${arm_num}_2"/>
-	<origin xyz="${props['Pitch_2_Ox']} ${props['Pitch_2_Oy']} ${props['Pitch_2_Oz']}" rpy="${props['Pitch_2_roll']} ${props['Pitch_2_pitch']} ${props['Pitch_2_yaw']}"/>
-	<axis xyz="0 1 0"/>
+<joint name="elbow_pitch_${arm_num}" type="revolute">
+	<parent link="elbow_pitch_motor_${arm_num}"/>
+	<child link="upper_arm_${arm_num}"/>
+	<origin xyz="${props['UpperArm_Ox']} ${props['UpperArm_Oy']} ${props['UpperArm_Oz']}" rpy="${props['UpperArm_roll']} ${props['UpperArm_pitch']} ${props['UpperArm_yaw']}"/>
+	<axis xyz="0 0 1"/>
 	<limit lower="${j_pitch_2_lower[arm_num-1]}" upper="${j_pitch_2_upper[arm_num-1]}" effort="${j_pitch_2_torque[arm_num-1]}" velocity="${j_pitch_2_velocity[arm_num-1]}"/>
 </joint>
 <!-- end effector  -->
-<joint name="j_hand_${arm_num}" type="fixed">
-	<parent link="arm${arm_num}_2"/>
+<joint name="hand_joint_${arm_num}" type="fixed">
+	<parent link="upper_arm_${arm_num}"/>
 	<child link="ball_arm_${arm_num}"/>
 	<origin xyz="${props['EndEffector_Ox']} ${props['EndEffector_Oy']} ${props['EndEffector_Oz']}" rpy="${props['EndEffector_roll']} ${props['EndEffector_pitch']} ${props['EndEffector_yaw']}"/>

File: cetc_sat_urdf/urdf/parts/cetc_sat_leg.urdf.xacro (robot description, xacro)
@@ -4,6 +4,30 @@
 <xacro:macro name="cetc_sat_leg" params="leg_num origin_x origin_y mirror">
 <!-- links -->
-<link name="hip_${leg_num}">
-	<origin xyz="0.0 0.0 0.0" rpy="0.0 0.0 0.0"/>
+<link name="hip_roll_motor_${leg_num}">
+	<inertial>
+		<origin xyz="0.0 0.0 0.0"/>
+		<mass value="${props_inertial['motorA_mass']}"/>
+		<inertia ixx="${MotorA_xx}" ixy="${MotorA_xy}" ixz="${MotorA_xz}" iyy="${MotorA_yy}" iyz="${MotorA_yz}" izz="${MotorA_zz}"/>
+	</inertial>
+	<visual>
+		<origin xyz="0.0 0.0 0.0"  rpy="0.0 0.0 0.0"/>
+	  	<geometry>
+	 		<cylinder radius="${props['cylinder_radius']}" length="${props['cylinder_length']}"/>
+	  	</geometry>
+  		<material name="dark_grey"/>
+	</visual>
+	<collision>
+		<origin xyz="0.0 0.0 0.0"  rpy="0.0 0.0 0.0"/>
+		<geometry>
+			<cylinder radius="${props['cylinder_radius']}" length="${props['cylinder_length']}"/>
+		</geometry>
+	</collision>
+</link>
+<link name="hip_pitch_motor_${leg_num}">
+	<inertial>
+		<origin xyz="0.0 0.0 0.0"/>
+		<mass value="${props_inertial['motorA_mass']}"/>
+		<inertia ixx="${MotorA_xx}" ixy="${MotorA_xy}" ixz="${MotorA_xz}" iyy="${MotorA_yy}" iyz="${MotorA_yz}" izz="${MotorA_zz}"/>
+	</inertial>
 	<visual>
 		<origin xyz="0.0 0.0 0.0"  rpy="0.0 0.0 0.0"/>
@@ -21,7 +45,12 @@
 </link>
 <link name="upper_leg_${leg_num}">
+	<inertial>
+		<origin xyz="0.0 0.0 0.0"/>
+		<mass value="${props_inertial['big_box_mass']}"/>
+		<inertia ixx="${BigBox_xx}" ixy="${BigBox_xy}" ixz="${BigBox_xz}" iyy="${BigBox_xx}" iyz="${BigBox_yz}" izz="${BigBox_zz}"/>
+	</inertial>
 	<origin xyz="0.0 0.0 0.0" rpy="0.0 0.0 0.0"/>
 	<visual>
-		<origin xyz="${props['Leg_3_Ox'] / 2} 0.0 0.0"  rpy="0.0 0.0 0.0"/>
+		<origin xyz="${props['KneePitch_Ox'] / 2} 0.0 0.0"  rpy="0.0 0.0 0.0"/>
 	  	<geometry>
 	 		<box size="${props['big_box_length']} ${props['big_box_width']} ${props['big_box_height']}"/>
@@ -30,5 +59,5 @@
 	</visual>
 	<collision>
-		<origin xyz="${props['Leg_3_Ox'] / 2} 0.0 0.0"  rpy="0.0 0.0 0.0"/>
+		<origin xyz="${props['KneePitch_Ox'] / 2} 0.0 0.0"  rpy="0.0 0.0 0.0"/>
 		<geometry>
 			<box size="${props['big_box_length']} ${props['big_box_width']} ${props['big_box_height']}"/>
@@ -36,6 +65,31 @@
 	</collision>
 </link>
+<link name="knee_pitch_motor_${leg_num}">
+	<inertial>
+		<origin xyz="0.0 0.0 0.0"/>
+		<mass value="${props_inertial['motorA_mass']}"/>
+		<inertia ixx="${MotorA_xx}" ixy="${MotorA_xy}" ixz="${MotorA_xz}" iyy="${MotorA_yy}" iyz="${MotorA_yz}" izz="${MotorA_zz}"/>
+	</inertial>
+	<visual>
+		<origin xyz="0.0 0.0 0.0"  rpy="0.0 0.0 0.0"/>
+	  	<geometry>
+	 		<cylinder radius="${props['cylinder_radius']}" length="${props['cylinder_length']}"/>
+	  	</geometry>
+  		<material name="dark_grey"/>
+	</visual>
+	<collision>
+		<origin xyz="0.0 0.0 0.0"  rpy="0.0 0.0 0.0"/>
+		<geometry>
+			<cylinder radius="${props['cylinder_radius']}" length="${props['cylinder_length']}"/>
+		</geometry>
+	</collision>
+</link>
 <link name="lower_leg_${leg_num}">
-<visual>
+	<inertial>
+		<origin xyz="0.0 0.0 0.0"/>
+		<mass value="${props_inertial['small_box_mass']}"/>
+		<inertia ixx="${SmallBox_xx}" ixy="${SmallBox_xy}" ixz="${SmallBox_xz}" iyy="${SmallBox_xx}" iyz="${SmallBox_yz}" izz="${SmallBox_zz}"/>
+	</inertial>
+	<visual>
 		<origin xyz="${props['Ankle_Ox'] / 2} 0.0 0.0"  rpy="0.0 0.0 0.0"/>
 	  	<geometry>
@@ -52,4 +106,9 @@
 </link>
 <link name="ball_${leg_num}">
+	<inertial>
+		<origin xyz="0.0 0.0 0.0"/>
+		<mass value="${props_inertial['ball_mass']}"/>
+		<inertia ixx="${Ball_xx}" ixy="${Ball_xy}" ixz="${Ball_xz}" iyy="${Ball_yy}" iyz="${Ball_yz}" izz="${Ball_zz}"/>
+	</inertial>
 	<visual>
 		<origin xyz="0.0 0.0 0.0" rpy="0.0 0.0 0.0"/>
@@ -68,21 +127,31 @@
 <joint name="hip_roll_${leg_num}" type="revolute">
 	<parent link="pelvis"/>
-	<child link="hip_${leg_num}"/>
-	<origin xyz="${origin_x*props['Leg_1_Ox'] / 2} ${origin_y*(-props['Leg_1_Oy'] / 2)} ${props['Leg_1_Oz']}" rpy="${props['Leg_1_roll']} ${props['Leg_1_pitch']} ${props['Leg_1_yaw']}"/>
+	<child link="hip_roll_motor_${leg_num}"/>
+	<origin xyz="${origin_x*props['HipRoll_Ox'] / 2} ${origin_y*(-props['HipRoll_Oy'] / 2)} ${props['HipRoll_Oz']}" rpy="${props['HipRoll_roll']} ${props['HipRoll_pitch']} ${props['HipRoll_yaw']}"/>
 	<axis xyz="0 0 1"/>
-   <limit lower="${hip_roll_lower[leg_num-1]}" upper="${hip_roll_upper[leg_num-1]}" effort="${motor_A_effort}" velocity="${motor_A_velocity}"/> <!-- 200 Nm, 1 rad/s-->
+    <limit lower="${hip_roll_lower[leg_num-1]}" upper="${hip_roll_upper[leg_num-1]}" effort="${motor_A_effort}" velocity="${motor_A_velocity}"/> <!-- 200 Nm, 1 rad/s-->
+</joint>
+<joint name="hip_pitch_stator_${leg_num}" type="fixed">
+	<parent link="hip_roll_motor_${leg_num}"/>
+	<child link="hip_pitch_motor_${leg_num}"/>
+	<origin xyz="${props['HipPitch_Ox']} ${mirror * (-props['HipPitch_Oy'])} ${props['HipPitch_Oz']}" rpy="${-props['HipPitch_roll']} ${props['HipPitch_pitch']} ${props['HipPitch_yaw']}"/>
 </joint>
 <joint name="hip_pitch_${leg_num}" type="revolute">
-	<parent link="hip_${leg_num}"/>
+	<parent link="hip_pitch_motor_${leg_num}"/>
 	<child link="upper_leg_${leg_num}"/>
-	<origin xyz="${props['Leg_2_Ox']} ${mirror*(-props['Leg_2_Oy']/2)} ${props['Leg_2_Oz']}" rpy="${props['Leg_2_roll']} ${props['Leg_2_pitch']} ${props['Leg_2_yaw']}"/>
-	<axis xyz="0 1 0"/>
+	<origin xyz="${props['UpperLeg_Ox']} ${mirror*(-props['UpperLeg_Oy']/2)} ${props['UpperLeg_Oz']}" rpy="${props['UpperLeg_roll']} ${props['UpperLeg_pitch']} ${props['UpperLeg_yaw']}"/>
+	<axis xyz="0 0 1"/>
    <limit lower="${hip_pitch_lower[leg_num-1]}" upper="${hip_pitch_upper[leg_num-1]}" effort="${motor_A_effort}" velocity="${motor_A_velocity}"/> <!-- 200 Nm, 1 rad/s-->
 </joint>
+<joint name="knee_pitch_stator_${leg_num}" type="fixed">
+	<parent link="upper_leg_${leg_num}"/>
+	<child link="knee_pitch_motor_${leg_num}"/>
+	<origin xyz="${props['KneePitch_Ox']} ${props['KneePitch_Oy']} ${props['KneePitch_Oz']}" rpy="${props['KneePitch_roll']} ${props['KneePitch_pitch']} ${props['KneePitch_yaw']}"/>
+</joint>
 <joint name="knee_pitch_${leg_num}" type="revolute">
-	<parent link="upper_leg_${leg_num}"/>
+	<parent link="knee_pitch_motor_${leg_num}"/>
 	<child link="lower_leg_${leg_num}"/>
-	<origin xyz="${props['Leg_3_Ox']} ${props['Leg_3_Oy']} ${props['Leg_3_Oz']}" rpy="${props['Leg_3_roll']} ${props['Leg_3_pitch']} ${props['Leg_3_yaw']}"/>
-	<axis xyz="0 1 0"/>
+	<origin xyz="${props['LowerLeg_Ox']} ${props['LowerLeg_Oy']} ${props['LowerLeg_Oz']}" rpy="${props['LowerLeg_roll']} ${props['LowerLeg_pitch']} ${props['LowerLeg_yaw']}"/>
+	<axis xyz="0 0 1"/>
    <limit lower="${knee_pitch_lower[leg_num-1]}" upper="${knee_pitch_upper[leg_num-1]}" effort="${motor_A_effort}" velocity="${motor_A_velocity}"/> <!-- 200 Nm, 1 rad/s-->
 </joint>
