Commit message: Ad urdf and srdf for xbot

File: cetc_sat_srdf/srdf/cetc_sat.srdf.xacro (robot description, xacro)
@@ -41,30 +41,44 @@
         </xacro:if>
         <xacro:if value="${ADD_UPPER_BODY}">
-        	<group name="left_arm"/>
-        	<group name="right_arm"/>
+            <group name="left_arm"/>
+            <group name="right_arm"/>
         </xacro:if>
     </group>
     <!-- Homing posture -->
     <group_state name="home" group="chains">
-    	<xacro:if value="${ADD_LEGS}">
-		    <joint name="hip_roll_1" value="0.0"/>
-		    <joint name="hip_pitch_1" value="0.7"/>
-		    <joint name="knee_pitch_1" value="-1.4"/>
-		    <joint name="hip_roll_2" value="0.0"/>
-		    <joint name="hip_pitch_2" value="0.7"/>
-		    <joint name="knee_pitch_2" value="-1.4"/>
-		    <joint name="hip_roll_3" value="0.0"/>
-		    <joint name="hip_pitch_3" value="0.7"/>
-		    <joint name="knee_pitch_3" value="-1.4"/>
-		    <joint name="hip_roll_4" value="0.0"/>
-		    <joint name="hip_pitch_4" value="0.7"/>
-		    <joint name="knee_pitch_4" value="-1.4"/>
-		    <joint name="shoulder_yaw_1" value="0.0"/>
-		    <joint name="shoulder_pitch_1" value="0.7"/>
-		    <joint name="elbow_pitch_1" value="1.4"/>
-		    <joint name="shoulder_yaw_2" value="0.0"/>
-		    <joint name="shoulder_pitch_2" value="0.7"/>
-		    <joint name="elbow_pitch_2" value="1.4"/>
-		</xacro:if>
+        <xacro:if value="${ADD_LEGS}">
+            <joint name="hip_roll_1" value="0.0"/>
+            <joint name="hip_pitch_1" value="0.7"/>
+            <joint name="knee_pitch_1" value="-1.4"/>
+            <joint name="hip_roll_2" value="0.0"/>
+            <joint name="hip_pitch_2" value="0.7"/>
+            <joint name="knee_pitch_2" value="-1.4"/>
+            <joint name="hip_roll_3" value="0.0"/>
+            <joint name="hip_pitch_3" value="0.7"/>
+            <joint name="knee_pitch_3" value="-1.4"/>
+            <joint name="hip_roll_4" value="0.0"/>
+            <joint name="hip_pitch_4" value="0.7"/>
+            <joint name="knee_pitch_4" value="-1.4"/>
+            <joint name="shoulder_yaw_1" value="0.0"/>
+            <joint name="shoulder_pitch_1" value="0.7"/>
+            <joint name="elbow_pitch_1" value="1.4"/>
+            <joint name="shoulder_yaw_2" value="0.0"/>
+            <joint name="shoulder_pitch_2" value="0.7"/>
+            <joint name="elbow_pitch_2" value="1.4"/>
+        </xacro:if>
+        <xacro:if value="${ADD_UPPER_BODY}">
+            <joint name="shoulder_yaw_1" value="0"/>
+            <joint name="shoulder_pitch_stator_1" value="0"/>
+            <joint name="shoulder_pitch_1" value="0"/>
+            <joint name="elbow_pitch_stator_1" value="0"/>
+            <joint name="elbow_pitch_1" value="0"/>
+            <joint name="hand_joint_1" value="0"/>
+            <joint name="shoulder_yaw_2" value="0"/>
+            <joint name="shoulder_pitch_stator_2" value="0"/>
+            <joint name="shoulder_pitch_2" value="0"/>
+            <joint name="elbow_pitch_stator_2" value="0"/>
+            <joint name="elbow_pitch_2" value="0"/>
+            <joint name="hand_joint_2" value="0"/>
+        </xacro:if>
     </group_state>
 </robot>

File: cetc_sat_urdf/urdf/cetc_sat_base.urdf.xacro (robot description, xacro)
@@ -1,8 +1,4 @@
 <?xml version="1.0"?>
 <robot xmlns:xacro="http://ros.org/wiki/xacro" name="cetc_sat">
-<!--
-  ROS urdf definition of the CETC-SAT quadruped robot by Istituto Italiano di Tecnologia
-  Author: Luca Rossini
--->
 <xacro:include filename="$(find cetc_sat_urdf)/urdf/utils.urdf.xacro" />
 <xacro:include filename="$(find cetc_sat_urdf)/urdf/parts/kinematics_properties.urdf.xacro" />
@@ -59,5 +55,5 @@
         color_height="720"
         color_fps="30">
-        <origin xyz="-0.1 0.22 0" rpy="0 0.25 1.57"/>
+        <origin xyz="-0.175 0.22 0" rpy="0 0.35 1.57"/>
     </xacro:sensor_d435i>
     <!-- RIGHT D435 CAMERA -->
@@ -80,5 +76,5 @@
         color_height="720"
         color_fps="30">
-        <origin xyz="-0.1 -0.22 0" rpy="0 0.25 -1.57"/>
+        <origin xyz="-0.175 -0.22 0" rpy="0 0.35 -1.57"/>
     </xacro:sensor_d435i>
     <!-- REAR D435 CAMERA -->
@@ -101,5 +97,5 @@
         color_height="720"
         color_fps="30">
-        <origin xyz="-0.39 0 0" rpy="0 0.25 3.14"/>
+        <origin xyz="-0.39 0 0" rpy="0 0.35 3.14"/>
     </xacro:sensor_d435i>
     <!-- FRONT1 D435 CAMERA -->
@@ -122,5 +118,5 @@
         color_height="720"
         color_fps="30">
-        <origin xyz="0.40 -0.075 0" rpy="1.57 0 0.21"/>
+        <origin xyz="0.40 -0.08 0" rpy="-1.57 0 0.34"/>
     </xacro:sensor_d435i>
     <!-- FRONT2 D435 CAMERA -->
@@ -143,5 +139,26 @@
         color_height="720"
         color_fps="30">
-        <origin xyz="0.40 0.075 0" rpy="1.57 0 -0.21"/>
+        <origin xyz="0.40 0.08 0" rpy="-1.57 0 -0.34"/>
+    </xacro:sensor_d435i>
+    <!-- FRONT3 (down) D435 CAMERA -->
+    <xacro:sensor_d435i parent="pelvis"
+        name="D435_front3"
+        topics_ns="D435_front3"
+        enable_pointCloud="true"
+        align_depth="true"
+        unite_imu_method="false"
+        visualize="true"
+        accel_fps="300"
+        gyro_fps="300"
+        depth_width="1280"
+        depth_height="720"
+        depth_fps="90"
+        infra_width="1280"
+        infra_height="720"
+        infra_fps="90"
+        color_width="1280"
+        color_height="720"
+        color_fps="30">
+        <origin xyz="0.37 0 -0.11" rpy="0 0.75 0"/>
     </xacro:sensor_d435i>
     <!-- Velodyne -->

File: cetc_sat_urdf/urdf/cetc_sat_robot.urdf.xacro (robot description, xacro)
@@ -1,9 +1,4 @@
 <?xml version="1.0"?>
 <robot xmlns:xacro="http://ros.org/wiki/xacro" name="cetc_sat">
-  <!--
-  ROS urdf definition of the PHOLUS humanoid robot by Istituto Italiano di Tecnologia
-  Author: Enrico Mingo
-  This file groups files to use cetc_sat in GAZEBO
-  -->
   <xacro:include filename="$(find cetc_sat_urdf)/urdf/cetc_sat.urdf.xacro" />
   <xacro:include filename="$(find cetc_sat_urdf)/urdf/gazebo/cetc_sat.gazebo.xacro" />

Commit message: Adjust xbot.gazebo and srdf

File: cetc_sat_srdf/srdf/cetc_sat.srdf.xacro (robot description, xacro)
@@ -60,24 +60,12 @@
             <joint name="hip_pitch_4" value="0.7"/>
             <joint name="knee_pitch_4" value="-1.4"/>
-            <joint name="shoulder_yaw_1" value="0.0"/>
-            <joint name="shoulder_pitch_1" value="0.7"/>
-            <joint name="elbow_pitch_1" value="1.4"/>
-            <joint name="shoulder_yaw_2" value="0.0"/>
-            <joint name="shoulder_pitch_2" value="0.7"/>
-            <joint name="elbow_pitch_2" value="1.4"/>
         </xacro:if>
         <xacro:if value="${ADD_UPPER_BODY}">
-            <joint name="shoulder_yaw_1" value="0"/>
-            <joint name="shoulder_pitch_stator_1" value="0"/>
-            <joint name="shoulder_pitch_1" value="0"/>
-            <joint name="elbow_pitch_stator_1" value="0"/>
-            <joint name="elbow_pitch_1" value="0"/>
-            <joint name="hand_joint_1" value="0"/>
-            <joint name="shoulder_yaw_2" value="0"/>
-            <joint name="shoulder_pitch_stator_2" value="0"/>
-            <joint name="shoulder_pitch_2" value="0"/>
-            <joint name="elbow_pitch_stator_2" value="0"/>
-            <joint name="elbow_pitch_2" value="0"/>
-            <joint name="hand_joint_2" value="0"/>
+            <joint name="shoulder_yaw_1" value="-0.05"/>
+            <joint name="shoulder_pitch_1" value="0.50"/>
+            <joint name="elbow_pitch_1" value="1.25"/>
+            <joint name="shoulder_yaw_2" value="0.05"/>
+            <joint name="shoulder_pitch_2" value="0.50"/>
+            <joint name="elbow_pitch_2" value="1.25"/>
         </xacro:if>
     </group_state>

File: cetc_sat_urdf/urdf/gazebo/cetc_sat.gazebo.xacro (robot description, xacro)
@@ -2,161 +2,5 @@
 <robot xmlns:xacro="http://ros.org/wiki/xacro">
     <xacro:if value="${ADD_LEGS}">
-<!--
-        <gazebo reference="imu_link">
-            <sensor name="imu_link" type="imu">
-                <always_on>1</always_on>
-                <update_rate>500</update_rate>
-                <visualize>true</visualize>
-                <topic>__default_topic__</topic>
-                <imu>
-                </imu>
-            </sensor>
-        </gazebo>
--->
-        <gazebo reference="ball_1">
-            <material>Gazebo/Residential </material>
-            <collision>
-                <surface>
-                    <friction>
-                        <!-- <torsional>
-                            <coefficient> 1.0 </coefficient>
-                            <use_patch_radius>true</use_patch_radius>
-                            <patch_radius>0.2</patch_radius>
-                        </torsional> -->
-                        <ode>
-                            <mu>1.0</mu>
-                            <mu2>1.0</mu2>
-                        </ode>
-                        <bullet>
-                            <friction>1.0</friction>
-                            <friction2>1.0</friction2>
-                        </bullet>
-                    </friction>
-                    <contact>
-                        <ode>
-                            <kp>2100000</kp>
-                            <kd>1</kd>
-                            <max_vel>100</max_vel>
-                        </ode>
-                        <bullet>
-                            <soft_cfm>0.007</soft_cfm>
-                            <soft_erp>0.25</soft_erp>
-                            <kp>1000000</kp>
-                            <kd>5</kd>
-                        </bullet>
-                    </contact>
-                </surface>
-            </collision>
-        </gazebo>
-        <gazebo reference="ball_2">
-            <material>Gazebo/Residential</material>
-            <collision>
-                <surface>
-                    <friction>
-                        <!-- <torsional>
-                            <coefficient> 1.0 </coefficient>
-                            <use_patch_radius>true</use_patch_radius>
-                            <patch_radius>0.2</patch_radius>
-                        </torsional> -->
-                        <ode>
-                            <mu>1.0</mu>
-                            <mu2>1.0</mu2>
-                        </ode>
-                        <bullet>
-                            <friction>1.0</friction>
-                            <friction2>1.0</friction2>
-                        </bullet>
-                    </friction>
-                    <contact>
-                        <ode>
-                            <kp>2100000</kp>
-                            <kd>1</kd>
-                            <max_vel>100</max_vel>
-                        </ode>
-                        <bullet>
-                            <soft_cfm>0.007</soft_cfm>
-                            <soft_erp>0.25</soft_erp>
-                            <kp>1000000</kp>
-                            <kd>5</kd>
-                        </bullet>
-                    </contact>
-                </surface>
-            </collision>
-        </gazebo>
-        <gazebo reference="ball_3">
-            <material>Gazebo/Residential </material>
-            <collision>
-                <surface>
-                    <friction>
-                        <!-- <torsional>
-                            <coefficient> 1.0 </coefficient>
-                            <use_patch_radius>true</use_patch_radius>
-                            <patch_radius>0.2</patch_radius>
-                        </torsional> -->
-                        <ode>
-                            <mu>1.0</mu>
-                            <mu2>1.0</mu2>
-                        </ode>
-                        <bullet>
-                            <friction>1.0</friction>
-                            <friction2>1.0</friction2>
-                        </bullet>
-                    </friction>
-                    <contact>
-                        <ode>
-                            <kp>2100000</kp>
-                            <kd>1</kd>
-                            <max_vel>100</max_vel>
-                        </ode>
-                        <bullet>
-                            <soft_cfm>0.007</soft_cfm>
-                            <soft_erp>0.25</soft_erp>
-                            <kp>1000000</kp>
-                            <kd>5</kd>
-                        </bullet>
-                    </contact>
-                </surface>
-            </collision>
-        </gazebo>
-        <gazebo reference="ball_4">
-            <material>Gazebo/Residential</material>
-            <collision>
-                <surface>
-                    <friction>
-                        <!-- <torsional>
-                            <coefficient> 1.0 </coefficient>
-                            <use_patch_radius>true</use_patch_radius>
-                            <patch_radius>0.2</patch_radius>
-                        </torsional> -->
-                        <ode>
-                            <mu>1.0</mu>
-                            <mu2>1.0</mu2>
-                        </ode>
-                        <bullet>
-                            <friction>1.0</friction>
-                            <friction2>1.0</friction2>
-                        </bullet>
-                    </friction>
-                    <contact>
-                        <ode>
-                            <kp>2100000</kp>
-                            <kd>1</kd>
-                            <max_vel>100</max_vel>
-                        </ode>
-                        <bullet>
-                            <soft_cfm>0.007</soft_cfm>
-                            <soft_erp>0.25</soft_erp>
-                            <kp>1000000</kp>
-                            <kd>5</kd>
-                        </bullet>
-                    </contact>
-                </surface>
-            </collision>
-        </gazebo>
         <gazebo reference="hip_roll_1">
-            <implicitSpringDamper>1</implicitSpringDamper>
-            <provideFeedback>true</provideFeedback>
-        </gazebo>
-        <gazebo reference="hip_pitch_stator_1">
             <implicitSpringDamper>1</implicitSpringDamper>
             <provideFeedback>true</provideFeedback>
@@ -166,13 +10,5 @@
             <provideFeedback>true</provideFeedback>
         </gazebo>
-        <gazebo reference="knee_pitch_stator_1">
-            <implicitSpringDamper>1</implicitSpringDamper>
-            <provideFeedback>true</provideFeedback>
-        </gazebo>
         <gazebo reference="knee_pitch_1">
-            <implicitSpringDamper>1</implicitSpringDamper>
-            <provideFeedback>true</provideFeedback>
-        </gazebo>
-        <gazebo reference="ball_joint_1">
             <implicitSpringDamper>1</implicitSpringDamper>
             <provideFeedback>true</provideFeedback>
@@ -182,13 +18,5 @@
             <provideFeedback>true</provideFeedback>
         </gazebo>
-        <gazebo reference="hip_pitch_stator_2">
-            <implicitSpringDamper>1</implicitSpringDamper>
-            <provideFeedback>true</provideFeedback>
-        </gazebo>
         <gazebo reference="hip_pitch_2">
-            <implicitSpringDamper>1</implicitSpringDamper>
-            <provideFeedback>true</provideFeedback>
-        </gazebo>
-        <gazebo reference="knee_pitch_stator_2">
             <implicitSpringDamper>1</implicitSpringDamper>
             <provideFeedback>true</provideFeedback>
@@ -198,13 +26,5 @@
             <provideFeedback>true</provideFeedback>
         </gazebo>
-        <gazebo reference="ball_joint_2">
-            <implicitSpringDamper>1</implicitSpringDamper>
-            <provideFeedback>true</provideFeedback>
-        </gazebo>
         <gazebo reference="hip_roll_3">
-            <implicitSpringDamper>1</implicitSpringDamper>
-            <provideFeedback>true</provideFeedback>
-        </gazebo>
-        <gazebo reference="hip_pitch_stator_3">
             <implicitSpringDamper>1</implicitSpringDamper>
             <provideFeedback>true</provideFeedback>
@@ -214,13 +34,5 @@
             <provideFeedback>true</provideFeedback>
         </gazebo>
-        <gazebo reference="knee_pitch_stator_3">
-            <implicitSpringDamper>1</implicitSpringDamper>
-            <provideFeedback>true</provideFeedback>
-        </gazebo>
         <gazebo reference="knee_pitch_3">
-            <implicitSpringDamper>1</implicitSpringDamper>
-            <provideFeedback>true</provideFeedback>
-        </gazebo>
-        <gazebo reference="ball_joint_3">
             <implicitSpringDamper>1</implicitSpringDamper>
             <provideFeedback>true</provideFeedback>
@@ -230,21 +42,9 @@
             <provideFeedback>true</provideFeedback>
         </gazebo>
-        <gazebo reference="hip_pitch_stator_4">
-            <implicitSpringDamper>1</implicitSpringDamper>
-            <provideFeedback>true</provideFeedback>
-        </gazebo>
         <gazebo reference="hip_pitch_4">
             <implicitSpringDamper>1</implicitSpringDamper>
             <provideFeedback>true</provideFeedback>
         </gazebo>
-        <gazebo reference="knee_pitch_stator_4">
-            <implicitSpringDamper>1</implicitSpringDamper>
-            <provideFeedback>true</provideFeedback>
-        </gazebo>
         <gazebo reference="knee_pitch_4">
-            <implicitSpringDamper>1</implicitSpringDamper>
-            <provideFeedback>true</provideFeedback>
-        </gazebo>
-        <gazebo reference="ball_joint_4">
             <implicitSpringDamper>1</implicitSpringDamper>
             <provideFeedback>true</provideFeedback>
@@ -256,13 +56,5 @@
             <provideFeedback>true</provideFeedback>
         </gazebo>
-        <gazebo reference="shoulder_pitch_stator_1">
-            <implicitSpringDamper>1</implicitSpringDamper>
-            <provideFeedback>true</provideFeedback>
-        </gazebo>
         <gazebo reference="shoulder_pitch_1">
-            <implicitSpringDamper>1</implicitSpringDamper>
-            <provideFeedback>true</provideFeedback>
-        </gazebo>
-        <gazebo reference="elbow_pitch_stator_1">
             <implicitSpringDamper>1</implicitSpringDamper>
             <provideFeedback>true</provideFeedback>
@@ -272,13 +64,5 @@
             <provideFeedback>true</provideFeedback>
         </gazebo>
-        <gazebo reference="hand_joint_1">
-            <implicitSpringDamper>1</implicitSpringDamper>
-            <provideFeedback>true</provideFeedback>
-        </gazebo>
         <gazebo reference="shoulder_yaw_2">
-            <implicitSpringDamper>1</implicitSpringDamper>
-            <provideFeedback>true</provideFeedback>
-        </gazebo>
-        <gazebo reference="shoulder_pitch_stator_2">
             <implicitSpringDamper>1</implicitSpringDamper>
             <provideFeedback>true</provideFeedback>
@@ -288,13 +72,5 @@
             <provideFeedback>true</provideFeedback>
         </gazebo>
-        <gazebo reference="elbow_pitch_stator_2">
-            <implicitSpringDamper>1</implicitSpringDamper>
-            <provideFeedback>true</provideFeedback>
-        </gazebo>
         <gazebo reference="elbow_pitch_2">
-            <implicitSpringDamper>1</implicitSpringDamper>
-            <provideFeedback>true</provideFeedback>
-        </gazebo>
-        <gazebo reference="hand_joint_2">
             <implicitSpringDamper>1</implicitSpringDamper>
             <provideFeedback>true</provideFeedback>

File: cetc_sat_urdf/urdf/gazebo/xbot.gazebo.xacro (robot description, xacro)
@@ -5,5 +5,4 @@
         <links>
             <link name="pelvis"/>
-            <link name="ball_1"/>
         </links>
     </plugin>
@@ -16,45 +15,22 @@
             <gain name="medium_mot" p="4000" d="40"/>
             <gain name="big_mot"    p="8000" d="50"/>
-            <gain name="wheel_mot"  p="25" d="5"/>
-            <pid name="neck_yaw" profile="lowpwr_mot"/>
-            <pid name="neck_pitch" profile="lowpwr_mot"/>
-            <pid name="neck_velodyne" p="0"  d="20"/>
             <pid name="shoulder_yaw_1" profile="medium_mot"/>
-            <pid name="shoulder_pitch_stator_1" profile="medium_mot"/>
             <pid name="shoulder_pitch_1" profile="medium_mot"/>
-            <pid name="elbow_pitch_stator_1" profile="medium_mot"/>
             <pid name="elbow_pitch_1" profile="small_mot"/>
-            <pid name="hand_joint_1" profile="small_mot"/>
-            <pid name="shoulder_yaw_1" profile="medium_mot"/>
-            <pid name="shoulder_pitch_stator_1" profile="medium_mot"/>
-            <pid name="shoulder_pitch_1" profile="medium_mot"/>
-            <pid name="elbow_pitch_stator_1" profile="medium_mot"/>
-            <pid name="elbow_pitch_1" profile="small_mot"/>
-            <pid name="hand_joint_1" profile="small_mot"/>
-            <pid name="torso_yaw" profile="big_mot"/>
+            <pid name="shoulder_yaw_2" profile="medium_mot"/>
+            <pid name="shoulder_pitch_2" profile="medium_mot"/>
+            <pid name="elbow_pitch_2" profile="small_mot"/>
             <pid name="hip_roll_1"     profile="big_mot"/>
-            <pid name="hip_pitch_stator_1"   profile="big_mot"/>
             <pid name="hip_pitch_1"  profile="big_mot"/>
-            <pid name="knee_pitch_stator_1" profile="medium_mot"/>
             <pid name="knee_pitch_1"   profile="medium_mot"/>
-            <pid name="ball_joint_1"     profile="wheel_mot"/>
             <pid name="hip_roll_2"     profile="big_mot"/>
-            <pid name="hip_pitch_stator_2"   profile="big_mot"/>
             <pid name="hip_pitch_2"  profile="big_mot"/>
-            <pid name="knee_pitch_stator_2" profile="medium_mot"/>
             <pid name="knee_pitch_2"   profile="medium_mot"/>
-            <pid name="ball_joint_2"     profile="wheel_mot"/>
             <pid name="hip_roll_3"     profile="big_mot"/>
-            <pid name="hip_pitch_stator_3"   profile="big_mot"/>
             <pid name="hip_pitch_3"  profile="big_mot"/>
-            <pid name="knee_pitch_stator_3" profile="medium_mot"/>
             <pid name="knee_pitch_3"   profile="medium_mot"/>
-            <pid name="ball_joint_3"     profile="wheel_mot"/>
             <pid name="hip_roll_4"     profile="big_mot"/>
-            <pid name="hip_pitch_stator_4"   profile="big_mot"/>
             <pid name="hip_pitch_4"  profile="big_mot"/>
-            <pid name="knee_pitch_stator_4" profile="medium_mot"/>
             <pid name="knee_pitch_4"   profile="medium_mot"/>
-            <pid name="ball_joint_4"     profile="wheel_mot"/>
         </pid>
     </plugin>
