Commit message: joint configuration

File: cetc_sat_srdf/srdf/cetc_sat.srdf.xacro (robot description, xacro)
@@ -27,8 +27,8 @@
     <xacro:if value="${ADD_UPPER_BODY}">
     	<group name="left_arm">
-    		<chain base_link="pelvis" tip_link="dagana_1_bottom_link"/>
+    		<chain base_link="pelvis" tip_link="wrist_1"/>
     	</group>
     	<group name="right_arm">
-    		<chain base_link="pelvis" tip_link="dagana_2_bottom_link"/>
+    		<chain base_link="pelvis" tip_link="wrist_2"/>
     	</group>
     </xacro:if>

File: cetc_sat_urdf/urdf/parts/cetc_sat_arm.urdf.xacro (robot description, xacro)
@@ -106,25 +106,26 @@
 </link>
 <!-- /shoulder-elbow -->
-<!--link name="ball_arm_${arm_num}">
-    <inertial>
+<link name="wrist_${arm_num}">
+	<inertial>
 		<origin xyz="0.0 0.0 0.0"/>
-		<mass value="${ball_mass}"/>
-		<inertia ixx="${Ball_xx}" ixy="${Ball_xy}" ixz="${Ball_xz}" iyy="${Ball_yy}" iyz="${Ball_yz}" izz="${Ball_zz}"/>
+		<mass value="${motorA_mass}"/>
+		<inertia ixx="${MotorA_xx}" ixy="${MotorA_xy}" ixz="${MotorA_xz}" iyy="${MotorA_yy}" iyz="${MotorA_yz}" izz="${MotorA_zz}"/>
 	</inertial>
 	<visual>
-		<origin xyz="0.0 0.0 0.0" rpy="0.0 0.0 0.0"/>
-		<geometry>
-			<sphere radius="${ball_radius}"/>
-		</geometry>
+		<origin xyz="0.0 0.0 0.0"  rpy="0.0 0.0 0.0"/>
+	  	<geometry>
+	 		<cylinder radius="${cylinder_radius}" length="${cylinder_length}"/>
+	  	</geometry>
+  		<material name="dark_grey"/>
 	</visual>
 	<collision>
-		<origin xyz="0.0 0.0 0.0" rpy="0.0 0.0 0.0"/>
+		<origin xyz="0.0 0.0 0.0"  rpy="0.0 0.0 0.0"/>
 		<geometry>
-			<sphere radius="${ball_radius}"/>
+			<cylinder radius="${cylinder_radius/2}" length="${cylinder_length/2}"/>
 		</geometry>
 	</collision>
-</link-->
-<xacro:dagana_gripper name="dagana_${arm_num}" parent_link="upper_arm_${arm_num}" joint_type="fixed">
-	<origin xyz="${EndEffector_Ox} ${EndEffector_Oy} ${EndEffector_Oz}" rpy="${EndEffector_roll} ${EndEffector_pitch} ${EndEffector_yaw}"/>
+</link>
+<xacro:dagana_gripper name="dagana_${arm_num}" parent_link="wrist_${arm_num}" joint_type="fixed">
+	<origin xyz="0 0 0" rpy="0 0 0"/>
 </xacro:dagana_gripper>
 <!-- /LINKS -->
@@ -165,9 +166,11 @@
 </joint>
 <!-- end effector  -->
-<!--joint name="hand_joint_${arm_num}" type="fixed">
+<joint name="wrist_joint_${arm_num}" type="revolute">
 	<parent link="upper_arm_${arm_num}"/>
-	<child link="ball_arm_${arm_num}"/>
+	<child link="wrist_${arm_num}"/>
 	<origin xyz="${EndEffector_Ox} ${EndEffector_Oy} ${EndEffector_Oz}" rpy="${EndEffector_roll} ${EndEffector_pitch} ${EndEffector_yaw}"/>
-</joint-->
+	<axis xyz="0 0 1"/>
+	<limit lower="${j_pitch_2_lower[arm_num-1]}" upper="${j_pitch_2_upper[arm_num-1]}" effort="${motor_effort}" velocity="${motor_velocity}"/>
+</joint>
 <xacro:if value="${PAYLOAD}">
 	<link name="payload_${arm_num}">

Commit message: params and joint configurations

File: cetc_sat_srdf/srdf/cetc_sat.srdf.xacro (robot description, xacro)
@@ -27,8 +27,8 @@
     <xacro:if value="${ADD_UPPER_BODY}">
     	<group name="left_arm">
-    		<chain base_link="pelvis" tip_link="wrist_1"/>
+    		<chain base_link="pelvis" tip_link="upper_arm3_1"/>
     	</group>
     	<group name="right_arm">
-    		<chain base_link="pelvis" tip_link="wrist_2"/>
+    		<chain base_link="pelvis" tip_link="upper_arm3_2"/>
     	</group>
     </xacro:if>

File: cetc_sat_urdf/urdf/parts/cetc_sat_arm.urdf.xacro (robot description, xacro)
@@ -48,5 +48,5 @@
 <link name="lower_arm_${arm_num}">
 	<inertial>
-		<origin xyz="${lower_arm_length / 2} 0.0 0.0"/>
+		<origin xyz="0.0 0.0 0.0"/>
 		<mass value="${lower_arm_mass}"/>
 		<inertia ixx="${LowerArm_xx}" ixy="${LowerArm_xy}" ixz="${LowerArm_xz}" iyy="${LowerArm_yy}" iyz="${LowerArm_yz}" izz="${LowerArm_zz}"/>
@@ -87,5 +87,5 @@
 <link name="upper_arm1_${arm_num}">
 	<inertial>
-		<origin xyz="${upper_arm1_length / 2} 0.0 0.0"/>
+		<origin xyz="0.0 0.0 0.0"/>
 		<mass value="${upper_arm1_mass}"/>
 		<inertia ixx="${UpperArm1_xx}" ixy="${UpperArm1_xy}" ixz="${UpperArm1_xz}" iyy="${UpperArm1_yy}" iyz="${UpperArm1_yz}" izz="${UpperArm1_zz}"/>
@@ -126,5 +126,5 @@
 <link name="upper_arm2_${arm_num}">
 	<inertial>
-		<origin xyz="${upper_arm2_length / 2} 0.0 0.0"/>
+		<origin xyz="0.0 0.0 0.0"/>
 		<mass value="${upper_arm2_mass}"/>
 		<inertia ixx="${UpperArm2_xx}" ixy="${UpperArm2_xy}" ixz="${UpperArm2_xz}" iyy="${UpperArm2_yy}" iyz="${UpperArm2_yz}" izz="${UpperArm2_zz}"/>
@@ -144,5 +144,5 @@
 </link>>
 <!-- /shoulder-elbow -->
-<link name="wrist_${arm_num}">
+<link name="wrist_yaw_motor_${arm_num}">
 	<inertial>
 		<origin xyz="0.0 0.0 0.0"/>
@@ -164,4 +164,23 @@
 	</collision>
 </link>
+<link name="upper_arm3_${arm_num}">
+	<inertial>
+		<origin xyz="0.0 0.0 0.0"/>
+		<mass value="${upper_arm3_mass}"/>
+		<inertia ixx="${UpperArm3_xx}" ixy="${UpperArm2_xy}" ixz="${UpperArm2_xz}" iyy="${UpperArm2_yy}" iyz="${UpperArm2_yz}" izz="${UpperArm2_zz}"/>
+	</inertial>
+	<visual>
+		<origin xyz="${upper_arm3_length / 2} 0.0 0.0"  rpy="0.0 0.0 0.0"/>
+		<geometry>
+			<box size="${upper_arm3_length} ${upper_arm2_width} ${upper_arm2_height}"/>
+		</geometry>
+	</visual>
+	<collision>
+		<origin xyz="${upper_arm3_length / 2} 0.0 0.0"  rpy="0.0 0.0 0.0"/>
+		<geometry>
+			<box size="${upper_arm3_length} ${upper_arm3_width} ${upper_arm3_height}"/>
+		</geometry>
+	</collision>
+</link>>
 <!--link name="ball_arm_${arm_num}">
 	<inertial>
@@ -183,6 +202,6 @@
 	</collision>
 </link-->
-<xacro:dagana_gripper name="dagana_${arm_num}" parent_link="wrist_${arm_num}" joint_type="fixed">
-	<origin xyz="0 0 0" rpy="0 0 0"/>
+<xacro:dagana_gripper name="dagana_${arm_num}" parent_link="upper_arm3_${arm_num}" joint_type="fixed">
+	<origin xyz="${EndEffector_Ox} ${EndEffector_Oy} ${EndEffector_Oz}" rpy="${EndEffector_roll} ${EndEffector_pitch} ${EndEffector_yaw}"/>
 </xacro:dagana_gripper>
 <!-- /LINKS -->
@@ -214,5 +233,5 @@
 	<origin xyz="${ElbowPitch_Ox} ${ElbowPitch_Oy} ${ElbowPitch_Oz}" rpy="${ElbowPitch_roll} ${ElbowPitch_pitch} ${ElbowPitch_yaw}"/>
 </joint>
-<!-- arm pitch 2 -->
+<!-- upper arm -->
 <joint name="elbow_pitch_${arm_num}" type="revolute">
 	<parent link="elbow_pitch_motor_${arm_num}"/>
@@ -222,21 +241,25 @@
 	<limit lower="${j_pitch_2_lower[arm_num-1]}" upper="${j_pitch_2_upper[arm_num-1]}" effort="${motor_effort}" velocity="${motor_velocity}"/>
 </joint>
+<joint name="wrist_yaw_stator_${arm_num}" type="fixed">
+	<parent link="upper_arm1_${arm_num}"/>
+	<child link="wrist_yaw_motor_${arm_num}"/>
+	<origin xyz="${WristYaw_Ox} ${WristYaw_Oy} ${WristYaw_Oz}" rpy="${WristYaw_roll} ${WristYaw_pitch} ${WristYaw_yaw}"/>
+</joint>
+<joint name="wrist_yaw_${arm_num}" type="revolute">
+	<parent link="wrist_yaw_motor_${arm_num}"/>
+	<child link="upper_arm2_${arm_num}"/>
+	<origin xyz="${UpperArm2_Ox} ${UpperArm2_Oy} ${UpperArm2_Oz}" rpy="${UpperArm2_roll} ${UpperArm2_pitch} ${UpperArm2_yaw}"/>
+	<axis xyz="1 0 0"/>
+	<limit lower="${j_pitch_2_lower[arm_num-1]}" upper="${j_pitch_2_upper[arm_num-1]}" effort="${motor_effort}" velocity="${motor_velocity}"/>
+</joint>
 <joint name="wrist_pitch_stator_${arm_num}" type="fixed">
-	<parent link="upper_arm1_${arm_num}"/>
+	<origin xyz="${WristPitch_Ox} ${WristPitch_Oy} ${WristPitch_Oz}" rpy="${WristPitch_roll} ${WristPitch_pitch} ${WristPitch_yaw}"/>
+	<parent link="upper_arm2_${arm_num}"/>
 	<child link="wrist_pitch_motor_${arm_num}"/>
-	<origin xyz="${WristPitch_Ox} ${WristPitch_Oy} ${WristPitch_Oz}" rpy="${WristPitch_roll} ${WristPitch_pitch} ${WristPitch_yaw}"/>
 </joint>
 <joint name="wrist_pitch_${arm_num}" type="revolute">
 	<parent link="wrist_pitch_motor_${arm_num}"/>
-	<child link="upper_arm2_${arm_num}"/>
-	<origin xyz="${UpperArm2_Ox} ${UpperArm2_Oy} ${UpperArm2_Oz}" rpy="${UpperArm2_roll} ${UpperArm2_pitch} ${UpperArm2_yaw}"/>
-	<axis xyz="0 0 1"/>
-	<limit lower="${j_pitch_2_lower[arm_num-1]}" upper="${j_pitch_2_upper[arm_num-1]}" effort="${motor_effort}" velocity="${motor_velocity}"/>
-</joint>
-<!-- end effector  -->
-<joint name="wrist_yaw_${arm_num}" type="revolute">
-	<parent link="upper_arm2_${arm_num}"/>
-	<child link="wrist_${arm_num}"/>
-	<origin xyz="${EndEffector_Ox} ${EndEffector_Oy} ${EndEffector_Oz}" rpy="${EndEffector_roll} ${EndEffector_pitch} ${EndEffector_yaw}"/>
+	<child link="upper_arm3_${arm_num}"/>
+	<origin xyz="${UpperArm3_Ox} ${UpperArm3_Oy} ${UpperArm3_Oz}" rpy="${UpperArm3_roll} ${UpperArm3_pitch} ${UpperArm3_yaw}"/>
 	<axis xyz="0 0 1"/>
 	<limit lower="${j_pitch_2_lower[arm_num-1]}" upper="${j_pitch_2_upper[arm_num-1]}" effort="${motor_effort}" velocity="${motor_velocity}"/>

File: cetc_sat_urdf/urdf/parts/inertial_properties.urdf.xacro (robot description, xacro)
@@ -11,4 +11,5 @@
         <xacro:property name="upper_arm1_mass" value="${inertial_props['upper_arm1_mass'][id]}"/>
         <xacro:property name="upper_arm2_mass" value="${inertial_props['upper_arm2_mass'][id]}"/>
+        <xacro:property name="upper_arm3_mass" value="${inertial_props['upper_arm3_mass'][id]}"/>
         <xacro:property name="lower_arm_mass" value="${inertial_props['lower_arm_mass'][id]}"/>
         <xacro:property name="ball_mass" value="${inertial_props['ball_mass'][id]}"/>
@@ -24,4 +25,5 @@
         <xacro:property name="upper_arm1_mass" value="${inertial_props['upper_arm1_mass']}"/>
         <xacro:property name="upper_arm2_mass" value="${inertial_props['upper_arm2_mass']}"/>
+        <xacro:property name="upper_arm3_mass" value="${inertial_props['upper_arm3_mass']}"/>
         <xacro:property name="lower_arm_mass" value="${inertial_props['lower_arm_mass']}"/>
         <xacro:property name="ball_mass" value="${inertial_props['ball_mass']}"/>
@@ -77,4 +79,10 @@
     <xacro:property name="UpperArm2_yz" value="0.0"/>
     <xacro:property name="UpperArm2_zz" value="${1/12 * upper_arm2_mass * (upper_arm2_width * upper_arm2_width + upper_arm2_length * upper_arm2_length)}"/>
+    <xacro:property name="UpperArm3_xx" value="${1/12 * upper_arm3_mass * (upper_arm3_width * upper_arm3_width + upper_arm3_height * upper_arm3_height)}"/>
+    <xacro:property name="UpperArm3_xy" value="0.0"/>
+    <xacro:property name="UpperArm3_xz" value="0.0"/>
+    <xacro:property name="UpperArm3_yy" value="${1/12 * upper_arm3_mass * (upper_arm3_length * upper_arm3_length + upper_arm3_height * upper_arm3_height)}"/>
+    <xacro:property name="UpperArm3_yz" value="0.0"/>
+    <xacro:property name="UpperArm3_zz" value="${1/12 * upper_arm3_mass * (upper_arm3_width * upper_arm3_width + upper_arm3_length * upper_arm3_length)}"/>
     <!-- Lower Arm -->
     <xacro:property name="LowerArm_xx" value="${1/12 * lower_arm_mass * (lower_arm_width * lower_arm_width + lower_arm_height * lower_arm_height)}"/>

File: cetc_sat_urdf/urdf/parts/kinematics_properties.urdf.xacro (robot description, xacro)
@@ -20,4 +20,7 @@
         <xacro:property name="upper_arm2_width" value="${kin_props['upper_arm2_width'][id]}"/>
         <xacro:property name="upper_arm2_height" value="${kin_props['upper_arm2_height'][id]}"/>
+        <xacro:property name="upper_arm3_length" value="${kin_props['upper_arm3_length'][id]}"/>
+        <xacro:property name="upper_arm3_width" value="${kin_props['upper_arm3_width'][id]}"/>
+        <xacro:property name="upper_arm3_height" value="${kin_props['upper_arm3_height'][id]}"/>
         <xacro:property name="lower_arm_length" value="${kin_props['lower_arm_length'][id]}"/>
         <xacro:property name="lower_arm_width" value="${kin_props['lower_arm_width'][id]}"/>
@@ -45,4 +48,7 @@
         <xacro:property name="upper_arm2_width" value="${kin_props['upper_arm2_width']}"/>
         <xacro:property name="upper_arm2_height" value="${kin_props['upper_arm2_height']}"/>
+        <xacro:property name="upper_arm3_length" value="${kin_props['upper_arm3_length']}"/>
+        <xacro:property name="upper_arm3_width" value="${kin_props['upper_arm3_width']}"/>
+        <xacro:property name="upper_arm3_height" value="${kin_props['upper_arm3_height']}"/>
         <xacro:property name="lower_arm_length" value="${kin_props['lower_arm_length']}"/>
         <xacro:property name="lower_arm_width" value="${kin_props['lower_arm_width']}"/>
@@ -98,6 +104,4 @@
     <xacro:property name="ShoulderYaw_Oy" value="${pelvis_width / 2}"/>
     <xacro:property name="ShoulderYaw_Oz" value="${pelvis_height / 2}"/>
-    <!--xacro:property name="ShoulderYaw_roll" value="0.5"/>
-    <xacro:property name="ShoulderYaw_pitch" value="0.4"/-->
     <xacro:property name="ShoulderYaw_roll" value="0.0"/>
     <xacro:property name="ShoulderYaw_pitch" value="0.0"/>
@@ -130,20 +134,32 @@
     <xacro:property name="UpperArm1_pitch" value="0.0"/>
     <xacro:property name="UpperArm1_yaw" value="0.0"/>
-    <xacro:property name="WristPitch_Ox" value="${upper_arm1_length}"/>
-	<xacro:property name="WristPitch_Oy" value="0.0"/>
-	<xacro:property name="WristPitch_Oz" value="0.0"/>
-	<xacro:property name="WristPitch_roll" value="0.0"/>
-	<xacro:property name="WristPitch_pitch" value="0.0"/>
-	<xacro:property name="WristPitch_yaw" value="0.0"/>
+    <xacro:property name="WristYaw_Ox" value="${upper_arm1_length}"/>
+	<xacro:property name="WristYaw_Oy" value="0.0"/>
+	<xacro:property name="WristYaw_Oz" value="0.0"/>
+	<xacro:property name="WristYaw_roll" value="0.0"/>
+	<xacro:property name="WristYaw_pitch" value="${PI_2}"/>
+	<xacro:property name="WristYaw_yaw" value="0.0"/>
 	<xacro:property name="UpperArm2_Ox" value="0.0"/>
     <xacro:property name="UpperArm2_Oy" value="0.0"/>
     <xacro:property name="UpperArm2_Oz" value="0.0"/>
     <xacro:property name="UpperArm2_roll" value="0.0"/>
-    <xacro:property name="UpperArm2_pitch" value="0.0"/>
+    <xacro:property name="UpperArm2_pitch" value="${-PI_2}"/>
     <xacro:property name="UpperArm2_yaw" value="0.0"/>
-    <xacro:property name="EndEffector_Ox" value="${upper_arm2_length}"/>
+	<xacro:property name="WristPitch_Ox" value="${upper_arm2_length}"/>
+    <xacro:property name="WristPitch_Oy" value="0.0"/>
+    <xacro:property name="WristPitch_Oz" value="0.0"/>
+    <xacro:property name="WristPitch_roll" value="0.0"/>
+    <xacro:property name="WristPitch_pitch" value="0.0"/>
+    <xacro:property name="WristPitch_yaw" value="0.0"/>
+    <xacro:property name="UpperArm3_Ox" value="0.0"/>
+    <xacro:property name="UpperArm3_Oy" value="0.0"/>
+    <xacro:property name="UpperArm3_Oz" value="0.0"/>
+    <xacro:property name="UpperArm3_roll" value="0.0"/>
+    <xacro:property name="UpperArm3_pitch" value="0.0"/>
+    <xacro:property name="UpperArm3_yaw" value="0.0"/>
+    <xacro:property name="EndEffector_Ox" value="${upper_arm3_length}"/>
     <xacro:property name="EndEffector_Oy" value="0.0"/>
     <xacro:property name="EndEffector_Oz" value="0.0"/>
-    <xacro:property name="EndEffector_roll" value="0.0	"/>
+    <xacro:property name="EndEffector_roll" value="0.0"/>
     <xacro:property name="EndEffector_pitch" value="${PI_2}"/>
     <xacro:property name="EndEffector_yaw" value="0.0"/>
