Commit message: fixed parameters

File: cetc_sat_urdf/urdf/parts/cetc_sat_arm.urdf.xacro (robot description, xacro)
@@ -130,5 +130,5 @@
 	<parent link="${parent}"/>
 	<child link="shoulder_yaw_motor_${arm_num}"/>
-	<origin xyz="${props['ShoulderYaw_Ox'] / 2 -0.1} ${rot*props['ShoulderYaw_Oy'] / 2 - rot*0.05} ${props['ShoulderYaw_Oz'] / 2}" rpy="${props['ShoulderYaw_roll']} ${props['ShoulderYaw_pitch']} ${props['ShoulderYaw_yaw']}"/>
+	<origin xyz="${ShoulderYaw_Ox - ShoulderYaw_OffsetX} ${rot * ShoulderYaw_Oy - rot * ShoulderYaw_OffsetY} ${ShoulderYaw_Oz - ShoulderYaw_OffsetZ}" rpy="${ShoulderYaw_roll} ${ShoulderYaw_pitch} ${ShoulderYaw_yaw}"/>
 	<axis xyz="0 0 1"/>
 	<limit lower="${j_shoulder_yaw_lower[arm_num-1]}" upper="${j_shoulder_yaw_upper[arm_num-1]}" effort="${j_shoulder_torque[arm_num-1]}" velocity="${j_shoulder_velocity[arm_num-1]}"/>
@@ -137,5 +137,5 @@
 	<parent link="shoulder_yaw_motor_${arm_num}"/>
 	<child link="shoulder_pitch_motor_${arm_num}"/>
-	<origin xyz="${props['ShoulderPitch_Ox']} ${props['ShoulderPitch_Oy']} ${props['ShoulderPitch_Oz'] / 2}" rpy="${-props['ShoulderPitch_roll']} ${props['ShoulderPitch_pitch']} ${props['ShoulderPitch_yaw']}"/>
+	<origin xyz="${ShoulderPitch_Ox} ${ShoulderPitch_Oy} ${ShoulderPitch_Oz}" rpy="${ShoulderPitch_roll} ${ShoulderPitch_pitch} ${ShoulderPitch_yaw}"/>
 </joint>
 <!-- arm pitch 1 -->
@@ -143,5 +143,5 @@
 	<parent link="shoulder_pitch_motor_${arm_num}"/>
 	<child link="lower_arm_${arm_num}"/>
-	<origin xyz="${props['LowerArm_Ox']} ${props['LowerArm_Oy']} ${props['LowerArm_Oz'] / 2}" rpy="${props['LowerArm_roll']} ${props['LowerArm_pitch']} ${-props['LowerArm_yaw']}"/>
+	<origin xyz="${LowerArm_Ox} ${LowerArm_Oy} ${LowerArm_Oz}" rpy="${LowerArm_roll} ${LowerArm_pitch} ${LowerArm_yaw}"/>
 	<axis xyz="0 0 1"/>
 	<limit lower="${j_pitch_1_lower[arm_num-1]}" upper="${j_pitch_1_upper[arm_num-1]}" effort="${j_pitch_1_torque[arm_num-1]}" velocity="${j_pitch_1_velocity[arm_num-1]}"/>
@@ -150,5 +150,5 @@
 	<parent link="lower_arm_${arm_num}"/>
 	<child link="elbow_pitch_motor_${arm_num}"/>
-	<origin xyz="${props['ElbowPitch_Ox']} ${props['ElbowPitch_Oy']} ${props['ElbowPitch_Oz']}" rpy="${props['ElbowPitch_roll']} ${props['ElbowPitch_pitch']} ${props['ElbowPitch_yaw']}"/>
+	<origin xyz="${ElbowPitch_Ox} ${ElbowPitch_Oy} ${ElbowPitch_Oz}" rpy="${ElbowPitch_roll} ${ElbowPitch_pitch} ${ElbowPitch_yaw}"/>
 </joint>
 <!-- arm pitch 2 -->
@@ -156,5 +156,5 @@
 	<parent link="elbow_pitch_motor_${arm_num}"/>
 	<child link="upper_arm_${arm_num}"/>
-	<origin xyz="${props['UpperArm_Ox']} ${props['UpperArm_Oy']} ${props['UpperArm_Oz']}" rpy="${props['UpperArm_roll']} ${props['UpperArm_pitch']} ${props['UpperArm_yaw']}"/>
+	<origin xyz="${UpperArm_Ox} ${UpperArm_Oy} ${UpperArm_Oz}" rpy="${UpperArm_roll} ${UpperArm_pitch} ${UpperArm_yaw}"/>
 	<axis xyz="0 0 1"/>
 	<limit lower="${j_pitch_2_lower[arm_num-1]}" upper="${j_pitch_2_upper[arm_num-1]}" effort="${j_pitch_2_torque[arm_num-1]}" velocity="${j_pitch_2_velocity[arm_num-1]}"/>
@@ -164,5 +164,5 @@
 	<parent link="upper_arm_${arm_num}"/>
 	<child link="ball_arm_${arm_num}"/>
-	<origin xyz="${props['EndEffector_Ox']} ${props['EndEffector_Oy']} ${props['EndEffector_Oz']}" rpy="${props['EndEffector_roll']} ${props['EndEffector_pitch']} ${props['EndEffector_yaw']}"/>
+	<origin xyz="${EndEffector_Ox} ${EndEffector_Oy} ${EndEffector_Oz}" rpy="${EndEffector_roll} ${EndEffector_pitch} ${EndEffector_yaw}"/>
 </joint>
 </xacro:macro>

File: cetc_sat_urdf/urdf/parts/cetc_sat_leg.urdf.xacro (robot description, xacro)
@@ -52,5 +52,5 @@
 	<origin xyz="0.0 0.0 0.0" rpy="0.0 0.0 0.0"/>
 	<visual>
-		<origin xyz="${props['KneePitch_Ox'] / 2} 0.0 0.0"  rpy="0.0 0.0 0.0"/>
+		<origin xyz="${props['big_box_length'] / 2} 0.0 0.0"  rpy="0.0 0.0 0.0"/>
 	  	<geometry>
 	 		<box size="${props['big_box_length']} ${props['big_box_width']} ${props['big_box_height']}"/>
@@ -59,5 +59,5 @@
 	</visual>
 	<collision>
-		<origin xyz="${props['KneePitch_Ox'] / 2} 0.0 0.0"  rpy="0.0 0.0 0.0"/>
+		<origin xyz="${props['big_box_length'] / 2} 0.0 0.0"  rpy="0.0 0.0 0.0"/>
 		<geometry>
 			<box size="${props['big_box_length']} ${props['big_box_width']} ${props['big_box_height']}"/>
@@ -92,5 +92,5 @@
 	</inertial>
 	<visual>
-		<origin xyz="${props['Ankle_Ox'] / 2} 0.0 0.0"  rpy="0.0 0.0 0.0"/>
+		<origin xyz="${props['small_box_length'] / 2} 0.0 0.0"  rpy="0.0 0.0 0.0"/>
 	  	<geometry>
 	 		<box size="${props['small_box_length']} ${props['small_box_width']} ${props['small_box_height']}"/>
@@ -99,5 +99,5 @@
 	</visual>
 	<collision>
-		<origin xyz="${props['Ankle_Ox'] / 2} 0.0 0.0"  rpy="0.0 0.0 0.0"/>
+		<origin xyz="${props['small_box_length'] / 2} 0.0 0.0"  rpy="0.0 0.0 0.0"/>
 		<geometry>
 	 		<box size="${props['small_box_length']} ${props['small_box_width']} ${props['small_box_height']}"/>
@@ -128,5 +128,5 @@
 	<parent link="pelvis"/>
 	<child link="hip_roll_motor_${leg_num}"/>
-	<origin xyz="${origin_x*props['HipRoll_Ox'] / 2} ${origin_y*(-props['HipRoll_Oy'] / 2)} ${props['HipRoll_Oz']}" rpy="${props['HipRoll_roll']} ${props['HipRoll_pitch']} ${props['HipRoll_yaw']}"/>
+	<origin xyz="${origin_x * HipRoll_Ox} ${origin_y * HipRoll_Oy} ${HipRoll_Oz}" rpy="${HipRoll_roll} ${HipRoll_pitch} ${HipRoll_yaw}"/>
 	<axis xyz="0 0 1"/>
     <limit lower="${hip_roll_lower[leg_num-1]}" upper="${hip_roll_upper[leg_num-1]}" effort="${motor_A_effort}" velocity="${motor_A_velocity}"/> <!-- 200 Nm, 1 rad/s-->
@@ -135,10 +135,10 @@
 	<parent link="hip_roll_motor_${leg_num}"/>
 	<child link="hip_pitch_motor_${leg_num}"/>
-	<origin xyz="${props['HipPitch_Ox']} ${mirror * (-props['HipPitch_Oy'])} ${props['HipPitch_Oz']}" rpy="${-props['HipPitch_roll']} ${props['HipPitch_pitch']} ${props['HipPitch_yaw']}"/>
+	<origin xyz="${HipPitch_Ox} ${mirror * (HipPitch_Oy)} ${HipPitch_Oz}" rpy="${HipPitch_roll} ${HipPitch_pitch} ${HipPitch_yaw}"/>
 </joint>
 <joint name="hip_pitch_${leg_num}" type="revolute">
 	<parent link="hip_pitch_motor_${leg_num}"/>
 	<child link="upper_leg_${leg_num}"/>
-	<origin xyz="${props['UpperLeg_Ox']} ${mirror*(-props['UpperLeg_Oy']/2)} ${props['UpperLeg_Oz']}" rpy="${props['UpperLeg_roll']} ${props['UpperLeg_pitch']} ${props['UpperLeg_yaw']}"/>
+	<origin xyz="${UpperLeg_Ox} ${mirror*(UpperLeg_Oy)} ${UpperLeg_Oz}" rpy="${UpperLeg_roll} ${UpperLeg_pitch} ${UpperLeg_yaw}"/>
 	<axis xyz="0 0 1"/>
    <limit lower="${hip_pitch_lower[leg_num-1]}" upper="${hip_pitch_upper[leg_num-1]}" effort="${motor_A_effort}" velocity="${motor_A_velocity}"/> <!-- 200 Nm, 1 rad/s-->
@@ -147,10 +147,10 @@
 	<parent link="upper_leg_${leg_num}"/>
 	<child link="knee_pitch_motor_${leg_num}"/>
-	<origin xyz="${props['KneePitch_Ox']} ${props['KneePitch_Oy']} ${props['KneePitch_Oz']}" rpy="${props['KneePitch_roll']} ${props['KneePitch_pitch']} ${props['KneePitch_yaw']}"/>
+	<origin xyz="${KneePitch_Ox} ${KneePitch_Oy} ${KneePitch_Oz}" rpy="${KneePitch_roll} ${KneePitch_pitch} ${KneePitch_yaw}"/>
 </joint>
 <joint name="knee_pitch_${leg_num}" type="revolute">
 	<parent link="knee_pitch_motor_${leg_num}"/>
 	<child link="lower_leg_${leg_num}"/>
-	<origin xyz="${props['LowerLeg_Ox']} ${props['LowerLeg_Oy']} ${props['LowerLeg_Oz']}" rpy="${props['LowerLeg_roll']} ${props['LowerLeg_pitch']} ${props['LowerLeg_yaw']}"/>
+	<origin xyz="${LowerLeg_Ox} ${LowerLeg_Oy} ${LowerLeg_Oz}" rpy="${LowerLeg_roll} ${LowerLeg_pitch} ${LowerLeg_yaw}"/>
 	<axis xyz="0 0 1"/>
    <limit lower="${knee_pitch_lower[leg_num-1]}" upper="${knee_pitch_upper[leg_num-1]}" effort="${motor_A_effort}" velocity="${motor_A_velocity}"/> <!-- 200 Nm, 1 rad/s-->
@@ -159,5 +159,5 @@
 	<parent link="lower_leg_${leg_num}"/>
 	<child link="ball_${leg_num}"/>
-	<origin xyz="${props['Ankle_Ox']} ${props['Ankle_Oy']} ${props['Ankle_Oz']}" rpy="${props['Ankle_roll']} ${props['Ankle_pitch']} ${props['Ankle_yaw']}"/>
+	<origin xyz="${Ankle_Ox} ${Ankle_Oy} ${Ankle_Oz}" rpy="${Ankle_roll} ${Ankle_pitch} ${Ankle_yaw}"/>
 </joint>
 </xacro:macro>

File: cetc_sat_urdf/urdf/parts/kinematics_properties.urdf.xacro (robot description, xacro)
@@ -1,14 +1,4 @@
 <!--<?xml version="1.0"?>-->
 <robot  xmlns:xacro="http://ros.org/wiki/xacro">
-<!-- link dimensions -->
-<!--xacro:property name="cylinder_radius" value="0.07"/>
-<xacro:property name="cylinder_length" value="0.1"/>
-<xacro:property name="big_box_length" value="0.4"/>
-<xacro:property name="big_box_width" value="0.1"/>
-<xacro:property name="big_box_height" value="0.1"/>
-<xacro:property name="small_box_length" value="0.4"/>
-<xacro:property name="small_box_width" value="0.05"/>
-<xacro:property name="small_box_height" value="0.05"/>
-<xacro:property name="ball_radius" value="0.05"/-->
 <!--pelvis dimensions: length: 0.80-1.1m, width: 0.45-0.60m-->
 <xacro:property name="pelvis_length" value="0.80"/>
@@ -16,24 +6,36 @@
 <xacro:property name="pelvis_height" value="0.20"/> <!-- random value to be defined -->
 <!-- Origin -->
-<xacro:property name="Leg_1_Ox" value="${pelvis_length / 2}"/>
-<xacro:property name="Leg_1_Oy" value="${-pelvis_width / 2}"/>
-<xacro:property name="Leg_1_Oz" value="${0.0 * mmTom}"/>
-<xacro:property name="Leg_1_roll" value="0.0"/>
-<xacro:property name="Leg_1_pitch" value="${PI_2}"/>
-<xacro:property name="Leg_1_yaw" value="0.0"/>
+<xacro:property name="HipRoll_Ox" value="${props['pelvis_length'] / 2}"/>
+<xacro:property name="HipRoll_Oy" value="${-props['pelvis_width'] / 2}"/>
+<xacro:property name="HipRoll_Oz" value="0.0"/>
+<xacro:property name="HipRoll_roll" value="0.0"/>
+<xacro:property name="HipRoll_pitch" value="${PI_2}"/>
+<xacro:property name="HipRoll_yaw" value="0.0"/>
 <!-- Origin -->
-<xacro:property name="Leg_2_Ox" value="0.0"/>
-<xacro:property name="Leg_2_Oy" value="-${props['cylinder_radius'] / 2}"/>
-<xacro:property name="Leg_2_Oz" value="0.0"/>
-<xacro:property name="Leg_2_roll" value="0.0"/>
-<xacro:property name="Leg_2_pitch" value="0.0"/>
-<xacro:property name="Leg_2_yaw" value="0.0"/>
+<xacro:property name="HipPitch_Ox" value="0.0"/>
+<xacro:property name="HipPitch_Oy" value="${-props['cylinder_radius']}"/>
+<xacro:property name="HipPitch_Oz" value="0.0"/>
+<xacro:property name="HipPitch_roll" value="${-PI_2}"/>
+<xacro:property name="HipPitch_pitch" value="0.0"/>
+<xacro:property name="HipPitch_yaw" value="0.0"/>
+<xacro:property name="UpperLeg_Ox" value="0.0"/>
+<xacro:property name="UpperLeg_Oy" value="0.0"/>
+<xacro:property name="UpperLeg_Oz" value="0.0"/>
+<xacro:property name="UpperLeg_roll" value="0.0"/>
+<xacro:property name="UpperLeg_pitch" value="0.0"/>
+<xacro:property name="UpperLeg_yaw" value="0.0"/>
 <!-- Origin -->
-<xacro:property name="Leg_3_Ox" value="${props['big_box_length']}"/>
-<xacro:property name="Leg_3_Oy" value="0.0"/>
-<xacro:property name="Leg_3_Oz" value="0.0"/>
-<xacro:property name="Leg_3_roll" value="0.0"/>
-<xacro:property name="Leg_3_pitch" value="0.0"/>
-<xacro:property name="Leg_3_yaw" value="0.0"/>
+<xacro:property name="KneePitch_Ox" value="${props['big_box_length']}"/>
+<xacro:property name="KneePitch_Oy" value="0.0"/>
+<xacro:property name="KneePitch_Oz" value="0.0"/>
+<xacro:property name="KneePitch_roll" value="0.0"/>
+<xacro:property name="KneePitch_pitch" value="0.0"/>
+<xacro:property name="KneePitch_yaw" value="0.0"/>
+<xacro:property name="LowerLeg_Ox" value="0.0"/>
+<xacro:property name="LowerLeg_Oy" value="0.0"/>
+<xacro:property name="LowerLeg_Oz" value="0.0"/>
+<xacro:property name="LowerLeg_roll" value="0.0"/>
+<xacro:property name="LowerLeg_pitch" value="0.0"/>
+<xacro:property name="LowerLeg_yaw" value="0.0"/>
 <!-- Origin -->
 <xacro:property name="Ankle_Ox" value="${props['big_box_length']}"/>
@@ -44,22 +46,37 @@
 <xacro:property name="Ankle_yaw" value="0.0"/>
 <!-- Arms -->
-<xacro:property name="Shoulder_Ox" value="${pelvis_length / 2 - 0.1}"/>
-<xacro:property name="Shoulder_Oy" value="${pelvis_width / 2 - 0.05}"/>
-<xacro:property name="Shoulder_Oz" value="${pelvis_height / 2}"/>
-<xacro:property name="Shoulder_roll" value="0.0"/>
-<xacro:property name="Shoulder_pitch" value="0.0"/>
-<xacro:property name="Shoulder_yaw" value="0.0"/>
-<xacro:property name="Pitch_1_Ox" value="0.0"/>
-<xacro:property name="Pitch_1_Oy" value="0.0"/>
-<xacro:property name="Pitch_1_Oz" value="${props['cylinder_length'] / 2}"/>
-<xacro:property name="Pitch_1_roll" value="0.0"/>
-<xacro:property name="Pitch_1_pitch" value="${-PI_2}"/>
-<xacro:property name="Pitch_1_yaw" value="0.0"/>
-<xacro:property name="Pitch_2_Ox" value="${props['big_box_length']}"/>
-<xacro:property name="Pitch_2_Oy" value="0.0"/>
-<xacro:property name="Pitch_2_Oz" value="0.0"/>
-<xacro:property name="Pitch_2_roll" value="0.0"/>
-<xacro:property name="Pitch_2_pitch" value="0.0"/>
-<xacro:property name="Pitch_2_yaw" value="0.0"/>
+<xacro:property name="ShoulderYaw_Ox" value="${pelvis_length / 2}"/>
+<xacro:property name="ShoulderYaw_Oy" value="${pelvis_width / 2}"/>
+<xacro:property name="ShoulderYaw_Oz" value="${pelvis_height / 2}"/>
+<xacro:property name="ShoulderYaw_roll" value="0.0"/>
+<xacro:property name="ShoulderYaw_pitch" value="0.0"/>
+<xacro:property name="ShoulderYaw_yaw" value="0.0"/>
+<xacro:property name="ShoulderYaw_OffsetX" value="0.1"/>
+<xacro:property name="ShoulderYaw_OffsetY" value="0.05"/>
+<xacro:property name="ShoulderYaw_OffsetZ" value="0.0"/>
+<xacro:property name="ShoulderPitch_Ox" value="0.0"/>
+<xacro:property name="ShoulderPitch_Oy" value="0.0"/>
+<xacro:property name="ShoulderPitch_Oz" value="${props['cylinder_length'] / 2}"/>
+<xacro:property name="ShoulderPitch_roll" value="${-PI_2}"/>
+<xacro:property name="ShoulderPitch_pitch" value="0.0"/>
+<xacro:property name="ShoulderPitch_yaw" value="0.0"/>
+<xacro:property name="LowerArm_Ox" value="0.0"/>
+<xacro:property name="LowerArm_Oy" value="0.0"/>
+<xacro:property name="LowerArm_Oz" value="0.0"/>
+<xacro:property name="LowerArm_roll" value="0.0"/>
+<xacro:property name="LowerArm_pitch" value="0.0"/>
+<xacro:property name="LowerArm_yaw" value="${-PI_2}"/>
+<xacro:property name="ElbowPitch_Ox" value="${props['big_box_length']}"/>
+<xacro:property name="ElbowPitch_Oy" value="0.0"/>
+<xacro:property name="ElbowPitch_Oz" value="0.0"/>
+<xacro:property name="ElbowPitch_roll" value="0.0"/>
+<xacro:property name="ElbowPitch_pitch" value="0.0"/>
+<xacro:property name="ElbowPitch_yaw" value="0.0"/>
+<xacro:property name="UpperArm_Ox" value="0.0"/>
+<xacro:property name="UpperArm_Oy" value="0.0"/>
+<xacro:property name="UpperArm_Oz" value="0.0"/>
+<xacro:property name="UpperArm_roll" value="0.0"/>
+<xacro:property name="UpperArm_pitch" value="0.0"/>
+<xacro:property name="UpperArm_yaw" value="0.0"/>
 <xacro:property name="EndEffector_Ox" value="${props['big_box_length']}"/>
 <xacro:property name="EndEffector_Oy" value="0.0"/>

Commit message: added dagana

File: cetc_sat_urdf/urdf/parts/cetc_sat_arm.urdf.xacro (robot description, xacro)
@@ -1,4 +1,5 @@
 <?xml version="1.0"?>
 <robot xmlns:xacro="http://ros.org/wiki/xacro">
+<xacro:include filename="$(find dagana_urdf)/urdf/dagana_macro.urdf.xacro"/>
 <!-- macro arms -->
 <xacro:macro name="cetc_sat_arm" params="arm_num rot parent">
@@ -105,5 +106,5 @@
 </link>
 <!-- /shoulder-elbow -->
-<link name="ball_arm_${arm_num}">
+<!--link name="ball_arm_${arm_num}">
     <inertial>
 		<origin xyz="0.0 0.0 0.0"/>
@@ -123,5 +124,8 @@
 		</geometry>
 	</collision>
-</link>
+</link-->
+<xacro:dagana_gripper name="dagana_${arm_num}" parent_link="upper_arm_${arm_num}" joint_type="fixed">
+	<origin xyz="${EndEffector_Ox} ${EndEffector_Oy} ${EndEffector_Oz}" rpy="${EndEffector_roll} ${EndEffector_pitch} ${EndEffector_yaw}"/>
+</xacro:dagana_gripper>
 <!-- /LINKS -->
 <!-- JOINTS -->
@@ -130,5 +134,5 @@
 	<parent link="${parent}"/>
 	<child link="shoulder_yaw_motor_${arm_num}"/>
-	<origin xyz="${ShoulderYaw_Ox - ShoulderYaw_OffsetX} ${rot * ShoulderYaw_Oy - rot * ShoulderYaw_OffsetY} ${ShoulderYaw_Oz - ShoulderYaw_OffsetZ}" rpy="${ShoulderYaw_roll} ${ShoulderYaw_pitch} ${ShoulderYaw_yaw}"/>
+	<origin xyz="${ShoulderYaw_Ox - ShoulderYaw_OffsetX} ${rot * ShoulderYaw_Oy - rot * ShoulderYaw_OffsetY} ${ShoulderYaw_Oz - ShoulderYaw_OffsetZ}" rpy="${-rot * ShoulderYaw_roll} ${ShoulderYaw_pitch} ${ShoulderYaw_yaw}"/>
 	<axis xyz="0 0 1"/>
 	<limit lower="${j_shoulder_yaw_lower[arm_num-1]}" upper="${j_shoulder_yaw_upper[arm_num-1]}" effort="${motor_effort}" velocity="${motor_velocity}"/>
@@ -161,9 +165,29 @@
 </joint>
 <!-- end effector  -->
-<joint name="hand_joint_${arm_num}" type="fixed">
+<!--joint name="hand_joint_${arm_num}" type="fixed">
 	<parent link="upper_arm_${arm_num}"/>
 	<child link="ball_arm_${arm_num}"/>
 	<origin xyz="${EndEffector_Ox} ${EndEffector_Oy} ${EndEffector_Oz}" rpy="${EndEffector_roll} ${EndEffector_pitch} ${EndEffector_yaw}"/>
-</joint>
+</joint-->
+<xacro:if value="${PAYLOAD}">
+	<link name="payload_${arm_num}">
+		<inertial>
+		    <origin xyz="0.0 0.0 0.0"/>
+			<mass value="4"/>
+			<inertia ixx="0.0267" iyy="0.0267" izz="0.0267" ixy="0" ixz="0" iyz="0"/>
+		</inertial>
+		<visual>
+			<origin xyz="0.0 0.0 0.0"  rpy="0.0 0.0 0.0"/>
+			<geometry>
+				<box size="0.2 0.2 0.2"/>
+			</geometry>
+			<material name="dark_grey"/>
+		</visual>
+	</link>
+	<joint name="hand_to_payload_${arm_num}" type="fixed">
+		<parent link="ball_arm_${arm_num}"/>
+		<child link="payload_${arm_num}"/>
+	</joint>
+</xacro:if>
 </xacro:macro>
 <!-- /macro arms -->

File: cetc_sat_urdf/urdf/parts/kinematics_properties.urdf.xacro (robot description, xacro)
@@ -92,6 +92,8 @@
     <xacro:property name="ShoulderYaw_Oy" value="${pelvis_width / 2}"/>
     <xacro:property name="ShoulderYaw_Oz" value="${pelvis_height / 2}"/>
-    <xacro:property name="ShoulderYaw_roll" value="0.0"/>
-    <xacro:property name="ShoulderYaw_pitch" value="0.0"/>
+    <xacro:property name="ShoulderYaw_roll" value="0.5"/>
+    <xacro:property name="ShoulderYaw_pitch" value="0.4"/>
+    <!--xacro:property name="ShoulderYaw_roll" value="0.0"/>
+    <xacro:property name="ShoulderYaw_pitch" value="0.0"/-->
     <xacro:property name="ShoulderYaw_yaw" value="0.0"/>
     <xacro:property name="ShoulderYaw_OffsetX" value="0.1"/>
@@ -125,6 +127,6 @@
     <xacro:property name="EndEffector_Oy" value="0.0"/>
     <xacro:property name="EndEffector_Oz" value="0.0"/>
-    <xacro:property name="EndEffector_roll" value="0.0"/>
-    <xacro:property name="EndEffector_pitch" value="0.0"/>
+    <xacro:property name="EndEffector_roll" value="0.0	"/>
+    <xacro:property name="EndEffector_pitch" value="${PI_2}"/>
     <xacro:property name="EndEffector_yaw" value="0.0"/>
 </robot>

Commit message: roll configuration

File: cetc_sat_urdf/urdf/parts/cetc_sat_arm.urdf.xacro (robot description, xacro)
@@ -41,4 +41,24 @@
 	<collision>
 		<origin xyz="0.0 0.0 0.0"  rpy="0.0 0.0 0.0"/>
+		<geometry>
+			<cylinder radius="${cylinder_radius}" length="${cylinder_length}"/>
+		</geometry>
+	</collision>
+</link>
+<link name="shoulder_roll_motor_${arm_num}">
+	<inertial>
+		<origin xyz="0.0 0.0 0.0"/>
+		<mass value="${motorA_mass}"/>
+		<inertia ixx="${MotorA_xx}" ixy="${MotorA_xy}" ixz="${MotorA_xz}" iyy="${MotorA_yy}" iyz="${MotorA_yz}" izz="${MotorA_zz}"/>
+	</inertial>
+	<visual>
+		<origin xyz="0.0 0.0 0.0"  rpy="0.0 ${PI_2} 0.0"/>
+	  	<geometry>
+	 		<cylinder radius="${cylinder_radius}" length="${cylinder_length}"/>
+	  	</geometry>
+  		<material name="dark_grey"/>
+	</visual>
+	<collision>
+		<origin xyz="0.0 0.0 0.0"  rpy="0.0 ${PI_2} 0.0"/>
 		<geometry>
 			<cylinder radius="${cylinder_radius}" length="${cylinder_length}"/>
@@ -138,6 +158,13 @@
 	<limit lower="${j_shoulder_yaw_lower[arm_num-1]}" upper="${j_shoulder_yaw_upper[arm_num-1]}" effort="${motor_effort}" velocity="${motor_velocity}"/>
 </joint>
+<joint name="shoulder_roll_${arm_num}" type="revolute">
+	<parent link="shoulder_yaw_motor_${arm_num}"/>
+	<child link="shoulder_roll_motor_${arm_num}"/>
+	<origin xyz="0. 0. 0." rpy="0. 0. 0."/>
+	<axis xyz="1 0 0"/>
+	<limit lower="${j_shoulder_yaw_lower[arm_num-1]}" upper="${j_shoulder_yaw_upper[arm_num-1]}" effort="${motor_effort}" velocity="${motor_velocity}"/>
+</joint>
 <joint name="shoulder_pitch_stator_${arm_num}" type="fixed">
-	<parent link="shoulder_yaw_motor_${arm_num}"/>
+	<parent link="shoulder_roll_motor_${arm_num}"/>
 	<child link="shoulder_pitch_motor_${arm_num}"/>
 	<origin xyz="${ShoulderPitch_Ox} ${ShoulderPitch_Oy} ${ShoulderPitch_Oz}" rpy="${ShoulderPitch_roll} ${ShoulderPitch_pitch} ${ShoulderPitch_yaw}"/>

File: cetc_sat_urdf/urdf/parts/kinematics_properties.urdf.xacro (robot description, xacro)
@@ -92,8 +92,8 @@
     <xacro:property name="ShoulderYaw_Oy" value="${pelvis_width / 2}"/>
     <xacro:property name="ShoulderYaw_Oz" value="${pelvis_height / 2}"/>
-    <xacro:property name="ShoulderYaw_roll" value="0.5"/>
-    <xacro:property name="ShoulderYaw_pitch" value="0.4"/>
-    <!--xacro:property name="ShoulderYaw_roll" value="0.0"/>
-    <xacro:property name="ShoulderYaw_pitch" value="0.0"/-->
+    <!--xacro:property name="ShoulderYaw_roll" value="0.5"/>
+    <xacro:property name="ShoulderYaw_pitch" value="0.4"/-->
+    <xacro:property name="ShoulderYaw_roll" value="0.0"/>
+    <xacro:property name="ShoulderYaw_pitch" value="0.0"/>
     <xacro:property name="ShoulderYaw_yaw" value="0.0"/>
     <xacro:property name="ShoulderYaw_OffsetX" value="0.1"/>
