Commit message: joint configuration

File: cetc_sat_urdf/urdf/parts/cetc_sat_arm.urdf.xacro (robot description, xacro)
@@ -126,25 +126,27 @@
 </link>
 <!-- /shoulder-elbow -->
-<!--link name="ball_arm_${arm_num}">
+<link name="wrist_${arm_num}">
     <inertial>
 		<origin xyz="0.0 0.0 0.0"/>
-		<mass value="${ball_mass}"/>
-		<inertia ixx="${Ball_xx}" ixy="${Ball_xy}" ixz="${Ball_xz}" iyy="${Ball_yy}" iyz="${Ball_yz}" izz="${Ball_zz}"/>
-	</inertial>
-	<visual>
-		<origin xyz="0.0 0.0 0.0" rpy="0.0 0.0 0.0"/>
-		<geometry>
-			<sphere radius="${ball_radius}"/>
-		</geometry>
-	</visual>
-	<collision>
-		<origin xyz="0.0 0.0 0.0" rpy="0.0 0.0 0.0"/>
-		<geometry>
-			<sphere radius="${ball_radius}"/>
-		</geometry>
-	</collision>
-</link-->
-<xacro:dagana_gripper name="dagana_${arm_num}" parent_link="upper_arm_${arm_num}" joint_type="fixed">
-	<origin xyz="${EndEffector_Ox} ${EndEffector_Oy} ${EndEffector_Oz}" rpy="${EndEffector_roll} ${EndEffector_pitch} ${EndEffector_yaw}"/>
+		<mass value="${motorA_mass}"/>
+		<inertia ixx="${MotorA_xx}" ixy="${MotorA_xy}" ixz="${MotorA_xz}" iyy="${MotorA_yy}" iyz="${MotorA_yz}" izz="${MotorA_zz}"/>
+	</inertial>
+	<visual>
+		<origin xyz="0.0 0.0 0.0"  rpy="0.0 0.0 0.0"/>
+	  	<geometry>
+	 		<cylinder radius="${cylinder_radius}" length="${cylinder_length}"/>
+	  	</geometry>
+  		<material name="dark_grey"/>
+	</visual>
+	<collision>
+		<origin xyz="0.0 0.0 0.0"  rpy="0.0 0.0 0.0"/>
+	  	<geometry>
+	 		<cylinder radius="${cylinder_radius}" length="${cylinder_length}"/>
+	  	</geometry>
+  		<material name="dark_grey"/>
+	</collision>
+</link>
+<xacro:dagana_gripper name="dagana_${arm_num}" parent_link="wrist_${arm_num}" joint_type="fixed">
+	<origin xyz="0 0 0" rpy="0 0 0"/>
 </xacro:dagana_gripper>
 <!-- /LINKS -->
@@ -192,9 +194,11 @@
 </joint>
 <!-- end effector  -->
-<!--joint name="hand_joint_${arm_num}" type="fixed">
+<joint name="wrist_joint_${arm_num}" type="revolute">
 	<parent link="upper_arm_${arm_num}"/>
-	<child link="ball_arm_${arm_num}"/>
+	<child link="wrist_${arm_num}"/>
 	<origin xyz="${EndEffector_Ox} ${EndEffector_Oy} ${EndEffector_Oz}" rpy="${EndEffector_roll} ${EndEffector_pitch} ${EndEffector_yaw}"/>
-</joint-->
+	<axis xyz="0 0 1"/>
+	<limit lower="${j_pitch_2_lower[arm_num-1]}" upper="${j_pitch_2_upper[arm_num-1]}" effort="${motor_effort}" velocity="${motor_velocity}"/>
+</joint>
 <xacro:if value="${PAYLOAD}">
 	<link name="payload_${arm_num}">

Commit message: params and joint configurations

File: cetc_sat_urdf/urdf/parts/cetc_sat_arm.urdf.xacro (robot description, xacro)
@@ -46,5 +46,5 @@
 	</collision>
 </link>
-<link name="shoulder_roll_motor_${arm_num}">
+<link name="shoulder_yaw2_motor_${arm_num}">
 	<inertial>
 		<origin xyz="0.0 0.0 0.0"/>
@@ -55,5 +55,5 @@
 		<origin xyz="0.0 0.0 0.0"  rpy="0.0 ${PI_2} 0.0"/>
 	  	<geometry>
-	 		<cylinder radius="${cylinder_radius}" length="${cylinder_length}"/>
+	 		<cylinder radius="${cylinder_radius}" length="${cylinder_length/6}"/>
 	  	</geometry>
   		<material name="dark_grey"/>
@@ -62,51 +62,70 @@
 		<origin xyz="0.0 0.0 0.0"  rpy="0.0 ${PI_2} 0.0"/>
 		<geometry>
-			<cylinder radius="${cylinder_radius}" length="${cylinder_length}"/>
-		</geometry>
-	</collision>
-</link>
-<link name="lower_arm_${arm_num}">
+			<cylinder radius="${cylinder_radius}" length="${cylinder_length/6}"/>
+		</geometry>
+	</collision>
+</link>
+<link name="lower_arm1_${arm_num}">
+	<inertial>
+		<origin xyz="0.0 0.0 0.0"/>
+		<mass value="${lower_arm1_mass}"/>
+		<inertia ixx="${LowerArm1_xx}" ixy="${LowerArm1_xy}" ixz="${LowerArm1_xz}" iyy="${LowerArm1_xx}" iyz="${LowerArm1_yz}" izz="${LowerArm1_zz}"/>
+	</inertial>
+	<visual>
+		<origin xyz="${lower_arm1_length / 2} 0.0 0.0"  rpy="0.0 0.0 0.0"/>
+		<geometry>
+			<box size="${lower_arm1_length} ${lower_arm1_width} ${lower_arm1_height}"/>
+		</geometry>
+	</visual>
+	<collision>
+		<origin xyz="${lower_arm1_length / 2} 0.0 0.0"  rpy="0.0 0.0 0.0"/>
+		<geometry>
+			<box size="${lower_arm1_length} ${lower_arm1_width} ${lower_arm1_height}"/>
+		</geometry>
+	</collision>
+</link>
+<link name="lower_arm2_${arm_num}">
+	<inertial>
+		<origin xyz="0.0 0.0 0.0"/>
+		<mass value="${lower_arm2_mass}"/>
+		<inertia ixx="${LowerArm2_xx}" ixy="${LowerArm2_xy}" ixz="${LowerArm2_xz}" iyy="${LowerArm2_xx}" iyz="${LowerArm2_yz}" izz="${LowerArm2_zz}"/>
+	</inertial>
+	<visual>
+		<origin xyz="${lower_arm2_length / 2} 0.0 0.0"  rpy="0.0 0.0 0.0"/>
+		<geometry>
+			<box size="${lower_arm2_length} ${lower_arm2_width} ${lower_arm2_height}"/>
+		</geometry>
+	</visual>
+	<collision>
+		<origin xyz="${lower_arm2_length / 2} 0.0 0.0"  rpy="0.0 0.0 0.0"/>
+		<geometry>
+			<box size="${lower_arm2_length} ${lower_arm2_width} ${lower_arm2_height}"/>
+		</geometry>
+	</collision>
+</link>
+<link name="elbow_pitch_motor_${arm_num}">
+	<inertial>
+		<origin xyz="0.0 0.0 0.0"/>
+		<mass value="${motorA_mass}"/>
+		<inertia ixx="${MotorA_xx}" ixy="${MotorA_xy}" ixz="${MotorA_xz}" iyy="${MotorA_yy}" iyz="${MotorA_yz}" izz="${MotorA_zz}"/>
+	</inertial>
+	<visual>
+		<origin xyz="0.0 0.0 0.0"  rpy="0.0 0.0 0.0"/>
+	  	<geometry>
+	 		<cylinder radius="${cylinder_radius}" length="${cylinder_length}"/>
+	  	</geometry>
+  		<material name="dark_grey"/>
+	</visual>
+	<collision>
+		<origin xyz="0.0 0.0 0.0"  rpy="0.0 0.0 0.0"/>
+		<geometry>
+			<cylinder radius="${cylinder_radius}" length="${cylinder_length}"/>
+		</geometry>
+	</collision>
+</link>
+<link name="upper_arm_${arm_num}">
 	<inertial>
 		<origin xyz="0.0 0.0 0.0"/>
 		<mass value="${upper_arm_mass}"/>
-		<inertia ixx="${LowerArm_xx}" ixy="${LowerArm_xy}" ixz="${LowerArm_xz}" iyy="${LowerArm_xx}" iyz="${LowerArm_yz}" izz="${LowerArm_zz}"/>
-	</inertial>
-	<visual>
-		<origin xyz="${lower_arm_length / 2} 0.0 0.0"  rpy="0.0 0.0 0.0"/>
-		<geometry>
-			<box size="${lower_arm_length} ${lower_arm_width} ${lower_arm_height}"/>
-		</geometry>
-	</visual>
-	<collision>
-		<origin xyz="${lower_arm_length / 2} 0.0 0.0"  rpy="0.0 0.0 0.0"/>
-		<geometry>
-			<box size="${lower_arm_length} ${lower_arm_width} ${lower_arm_height}"/>
-		</geometry>
-	</collision>
-</link>
-<link name="elbow_pitch_motor_${arm_num}">
-	<inertial>
-		<origin xyz="0.0 0.0 0.0"/>
-		<mass value="${motorA_mass}"/>
-		<inertia ixx="${MotorA_xx}" ixy="${MotorA_xy}" ixz="${MotorA_xz}" iyy="${MotorA_yy}" iyz="${MotorA_yz}" izz="${MotorA_zz}"/>
-	</inertial>
-	<visual>
-		<origin xyz="0.0 0.0 0.0"  rpy="0.0 0.0 0.0"/>
-	  	<geometry>
-	 		<cylinder radius="${cylinder_radius}" length="${cylinder_length}"/>
-	  	</geometry>
-  		<material name="dark_grey"/>
-	</visual>
-	<collision>
-		<origin xyz="0.0 0.0 0.0"  rpy="0.0 0.0 0.0"/>
-		<geometry>
-			<cylinder radius="${cylinder_radius}" length="${cylinder_length}"/>
-		</geometry>
-	</collision>
-</link>
-<link name="upper_arm_${arm_num}">
-	<inertial>
-		<origin xyz="0.0 0.0 0.0"/>
-		<mass value="${lower_arm_mass}"/>
 		<inertia ixx="${UpperArm_xx}" ixy="${UpperArm_xy}" ixz="${UpperArm_xz}" iyy="${UpperArm_xx}" iyz="${UpperArm_yz}" izz="${UpperArm_zz}"/>
 	</inertial>
@@ -119,5 +138,5 @@
 	</visual>
 	<collision>
-		<origin xyz="${lower_arm_length / 2} 0.0 0.0"  rpy="0.0 0.0 0.0"/>
+		<origin xyz="${upper_arm_length / 2} 0.0 0.0"  rpy="0.0 0.0 0.0"/>
 		<geometry>
 			<box size="${upper_arm_length} ${upper_arm_width} ${upper_arm_height}"/>
@@ -160,26 +179,31 @@
 	<limit lower="${j_shoulder_yaw_lower[arm_num-1]}" upper="${j_shoulder_yaw_upper[arm_num-1]}" effort="${motor_effort}" velocity="${motor_velocity}"/>
 </joint>
-<joint name="shoulder_roll_${arm_num}" type="revolute">
+<joint name="shoulder_pitch_stator_${arm_num}" type="fixed">
 	<parent link="shoulder_yaw_motor_${arm_num}"/>
-	<child link="shoulder_roll_motor_${arm_num}"/>
+	<child link="shoulder_pitch_motor_${arm_num}"/>
+	<origin xyz="${ShoulderPitch_Ox} ${ShoulderPitch_Oy} ${ShoulderPitch_Oz}" rpy="${ShoulderPitch_roll} ${ShoulderPitch_pitch} ${ShoulderPitch_yaw}"/>
+</joint>
+<!-- arm pitch 1 -->
+<joint name="shoulder_pitch_${arm_num}" type="revolute">
+	<parent link="shoulder_pitch_motor_${arm_num}"/>
+	<child link="lower_arm1_${arm_num}"/>
+	<origin xyz="${LowerArm1_Ox} ${LowerArm1_Oy} ${LowerArm1_Oz}" rpy="${LowerArm1_roll} ${LowerArm1_pitch} ${LowerArm1_yaw}"/>
+	<axis xyz="0 0 1"/>
+	<limit lower="${j_pitch_1_lower[arm_num-1]}" upper="${j_pitch_1_upper[arm_num-1]}" effort="${motor_effort}" velocity="${motor_velocity}"/>
+</joint>
+<joint name="shoulder_yaw2_stator${arm_num}" type="fixed">
+	<parent link="lower_arm1_${arm_num}"/>
+	<child link="shoulder_yaw2_motor_${arm_num}"/>
+	<origin xyz="${LowerArm2_Ox} ${LowerArm2_Oy} ${LowerArm2_Oz}" rpy="${LowerArm2_roll} ${LowerArm2_pitch} ${LowerArm2_yaw}"/>
+</joint>
+<joint name="shoulder_yaw2_${arm_num}" type="revolute">
+	<parent link="shoulder_yaw2_motor_${arm_num}"/>
+	<child link="lower_arm2_${arm_num}"/>
 	<origin xyz="0. 0. 0." rpy="0. 0. 0."/>
 	<axis xyz="1 0 0"/>
 	<limit lower="${j_shoulder_yaw_lower[arm_num-1]}" upper="${j_shoulder_yaw_upper[arm_num-1]}" effort="${motor_effort}" velocity="${motor_velocity}"/>
 </joint>
-<joint name="shoulder_pitch_stator_${arm_num}" type="fixed">
-	<parent link="shoulder_roll_motor_${arm_num}"/>
-	<child link="shoulder_pitch_motor_${arm_num}"/>
-	<origin xyz="${ShoulderPitch_Ox} ${ShoulderPitch_Oy} ${ShoulderPitch_Oz}" rpy="${ShoulderPitch_roll} ${ShoulderPitch_pitch} ${ShoulderPitch_yaw}"/>
-</joint>
-<!-- arm pitch 1 -->
-<joint name="shoulder_pitch_${arm_num}" type="revolute">
-	<parent link="shoulder_pitch_motor_${arm_num}"/>
-	<child link="lower_arm_${arm_num}"/>
-	<origin xyz="${LowerArm_Ox} ${LowerArm_Oy} ${LowerArm_Oz}" rpy="${LowerArm_roll} ${LowerArm_pitch} ${LowerArm_yaw}"/>
-	<axis xyz="0 0 1"/>
-	<limit lower="${j_pitch_1_lower[arm_num-1]}" upper="${j_pitch_1_upper[arm_num-1]}" effort="${motor_effort}" velocity="${motor_velocity}"/>
-</joint>
 <joint name="elbow_pitch_stator_${arm_num}" type="fixed">
-	<parent link="lower_arm_${arm_num}"/>
+	<parent link="lower_arm2_${arm_num}"/>
 	<child link="elbow_pitch_motor_${arm_num}"/>
 	<origin xyz="${ElbowPitch_Ox} ${ElbowPitch_Oy} ${ElbowPitch_Oz}" rpy="${ElbowPitch_roll} ${ElbowPitch_pitch} ${ElbowPitch_yaw}"/>

File: cetc_sat_urdf/urdf/parts/inertial_properties.urdf.xacro (robot description, xacro)
@@ -10,5 +10,6 @@
         <xacro:property name="lower_leg_mass" value="${inertial_props['lower_leg_mass'][id]}"/>
         <xacro:property name="upper_arm_mass" value="${inertial_props['upper_arm_mass'][id]}"/>
-        <xacro:property name="lower_arm_mass" value="${inertial_props['lower_arm_mass'][id]}"/>
+        <xacro:property name="lower_arm1_mass" value="${inertial_props['lower_arm1_mass'][id]}"/>
+        <xacro:property name="lower_arm2_mass" value="${inertial_props['lower_arm2_mass'][id]}"/>
         <xacro:property name="ball_mass" value="${inertial_props['ball_mass'][id]}"/>
         <xacro:property name="motorA_mass" value="${inertial_props['motorA_mass'][id]}"/>
@@ -22,5 +23,6 @@
         <xacro:property name="lower_leg_mass" value="${inertial_props['lower_leg_mass']}"/>
         <xacro:property name="upper_arm_mass" value="${inertial_props['upper_arm_mass']}"/>
-        <xacro:property name="lower_arm_mass" value="${inertial_props['lower_arm_mass']}"/>
+        <xacro:property name="lower_arm1_mass" value="${inertial_props['lower_arm1_mass']}"/>
+        <xacro:property name="lower_arm2_mass" value="${inertial_props['lower_arm2_mass']}"/>
         <xacro:property name="ball_mass" value="${inertial_props['ball_mass']}"/>
         <xacro:property name="motorA_mass" value="${inertial_props['motorA_mass']}"/>
@@ -70,10 +72,16 @@
     <xacro:property name="UpperArm_zz" value="${1/3 * upper_arm_mass * (upper_arm_width * upper_arm_width + upper_arm_length * upper_arm_length)}"/>
     <!-- Lower Arm -->
-    <xacro:property name="LowerArm_xx" value="${1/3 * lower_arm_mass * (lower_arm_width * lower_arm_width + lower_arm_height * lower_arm_height)}"/>
-    <xacro:property name="LowerArm_xy" value="0.0"/>
-    <xacro:property name="LowerArm_xz" value="0.0"/>
-    <xacro:property name="LowerArm_yy" value="${1/3 * lower_arm_mass * (lower_arm_length * lower_arm_length + lower_arm_height * lower_arm_height)}"/>
-    <xacro:property name="LowerArm_yz" value="0.0"/>
-    <xacro:property name="LowerArm_zz" value="${1/3 * lower_arm_mass * (lower_arm_width * lower_arm_width + lower_arm_length * lower_arm_length)}"/>
+    <xacro:property name="LowerArm1_xx" value="${1/3 * lower_arm1_mass * (lower_arm1_width * lower_arm1_width + lower_arm1_height * lower_arm1_height)}"/>
+    <xacro:property name="LowerArm1_xy" value="0.0"/>
+    <xacro:property name="LowerArm1_xz" value="0.0"/>
+    <xacro:property name="LowerArm1_yy" value="${1/3 * lower_arm1_mass * (lower_arm1_length * lower_arm1_length + lower_arm1_height * lower_arm1_height)}"/>
+    <xacro:property name="LowerArm1_yz" value="0.0"/>
+    <xacro:property name="LowerArm1_zz" value="${1/3 * lower_arm1_mass * (lower_arm1_width * lower_arm1_width + lower_arm1_length * lower_arm1_length)}"/>
+    <xacro:property name="LowerArm2_xx" value="${1/3 * lower_arm2_mass * (lower_arm2_width * lower_arm2_width + lower_arm2_height * lower_arm2_height)}"/>
+    <xacro:property name="LowerArm2_xy" value="0.0"/>
+    <xacro:property name="LowerArm2_xz" value="0.0"/>
+    <xacro:property name="LowerArm2_yy" value="${1/3 * lower_arm2_mass * (lower_arm2_length * lower_arm2_length + lower_arm2_height * lower_arm2_height)}"/>
+    <xacro:property name="LowerArm2_yz" value="0.0"/>
+    <xacro:property name="LowerArm2_zz" value="${1/3 * lower_arm2_mass * (lower_arm2_width * lower_arm2_width + lower_arm2_length * lower_arm2_length)}"/>
     <!-- Ball (hollow sphere) -->
     <xacro:property name="Ball_xx" value="${2/3 * ball_mass * ball_radius * ball_radius}"/>

File: cetc_sat_urdf/urdf/parts/kinematics_properties.urdf.xacro (robot description, xacro)
@@ -17,7 +17,10 @@
         <xacro:property name="upper_arm_width" value="${kin_props['upper_arm_width'][id]}"/>
         <xacro:property name="upper_arm_height" value="${kin_props['upper_arm_height'][id]}"/>
-        <xacro:property name="lower_arm_length" value="${kin_props['lower_arm_length'][id]}"/>
-        <xacro:property name="lower_arm_width" value="${kin_props['lower_arm_width'][id]}"/>
-        <xacro:property name="lower_arm_height" value="${kin_props['lower_arm_height'][id]}"/>
+        <xacro:property name="lower_arm1_length" value="${kin_props['lower_arm1_length'][id]}"/>
+        <xacro:property name="lower_arm1_width" value="${kin_props['lower_arm1_width'][id]}"/>
+        <xacro:property name="lower_arm1_height" value="${kin_props['lower_arm1_height'][id]}"/>
+        <xacro:property name="lower_arm2_length" value="${kin_props['lower_arm2_length'][id]}"/>
+        <xacro:property name="lower_arm2_width" value="${kin_props['lower_arm2_width'][id]}"/>
+        <xacro:property name="lower_arm2_height" value="${kin_props['lower_arm2_height'][id]}"/>
         <xacro:property name="ball_radius" value="${kin_props['ball_radius'][id]}"/>
         <xacro:property name="pelvis_length" value="${kin_props['pelvis_length'][id]}"/>
@@ -39,7 +42,10 @@
         <xacro:property name="upper_arm_width" value="${kin_props['upper_arm_width']}"/>
         <xacro:property name="upper_arm_height" value="${kin_props['upper_arm_height']}"/>
-        <xacro:property name="lower_arm_length" value="${kin_props['lower_arm_length']}"/>
-        <xacro:property name="lower_arm_width" value="${kin_props['lower_arm_width']}"/>
-        <xacro:property name="lower_arm_height" value="${kin_props['lower_arm_height']}"/>
+        <xacro:property name="lower_arm1_length" value="${kin_props['lower_arm1_length']}"/>
+        <xacro:property name="lower_arm1_width" value="${kin_props['lower_arm1_width']}"/>
+        <xacro:property name="lower_arm1_height" value="${kin_props['lower_arm1_height']}"/>
+        <xacro:property name="lower_arm2_length" value="${kin_props['lower_arm2_length']}"/>
+        <xacro:property name="lower_arm2_width" value="${kin_props['lower_arm2_width']}"/>
+        <xacro:property name="lower_arm2_height" value="${kin_props['lower_arm2_height']}"/>
         <xacro:property name="ball_radius" value="${kin_props['ball_radius']}"/>
         <xacro:property name="pelvis_length" value="${kin_props['pelvis_length']}"/>
@@ -106,11 +112,17 @@
     <xacro:property name="ShoulderPitch_pitch" value="0.0"/>
     <xacro:property name="ShoulderPitch_yaw" value="0.0"/>
-    <xacro:property name="LowerArm_Ox" value="0.0"/>
-    <xacro:property name="LowerArm_Oy" value="0.0"/>
-    <xacro:property name="LowerArm_Oz" value="0.0"/>
-    <xacro:property name="LowerArm_roll" value="0.0"/>
-    <xacro:property name="LowerArm_pitch" value="0.0"/>
-    <xacro:property name="LowerArm_yaw" value="${-PI_2}"/>
-    <xacro:property name="ElbowPitch_Ox" value="${lower_arm_length}"/>
+    <xacro:property name="LowerArm1_Ox" value="0.0"/>
+    <xacro:property name="LowerArm1_Oy" value="0.0"/>
+    <xacro:property name="LowerArm1_Oz" value="0.0"/>
+    <xacro:property name="LowerArm1_roll" value="0.0"/>
+    <xacro:property name="LowerArm1_pitch" value="0.0"/>
+    <xacro:property name="LowerArm1_yaw" value="${-PI_2}"/>
+    <xacro:property name="LowerArm2_Ox" value="${lower_arm1_length}"/>
+    <xacro:property name="LowerArm2_Oy" value="0.0"/>
+    <xacro:property name="LowerArm2_Oz" value="0.0"/>
+    <xacro:property name="LowerArm2_roll" value="0.0"/>
+    <xacro:property name="LowerArm2_pitch" value="0.0"/>
+    <xacro:property name="LowerArm2_yaw" value="0.0"/>
+    <xacro:property name="ElbowPitch_Ox" value="${lower_arm2_length}"/>
     <xacro:property name="ElbowPitch_Oy" value="0.0"/>
     <xacro:property name="ElbowPitch_Oz" value="0.0"/>
