Commit message: joints and params configuration

File: cetc_sat_urdf/urdf/parts/cetc_sat_arm.urdf.xacro (robot description, xacro)
@@ -49,5 +49,5 @@
 	<inertial>
 		<origin xyz="0.0 0.0 0.0"/>
-		<mass value="${upper_arm_mass}"/>
+		<mass value="${lower_arm_mass}"/>
 		<inertia ixx="${LowerArm_xx}" ixy="${LowerArm_xy}" ixz="${LowerArm_xz}" iyy="${LowerArm_xx}" iyz="${LowerArm_yz}" izz="${LowerArm_zz}"/>
 	</inertial>
@@ -85,14 +85,14 @@
 	</collision>
 </link>
-<link name="upper_arm_${arm_num}">
-	<inertial>
-		<origin xyz="0.0 0.0 0.0"/>
-		<mass value="${lower_arm_mass}"/>
-		<inertia ixx="${UpperArm_xx}" ixy="${UpperArm_xy}" ixz="${UpperArm_xz}" iyy="${UpperArm_xx}" iyz="${UpperArm_yz}" izz="${UpperArm_zz}"/>
-	</inertial>
-	<visual>
-		<origin xyz="${upper_arm_length / 2} 0.0 0.0"  rpy="0.0 0.0 0.0"/>
-		<geometry>
-			<box size="${upper_arm_length} ${upper_arm_width} ${upper_arm_height}"/>
+<link name="upper_arm1_${arm_num}">
+	<inertial>
+		<origin xyz="0.0 0.0 0.0"/>
+		<mass value="${upper_arm1_mass}"/>
+		<inertia ixx="${UpperArm1_xx}" ixy="${UpperArm1_xy}" ixz="${UpperArm1_xz}" iyy="${UpperArm1_xx}" iyz="${UpperArm1_yz}" izz="${UpperArm1_zz}"/>
+	</inertial>
+	<visual>
+		<origin xyz="${upper_arm1_length / 2} 0.0 0.0"  rpy="0.0 0.0 0.0"/>
+		<geometry>
+			<box size="${upper_arm1_length} ${upper_arm1_width} ${upper_arm1_height}"/>
 		</geometry>
 		<material name="dark_grey"/>
@@ -101,5 +101,45 @@
 		<origin xyz="${lower_arm_length / 2} 0.0 0.0"  rpy="0.0 0.0 0.0"/>
 		<geometry>
-			<box size="${upper_arm_length} ${upper_arm_width} ${upper_arm_height}"/>
+			<box size="${upper_arm1_length} ${upper_arm1_width} ${upper_arm1_height}"/>
+		</geometry>
+	</collision>
+</link>
+<link name="wrist_pitch_motor_${arm_num}">
+	<inertial>
+		<origin xyz="0.0 0.0 0.0"/>
+		<mass value="${motorA_mass}"/>
+		<inertia ixx="${MotorA_xx}" ixy="${MotorA_xy}" ixz="${MotorA_xz}" iyy="${MotorA_yy}" iyz="${MotorA_yz}" izz="${MotorA_zz}"/>
+	</inertial>
+	<visual>
+		<origin xyz="0.0 0.0 0.0"  rpy="0.0 0.0 0.0"/>
+	  	<geometry>
+	 		<cylinder radius="${cylinder_radius / 2}" length="${cylinder_length / 2}"/>
+	  	</geometry>
+  		<material name="dark_grey"/>
+	</visual>
+	<collision>
+		<origin xyz="0.0 0.0 0.0"  rpy="0.0 0.0 0.0"/>
+		<geometry>
+			<cylinder radius="${cylinder_radius}" length="${cylinder_length}"/>
+		</geometry>
+	</collision>
+</link>
+<link name="upper_arm2_${arm_num}">
+	<inertial>
+		<origin xyz="0.0 0.0 0.0"/>
+		<mass value="${upper_arm2_mass}"/>
+		<inertia ixx="${UpperArm2_xx}" ixy="${UpperArm2_xy}" ixz="${UpperArm2_xz}" iyy="${UpperArm2_xx}" iyz="${UpperArm2_yz}" izz="${UpperArm2_zz}"/>
+	</inertial>
+	<visual>
+		<origin xyz="${upper_arm2_length / 2} 0.0 0.0"  rpy="0.0 0.0 0.0"/>
+		<geometry>
+			<box size="${upper_arm2_length} ${upper_arm2_width} ${upper_arm2_height}"/>
+		</geometry>
+		<material name="dark_grey"/>
+	</visual>
+	<collision>
+		<origin xyz="${upper_arm1_length / 2} 0.0 0.0"  rpy="0.0 0.0 0.0"/>
+		<geometry>
+			<box size="${upper_arm2_length} ${upper_arm2_width} ${upper_arm2_height}"/>
 		</geometry>
 	</collision>
@@ -115,5 +155,5 @@
 		<origin xyz="0.0 0.0 0.0"  rpy="0.0 0.0 0.0"/>
 	  	<geometry>
-	 		<cylinder radius="${cylinder_radius}" length="${cylinder_length}"/>
+	 		<cylinder radius="${cylinder_radius}" length="${cylinder_length / 6}"/>
 	  	</geometry>
   		<material name="dark_grey"/>
@@ -160,12 +200,24 @@
 <joint name="elbow_pitch_${arm_num}" type="revolute">
 	<parent link="elbow_pitch_motor_${arm_num}"/>
-	<child link="upper_arm_${arm_num}"/>
-	<origin xyz="${UpperArm_Ox} ${UpperArm_Oy} ${UpperArm_Oz}" rpy="${UpperArm_roll} ${UpperArm_pitch} ${UpperArm_yaw}"/>
+	<child link="upper_arm1_${arm_num}"/>
+	<origin xyz="${UpperArm1_Ox} ${UpperArm1_Oy} ${UpperArm1_Oz}" rpy="${UpperArm1_roll} ${UpperArm1_pitch} ${UpperArm1_yaw}"/>
 	<axis xyz="0 0 1"/>
 	<limit lower="${j_pitch_2_lower[arm_num-1]}" upper="${j_pitch_2_upper[arm_num-1]}" effort="${motor_effort}" velocity="${motor_velocity}"/>
 </joint>
+<joint name="wrist_pitch_motor_${arm_num}" type="fixed">
+	<parent link="upper_arm1_${arm_num}"/>
+	<child link="wrist_pitch_motor_${arm_num}"/>
+	<origin xyz="${WristPitch_Ox} ${WristPitch_Oy} ${WristPitch_Oz}" rpy="${WristPitch_roll} ${WristPitch_pitch} ${WristPitch_yaw}"/>
+</joint>
+<joint name="wrist_pitch_joint_${arm_num}" type="revolute">
+	<parent link="wrist_pitch_motor_${arm_num}"/>
+	<child link="upper_arm2_${arm_num}"/>
+	<origin xyz="${UpperArm2_Ox} ${UpperArm2_Oy} ${UpperArm2_Oz}" rpy="${UpperArm2_roll} ${UpperArm2_pitch} ${UpperArm2_yaw}"/>
+	<axis xyz="0 0 1"/>
+	<limit lower="${j_pitch_2_lower[arm_num-1]}" upper="${j_pitch_2_upper[arm_num-1]}" effort="${motor_effort}" velocity="${motor_velocity}"/>
+</joint>
 <!-- end effector  -->
-<joint name="wrist_joint_${arm_num}" type="revolute">
-	<parent link="upper_arm_${arm_num}"/>
+<joint name="wrist_yaw_joint_${arm_num}" type="revolute">
+	<parent link="upper_arm2_${arm_num}"/>
 	<child link="wrist_${arm_num}"/>
 	<origin xyz="${EndEffector_Ox} ${EndEffector_Oy} ${EndEffector_Oz}" rpy="${EndEffector_roll} ${EndEffector_pitch} ${EndEffector_yaw}"/>

File: cetc_sat_urdf/urdf/parts/inertial_properties.urdf.xacro (robot description, xacro)
@@ -9,5 +9,6 @@
         <xacro:property name="upper_leg_mass" value="${inertial_props['upper_leg_mass'][id]}"/>
         <xacro:property name="lower_leg_mass" value="${inertial_props['lower_leg_mass'][id]}"/>
-        <xacro:property name="upper_arm_mass" value="${inertial_props['upper_arm_mass'][id]}"/>
+        <xacro:property name="upper_arm1_mass" value="${inertial_props['upper_arm1_mass'][id]}"/>
+        <xacro:property name="upper_arm2_mass" value="${inertial_props['upper_arm2_mass'][id]}"/>
         <xacro:property name="lower_arm_mass" value="${inertial_props['lower_arm_mass'][id]}"/>
         <xacro:property name="ball_mass" value="${inertial_props['ball_mass'][id]}"/>
@@ -21,5 +22,6 @@
         <xacro:property name="upper_leg_mass" value="${inertial_props['upper_leg_mass']}"/>
         <xacro:property name="lower_leg_mass" value="${inertial_props['lower_leg_mass']}"/>
-        <xacro:property name="upper_arm_mass" value="${inertial_props['upper_arm_mass']}"/>
+        <xacro:property name="upper_arm1_mass" value="${inertial_props['upper_arm1_mass']}"/>
+        <xacro:property name="upper_arm2_mass" value="${inertial_props['upper_arm2_mass']}"/>
         <xacro:property name="lower_arm_mass" value="${inertial_props['lower_arm_mass']}"/>
         <xacro:property name="ball_mass" value="${inertial_props['ball_mass']}"/>
@@ -63,10 +65,16 @@
     <xacro:property name="LowerLeg_zz" value="${1/3 * lower_leg_mass * (lower_leg_width * lower_leg_width + lower_leg_length * lower_leg_length)}"/>
     <!-- Upper Arm -->
-    <xacro:property name="UpperArm_xx" value="${1/3 * upper_arm_mass * (upper_arm_width * upper_arm_width + upper_arm_height * upper_arm_height)}"/>
-    <xacro:property name="UpperArm_xy" value="0.0"/>
-    <xacro:property name="UpperArm_xz" value="0.0"/>
-    <xacro:property name="UpperArm_yy" value="${1/3 * upper_arm_mass * (upper_arm_length * upper_arm_length + upper_arm_height * upper_arm_height)}"/>
-    <xacro:property name="UpperArm_yz" value="0.0"/>
-    <xacro:property name="UpperArm_zz" value="${1/3 * upper_arm_mass * (upper_arm_width * upper_arm_width + upper_arm_length * upper_arm_length)}"/>
+    <xacro:property name="UpperArm1_xx" value="${1/3 * upper_arm1_mass * (upper_arm1_width * upper_arm1_width + upper_arm1_height * upper_arm1_height)}"/>
+    <xacro:property name="UpperArm1_xy" value="0.0"/>
+    <xacro:property name="UpperArm1_xz" value="0.0"/>
+    <xacro:property name="UpperArm1_yy" value="${1/3 * upper_arm1_mass * (upper_arm1_length * upper_arm1_length + upper_arm1_height * upper_arm1_height)}"/>
+    <xacro:property name="UpperArm1_yz" value="0.0"/>
+    <xacro:property name="UpperArm1_zz" value="${1/3 * upper_arm1_mass * (upper_arm1_width * upper_arm1_width + upper_arm1_length * upper_arm1_length)}"/>
+    <xacro:property name="UpperArm2_xx" value="${1/3 * upper_arm2_mass * (upper_arm2_width * upper_arm2_width + upper_arm2_height * upper_arm2_height)}"/>
+    <xacro:property name="UpperArm2_xy" value="0.0"/>
+    <xacro:property name="UpperArm2_xz" value="0.0"/>
+    <xacro:property name="UpperArm2_yy" value="${1/3 * upper_arm2_mass * (upper_arm2_length * upper_arm2_length + upper_arm2_height * upper_arm2_height)}"/>
+    <xacro:property name="UpperArm2_yz" value="0.0"/>
+    <xacro:property name="UpperArm2_zz" value="${1/3 * upper_arm2_mass * (upper_arm2_width * upper_arm2_width + upper_arm2_length * upper_arm2_length)}"/>
     <!-- Lower Arm -->
     <xacro:property name="LowerArm_xx" value="${1/3 * lower_arm_mass * (lower_arm_width * lower_arm_width + lower_arm_height * lower_arm_height)}"/>

File: cetc_sat_urdf/urdf/parts/kinematics_properties.urdf.xacro (robot description, xacro)
@@ -14,7 +14,10 @@
         <xacro:property name="lower_upper_leg_width" value="${kin_props['lower_leg_width'][id]}"/>
         <xacro:property name="lower_upper_leg_height" value="${kin_props['lower_leg_height'][id]}"/>
-        <xacro:property name="upper_arm_length" value="${kin_props['upper_arm_length'][id]}"/>
-        <xacro:property name="upper_arm_width" value="${kin_props['upper_arm_width'][id]}"/>
-        <xacro:property name="upper_arm_height" value="${kin_props['upper_arm_height'][id]}"/>
+        <xacro:property name="upper_arm1_length" value="${kin_props['upper_arm1_length'][id]}"/>
+        <xacro:property name="upper_arm1_width" value="${kin_props['upper_arm1_width'][id]}"/>
+        <xacro:property name="upper_arm1_height" value="${kin_props['upper_arm1_height'][id]}"/>
+        <xacro:property name="upper_arm2_length" value="${kin_props['upper_arm2_length'][id]}"/>
+        <xacro:property name="upper_arm2_width" value="${kin_props['upper_arm2_width'][id]}"/>
+        <xacro:property name="upper_arm2_height" value="${kin_props['upper_arm2_height'][id]}"/>
         <xacro:property name="lower_arm_length" value="${kin_props['lower_arm_length'][id]}"/>
         <xacro:property name="lower_arm_width" value="${kin_props['lower_arm_width'][id]}"/>
@@ -36,7 +39,10 @@
         <xacro:property name="lower_leg_width" value="${kin_props['lower_leg_width']}"/>
         <xacro:property name="lower_leg_height" value="${kin_props['lower_leg_height']}"/>
-        <xacro:property name="upper_arm_length" value="${kin_props['upper_arm_length']}"/>
-        <xacro:property name="upper_arm_width" value="${kin_props['upper_arm_width']}"/>
-        <xacro:property name="upper_arm_height" value="${kin_props['upper_arm_height']}"/>
+        <xacro:property name="upper_arm1_length" value="${kin_props['upper_arm1_length']}"/>
+        <xacro:property name="upper_arm1_width" value="${kin_props['upper_arm1_width']}"/>
+        <xacro:property name="upper_arm1_height" value="${kin_props['upper_arm1_height']}"/>
+        <xacro:property name="upper_arm2_length" value="${kin_props['upper_arm2_length']}"/>
+        <xacro:property name="upper_arm2_width" value="${kin_props['upper_arm2_width']}"/>
+        <xacro:property name="upper_arm2_height" value="${kin_props['upper_arm2_height']}"/>
         <xacro:property name="lower_arm_length" value="${kin_props['lower_arm_length']}"/>
         <xacro:property name="lower_arm_width" value="${kin_props['lower_arm_width']}"/>
@@ -118,11 +124,23 @@
     <xacro:property name="ElbowPitch_pitch" value="0.0"/>
     <xacro:property name="ElbowPitch_yaw" value="0.0"/>
-    <xacro:property name="UpperArm_Ox" value="0.0"/>
-    <xacro:property name="UpperArm_Oy" value="0.0"/>
-    <xacro:property name="UpperArm_Oz" value="0.0"/>
-    <xacro:property name="UpperArm_roll" value="0.0"/>
-    <xacro:property name="UpperArm_pitch" value="0.0"/>
-    <xacro:property name="UpperArm_yaw" value="0.0"/>
-    <xacro:property name="EndEffector_Ox" value="${upper_arm_length}"/>
+    <xacro:property name="UpperArm1_Ox" value="0.0"/>
+    <xacro:property name="UpperArm1_Oy" value="0.0"/>
+    <xacro:property name="UpperArm1_Oz" value="0.0"/>
+    <xacro:property name="UpperArm1_roll" value="0.0"/>
+    <xacro:property name="UpperArm1_pitch" value="0.0"/>
+    <xacro:property name="UpperArm1_yaw" value="0.0"/>
+    <xacro:property name="WristPitch_Ox" value="${upper_arm1_length}"/>
+	<xacro:property name="WristPitch_Oy" value="0.0"/>
+	<xacro:property name="WristPitch_Oz" value="0.0"/>
+	<xacro:property name="WristPitch_roll" value="0.0"/>
+	<xacro:property name="WristPitch_pitch" value="0.0"/>
+	<xacro:property name="WristPitch_yaw" value="0.0"/>
+	<xacro:property name="UpperArm2_Ox" value="0.0"/>
+    <xacro:property name="UpperArm2_Oy" value="0.0"/>
+    <xacro:property name="UpperArm2_Oz" value="0.0"/>
+    <xacro:property name="UpperArm2_roll" value="0.0"/>
+    <xacro:property name="UpperArm2_pitch" value="0.0"/>
+    <xacro:property name="UpperArm2_yaw" value="0.0"/>
+    <xacro:property name="EndEffector_Ox" value="${upper_arm2_length}"/>
     <xacro:property name="EndEffector_Oy" value="0.0"/>
     <xacro:property name="EndEffector_Oz" value="0.0"/>

Commit message: roll joint

File: cetc_sat_urdf/urdf/parts/cetc_sat_arm.urdf.xacro (robot description, xacro)
@@ -214,5 +214,5 @@
 	<child link="upper_arm2_${arm_num}"/>
 	<origin xyz="${UpperArm2_Ox} ${UpperArm2_Oy} ${UpperArm2_Oz}" rpy="${UpperArm2_roll} ${UpperArm2_pitch} ${UpperArm2_yaw}"/>
-	<axis xyz="0 0 1"/>
+	<axis xyz="0 1 0"/>
 	<limit lower="${j_pitch_2_lower[arm_num-1]}" upper="${j_pitch_2_upper[arm_num-1]}" effort="${motor_effort}" velocity="${motor_velocity}"/>
 </joint>

File: cetc_sat_urdf/urdf/parts/kinematics_properties.urdf.xacro (robot description, xacro)
@@ -133,5 +133,5 @@
 	<xacro:property name="WristPitch_Oy" value="0.0"/>
 	<xacro:property name="WristPitch_Oz" value="0.0"/>
-	<xacro:property name="WristPitch_roll" value="0.0"/>
+	<xacro:property name="WristPitch_roll" value="${PI_2}"/>
 	<xacro:property name="WristPitch_pitch" value="0.0"/>
 	<xacro:property name="WristPitch_yaw" value="0.0"/>
@@ -139,5 +139,5 @@
     <xacro:property name="UpperArm2_Oy" value="0.0"/>
     <xacro:property name="UpperArm2_Oz" value="0.0"/>
-    <xacro:property name="UpperArm2_roll" value="0.0"/>
+    <xacro:property name="UpperArm2_roll" value="${-PI_2}"/>
     <xacro:property name="UpperArm2_pitch" value="0.0"/>
     <xacro:property name="UpperArm2_yaw" value="0.0"/>
@@ -145,5 +145,5 @@
     <xacro:property name="EndEffector_Oy" value="0.0"/>
     <xacro:property name="EndEffector_Oz" value="0.0"/>
-    <xacro:property name="EndEffector_roll" value="0.0	"/>
+    <xacro:property name="EndEffector_roll" value="0.0"/>
     <xacro:property name="EndEffector_pitch" value="${PI_2}"/>
     <xacro:property name="EndEffector_yaw" value="0.0"/>

Commit message: colors

File: cetc_sat_urdf/urdf/parts/cetc_sat_arm.urdf.xacro (robot description, xacro)
@@ -96,5 +96,4 @@
 			<box size="${upper_arm1_length} ${upper_arm1_width} ${upper_arm1_height}"/>
 		</geometry>
-		<material name="dark_grey"/>
 	</visual>
 	<collision>
@@ -136,5 +135,4 @@
 			<box size="${upper_arm2_length} ${upper_arm2_width} ${upper_arm2_height}"/>
 		</geometry>
-		<material name="dark_grey"/>
 	</visual>
 	<collision>

Commit message: fixed inertias

File: cetc_sat_urdf/urdf/parts/cetc_sat_arm.urdf.xacro (robot description, xacro)
@@ -48,7 +48,7 @@
 <link name="lower_arm_${arm_num}">
 	<inertial>
-		<origin xyz="0.0 0.0 0.0"/>
+		<origin xyz="${lower_arm_length / 2} 0.0 0.0"/>
 		<mass value="${lower_arm_mass}"/>
-		<inertia ixx="${LowerArm_xx}" ixy="${LowerArm_xy}" ixz="${LowerArm_xz}" iyy="${LowerArm_xx}" iyz="${LowerArm_yz}" izz="${LowerArm_zz}"/>
+		<inertia ixx="${LowerArm_xx}" ixy="${LowerArm_xy}" ixz="${LowerArm_xz}" iyy="${LowerArm_yy}" iyz="${LowerArm_yz}" izz="${LowerArm_zz}"/>
 	</inertial>
 	<visual>
@@ -87,7 +87,7 @@
 <link name="upper_arm1_${arm_num}">
 	<inertial>
-		<origin xyz="0.0 0.0 0.0"/>
+		<origin xyz="${upper_arm1_length / 2} 0.0 0.0"/>
 		<mass value="${upper_arm1_mass}"/>
-		<inertia ixx="${UpperArm1_xx}" ixy="${UpperArm1_xy}" ixz="${UpperArm1_xz}" iyy="${UpperArm1_xx}" iyz="${UpperArm1_yz}" izz="${UpperArm1_zz}"/>
+		<inertia ixx="${UpperArm1_xx}" ixy="${UpperArm1_xy}" ixz="${UpperArm1_xz}" iyy="${UpperArm1_yy}" iyz="${UpperArm1_yz}" izz="${UpperArm1_zz}"/>
 	</inertial>
 	<visual>
@@ -126,7 +126,7 @@
 <link name="upper_arm2_${arm_num}">
 	<inertial>
-		<origin xyz="0.0 0.0 0.0"/>
+		<origin xyz="${upper_arm2_length / 2} 0.0 0.0"/>
 		<mass value="${upper_arm2_mass}"/>
-		<inertia ixx="${UpperArm2_xx}" ixy="${UpperArm2_xy}" ixz="${UpperArm2_xz}" iyy="${UpperArm2_xx}" iyz="${UpperArm2_yz}" izz="${UpperArm2_zz}"/>
+		<inertia ixx="${UpperArm2_xx}" ixy="${UpperArm2_xy}" ixz="${UpperArm2_xz}" iyy="${UpperArm2_yy}" iyz="${UpperArm2_yz}" izz="${UpperArm2_zz}"/>
 	</inertial>
 	<visual>
