Commit message: fixed inertias

File: cetc_sat_urdf/urdf/parts/cetc_sat_arm.urdf.xacro (robot description, xacro)
@@ -68,7 +68,7 @@
 <link name="lower_arm1_${arm_num}">
 	<inertial>
-		<origin xyz="0.0 0.0 0.0"/>
+		<origin xyz="${lower_arm1_length / 2} 0.0 0.0"/>
 		<mass value="${lower_arm1_mass}"/>
-		<inertia ixx="${LowerArm1_xx}" ixy="${LowerArm1_xy}" ixz="${LowerArm1_xz}" iyy="${LowerArm1_xx}" iyz="${LowerArm1_yz}" izz="${LowerArm1_zz}"/>
+		<inertia ixx="${LowerArm1_xx}" ixy="${LowerArm1_xy}" ixz="${LowerArm1_xz}" iyy="${LowerArm1_yy}" iyz="${LowerArm1_yz}" izz="${LowerArm1_zz}"/>
 	</inertial>
 	<visual>
@@ -87,7 +87,7 @@
 <link name="lower_arm2_${arm_num}">
 	<inertial>
-		<origin xyz="0.0 0.0 0.0"/>
+		<origin xyz="${lower_arm2_length / 2} 0.0 0.0"/>
 		<mass value="${lower_arm2_mass}"/>
-		<inertia ixx="${LowerArm2_xx}" ixy="${LowerArm2_xy}" ixz="${LowerArm2_xz}" iyy="${LowerArm2_xx}" iyz="${LowerArm2_yz}" izz="${LowerArm2_zz}"/>
+		<inertia ixx="${LowerArm2_xx}" ixy="${LowerArm2_xy}" ixz="${LowerArm2_xz}" iyy="${LowerArm2_yy}" iyz="${LowerArm2_yz}" izz="${LowerArm2_zz}"/>
 	</inertial>
 	<visual>
@@ -126,7 +126,7 @@
 <link name="upper_arm_${arm_num}">
 	<inertial>
-		<origin xyz="0.0 0.0 0.0"/>
+		<origin xyz="${upper_arm_length / 2} 0.0 0.0"/>
 		<mass value="${upper_arm_mass}"/>
-		<inertia ixx="${UpperArm_xx}" ixy="${UpperArm_xy}" ixz="${UpperArm_xz}" iyy="${UpperArm_xx}" iyz="${UpperArm_yz}" izz="${UpperArm_zz}"/>
+		<inertia ixx="${UpperArm_xx}" ixy="${UpperArm_xy}" ixz="${UpperArm_xz}" iyy="${UpperArm_yy}" iyz="${UpperArm_yz}" izz="${UpperArm_zz}"/>
 	</inertial>
 	<visual>

File: cetc_sat_urdf/urdf/parts/inertial_properties.urdf.xacro (robot description, xacro)
@@ -51,37 +51,37 @@
     <xacro:property name="Pelvis_zz" value="${1/12 * pelvis_mass * (pelvis_width * pelvis_width + pelvis_length * pelvis_length)}"/>
     <!-- Upper Leg -->
-    <xacro:property name="UpperLeg_xx" value="${1/3 * upper_leg_mass * (upper_leg_width * upper_leg_width + upper_leg_height * upper_leg_height)}"/>
+    <xacro:property name="UpperLeg_xx" value="${1/12 * upper_leg_mass * (upper_leg_width * upper_leg_width + upper_leg_height * upper_leg_height)}"/>
     <xacro:property name="UpperLeg_xy" value="0.0"/>
     <xacro:property name="UpperLeg_xz" value="0.0"/>
-    <xacro:property name="UpperLeg_yy" value="${1/3 * upper_leg_mass * (upper_leg_length * upper_leg_length + upper_leg_height * upper_leg_height)}"/>
+    <xacro:property name="UpperLeg_yy" value="${1/12 * upper_leg_mass * (upper_leg_length * upper_leg_length + upper_leg_height * upper_leg_height)}"/>
     <xacro:property name="UpperLeg_yz" value="0.0"/>
-    <xacro:property name="UpperLeg_zz" value="${1/3 * upper_leg_mass * (upper_leg_width * upper_leg_width + upper_leg_length * upper_leg_length)}"/>
+    <xacro:property name="UpperLeg_zz" value="${1/12 * upper_leg_mass * (upper_leg_width * upper_leg_width + upper_leg_length * upper_leg_length)}"/>
     <!-- Lower Leg -->
-    <xacro:property name="LowerLeg_xx" value="${1/3 * lower_leg_mass * (lower_leg_width * lower_leg_width + lower_leg_height * lower_leg_height)}"/>
+    <xacro:property name="LowerLeg_xx" value="${1/12 * lower_leg_mass * (lower_leg_width * lower_leg_width + lower_leg_height * lower_leg_height)}"/>
     <xacro:property name="LowerLeg_xy" value="0.0"/>
     <xacro:property name="LowerLeg_xz" value="0.0"/>
-    <xacro:property name="LowerLeg_yy" value="${1/3 * lower_leg_mass * (lower_leg_length * lower_leg_length + lower_leg_height * lower_leg_height)}"/>
+    <xacro:property name="LowerLeg_yy" value="${1/12 * lower_leg_mass * (lower_leg_length * lower_leg_length + lower_leg_height * lower_leg_height)}"/>
     <xacro:property name="LowerLeg_yz" value="0.0"/>
-    <xacro:property name="LowerLeg_zz" value="${1/3 * lower_leg_mass * (lower_leg_width * lower_leg_width + lower_leg_length * lower_leg_length)}"/>
+    <xacro:property name="LowerLeg_zz" value="${1/12 * lower_leg_mass * (lower_leg_width * lower_leg_width + lower_leg_length * lower_leg_length)}"/>
     <!-- Upper Arm -->
-    <xacro:property name="UpperArm_xx" value="${1/3 * upper_arm_mass * (upper_arm_width * upper_arm_width + upper_arm_height * upper_arm_height)}"/>
+    <xacro:property name="UpperArm_xx" value="${1/12 * upper_arm_mass * (upper_arm_width * upper_arm_width + upper_arm_height * upper_arm_height)}"/>
     <xacro:property name="UpperArm_xy" value="0.0"/>
     <xacro:property name="UpperArm_xz" value="0.0"/>
-    <xacro:property name="UpperArm_yy" value="${1/3 * upper_arm_mass * (upper_arm_length * upper_arm_length + upper_arm_height * upper_arm_height)}"/>
+    <xacro:property name="UpperArm_yy" value="${1/12 * upper_arm_mass * (upper_arm_length * upper_arm_length + upper_arm_height * upper_arm_height)}"/>
     <xacro:property name="UpperArm_yz" value="0.0"/>
-    <xacro:property name="UpperArm_zz" value="${1/3 * upper_arm_mass * (upper_arm_width * upper_arm_width + upper_arm_length * upper_arm_length)}"/>
+    <xacro:property name="UpperArm_zz" value="${1/12 * upper_arm_mass * (upper_arm_width * upper_arm_width + upper_arm_length * upper_arm_length)}"/>
     <!-- Lower Arm -->
-    <xacro:property name="LowerArm1_xx" value="${1/3 * lower_arm1_mass * (lower_arm1_width * lower_arm1_width + lower_arm1_height * lower_arm1_height)}"/>
+    <xacro:property name="LowerArm1_xx" value="${1/12 * lower_arm1_mass * (lower_arm1_width * lower_arm1_width + lower_arm1_height * lower_arm1_height)}"/>
     <xacro:property name="LowerArm1_xy" value="0.0"/>
     <xacro:property name="LowerArm1_xz" value="0.0"/>
-    <xacro:property name="LowerArm1_yy" value="${1/3 * lower_arm1_mass * (lower_arm1_length * lower_arm1_length + lower_arm1_height * lower_arm1_height)}"/>
+    <xacro:property name="LowerArm1_yy" value="${1/12 * lower_arm1_mass * (lower_arm1_length * lower_arm1_length + lower_arm1_height * lower_arm1_height)}"/>
     <xacro:property name="LowerArm1_yz" value="0.0"/>
-    <xacro:property name="LowerArm1_zz" value="${1/3 * lower_arm1_mass * (lower_arm1_width * lower_arm1_width + lower_arm1_length * lower_arm1_length)}"/>
-    <xacro:property name="LowerArm2_xx" value="${1/3 * lower_arm2_mass * (lower_arm2_width * lower_arm2_width + lower_arm2_height * lower_arm2_height)}"/>
+    <xacro:property name="LowerArm1_zz" value="${1/12 * lower_arm1_mass * (lower_arm1_width * lower_arm1_width + lower_arm1_length * lower_arm1_length)}"/>
+    <xacro:property name="LowerArm2_xx" value="${1/12 * lower_arm2_mass * (lower_arm2_width * lower_arm2_width + lower_arm2_height * lower_arm2_height)}"/>
     <xacro:property name="LowerArm2_xy" value="0.0"/>
     <xacro:property name="LowerArm2_xz" value="0.0"/>
-    <xacro:property name="LowerArm2_yy" value="${1/3 * lower_arm2_mass * (lower_arm2_length * lower_arm2_length + lower_arm2_height * lower_arm2_height)}"/>
+    <xacro:property name="LowerArm2_yy" value="${1/12 * lower_arm2_mass * (lower_arm2_length * lower_arm2_length + lower_arm2_height * lower_arm2_height)}"/>
     <xacro:property name="LowerArm2_yz" value="0.0"/>
-    <xacro:property name="LowerArm2_zz" value="${1/3 * lower_arm2_mass * (lower_arm2_width * lower_arm2_width + lower_arm2_length * lower_arm2_length)}"/>
+    <xacro:property name="LowerArm2_zz" value="${1/12 * lower_arm2_mass * (lower_arm2_width * lower_arm2_width + lower_arm2_length * lower_arm2_length)}"/>
     <!-- Ball (hollow sphere) -->
     <xacro:property name="Ball_xx" value="${2/3 * ball_mass * ball_radius * ball_radius}"/>

Commit message: reduced wrist length

File: cetc_sat_urdf/urdf/parts/cetc_sat_arm.urdf.xacro (robot description, xacro)
@@ -154,12 +154,12 @@
 		<origin xyz="0.0 0.0 0.0"  rpy="0.0 0.0 0.0"/>
 	  	<geometry>
-	 		<cylinder radius="${cylinder_radius}" length="${cylinder_length}"/>
-	  	</geometry>
-  		<material name="dark_grey"/>
-	</visual>
-	<collision>
-		<origin xyz="0.0 0.0 0.0"  rpy="0.0 0.0 0.0"/>
-	  	<geometry>
-	 		<cylinder radius="${cylinder_radius}" length="${cylinder_length}"/>
+	 		<cylinder radius="${cylinder_radius}" length="${cylinder_length / 6}"/>
+	  	</geometry>
+  		<material name="dark_grey"/>
+	</visual>
+	<collision>
+		<origin xyz="0.0 0.0 0.0"  rpy="0.0 0.0 0.0"/>
+	  	<geometry>
+	 		<cylinder radius="${cylinder_radius}" length="${cylinder_length / 6}"/>
 	  	</geometry>
   		<material name="dark_grey"/>
