Commit message: fix limits again

File: kyon_urdf/urdf/parts/kyon_arm.urdf.xacro (robot description, xacro)
@@ -117,5 +117,5 @@
 	<origin xyz="${ShoulderYaw_Ox} ${rot * ShoulderYaw_Oy} ${ShoulderYaw_Oz}" rpy="${rot * ShoulderYaw_roll} ${ShoulderYaw_pitch} ${ShoulderYaw_yaw}"/>
 	<axis xyz="0 0 -1"/>
-	<limit lower="${j_shoulder_yaw_lower[arm_num-1]}" upper="${j_shoulder_yaw_upper[arm_num-1]}" effort="${motorB_effort}" velocity="${motorB_velocity}"/>
+	<limit lower="${j_shoulder_yaw_lower[arm_num-1]}" upper="${j_shoulder_yaw_upper[arm_num-1]}" effort="${motorC_effort}" velocity="${motorC_velocity}"/>
 </joint>
 <!-- arm pitch 1 -->
@@ -125,5 +125,5 @@
 	<origin xyz="${ShoulderPitch_Ox} ${ShoulderPitch_Oy} ${ShoulderPitch_Oz}" rpy="${ShoulderPitch_roll} ${ShoulderPitch_pitch} ${ShoulderPitch_yaw + rot * PI_2}"/>
 	<axis xyz="0 0 1"/>
-	<limit lower="${j_pitch_1_lower[arm_num-1]}" upper="${j_pitch_1_upper[arm_num-1]}" effort="${motorC_effort}" velocity="${motorC_velocity}"/>
+	<limit lower="${j_pitch_1_lower[arm_num-1]}" upper="${j_pitch_1_upper[arm_num-1]}" effort="${motorB_effort}" velocity="${motorB_velocity}"/>
 </joint>
 <joint name="elbow_pitch_${arm_num}" type="revolute">
@@ -132,5 +132,5 @@
 	<origin xyz="${ElbowPitch_Ox} ${ElbowPitch_Oy} ${ElbowPitch_Oz}" rpy="${ElbowPitch_roll} ${ElbowPitch_pitch} ${ElbowPitch_yaw}"/>
 	<axis xyz="0 0 -1"/>
-	<limit lower="${j_pitch_1_lower[arm_num-1]}" upper="${j_pitch_1_upper[arm_num-1]}" effort="${motorC_effort}" velocity="${motorC_velocity}"/>
+	<limit lower="${j_pitch_2_lower[arm_num-1]}" upper="${j_pitch_2_upper[arm_num-1]}" effort="${motorC_effort}" velocity="${motorC_velocity}"/>
 </joint>
 <joint name="wrist_pitch_${arm_num}" type="revolute">
@@ -139,5 +139,5 @@
 	<origin xyz="${WristPitch_Ox} ${WristPitch_Oy} ${WristPitch_Oz}" rpy="${WristPitch_roll} ${WristPitch_pitch} ${WristPitch_yaw}"/>
 	<axis xyz="0 0 -1"/>
-	<limit lower="${j_pitch_2_lower[arm_num-1]}" upper="${j_pitch_2_upper[arm_num-1]}" effort="${motorD_effort}" velocity="${motorD_velocity}"/>
+	<limit lower="${j_wrist_pitch_lower[arm_num-1]}" upper="${j_wrist_pitch_upper[arm_num-1]}" effort="${motorD_effort}" velocity="${motorD_velocity}"/>
 </joint>
 <joint name="wrist_yaw_${arm_num}" type="revolute">
@@ -146,5 +146,5 @@
 	<origin xyz="${WristYaw_Ox} ${WristYaw_Oy} ${WristYaw_Oz}" rpy="${WristYaw_roll} ${WristYaw_pitch} ${WristYaw_yaw}"/>
 	<axis xyz="0 0 1"/>
-	<limit lower="${j_pitch_2_lower[arm_num-1]}" upper="${j_pitch_2_upper[arm_num-1]}" effort="${motorD_effort}" velocity="${motorD_velocity}"/>
+	<limit lower="${j_wrist_yaw_lower[arm_num-1]}" upper="${j_wrist_yaw_upper[arm_num-1]}" effort="${motorD_effort}" velocity="${motorD_velocity}"/>
 </joint>
 <xacro:if value="${ADD_DAGANA}">

File: kyon_urdf/urdf/parts/limits.urdf.xacro (robot description, xacro)
@@ -35,5 +35,5 @@
 <xacro:property name="motorC_velocity" value="4.6"/>
 <xacro:property name="motorD_velocity" value="14"/>
-<xacro:property name="motorWheel_velocity" value="20"/>
+<xacro:property name="motorWheel_velocity" value="30"/>
 <!-- Motor effort -->
 <xacro:property name="motorA_effort" value="185"/>
