Commit message: corrected pelvis to shoulder transformation

File: kyon_urdf/urdf/parts/kinematics_properties.urdf.xacro (robot description, xacro)
@@ -61,7 +61,7 @@
     <xacro:property name="Wheel_yaw" value="0.0"/>
     <!-- Arms -->
-    <xacro:property name="ShoulderYaw_Ox" value="${270.00 * mTomm}"/>
-    <xacro:property name="ShoulderYaw_Oy" value="${102.996 * mTomm}"/>
-    <xacro:property name="ShoulderYaw_Oz" value="${187.217 * mTomm}"/>
+    <xacro:property name="ShoulderYaw_Ox" value="${280.00 * mTomm}"/>
+    <xacro:property name="ShoulderYaw_Oy" value="${96.6072 * mTomm}"/>
+    <xacro:property name="ShoulderYaw_Oz" value="${203.559 * mTomm}"/>
     <xacro:property name="ShoulderYaw_roll" value="0.3490656"/>
     <xacro:property name="ShoulderYaw_pitch" value="0.0"/>

File: kyon_urdf/urdf/parts/limits.urdf.xacro (robot description, xacro)
@@ -6,6 +6,6 @@
 <xacro:property name="hip_pitch_lower" value="${[-2.4056, -2.3266, -2.4696, -2.3426]}"/>
 <xacro:property name="hip_pitch_upper" value="${[2.4056, 2.3266, 2.4696, 2.3426]}"/>
-<xacro:property name="knee_pitch_lower" value="${[-2.4056, -2.3266, -2.4696, -2.3426]}"/>
-<xacro:property name="knee_pitch_upper" value="${[2.4056, 2.3266, 2.4696, 2.3426]}"/>
+<xacro:property name="knee_pitch_lower" value="${[-3.4056, -3.3266, -3.4696, -3.3426]}"/>
+<xacro:property name="knee_pitch_upper" value="${[3.4056, 3.3266, 3.4696, 3.3426]}"/>
 <!-- Arms -->
 <xacro:property name="j_shoulder_yaw_lower" value="${[-3.312, -3.3458]}"/>

Commit message: fixed coarse visual mesh being used for collison

File: kyon_urdf/urdf/parts/kinematics_properties.urdf.xacro (robot description, xacro)
@@ -24,4 +24,6 @@
     <xacro:property name="pelvis_width" value="${kin_props['pelvis_width']}"/>
     <xacro:property name="pelvis_height" value="${kin_props['pelvis_height']}"/>
+    <xacro:property name="wheel_radius" value="${kin_props['wheel_radius']}"/>
+    <xacro:property name="wheel_depth" value="${kin_props['wheel_depth']}"/>
     <!-- Compound properties (i.e. based on the props parsed from the yaml) -->
     <!-- Origin -->

File: kyon_urdf/urdf/parts/kyon_leg.urdf.xacro (robot description, xacro)
@@ -149,8 +149,11 @@
             <collision>
                 <origin xyz="0 0 0" rpy="0 0 0" />
-                <geometry>
+				<geometry>
+					<cylinder radius="${wheel_radius}" length="${wheel_depth}"/>
+				</geometry>
+                <!-- <geometry>
                     <mesh filename="${MESH_PATH}/collision/mesh_wheel23.stl"
                         scale="0.001 0.001 ${mirror*0.001}" />
-                </geometry>
+                </geometry> -->
                 <material name="black" />
             </collision>

Commit message: fixed coarse mesh being used for wheel collision

File: kyon_urdf/urdf/parts/kinematics_properties.urdf.xacro (robot description, xacro)
@@ -24,4 +24,6 @@
     <xacro:property name="pelvis_width" value="${kin_props['pelvis_width']}"/>
     <xacro:property name="pelvis_height" value="${kin_props['pelvis_height']}"/>
+    <xacro:property name="wheel_radius" value="${kin_props['wheel_radius']}"/>
+    <xacro:property name="wheel_depth" value="${kin_props['wheel_depth']}"/>
     <!-- Compound properties (i.e. based on the props parsed from the yaml) -->
     <!-- Origin -->

Commit message: dagana upd

File: kyon_urdf/urdf/parts/kinematics_properties.urdf.xacro (robot description, xacro)
@@ -104,5 +104,5 @@
     <xacro:property name="DaganaBase_roll" value="0.0"/>
     <xacro:property name="DaganaBase_pitch" value="0.0"/>
-    <xacro:property name="DaganaBase_yaw" value="0.0"/>
+    <xacro:property name="DaganaBase_yaw" value="${-PI_2}"/>
     <xacro:property name="DaganaClamp_Ox" value="${36.1625 * mmTom}"/>
     <xacro:property name="DaganaClamp_Oy" value="${16.000 * mmTom}"/>

File: kyon_urdf/urdf/parts/kyon_dagana.urdf.xacro (robot description, xacro)
@@ -58,5 +58,5 @@
     <parent link="${parent}"/>
     <child link="dagana_${arm_num}_base"/>
-    <origin xyz="${DaganaBase_Ox} ${DaganaBase_Oy} ${DaganaBase_Oz}" rpy="${DaganaBase_roll} ${DaganaBase_pitch} ${DaganaBase_yaw}"/>
+    <origin xyz="${DaganaBase_Ox} ${DaganaBase_Oy} ${DaganaBase_Oz}" rpy="${DaganaBase_roll} ${DaganaBase_pitch} ${DaganaBase_yaw * (1.0 if arm_num == 1 else -1)}"/>
 </joint>
 <joint name="dagana_${arm_num}_clamp_joint" type="revolute">
@@ -64,5 +64,5 @@
     <child link="dagana_${arm_num}_claw"/>
     <origin xyz="${DaganaClamp_Ox} ${DaganaClamp_Oy} ${DaganaClamp_Oz}" rpy="${DaganaClamp_roll} ${DaganaClamp_pitch} ${DaganaClamp_yaw}"/>
-    <axis xyz="0 0 1"/>
+    <axis xyz="0 0 -1"/>
     <limit lower="${dagana_lower[arm_num-1]}" upper="${dagana_upper[arm_num-1]}" effort="${motorD_effort}" velocity="${motorD_velocity}"/>
 </joint>

File: kyon_urdf/urdf/parts/limits.urdf.xacro (robot description, xacro)
@@ -28,6 +28,6 @@
 <xacro:property name="j_pitch_2_torque" value="${[147.00, 147.00 ]}"/>
 <!-- Dagana -->
-<xacro:property name="dagana_lower" value="${[-3.4056, -3.3266]}"/>
-<xacro:property name="dagana_upper" value="${[3.4056, 3.3266]}"/>
+<xacro:property name="dagana_lower" value="${[0, 0]}"/>
+<xacro:property name="dagana_upper" value="${[1.2, 1.2]}"/>
 <!-- Motor velocities -->
 <xacro:property name="motorA_velocity" value="7.6"/>
