Commit message: updated effort and velocity limits

File: kyon_urdf/urdf/parts/limits.urdf.xacro (robot description, xacro)
@@ -25,6 +25,12 @@
 <xacro:property name="dagana_upper" value="${[3.4056, 3.3266]}"/>
 <!-- Motor velocities -->
-<xacro:property name="motor_velocity" value="15.5"/>
+<xacro:property name="motorA_velocity" value="7.6"/>
+<xacro:property name="motorB_velocity" value="3.8"/>
+<xacro:property name="motorC_velocity" value="4.6"/>
+<xacro:property name="motorD_velocity" value="14"/>
 <!-- Motor effort -->
-<xacro:property name="motor_effort" value="132"/>
+<xacro:property name="motorA_effort" value="185"/>
+<xacro:property name="motorA_effort" value="146"/>
+<xacro:property name="motorA_effort" value="122"/>
+<xacro:property name="motorA_effort" value="25"/>
 </robot>

Commit message: continuous wheels

File: kyon_urdf/urdf/parts/limits.urdf.xacro (robot description, xacro)
@@ -8,4 +8,6 @@
 <xacro:property name="knee_pitch_lower" value="${[-3.4056, -3.3266, -3.4696, -3.3426]}"/>
 <xacro:property name="knee_pitch_upper" value="${[3.4056, 3.3266, 3.4696, 3.3426]}"/>
+<xacro:property name="ankle_yaw_lower" value="${[3.4056, 3.3266, 3.4696, 3.3426]}"/>
+<xacro:property name="ankle_yaw_upper" value="${[3.4056, 3.3266, 3.4696, 3.3426]}"/>
 <!-- Arms -->
 <xacro:property name="j_shoulder_yaw_lower" value="${[-3.312, -3.3458]}"/>

File: kyon_urdf/urdf/parts/steering_wheel.urdf.xacro (robot description, xacro)
@@ -82,12 +82,12 @@
     <origin xyz="${AnkleYaw_Ox} ${AnkleYaw_Oy} ${AnkleYaw_Oz}" rpy="${AnkleYaw_roll} ${AnkleYaw_pitch} ${AnkleYaw_yaw}"/>
     <axis xyz="0 0 1"/>
-    <limit lower="${knee_pitch_lower[leg_num-1]}" upper="${knee_pitch_upper[leg_num-1]}" effort="${motorA_effort}" velocity="${motorA_velocity}"/>
+    <limit lower="${ankle_yaw_lower[leg_num-1]}" upper="${ankle_yaw_upper[leg_num-1]}" effort="${motorA_effort}" velocity="${motorA_velocity}"/>
 </joint>
-<joint name="wheel_joint_${leg_num}" type="revolute">
+<joint name="wheel_joint_${leg_num}" type="continuous">
     <parent link="ankle_yaw_${leg_num}_link"/>
     <child link="wheel_${leg_num}"/>
     <origin xyz="${SteeringWheel_Ox} ${SteeringWheel_Oy} ${SteeringWheel_Oz}" rpy="${SteeringWheel_roll} ${SteeringWheel_pitch} ${SteeringWheel_yaw}"/>
     <axis xyz="0 0 1"/>
-    <limit lower="-1e9" upper="1e9" effort="${motorWheel_effort}" velocity="${motorWheel_velocity}"/>
+    <limit effort="${motorWheel_effort}" velocity="${motorWheel_velocity}"/>
 </joint>
 </xacro:macro>

File: kyon_urdf/urdf/parts/wheel_leg.urdf.xacro (robot description, xacro)
@@ -52,10 +52,10 @@
     <limit lower="${knee_pitch_lower[leg_num-1]}" upper="${knee_pitch_upper[leg_num-1]}" effort="${motorA_effort}" velocity="${motorA_velocity}"/>
 </joint>
-<joint name="wheel_joint_${leg_num}" type="revolute">
+<joint name="wheel_joint_${leg_num}" type="continuous">
     <parent link="knee_pitch_${leg_num}_link"/>
     <child link="wheel_${leg_num}"/>
     <origin xyz="${Wheel_Ox} ${Wheel_Oy} ${Wheel_Oz}" rpy="${Wheel_roll} ${Wheel_pitch} ${Wheel_yaw}"/>
     <axis xyz="0 0 1"/>
-    <limit lower="-10000000" upper="10000000" effort="${motorWheel_effort}" velocity="${motorWheel_velocity}"/>
+    <limit effort="${motorWheel_effort}" velocity="${motorWheel_velocity}"/>
 </joint>
 <joint name="contact_${leg_num}_joint" type="fixed">

Commit message: typo

File: kyon_urdf/urdf/parts/limits.urdf.xacro (robot description, xacro)
@@ -8,5 +8,5 @@
 <xacro:property name="knee_pitch_lower" value="${[-3.4056, -3.3266, -3.4696, -3.3426]}"/>
 <xacro:property name="knee_pitch_upper" value="${[3.4056, 3.3266, 3.4696, 3.3426]}"/>
-<xacro:property name="ankle_yaw_lower" value="${[3.4056, 3.3266, 3.4696, 3.3426]}"/>
+<xacro:property name="ankle_yaw_lower" value="${[-3.4056, -3.3266, -3.4696, -3.3426]}"/>
 <xacro:property name="ankle_yaw_upper" value="${[3.4056, 3.3266, 3.4696, 3.3426]}"/>
 <!-- Arms -->

Commit message: hip roll and ankle limits

File: kyon_urdf/urdf/parts/limits.urdf.xacro (robot description, xacro)
@@ -2,10 +2,12 @@
 <robot  xmlns:xacro="http://ros.org/wiki/xacro">
 <!-- Legs -->
-<xacro:property name="hip_roll_lower" value="${[-2.030,-2.510, -2.510 ,-2.030]}"/>
-<xacro:property name="hip_roll_upper" value="${[ 2.510, 2.030,  2.030 , 2.510]}"/>
+<xacro:property name="hip_roll_lower" value="${[-0.65,-0.65, -0.65 ,-0.65]}"/>
+<xacro:property name="hip_roll_upper" value="${[ 0.65, 0.65,  0.65 , 0.65]}"/>
 <xacro:property name="hip_pitch_lower" value="${[-2.4056, -2.3266, -2.4696, -2.3426]}"/>
 <xacro:property name="hip_pitch_upper" value="${[2.4056, 2.3266, 2.4696, 2.3426]}"/>
-<xacro:property name="knee_pitch_lower" value="${[-3.4056, -3.3266, -3.4696, -3.3426]}"/>
-<xacro:property name="knee_pitch_upper" value="${[3.4056, 3.3266, 3.4696, 3.3426]}"/>
+<xacro:property name="knee_pitch_lower" value="${[-3.2, -3.2, -3.2, -3.2]}"/>
+<xacro:property name="knee_pitch_upper" value="${[3.2, 3.2, 3.2, 3.2]}"/>
+<xacro:property name="ankle_yaw_lower" value="${[-3.0, -3.0, -3.0, -3.0]}"/>
+<xacro:property name="ankle_yaw_upper" value="${[ 3.0,  3.0,  3.0,  3.0]}"/>
 <!-- Arms -->
 <xacro:property name="j_shoulder_yaw_lower" value="${[-3.312, -3.3458]}"/>

Commit message: upd limits

File: kyon_urdf/urdf/parts/limits.urdf.xacro (robot description, xacro)
@@ -2,19 +2,23 @@
 <robot  xmlns:xacro="http://ros.org/wiki/xacro">
 <!-- Legs -->
-<xacro:property name="hip_roll_lower" value="${[-2.030,-2.510, -2.510 ,-2.030]}"/>
-<xacro:property name="hip_roll_upper" value="${[ 2.510, 2.030,  2.030 , 2.510]}"/>
+<xacro:property name="hip_roll_lower" value="${[-0.65,-0.65, -0.65 ,-0.65]}"/>
+<xacro:property name="hip_roll_upper" value="${[ 0.65, 0.65,  0.65 , 0.65]}"/>
 <xacro:property name="hip_pitch_lower" value="${[-2.4056, -2.3266, -2.4696, -2.3426]}"/>
 <xacro:property name="hip_pitch_upper" value="${[2.4056, 2.3266, 2.4696, 2.3426]}"/>
-<xacro:property name="knee_pitch_lower" value="${[-3.4056, -3.3266, -3.4696, -3.3426]}"/>
-<xacro:property name="knee_pitch_upper" value="${[3.4056, 3.3266, 3.4696, 3.3426]}"/>
-<xacro:property name="ankle_yaw_lower" value="${[-3.4056, -3.3266, -3.4696, -3.3426]}"/>
-<xacro:property name="ankle_yaw_upper" value="${[3.4056, 3.3266, 3.4696, 3.3426]}"/>
+<xacro:property name="knee_pitch_lower" value="${[-3.0, -3.0, -3.0, -3.0]}"/>
+<xacro:property name="knee_pitch_upper" value="${[3.0, 3.0, 3.0, 3.0]}"/>
+<xacro:property name="ankle_yaw_lower" value="${[-3.0, -3.0, -3.0, -3.0]}"/>
+<xacro:property name="ankle_yaw_upper" value="${[ 3.0,  3.0,  3.0,  3.0]}"/>
 <!-- Arms -->
-<xacro:property name="j_shoulder_yaw_lower" value="${[-3.312, -3.3458]}"/>
-<xacro:property name="j_shoulder_yaw_upper" value="${[3.312, 3.3458]}"/>
-<xacro:property name="j_pitch_1_lower" value="${[-3, -3]}"/>
-<xacro:property name="j_pitch_1_upper" value="${[3, 3]}"/>
-<xacro:property name="j_pitch_2_lower" value="${[-2.4056, -2.3266, -2.4696, -2.3426]}"/>
-<xacro:property name="j_pitch_2_upper" value="${[2.4056, 2.3266, 2.4696, 2.3426]}"/>
+<xacro:property name="j_shoulder_yaw_lower" value="${[-3.0, -3.0]}"/>
+<xacro:property name="j_shoulder_yaw_upper" value="${[3.0, 3.0]}"/>
+<xacro:property name="j_pitch_1_lower" value="${[-2.2, -2.2]}"/>
+<xacro:property name="j_pitch_1_upper" value="${[2.2, 2.2]}"/>
+<xacro:property name="j_pitch_2_lower" value="${[-2.8, -2.8]}"/>
+<xacro:property name="j_pitch_2_upper" value="${[2.8, 2.8]}"/>
+<xacro:property name="j_wrist_pitch_lower" value="${[-1.6, -1.6]}"/>
+<xacro:property name="j_wrist_pitch_upper" value="${[1.6, 1.6]}"/>
+<xacro:property name="j_wrist_yaw_lower" value="${[-2.7, -2.7]}"/>
+<xacro:property name="j_wrist_yaw_upper" value="${[2.7, 2.7]}"/>
 <xacro:property name="j_shoulder_velocity" value="${[3.86, 3.86 ]}"/>
 <xacro:property name="j_pitch_1_velocity" value="${[3.86, 3.86 ]}"/>

Commit message: knee limits to allow parking

File: kyon_urdf/urdf/parts/limits.urdf.xacro (robot description, xacro)
@@ -6,6 +6,6 @@
 <xacro:property name="hip_pitch_lower" value="${[-2.4056, -2.3266, -2.4696, -2.3426]}"/>
 <xacro:property name="hip_pitch_upper" value="${[2.4056, 2.3266, 2.4696, 2.3426]}"/>
-<xacro:property name="knee_pitch_lower" value="${[-3.0, -3.0, -3.0, -3.0]}"/>
-<xacro:property name="knee_pitch_upper" value="${[3.0, 3.0, 3.0, 3.0]}"/>
+<xacro:property name="knee_pitch_lower" value="${[-3.20, -3.20, -3.20, -3.20]}"/>
+<xacro:property name="knee_pitch_upper" value="${[3.20, 3.20, 3.20, 3.20]}"/>
 <xacro:property name="ankle_yaw_lower" value="${[-3.0, -3.0, -3.0, -3.0]}"/>
 <xacro:property name="ankle_yaw_upper" value="${[ 3.0,  3.0,  3.0,  3.0]}"/>
