Commit message: fix limits for wheel modules

File: kyon_urdf/urdf/parts/limits.urdf.xacro (robot description, xacro)
@@ -35,5 +35,5 @@
 <xacro:property name="motorC_velocity" value="4.6"/>
 <xacro:property name="motorD_velocity" value="14"/>
-<xacro:property name="motorWheel_velocity" value="30"/>
+<xacro:property name="motorWheel_velocity" value="24"/>
 <!-- Motor effort -->
 <xacro:property name="motorA_effort" value="185"/>
@@ -41,4 +41,4 @@
 <xacro:property name="motorC_effort" value="122"/>
 <xacro:property name="motorD_effort" value="25"/>
-<xacro:property name="motorWheel_effort" value="100"/>
+<xacro:property name="motorWheel_effort" value="25"/>
 </robot>

File: kyon_urdf/urdf/parts/steering_wheel.urdf.xacro (robot description, xacro)
@@ -82,5 +82,5 @@
     <origin xyz="${AnkleYaw_Ox} ${AnkleYaw_Oy} ${AnkleYaw_Oz}" rpy="${AnkleYaw_roll} ${AnkleYaw_pitch} ${AnkleYaw_yaw}"/>
     <axis xyz="0 0 1"/>
-    <limit lower="${ankle_yaw_lower[leg_num-1]}" upper="${ankle_yaw_upper[leg_num-1]}" effort="${motorA_effort}" velocity="${motorA_velocity}"/>
+    <limit lower="${ankle_yaw_lower[leg_num-1]}" upper="${ankle_yaw_upper[leg_num-1]}" effort="${motorC_effort}" velocity="${motorC_velocity}"/>
 </joint>
 <joint name="wheel_joint_${leg_num}" type="revolute">
