Commit message: quick fix

File: kyon_urdf/urdf/parts/wheel_leg.urdf.xacro (robot description, xacro)
@@ -55,5 +55,5 @@
     <origin xyz="${Wheel_Ox} ${Wheel_Oy} ${Wheel_Oz}" rpy="${Wheel_roll} ${Wheel_pitch} ${Wheel_yaw}"/>
     <axis xyz="0 0 1"/>
-    <limit lower="${knee_pitch_lower[leg_num-1]}" upper="${knee_pitch_upper[leg_num-1]}" effort="${motorWheel_effort}" velocity="${motorWheel_velocity}"/>
+    <limit lower="-10000000" upper="10000000" effort="${motorWheel_effort}" velocity="${motorWheel_velocity}"/>
 </joint>
 </xacro:macro>

Commit message: contact link

File: kyon_urdf/urdf/parts/wheel_leg.urdf.xacro (robot description, xacro)
@@ -39,8 +39,10 @@
 		<origin xyz="0.0 0.0 0.0"  rpy="0.0 0.0 0.0"/>
 		<geometry>
-			<mesh filename="package://kyon_urdf/meshes/collision/mesh_wheel.stl" scale="0.001 0.001 0.001"/>
+			<!--mesh filename="package://kyon_urdf/meshes/collision/mesh_wheel.stl" scale="0.001 0.001 0.001"/-->
+			<cylinder radius="0.11" length="0.045"/>
 		</geometry>
 	</collision>
 </link>
+<link name="contact_${leg_num}"/>
 <joint name="knee_pitch_${leg_num}" type="revolute">
     <parent link="${parent}"/>
@@ -57,4 +59,8 @@
     <limit lower="-10000000" upper="10000000" effort="${motorWheel_effort}" velocity="${motorWheel_velocity}"/>
 </joint>
+<joint name="contact_${leg_num}_joint" type="fixed">
+    <parent link="wheel_${leg_num}"/>
+    <child link="contact_${leg_num}"/>
+</joint>
 </xacro:macro>
 </robot>

Commit message: contact in the center of the wheel (kyon_mjx purposes)

File: kyon_urdf/urdf/parts/wheel_leg.urdf.xacro (robot description, xacro)
@@ -39,8 +39,10 @@
 		<origin xyz="0.0 0.0 0.0"  rpy="0.0 0.0 0.0"/>
 		<geometry>
-			<mesh filename="package://kyon_urdf/meshes/collision/mesh_wheel.stl" scale="0.001 0.001 0.001"/>
+			<!-- <mesh filename="package://kyon_urdf/meshes/collision/mesh_wheel.stl" scale="0.001 0.001 0.001"/> -->
+            <cylinder radius="0.11" length="0.045"/>
 		</geometry>
 	</collision>
 </link>
+<link name="contact_${leg_num}"/>
 <joint name="knee_pitch_${leg_num}" type="revolute">
     <parent link="${parent}"/>
@@ -57,4 +59,8 @@
     <limit lower="-10000000" upper="10000000" effort="${motorWheel_effort}" velocity="${motorWheel_velocity}"/>
 </joint>
+<joint name="contact_${leg_num}_joint" type="fixed">
+    <parent link="wheel_${leg_num}"/>
+    <child link="contact_${leg_num}"/>
+</joint>
 </xacro:macro>
 </robot>

Commit message: adjusted collision cylinder depth

File: kyon_urdf/urdf/parts/wheel_leg.urdf.xacro (robot description, xacro)
@@ -40,5 +40,5 @@
 		<geometry>
 			<!-- <mesh filename="${MESH_PATH}/collision/mesh_wheel.stl" scale="0.001 0.001 0.001"/> -->
-            <cylinder radius="0.11" length="0.045"/>
+            <cylinder radius="0.1066" length="0.03"/>
 		</geometry>
 	</collision>
