Commit message: linking to wrong mesh file

File: kyon_urdf/urdf/parts/kyon_leg.urdf.xacro (robot description, xacro)
@@ -142,5 +142,5 @@
                 <origin xyz="0.0 0.0 0.0" rpy="0.0 0.0 0.0" />
                 <geometry>
-                    <mesh filename="package://centauro_urdf/meshes/v2/mesh_wheel23.stl"
+                    <mesh filename="package://kyon_urdf/meshes/v2/mesh_wheel23.stl"
                         scale="0.001 0.001 ${mirror*0.001}" />
                 </geometry>
@@ -150,5 +150,5 @@
                 <origin xyz="0 0 0" rpy="0 0 0" />
                 <geometry>
-                    <mesh filename="package://centauro_urdf/meshes/v2/collision/mesh_wheel23.stl"
+                    <mesh filename="package://kyon_urdf/meshes/v2/collision/mesh_wheel23.stl"
                         scale="0.001 0.001 ${mirror*0.001}" />
                 </geometry>

Commit message: fix

File: kyon_urdf/urdf/parts/kyon_leg.urdf.xacro (robot description, xacro)
@@ -142,5 +142,5 @@
                 <origin xyz="0.0 0.0 0.0" rpy="0.0 0.0 0.0" />
                 <geometry>
-                    <mesh filename="package://kyon_urdf/meshes/v2/mesh_wheel23.stl"
+                    <mesh filename="package://kyon_urdf/meshes/mesh_wheel23.stl"
                         scale="0.001 0.001 ${mirror*0.001}" />
                 </geometry>
@@ -150,5 +150,5 @@
                 <origin xyz="0 0 0" rpy="0 0 0" />
                 <geometry>
-                    <mesh filename="package://kyon_urdf/meshes/v2/collision/mesh_wheel23.stl"
+                    <mesh filename="package://kyon_urdf/meshes/collision/mesh_wheel23.stl"
                         scale="0.001 0.001 ${mirror*0.001}" />
                 </geometry>

Commit message: added separate property for wheels

File: kyon_urdf/urdf/parts/kyon_leg.urdf.xacro (robot description, xacro)
@@ -130,5 +130,5 @@
             <origin xyz="${Wheel23_Ox} ${Wheel23_Oy} ${-mirror*Wheel23_Oz}" rpy="${Wheel23_roll} ${Wheel23_pitch} ${Wheel23_yaw}" />
             <axis xyz="0 0 ${mirror}"/>
-            <limit effort="${motor_effort}" velocity="${motor_velocity}" />  <!-- 23 Nm, 1
+            <limit effort="${motor_effort}" velocity="${wheel_motor_velocity}" />  <!-- 23 Nm, 1
             rad/s-->
         </joint>

File: kyon_urdf/urdf/parts/limits.urdf.xacro (robot description, xacro)
@@ -28,4 +28,5 @@
 	<xacro:property name="motor_velocity" value="9.3"/>
 </xacro:if>
+<xacro:property name="wheel_motor_velocity" value="60.0"/>
 <!-- Motor effort -->
 <xacro:if value="${inertial_props['gear_ratio'] == 30}">

Commit message: fixed meshes that were colliding even in homing

File: kyon_urdf/urdf/parts/kyon_leg.urdf.xacro (robot description, xacro)
@@ -22,11 +22,10 @@
   		<material name="dark_grey"/>
 	</visual>
-	<collision>
+	<!-- <collision>
 		<origin xyz="0.0 0.0 0.0"  rpy="0.0 0.0 0.0"/>
 		<geometry>
-	 		<!-- <cylinder radius="${cylinder_radius}" length="${cylinder_length}"/> -->
 			<mesh filename="${MESH_PATH}/collision/mesh_hip-roll.stl" scale="0.001 ${mirror*0.001} 0.001"/>
 		</geometry>
-	</collision>
+	</collision> -->
 </link>
 <link name="hip_pitch_${leg_num}_link">
@@ -53,5 +52,5 @@
 		<origin xyz="0.0 0.0 0.0"  rpy="0.0 0.0 0.0"/>
 		<geometry>
-			<mesh filename="${MESH_PATH}/collision/mesh_hip-pitch.stl" scale="0.001 0.001 0.001"/>
+			<mesh filename="${MESH_PATH}/collision/mesh_hip-pitch_cut.stl" scale="0.001 0.001 0.001"/>
 		</geometry>
 		<material name="kyon_orange"/>

File: kyon_urdf/urdf/parts/steering_wheel.urdf.xacro (robot description, xacro)
@@ -21,5 +21,5 @@
 		<geometry>
 	 		<!-- <cylinder radius="${cylinder_radius}" length="${cylinder_length}"/> -->
-			<mesh filename="${MESH_PATH}/collision/mesh_knee-steering.stl" scale="0.001 0.001 0.001"/>
+			<mesh filename="${MESH_PATH}/collision/mesh_knee-steering_cut.stl" scale="0.001 0.001 0.001"/>
 		</geometry>
 	</collision>
@@ -43,5 +43,5 @@
 		<geometry>
 	 		<!-- <cylinder radius="${cylinder_radius}" length="${cylinder_length}"/> -->
-			<mesh filename="${MESH_PATH}/collision/mesh_ankle-yaw.stl" scale="0.001 0.001 0.001"/>
+			<mesh filename="${MESH_PATH}/collision/mesh_ankle-yaw_cut.stl" scale="0.001 0.001 0.001"/>
 		</geometry>
 	</collision>
@@ -64,5 +64,5 @@
 		<origin xyz="0.0 0.0 0.0"  rpy="0.0 0.0 0.0"/>
 		<geometry>
-	 		<cylinder radius="0.1066" length="0.05"/>
+	 		<cylinder radius="0.1066" length="0.03"/>
 			<!-- <mesh filename="${MESH_PATH}/collision/mesh_wheel.stl" scale="0.001 0.001 0.001"/> -->
 		</geometry>
