Commit message: fixed dagana inertias

File: kyon_urdf/urdf/parts/inertial_properties.urdf.xacro (robot description, xacro)
@@ -118,4 +118,15 @@
 	<xacro:property name="SteeringWheel_yz" value="${0.0 * mm2Tom2}"/>
 	<xacro:property name="SteeringWheel_zz" value="${7.9333497e+03 * mm2Tom2}"/>
+    <!-- Wheel-->
+    <xacro:property name="Wheel_mass" value="1.2638390"/>
+	<xacro:property name="Wheel_x" value="${0.0 * mmTom}"/>
+	<xacro:property name="Wheel_y" value="${0.0 * mmTom}"/>
+	<xacro:property name="Wheel_z" value="${1.4437817e+00 * mmTom}"/>
+	<xacro:property name="Wheel_xx" value="${4.1796417e+03 * mm2Tom2}"/>
+	<xacro:property name="Wheel_xy" value="${4.4497596e-03 * mm2Tom2}"/>
+	<xacro:property name="Wheel_xz" value="${0.0000000e+00 * mm2Tom2}"/>
+	<xacro:property name="Wheel_yy" value="${4.1796381e+03 * mm2Tom2}"/>
+	<xacro:property name="Wheel_yz" value="${0.0 * mm2Tom2}"/>
+	<xacro:property name="Wheel_zz" value="${7.9333497e+03 * mm2Tom2}"/>
     <!-- Shoulder Yaw -->
     <xacro:property name="ShoulderYaw_mass" value="0.67826074"/>
@@ -173,3 +184,25 @@
     <xacro:property name="WristYaw_yz" value="${-2.5372645e-02 * mm2Tom2}"/>
     <xacro:property name="WristYaw_zz" value="${1.1802904e+02 * mm2Tom2}"/>
+    <!-- Dagana -->
+    <xacro:property name="Dagana_mass" value="0.96534359"/>
+    <xacro:property name="Dagana_x" value="${-4.2244666e+00 * mmTom}"/>
+    <xacro:property name="Dagana_y" value="${-2.7238215e+00 * mmTom}"/>
+    <xacro:property name="Dagana_z" value="${5.3670845e+01 * mmTom}"/>
+    <xacro:property name="Dagana_xx" value="${2.0957096e+03 * mm2Tom2}"/>
+    <xacro:property name="Dagana_xy" value="${-6.4554109e+01 * mm2Tom2}"/>
+    <xacro:property name="Dagana_xz" value="${4.4955881e+01 * mm2Tom2}"/>
+    <xacro:property name="Dagana_yy" value="${2.1216529e+03 * mm2Tom2}"/>
+    <xacro:property name="Dagana_yz" value="${3.7094613e+02 * mm2Tom2}"/>
+    <xacro:property name="Dagana_zz" value="${1.1572224e+03 * mm2Tom2}"/>
+    <!-- Dagana Claw -->
+    <xacro:property name="DaganaClaw_mass" value="0.25739835"/>
+    <xacro:property name="DaganaClaw_x" value="${-5.1620300e+01 * mmTom}"/>
+    <xacro:property name="DaganaClaw_y" value="${8.0601187e+00 * mmTom}"/>
+    <xacro:property name="DaganaClaw_z" value="${-3.7212096e+01 * mmTom}"/>
+    <xacro:property name="DaganaClaw_xx" value="${2.9169897e+02 * mm2Tom2}"/>
+    <xacro:property name="DaganaClaw_xy" value="${8.3015178e+00 * mm2Tom2}"/>
+    <xacro:property name="DaganaClaw_xz" value="${1.3355847e+01 * mm2Tom2}"/>
+    <xacro:property name="DaganaClaw_yy" value="${7.3268589e+02 * mm2Tom2}"/>
+    <xacro:property name="DaganaClaw_yz" value="${-2.1083033e+00 * mm2Tom2}"/>
+    <xacro:property name="DaganaClaw_zz" value="${5.1112938e+02 * mm2Tom2}"/>
 </robot>

File: kyon_urdf/urdf/parts/kyon_dagana.urdf.xacro (robot description, xacro)
@@ -5,7 +5,7 @@
 <link name="dagana_${arm_num}_base">
     <inertial>
-        <origin xyz="0.0 0.0 0.0"/>
-        <mass value="${motorA_mass}"/>
-        <inertia ixx="${MotorA_xx}" ixy="${MotorA_xy}" ixz="${MotorA_xz}" iyy="${MotorA_yy}" iyz="${MotorA_yz}" izz="${MotorA_zz}"/>
+        <origin xyz="${Dagana_x} ${Dagana_y} ${Dagana_z}"/>
+        <mass value="${Dagana_mass}"/>
+        <inertia ixx="${Dagana_xx}" ixy="${Dagana_xy}" ixz="${Dagana_xz}" iyy="${Dagana_yy}" iyz="${Dagana_yz}" izz="${Dagana_zz}"/>
     </inertial>
     <visual>
@@ -23,9 +23,9 @@
     </collision>
 </link>
-<link name="dagana_${arm_num}_clamp">
+<link name="dagana_${arm_num}_claw">
     <inertial>
-        <origin xyz="0.0 0.0 0.0"/>
-        <mass value="${motorA_mass}"/>
-        <inertia ixx="${MotorA_xx}" ixy="${MotorA_xy}" ixz="${MotorA_xz}" iyy="${MotorA_yy}" iyz="${MotorA_yz}" izz="${MotorA_zz}"/>
+        <origin xyz="${DaganaClaw_x} ${DaganaClaw_y} ${DaganaClaw_z}"/>
+        <mass value="${DaganaClaw_mass}"/>
+        <inertia ixx="${DaganaClaw_xx}" ixy="${DaganaClaw_xy}" ixz="${DaganaClaw_xz}" iyy="${DaganaClaw_yy}" iyz="${DaganaClaw_yz}" izz="${DaganaClaw_zz}"/>
     </inertial>
     <visual>
@@ -50,5 +50,5 @@
 <joint name="dagana_${arm_num}_clamp_joint" type="revolute">
     <parent link="dagana_${arm_num}_base"/>
-    <child link="dagana_${arm_num}_clamp"/>
+    <child link="dagana_${arm_num}_claw"/>
     <origin xyz="${DaganaClamp_Ox} ${DaganaClamp_Oy} ${DaganaClamp_Oz}" rpy="${DaganaClamp_roll} ${DaganaClamp_pitch} ${DaganaClamp_yaw}"/>
     <axis xyz="0 0 1"/>

Commit message: overwrite wheel_leg inertia (temporary)
inertia has to be modified since the original values are not correct

File: kyon_urdf/urdf/parts/inertial_properties.urdf.xacro (robot description, xacro)
@@ -60,10 +60,20 @@
     <xacro:property name="KneePitchWheel_y" value="${-2.5371445e+02 * mmTom}"/>
     <xacro:property name="KneePitchWheel_z" value="${4.1781751e+01 * mmTom}"/>
-    <xacro:property name="KneePitchWheel_xx" value="${1.1851050e+04 * mm2Tom2}"/>
+    <!-- <xacro:property name="KneePitchWheel_xx" value="${1.1851050e+04 * mm2Tom2}"/>
     <xacro:property name="KneePitchWheel_xy" value="${5.3594921e+02 * mm2Tom2}"/>
     <xacro:property name="KneePitchWheel_xz" value="${-1.9109120e+03 * mm2Tom2}"/>
     <xacro:property name="KneePitchWheel_yy" value="${-2.2822244e+03 * mm2Tom2}"/>
     <xacro:property name="KneePitchWheel_yz" value="${1.4122439e+03 * mm2Tom2}"/>
-    <xacro:property name="KneePitchWheel_zz" value="${1.2166274e+04 * mm2Tom2}"/>
+    <xacro:property name="KneePitchWheel_zz" value="${1.2166274e+04 * mm2Tom2}"/> -->
+    <xacro:property name="lower_leg_mass" value="1.0"/>
+    <xacro:property name="lower_leg_length" value="0.3"/>
+    <xacro:property name="lower_leg_width" value="0.05"/>
+    <xacro:property name="lower_leg_height" value="0.05"/>
+    <xacro:property name="KneePitchWheel_xx" value="${1/3 * lower_leg_mass * (lower_leg_width * lower_leg_width + lower_leg_height * lower_leg_height)}"/>
+    <xacro:property name="KneePitchWheel_xy" value="0.0"/>
+    <xacro:property name="KneePitchWheel_xz" value="0.0"/>
+    <xacro:property name="KneePitchWheel_yy" value="${1/3 * lower_leg_mass * (lower_leg_length * lower_leg_length + lower_leg_height * lower_leg_height)}"/>
+    <xacro:property name="KneePitchWheel_yz" value="0.0"/>
+    <xacro:property name="KneePitchWheel_zz" value="${1/3 * lower_leg_mass * (lower_leg_width * lower_leg_width + lower_leg_length * lower_leg_length)}"/>
     <!-- Ankle Yaw -->
     <xacro:property name="AnkleYaw_mass" value="1.4941965"/>

Commit message: removed unfeasible inertias

File: kyon_urdf/urdf/parts/inertial_properties.urdf.xacro (robot description, xacro)
@@ -61,8 +61,8 @@
     <xacro:property name="KneePitchWheel_z" value="${4.1781751e+01 * mmTom}"/>
     <xacro:property name="KneePitchWheel_xx" value="${1.1851050e+04 * mm2Tom2}"/>
-    <xacro:property name="KneePitchWheel_xy" value="${5.3594921e+02 * mm2Tom2}"/>
-    <xacro:property name="KneePitchWheel_xz" value="${-1.9109120e+03 * mm2Tom2}"/>
-    <xacro:property name="KneePitchWheel_yy" value="${-2.2822244e+03 * mm2Tom2}"/>
-    <xacro:property name="KneePitchWheel_yz" value="${1.4122439e+03 * mm2Tom2}"/>
+    <xacro:property name="KneePitchWheel_xy" value="${0* mm2Tom2}"/>
+    <xacro:property name="KneePitchWheel_xz" value="${0 * mm2Tom2}"/>
+    <xacro:property name="KneePitchWheel_yy" value="${2.2822244e+03 * mm2Tom2}"/>
+    <xacro:property name="KneePitchWheel_yz" value="${0 * mm2Tom2}"/>
     <xacro:property name="KneePitchWheel_zz" value="${1.2166274e+04 * mm2Tom2}"/>
     <!-- Ankle Yaw -->

Commit message: pelvis mass with battery

File: kyon_urdf/urdf/parts/inertial_properties.urdf.xacro (robot description, xacro)
@@ -3,5 +3,5 @@
     <xacro:property name="mm2Tom2" value="${0.001*0.001}"/>
     <!-- Pelvis -->
-    <xacro:property name="Pelvis_mass" value="23.024083"/>
+    <xacro:property name="Pelvis_mass" value="27.724083"/>  <!-- ERA 23 poi 15 poi 18 -->
     <xacro:property name="Pelvis_x" value="${4.9723680e+01 * mmTom}"/>
     <xacro:property name="Pelvis_y" value="${2.2995169e+00 * mmTom}"/>

Commit message: Fix inertial properties in inertial_properties.urdf.xacro

File: kyon_urdf/urdf/parts/inertial_properties.urdf.xacro (robot description, xacro)
@@ -45,5 +45,5 @@
     <xacro:property name="HipPitch_xy" value="${-6.4677573e+02 * mm2Tom2}"/>
     <xacro:property name="HipPitch_xz" value="${-5.7668584e+01 * mm2Tom2}"/>
-    <xacro:property name="HipPitch_yy" value="${2.7586781e+04 * mm2Tom2}"/>
+    <xacro:property name="HipPitch_yy" value="${3.3682020e+04 * mm2Tom2}"/>
     <xacro:property name="HipPitch_yz" value="${2.7586781e+04 * mm2Tom2}"/>
     <xacro:property name="HipPitch_zz" value="${1.0048465e+05 * mm2Tom2}"/>
@@ -165,5 +165,5 @@
     <xacro:property name="WristYaw_xz" value="${-1.2366562e-01 * mm2Tom2}"/>
     <xacro:property name="WristYaw_yy" value="${7.7918818e+01 * mm2Tom2}"/>
-    <xacro:property name="WristYaw_yz" value="${--8.8392181e-01 * mm2Tom2}"/>
+    <xacro:property name="WristYaw_yz" value="${-8.8392181e-01 * mm2Tom2}"/>
     <xacro:property name="WristYaw_zz" value="${1.2246055e+02 * mm2Tom2}"/>
     <!-- Dagana -->
