Commit message: fix knee sign when using steering

File: kyon_urdf/urdf/parts/steering_wheel.urdf.xacro (robot description, xacro)
@@ -73,5 +73,5 @@
     <child link="knee_pitch_${leg_num}_link"/>
     <origin xyz="${KneePitch_Ox} ${KneePitch_Oy} ${KneePitch_Oz}" rpy="${KneePitch_roll} ${KneePitch_pitch} ${KneePitch_yaw}"/>
-    <axis xyz="0 0 1"/>
+    <axis xyz="0 0 -1"/>
     <limit lower="${knee_pitch_lower[leg_num-1]}" upper="${knee_pitch_upper[leg_num-1]}" effort="${motorA_effort}" velocity="${motorA_velocity}"/>
 </joint>
@@ -81,5 +81,5 @@
     <origin xyz="${AnkleYaw_Ox} ${AnkleYaw_Oy} ${AnkleYaw_Oz}" rpy="${AnkleYaw_roll} ${AnkleYaw_pitch} ${AnkleYaw_yaw}"/>
     <axis xyz="0 0 1"/>
-    <limit lower="${knee_pitch_lower[leg_num-1]}" upper="${knee_pitch_upper[leg_num-1]}" effort="${motorA_effort}" velocity="${motorA_velocity}"/>
+    <limit lower="${ankle_yaw_lower[leg_num-1]}" upper="${ankle_yaw_upper[leg_num-1]}" effort="${motorA_effort}" velocity="${motorA_velocity}"/>
 </joint>
 <joint name="wheel_joint_${leg_num}" type="revolute">
@@ -88,5 +88,5 @@
     <origin xyz="${SteeringWheel_Ox} ${SteeringWheel_Oy} ${SteeringWheel_Oz}" rpy="${SteeringWheel_roll} ${SteeringWheel_pitch} ${SteeringWheel_yaw}"/>
     <axis xyz="0 0 1"/>
-    <limit lower="${knee_pitch_lower[leg_num-1]}" upper="${knee_pitch_upper[leg_num-1]}" effort="${motorWheel_effort}" velocity="${motorWheel_velocity}"/>
+    <limit lower="-1e9" upper="1e9" effort="${motorWheel_effort}" velocity="${motorWheel_velocity}"/>
 </joint>
 </xacro:macro>

Commit message: back to revolute joints

File: kyon_urdf/urdf/parts/steering_wheel.urdf.xacro (robot description, xacro)
@@ -84,10 +84,10 @@
     <limit lower="${ankle_yaw_lower[leg_num-1]}" upper="${ankle_yaw_upper[leg_num-1]}" effort="${motorA_effort}" velocity="${motorA_velocity}"/>
 </joint>
-<joint name="wheel_joint_${leg_num}" type="continuous">
+<joint name="wheel_joint_${leg_num}" type="revolute">
     <parent link="ankle_yaw_${leg_num}_link"/>
     <child link="wheel_${leg_num}"/>
     <origin xyz="${SteeringWheel_Ox} ${SteeringWheel_Oy} ${SteeringWheel_Oz}" rpy="${SteeringWheel_roll} ${SteeringWheel_pitch} ${SteeringWheel_yaw}"/>
     <axis xyz="0 0 1"/>
-    <limit effort="${motorWheel_effort}" velocity="${motorWheel_velocity}"/>
+    <limit lower="-1e9" upper="1e9" effort="${motorWheel_effort}" velocity="${motorWheel_velocity}"/>
 </joint>
 </xacro:macro>

Commit message: add contact link to steering wheel

File: kyon_urdf/urdf/parts/steering_wheel.urdf.xacro (robot description, xacro)
@@ -91,4 +91,10 @@
     <limit lower="-1e9" upper="1e9" effort="${motorWheel_effort}" velocity="${motorWheel_velocity}"/>
 </joint>
+<joint name="contact_joint_${leg_num}" type="fixed">
+	<parent link="ankle_yaw_${leg_num}_link"/>
+    <child link="contact_${leg_num}"/>
+    <origin xyz="${SteeringWheel_Ox} ${SteeringWheel_Oy}  ${SteeringWheel_Oz - 0.107}"/>
+</joint>
+<link name="contact_${leg_num}"/>
 </xacro:macro>
 </robot>

Commit message: radius fix + wheel collision is now a cylinder by default

File: kyon_urdf/urdf/parts/steering_wheel.urdf.xacro (robot description, xacro)
@@ -64,6 +64,6 @@
 		<origin xyz="0.0 0.0 0.0"  rpy="0.0 0.0 0.0"/>
 		<geometry>
-	 		<!-- <cylinder radius="${cylinder_radius}" length="${cylinder_length}"/> -->
-			<mesh filename="${MESH_PATH}/collision/mesh_wheel.stl" scale="0.001 0.001 0.001"/>
+	 		<cylinder radius="0.1066" length="0.05"/>
+			<!-- <mesh filename="${MESH_PATH}/collision/mesh_wheel.stl" scale="0.001 0.001 0.001"/> -->
 		</geometry>
 		<material name="light_grey"/>
@@ -97,4 +97,10 @@
 </joint>
 <link name="contact_${leg_num}"/>
+<joint name="ball_joint_${leg_num}" type="fixed">
+	<parent link="ankle_yaw_${leg_num}_link"/>
+    <child link="ball_${leg_num}"/>
+    <origin xyz="${SteeringWheel_Ox} ${SteeringWheel_Oy} ${SteeringWheel_Oz}" rpy="${SteeringWheel_roll} ${SteeringWheel_pitch} ${SteeringWheel_yaw}"/>
+</joint>
+<link name="ball_${leg_num}"/>
 </xacro:macro>
 </robot>

Commit message: contact frames with wheels fix

File: kyon_urdf/urdf/parts/steering_wheel.urdf.xacro (robot description, xacro)
@@ -94,5 +94,5 @@
 	<parent link="ankle_yaw_${leg_num}_link"/>
     <child link="contact_${leg_num}"/>
-    <origin xyz="${SteeringWheel_Ox} ${SteeringWheel_Oy}  ${SteeringWheel_Oz - 0.107}"/>
+    <origin xyz="${SteeringWheel_Ox-0.0753775*mirror} ${SteeringWheel_Oy}  ${SteeringWheel_Oz-0.0753775} " rpy="0.0 ${0.785*mirror} 0.0"/>
 </joint>
 <link name="contact_${leg_num}"/>

Commit message: adjusted collision cylinder depth

File: kyon_urdf/urdf/parts/steering_wheel.urdf.xacro (robot description, xacro)
@@ -64,5 +64,5 @@
 		<origin xyz="0.0 0.0 0.0"  rpy="0.0 0.0 0.0"/>
 		<geometry>
-	 		<cylinder radius="0.1066" length="0.05"/>
+	 		<cylinder radius="0.1066" length="0.03"/>
 			<!-- <mesh filename="${MESH_PATH}/collision/mesh_wheel.stl" scale="0.001 0.001 0.001"/> -->
 		</geometry>

File: kyon_urdf/urdf/parts/wheel_leg.urdf.xacro (robot description, xacro)
@@ -40,5 +40,5 @@
 		<geometry>
 			<!-- <mesh filename="${MESH_PATH}/collision/mesh_wheel.stl" scale="0.001 0.001 0.001"/> -->
-            <cylinder radius="0.11" length="0.045"/>
+            <cylinder radius="0.11" length="0.03"/>
 		</geometry>
 	</collision>

Commit message: fixed meshes that were colliding even in homing

File: kyon_urdf/urdf/parts/steering_wheel.urdf.xacro (robot description, xacro)
@@ -21,5 +21,5 @@
 		<geometry>
 	 		<!-- <cylinder radius="${cylinder_radius}" length="${cylinder_length}"/> -->
-			<mesh filename="${MESH_PATH}/collision/mesh_knee-steering.stl" scale="0.001 0.001 0.001"/>
+			<mesh filename="${MESH_PATH}/collision/mesh_knee-steering_cut.stl" scale="0.001 0.001 0.001"/>
 		</geometry>
 	</collision>
@@ -43,5 +43,5 @@
 		<geometry>
 	 		<!-- <cylinder radius="${cylinder_radius}" length="${cylinder_length}"/> -->
-			<mesh filename="${MESH_PATH}/collision/mesh_ankle-yaw.stl" scale="0.001 0.001 0.001"/>
+			<mesh filename="${MESH_PATH}/collision/mesh_ankle-yaw_cut.stl" scale="0.001 0.001 0.001"/>
 		</geometry>
 	</collision>

Commit message: add name to wheel geom for replacing

File: kyon_urdf/urdf/parts/steering_wheel.urdf.xacro (robot description, xacro)
@@ -63,5 +63,5 @@
 	<collision>
 		<origin xyz="0.0 0.0 0.0"  rpy="0.0 0.0 0.0"/>
-		<geometry>
+		<geometry name="wheel_${leg_num}_collision">
 	 		<!-- <cylinder radius="${cylinder_radius}" length="${cylinder_length}"/> -->
 			<mesh filename="package://kyon_urdf/meshes/collision/mesh_wheel.stl" scale="0.001 0.001 0.001"/>
