Commit message: removed useless files

File: kyon_urdf/urdf/parts/foot_leg.urdf.xacro (robot description, xacro)
@@ -5,7 +5,7 @@
 <link name="knee_pitch_${leg_num}_link">
     <inertial>
-        <origin xyz="${StickLeg_x} ${StickLeg_y} ${StickLeg_z}"/>
-        <mass value="${StickLeg_mass}"/>
-        <inertia ixx="${StickLeg_xx}" ixy="${mirror*StickLeg_xy}" ixz="${mirror*StickLeg_xz}" iyy="${StickLeg_yy}" iyz="${StickLeg_yz}" izz="${StickLeg_zz}"/>
+        <origin xyz="${KneePitch_x} ${KneePitch_y} ${KneePitch_z}"/>
+        <mass value="${KneePitch_mass}"/>
+        <inertia ixx="${KneePitch_xx}" ixy="${mirror*KneePitch_xy}" ixz="${mirror*KneePitch_xz}" iyy="${KneePitch_yy}" iyz="${KneePitch_yz}" izz="${KneePitch_zz}"/>
     </inertial>
     <visual>

File: kyon_urdf/urdf/parts/inertial_properties.urdf.xacro (robot description, xacro)
@@ -2,43 +2,4 @@
 <robot  xmlns:xacro="http://ros.org/wiki/xacro">
     <xacro:property name="mm2Tom2" value="${0.001*0.001}"/>
-    <xacro:property name="inertial_yaml_file" value="$(find kyon_urdf)/urdf/config/inertial_properties.yaml" />
-    <xacro:property name="inertial_props" value="${xacro.load_yaml(inertial_yaml_file)}"/>
-    <xacro:property name="pelvis_mass" value="${inertial_props['pelvis_mass']}"/>
-    <xacro:property name="upper_leg_mass" value="${inertial_props['upper_leg_mass']}"/>
-    <xacro:property name="lower_leg_mass" value="${inertial_props['lower_leg_mass']}"/>
-    <xacro:property name="upper_arm1_mass" value="${inertial_props['upper_arm1_mass']}"/>
-    <xacro:property name="upper_arm2_mass" value="${inertial_props['upper_arm2_mass']}"/>
-    <xacro:property name="lower_arm_mass" value="${inertial_props['lower_arm_mass']}"/>
-    <xacro:property name="ball_mass" value="${inertial_props['ball_mass']}"/>
-    <xacro:property name="motorA_mass" value="${inertial_props['motorA_mass']}"/>
-    <xacro:property name="motor_arm1_mass" value="${inertial_props['motor_arm1_mass']}"/>
-    <xacro:property name="motor_arm2_mass" value="${inertial_props['motor_arm2_mass']}"/>
-    <xacro:property name="motor_arm3_mass" value="${inertial_props['motor_arm3_mass']}"/>
-    <!-- Compound properties (i.e. based on the props parsed from the yaml) -->
-    <!-- Motor -->
-    <xacro:property name="MotorA_xx" value="${1/12 * motor_arm1_mass * (3 * cylinder_radius * cylinder_radius + cylinder_length * cylinder_length)}"/>
-    <xacro:property name="MotorA_xy" value="0.0"/>
-    <xacro:property name="MotorA_xz" value="0.0"/>
-    <xacro:property name="MotorA_yy" value="${1/12 * motor_arm1_mass * (3 * cylinder_radius * cylinder_radius + cylinder_length * cylinder_length)}"/>
-    <xacro:property name="MotorA_yz" value="0.0"/>
-    <xacro:property name="MotorA_zz" value="${1/2 * motor_arm1_mass * cylinder_radius * cylinder_radius}"/>
-    <xacro:property name="MotorArm1_xx" value="${1/12 * motor_arm1_mass * (3 * cylinder_radius * cylinder_radius + cylinder_length * cylinder_length)}"/>
-    <xacro:property name="MotorArm1_xy" value="0.0"/>
-    <xacro:property name="MotorArm1_xz" value="0.0"/>
-    <xacro:property name="MotorArm1_yy" value="${1/12 * motor_arm1_mass * (3 * cylinder_radius * cylinder_radius + cylinder_length * cylinder_length)}"/>
-    <xacro:property name="MotorArm1_yz" value="0.0"/>
-    <xacro:property name="MotorArm1_zz" value="${1/2 * motor_arm1_mass * cylinder_radius * cylinder_radius}"/>
-    <xacro:property name="MotorArm2_xx" value="${1/12 * motor_arm2_mass * (3 * cylinder_radius * cylinder_radius + cylinder_length * cylinder_length)}"/>
-    <xacro:property name="MotorArm2_xy" value="0.0"/>
-    <xacro:property name="MotorArm2_xz" value="0.0"/>
-    <xacro:property name="MotorArm2_yy" value="${1/12 * motor_arm2_mass * (3 * cylinder_radius * cylinder_radius + cylinder_length * cylinder_length)}"/>
-    <xacro:property name="MotorArm2_yz" value="0.0"/>
-    <xacro:property name="MotorArm2_zz" value="${1/2 * motor_arm2_mass * cylinder_radius * cylinder_radius}"/>
-    <xacro:property name="MotorArm3_xx" value="${1/12 * motor_arm3_mass * (3 * cylinder_radius * cylinder_radius + cylinder_length * cylinder_length)}"/>
-    <xacro:property name="MotorArm3_xy" value="0.0"/>
-    <xacro:property name="MotorArm3_xz" value="0.0"/>
-    <xacro:property name="MotorArm3_yy" value="${1/12 * motor_arm3_mass * (3 * cylinder_radius * cylinder_radius + cylinder_length * cylinder_length)}"/>
-    <xacro:property name="MotorArm3_yz" value="0.0"/>
-    <xacro:property name="MotorArm3_zz" value="${1/2 * motor_arm3_mass * cylinder_radius * cylinder_radius}"/>
     <!-- Pelvis -->
     <xacro:property name="Pelvis_mass" value="23.024083"/>
@@ -74,26 +35,35 @@
     <xacro:property name="HipPitch_yz" value="${2.8582838e+04 * mm2Tom2}"/>
     <xacro:property name="HipPitch_zz" value="${1.0356313e+05 * mm2Tom2}"/>
-    <!-- Stick Leg -->
-    <xacro:property name="StickLeg_mass" value="0.70900216"/>
-    <xacro:property name="StickLeg_x" value="${5.1193011e-03 * mmTom}"/>
-    <xacro:property name="StickLeg_y" value="${-1.0291595e+02 * mmTom}"/>
-    <xacro:property name="StickLeg_z" value="${-1.2895495e+00 * mmTom}"/>
-    <xacro:property name="StickLeg_xx" value="${1.2517512e+04 * mm2Tom2}"/>
-    <xacro:property name="StickLeg_xy" value="${-5.4385779e-01 * mm2Tom2}"/>
-    <xacro:property name="StickLeg_xz" value="${1.4538899e-01 * mm2Tom2}"/>
-    <xacro:property name="StickLeg_yy" value="${8.0474409e+02 * mm2Tom2}"/>
-    <xacro:property name="StickLeg_yz" value="${1.7446290e+03 * mm2Tom2}"/>
-    <xacro:property name="StickLeg_zz" value="${1.2307020e+04 * mm2Tom2}"/>
     <!-- Knee Pitch -->
-    <xacro:property name="KneePitch_mass" value="1.4555296"/>
-    <xacro:property name="KneePitch_x" value="${-5.1135441e-01 * mmTom}"/>
-    <xacro:property name="KneePitch_y" value="${-1.7451804e+01 * mmTom}"/>
-    <xacro:property name="KneePitch_z" value="${3.7226616e+01 * mmTom}"/>
-    <xacro:property name="KneePitch_xx" value="${3.8934930e+03 * mm2Tom2}"/>
-    <xacro:property name="KneePitch_xy" value="${2.4351251e+01 * mm2Tom2}"/>
-    <xacro:property name="KneePitch_xz" value="${2.2649175e+01 * mm2Tom2}"/>
-    <xacro:property name="KneePitch_yy" value="${3.2260304e+03 * mm2Tom2}"/>
-    <xacro:property name="KneePitch_yz" value="${5.5514749e+02 * mm2Tom2}"/>
-    <xacro:property name="KneePitch_zz" value="${2.0709191e+03 * mm2Tom2}"/>
+    <xacro:property name="KneePitch_mass" value="0.70900216"/>
+    <xacro:property name="KneePitch_x" value="${5.1193011e-03 * mmTom}"/>
+    <xacro:property name="KneePitch_y" value="${-1.0291595e+02 * mmTom}"/>
+    <xacro:property name="KneePitch_z" value="${-1.2895495e+00 * mmTom}"/>
+    <xacro:property name="KneePitch_xx" value="${1.2517512e+04 * mm2Tom2}"/>
+    <xacro:property name="KneePitch_xy" value="${-5.4385779e-01 * mm2Tom2}"/>
+    <xacro:property name="KneePitch_xz" value="${1.4538899e-01 * mm2Tom2}"/>
+    <xacro:property name="KneePitch_yy" value="${8.0474409e+02 * mm2Tom2}"/>
+    <xacro:property name="KneePitch_yz" value="${1.7446290e+03 * mm2Tom2}"/>
+    <xacro:property name="KneePitch_zz" value="${1.2307020e+04 * mm2Tom2}"/>
+    <xacro:property name="KneePitchSteeringWheel_mass" value="1.4555296"/>
+    <xacro:property name="KneePitchSteeringWheel_x" value="${-5.1135441e-01 * mmTom}"/>
+    <xacro:property name="KneePitchSteeringWheel_y" value="${-1.7451804e+01 * mmTom}"/>
+    <xacro:property name="KneePitchSteeringWheel_z" value="${3.7226616e+01 * mmTom}"/>
+    <xacro:property name="KneePitchSteeringWheel_xx" value="${3.8934930e+03 * mm2Tom2}"/>
+    <xacro:property name="KneePitchSteeringWheel_xy" value="${2.4351251e+01 * mm2Tom2}"/>
+    <xacro:property name="KneePitchSteeringWheel_xz" value="${2.2649175e+01 * mm2Tom2}"/>
+    <xacro:property name="KneePitchSteeringWheel_yy" value="${3.2260304e+03 * mm2Tom2}"/>
+    <xacro:property name="KneePitchSteeringWheel_yz" value="${5.5514749e+02 * mm2Tom2}"/>
+    <xacro:property name="KneePitchSteeringWheel_zz" value="${2.0709191e+03 * mm2Tom2}"/>
+    <xacro:property name="KneePitchWheel_mass" value="0.70900216"/>
+    <xacro:property name="KneePitchWheel_xx" value="${5.1193011e-03 * mmTom}"/>
+    <xacro:property name="KneePitchWheel_y" value="${-1.0291595e+02 * mmTom}"/>
+    <xacro:property name="KneePitchWheel_z" value="${-1.2895495e+00 * mmTom}"/>
+    <xacro:property name="KneePitchWheel_xx" value="${1.2517512e+04 * mm2Tom2}"/>
+    <xacro:property name="KneePitchWheel_xy" value="${-5.4385779e-01 * mm2Tom2}"/>
+    <xacro:property name="KneePitchWheel_xz" value="${1.4538899e-01 * mm2Tom2}"/>
+    <xacro:property name="KneePitchWheel_yy" value="${8.0474409e+02 * mm2Tom2}"/>
+    <xacro:property name="KneePitchWheel_yz" value="${1.7446290e+03 * mm2Tom2}"/>
+    <xacro:property name="KneePitchWheel_zz" value="${1.2307020e+04 * mm2Tom2}"/>
     <!-- Ankle Yaw -->
     <xacro:property name="AnkleYaw_mass" value="1.4941965"/>

File: kyon_urdf/urdf/parts/kinematics_properties.urdf.xacro (robot description, xacro)
@@ -3,27 +3,4 @@
     <xacro:property name="mmTom" value="0.001"/>
     <xacro:property name="degTorad" value="0.01744"/>
-    <xacro:property name="kin_yaml_file" value="$(find kyon_urdf)/urdf/config/kinematics_properties.yaml" />
-    <xacro:property name="kin_props" value="${xacro.load_yaml(kin_yaml_file)}"/>
-    <xacro:property name="cylinder_radius" value="${kin_props['cylinder_radius']}"/>
-    <xacro:property name="cylinder_length" value="${kin_props['cylinder_length']}"/>
-    <xacro:property name="upper_leg_length" value="${kin_props['upper_leg_length']}"/>
-    <xacro:property name="upper_leg_width" value="${kin_props['upper_leg_width']}"/>
-    <xacro:property name="upper_leg_height" value="${kin_props['upper_leg_height']}"/>
-    <xacro:property name="lower_leg_length" value="${kin_props['lower_leg_length']}"/>
-    <xacro:property name="lower_leg_width" value="${kin_props['lower_leg_width']}"/>
-    <xacro:property name="lower_leg_height" value="${kin_props['lower_leg_height']}"/>
-    <xacro:property name="upper_arm1_length" value="${kin_props['upper_arm1_length']}"/>
-    <xacro:property name="upper_arm1_width" value="${kin_props['upper_arm1_width']}"/>
-    <xacro:property name="upper_arm1_height" value="${kin_props['upper_arm1_height']}"/>
-    <xacro:property name="upper_arm2_length" value="${kin_props['upper_arm2_length']}"/>
-    <xacro:property name="upper_arm2_width" value="${kin_props['upper_arm2_width']}"/>
-    <xacro:property name="upper_arm2_height" value="${kin_props['upper_arm2_height']}"/>
-    <xacro:property name="lower_arm_length" value="${kin_props['lower_arm_length']}"/>
-    <xacro:property name="lower_arm_width" value="${kin_props['lower_arm_width']}"/>
-    <xacro:property name="lower_arm_height" value="${kin_props['lower_arm_height']}"/>
-    <xacro:property name="ball_radius" value="${kin_props['ball_radius']}"/>
-    <xacro:property name="pelvis_length" value="${kin_props['pelvis_length']}"/>
-    <xacro:property name="pelvis_width" value="${kin_props['pelvis_width']}"/>
-    <xacro:property name="pelvis_height" value="${kin_props['pelvis_height']}"/>
     <!-- Compound properties (i.e. based on the props parsed from the yaml) -->
     <!-- Origin -->

File: kyon_urdf/urdf/parts/limits.urdf.xacro (robot description, xacro)
@@ -25,16 +25,6 @@
 <xacro:property name="dagana_upper" value="${[3.4056, 3.3266]}"/>
 <!-- Motor velocities -->
-<xacro:if value="${inertial_props['gear_ratio'] == 30}">
-	<xacro:property name="motor_velocity" value="15.5"/>
-</xacro:if>
-<xacro:if value="${inertial_props['gear_ratio'] == 50}">
-	<xacro:property name="motor_velocity" value="9.3"/>
-</xacro:if>
+<xacro:property name="motor_velocity" value="15.5"/>
 <!-- Motor effort -->
-<xacro:if value="${inertial_props['gear_ratio'] == 30}">
-	<xacro:property name="motor_effort" value="132"/>
-</xacro:if>
-<xacro:if value="${inertial_props['gear_ratio'] == 50}">
-	<xacro:property name="motor_effort" value="220"/>
-</xacro:if>
+<xacro:property name="motor_effort" value="132"/>
 </robot>

File: kyon_urdf/urdf/parts/steering_wheel.urdf.xacro (robot description, xacro)
@@ -5,7 +5,7 @@
 <link name="knee_pitch_${leg_num}_link">
     <inertial>
-		<origin xyz="${KneePitch_x} ${KneePitch_y} ${KneePitch_z}"/>
-		<mass value="${KneePitch_mass}"/>
-		<inertia ixx="${KneePitch_xx}" ixy="${KneePitch_xy}" ixz="${KneePitch_xz}" iyy="${KneePitch_yy}" iyz="${KneePitch_yz}" izz="${KneePitch_zz}"/>
+		<origin xyz="${KneePitchSteeringWheel_x} ${KneePitchSteeringWheel_y} ${KneePitchSteeringWheel_z}"/>
+		<mass value="${KneePitchSteeringWheel_mass}"/>
+		<inertia ixx="${KneePitchSteeringWheel_xx}" ixy="${KneePitchSteeringWheel_xy}" ixz="${KneePitchSteeringWheel_xz}" iyy="${KneePitchSteeringWheel_yy}" iyz="${KneePitchSteeringWheel_yz}" izz="${KneePitchSteeringWheel_zz}"/>
 	</inertial>
 	<visual>

File: kyon_urdf/urdf/parts/wheel_leg.urdf.xacro (robot description, xacro)
@@ -6,6 +6,6 @@
     <inertial>
         <origin xyz="0.0 0.0 0.0"/>
-        <mass value="${motorA_mass}"/>
-        <inertia ixx="${MotorA_xx}" ixy="${mirror*MotorA_xy}" ixz="${mirror*MotorA_xz}" iyy="${MotorA_yy}" iyz="${MotorA_yz}" izz="${MotorA_zz}"/>
+        <mass value="${KneePitchWheel_mass}"/>
+        <inertia ixx="${KneePitchWheel_xx}" ixy="${mirror*KneePitchWheel_xy}" ixz="${mirror*KneePitchWheel_xz}" iyy="${KneePitchWheel_yy}" iyz="${KneePitchWheel_yz}" izz="${KneePitchWheel_zz}"/>
     </inertial>
     <visual>

Commit message: updated effort and velocity limits

File: kyon_urdf/urdf/parts/foot_leg.urdf.xacro (robot description, xacro)
@@ -28,5 +28,5 @@
     <origin xyz="${KneePitch_Ox} ${KneePitch_Oy} ${KneePitch_Oz}" rpy="${KneePitch_roll} ${KneePitch_pitch} ${KneePitch_yaw}"/>
     <axis xyz="0 0 1"/>
-    <limit lower="${knee_pitch_lower[leg_num-1]}" upper="${knee_pitch_upper[leg_num-1]}" effort="${motor_effort}" velocity="${motor_velocity}"/>
+    <limit lower="${knee_pitch_lower[leg_num-1]}" upper="${knee_pitch_upper[leg_num-1]}" effort="${motorA_effort}" velocity="${motorA_velocity}"/>
 </joint>
 <link name="contact_${leg_num}"/>

File: kyon_urdf/urdf/parts/kyon_arm.urdf.xacro (robot description, xacro)
@@ -109,5 +109,5 @@
 	<origin xyz="${ShoulderYaw_Ox} ${rot * ShoulderYaw_Oy} ${ShoulderYaw_Oz}" rpy="${rot * ShoulderYaw_roll} ${ShoulderYaw_pitch} ${ShoulderYaw_yaw}"/>
 	<axis xyz="0 0 1"/>
-	<limit lower="${j_shoulder_yaw_lower[arm_num-1]}" upper="${j_shoulder_yaw_upper[arm_num-1]}" effort="${motor_effort}" velocity="${motor_velocity}"/>
+	<limit lower="${j_shoulder_yaw_lower[arm_num-1]}" upper="${j_shoulder_yaw_upper[arm_num-1]}" effort="${motorB_effort}" velocity="${motorB_velocity}"/>
 </joint>
 <!-- arm pitch 1 -->
@@ -117,5 +117,5 @@
 	<origin xyz="${ShoulderPitch_Ox} ${ShoulderPitch_Oy} ${ShoulderPitch_Oz}" rpy="${ShoulderPitch_roll} ${ShoulderPitch_pitch} ${ShoulderPitch_yaw + rot * PI_2}"/>
 	<axis xyz="0 0 1"/>
-	<limit lower="${j_pitch_1_lower[arm_num-1]}" upper="${j_pitch_1_upper[arm_num-1]}" effort="${motor_effort}" velocity="${motor_velocity}"/>
+	<limit lower="${j_pitch_1_lower[arm_num-1]}" upper="${j_pitch_1_upper[arm_num-1]}" effort="${motorC_effort}" velocity="${motorC_velocity}"/>
 </joint>
 <joint name="elbow_pitch_${arm_num}" type="revolute">
@@ -124,5 +124,5 @@
 	<origin xyz="${ElbowPitch_Ox} ${ElbowPitch_Oy} ${ElbowPitch_Oz}" rpy="${ElbowPitch_roll} ${ElbowPitch_pitch} ${ElbowPitch_yaw}"/>
 	<axis xyz="0 0 1"/>
-	<limit lower="${j_pitch_1_lower[arm_num-1]}" upper="${j_pitch_1_upper[arm_num-1]}" effort="${motor_effort}" velocity="${motor_velocity}"/>
+	<limit lower="${j_pitch_1_lower[arm_num-1]}" upper="${j_pitch_1_upper[arm_num-1]}" effort="${motorC_effort}" velocity="${motorC_velocity}"/>
 </joint>
 <joint name="wrist_pitch_${arm_num}" type="revolute">
@@ -131,5 +131,5 @@
 	<origin xyz="${WristPitch_Ox} ${WristPitch_Oy} ${WristPitch_Oz}" rpy="${WristPitch_roll} ${WristPitch_pitch} ${WristPitch_yaw}"/>
 	<axis xyz="0 0 1"/>
-	<limit lower="${j_pitch_2_lower[arm_num-1]}" upper="${j_pitch_2_upper[arm_num-1]}" effort="${motor_effort}" velocity="${motor_velocity}"/>
+	<limit lower="${j_pitch_2_lower[arm_num-1]}" upper="${j_pitch_2_upper[arm_num-1]}" effort="${motorD_effort}" velocity="${motorD_velocity}"/>
 </joint>
 <joint name="wrist_yaw_${arm_num}" type="revolute">
@@ -138,5 +138,5 @@
 	<origin xyz="${WristYaw_Ox} ${WristYaw_Oy} ${WristYaw_Oz}" rpy="${WristYaw_roll} ${WristYaw_pitch} ${WristYaw_yaw}"/>
 	<axis xyz="0 0 1"/>
-	<limit lower="${j_pitch_2_lower[arm_num-1]}" upper="${j_pitch_2_upper[arm_num-1]}" effort="${motor_effort}" velocity="${motor_velocity}"/>
+	<limit lower="${j_pitch_2_lower[arm_num-1]}" upper="${j_pitch_2_upper[arm_num-1]}" effort="${motorD_effort}" velocity="${motorD_velocity}"/>
 </joint>
 <xacro:kyon_dagana arm_num="${arm_num}" parent="wrist_yaw_${arm_num}_link"/>

File: kyon_urdf/urdf/parts/kyon_dagana.urdf.xacro (robot description, xacro)
@@ -53,5 +53,5 @@
     <origin xyz="${DaganaClamp_Ox} ${DaganaClamp_Oy} ${DaganaClamp_Oz}" rpy="${DaganaClamp_roll} ${DaganaClamp_pitch} ${DaganaClamp_yaw}"/>
     <axis xyz="0 0 1"/>
-    <limit lower="${dagana_lower[arm_num-1]}" upper="${dagana_upper[arm_num-1]}" effort="${motor_effort}" velocity="${motor_velocity}"/>
+    <limit lower="${dagana_lower[arm_num-1]}" upper="${dagana_upper[arm_num-1]}" effort="${motorD_effort}" velocity="${motorD_velocity}"/>
 </joint>
 </xacro:macro>

File: kyon_urdf/urdf/parts/kyon_leg.urdf.xacro (robot description, xacro)
@@ -56,5 +56,5 @@
 	<origin xyz="${origin_x * HipRoll_Ox} ${origin_y * HipRoll_Oy} ${HipRoll_Oz}" rpy="${HipRoll_roll} ${origin_x*HipRoll_pitch} ${HipRoll_yaw}"/>
 	<axis xyz="0 0 1"/>
-    <limit lower="${hip_roll_lower[leg_num-1]}" upper="${hip_roll_upper[leg_num-1]}" effort="${motor_effort}" velocity="${motor_velocity}"/>
+    <limit lower="${hip_roll_lower[leg_num-1]}" upper="${hip_roll_upper[leg_num-1]}" effort="${motorA_effort}" velocity="${motorA_velocity}"/>
 </joint>
 <joint name="hip_pitch_${leg_num}" type="revolute">
@@ -63,5 +63,5 @@
 	<origin xyz="${HipPitch_Ox} ${origin_y * HipPitch_Oy} ${HipPitch_Oz}" rpy="${HipPitch_roll} ${origin_x * origin_y * HipPitch_pitch} ${origin_x * HipPitch_yaw}"/>
 	<axis xyz="0 0 1"/>
-	<limit lower="${hip_pitch_lower[leg_num-1]}" upper="${hip_pitch_upper[leg_num-1]}" effort="${motor_effort}" velocity="${motor_velocity}"/>
+	<limit lower="${hip_pitch_lower[leg_num-1]}" upper="${hip_pitch_upper[leg_num-1]}" effort="${motorA_effort}" velocity="${motorA_velocity}"/>
 </joint>
 <xacro:if value="${ADD_FEET}">

File: kyon_urdf/urdf/parts/limits.urdf.xacro (robot description, xacro)
@@ -29,8 +29,10 @@
 <xacro:property name="motorC_velocity" value="4.6"/>
 <xacro:property name="motorD_velocity" value="14"/>
+<xacro:property name="motorWheel_velocity" value="20"/>
 <!-- Motor effort -->
 <xacro:property name="motorA_effort" value="185"/>
-<xacro:property name="motorA_effort" value="146"/>
-<xacro:property name="motorA_effort" value="122"/>
-<xacro:property name="motorA_effort" value="25"/>
+<xacro:property name="motorB_effort" value="146"/>
+<xacro:property name="motorC_effort" value="122"/>
+<xacro:property name="motorD_effort" value="25"/>
+<xacro:property name="motorWheel_effort" value="100"/>
 </robot>

File: kyon_urdf/urdf/parts/steering_wheel.urdf.xacro (robot description, xacro)
@@ -74,5 +74,5 @@
     <origin xyz="${KneePitch_Ox} ${KneePitch_Oy} ${KneePitch_Oz}" rpy="${KneePitch_roll} ${KneePitch_pitch} ${KneePitch_yaw}"/>
     <axis xyz="0 0 1"/>
-    <limit lower="${knee_pitch_lower[leg_num-1]}" upper="${knee_pitch_upper[leg_num-1]}" effort="${motor_effort}" velocity="${motor_velocity}"/>
+    <limit lower="${knee_pitch_lower[leg_num-1]}" upper="${knee_pitch_upper[leg_num-1]}" effort="${motorA_effort}" velocity="${motorA_velocity}"/>
 </joint>
 <joint name="ankle_yaw_${leg_num}" type="revolute">
@@ -81,5 +81,5 @@
     <origin xyz="${AnkleYaw_Ox} ${AnkleYaw_Oy} ${AnkleYaw_Oz}" rpy="${AnkleYaw_roll} ${AnkleYaw_pitch} ${AnkleYaw_yaw}"/>
     <axis xyz="0 0 1"/>
-    <limit lower="${knee_pitch_lower[leg_num-1]}" upper="${knee_pitch_upper[leg_num-1]}" effort="${motor_effort}" velocity="${motor_velocity}"/>
+    <limit lower="${knee_pitch_lower[leg_num-1]}" upper="${knee_pitch_upper[leg_num-1]}" effort="${motorA_effort}" velocity="${motorA_velocity}"/>
 </joint>
 <joint name="wheel_joint_${leg_num}" type="revolute">
@@ -88,5 +88,5 @@
     <origin xyz="${SteeringWheel_Ox} ${SteeringWheel_Oy} ${SteeringWheel_Oz}" rpy="${SteeringWheel_roll} ${SteeringWheel_pitch} ${SteeringWheel_yaw}"/>
     <axis xyz="0 0 1"/>
-    <limit lower="${knee_pitch_lower[leg_num-1]}" upper="${knee_pitch_upper[leg_num-1]}" effort="${motor_effort}" velocity="${motor_velocity}"/>
+    <limit lower="${knee_pitch_lower[leg_num-1]}" upper="${knee_pitch_upper[leg_num-1]}" effort="${motorWheel_effort}" velocity="${motorWheel_velocity}"/>
 </joint>
 </xacro:macro>

File: kyon_urdf/urdf/parts/wheel_leg.urdf.xacro (robot description, xacro)
@@ -48,5 +48,5 @@
     <origin xyz="${KneePitch_Ox} ${KneePitch_Oy} ${KneePitch_Oz}" rpy="${KneePitch_roll} ${KneePitch_pitch} ${KneePitch_yaw}"/>
     <axis xyz="0 0 1"/>
-    <limit lower="${knee_pitch_lower[leg_num-1]}" upper="${knee_pitch_upper[leg_num-1]}" effort="${motor_effort}" velocity="${motor_velocity}"/>
+    <limit lower="${knee_pitch_lower[leg_num-1]}" upper="${knee_pitch_upper[leg_num-1]}" effort="${motorA_effort}" velocity="${motorA_velocity}"/>
 </joint>
 <joint name="wheel_joint_${leg_num}" type="revolute">
@@ -55,5 +55,5 @@
     <origin xyz="${Wheel_Ox} ${Wheel_Oy} ${Wheel_Oz}" rpy="${Wheel_roll} ${Wheel_pitch} ${Wheel_yaw}"/>
     <axis xyz="0 0 1"/>
-    <limit lower="${knee_pitch_lower[leg_num-1]}" upper="${knee_pitch_upper[leg_num-1]}" effort="${motor_effort}" velocity="${motor_velocity}"/>
+    <limit lower="${knee_pitch_lower[leg_num-1]}" upper="${knee_pitch_upper[leg_num-1]}" effort="${motorWheel_effort}" velocity="${motorWheel_velocity}"/>
 </joint>
 </xacro:macro>
