Commit message: leg signs

File: kyon_urdf/urdf/parts/foot_leg.urdf.xacro (robot description, xacro)
@@ -27,5 +27,5 @@
     <child link="knee_pitch_${leg_num}_link"/>
     <origin xyz="${KneePitch_Ox} ${KneePitch_Oy} ${KneePitch_Oz}" rpy="${KneePitch_roll} ${KneePitch_pitch} ${KneePitch_yaw}"/>
-    <axis xyz="0 0 1"/>
+    <axis xyz="0 0 -1"/>
     <limit lower="${knee_pitch_lower[leg_num-1]}" upper="${knee_pitch_upper[leg_num-1]}" effort="${motorA_effort}" velocity="${motorA_velocity}"/>
 </joint>

File: kyon_urdf/urdf/parts/kyon_leg.urdf.xacro (robot description, xacro)
@@ -55,5 +55,5 @@
 	<child link="hip_roll_${leg_num}_link"/>
 	<origin xyz="${origin_x * HipRoll_Ox} ${origin_y * HipRoll_Oy} ${HipRoll_Oz}" rpy="${HipRoll_roll} ${origin_x*HipRoll_pitch} ${HipRoll_yaw}"/>
-	<axis xyz="0 0 1"/>
+	<axis xyz="0 0 -1"/>
     <limit lower="${hip_roll_lower[leg_num-1]}" upper="${hip_roll_upper[leg_num-1]}" effort="${motorA_effort}" velocity="${motorA_velocity}"/>
 </joint>
@@ -62,5 +62,5 @@
 	<child link="hip_pitch_${leg_num}_link"/>
 	<origin xyz="${HipPitch_Ox} ${origin_y * HipPitch_Oy} ${HipPitch_Oz}" rpy="${HipPitch_roll} ${origin_x * origin_y * HipPitch_pitch} ${origin_x * HipPitch_yaw}"/>
-	<axis xyz="0 0 1"/>
+	<axis xyz="0 0 -1"/>
 	<limit lower="${hip_pitch_lower[leg_num-1]}" upper="${hip_pitch_upper[leg_num-1]}" effort="${motorA_effort}" velocity="${motorA_velocity}"/>
 </joint>

Commit message: fixed foot contact sphere size/location

File: kyon_urdf/urdf/parts/foot_leg.urdf.xacro (robot description, xacro)
@@ -43,5 +43,5 @@
                     <origin xyz="0.0 0.0 0.0" rpy="0.0 0.0 0.0" />
                     <geometry>
-                        <sphere radius="0.03" />
+                        <sphere radius="0.039" />
                     </geometry>
                     <material>
@@ -54,5 +54,5 @@
             <parent link="knee_pitch_${leg_num}_link" />
             <child link="contact_${leg_num}" />
-            <origin xyz="${-mirror*0.0} -0.31 0.022"
+            <origin xyz="${-mirror*0.0} -0.305 0.022"
                 rpy="${1.57*mirror} ${0} ${0.785 if mirror == -1 else 2.356}" />
         </joint>

Commit message: moved contacts inward

File: kyon_urdf/urdf/parts/foot_leg.urdf.xacro (robot description, xacro)
@@ -46,5 +46,5 @@
     <parent link="knee_pitch_${leg_num}_link"/>
     <child link="contact_${leg_num}"/>
-    <origin xyz="${-mirror*0.0} -0.305 0.054" rpy="${1.57*mirror} ${0} ${0.785 if mirror == -1 else 2.356}"/>
+    <origin xyz="${-mirror*0.0} -0.305 0.022" rpy="${1.57*mirror} ${0} ${0.785 if mirror == -1 else 2.356}"/>
 </joint>
 </xacro:macro>

Commit message: fixed sphere collision position

File: kyon_urdf/urdf/parts/foot_leg.urdf.xacro (robot description, xacro)
@@ -50,5 +50,5 @@
     <parent link="knee_pitch_${leg_num}_link"/>
     <child link="contact_${leg_num}"/>
-    <origin xyz="${-mirror*0.0} -0.3 0.054" rpy="${1.57*mirror} ${0} ${0.785 if mirror == -1 else 2.356}"/>
+    <origin xyz="${-mirror*0.0} -0.312 0.024" rpy="${1.57*mirror} ${0} ${0.785 if mirror == -1 else 2.356}"/>
 </joint>
 </xacro:macro>

Commit message: Added inertia to feet contact links (otherwise Mujoco may compute it by itself)

File: kyon_urdf/urdf/parts/foot_leg.urdf.xacro (robot description, xacro)
@@ -33,4 +33,9 @@
 </joint>
 <link name="contact_${leg_num}">
+    <inertial>
+        <origin xyz="0 0 0"/>
+        <mass value="0.001"/>
+        <inertia ixx="6.4e-7" ixy="0.0" ixz="0.0" iyy="6.4e-7" iyz="0.0" izz="6.4e-7"/>
+    </inertial>
     <visual>
         <origin xyz="0 0 0" rpy="0 0 0"/>

Commit message: avoid contact spheres and add steering

File: kyon_urdf/urdf/parts/foot_leg.urdf.xacro (robot description, xacro)
@@ -32,19 +32,5 @@
     <limit lower="${knee_pitch_lower[leg_num-1]}" upper="${knee_pitch_upper[leg_num-1]}" effort="${motorA_effort}" velocity="${motorA_velocity}"/>
 </joint>
-<link name="contact_${leg_num}">
-    <visual>
-        <origin xyz="0 0 0" rpy="0 0 0"/>
-        <geometry>
-            <sphere radius="0.03"/>
-        </geometry>
-        <material name="white"/>
-    </visual>
-    <collision name="contact_${leg_num}">
-        <origin xyz="0 0 0" rpy="0 0 0"/>
-        <geometry>
-            <sphere radius="0.03"/>
-        </geometry>
-    </collision>
-</link>
+<link name="contact_${leg_num}"/>
 <joint name="contact_${leg_num}_joint" type="fixed">
     <parent link="knee_pitch_${leg_num}_link"/>

File: kyon_urdf/urdf/parts/kyon_leg.urdf.xacro (robot description, xacro)
@@ -80,10 +80,10 @@
 	<xacro:foot_leg leg_num="${leg_num}" parent="hip_pitch_${leg_num}_link" origin_x="${origin_x}" origin_y="${origin_y}" mirror="${mirror}"/>
 </xacro:unless>
-<!-- <xacro:if value="${ADD_WHEELS}"> -->
-	<!-- <xacro:steering_wheel leg_num="${leg_num}" parent="hip_pitch_${leg_num}_link" origin_x="${origin_x}" origin_y="${origin_y}" mirror="${mirror}"/> -->
-<!-- </xacro:if> -->
 <xacro:if value="${ADD_WHEELS}">
+	<xacro:steering_wheel leg_num="${leg_num}" parent="hip_pitch_${leg_num}_link" origin_x="${origin_x}" origin_y="${origin_y}" mirror="${mirror}"/>
+</xacro:if>
+<!-- <xacro:if value="${ADD_WHEELS}">
     <xacro:wheel_leg leg_num="${leg_num}" parent="hip_pitch_${leg_num}_link" origin_x="${origin_x}" origin_y="${origin_y}" mirror="${mirror}"/>
-</xacro:if>
+</xacro:if> -->
 </xacro:macro>
 <!-- /macro legs -->

Commit message: remove negative scale for foot leg left (isaac hasa issues)

File: kyon_urdf/urdf/parts/foot_leg.urdf.xacro (robot description, xacro)
@@ -12,5 +12,10 @@
         <origin xyz="0.0 0.0 0.0"  rpy="0.0 0.0 0.0"/>
         <geometry>
-            <mesh filename="${MESH_PATH}/mesh_foot-leg.stl" scale="${mirror*0.001} 0.001 0.001"/>
+            <xacro:if value="${mirror == -1}">
+                <mesh filename="${MESH_PATH}/mesh_foot_leg_left.stl" scale="0.001 0.001 0.001"/>
+            </xacro:if>
+            <xacro:unless value="${mirror == -1}">
+                <mesh filename="${MESH_PATH}/mesh_foot-leg.stl" scale="0.001 0.001 0.001"/>
+            </xacro:unless>
         </geometry>
         <material name="dark_grey"/>
@@ -19,5 +24,10 @@
         <origin xyz="0.0 0.0 0.0"  rpy="0.0 0.0 0.0"/>
         <geometry>
-            <mesh filename="${MESH_PATH}/collision/mesh_foot-leg.stl" scale="${mirror*0.001} 0.001 0.001"/>
+            <xacro:if value="${mirror == -1}">
+                <mesh filename="${MESH_PATH}/collision/mesh_foot_leg_left.stl" scale="0.001 0.001 0.001"/>
+            </xacro:if>
+            <xacro:unless value="${mirror == -1}">
+                <mesh filename="${MESH_PATH}/collision/mesh_foot-leg.stl" scale="0.001 0.001 0.001"/>
+            </xacro:unless>
         </geometry>
     </collision>
