Commit message: split dagana meshes to improve coll

File: kyon_urdf/urdf/parts/kyon_dagana.urdf.xacro (robot description, xacro)
@@ -19,5 +19,11 @@
         <origin xyz="0.0 0.0 0.0"  rpy="0.0 0.0 0.0"/>
         <geometry>
-            <mesh filename="package://kyon_urdf/meshes/collision/mesh_dagana-base.stl" scale="0.001 0.001 0.001"/>
+            <mesh filename="package://kyon_urdf/meshes/collision/mesh_dagana-base-simplified.stl" scale="0.001 0.001 0.001"/>
+        </geometry>
+    </collision>
+    <collision>
+        <origin xyz="0.0 0.0 0.0"  rpy="0.0 0.0 0.0"/>
+        <geometry>
+            <mesh filename="package://kyon_urdf/meshes/collision/mesh_dagana-base-base-simplified.stl" scale="0.001 0.001 0.001"/>
         </geometry>
     </collision>
@@ -39,5 +45,11 @@
         <origin xyz="0.0 0.0 0.0"  rpy="0.0 0.0 0.0"/>
         <geometry>
-            <mesh filename="package://kyon_urdf/meshes/collision/mesh_dagana-clamp.stl" scale="0.001 0.001 0.001"/>
+            <mesh filename="package://kyon_urdf/meshes/collision/mesh_dagana-clamp-base-simplified.stl" scale="0.001 0.001 0.001"/>
+        </geometry>
+    </collision>
+    <collision>
+        <origin xyz="0.0 0.0 0.0"  rpy="0.0 0.0 0.0"/>
+        <geometry>
+            <mesh filename="package://kyon_urdf/meshes/collision/mesh_dagana-clamp-simplified.stl" scale="0.001 0.001 0.001"/>
         </geometry>
     </collision>

Commit message: bugfix

File: kyon_urdf/urdf/parts/kyon_dagana.urdf.xacro (robot description, xacro)
@@ -41,10 +41,10 @@
         </geometry>
     </collision>
-    <visual>
+    <collision>
         <origin xyz="0.0 0.0007432 0.0405" rpy="0 0 0" />
         <geometry>
             <box size="0.0879  0.0844864 0.081"/>
         </geometry>
-    </visual>
+    </collision>
     <!-- <collision>
         <origin xyz="0.0 0.0 0.0"  rpy="0.0 0.0 0.0"/>
