Commit message: modified to revolute for controller purposes

File: kyon_urdf/urdf/gazebo/xbot.gazebo.xacro (robot description, xacro)
@@ -11,8 +11,8 @@
     <plugin name="xbot2_joint_driver" filename="libxbot2_gz_joint_server.so">
         <pid>
-            <gain name="lowpwr_mot" p="50"  d="5"/>
-            <gain name="small_mot"  p="200"  d="10"/>
-            <gain name="medium_mot" p="500" d="20"/>
-            <gain name="big_mot"    p="1000" d="30"/>
+            <gain name="lowpwr_mot" p="100"  d="1"/>
+            <gain name="small_mot"  p="500"  d="5"/>
+            <gain name="medium_mot" p="1000" d="10"/>
+            <gain name="big_mot"    p="1500" d="20"/>
             <pid name="shoulder_yaw_1" profile="medium_mot"/>
             <pid name="shoulder_pitch_1" profile="medium_mot"/>
@@ -27,14 +27,14 @@
             <pid name="hip_roll_1"     profile="big_mot"/>
             <pid name="hip_pitch_1"  profile="big_mot"/>
-            <pid name="knee_pitch_1"   profile="medium_mot"/>
+            <pid name="knee_pitch_1"   profile="big_mot"/>
             <pid name="hip_roll_2"     profile="big_mot"/>
             <pid name="hip_pitch_2"  profile="big_mot"/>
-            <pid name="knee_pitch_2"   profile="medium_mot"/>
+            <pid name="knee_pitch_2"   profile="big_mot"/>
             <pid name="hip_roll_3"     profile="big_mot"/>
             <pid name="hip_pitch_3"  profile="big_mot"/>
-            <pid name="knee_pitch_3"   profile="medium_mot"/>
+            <pid name="knee_pitch_3"   profile="big_mot"/>
             <pid name="hip_roll_4"     profile="big_mot"/>
             <pid name="hip_pitch_4"  profile="big_mot"/>
-            <pid name="knee_pitch_4"   profile="medium_mot"/>
+            <pid name="knee_pitch_4"   profile="big_mot"/>
         </pid>
     </plugin>

File: kyon_urdf/urdf/parts/kyon_leg.urdf.xacro (robot description, xacro)
@@ -125,5 +125,5 @@
 </link>
 <xacro:if value="${ADD_WHEELS}">
-	<joint name="wheel_joint_${leg_num}" type="continuous">
+	<joint name="wheel_joint_${leg_num}" type="revolute">
             <parent link="ball_${leg_num}" />
             <child link="wheel_${leg_num}" />
