Commit message: fixed last simulator small issues

File: kyon_urdf/urdf/gazebo/kyon.gazebo.xacro (robot description, xacro)
@@ -200,4 +200,12 @@
             <provideFeedback>true</provideFeedback>
         </gazebo>
+        <gazebo reference="wrist_pitch_1">
+            <implicitSpringDamper>1</implicitSpringDamper>
+            <provideFeedback>true</provideFeedback>
+        </gazebo>
+        <gazebo reference="wrist_yaw_1">
+            <implicitSpringDamper>1</implicitSpringDamper>
+            <provideFeedback>true</provideFeedback>
+        </gazebo>
         <gazebo reference="shoulder_yaw_2">
             <implicitSpringDamper>1</implicitSpringDamper>
@@ -209,4 +217,12 @@
         </gazebo>
         <gazebo reference="elbow_pitch_2">
+            <implicitSpringDamper>1</implicitSpringDamper>
+            <provideFeedback>true</provideFeedback>
+        </gazebo>
+        <gazebo reference="wrist_pitch_2">
+            <implicitSpringDamper>1</implicitSpringDamper>
+            <provideFeedback>true</provideFeedback>
+        </gazebo>
+        <gazebo reference="wrist_yaw_2">
             <implicitSpringDamper>1</implicitSpringDamper>
             <provideFeedback>true</provideFeedback>

File: kyon_urdf/urdf/gazebo/materials.gazebo.xacro (robot description, xacro)
@@ -42,5 +42,5 @@
 </xacro:macro>
 <gazebo reference="pelvis">
-	<material>Gazebo/LightBlueLaser</material>
+	<material>Gazebo/SkyBlue</material>
 </gazebo>
 <xacro:if value="${ADD_LEGS}">
@@ -60,3 +60,16 @@
 </gazebo>
 </xacro:if>
+<xacro:if value="${ADD_WHEELS}"/>
+    <gazebo reference="wheel_1">
+        <material>Gazebo/DarkGrey</material>
+    </gazebo>
+    <gazebo reference="wheel_2">
+        <material>Gazebo/DarkGrey</material>
+    </gazebo>
+    <gazebo reference="wheel_3">
+        <material>Gazebo/DarkGrey</material>
+    </gazebo>
+    <gazebo reference="wheel_4">
+        <material>Gazebo/DarkGrey</material>
+    </gazebo>
 </robot>

File: kyon_urdf/urdf/gazebo/xbot.gazebo.xacro (robot description, xacro)
@@ -18,7 +18,11 @@
             <pid name="shoulder_pitch_1" profile="medium_mot"/>
             <pid name="elbow_pitch_1" profile="small_mot"/>
+            <pid name="wrist_pitch_1" profile="small_mot"/>
+            <pid name="wrist_yaw_1" profile="small_mot"/>
             <pid name="shoulder_yaw_2" profile="medium_mot"/>
             <pid name="shoulder_pitch_2" profile="medium_mot"/>
             <pid name="elbow_pitch_2" profile="small_mot"/>
+            <pid name="wrist_pitch_2" profile="small_mot"/>
+            <pid name="wrist_yaw_2" profile="small_mot"/>
             <pid name="hip_roll_1"     profile="big_mot"/>
             <pid name="hip_pitch_1"  profile="big_mot"/>

File: kyon_urdf/urdf/kyon.urdf (robot description, URDF)
Before this commit: robot kyon, 135 links, 134 joints
Links:
- removed link D435_front1_accel_frame
- removed link D435_front1_accel_optical_frame
- removed link D435_front1_bottom_screw_frame
- removed link D435_front1_color_frame
- removed link D435_front1_color_optical_frame
- removed link D435_front1_depth_frame
- removed link D435_front1_depth_optical_frame
- removed link D435_front1_gyro_frame
- removed link D435_front1_gyro_optical_frame
- removed link D435_front1_left_ir_frame
- removed link D435_front1_left_ir_optical_frame
- removed link D435_front1_link
- removed link D435_front1_right_ir_frame
- removed link D435_front1_right_ir_optical_frame
- removed link D435_front2_accel_frame
- removed link D435_front2_accel_optical_frame
- removed link D435_front2_bottom_screw_frame
- removed link D435_front2_color_frame
- removed link D435_front2_color_optical_frame
- removed link D435_front2_depth_frame
- removed link D435_front2_depth_optical_frame
- removed link D435_front2_gyro_frame
- removed link D435_front2_gyro_optical_frame
- removed link D435_front2_left_ir_frame
- removed link D435_front2_left_ir_optical_frame
- removed link D435_front2_link
- removed link D435_front2_right_ir_frame
- removed link D435_front2_right_ir_optical_frame
- removed link D435_front3_accel_frame
- removed link D435_front3_accel_optical_frame
- removed link D435_front3_bottom_screw_frame
- removed link D435_front3_color_frame
- removed link D435_front3_color_optical_frame
- removed link D435_front3_depth_frame
- removed link D435_front3_depth_optical_frame
- removed link D435_front3_gyro_frame
- removed link D435_front3_gyro_optical_frame
- removed link D435_front3_left_ir_frame
- removed link D435_front3_left_ir_optical_frame
- removed link D435_front3_link
- removed link D435_front3_right_ir_frame
- removed link D435_front3_right_ir_optical_frame
- removed link D435_left_accel_frame
- removed link D435_left_accel_optical_frame
- removed link D435_left_bottom_screw_frame
- removed link D435_left_color_frame
- removed link D435_left_color_optical_frame
- removed link D435_left_depth_frame
- removed link D435_left_depth_optical_frame
- removed link D435_left_gyro_frame
- removed link D435_left_gyro_optical_frame
- removed link D435_left_left_ir_frame
- removed link D435_left_left_ir_optical_frame
- removed link D435_left_link
- removed link D435_left_right_ir_frame
- removed link D435_left_right_ir_optical_frame
- removed link D435_rear_accel_frame
- removed link D435_rear_accel_optical_frame
- removed link D435_rear_bottom_screw_frame
- removed link D435_rear_color_frame
- removed link D435_rear_color_optical_frame
- removed link D435_rear_depth_frame
- removed link D435_rear_depth_optical_frame
- removed link D435_rear_gyro_frame
- removed link D435_rear_gyro_optical_frame
- removed link D435_rear_left_ir_frame
- removed link D435_rear_left_ir_optical_frame
- removed link D435_rear_link
- removed link D435_rear_right_ir_frame
- removed link D435_rear_right_ir_optical_frame
- removed link D435_right_accel_frame
- removed link D435_right_accel_optical_frame
- removed link D435_right_bottom_screw_frame
- removed link D435_right_color_frame
- removed link D435_right_color_optical_frame
- removed link D435_right_depth_frame
- removed link D435_right_depth_optical_frame
- removed link D435_right_gyro_frame
- removed link D435_right_gyro_optical_frame
- removed link D435_right_left_ir_frame
- removed link D435_right_left_ir_optical_frame
- removed link D435_right_link
- removed link D435_right_right_ir_frame
- removed link D435_right_right_ir_optical_frame
- removed link dagana_1_bottom_link
- removed link dagana_1_tcp
- removed link dagana_1_top_link
- removed link dagana_2_bottom_link
- removed link dagana_2_tcp
- removed link dagana_2_top_link
- removed link elbow_pitch_motor_1
- removed link elbow_pitch_motor_2
- removed link lower_arm_1
- removed link lower_arm_2
- removed link shoulder_pitch_motor_1
- removed link shoulder_pitch_motor_2
- removed link shoulder_yaw_motor_1
- removed link shoulder_yaw_motor_2
- removed link upper_arm1_1
- removed link upper_arm1_2
- removed link upper_arm2_1
- removed link upper_arm2_2
- removed link velodyne
- removed link velodyne_base_link
- removed link wrist_1
- removed link wrist_2
- removed link wrist_pitch_motor_1
- removed link wrist_pitch_motor_2
- added link wheel_1, mass 1.8569388; collision mesh filename=package://kyon_urdf/meshes/collision/mesh_wheel23.stl scale=0.001 0.001 -0.001; visual mesh filename=package://kyon_urdf/meshes/mesh_wheel23.stl scale=0.001 0.001 -0.001
- added link wheel_2, mass 1.8569388; collision mesh filename=package://kyon_urdf/meshes/collision/mesh_wheel23.stl scale=0.001 0.001 0.001; visual mesh filename=package://kyon_urdf/meshes/mesh_wheel23.stl scale=0.001 0.001 0.001
- added link wheel_3, mass 1.8569388; collision mesh filename=package://kyon_urdf/meshes/collision/mesh_wheel23.stl scale=0.001 0.001 -0.001; visual mesh filename=package://kyon_urdf/meshes/mesh_wheel23.stl scale=0.001 0.001 -0.001
- added link wheel_4, mass 1.8569388; collision mesh filename=package://kyon_urdf/meshes/collision/mesh_wheel23.stl scale=0.001 0.001 0.001; visual mesh filename=package://kyon_urdf/meshes/mesh_wheel23.stl scale=0.001 0.001 0.001
- link pelvis: mass 14 -> 32
Joints:
- removed joint D435_front1_accel_joint
- removed joint D435_front1_accel_optical_joint
- removed joint D435_front1_color_joint
- removed joint D435_front1_color_optical_joint
- removed joint D435_front1_depth_joint
- removed joint D435_front1_depth_optical_joint
- removed joint D435_front1_gyro_joint
- removed joint D435_front1_gyro_optical_joint
- removed joint D435_front1_joint
- removed joint D435_front1_left_ir_joint
- removed joint D435_front1_left_ir_optical_joint
- removed joint D435_front1_link_joint
- removed joint D435_front1_right_ir_joint
- removed joint D435_front1_right_ir_optical_joint
- removed joint D435_front2_accel_joint
- removed joint D435_front2_accel_optical_joint
- removed joint D435_front2_color_joint
- removed joint D435_front2_color_optical_joint
- removed joint D435_front2_depth_joint
- removed joint D435_front2_depth_optical_joint
- removed joint D435_front2_gyro_joint
- removed joint D435_front2_gyro_optical_joint
- removed joint D435_front2_joint
- removed joint D435_front2_left_ir_joint
- removed joint D435_front2_left_ir_optical_joint
- removed joint D435_front2_link_joint
- removed joint D435_front2_right_ir_joint
- removed joint D435_front2_right_ir_optical_joint
- removed joint D435_front3_accel_joint
- removed joint D435_front3_accel_optical_joint
- removed joint D435_front3_color_joint
- removed joint D435_front3_color_optical_joint
- removed joint D435_front3_depth_joint
- removed joint D435_front3_depth_optical_joint
- removed joint D435_front3_gyro_joint
- removed joint D435_front3_gyro_optical_joint
- removed joint D435_front3_joint
- removed joint D435_front3_left_ir_joint
- removed joint D435_front3_left_ir_optical_joint
- removed joint D435_front3_link_joint
- removed joint D435_front3_right_ir_joint
- removed joint D435_front3_right_ir_optical_joint
- removed joint D435_left_accel_joint
- removed joint D435_left_accel_optical_joint
- removed joint D435_left_color_joint
- removed joint D435_left_color_optical_joint
- removed joint D435_left_depth_joint
- removed joint D435_left_depth_optical_joint
- removed joint D435_left_gyro_joint
- removed joint D435_left_gyro_optical_joint
- removed joint D435_left_joint
- removed joint D435_left_left_ir_joint
- removed joint D435_left_left_ir_optical_joint
- removed joint D435_left_link_joint
- removed joint D435_left_right_ir_joint
- removed joint D435_left_right_ir_optical_joint
- removed joint D435_rear_accel_joint
- removed joint D435_rear_accel_optical_joint
- removed joint D435_rear_color_joint
- removed joint D435_rear_color_optical_joint
- removed joint D435_rear_depth_joint
- removed joint D435_rear_depth_optical_joint
- removed joint D435_rear_gyro_joint
- removed joint D435_rear_gyro_optical_joint
- removed joint D435_rear_joint
- removed joint D435_rear_left_ir_joint
- removed joint D435_rear_left_ir_optical_joint
- removed joint D435_rear_link_joint
- removed joint D435_rear_right_ir_joint
- removed joint D435_rear_right_ir_optical_joint
- removed joint D435_right_accel_joint
- removed joint D435_right_accel_optical_joint
- removed joint D435_right_color_joint
- removed joint D435_right_color_optical_joint
- removed joint D435_right_depth_joint
- removed joint D435_right_depth_optical_joint
- removed joint D435_right_gyro_joint
- removed joint D435_right_gyro_optical_joint
- removed joint D435_right_joint
- removed joint D435_right_left_ir_joint
- removed joint D435_right_left_ir_optical_joint
- removed joint D435_right_link_joint
- removed joint D435_right_right_ir_joint
- removed joint D435_right_right_ir_optical_joint
- removed joint dagana_1_claw_joint
- removed joint dagana_1_mount_joint
- removed joint dagana_1_tcp_joint
- removed joint dagana_2_claw_joint
- removed joint dagana_2_mount_joint
- removed joint dagana_2_tcp_joint
- removed joint elbow_pitch_1
- removed joint elbow_pitch_2
- removed joint elbow_pitch_stator_1
- removed joint elbow_pitch_stator_2
- removed joint shoulder_pitch_1
- removed joint shoulder_pitch_2
- removed joint shoulder_pitch_stator_1
- removed joint shoulder_pitch_stator_2
- removed joint shoulder_yaw_1
- removed joint shoulder_yaw_2
- removed joint velodyne_base_mount_joint
- removed joint velodyne_base_scan_joint
- removed joint wrist_pitch_1
- removed joint wrist_pitch_2
- removed joint wrist_pitch_stator_1
- removed joint wrist_pitch_stator_2
- removed joint wrist_yaw_1
- removed joint wrist_yaw_2
- added joint wheel_joint_1: type continuous, parent ball_1, child wheel_1, origin xyz=0.0 0.0 0.05 rpy=0.0 0.0 0.0, axis 0 0 -1, limit lower=-1e6 upper=1e6 effort=132 velocity=30.
- added joint wheel_joint_2: type continuous, parent ball_2, child wheel_2, origin xyz=0.0 0.0 -0.05 rpy=0.0 0.0 0.0, axis 0 0 1, limit lower=-1e6 upper=1e6 effort=132 velocity=30.
- added joint wheel_joint_3: type continuous, parent ball_3, child wheel_3, origin xyz=0.0 0.0 0.05 rpy=0.0 0.0 0.0, axis 0 0 -1, limit lower=-1e6 upper=1e6 effort=132 velocity=30.
- added joint wheel_joint_4: type continuous, parent ball_4, child wheel_4, origin xyz=0.0 0.0 -0.05 rpy=0.0 0.0 0.0, axis 0 0 1, limit lower=-1e6 upper=1e6 effort=132 velocity=30.

File: kyon_urdf/urdf/parts/arms.urdf.xacro (robot description, xacro)
@@ -33,5 +33,5 @@
 		<joint name="hand_to_payload_1" type="fixed">
 			<origin xyz="0 0.1 0.0" rpy="0 0 0"/>
-			<parent link="dagana_1_palm_frame"/>
+			<parent link="dagana_1_bottom_link"/>
 			<child link="payload_1"/>
 		</joint>
@@ -52,5 +52,5 @@
 		<joint name="hand_to_payload_2" type="fixed">
 			<origin xyz="0 0.1 0.0" rpy="0 0 0"/>
-			<parent link="dagana_2_palm_frame"/>
+			<parent link="dagana_2_bottom_link"/>
 			<child link="payload_2"/>
 		</joint>

File: kyon_urdf/urdf/parts/kyon_leg.urdf.xacro (robot description, xacro)
@@ -130,6 +130,6 @@
             <origin xyz="${Wheel23_Ox} ${Wheel23_Oy} ${-mirror*Wheel23_Oz}" rpy="${Wheel23_roll} ${Wheel23_pitch} ${Wheel23_yaw}" />
             <axis xyz="0 0 ${mirror}"/>
-            <limit effort="${motor_effort}" velocity="${motor_velocity}" />  <!-- 23 Nm, 1
-            rad/s-->
+            <limit lower="-1e6" upper="1e6" effort="${motor_effort}" velocity="30." />
+            <!--limit effort="${motor_effort}" velocity="${motor_velocity}" /-->
         </joint>
         <link name="wheel_${leg_num}">

Commit message: fixed contact and wheel_4 stiffness

File: kyon_urdf/urdf/gazebo/kyon.gazebo.xacro (robot description, xacro)
@@ -51,138 +51,34 @@
         </gazebo>
         <gazebo reference="ball_1">
-        	<collision>
-		        <surface>
-		            <friction>
-		                <!-- <torsional>
-		                    <coefficient> 1.0 </coefficient>
-		                    <use_patch_radius>true</use_patch_radius>
-		                    <patch_radius>0.2</patch_radius>
-		                </torsional> -->
-		                <ode>
-		                    <mu>1.0</mu>
-		                    <mu2>1.0</mu2>
-		                </ode>
-		                <bullet>
-		                    <friction>1.0</friction>
-		                    <friction2>1.0</friction2>
-		                </bullet>
-		            </friction>
-		            <contact>
-		                <ode>
-		                    <kp>2100000</kp>
-		                    <kd>1</kd>
-		                    <max_vel>100</max_vel>
-		                </ode>
-		                <bullet>
-		                    <soft_cfm>0.007</soft_cfm>
-		                    <soft_erp>0.25</soft_erp>
-		                    <kp>1000000</kp>
-		                    <kd>5</kd>
-		                </bullet>
-		            </contact>
-		        </surface>
-		    </collision>
+        	<kp>1000000.0</kp>
+			<kd>100.0</kd>
+			<mu1>1.0</mu1>
+			<mu2>1.0</mu2>
+			<maxVel>1.0</maxVel>
+			<maxContacts>1</maxContacts>
 		</gazebo>
 		<gazebo reference="ball_2">
-        	<collision>
-		        <surface>
-		            <friction>
-		                <!-- <torsional>
-		                    <coefficient> 1.0 </coefficient>
-		                    <use_patch_radius>true</use_patch_radius>
-		                    <patch_radius>0.2</patch_radius>
-		                </torsional> -->
-		                <ode>
-		                    <mu>1.0</mu>
-		                    <mu2>1.0</mu2>
-		                </ode>
-		                <bullet>
-		                    <friction>1.0</friction>
-		                    <friction2>1.0</friction2>
-		                </bullet>
-		            </friction>
-		            <contact>
-		                <ode>
-		                    <kp>2100000</kp>
-		                    <kd>1</kd>
-		                    <max_vel>100</max_vel>
-		                </ode>
-		                <bullet>
-		                    <soft_cfm>0.007</soft_cfm>
-		                    <soft_erp>0.25</soft_erp>
-		                    <kp>1000000</kp>
-		                    <kd>5</kd>
-		                </bullet>
-		            </contact>
-		        </surface>
-		    </collision>
+        	<kp>1000000.0</kp>
+			<kd>100.0</kd>
+			<mu1>1.0</mu1>
+			<mu2>1.0</mu2>
+			<maxVel>1.0</maxVel>
+			<maxContacts>1</maxContacts>
 		</gazebo>
 		<gazebo reference="ball_3">
-        	<collision>
-		        <surface>
-		            <friction>
-		                <!-- <torsional>
-		                    <coefficient> 1.0 </coefficient>
-		                    <use_patch_radius>true</use_patch_radius>
-		                    <patch_radius>0.2</patch_radius>
-		                </torsional> -->
-		                <ode>
-		                    <mu>1.0</mu>
-		                    <mu2>1.0</mu2>
-		                </ode>
-		                <bullet>
-		                    <friction>1.0</friction>
-		                    <friction2>1.0</friction2>
-		                </bullet>
-		            </friction>
-		            <contact>
-		                <ode>
-		                    <kp>2100000</kp>
-		                    <kd>1</kd>
-		                    <max_vel>100</max_vel>
-		                </ode>
-		                <bullet>
-		                    <soft_cfm>0.007</soft_cfm>
-		                    <soft_erp>0.25</soft_erp>
-		                    <kp>1000000</kp>
-		                    <kd>5</kd>
-		                </bullet>
-		            </contact>
-		        </surface>
-		    </collision>
+        	<kp>1000000.0</kp>
+			<kd>100.0</kd>
+			<mu1>1.0</mu1>
+			<mu2>1.0</mu2>
+			<maxVel>1.0</maxVel>
+			<maxContacts>1</maxContacts>
 		</gazebo>
 		<gazebo reference="ball_4">
-        	<collision>
-		        <surface>
-		            <friction>
-		                <!-- <torsional>
-		                    <coefficient> 1.0 </coefficient>
-		                    <use_patch_radius>true</use_patch_radius>
-		                    <patch_radius>0.2</patch_radius>
-		                </torsional> -->
-		                <ode>
-		                    <mu>1.0</mu>
-		                    <mu2>1.0</mu2>
-		                </ode>
-		                <bullet>
-		                    <friction>1.0</friction>
-		                    <friction2>1.0</friction2>
-		                </bullet>
-		            </friction>
-		            <contact>
-		                <ode>
-		                    <kp>2100000</kp>
-		                    <kd>1</kd>
-		                    <max_vel>100</max_vel>
-		                </ode>
-		                <bullet>
-		                    <soft_cfm>0.007</soft_cfm>
-		                    <soft_erp>0.25</soft_erp>
-		                    <kp>1000000</kp>
-		                    <kd>5</kd>
-		                </bullet>
-		            </contact>
-		        </surface>
-		    </collision>
+        	<kp>1000000.0</kp>
+			<kd>100.0</kd>
+			<mu1>1.0</mu1>
+			<mu2>1.0</mu2>
+			<maxVel>1.0</maxVel>
+			<maxContacts>1</maxContacts>
 		</gazebo>
     </xacro:if>
@@ -229,4 +125,38 @@
         </gazebo>
     </xacro:if>
+    <xacro:if value="${ADD_WHEELS}">
+        <gazebo reference="wheel_1">
+            <kp>1000000.0</kp>
+			<kd>100.0</kd>
+			<mu1>1.0</mu1>
+			<mu2>1.0</mu2>
+			<maxVel>1.0</maxVel>
+			<maxContacts>1</maxContacts>
+	    </gazebo>
+	    <gazebo reference="wheel_2">
+            <kp>1000000.0</kp>
+			<kd>100.0</kd>
+			<mu1>1.0</mu1>
+			<mu2>1.0</mu2>
+			<maxVel>1.0</maxVel>
+			<maxContacts>1</maxContacts>
+	    </gazebo>
+	    <gazebo reference="wheel_3">
+            <kp>1000000.0</kp>
+			<kd>100.0</kd>
+			<mu1>1.0</mu1>
+			<mu2>1.0</mu2>
+			<maxVel>1.0</maxVel>
+			<maxContacts>1</maxContacts>
+	    </gazebo>
+	    <gazebo reference="wheel_4">
+            <kp>1000000.0</kp>
+			<kd>100.0</kd>
+			<mu1>1.0</mu1>
+			<mu2>1.0</mu2>
+			<maxVel>1.0</maxVel>
+			<maxContacts>1</maxContacts>
+	    </gazebo>
+	</xacro:if>
 	<xacro:if value="${ADD_FT_SENSORS}">
 		<xacro:include filename="$(find kyon_urdf)/urdf/gazebo/ft_sensors.gazebo.xacro" />

File: kyon_urdf/urdf/gazebo/xbot.gazebo.xacro (robot description, xacro)
@@ -41,5 +41,5 @@
             <pid name="hip_pitch_4"  profile="big_mot"/>
             <pid name="knee_pitch_4"   profile="big_mot"/>
-            <pid name="wheel_joint_1" profile="wheel"/>
+            <pid name="wheel_joint_4" profile="wheel"/>
         </pid>
     </plugin>
