Commit message: fixed floating joint to have base link as child
Signed-off-by: Andrea Patrizi <andreapatrizi1b6e6@gmail.com>

File: kyon_urdf/urdf/kyon.urdf.xacro (robot description, xacro)
@@ -27,5 +27,5 @@
 	<joint name="reference" type="floating">
 		<parent link="world"/>
-		<child link="pelvis"/>
+		<child link="base_link"/>
 	</joint>
 </xacro:if>

File: kyon_urdf/urdf/kyon_robot.urdf.xacro (robot description, xacro)
@@ -13,5 +13,5 @@
       <joint name="reference" type="fixed">
       <parent link="world"/>
-      <child link="pelvis"/>
+      <child link="base_link"/>
     </joint>
   </xacro:unless>

Commit message: fixed wrong mesh path in case of use with RViz
Signed-off-by: Andrea Patrizi <andreapatrizi1b6e6@gmail.com>

File: kyon_urdf/urdf/kyon.urdf.xacro (robot description, xacro)
@@ -5,4 +5,15 @@
 <xacro:arg name="kyon_root" default="$(find kyon_urdf)" />
 <xacro:property name="KYON_ROOT" value="$(arg kyon_root)" />
+<!-- setting use_abs_mesh_paths should be kept to false
+for use with tools like RViz, which does not accept plain
+abolute paths for mesh paths-->
+<xacro:arg name="use_abs_mesh_paths" default="false" />
+<xacro:property name="USE_ABS_MESH_PATHS" value="$(arg use_abs_mesh_paths)" />
+<xacro:if value="${USE_ABS_MESH_PATHS}">
+  <xacro:property name="MESH_PATH" value="${KYON_ROOT}/meshes" />
+</xacro:if>
+<xacro:unless value="${USE_ABS_MESH_PATHS}">
+  <xacro:property name="MESH_PATH" value="package://kyon_urdf/meshes" />
+</xacro:unless>
 <xacro:arg name="config" default="${KYON_ROOT}/urdf/config/kyon.urdf.xacro"/>
 <!-- ************ MODEL CONFIGURATION ************ -->

File: kyon_urdf/urdf/kyon_robot.urdf.xacro (robot description, xacro)
@@ -5,4 +5,15 @@
   <xacro:arg name="kyon_root" default="$(find kyon_urdf)" />
   <xacro:property name="KYON_ROOT" value="$(arg kyon_root)" />
+  <!-- setting use_abs_mesh_paths should be kept to false
+  for use with tools like RViz, which does not accept plain
+  abolute paths for mesh paths-->
+  <xacro:arg name="use_abs_mesh_paths" default="false" />
+  <xacro:property name="USE_ABS_MESH_PATHS" value="$(arg use_abs_mesh_paths)" />
+  <xacro:if value="${USE_ABS_MESH_PATHS}">
+    <xacro:property name="MESH_PATH" value="${KYON_ROOT}/meshes" />
+  </xacro:if>
+  <xacro:unless value="${USE_ABS_MESH_PATHS}">
+    <xacro:property name="MESH_PATH" value="package://kyon_urdf/meshes" />
+  </xacro:unless>
   <xacro:include filename="${KYON_ROOT}/urdf/kyon.urdf.xacro" />
   <xacro:include filename="${KYON_ROOT}/urdf/gazebo/kyon.gazebo.xacro" />

File: kyon_urdf/urdf/parts/kyon_leg.urdf.xacro (robot description, xacro)
@@ -142,5 +142,5 @@
                 <origin xyz="0.0 0.0 0.0" rpy="0.0 0.0 0.0" />
                 <geometry>
-                    <mesh filename="${KYON_ROOT}/meshes/mesh_wheel23.stl"
+                    <mesh filename="${MESH_PATH}/mesh_wheel23.stl"
                         scale="0.001 0.001 ${mirror*0.001}" />
                 </geometry>
@@ -150,5 +150,5 @@
                 <origin xyz="0 0 0" rpy="0 0 0" />
                 <geometry>
-                    <mesh filename="${KYON_ROOT}/meshes/collision/mesh_wheel23.stl"
+                    <mesh filename="${MESH_PATH}/collision/mesh_wheel23.stl"
                         scale="0.001 0.001 ${mirror*0.001}" />
                 </geometry>

Commit message: added flag to allow use with manual path and rviz

File: kyon_urdf/urdf/kyon.urdf.xacro (robot description, xacro)
@@ -9,10 +9,17 @@
 abolute paths for mesh paths-->
 <xacro:arg name="use_abs_mesh_paths" default="false" />
+<xacro:arg name="use_local_filesys_for_meshes" default="false" />
 <xacro:property name="USE_ABS_MESH_PATHS" value="$(arg use_abs_mesh_paths)" />
+<xacro:property name="USE_LOCAL_FILESYS_FOR_MESHES" value="$(arg use_local_filesys_for_meshes)" />
 <xacro:if value="${USE_ABS_MESH_PATHS}">
-  <xacro:property name="MESH_PATH" value="${KYON_ROOT}/meshes" />
-</xacro:if>
+	<xacro:if value="${USE_LOCAL_FILESYS_FOR_MESHES}">
+	<xacro:property name="MESH_PATH" value="file://${KYON_ROOT}/meshes" />
+	</xacro:if>
+	<xacro:unless value="${USE_ABS_MESH_PATHS}">
+	<xacro:property name="MESH_PATH" value="${KYON_ROOT}/meshes" />
+	</xacro:unless>
+	</xacro:if>
 <xacro:unless value="${USE_ABS_MESH_PATHS}">
-  <xacro:property name="MESH_PATH" value="package://kyon_urdf/meshes" />
+<xacro:property name="MESH_PATH" value="package://kyon_urdf/meshes" />
 </xacro:unless>
 <xacro:arg name="config" default="${KYON_ROOT}/urdf/config/kyon.urdf.xacro"/>

Commit message: adjust urdf floating base height

File: kyon_urdf/urdf/kyon.urdf.xacro (robot description, xacro)
@@ -13,4 +13,5 @@
 		<parent link="world"/>
 		<child link="pelvis"/>
+		<origin xyz="0 0 0.6"/>
 	</joint>
 </xacro:if>
