Commit message: corrected mass

File: kyon_urdf/urdf/kyon.urdf (robot description, URDF)
Before this commit: robot kyon, 31 links, 30 joints
Links:
- removed link wheel_1
- removed link wheel_2
- removed link wheel_3
- removed link wheel_4
- added link D435_front1_accel_frame
- added link D435_front1_accel_optical_frame
- added link D435_front1_bottom_screw_frame
- added link D435_front1_color_frame
- added link D435_front1_color_optical_frame
- added link D435_front1_depth_frame
- added link D435_front1_depth_optical_frame
- added link D435_front1_gyro_frame
- added link D435_front1_gyro_optical_frame
- added link D435_front1_left_ir_frame
- added link D435_front1_left_ir_optical_frame
- added link D435_front1_link, mass 0.564; collision box size=0.02505 0.09 0.025; visual mesh filename=package://realsense2_description/meshes/d435.dae
- added link D435_front1_right_ir_frame
- added link D435_front1_right_ir_optical_frame
- added link D435_front2_accel_frame
- added link D435_front2_accel_optical_frame
- added link D435_front2_bottom_screw_frame
- added link D435_front2_color_frame
- added link D435_front2_color_optical_frame
- added link D435_front2_depth_frame
- added link D435_front2_depth_optical_frame
- added link D435_front2_gyro_frame
- added link D435_front2_gyro_optical_frame
- added link D435_front2_left_ir_frame
- added link D435_front2_left_ir_optical_frame
- added link D435_front2_link, mass 0.564; collision box size=0.02505 0.09 0.025; visual mesh filename=package://realsense2_description/meshes/d435.dae
- added link D435_front2_right_ir_frame
- added link D435_front2_right_ir_optical_frame
- added link D435_front3_accel_frame
- added link D435_front3_accel_optical_frame
- added link D435_front3_bottom_screw_frame
- added link D435_front3_color_frame
- added link D435_front3_color_optical_frame
- added link D435_front3_depth_frame
- added link D435_front3_depth_optical_frame
- added link D435_front3_gyro_frame
- added link D435_front3_gyro_optical_frame
- added link D435_front3_left_ir_frame
- added link D435_front3_left_ir_optical_frame
- added link D435_front3_link, mass 0.564; collision box size=0.02505 0.09 0.025; visual mesh filename=package://realsense2_description/meshes/d435.dae
- added link D435_front3_right_ir_frame
- added link D435_front3_right_ir_optical_frame
- added link D435_left_accel_frame
- added link D435_left_accel_optical_frame
- added link D435_left_bottom_screw_frame
- added link D435_left_color_frame
- added link D435_left_color_optical_frame
- added link D435_left_depth_frame
- added link D435_left_depth_optical_frame
- added link D435_left_gyro_frame
- added link D435_left_gyro_optical_frame
- added link D435_left_left_ir_frame
- added link D435_left_left_ir_optical_frame
- added link D435_left_link, mass 0.564; collision box size=0.02505 0.09 0.025; visual mesh filename=package://realsense2_description/meshes/d435.dae
- added link D435_left_right_ir_frame
- added link D435_left_right_ir_optical_frame
- added link D435_rear_accel_frame
- added link D435_rear_accel_optical_frame
- added link D435_rear_bottom_screw_frame
- added link D435_rear_color_frame
- added link D435_rear_color_optical_frame
- added link D435_rear_depth_frame
- added link D435_rear_depth_optical_frame
- added link D435_rear_gyro_frame
- added link D435_rear_gyro_optical_frame
- added link D435_rear_left_ir_frame
- added link D435_rear_left_ir_optical_frame
- added link D435_rear_link, mass 0.564; collision box size=0.02505 0.09 0.025; visual mesh filename=package://realsense2_description/meshes/d435.dae
- added link D435_rear_right_ir_frame
- added link D435_rear_right_ir_optical_frame
- added link D435_right_accel_frame
- added link D435_right_accel_optical_frame
- added link D435_right_bottom_screw_frame
- added link D435_right_color_frame
- added link D435_right_color_optical_frame
- added link D435_right_depth_frame
- added link D435_right_depth_optical_frame
- added link D435_right_gyro_frame
- added link D435_right_gyro_optical_frame
- added link D435_right_left_ir_frame
- added link D435_right_left_ir_optical_frame
- added link D435_right_link, mass 0.564; collision box size=0.02505 0.09 0.025; visual mesh filename=package://realsense2_description/meshes/d435.dae
- added link D435_right_right_ir_frame
- added link D435_right_right_ir_optical_frame
- added link ball_arm_1, mass 0.1; collision sphere radius=0.05; visual sphere radius=0.05
- added link ball_arm_2, mass 0.1; collision sphere radius=0.05; visual sphere radius=0.05
- added link elbow_pitch_motor_1, mass 0.8; collision cylinder length=0.1 radius=0.07; visual cylinder length=0.1 radius=0.07
- added link elbow_pitch_motor_2, mass 0.8; collision cylinder length=0.1 radius=0.07; visual cylinder length=0.1 radius=0.07
- added link lower_arm_1, mass 1.0; collision box size=0.32 0.1 0.1; visual box size=0.32 0.1 0.1
- added link lower_arm_2, mass 1.0; collision box size=0.32 0.1 0.1; visual box size=0.32 0.1 0.1
- added link shoulder_pitch_motor_1, mass 0.8; collision cylinder length=0.1 radius=0.07; visual cylinder length=0.1 radius=0.07
- added link shoulder_pitch_motor_2, mass 0.8; collision cylinder length=0.1 radius=0.07; visual cylinder length=0.1 radius=0.07
- added link shoulder_yaw_motor_1, mass 1.6; collision cylinder length=0.1 radius=0.07; visual cylinder length=0.1 radius=0.07
- added link shoulder_yaw_motor_2, mass 1.6; collision cylinder length=0.1 radius=0.07; visual cylinder length=0.1 radius=0.07
- added link upper_arm1_1, mass 0.77; collision box size=0.3 0.05 0.05; visual box size=0.3 0.05 0.05
- added link upper_arm1_2, mass 0.77; collision box size=0.3 0.05 0.05; visual box size=0.3 0.05 0.05
- added link upper_arm2_1, mass 2.0; collision box size=0.1 0.05 0.05; visual box size=0.1 0.05 0.05
- added link upper_arm2_2, mass 2.0; collision box size=0.1 0.05 0.05; visual box size=0.1 0.05 0.05
- added link velodyne, mass 0.01; collision sphere radius=0; visual mesh filename=package://velodyne_description/meshes/VLP16_scan.dae
- added link velodyne_base_link, mass 0.83; collision cylinder length=0.0717 radius=0.0516; visual mesh filename=package://velodyne_description/meshes/VLP16_base_1.dae
- added link wrist_1, mass 0.63; collision cylinder length=0.05 radius=0.035; visual cylinder length=0.016666666666666666 radius=0.07
- added link wrist_2, mass 0.63; collision cylinder length=0.05 radius=0.035; visual cylinder length=0.016666666666666666 radius=0.07
- added link wrist_pitch_motor_1, mass 0.63; collision cylinder length=0.1 radius=0.07; visual cylinder length=0.05 radius=0.035
- added link wrist_pitch_motor_2, mass 0.63; collision cylinder length=0.1 radius=0.07; visual cylinder length=0.05 radius=0.035
- link pelvis: mass 32 -> 14
Joints:
- removed joint wheel_joint_1
- removed joint wheel_joint_2
- removed joint wheel_joint_3
- removed joint wheel_joint_4
- added joint D435_front1_accel_joint: type fixed, parent D435_front1_link, child D435_front1_accel_frame, origin xyz=-0.00174 0.00552 0.0176 rpy=0 0 0
- added joint D435_front1_accel_optical_joint: type fixed, parent D435_front1_accel_frame, child D435_front1_accel_optical_frame, origin xyz=0 0 0 rpy=-1.5707963267948966 0 -1.5707963267948966
- added joint D435_front1_color_joint: type fixed, parent D435_front1_depth_frame, child D435_front1_color_frame, origin xyz=0 0.015 0 rpy=0 0 0
- added joint D435_front1_color_optical_joint: type fixed, parent D435_front1_color_frame, child D435_front1_color_optical_frame, origin xyz=0 0 0 rpy=-1.5707963267948966 0 -1.5707963267948966
- added joint D435_front1_depth_joint: type fixed, parent D435_front1_link, child D435_front1_depth_frame, origin xyz=0 0 0 rpy=0 0 0
- added joint D435_front1_depth_optical_joint: type fixed, parent D435_front1_depth_frame, child D435_front1_depth_optical_frame, origin xyz=0 0 0 rpy=-1.5707963267948966 0 -1.5707963267948966
- added joint D435_front1_gyro_joint: type fixed, parent D435_front1_link, child D435_front1_gyro_frame, origin xyz=-0.00174 0.00552 0.0176 rpy=0 0 0
- added joint D435_front1_gyro_optical_joint: type fixed, parent D435_front1_gyro_frame, child D435_front1_gyro_optical_frame, origin xyz=0 0 0 rpy=-1.5707963267948966 0 -1.5707963267948966
- added joint D435_front1_joint: type fixed, parent pelvis, child D435_front1_bottom_screw_frame, origin xyz=0.40 -0.08 0 rpy=-1.57 0 0.34
- added joint D435_front1_left_ir_joint: type fixed, parent D435_front1_depth_frame, child D435_front1_left_ir_frame, origin xyz=0 0.0 0 rpy=0 0 0
- added joint D435_front1_left_ir_optical_joint: type fixed, parent D435_front1_left_ir_frame, child D435_front1_left_ir_optical_frame, origin xyz=0 0 0 rpy=-1.5707963267948966 0 -1.5707963267948966
- added joint D435_front1_link_joint: type fixed, parent D435_front1_bottom_screw_frame, child D435_front1_link, origin xyz=0 0.0175 0.0125 rpy=0 0 0
- added joint D435_front1_right_ir_joint: type fixed, parent D435_front1_depth_frame, child D435_front1_right_ir_frame, origin xyz=0 -0.05 0 rpy=0 0 0
- added joint D435_front1_right_ir_optical_joint: type fixed, parent D435_front1_right_ir_frame, child D435_front1_right_ir_optical_frame, origin xyz=0 0 0 rpy=-1.5707963267948966 0 -1.5707963267948966
- added joint D435_front2_accel_joint: type fixed, parent D435_front2_link, child D435_front2_accel_frame, origin xyz=-0.00174 0.00552 0.0176 rpy=0 0 0
- added joint D435_front2_accel_optical_joint: type fixed, parent D435_front2_accel_frame, child D435_front2_accel_optical_frame, origin xyz=0 0 0 rpy=-1.5707963267948966 0 -1.5707963267948966
- added joint D435_front2_color_joint: type fixed, parent D435_front2_depth_frame, child D435_front2_color_frame, origin xyz=0 0.015 0 rpy=0 0 0
- added joint D435_front2_color_optical_joint: type fixed, parent D435_front2_color_frame, child D435_front2_color_optical_frame, origin xyz=0 0 0 rpy=-1.5707963267948966 0 -1.5707963267948966
- added joint D435_front2_depth_joint: type fixed, parent D435_front2_link, child D435_front2_depth_frame, origin xyz=0 0 0 rpy=0 0 0
- added joint D435_front2_depth_optical_joint: type fixed, parent D435_front2_depth_frame, child D435_front2_depth_optical_frame, origin xyz=0 0 0 rpy=-1.5707963267948966 0 -1.5707963267948966
- added joint D435_front2_gyro_joint: type fixed, parent D435_front2_link, child D435_front2_gyro_frame, origin xyz=-0.00174 0.00552 0.0176 rpy=0 0 0
- added joint D435_front2_gyro_optical_joint: type fixed, parent D435_front2_gyro_frame, child D435_front2_gyro_optical_frame, origin xyz=0 0 0 rpy=-1.5707963267948966 0 -1.5707963267948966
- added joint D435_front2_joint: type fixed, parent pelvis, child D435_front2_bottom_screw_frame, origin xyz=0.40 0.08 0 rpy=-1.57 0 -0.34
- added joint D435_front2_left_ir_joint: type fixed, parent D435_front2_depth_frame, child D435_front2_left_ir_frame, origin xyz=0 0.0 0 rpy=0 0 0
- added joint D435_front2_left_ir_optical_joint: type fixed, parent D435_front2_left_ir_frame, child D435_front2_left_ir_optical_frame, origin xyz=0 0 0 rpy=-1.5707963267948966 0 -1.5707963267948966
- added joint D435_front2_link_joint: type fixed, parent D435_front2_bottom_screw_frame, child D435_front2_link, origin xyz=0 0.0175 0.0125 rpy=0 0 0
- added joint D435_front2_right_ir_joint: type fixed, parent D435_front2_depth_frame, child D435_front2_right_ir_frame, origin xyz=0 -0.05 0 rpy=0 0 0
- added joint D435_front2_right_ir_optical_joint: type fixed, parent D435_front2_right_ir_frame, child D435_front2_right_ir_optical_frame, origin xyz=0 0 0 rpy=-1.5707963267948966 0 -1.5707963267948966
- added joint D435_front3_accel_joint: type fixed, parent D435_front3_link, child D435_front3_accel_frame, origin xyz=-0.00174 0.00552 0.0176 rpy=0 0 0
- added joint D435_front3_accel_optical_joint: type fixed, parent D435_front3_accel_frame, child D435_front3_accel_optical_frame, origin xyz=0 0 0 rpy=-1.5707963267948966 0 -1.5707963267948966
- added joint D435_front3_color_joint: type fixed, parent D435_front3_depth_frame, child D435_front3_color_frame, origin xyz=0 0.015 0 rpy=0 0 0
- added joint D435_front3_color_optical_joint: type fixed, parent D435_front3_color_frame, child D435_front3_color_optical_frame, origin xyz=0 0 0 rpy=-1.5707963267948966 0 -1.5707963267948966
- added joint D435_front3_depth_joint: type fixed, parent D435_front3_link, child D435_front3_depth_frame, origin xyz=0 0 0 rpy=0 0 0
- added joint D435_front3_depth_optical_joint: type fixed, parent D435_front3_depth_frame, child D435_front3_depth_optical_frame, origin xyz=0 0 0 rpy=-1.5707963267948966 0 -1.5707963267948966
- added joint D435_front3_gyro_joint: type fixed, parent D435_front3_link, child D435_front3_gyro_frame, origin xyz=-0.00174 0.00552 0.0176 rpy=0 0 0
- added joint D435_front3_gyro_optical_joint: type fixed, parent D435_front3_gyro_frame, child D435_front3_gyro_optical_frame, origin xyz=0 0 0 rpy=-1.5707963267948966 0 -1.5707963267948966
- added joint D435_front3_joint: type fixed, parent pelvis, child D435_front3_bottom_screw_frame, origin xyz=0.37 0 -0.11 rpy=0 0.75 0
- added joint D435_front3_left_ir_joint: type fixed, parent D435_front3_depth_frame, child D435_front3_left_ir_frame, origin xyz=0 0.0 0 rpy=0 0 0
- added joint D435_front3_left_ir_optical_joint: type fixed, parent D435_front3_left_ir_frame, child D435_front3_left_ir_optical_frame, origin xyz=0 0 0 rpy=-1.5707963267948966 0 -1.5707963267948966
- added joint D435_front3_link_joint: type fixed, parent D435_front3_bottom_screw_frame, child D435_front3_link, origin xyz=0 0.0175 0.0125 rpy=0 0 0
- added joint D435_front3_right_ir_joint: type fixed, parent D435_front3_depth_frame, child D435_front3_right_ir_frame, origin xyz=0 -0.05 0 rpy=0 0 0
- added joint D435_front3_right_ir_optical_joint: type fixed, parent D435_front3_right_ir_frame, child D435_front3_right_ir_optical_frame, origin xyz=0 0 0 rpy=-1.5707963267948966 0 -1.5707963267948966
- added joint D435_left_accel_joint: type fixed, parent D435_left_link, child D435_left_accel_frame, origin xyz=-0.00174 0.00552 0.0176 rpy=0 0 0
- added joint D435_left_accel_optical_joint: type fixed, parent D435_left_accel_frame, child D435_left_accel_optical_frame, origin xyz=0 0 0 rpy=-1.5707963267948966 0 -1.5707963267948966
- added joint D435_left_color_joint: type fixed, parent D435_left_depth_frame, child D435_left_color_frame, origin xyz=0 0.015 0 rpy=0 0 0
- added joint D435_left_color_optical_joint: type fixed, parent D435_left_color_frame, child D435_left_color_optical_frame, origin xyz=0 0 0 rpy=-1.5707963267948966 0 -1.5707963267948966
- added joint D435_left_depth_joint: type fixed, parent D435_left_link, child D435_left_depth_frame, origin xyz=0 0 0 rpy=0 0 0
- added joint D435_left_depth_optical_joint: type fixed, parent D435_left_depth_frame, child D435_left_depth_optical_frame, origin xyz=0 0 0 rpy=-1.5707963267948966 0 -1.5707963267948966
- added joint D435_left_gyro_joint: type fixed, parent D435_left_link, child D435_left_gyro_frame, origin xyz=-0.00174 0.00552 0.0176 rpy=0 0 0
- added joint D435_left_gyro_optical_joint: type fixed, parent D435_left_gyro_frame, child D435_left_gyro_optical_frame, origin xyz=0 0 0 rpy=-1.5707963267948966 0 -1.5707963267948966
- added joint D435_left_joint: type fixed, parent pelvis, child D435_left_bottom_screw_frame, origin xyz=-0.175 0.22 0 rpy=0 0.35 1.57
- added joint D435_left_left_ir_joint: type fixed, parent D435_left_depth_frame, child D435_left_left_ir_frame, origin xyz=0 0.0 0 rpy=0 0 0
- added joint D435_left_left_ir_optical_joint: type fixed, parent D435_left_left_ir_frame, child D435_left_left_ir_optical_frame, origin xyz=0 0 0 rpy=-1.5707963267948966 0 -1.5707963267948966
- added joint D435_left_link_joint: type fixed, parent D435_left_bottom_screw_frame, child D435_left_link, origin xyz=0 0.0175 0.0125 rpy=0 0 0
- added joint D435_left_right_ir_joint: type fixed, parent D435_left_depth_frame, child D435_left_right_ir_frame, origin xyz=0 -0.05 0 rpy=0 0 0
- added joint D435_left_right_ir_optical_joint: type fixed, parent D435_left_right_ir_frame, child D435_left_right_ir_optical_frame, origin xyz=0 0 0 rpy=-1.5707963267948966 0 -1.5707963267948966
- added joint D435_rear_accel_joint: type fixed, parent D435_rear_link, child D435_rear_accel_frame, origin xyz=-0.00174 0.00552 0.0176 rpy=0 0 0
- added joint D435_rear_accel_optical_joint: type fixed, parent D435_rear_accel_frame, child D435_rear_accel_optical_frame, origin xyz=0 0 0 rpy=-1.5707963267948966 0 -1.5707963267948966
- added joint D435_rear_color_joint: type fixed, parent D435_rear_depth_frame, child D435_rear_color_frame, origin xyz=0 0.015 0 rpy=0 0 0
- added joint D435_rear_color_optical_joint: type fixed, parent D435_rear_color_frame, child D435_rear_color_optical_frame, origin xyz=0 0 0 rpy=-1.5707963267948966 0 -1.5707963267948966
- added joint D435_rear_depth_joint: type fixed, parent D435_rear_link, child D435_rear_depth_frame, origin xyz=0 0 0 rpy=0 0 0
- added joint D435_rear_depth_optical_joint: type fixed, parent D435_rear_depth_frame, child D435_rear_depth_optical_frame, origin xyz=0 0 0 rpy=-1.5707963267948966 0 -1.5707963267948966
- added joint D435_rear_gyro_joint: type fixed, parent D435_rear_link, child D435_rear_gyro_frame, origin xyz=-0.00174 0.00552 0.0176 rpy=0 0 0
- added joint D435_rear_gyro_optical_joint: type fixed, parent D435_rear_gyro_frame, child D435_rear_gyro_optical_frame, origin xyz=0 0 0 rpy=-1.5707963267948966 0 -1.5707963267948966
- added joint D435_rear_joint: type fixed, parent pelvis, child D435_rear_bottom_screw_frame, origin xyz=-0.39 0 0 rpy=0 0.35 3.14
- added joint D435_rear_left_ir_joint: type fixed, parent D435_rear_depth_frame, child D435_rear_left_ir_frame, origin xyz=0 0.0 0 rpy=0 0 0
- added joint D435_rear_left_ir_optical_joint: type fixed, parent D435_rear_left_ir_frame, child D435_rear_left_ir_optical_frame, origin xyz=0 0 0 rpy=-1.5707963267948966 0 -1.5707963267948966
- added joint D435_rear_link_joint: type fixed, parent D435_rear_bottom_screw_frame, child D435_rear_link, origin xyz=0 0.0175 0.0125 rpy=0 0 0
- added joint D435_rear_right_ir_joint: type fixed, parent D435_rear_depth_frame, child D435_rear_right_ir_frame, origin xyz=0 -0.05 0 rpy=0 0 0
- added joint D435_rear_right_ir_optical_joint: type fixed, parent D435_rear_right_ir_frame, child D435_rear_right_ir_optical_frame, origin xyz=0 0 0 rpy=-1.5707963267948966 0 -1.5707963267948966
- added joint D435_right_accel_joint: type fixed, parent D435_right_link, child D435_right_accel_frame, origin xyz=-0.00174 0.00552 0.0176 rpy=0 0 0
- added joint D435_right_accel_optical_joint: type fixed, parent D435_right_accel_frame, child D435_right_accel_optical_frame, origin xyz=0 0 0 rpy=-1.5707963267948966 0 -1.5707963267948966
- added joint D435_right_color_joint: type fixed, parent D435_right_depth_frame, child D435_right_color_frame, origin xyz=0 0.015 0 rpy=0 0 0
- added joint D435_right_color_optical_joint: type fixed, parent D435_right_color_frame, child D435_right_color_optical_frame, origin xyz=0 0 0 rpy=-1.5707963267948966 0 -1.5707963267948966
- added joint D435_right_depth_joint: type fixed, parent D435_right_link, child D435_right_depth_frame, origin xyz=0 0 0 rpy=0 0 0
- added joint D435_right_depth_optical_joint: type fixed, parent D435_right_depth_frame, child D435_right_depth_optical_frame, origin xyz=0 0 0 rpy=-1.5707963267948966 0 -1.5707963267948966
- added joint D435_right_gyro_joint: type fixed, parent D435_right_link, child D435_right_gyro_frame, origin xyz=-0.00174 0.00552 0.0176 rpy=0 0 0
- added joint D435_right_gyro_optical_joint: type fixed, parent D435_right_gyro_frame, child D435_right_gyro_optical_frame, origin xyz=0 0 0 rpy=-1.5707963267948966 0 -1.5707963267948966
- added joint D435_right_joint: type fixed, parent pelvis, child D435_right_bottom_screw_frame, origin xyz=-0.175 -0.22 0 rpy=0 0.35 -1.57
- added joint D435_right_left_ir_joint: type fixed, parent D435_right_depth_frame, child D435_right_left_ir_frame, origin xyz=0 0.0 0 rpy=0 0 0
- added joint D435_right_left_ir_optical_joint: type fixed, parent D435_right_left_ir_frame, child D435_right_left_ir_optical_frame, origin xyz=0 0 0 rpy=-1.5707963267948966 0 -1.5707963267948966
- added joint D435_right_link_joint: type fixed, parent D435_right_bottom_screw_frame, child D435_right_link, origin xyz=0 0.0175 0.0125 rpy=0 0 0
- added joint D435_right_right_ir_joint: type fixed, parent D435_right_depth_frame, child D435_right_right_ir_frame, origin xyz=0 -0.05 0 rpy=0 0 0
- added joint D435_right_right_ir_optical_joint: type fixed, parent D435_right_right_ir_frame, child D435_right_right_ir_optical_frame, origin xyz=0 0 0 rpy=-1.5707963267948966 0 -1.5707963267948966
- added joint elbow_pitch_1: type revolute, parent elbow_pitch_motor_1, child upper_arm1_1, origin xyz=0.0 0.0 0.0 rpy=0.0 0.0 0.0, axis 0 0 1, limit lower=-2.4056 upper=2.4056 effort=132 velocity=15.5
- added joint elbow_pitch_2: type revolute, parent elbow_pitch_motor_2, child upper_arm1_2, origin xyz=0.0 0.0 0.0 rpy=0.0 0.0 0.0, axis 0 0 1, limit lower=-2.3266 upper=2.3266 effort=132 velocity=15.5
- added joint elbow_pitch_stator_1: type fixed, parent lower_arm_1, child elbow_pitch_motor_1, origin xyz=0.32 0.0 0.0 rpy=0.0 0.0 0.0
- added joint elbow_pitch_stator_2: type fixed, parent lower_arm_2, child elbow_pitch_motor_2, origin xyz=0.32 0.0 0.0 rpy=0.0 0.0 0.0
- added joint hand_joint_1: type fixed, parent wrist_1, child ball_arm_1, origin xyz=0 0 0.05 rpy=0 0 0
- added joint hand_joint_2: type fixed, parent wrist_2, child ball_arm_2, origin xyz=0 0 0.05 rpy=0 0 0
- added joint shoulder_pitch_1: type revolute, parent shoulder_pitch_motor_1, child lower_arm_1, origin xyz=0.0 0.0 0.0 rpy=0.0 0.0 -1.57079632679, axis 0 0 1, limit lower=-2.4056 upper=2.4056 effort=132 velocity=15.5
- added joint shoulder_pitch_2: type revolute, parent shoulder_pitch_motor_2, child lower_arm_2, origin xyz=0.0 0.0 0.0 rpy=0.0 0.0 -1.57079632679, axis 0 0 1, limit lower=-2.3266 upper=2.3266 effort=132 velocity=15.5
- added joint shoulder_pitch_stator_1: type fixed, parent shoulder_yaw_motor_1, child shoulder_pitch_motor_1, origin xyz=0.0 0.0 0.05 rpy=-1.57079632679 0.0 0.0
- added joint shoulder_pitch_stator_2: type fixed, parent shoulder_yaw_motor_2, child shoulder_pitch_motor_2, origin xyz=0.0 0.0 0.05 rpy=-1.57079632679 0.0 0.0
- added joint shoulder_yaw_1: type revolute, parent pelvis, child shoulder_yaw_motor_1, origin xyz=0.30000000000000004 0.175 0.1 rpy=-0.0 0.0 0.0, axis 0 0 1, limit lower=-3.312 upper=3.312 effort=132 velocity=15.5
- added joint shoulder_yaw_2: type revolute, parent pelvis, child shoulder_yaw_motor_2, origin xyz=0.30000000000000004 -0.175 0.1 rpy=0.0 0.0 0.0, axis 0 0 1, limit lower=-3.3458 upper=3.3458 effort=132 velocity=15.5
- added joint velodyne_base_mount_joint: type fixed, parent pelvis, child velodyne_base_link, origin xyz=0.36 0 0.11 rpy=0 0 0
- added joint velodyne_base_scan_joint: type fixed, parent velodyne_base_link, child velodyne, origin xyz=0 0 0.0377 rpy=0 0 0
- added joint wrist_pitch_1: type revolute, parent wrist_pitch_motor_1, child upper_arm2_1, origin xyz=0.0 0.0 0.0 rpy=0.0 0.0 0.0, axis 0 0 1, limit lower=-2.4056 upper=2.4056 effort=132 velocity=15.5
- added joint wrist_pitch_2: type revolute, parent wrist_pitch_motor_2, child upper_arm2_2, origin xyz=0.0 0.0 0.0 rpy=0.0 0.0 0.0, axis 0 0 1, limit lower=-2.3266 upper=2.3266 effort=132 velocity=15.5
- added joint wrist_pitch_stator_1: type fixed, parent upper_arm1_1, child wrist_pitch_motor_1, origin xyz=0.3 0.0 0.0 rpy=0.0 0.0 0.0
- added joint wrist_pitch_stator_2: type fixed, parent upper_arm1_2, child wrist_pitch_motor_2, origin xyz=0.3 0.0 0.0 rpy=0.0 0.0 0.0
- added joint wrist_yaw_1: type revolute, parent upper_arm2_1, child wrist_1, origin xyz=0.1 0.0 0.0 rpy=0.0 1.57079632679 0.0, axis 0 0 1, limit lower=-2.4056 upper=2.4056 effort=132 velocity=15.5
- added joint wrist_yaw_2: type revolute, parent upper_arm2_2, child wrist_2, origin xyz=0.1 0.0 0.0 rpy=0.0 1.57079632679 0.0, axis 0 0 1, limit lower=-2.3266 upper=2.3266 effort=132 velocity=15.5
