Commit message: corrected mass

File: kyon_urdf/urdf/parts/kyon_leg.urdf.xacro (robot description, xacro)
@@ -150,6 +150,7 @@
                 <origin xyz="0 0 0" rpy="0 0 0" />
                 <geometry>
-                    <mesh filename="package://kyon_urdf/meshes/collision/mesh_wheel23.stl"
-                        scale="0.001 0.001 ${mirror*0.001}" />
+                    <!--mesh filename="package://kyon_urdf/meshes/collision/mesh_wheel23.stl"
+                        scale="0.001 0.001 ${mirror*0.001}" /-->
+                    <sphere radius="0.125"/>
                 </geometry>
                 <material name="black" />

Commit message: added wrist and wheel_leg

File: kyon_urdf/urdf/kyon.urdf (robot description, URDF)
Before this commit: robot kyon, 30 links, 29 joints
Links:
- removed link ball_arm_1
- removed link ball_arm_2
- removed link upper_arm2_1
- removed link upper_arm2_2
- removed link wrist_1
- removed link wrist_2
- removed link wrist_pitch_motor_1
- removed link wrist_pitch_motor_2
- added link wheel_1, mass 1.8; collision mesh filename=package://kyon_urdf/meshes/collision/mesh_wheel.stl scale=0.001 0.001 0.001; visual mesh filename=package://kyon_urdf/meshes/mesh_wheel.stl scale=0.001 0.001 0.001
- added link wheel_2, mass 1.8; collision mesh filename=package://kyon_urdf/meshes/collision/mesh_wheel.stl scale=0.001 0.001 0.001; visual mesh filename=package://kyon_urdf/meshes/mesh_wheel.stl scale=0.001 0.001 0.001
- added link wheel_3, mass 1.8; collision mesh filename=package://kyon_urdf/meshes/collision/mesh_wheel.stl scale=0.001 0.001 0.001; visual mesh filename=package://kyon_urdf/meshes/mesh_wheel.stl scale=0.001 0.001 0.001
- added link wheel_4, mass 1.8; collision mesh filename=package://kyon_urdf/meshes/collision/mesh_wheel.stl scale=0.001 0.001 0.001; visual mesh filename=package://kyon_urdf/meshes/mesh_wheel.stl scale=0.001 0.001 0.001
- added link wrist_pitch_1, mass 0.63; collision mesh filename=package://kyon_urdf/meshes/collision/mesh_wrist-pitch.stl scale=0.001 0.001 0.001; visual mesh filename=package://kyon_urdf/meshes/mesh_wrist-pitch.stl scale=0.001 0.001 0.001
- added link wrist_pitch_2, mass 0.63; collision mesh filename=package://kyon_urdf/meshes/collision/mesh_wrist-pitch.stl scale=0.001 0.001 0.001; visual mesh filename=package://kyon_urdf/meshes/mesh_wrist-pitch.stl scale=0.001 0.001 0.001
- added link wrist_yaw_1, mass 0.63; collision mesh filename=package://kyon_urdf/meshes/collision/mesh_wrist-yaw.stl scale=0.001 0.001 0.001; visual mesh filename=package://kyon_urdf/meshes/mesh_wrist-yaw.stl scale=0.001 0.001 0.001
- added link wrist_yaw_2, mass 0.63; collision mesh filename=package://kyon_urdf/meshes/collision/mesh_wrist-yaw.stl scale=0.001 0.001 0.001; visual mesh filename=package://kyon_urdf/meshes/mesh_wrist-yaw.stl scale=0.001 0.001 0.001
- link knee_pitch_1: geometry collision mesh filename=package://kyon_urdf/meshes/collision/mesh_fixed-wheel-leg.s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 scale=-0.001 0.001 0.001; visual mesh filename=package://kyon_urdf/meshes/mesh_fixed-wheel-leg.stl scale=-0.001 0.001 0.001
- link knee_pitch_2: geometry collision mesh filename=package://kyon_urdf/meshes/collision/mesh_fixed-wheel-leg.s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 scale=0.001 0.001 0.001; visual mesh filename=package://kyon_urdf/meshes/mesh_fixed-wheel-leg.stl scale=0.001 0.001 0.001
- link knee_pitch_3: geometry collision mesh filename=package://kyon_urdf/meshes/collision/mesh_fixed-wheel-leg.s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 scale=-0.001 0.001 0.001; visual mesh filename=package://kyon_urdf/meshes/mesh_fixed-wheel-leg.stl scale=-0.001 0.001 0.001
- link knee_pitch_4: geometry collision mesh filename=package://kyon_urdf/meshes/collision/mesh_fixed-wheel-leg.s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 scale=0.001 0.001 0.001; visual mesh filename=package://kyon_urdf/meshes/mesh_fixed-wheel-leg.stl scale=0.001 0.001 0.001
Joints:
- removed joint hand_joint_1
- removed joint hand_joint_2
- removed joint wrist_pitch_stator_1
- removed joint wrist_pitch_stator_2
- added joint wheel_joint_1: type revolute, parent knee_pitch_1, child wheel_1, origin xyz=0.0 -0.3 0.054 rpy=0.0 0.0 0.0, axis 0 0 1, limit lower=-3.4056 upper=3.4056 effort=132 velocity=15.5
- added joint wheel_joint_2: type revolute, parent knee_pitch_2, child wheel_2, origin xyz=0.0 -0.3 0.054 rpy=0.0 0.0 0.0, axis 0 0 1, limit lower=-3.3266 upper=3.3266 effort=132 velocity=15.5
- added joint wheel_joint_3: type revolute, parent knee_pitch_3, child wheel_3, origin xyz=0.0 -0.3 0.054 rpy=0.0 0.0 0.0, axis 0 0 1, limit lower=-3.4696 upper=3.4696 effort=132 velocity=15.5
- added joint wheel_joint_4: type revolute, parent knee_pitch_4, child wheel_4, origin xyz=0.0 -0.3 0.054 rpy=0.0 0.0 0.0, axis 0 0 1, limit lower=-3.3426 upper=3.3426 effort=132 velocity=15.5
- joint knee_pitch_1: limit lower=-2.4056 upper=2.4056 effort=132 velocity=15.5 -> lower=-3.4056 upper=3.4056 effort=132 velocity=15.5
- joint knee_pitch_2: limit lower=-2.3266 upper=2.3266 effort=132 velocity=15.5 -> lower=-3.3266 upper=3.3266 effort=132 velocity=15.5
- joint knee_pitch_3: limit lower=-2.4696 upper=2.4696 effort=132 velocity=15.5 -> lower=-3.4696 upper=3.4696 effort=132 velocity=15.5
- joint knee_pitch_4: limit lower=-2.3426 upper=2.3426 effort=132 velocity=15.5 -> lower=-3.3426 upper=3.3426 effort=132 velocity=15.5
- joint shoulder_yaw_1: origin xyz=0.27 0.10299599999999999 0.18721700000000002 rpy=-0.3490656 0.0 0.0 -> xyz=0.28 0.0966072 0.203559 rpy=-0.3490656 0.0 0.0
- joint shoulder_yaw_2: origin xyz=0.27 -0.10299599999999999 0.18721700000000002 rpy=0.3490656 0.0 0.0 -> xyz=0.28 -0.0966072 0.203559 rpy=0.3490656 0.0 0.0
- joint wrist_pitch_1: child upper_arm2_1 -> wrist_pitch_1; origin xyz=0.0 0.0 0.0 rpy=0.0 0.0 0.0 -> xyz=0.0 -0.25 -0.020502500000000003 rpy=-3.14159265359 0.0 0.0; parent wrist_pitch_motor_1 -> elbow_pitch_1
- joint wrist_pitch_2: child upper_arm2_2 -> wrist_pitch_2; origin xyz=0.0 0.0 0.0 rpy=0.0 0.0 0.0 -> xyz=0.0 -0.25 -0.020502500000000003 rpy=-3.14159265359 0.0 0.0; parent wrist_pitch_motor_2 -> elbow_pitch_2
- joint wrist_yaw_1: child wrist_1 -> wrist_yaw_1; origin xyz=0.1 0.0 0.0 rpy=0.0 1.57079632679 0.0 -> xyz=0.0 0.11586199999999999 -0.02036 rpy=-1.57079632679 0.0 0.0; parent upper_arm2_1 -> wrist_pitch_1
- joint wrist_yaw_2: child wrist_2 -> wrist_yaw_2; origin xyz=0.1 0.0 0.0 rpy=0.0 1.57079632679 0.0 -> xyz=0.0 0.11586199999999999 -0.02036 rpy=-1.57079632679 0.0 0.0; parent upper_arm2_2 -> wrist_pitch_2

File: kyon_urdf/urdf/parts/arms.urdf.xacro (robot description, xacro)
@@ -2,6 +2,4 @@
 <robot xmlns:xacro="http://ros.org/wiki/xacro">
 <xacro:include filename="$(find kyon_urdf)/urdf/parts/kyon_arm.urdf.xacro"/>
-<xacro:include filename="$(find kyon_urdf)/urdf/parts/kyon_ball_ee.xacro"/>
-<xacro:include filename="$(find dagana_urdf)/urdf/dagana_macro.urdf.xacro"/>
 <!-- arms -->
 <xacro:kyon_arm arm_num="1"  rot="1"  parent="pelvis">
@@ -9,55 +7,43 @@
 <xacro:kyon_arm arm_num="2" rot="-1"  parent="pelvis">
 </xacro:kyon_arm>
-<xacro:if value="${ADD_DAGANA}">
-	<xacro:dagana_gripper name="dagana_1" parent_link="wrist_1" joint_type="fixed">
-		<origin xyz="0 0 0" rpy="0 0 0"/>
-	</xacro:dagana_gripper>
-	<xacro:dagana_gripper name="dagana_2" parent_link="wrist_2" joint_type="fixed">
-		<origin xyz="0 0 0" rpy="0 0 0"/>
-	</xacro:dagana_gripper>
-	<xacro:if value="${PAYLOAD}">
-		<link name="payload_1">
-			<inertial>
-				<origin xyz="0.0 0.0 0.0"/>
-				<mass value="4"/>
-				<inertia ixx="0.0267" iyy="0.0267" izz="0.0267" ixy="0" ixz="0" iyz="0"/>
-			</inertial>
-			<visual>
-				<origin xyz="0.0 0.0 0.0"  rpy="0.0 0.0 0.0"/>
-				<geometry>
-					<box size="0.2 0.2 0.2"/>
-				</geometry>
-				<material name="dark_grey"/>
-			</visual>
-		</link>
-		<joint name="hand_to_payload_1" type="fixed">
-			<origin xyz="0 0.1 0.0" rpy="0 0 0"/>
-			<parent link="dagana_1_bottom_link"/>
-			<child link="payload_1"/>
-		</joint>
-		<link name="payload_2">
-			<inertial>
-				<origin xyz="0.0 0.0 0.0"/>
-				<mass value="4"/>
-				<inertia ixx="0.0267" iyy="0.0267" izz="0.0267" ixy="0" ixz="0" iyz="0"/>
-			</inertial>
-			<visual>
-				<origin xyz="0.0 0.0 0.0"  rpy="0.0 0.0 0.0"/>
-				<geometry>
-					<box size="0.2 0.2 0.2"/>
-				</geometry>
-				<material name="dark_grey"/>
-			</visual>
-		</link>
-		<joint name="hand_to_payload_2" type="fixed">
-			<origin xyz="0 0.1 0.0" rpy="0 0 0"/>
-			<parent link="dagana_2_bottom_link"/>
-			<child link="payload_2"/>
-		</joint>
-	</xacro:if>
+<xacro:if value="${PAYLOAD}">
+	<link name="payload_1">
+		<inertial>
+			<origin xyz="0.0 0.0 0.0"/>
+			<mass value="4"/>
+			<inertia ixx="0.0267" iyy="0.0267" izz="0.0267" ixy="0" ixz="0" iyz="0"/>
+		</inertial>
+		<visual>
+			<origin xyz="0.0 0.0 0.0"  rpy="0.0 0.0 0.0"/>
+			<geometry>
+				<box size="0.2 0.2 0.2"/>
+			</geometry>
+			<material name="dark_grey"/>
+		</visual>
+	</link>
+	<joint name="hand_to_payload_1" type="fixed">
+		<origin xyz="0 0.1 0.0" rpy="0 0 0"/>
+		<parent link="dagana_1_bottom_link"/>
+		<child link="payload_1"/>
+	</joint>
+	<link name="payload_2">
+		<inertial>
+			<origin xyz="0.0 0.0 0.0"/>
+			<mass value="4"/>
+			<inertia ixx="0.0267" iyy="0.0267" izz="0.0267" ixy="0" ixz="0" iyz="0"/>
+		</inertial>
+		<visual>
+			<origin xyz="0.0 0.0 0.0"  rpy="0.0 0.0 0.0"/>
+			<geometry>
+				<box size="0.2 0.2 0.2"/>
+			</geometry>
+			<material name="dark_grey"/>
+		</visual>
+	</link>
+	<joint name="hand_to_payload_2" type="fixed">
+		<origin xyz="0 0.1 0.0" rpy="0 0 0"/>
+		<parent link="dagana_2_bottom_link"/>
+		<child link="payload_2"/>
+	</joint>
 </xacro:if>
-<xacro:unless value="${ADD_DAGANA}">
-	<xacro:ball_ee arm_num="1" parent="wrist_1" payload="${PAYLOAD}"/>
-	<xacro:ball_ee arm_num="2" parent="wrist_2" payload="${PAYLOAD}"/>
-</xacro:unless>
 </robot>

File: kyon_urdf/urdf/parts/kinematics_properties.urdf.xacro (robot description, xacro)
@@ -1,5 +1,5 @@
 <?xml version="1.0"?>
 <robot  xmlns:xacro="http://ros.org/wiki/xacro">
-    <xacro:property name="mTomm" value="0.001"/>
+    <xacro:property name="mmTom" value="0.001"/>
     <xacro:property name="kin_yaml_file" value="$(find kyon_urdf)/urdf/config/kinematics_properties.yaml" />
     <xacro:property name="kin_props" value="${xacro.load_yaml(kin_yaml_file)}"/>
@@ -27,6 +27,6 @@
     <!-- Compound properties (i.e. based on the props parsed from the yaml) -->
     <!-- Origin -->
-    <xacro:property name="HipRoll_Ox" value="${409.360 * mTomm}"/>
-    <xacro:property name="HipRoll_Oy" value="${77.500 * mTomm}"/>
+    <xacro:property name="HipRoll_Ox" value="${409.360 * mmTom}"/>
+    <xacro:property name="HipRoll_Oy" value="${77.500 * mmTom}"/>
     <xacro:property name="HipRoll_Oz" value="0.0"/>
     <xacro:property name="HipRoll_roll" value="0.0"/>
@@ -55,13 +55,19 @@
     <!-- Origin -->
     <xacro:property name="Wheel_Ox" value="0.0"/>
-    <xacro:property name="Wheel_Oy" value="0.0"/>
-    <xacro:property name="Wheel_Oz" value="${-290.000 * mmTom}"/>
-    <xacro:property name="Wheel_roll" value="${PI_2}"/>
+    <xacro:property name="Wheel_Oy" value="${-300.000 * mmTom}"/>
+    <xacro:property name="Wheel_Oz" value="${54.000 * mmTom}"/>
+    <xacro:property name="Wheel_roll" value="0.0"/>
     <xacro:property name="Wheel_pitch" value="0.0"/>
     <xacro:property name="Wheel_yaw" value="0.0"/>
+    <xacro:property name="SteeringWheel_Ox" value="0.0"/>
+    <xacro:property name="SteeringWheel_Oy" value="0.0"/>
+    <xacro:property name="SteeringWheel_Oz" value="${-290.000 * mmTom}"/>
+    <xacro:property name="SteeringWheel_roll" value="${PI_2}"/>
+    <xacro:property name="SteeringWheel_pitch" value="0.0"/>
+    <xacro:property name="SteeringWheel_yaw" value="0.0"/>
     <!-- Arms -->
-    <xacro:property name="ShoulderYaw_Ox" value="${280.00 * mTomm}"/>
-    <xacro:property name="ShoulderYaw_Oy" value="${96.6072 * mTomm}"/>
-    <xacro:property name="ShoulderYaw_Oz" value="${203.559 * mTomm}"/>
+    <xacro:property name="ShoulderYaw_Ox" value="${280.00 * mmTom}"/>
+    <xacro:property name="ShoulderYaw_Oy" value="${96.6072 * mmTom}"/>
+    <xacro:property name="ShoulderYaw_Oz" value="${203.559 * mmTom}"/>
     <xacro:property name="ShoulderYaw_roll" value="0.3490656"/>
     <xacro:property name="ShoulderYaw_pitch" value="0.0"/>
@@ -69,5 +75,5 @@
     <xacro:property name="ShoulderPitch_Ox" value="0.0"/>
     <xacro:property name="ShoulderPitch_Oy" value="0.0"/>
-    <xacro:property name="ShoulderPitch_Oz" value="${73.5 * mTomm}"/>
+    <xacro:property name="ShoulderPitch_Oz" value="${73.5 * mmTom}"/>
     <xacro:property name="ShoulderPitch_roll" value="0.0"/>
     <xacro:property name="ShoulderPitch_pitch" value="0.0"/>
@@ -75,26 +81,20 @@
     <xacro:property name="ElbowPitch_Ox" value="0.0"/>
     <xacro:property name="ElbowPitch_Oy" value="0.0"/>
-    <xacro:property name="ElbowPitch_Oz" value="${320.00 * mTomm}"/>
+    <xacro:property name="ElbowPitch_Oz" value="${320.00 * mmTom}"/>
     <xacro:property name="ElbowPitch_roll" value="${-PI_2}"/>
     <xacro:property name="ElbowPitch_pitch" value="0.0"/>
     <xacro:property name="ElbowPitch_yaw" value="0.0"/>
-    <xacro:property name="UpperArm1_Ox" value="0.0"/>
-    <xacro:property name="UpperArm1_Oy" value="0.0"/>
-    <xacro:property name="UpperArm1_Oz" value="0.0"/>
-    <xacro:property name="UpperArm1_roll" value="0.0"/>
-    <xacro:property name="UpperArm1_pitch" value="0.0"/>
-    <xacro:property name="UpperArm1_yaw" value="0.0"/>
     <xacro:property name="WristPitch_Ox" value="0.0"/>
-	<xacro:property name="WristPitch_Oy" value="${-250.00 * mTomm}"/>
-	<xacro:property name="WristPitch_Oz" value="0.0"/>
-	<xacro:property name="WristPitch_roll" value="0.0"/>
+	<xacro:property name="WristPitch_Oy" value="${-250.00 * mmTom}"/>
+	<xacro:property name="WristPitch_Oz" value="${-20.5025 * mmTom}"/>
+	<xacro:property name="WristPitch_roll" value="${-PI}"/>
 	<xacro:property name="WristPitch_pitch" value="0.0"/>
-	<xacro:property name="WristPitch_yaw" value="${-PI_2}"/>
-	<xacro:property name="UpperArm2_Ox" value="0.0"/>
-    <xacro:property name="UpperArm2_Oy" value="0.0"/>
-    <xacro:property name="UpperArm2_Oz" value="0.0"/>
-    <xacro:property name="UpperArm2_roll" value="0.0"/>
-    <xacro:property name="UpperArm2_pitch" value="0.0"/>
-    <xacro:property name="UpperArm2_yaw" value="0.0"/>
+	<xacro:property name="WristPitch_yaw" value="0.0"/>
+    <xacro:property name="WristYaw_Ox" value="0.0"/>
+	<xacro:property name="WristYaw_Oy" value="${115.862 * mmTom}"/>
+	<xacro:property name="WristYaw_Oz" value="${-20.360 * mmTom}"/>
+	<xacro:property name="WristYaw_roll" value="${-PI_2}"/>
+	<xacro:property name="WristYaw_pitch" value="0.0"/>
+	<xacro:property name="WristYaw_yaw" value="0.0"/>
     <xacro:property name="EndEffector_Ox" value="${upper_arm2_length}"/>
     <xacro:property name="EndEffector_Oy" value="0.0"/>
@@ -103,9 +103,3 @@
     <xacro:property name="EndEffector_pitch" value="${PI_2}"/>
     <xacro:property name="EndEffector_yaw" value="0.0"/>
-    <xacro:property name="Wheel23_Ox" value="0.0"/>
-    <xacro:property name="Wheel23_Oy" value="0.0"/>
-    <xacro:property name="Wheel23_Oz" value="${ball_radius}"/>
-    <xacro:property name="Wheel23_roll" value="0.0"/>
-    <xacro:property name="Wheel23_pitch" value="0.0"/>
-    <xacro:property name="Wheel23_yaw" value="0.0"/>
 </robot>

File: kyon_urdf/urdf/parts/kyon_arm.urdf.xacro (robot description, xacro)
@@ -8,5 +8,5 @@
 	<inertial>
 		<origin xyz="0.0 0.0 0.0"/>
-		<mass value="${motor_arm1_mass + 0.68}"/>   <!-- hardcoded weight for the arm's base mass-->
+		<mass value="${motor_arm1_mass + 0.68}"/>
 		<inertia ixx="${MotorArm1_xx}" ixy="${MotorArm1_xy}" ixz="${MotorArm1_xz}" iyy="${MotorArm1_yy}" iyz="${MotorArm1_yz}" izz="${MotorArm1_zz}"/>
 	</inertial>
@@ -14,5 +14,4 @@
 		<origin xyz="0.0 0.0 0.0"  rpy="0.0 0.0 0.0"/>
 		<geometry>
-			<!--cylinder radius="${cylinder_radius}" length="${cylinder_length}"/-->
 			<mesh filename="package://kyon_urdf/meshes/mesh_sh-yaw.stl" scale="0.001 0.001 0.001"/>
 		</geometry>
@@ -22,5 +21,4 @@
 		<origin xyz="0.0 0.0 0.0"  rpy="0.0 0.0 0.0"/>
 		<geometry>
-			<!--cylinder radius="${cylinder_radius}" length="${cylinder_length}"/-->
 			<mesh filename="package://kyon_urdf/meshes/collision/mesh_sh-yaw.stl" scale="0.001 0.001 0.001"/>
 		</geometry>
@@ -34,7 +32,5 @@
 	</inertial>
 	<visual>
-		<!--origin xyz="${lower_arm_length / 2} 0.0 0.0"  rpy="0.0 0.0 0.0"/-->
 	  	<geometry>
-			<!--box size="${lower_arm_length} ${lower_arm_width} ${lower_arm_height}"/-->
 	 		<mesh filename="package://kyon_urdf/meshes/mesh_sh-pitch.stl" scale="0.001 0.001 0.001"/>
 	  	</geometry>
@@ -42,7 +38,5 @@
 	</visual>
 	<collision>
-		<!--origin xyz="${lower_arm_length / 2} 0.0 0.0"  rpy="0.0 0.0 0.0"/-->
 	  	<geometry>
-			<!--box size="${lower_arm_length} ${lower_arm_width} ${lower_arm_height}"/-->
 			<mesh filename="package://kyon_urdf/meshes/collision/mesh_sh-pitch.stl" scale="0.001 0.001 0.001"/>
 		</geometry>
@@ -56,19 +50,15 @@
 	</inertial>
 	<visual>
-		<!--origin xyz="${upper_arm1_length / 2} 0.0 0.0"  rpy="0.0 0.0 0.0"/-->
 		<geometry>
-			<!--box size="${upper_arm1_length} ${upper_arm1_width} ${upper_arm1_height}"/-->
 			<mesh filename="package://kyon_urdf/meshes/mesh_elbow.stl" scale="0.001 0.001 0.001"/>
 		</geometry>
 	</visual>
 	<collision>
-		<!--origin xyz="${lower_arm_length / 2} 0.0 0.0"  rpy="0.0 0.0 0.0"/-->
 		<geometry>
-			<!--box size="${upper_arm1_length} ${upper_arm1_width} ${upper_arm1_height}"/-->
 			<mesh filename="package://kyon_urdf/meshes/mesh_elbow.stl" scale="0.001 0.001 0.001"/>
 		</geometry>
 	</collision>
 </link>
-<link name="wrist_pitch_motor_${arm_num}">
+<link name="wrist_pitch_${arm_num}">
 	<inertial>
 		<origin xyz="0.0 0.0 0.0"/>
@@ -79,5 +69,5 @@
 		<origin xyz="0.0 0.0 0.0"  rpy="0.0 0.0 0.0"/>
 	  	<geometry>
-	 		<cylinder radius="${cylinder_radius / 2}" length="${cylinder_length / 2}"/>
+	 		<mesh filename="package://kyon_urdf/meshes/mesh_wrist-pitch.stl" scale="0.001 0.001 0.001"/>
 	  	</geometry>
   		<material name="dark_grey"/>
@@ -86,29 +76,9 @@
 		<origin xyz="0.0 0.0 0.0"  rpy="0.0 0.0 0.0"/>
 		<geometry>
-			<cylinder radius="${cylinder_radius}" length="${cylinder_length}"/>
+			<mesh filename="package://kyon_urdf/meshes/collision/mesh_wrist-pitch.stl" scale="0.001 0.001 0.001"/>
 		</geometry>
 	</collision>
 </link>
-<link name="upper_arm2_${arm_num}">
-	<inertial>
-		<origin xyz="${upper_arm2_length / 2} 0.0 0.0"/>
-		<mass value="${upper_arm2_mass}"/>
-		<inertia ixx="${UpperArm2_xx}" ixy="${UpperArm2_xy}" ixz="${UpperArm2_xz}" iyy="${UpperArm2_yy}" iyz="${UpperArm2_yz}" izz="${UpperArm2_zz}"/>
-	</inertial>
-	<visual>
-		<origin xyz="${upper_arm2_length / 2} 0.0 0.0"  rpy="0.0 0.0 0.0"/>
-		<geometry>
-			<box size="${upper_arm2_length} ${upper_arm2_width} ${upper_arm2_height}"/>
-		</geometry>
-	</visual>
-	<collision>
-		<origin xyz="${upper_arm1_length / 2} 0.0 0.0"  rpy="0.0 0.0 0.0"/>
-		<geometry>
-			<box size="${upper_arm2_length} ${upper_arm2_width} ${upper_arm2_height}"/>
-		</geometry>
-	</collision>
-</link>>
-<!-- /shoulder-elbow -->
-<link name="wrist_${arm_num}">
+<link name="wrist_yaw_${arm_num}">
 	<inertial>
 		<origin xyz="0.0 0.0 0.0"/>
@@ -119,5 +89,5 @@
 		<origin xyz="0.0 0.0 0.0"  rpy="0.0 0.0 0.0"/>
 	  	<geometry>
-	 		<cylinder radius="${cylinder_radius}" length="${cylinder_length / 6}"/>
+	 		<mesh filename="package://kyon_urdf/meshes/mesh_wrist-yaw.stl" scale="0.001 0.001 0.001"/>
 	  	</geometry>
   		<material name="dark_grey"/>
@@ -126,5 +96,5 @@
 		<origin xyz="0.0 0.0 0.0"  rpy="0.0 0.0 0.0"/>
 		<geometry>
-			<cylinder radius="${cylinder_radius/2}" length="${cylinder_length/2}"/>
+			<mesh filename="package://kyon_urdf/meshes/collision/mesh_wrist-yaw.stl" scale="0.001 0.001 0.001"/>
 		</geometry>
 	</collision>
@@ -155,21 +125,15 @@
 	<limit lower="${j_pitch_1_lower[arm_num-1]}" upper="${j_pitch_1_upper[arm_num-1]}" effort="${motor_effort}" velocity="${motor_velocity}"/>
 </joint>
-<joint name="wrist_pitch_stator_${arm_num}" type="fixed">
+<joint name="wrist_pitch_${arm_num}" type="revolute">
 	<parent link="elbow_pitch_${arm_num}"/>
-	<child link="wrist_pitch_motor_${arm_num}"/>
+	<child link="wrist_pitch_${arm_num}"/>
 	<origin xyz="${WristPitch_Ox} ${WristPitch_Oy} ${WristPitch_Oz}" rpy="${WristPitch_roll} ${WristPitch_pitch} ${WristPitch_yaw}"/>
-</joint>
-<joint name="wrist_pitch_${arm_num}" type="revolute">
-	<parent link="wrist_pitch_motor_${arm_num}"/>
-	<child link="upper_arm2_${arm_num}"/>
-	<origin xyz="${UpperArm2_Ox} ${UpperArm2_Oy} ${UpperArm2_Oz}" rpy="${UpperArm2_roll} ${UpperArm2_pitch} ${UpperArm2_yaw}"/>
 	<axis xyz="0 0 1"/>
 	<limit lower="${j_pitch_2_lower[arm_num-1]}" upper="${j_pitch_2_upper[arm_num-1]}" effort="${motor_effort}" velocity="${motor_velocity}"/>
 </joint>
-<!-- end effector  -->
 <joint name="wrist_yaw_${arm_num}" type="revolute">
-	<parent link="upper_arm2_${arm_num}"/>
-	<child link="wrist_${arm_num}"/>
-	<origin xyz="${EndEffector_Ox} ${EndEffector_Oy} ${EndEffector_Oz}" rpy="${EndEffector_roll} ${EndEffector_pitch} ${EndEffector_yaw}"/>
+	<parent link="wrist_pitch_${arm_num}"/>
+	<child link="wrist_yaw_${arm_num}"/>
+	<origin xyz="${WristYaw_Ox} ${WristYaw_Oy} ${WristYaw_Oz}" rpy="${WristYaw_roll} ${WristYaw_pitch} ${WristYaw_yaw}"/>
 	<axis xyz="0 0 1"/>
 	<limit lower="${j_pitch_2_lower[arm_num-1]}" upper="${j_pitch_2_upper[arm_num-1]}" effort="${motor_effort}" velocity="${motor_velocity}"/>

File: kyon_urdf/urdf/parts/kyon_leg.urdf.xacro (robot description, xacro)
@@ -2,6 +2,7 @@
 <robot xmlns:xacro="http://ros.org/wiki/xacro">
 <!-- include end-effectors -->
-<xacro:include filename="$(find kyon_urdf)/urdf/parts/foot_leg.urdf.xacro" />
-<xacro:include filename="$(find kyon_urdf)/urdf/parts/steering_wheel.urdf.xacro" />
+<xacro:include filename="$(find kyon_urdf)/urdf/parts/foot_leg.urdf.xacro"/>
+<xacro:include filename="$(find kyon_urdf)/urdf/parts/steering_wheel.urdf.xacro"/>
+<xacro:include filename="$(find kyon_urdf)/urdf/parts/wheel_leg.urdf.xacro"/>
 <!-- macro legs -->
 <xacro:macro name="kyon_leg" params="leg_num origin_x origin_y mirror">
@@ -70,4 +71,7 @@
 	<xacro:steering_wheel leg_num="${leg_num}" parent="hip_pitch_${leg_num}" origin_x="${origin_x}" origin_y="${origin_y}" mirror="${mirror}"/>
 </xacro:if>
+<xacro:if value="${ADD_WHEELS}">
+	<xacro:wheel_leg leg_num="${leg_num}" parent="hip_pitch_${leg_num}" origin_x="${origin_x}" origin_y="${origin_y}" mirror="${mirror}"/>
+</xacro:if>
 </xacro:macro>
 <!-- /macro legs -->

File: kyon_urdf/urdf/parts/steering_wheel.urdf.xacro (robot description, xacro)
@@ -86,5 +86,5 @@
     <parent link="ankle_yaw_${leg_num}"/>
     <child link="wheel_${leg_num}"/>
-    <origin xyz="${Wheel_Ox} ${Wheel_Oy} ${Wheel_Oz}" rpy="${Wheel_roll} ${Wheel_pitch} ${Wheel_yaw}"/>
+    <origin xyz="${SteeringWheel_Ox} ${SteeringWheel_Oy} ${SteeringWheel_Oz}" rpy="${SteeringWheel_roll} ${SteeringWheel_pitch} ${SteeringWheel_yaw}"/>
     <axis xyz="0 0 1"/>
     <limit lower="${knee_pitch_lower[leg_num-1]}" upper="${knee_pitch_upper[leg_num-1]}" effort="${motor_effort}" velocity="${motor_velocity}"/>
