Commit message: added dagana. missing inertia

File: kyon_urdf/urdf/kyon.urdf (robot description, URDF)
Before this commit: robot kyon, 30 links, 29 joints
Links:
- added link ankle_yaw_1, mass 1.8; collision mesh filename=package://kyon_urdf/meshes/collision/mesh_ankle-yaw.stl scale=0.001 0.001 0.001; visual mesh filename=package://kyon_urdf/meshes/mesh_ankle-yaw.stl scale=0.001 0.001 0.001
- added link ankle_yaw_2, mass 1.8; collision mesh filename=package://kyon_urdf/meshes/collision/mesh_ankle-yaw.stl scale=0.001 0.001 0.001; visual mesh filename=package://kyon_urdf/meshes/mesh_ankle-yaw.stl scale=0.001 0.001 0.001
- added link ankle_yaw_3, mass 1.8; collision mesh filename=package://kyon_urdf/meshes/collision/mesh_ankle-yaw.stl scale=0.001 0.001 0.001; visual mesh filename=package://kyon_urdf/meshes/mesh_ankle-yaw.stl scale=0.001 0.001 0.001
- added link ankle_yaw_4, mass 1.8; collision mesh filename=package://kyon_urdf/meshes/collision/mesh_ankle-yaw.stl scale=0.001 0.001 0.001; visual mesh filename=package://kyon_urdf/meshes/mesh_ankle-yaw.stl scale=0.001 0.001 0.001
- added link dagana1_base, mass 1.8; collision mesh filename=package://kyon_urdf/meshes/collision/mesh_dagana-base.stl scale=0.001 0.001 0.001; visual mesh filename=package://kyon_urdf/meshes/mesh_dagana-base.stl scale=0.001 0.001 0.001
- added link dagana1_clamp, mass 1.8; collision mesh filename=package://kyon_urdf/meshes/collision/mesh_dagana-clamp.stl scale=0.001 0.001 0.001; visual mesh filename=package://kyon_urdf/meshes/mesh_dagana-clamp.stl scale=0.001 0.001 0.001
- added link dagana2_base, mass 1.8; collision mesh filename=package://kyon_urdf/meshes/collision/mesh_dagana-base.stl scale=0.001 0.001 0.001; visual mesh filename=package://kyon_urdf/meshes/mesh_dagana-base.stl scale=0.001 0.001 0.001
- added link dagana2_clamp, mass 1.8; collision mesh filename=package://kyon_urdf/meshes/collision/mesh_dagana-clamp.stl scale=0.001 0.001 0.001; visual mesh filename=package://kyon_urdf/meshes/mesh_dagana-clamp.stl scale=0.001 0.001 0.001
- link knee_pitch_1: geometry collision mesh filename=package://kyon_urdf/meshes/collision/mesh_knee-steering.stl scale=0.001 0.001 0.001; visual mesh filename=package://kyon_urdf/meshes/mesh_knee-steering.stl scale=0.001 0.001 0.001
- link knee_pitch_2: geometry collision mesh filename=package://kyon_urdf/meshes/collision/mesh_knee-steering.stl scale=0.001 0.001 0.001; visual mesh filename=package://kyon_urdf/meshes/mesh_knee-steering.stl scale=0.001 0.001 0.001
- link knee_pitch_3: geometry collision mesh filename=package://kyon_urdf/meshes/collision/mesh_knee-steering.stl scale=0.001 0.001 0.001; visual mesh filename=package://kyon_urdf/meshes/mesh_knee-steering.stl scale=0.001 0.001 0.001
- link knee_pitch_4: geometry collision mesh filename=package://kyon_urdf/meshes/collision/mesh_knee-steering.stl scale=0.001 0.001 0.001; visual mesh filename=package://kyon_urdf/meshes/mesh_knee-steering.stl scale=0.001 0.001 0.001
Joints:
- added joint ankle_yaw_1: type revolute, parent knee_pitch_1, child ankle_yaw_1, origin xyz=0.0 -0.01 0.067 rpy=-1.57079632679 0.0 0.0, axis 0 0 1, limit lower=-3.4056 upper=3.4056 effort=132 velocity=15.5
- added joint ankle_yaw_2: type revolute, parent knee_pitch_2, child ankle_yaw_2, origin xyz=0.0 -0.01 0.067 rpy=-1.57079632679 0.0 0.0, axis 0 0 1, limit lower=-3.3266 upper=3.3266 effort=132 velocity=15.5
- added joint ankle_yaw_3: type revolute, parent knee_pitch_3, child ankle_yaw_3, origin xyz=0.0 -0.01 0.067 rpy=-1.57079632679 0.0 0.0, axis 0 0 1, limit lower=-3.4696 upper=3.4696 effort=132 velocity=15.5
- added joint ankle_yaw_4: type revolute, parent knee_pitch_4, child ankle_yaw_4, origin xyz=0.0 -0.01 0.067 rpy=-1.57079632679 0.0 0.0, axis 0 0 1, limit lower=-3.3426 upper=3.3426 effort=132 velocity=15.5
- added joint dagana1_base_joint: type fixed, parent wrist_yaw_1, child dagana1_base, origin xyz=0.0 0.0 0.0 rpy=0.0 0.0 0.0
- added joint dagana1_clamp_joint: type revolute, parent dagana1_base, child dagana1_clamp, origin xyz=0.0361625 0.016 0.044 rpy=0.0 1.57079632679 0.0, axis 0 0 1, limit lower=-3.4056 upper=3.4056 effort=132 velocity=15.5
- added joint dagana2_base_joint: type fixed, parent wrist_yaw_2, child dagana2_base, origin xyz=0.0 0.0 0.0 rpy=0.0 0.0 0.0
- added joint dagana2_clamp_joint: type revolute, parent dagana2_base, child dagana2_clamp, origin xyz=0.0361625 0.016 0.044 rpy=0.0 1.57079632679 0.0, axis 0 0 1, limit lower=-3.3266 upper=3.3266 effort=132 velocity=15.5
- joint wheel_joint_1: origin xyz=0.0 -0.3 0.054 rpy=0.0 0.0 0.0 -> xyz=0.0 0.0 -0.29 rpy=1.57079632679 0.0 0.0; parent knee_pitch_1 -> ankle_yaw_1
- joint wheel_joint_2: origin xyz=0.0 -0.3 0.054 rpy=0.0 0.0 0.0 -> xyz=0.0 0.0 -0.29 rpy=1.57079632679 0.0 0.0; parent knee_pitch_2 -> ankle_yaw_2
- joint wheel_joint_3: origin xyz=0.0 -0.3 0.054 rpy=0.0 0.0 0.0 -> xyz=0.0 0.0 -0.29 rpy=1.57079632679 0.0 0.0; parent knee_pitch_3 -> ankle_yaw_3
- joint wheel_joint_4: origin xyz=0.0 -0.3 0.054 rpy=0.0 0.0 0.0 -> xyz=0.0 0.0 -0.29 rpy=1.57079632679 0.0 0.0; parent knee_pitch_4 -> ankle_yaw_4

File: kyon_urdf/urdf/parts/kinematics_properties.urdf.xacro (robot description, xacro)
@@ -2,4 +2,5 @@
 <robot  xmlns:xacro="http://ros.org/wiki/xacro">
     <xacro:property name="mmTom" value="0.001"/>
+    <xacro:property name="degTorad" value="0.01744"/>
     <xacro:property name="kin_yaml_file" value="$(find kyon_urdf)/urdf/config/kinematics_properties.yaml" />
     <xacro:property name="kin_props" value="${xacro.load_yaml(kin_yaml_file)}"/>
@@ -97,9 +98,15 @@
 	<xacro:property name="WristYaw_pitch" value="0.0"/>
 	<xacro:property name="WristYaw_yaw" value="0.0"/>
-    <xacro:property name="EndEffector_Ox" value="${upper_arm2_length}"/>
-    <xacro:property name="EndEffector_Oy" value="0.0"/>
-    <xacro:property name="EndEffector_Oz" value="0.0"/>
-    <xacro:property name="EndEffector_roll" value="0.0	"/>
-    <xacro:property name="EndEffector_pitch" value="${PI_2}"/>
-    <xacro:property name="EndEffector_yaw" value="0.0"/>
+    <xacro:property name="DaganaBase_Ox" value="0.0"/>
+    <xacro:property name="DaganaBase_Oy" value="0.0"/>
+    <xacro:property name="DaganaBase_Oz" value="0.0"/>
+    <xacro:property name="DaganaBase_roll" value="0.0"/>
+    <xacro:property name="DaganaBase_pitch" value="0.0"/>
+    <xacro:property name="DaganaBase_yaw" value="0.0"/>
+    <xacro:property name="DaganaClamp_Ox" value="${36.1625 * mmTom}"/>
+    <xacro:property name="DaganaClamp_Oy" value="${16.000 * mmTom}"/>
+    <xacro:property name="DaganaClamp_Oz" value="${44.000 * mmTom}"/>
+    <xacro:property name="DaganaClamp_roll" value="0.0"/>
+    <xacro:property name="DaganaClamp_pitch" value="${PI_2}"/>
+    <xacro:property name="DaganaClamp_yaw" value="0.0"/>
 </robot>

File: kyon_urdf/urdf/parts/kyon_arm.urdf.xacro (robot description, xacro)
@@ -1,4 +1,5 @@
 <?xml version="1.0"?>
 <robot xmlns:xacro="http://ros.org/wiki/xacro">
+<xacro:include filename="$(find kyon_urdf)/urdf/parts/kyon_dagana.urdf.xacro"/>
 <!-- macro arms -->
 <xacro:macro name="kyon_arm" params="arm_num rot parent">
@@ -139,4 +140,7 @@
 	<limit lower="${j_pitch_2_lower[arm_num-1]}" upper="${j_pitch_2_upper[arm_num-1]}" effort="${motor_effort}" velocity="${motor_velocity}"/>
 </joint>
+<xacro:if value="${ADD_DAGANA}">
+	<xacro:kyon_dagana arm_num="${arm_num}" parent="wrist_yaw_${arm_num}"/>
+</xacro:if>
 </xacro:macro>
 <!-- /macro arms -->

File: kyon_urdf/urdf/parts/limits.urdf.xacro (robot description, xacro)
@@ -21,4 +21,7 @@
 <xacro:property name="j_pitch_1_torque" value="${[147.00, 147.00 ]}"/>
 <xacro:property name="j_pitch_2_torque" value="${[147.00, 147.00 ]}"/>
+<!-- Dagana -->
+<xacro:property name="dagana_lower" value="${[-3.4056, -3.3266]}"/>
+<xacro:property name="dagana_upper" value="${[3.4056, 3.3266]}"/>
 <!-- Motor velocities -->
 <xacro:if value="${inertial_props['gear_ratio'] == 30}">
