Commit message: masses and inertias

File: kyon_urdf/urdf/kyon.urdf (robot description, URDF)
Before this commit: robot kyon, 38 links, 37 joints
Links:
- removed link ankle_yaw_1
- removed link ankle_yaw_2
- removed link ankle_yaw_3
- removed link ankle_yaw_4
- removed link dagana1_base
- removed link dagana1_clamp
- removed link dagana2_base
- removed link dagana2_clamp
- removed link elbow_pitch_1
- removed link elbow_pitch_2
- removed link hip_pitch_1
- removed link hip_pitch_2
- removed link hip_pitch_3
- removed link hip_pitch_4
- removed link hip_roll_1
- removed link hip_roll_2
- removed link hip_roll_3
- removed link hip_roll_4
- removed link knee_pitch_1
- removed link knee_pitch_2
- removed link knee_pitch_3
- removed link knee_pitch_4
- removed link shoulder_pitch_1
- removed link shoulder_pitch_2
- removed link shoulder_yaw_1
- removed link shoulder_yaw_2
- removed link wheel_1
- removed link wheel_2
- removed link wheel_3
- removed link wheel_4
- removed link wrist_pitch_1
- removed link wrist_pitch_2
- removed link wrist_yaw_1
- removed link wrist_yaw_2
- added link ankle_yaw_1_link, mass 1.4941965; collision mesh filename=package://kyon_urdf/meshes/collision/mesh_ankle-yaw.stl scale=0.001 0.001 0.001; visual mesh filename=package://kyon_urdf/meshes/mesh_ankle-yaw.stl scale=0.001 0.001 0.001
- added link ankle_yaw_2_link, mass 1.4941965; collision mesh filename=package://kyon_urdf/meshes/collision/mesh_ankle-yaw.stl scale=0.001 0.001 0.001; visual mesh filename=package://kyon_urdf/meshes/mesh_ankle-yaw.stl scale=0.001 0.001 0.001
- added link ankle_yaw_3_link, mass 1.4941965; collision mesh filename=package://kyon_urdf/meshes/collision/mesh_ankle-yaw.stl scale=0.001 0.001 0.001; visual mesh filename=package://kyon_urdf/meshes/mesh_ankle-yaw.stl scale=0.001 0.001 0.001
- added link ankle_yaw_4_link, mass 1.4941965; collision mesh filename=package://kyon_urdf/meshes/collision/mesh_ankle-yaw.stl scale=0.001 0.001 0.001; visual mesh filename=package://kyon_urdf/meshes/mesh_ankle-yaw.stl scale=0.001 0.001 0.001
- added link dagana_1_base, mass 1.8; collision mesh filename=package://kyon_urdf/meshes/collision/mesh_dagana-base.stl scale=0.001 0.001 0.001; visual mesh filename=package://kyon_urdf/meshes/mesh_dagana-base.stl scale=0.001 0.001 0.001
- added link dagana_1_clamp, mass 1.8; collision mesh filename=package://kyon_urdf/meshes/collision/mesh_dagana-clamp.stl scale=0.001 0.001 0.001; visual mesh filename=package://kyon_urdf/meshes/mesh_dagana-clamp.stl scale=0.001 0.001 0.001
- added link dagana_2_base, mass 1.8; collision mesh filename=package://kyon_urdf/meshes/collision/mesh_dagana-base.stl scale=0.001 0.001 0.001; visual mesh filename=package://kyon_urdf/meshes/mesh_dagana-base.stl scale=0.001 0.001 0.001
- added link dagana_2_clamp, mass 1.8; collision mesh filename=package://kyon_urdf/meshes/collision/mesh_dagana-clamp.stl scale=0.001 0.001 0.001; visual mesh filename=package://kyon_urdf/meshes/mesh_dagana-clamp.stl scale=0.001 0.001 0.001
- added link elbow_pitch_1_link, mass 0.77; collision mesh filename=package://kyon_urdf/meshes/mesh_elbow.stl scale=0.001 0.001 0.001; visual mesh filename=package://kyon_urdf/meshes/mesh_elbow.stl scale=0.001 0.001 0.001
- added link elbow_pitch_2_link, mass 0.77; collision mesh filename=package://kyon_urdf/meshes/mesh_elbow.stl scale=0.001 0.001 0.001; visual mesh filename=package://kyon_urdf/meshes/mesh_elbow.stl scale=0.001 0.001 0.001
- added link hip_pitch_1_link, mass 6.6449096; collision mesh filename=package://kyon_urdf/meshes/collision/mesh_hip-pitch.stl scale=0.001 0.001 0.001; visual mesh filename=package://kyon_urdf/meshes/mesh_hip-pitch.stl scale=0.001 0.001 0.001
- added link hip_pitch_2_link, mass 6.6449096; collision mesh filename=package://kyon_urdf/meshes/collision/mesh_hip-pitch.stl scale=0.001 0.001 0.001; visual mesh filename=package://kyon_urdf/meshes/mesh_hip-pitch.stl scale=0.001 0.001 0.001
- added link hip_pitch_3_link, mass 6.6449096; collision mesh filename=package://kyon_urdf/meshes/collision/mesh_hip-pitch.stl scale=0.001 0.001 0.001; visual mesh filename=package://kyon_urdf/meshes/mesh_hip-pitch.stl scale=0.001 0.001 0.001
- added link hip_pitch_4_link, mass 6.6449096; collision mesh filename=package://kyon_urdf/meshes/collision/mesh_hip-pitch.stl scale=0.001 0.001 0.001; visual mesh filename=package://kyon_urdf/meshes/mesh_hip-pitch.stl scale=0.001 0.001 0.001
- added link hip_roll_1_link, mass 2.7479472; collision mesh filename=package://kyon_urdf/meshes/collision/mesh_hip-roll.stl scale=0.001 -0.001 0.001; visual mesh filename=package://kyon_urdf/meshes/mesh_hip-roll.stl scale=0.001 -0.001 0.001
- added link hip_roll_2_link, mass 2.7479472; collision mesh filename=package://kyon_urdf/meshes/collision/mesh_hip-roll.stl scale=0.001 0.001 0.001; visual mesh filename=package://kyon_urdf/meshes/mesh_hip-roll.stl scale=0.001 0.001 0.001
- added link hip_roll_3_link, mass 2.7479472; collision mesh filename=package://kyon_urdf/meshes/collision/mesh_hip-roll.stl scale=0.001 -0.001 0.001; visual mesh filename=package://kyon_urdf/meshes/mesh_hip-roll.stl scale=0.001 -0.001 0.001
- added link hip_roll_4_link, mass 2.7479472; collision mesh filename=package://kyon_urdf/meshes/collision/mesh_hip-roll.stl scale=0.001 0.001 0.001; visual mesh filename=package://kyon_urdf/meshes/mesh_hip-roll.stl scale=0.001 0.001 0.001
- added link knee_pitch_1_link, mass 1.4555296; collision mesh filename=package://kyon_urdf/meshes/collision/mesh_knee-steering.stl scale=0.001 0.001 0.001; visual mesh filename=package://kyon_urdf/meshes/mesh_knee-steering.stl scale=0.001 0.001 0.001
- added link knee_pitch_2_link, mass 1.4555296; collision mesh filename=package://kyon_urdf/meshes/collision/mesh_knee-steering.stl scale=0.001 0.001 0.001; visual mesh filename=package://kyon_urdf/meshes/mesh_knee-steering.stl scale=0.001 0.001 0.001
- added link knee_pitch_3_link, mass 1.4555296; collision mesh filename=package://kyon_urdf/meshes/collision/mesh_knee-steering.stl scale=0.001 0.001 0.001; visual mesh filename=package://kyon_urdf/meshes/mesh_knee-steering.stl scale=0.001 0.001 0.001
- added link knee_pitch_4_link, mass 1.4555296; collision mesh filename=package://kyon_urdf/meshes/collision/mesh_knee-steering.stl scale=0.001 0.001 0.001; visual mesh filename=package://kyon_urdf/meshes/mesh_knee-steering.stl scale=0.001 0.001 0.001
- added link shoulder_pitch_1_link, mass 1.8; collision mesh filename=package://kyon_urdf/meshes/collision/mesh_sh-pitch.stl scale=0.001 0.001 0.001; visual mesh filename=package://kyon_urdf/meshes/mesh_sh-pitch.stl scale=0.001 0.001 0.001
- added link shoulder_pitch_2_link, mass 1.8; collision mesh filename=package://kyon_urdf/meshes/collision/mesh_sh-pitch.stl scale=0.001 0.001 0.001; visual mesh filename=package://kyon_urdf/meshes/mesh_sh-pitch.stl scale=0.001 0.001 0.001
- added link shoulder_yaw_1_link, mass 1.6; collision mesh filename=package://kyon_urdf/meshes/collision/mesh_sh-yaw.stl scale=0.001 0.001 0.001; visual mesh filename=package://kyon_urdf/meshes/mesh_sh-yaw.stl scale=0.001 0.001 0.001
- added link shoulder_yaw_2_link, mass 1.6; collision mesh filename=package://kyon_urdf/meshes/collision/mesh_sh-yaw.stl scale=0.001 0.001 0.001; visual mesh filename=package://kyon_urdf/meshes/mesh_sh-yaw.stl scale=0.001 0.001 0.001
- added link wheel_1_link, mass 1.263839; collision mesh filename=package://kyon_urdf/meshes/collision/mesh_wheel.stl scale=0.001 0.001 0.001; visual mesh filename=package://kyon_urdf/meshes/mesh_wheel.stl scale=0.001 0.001 0.001
- added link wheel_2_link, mass 1.263839; collision mesh filename=package://kyon_urdf/meshes/collision/mesh_wheel.stl scale=0.001 0.001 0.001; visual mesh filename=package://kyon_urdf/meshes/mesh_wheel.stl scale=0.001 0.001 0.001
- added link wheel_3_link, mass 1.263839; collision mesh filename=package://kyon_urdf/meshes/collision/mesh_wheel.stl scale=0.001 0.001 0.001; visual mesh filename=package://kyon_urdf/meshes/mesh_wheel.stl scale=0.001 0.001 0.001
- added link wheel_4_link, mass 1.263839; collision mesh filename=package://kyon_urdf/meshes/collision/mesh_wheel.stl scale=0.001 0.001 0.001; visual mesh filename=package://kyon_urdf/meshes/mesh_wheel.stl scale=0.001 0.001 0.001
- added link wrist_pitch_1_link, mass 0.63; collision mesh filename=package://kyon_urdf/meshes/collision/mesh_wrist-pitch.stl scale=0.001 0.001 0.001; visual mesh filename=package://kyon_urdf/meshes/mesh_wrist-pitch.stl scale=0.001 0.001 0.001
- added link wrist_pitch_2_link, mass 0.63; collision mesh filename=package://kyon_urdf/meshes/collision/mesh_wrist-pitch.stl scale=0.001 0.001 0.001; visual mesh filename=package://kyon_urdf/meshes/mesh_wrist-pitch.stl scale=0.001 0.001 0.001
- added link wrist_yaw_1_link, mass 0.63; collision mesh filename=package://kyon_urdf/meshes/collision/mesh_wrist-yaw.stl scale=0.001 0.001 0.001; visual mesh filename=package://kyon_urdf/meshes/mesh_wrist-yaw.stl scale=0.001 0.001 0.001
- added link wrist_yaw_2_link, mass 0.63; collision mesh filename=package://kyon_urdf/meshes/collision/mesh_wrist-yaw.stl scale=0.001 0.001 0.001; visual mesh filename=package://kyon_urdf/meshes/mesh_wrist-yaw.stl scale=0.001 0.001 0.001
- link pelvis: mass 14 -> 32.642743
Joints:
- removed joint dagana1_base_joint
- removed joint dagana1_clamp_joint
- removed joint dagana2_base_joint
- removed joint dagana2_clamp_joint
- added joint dagana_1_base_joint: type fixed, parent wrist_yaw_1_link, child dagana_1_base, origin xyz=0.0 0.0 0.0 rpy=0.0 0.0 0.0
- added joint dagana_1_clamp_joint: type revolute, parent dagana_1_base, child dagana_1_clamp, origin xyz=0.0361625 0.016 0.044 rpy=0.0 1.57079632679 0.0, axis 0 0 1, limit lower=-3.4056 upper=3.4056 effort=132 velocity=15.5
- added joint dagana_2_base_joint: type fixed, parent wrist_yaw_2_link, child dagana_2_base, origin xyz=0.0 0.0 0.0 rpy=0.0 0.0 0.0
- added joint dagana_2_clamp_joint: type revolute, parent dagana_2_base, child dagana_2_clamp, origin xyz=0.0361625 0.016 0.044 rpy=0.0 1.57079632679 0.0, axis 0 0 1, limit lower=-3.3266 upper=3.3266 effort=132 velocity=15.5
- joint ankle_yaw_1: child ankle_yaw_1 -> ankle_yaw_1_link; origin xyz=0.0 -0.01 0.067 rpy=-1.57079632679 0.0 0.0 -> xyz=0.0 -0.0735 0.059000000000000004 rpy=-1.57079632679 0.0 0.0; parent knee_pitch_1 -> knee_pitch_1_link
- joint ankle_yaw_2: child ankle_yaw_2 -> ankle_yaw_2_link; origin xyz=0.0 -0.01 0.067 rpy=-1.57079632679 0.0 0.0 -> xyz=0.0 -0.0735 0.059000000000000004 rpy=-1.57079632679 0.0 0.0; parent knee_pitch_2 -> knee_pitch_2_link
- joint ankle_yaw_3: child ankle_yaw_3 -> ankle_yaw_3_link; origin xyz=0.0 -0.01 0.067 rpy=-1.57079632679 0.0 0.0 -> xyz=0.0 -0.0735 0.059000000000000004 rpy=-1.57079632679 0.0 0.0; parent knee_pitch_3 -> knee_pitch_3_link
- joint ankle_yaw_4: child ankle_yaw_4 -> ankle_yaw_4_link; origin xyz=0.0 -0.01 0.067 rpy=-1.57079632679 0.0 0.0 -> xyz=0.0 -0.0735 0.059000000000000004 rpy=-1.57079632679 0.0 0.0; parent knee_pitch_4 -> knee_pitch_4_link
- joint elbow_pitch_1: child elbow_pitch_1 -> elbow_pitch_1_link; limit lower=-2.4056 upper=2.4056 effort=132 velocity=15.5 -> lower=-3 upper=3 effort=132 velocity=15.5; parent shoulder_pitch_1 -> shoulder_pitch_1_link
- joint elbow_pitch_2: child elbow_pitch_2 -> elbow_pitch_2_link; limit lower=-2.3266 upper=2.3266 effort=132 velocity=15.5 -> lower=-3 upper=3 effort=132 velocity=15.5; parent shoulder_pitch_2 -> shoulder_pitch_2_link
- joint hip_pitch_1: child hip_pitch_1 -> hip_pitch_1_link; origin xyz=0.0 0.05086 0.0 rpy=-1.57079632679 1.57079632679 0.0 -> xyz=0.0 -0.04746 0.0 rpy=0.0 1.57079632679 1.57079632679; parent hip_roll_1 -> hip_roll_1_link
- joint hip_pitch_2: child hip_pitch_2 -> hip_pitch_2_link; origin xyz=0.0 -0.05086 0.0 rpy=1.57079632679 -1.57079632679 0.0 -> xyz=0.0 0.04746 0.0 rpy=0.0 -1.57079632679 1.57079632679; parent hip_roll_2 -> hip_roll_2_link
- joint hip_pitch_3: child hip_pitch_3 -> hip_pitch_3_link; origin xyz=-0.0 0.05086 0.0 rpy=-1.57079632679 -1.57079632679 0.0 -> xyz=0.0 -0.04746 0.0 rpy=0.0 -1.57079632679 -1.57079632679; parent hip_roll_3 -> hip_roll_3_link
- joint hip_pitch_4: child hip_pitch_4 -> hip_pitch_4_link; origin xyz=-0.0 -0.05086 0.0 rpy=1.57079632679 1.57079632679 0.0 -> xyz=0.0 0.04746 0.0 rpy=0.0 1.57079632679 -1.57079632679; parent hip_roll_4 -> hip_roll_4_link
- joint hip_roll_1: child hip_roll_1 -> hip_roll_1_link; origin xyz=0.40936 0.0775 0.0 rpy=0.0 1.57079632679 0.0 -> xyz=0.41100000000000003 0.0775 0.0 rpy=0.0 1.57079632679 0.0
- joint hip_roll_2: child hip_roll_2 -> hip_roll_2_link; origin xyz=0.40936 -0.0775 0.0 rpy=0.0 1.57079632679 0.0 -> xyz=0.41100000000000003 -0.0775 0.0 rpy=0.0 1.57079632679 0.0
- joint hip_roll_3: child hip_roll_3 -> hip_roll_3_link; origin xyz=-0.40936 0.0775 0.0 rpy=0.0 -1.57079632679 0.0 -> xyz=-0.41100000000000003 0.0775 0.0 rpy=0.0 -1.57079632679 0.0
- joint hip_roll_4: child hip_roll_4 -> hip_roll_4_link; origin xyz=-0.40936 -0.0775 0.0 rpy=0.0 -1.57079632679 0.0 -> xyz=-0.41100000000000003 -0.0775 0.0 rpy=0.0 -1.57079632679 0.0
- joint knee_pitch_1: child knee_pitch_1 -> knee_pitch_1_link; origin xyz=0.0 -0.34600000000000003 0.16671000000000002 rpy=0.0 0.0 0.0 -> xyz=0.0 -0.34600000000000003 0.24606 rpy=0.0 0.0 0.0; parent hip_pitch_1 -> hip_pitch_1_link
- joint knee_pitch_2: child knee_pitch_2 -> knee_pitch_2_link; origin xyz=0.0 -0.34600000000000003 0.16671000000000002 rpy=0.0 0.0 0.0 -> xyz=0.0 -0.34600000000000003 0.24606 rpy=0.0 0.0 0.0; parent hip_pitch_2 -> hip_pitch_2_link
- joint knee_pitch_3: child knee_pitch_3 -> knee_pitch_3_link; origin xyz=0.0 -0.34600000000000003 0.16671000000000002 rpy=0.0 0.0 0.0 -> xyz=0.0 -0.34600000000000003 0.24606 rpy=0.0 0.0 0.0; parent hip_pitch_3 -> hip_pitch_3_link
- joint knee_pitch_4: child knee_pitch_4 -> knee_pitch_4_link; origin xyz=0.0 -0.34600000000000003 0.16671000000000002 rpy=0.0 0.0 0.0 -> xyz=0.0 -0.34600000000000003 0.24606 rpy=0.0 0.0 0.0; parent hip_pitch_4 -> hip_pitch_4_link
- joint shoulder_pitch_1: child shoulder_pitch_1 -> shoulder_pitch_1_link; limit lower=-2.4056 upper=2.4056 effort=132 velocity=15.5 -> lower=-3 upper=3 effort=132 velocity=15.5; parent shoulder_yaw_1 -> shoulder_yaw_1_link
- joint shoulder_pitch_2: child shoulder_pitch_2 -> shoulder_pitch_2_link; limit lower=-2.3266 upper=2.3266 effort=132 velocity=15.5 -> lower=-3 upper=3 effort=132 velocity=15.5; parent shoulder_yaw_2 -> shoulder_yaw_2_link
- joint shoulder_yaw_1: child shoulder_yaw_1 -> shoulder_yaw_1_link
- joint shoulder_yaw_2: child shoulder_yaw_2 -> shoulder_yaw_2_link
- joint wheel_joint_1: child wheel_1 -> wheel_1_link; origin xyz=0.0 0.0 -0.29 rpy=1.57079632679 0.0 0.0 -> xyz=0.0 0.0 -0.2265 rpy=-1.57079632679 0.0 0.0; parent ankle_yaw_1 -> ankle_yaw_1_link
- joint wheel_joint_2: child wheel_2 -> wheel_2_link; origin xyz=0.0 0.0 -0.29 rpy=1.57079632679 0.0 0.0 -> xyz=0.0 0.0 -0.2265 rpy=-1.57079632679 0.0 0.0; parent ankle_yaw_2 -> ankle_yaw_2_link
- joint wheel_joint_3: child wheel_3 -> wheel_3_link; origin xyz=0.0 0.0 -0.29 rpy=1.57079632679 0.0 0.0 -> xyz=0.0 0.0 -0.2265 rpy=-1.57079632679 0.0 0.0; parent ankle_yaw_3 -> ankle_yaw_3_link
- joint wheel_joint_4: child wheel_4 -> wheel_4_link; origin xyz=0.0 0.0 -0.29 rpy=1.57079632679 0.0 0.0 -> xyz=0.0 0.0 -0.2265 rpy=-1.57079632679 0.0 0.0; parent ankle_yaw_4 -> ankle_yaw_4_link
- joint wrist_pitch_1: child wrist_pitch_1 -> wrist_pitch_1_link; parent elbow_pitch_1 -> elbow_pitch_1_link
- joint wrist_pitch_2: child wrist_pitch_2 -> wrist_pitch_2_link; parent elbow_pitch_2 -> elbow_pitch_2_link
- joint wrist_yaw_1: child wrist_yaw_1 -> wrist_yaw_1_link; parent wrist_pitch_1 -> wrist_pitch_1_link
- joint wrist_yaw_2: child wrist_yaw_2 -> wrist_yaw_2_link; parent wrist_pitch_2 -> wrist_pitch_2_link

File: kyon_urdf/urdf/kyon_base.urdf.xacro (robot description, xacro)
@@ -11,6 +11,6 @@
 <link name="pelvis">
 	<inertial>
-		<origin xyz="0.0 0.0 0.0"/>
-		<mass value="${pelvis_mass}"/>
+		<origin xyz="${Pelvis_x} ${Pelvis_y} ${Pelvis_z}"/>
+		<mass value="${Pelvis_mass}"/>
 		<inertia ixx="${Pelvis_xx}" ixy="${Pelvis_xy}" ixz="${Pelvis_xz}" iyy="${Pelvis_yy}" iyz="${Pelvis_yz}" izz="${Pelvis_zz}"/>
 	</inertial>
@@ -18,5 +18,4 @@
 		<origin xyz="0.0 0 0.0"  rpy="0.0 0.0 0.0"/>
 		<geometry>
-	 		<!--box size="${pelvis_length} ${pelvis_width} ${pelvis_height}"/-->
 	 		<mesh filename="package://kyon_urdf/meshes/mesh_pelvis.stl" scale="0.001 0.001 0.001"/>
 		</geometry>
@@ -25,5 +24,4 @@
 		<origin xyz="0.0 0 0.0"  rpy="0.0 0.0 0.0"/>
 		<geometry>
-	  		<!--box size="${pelvis_length} ${pelvis_width} ${pelvis_height}"/-->
 	  		<mesh filename="package://kyon_urdf/meshes/collision/mesh_pelvis.stl" scale="0.001 0.001 0.001"/>
 		</geometry>

File: kyon_urdf/urdf/parts/foot_leg.urdf.xacro (robot description, xacro)
@@ -5,7 +5,7 @@
 <link name="knee_pitch_${leg_num}_link">
     <inertial>
-        <origin xyz="0.0 0.0 0.0"/>
-        <mass value="${motorA_mass}"/>
-        <inertia ixx="${MotorA_xx}" ixy="${mirror*MotorA_xy}" ixz="${mirror*MotorA_xz}" iyy="${MotorA_yy}" iyz="${MotorA_yz}" izz="${MotorA_zz}"/>
+        <origin xyz="${StickLeg_x} ${StickLeg_y} ${StickLeg_z}"/>
+        <mass value="${StickLeg_mass}"/>
+        <inertia ixx="${StickLeg_xx}" ixy="${mirror*StickLeg_xy}" ixz="${mirror*StickLeg_xz}" iyy="${StickLeg_yy}" iyz="${StickLeg_yz}" izz="${StickLeg_zz}"/>
     </inertial>
     <visual>
