Commit message: masses and inertias

File: kyon_urdf/urdf/parts/inertial_properties.urdf.xacro (robot description, xacro)
@@ -1,4 +1,5 @@
 <?xml version="1.0"?>
 <robot  xmlns:xacro="http://ros.org/wiki/xacro">
+    <xacro:property name="mm2Tom2" value="${0.001*0.001}"/>
     <xacro:property name="inertial_yaml_file" value="$(find kyon_urdf)/urdf/config/inertial_properties.yaml" />
     <xacro:property name="inertial_props" value="${xacro.load_yaml(inertial_yaml_file)}"/>
@@ -41,24 +42,80 @@
     <xacro:property name="MotorArm3_zz" value="${1/2 * motor_arm3_mass * cylinder_radius * cylinder_radius}"/>
     <!-- Pelvis -->
-    <xacro:property name="Pelvis_xx" value="${1/12 * pelvis_mass * (pelvis_width * pelvis_width + pelvis_height * pelvis_height)}"/>
-    <xacro:property name="Pelvis_xy" value="0.0"/>
-    <xacro:property name="Pelvis_xz" value="0.0"/>
-    <xacro:property name="Pelvis_yy" value="${1/12 * pelvis_mass * (pelvis_length * pelvis_length + pelvis_height * pelvis_height)}"/>
-    <xacro:property name="Pelvis_yz" value="0.0"/>
-    <xacro:property name="Pelvis_zz" value="${1/12 * pelvis_mass * (pelvis_width * pelvis_width + pelvis_length * pelvis_length)}"/>
-    <!-- Upper Leg -->
-    <xacro:property name="UpperLeg_xx" value="${1/12 * upper_leg_mass * (upper_leg_width * upper_leg_width + upper_leg_height * upper_leg_height)}"/>
-    <xacro:property name="UpperLeg_xy" value="0.0"/>
-    <xacro:property name="UpperLeg_xz" value="0.0"/>
-    <xacro:property name="UpperLeg_yy" value="${1/12 * upper_leg_mass * (upper_leg_length * upper_leg_length + upper_leg_height * upper_leg_height)}"/>
-    <xacro:property name="UpperLeg_yz" value="0.0"/>
-    <xacro:property name="UpperLeg_zz" value="${1/12 * upper_leg_mass * (upper_leg_width * upper_leg_width + upper_leg_length * upper_leg_length)}"/>
-    <!-- Lower Leg -->
-    <xacro:property name="LowerLeg_xx" value="${1/12 * lower_leg_mass * (lower_leg_width * lower_leg_width + lower_leg_height * lower_leg_height)}"/>
-    <xacro:property name="LowerLeg_xy" value="0.0"/>
-    <xacro:property name="LowerLeg_xz" value="0.0"/>
-    <xacro:property name="LowerLeg_yy" value="${1/12 * lower_leg_mass * (lower_leg_length * lower_leg_length + lower_leg_height * lower_leg_height)}"/>
-    <xacro:property name="LowerLeg_yz" value="0.0"/>
-    <xacro:property name="LowerLeg_zz" value="${1/12 * lower_leg_mass * (lower_leg_width * lower_leg_width + lower_leg_length * lower_leg_length)}"/>
+    <xacro:property name="Pelvis_mass" value="32.642743"/>
+    <xacro:property name="Pelvis_x" value="${3.5990152e+01 * mmTom}"/>
+    <xacro:property name="Pelvis_y" value="${-3.0735925e+01 * mmTom}"/>
+    <xacro:property name="Pelvis_z" value="${3.7859444e+01 * mmTom}"/>
+    <xacro:property name="Pelvis_xx" value="${3.5499677e+05 * mm2Tom2}"/>
+    <xacro:property name="Pelvis_xy" value="${-3.9512772e+04 * mm2Tom2}"/>
+    <xacro:property name="Pelvis_xz" value="${-9.9657679e+04 * mm2Tom2}"/>
+    <xacro:property name="Pelvis_yy" value="${1.2528724e+06 * mm2Tom2}"/>
+    <xacro:property name="Pelvis_yz" value="${-5.5537486e+04 * mm2Tom2}"/>
+    <xacro:property name="Pelvis_zz" value="${1.2807784e+06 * mm2Tom2}"/>
+    <!-- Hip Roll -->
+    <xacro:property name="HipRoll_mass" value="2.7479472"/>
+    <xacro:property name="HipRoll_x" value="${-4.8748556e-01 * mmTom}"/>
+    <xacro:property name="HipRoll_y" value="${6.3409270e+00 * mmTom}"/>
+    <xacro:property name="HipRoll_z" value="${-1.1484611e+02 * mmTom}"/>
+    <xacro:property name="HipRoll_xx" value="${1.4719608e+04 * mm2Tom2}"/>
+    <xacro:property name="HipRoll_xy" value="${-1.1262382e+01 * mm2Tom2}"/>
+    <xacro:property name="HipRoll_xz" value="${3.2414002e+01 * mm2Tom2}"/>
+    <xacro:property name="HipRoll_yy" value="${1.4797973e+04 * mm2Tom2}"/>
+    <xacro:property name="HipRoll_yz" value="${-1.7237369e+03 * mm2Tom2}"/>
+    <xacro:property name="HipRoll_zz" value="${4.9076886e+03 * mm2Tom2}"/>
+    <!-- Hip Pitch -->
+    <xacro:property name="HipPitch_mass" value="6.6449096"/>
+    <xacro:property name="HipPitch_x" value="${6.4486994e-02 * mmTom}"/>
+    <xacro:property name="HipPitch_y" value="${-7.8127559e+01 * mmTom}"/>
+    <xacro:property name="HipPitch_z" value="${1.4684759e+02 * mmTom}"/>
+    <xacro:property name="HipPitch_xx" value="${1.2473067e+05 * mm2Tom2}"/>
+    <xacro:property name="HipPitch_xy" value="${-6.7511845e+02 * mm2Tom2}"/>
+    <xacro:property name="HipPitch_xz" value="${-5.3841528e+01 * mm2Tom2}"/>
+    <xacro:property name="HipPitch_yy" value="${3.4322669e+04 * mm2Tom2}"/>
+    <xacro:property name="HipPitch_yz" value="${2.8582838e+04 * mm2Tom2}"/>
+    <xacro:property name="HipPitch_zz" value="${1.0356313e+05 * mm2Tom2}"/>
+    <!-- Stick Leg -->
+    <xacro:property name="StickLeg_mass" value="0.70900216"/>
+    <xacro:property name="StickLeg_x" value="${5.1193011e-03 * mmTom}"/>
+    <xacro:property name="StickLeg_y" value="${-1.0291595e+02 * mmTom}"/>
+    <xacro:property name="StickLeg_z" value="${-1.2895495e+00 * mmTom}"/>
+    <xacro:property name="StickLeg_xx" value="${1.2517512e+04 * mm2Tom2}"/>
+    <xacro:property name="StickLeg_xy" value="${-5.4385779e-01 * mm2Tom2}"/>
+    <xacro:property name="StickLeg_xz" value="${1.4538899e-01 * mm2Tom2}"/>
+    <xacro:property name="StickLeg_yy" value="${8.0474409e+02 * mm2Tom2}"/>
+    <xacro:property name="StickLeg_yz" value="${1.7446290e+03 * mm2Tom2}"/>
+    <xacro:property name="StickLeg_zz" value="${1.2307020e+04 * mm2Tom2}"/>
+    <!-- Knee Pitch -->
+    <xacro:property name="KneePitch_mass" value="1.4555296"/>
+    <xacro:property name="KneePitch_x" value="${-5.1135441e-01 * mmTom}"/>
+    <xacro:property name="KneePitch_y" value="${-1.7451804e+01 * mmTom}"/>
+    <xacro:property name="KneePitch_z" value="${3.7226616e+01 * mmTom}"/>
+    <xacro:property name="KneePitch_xx" value="${3.8934930e+03 * mm2Tom2}"/>
+    <xacro:property name="KneePitch_xy" value="${2.4351251e+01 * mm2Tom2}"/>
+    <xacro:property name="KneePitch_xz" value="${2.2649175e+01 * mm2Tom2}"/>
+    <xacro:property name="KneePitch_yy" value="${3.2260304e+03 * mm2Tom2}"/>
+    <xacro:property name="KneePitch_yz" value="${5.5514749e+02 * mm2Tom2}"/>
+    <xacro:property name="KneePitch_zz" value="${2.0709191e+03 * mm2Tom2}"/>
+    <!-- Ankle Yaw -->
+    <xacro:property name="AnkleYaw_mass" value="1.4941965"/>
+    <xacro:property name="AnkleYaw_x" value="${1.6741030e-01 * mmTom}"/>
+    <xacro:property name="AnkleYaw_y" value="${-9.4968142e+00 * mmTom}"/>
+    <xacro:property name="AnkleYaw_z" value="${-1.7017490e+02 * mmTom}"/>
+    <xacro:property name="AnkleYaw_xx" value="${1.2013025e+04 * mm2Tom2}"/>
+    <xacro:property name="AnkleYaw_xy" value="${-1.9404017e+03 * mm2Tom2}"/>
+    <xacro:property name="AnkleYaw_xz" value="${3.9733307e+02 * mm2Tom2}"/>
+    <xacro:property name="AnkleYaw_yy" value="${1.1965900e+04 * mm2Tom2}"/>
+    <xacro:property name="AnkleYaw_yz" value="${-2.9154923e+02 * mm2Tom2}"/>
+    <xacro:property name="AnkleYaw_zz" value="${-2.0271262e+03 * mm2Tom2}"/>
+    <!-- Steering Wheel-->
+    <xacro:property name="SteeringWheel_mass" value="1.2638390"/>
+	<xacro:property name="SteeringWheel_x" value="${0.0 * mmTom}"/>
+	<xacro:property name="SteeringWheel_y" value="${0.0 * mmTom}"/>
+	<xacro:property name="SteeringWheel_z" value="${1.4437817e+00 * mmTom}"/>
+	<xacro:property name="SteeringWheel_xx" value="${4.1796417e+03 * mm2Tom2}"/>
+	<xacro:property name="SteeringWheel_xy" value="${4.4497596e-03 * mm2Tom2}"/>
+	<xacro:property name="SteeringWheel_xz" value="${0.0000000e+00 * mm2Tom2}"/>
+	<xacro:property name="SteeringWheel_yy" value="${4.1796381e+03 * mm2Tom2}"/>
+	<xacro:property name="SteeringWheel_yz" value="${0.0 * mm2Tom2}"/>
+	<xacro:property name="SteeringWheel_zz" value="${7.9333497e+03 * mm2Tom2}"/>
     <!-- Upper Arm -->
     <xacro:property name="UpperArm1_xx" value="${1/12 * upper_arm1_mass * (upper_arm1_width * upper_arm1_width + upper_arm1_height * upper_arm1_height)}"/>
@@ -88,15 +145,3 @@
     <xacro:property name="Ball_yz" value="0.0"/>
     <xacro:property name="Ball_zz" value="${2/3 * ball_mass * ball_radius * ball_radius}"/>
-    <xacro:property name="Wheel23_mass" value="1.8569388e+00"/>
-    <!-- Center of Mass -->
-	<xacro:property name="Wheel23_x" value="${0.0 * mmTom}"/>
-	<xacro:property name="Wheel23_y" value="${0.0 * mmTom}"/>
-	<xacro:property name="Wheel23_z" value="${-1.5403767e-01 * mmTom}"/>
-	<!-- Inertia -->
-	<xacro:property name="Wheel23_xx" value="${8.6373591e+03 * mm2Tom2}"/>
-	<xacro:property name="Wheel23_yy" value="${8.6373644e+03 * mm2Tom2}"/>
-	<xacro:property name="Wheel23_zz" value="${1.6376551e+04 * mm2Tom2}"/>
-	<xacro:property name="Wheel23_xy" value="${0.0 * mm2Tom2}"/>
-	<xacro:property name="Wheel23_xz" value="${0.0 * mm2Tom2}"/>
-	<xacro:property name="Wheel23_yz" value="${0.0 * mm2Tom2}"/>
 </robot>

File: kyon_urdf/urdf/parts/kinematics_properties.urdf.xacro (robot description, xacro)
@@ -28,6 +28,6 @@
     <!-- Compound properties (i.e. based on the props parsed from the yaml) -->
     <!-- Origin -->
-    <xacro:property name="HipRoll_Ox" value="${409.360 * mmTom}"/>
-    <xacro:property name="HipRoll_Oy" value="${77.500 * mmTom}"/>
+    <xacro:property name="HipRoll_Ox" value="${411.000 * mmTom}"/>
+    <xacro:property name="HipRoll_Oy" value="${-77.500 * mmTom}"/>
     <xacro:property name="HipRoll_Oz" value="0.0"/>
     <xacro:property name="HipRoll_roll" value="0.0"/>
@@ -36,19 +36,19 @@
     <!-- Origin -->
     <xacro:property name="HipPitch_Ox" value="0.0"/>
-    <xacro:property name="HipPitch_Oy" value="${50.860 * mmTom}"/>
+    <xacro:property name="HipPitch_Oy" value="${47.460 * mmTom}"/>
     <xacro:property name="HipPitch_Oz" value="0.0"/>
-    <xacro:property name="HipPitch_roll" value="${-PI_2}"/>
-    <xacro:property name="HipPitch_pitch" value="${PI_2}"/>
-    <xacro:property name="HipPitch_yaw" value="0.0"/>
+    <xacro:property name="HipPitch_roll" value="0.0"/>
+    <xacro:property name="HipPitch_pitch" value="${-PI_2}"/>
+    <xacro:property name="HipPitch_yaw" value="${PI_2}"/>
     <!-- Origin -->
     <xacro:property name="KneePitch_Ox" value="0.0"/>
     <xacro:property name="KneePitch_Oy" value="${-346.000 * mmTom}"/>
-    <xacro:property name="KneePitch_Oz" value="${166.710 * mmTom}"/>
+    <xacro:property name="KneePitch_Oz" value="${246.060 * mmTom}"/>
     <xacro:property name="KneePitch_roll" value="0.0"/>
     <xacro:property name="KneePitch_pitch" value="0.0"/>
     <xacro:property name="KneePitch_yaw" value="0.0"/>
     <xacro:property name="AnkleYaw_Ox" value="0.0"/>
-    <xacro:property name="AnkleYaw_Oy" value="${-10.000 * mmTom}"/>
-    <xacro:property name="AnkleYaw_Oz" value="${67.000 * mmTom}"/>
+    <xacro:property name="AnkleYaw_Oy" value="${-73.500 * mmTom}"/>
+    <xacro:property name="AnkleYaw_Oz" value="${59.000 * mmTom}"/>
     <xacro:property name="AnkleYaw_roll" value="-${PI_2}"/>
     <xacro:property name="AnkleYaw_pitch" value="0.0"/>
@@ -63,6 +63,6 @@
     <xacro:property name="SteeringWheel_Ox" value="0.0"/>
     <xacro:property name="SteeringWheel_Oy" value="0.0"/>
-    <xacro:property name="SteeringWheel_Oz" value="${-290.000 * mmTom}"/>
-    <xacro:property name="SteeringWheel_roll" value="${PI_2}"/>
+    <xacro:property name="SteeringWheel_Oz" value="${-226.500 * mmTom}"/>
+    <xacro:property name="SteeringWheel_roll" value="-${PI_2}"/>
     <xacro:property name="SteeringWheel_pitch" value="0.0"/>
     <xacro:property name="SteeringWheel_yaw" value="0.0"/>

File: kyon_urdf/urdf/parts/kyon_leg.urdf.xacro (robot description, xacro)
@@ -10,7 +10,7 @@
 <link name="hip_roll_${leg_num}_link">
 	<inertial>
-		<origin xyz="0.0 0.0 0.0"/>
-		<mass value="${motorA_mass}"/>
-		<inertia ixx="${MotorA_xx}" ixy="${mirror*MotorA_xy}" ixz="${MotorA_xz}" iyy="${MotorA_yy}" iyz="${mirror*MotorA_yz}" izz="${MotorA_zz}"/>
+		<origin xyz="${HipRoll_x} ${HipRoll_y} ${HipRoll_z}"/>
+		<mass value="${HipRoll_mass}"/>
+		<inertia ixx="${HipRoll_xx}" ixy="${mirror*HipRoll_xy}" ixz="${HipRoll_xz}" iyy="${HipRoll_yy}" iyz="${mirror*HipRoll_yz}" izz="${HipRoll_zz}"/>
 	</inertial>
 	<visual>
@@ -32,7 +32,7 @@
 <link name="hip_pitch_${leg_num}_link">
 	<inertial>
-		<origin xyz="0.0 0.0 0.0"/>
-		<mass value="${motorA_mass}"/>
-		<inertia ixx="${MotorA_xx}" ixy="${MotorA_xy}" ixz="${MotorA_xz}" iyy="${MotorA_yy}" iyz="${MotorA_yz}" izz="${MotorA_zz}"/>
+		<origin xyz="${HipPitch_x} ${HipPitch_y} ${HipPitch_z}"/>
+		<mass value="${HipPitch_mass}"/>
+		<inertia ixx="${HipPitch_xx}" ixy="${HipPitch_xy}" ixz="${HipPitch_xz}" iyy="${HipPitch_yy}" iyz="${HipPitch_yz}" izz="${HipPitch_zz}"/>
 	</inertial>
 	<visual>
@@ -61,5 +61,5 @@
 	<parent link="hip_roll_${leg_num}_link"/>
 	<child link="hip_pitch_${leg_num}_link"/>
-	<origin xyz="${origin_x * HipPitch_Ox} ${origin_y * HipPitch_Oy} ${HipPitch_Oz}" rpy="${origin_y*HipPitch_roll} ${origin_x*origin_y*HipPitch_pitch} ${HipPitch_yaw}"/>
+	<origin xyz="${HipPitch_Ox} ${origin_y * HipPitch_Oy} ${HipPitch_Oz}" rpy="${HipPitch_roll} ${origin_x * origin_y * HipPitch_pitch} ${origin_x * HipPitch_yaw}"/>
 	<axis xyz="0 0 1"/>
 	<limit lower="${hip_pitch_lower[leg_num-1]}" upper="${hip_pitch_upper[leg_num-1]}" effort="${motor_effort}" velocity="${motor_velocity}"/>

File: kyon_urdf/urdf/parts/legs.urdf.xacro (robot description, xacro)
@@ -2,11 +2,11 @@
 <robot xmlns:xacro="http://ros.org/wiki/xacro">
 <xacro:include filename="$(find kyon_urdf)/urdf/parts/kyon_leg.urdf.xacro" />
-<xacro:kyon_leg leg_num="1" origin_x="1" origin_y="1" mirror="-1">
+<xacro:kyon_leg leg_num="1" origin_x="1" origin_y="-1" mirror="-1">
 </xacro:kyon_leg>
-<xacro:kyon_leg leg_num="2" origin_x="1" origin_y="-1" mirror="1">
+<xacro:kyon_leg leg_num="2" origin_x="1" origin_y="1" mirror="1">
 </xacro:kyon_leg>
-<xacro:kyon_leg leg_num="3" origin_x="-1" origin_y="1" mirror="-1">
+<xacro:kyon_leg leg_num="3" origin_x="-1" origin_y="-1" mirror="-1">
 </xacro:kyon_leg>
-<xacro:kyon_leg leg_num="4" origin_x="-1" origin_y="-1" mirror="1">
+<xacro:kyon_leg leg_num="4" origin_x="-1" origin_y="1" mirror="1">
 </xacro:kyon_leg>
 </robot>

File: kyon_urdf/urdf/parts/steering_wheel.urdf.xacro (robot description, xacro)
@@ -5,7 +5,7 @@
 <link name="knee_pitch_${leg_num}_link">
     <inertial>
-		<origin xyz="0.0 0.0 0.0"/>
-		<mass value="${motorA_mass}"/>
-		<inertia ixx="${MotorA_xx}" ixy="${mirror*MotorA_xy}" ixz="${MotorA_xz}" iyy="${MotorA_yy}" iyz="${mirror*MotorA_yz}" izz="${MotorA_zz}"/>
+		<origin xyz="${KneePitch_x} ${KneePitch_y} ${KneePitch_z}"/>
+		<mass value="${KneePitch_mass}"/>
+		<inertia ixx="${KneePitch_xx}" ixy="${KneePitch_xy}" ixz="${KneePitch_xz}" iyy="${KneePitch_yy}" iyz="${KneePitch_yz}" izz="${KneePitch_zz}"/>
 	</inertial>
 	<visual>
@@ -27,7 +27,7 @@
 <link name="ankle_yaw_${leg_num}_link">
     <inertial>
-		<origin xyz="0.0 0.0 0.0"/>
-		<mass value="${motorA_mass}"/>
-		<inertia ixx="${MotorA_xx}" ixy="${mirror*MotorA_xy}" ixz="${MotorA_xz}" iyy="${MotorA_yy}" iyz="${mirror*MotorA_yz}" izz="${MotorA_zz}"/>
+		<origin xyz="${AnkleYaw_x} ${AnkleYaw_y} ${AnkleYaw_z}"/>
+		<mass value="${AnkleYaw_mass}"/>
+		<inertia ixx="${AnkleYaw_xx}" ixy="${AnkleYaw_xy}" ixz="${AnkleYaw_xz}" iyy="${AnkleYaw_yy}" iyz="${AnkleYaw_yz}" izz="${AnkleYaw_zz}"/>
 	</inertial>
 	<visual>
@@ -49,7 +49,7 @@
 <link name="wheel_${leg_num}_link">
     <inertial>
-		<origin xyz="0.0 0.0 0.0"/>
-		<mass value="${motorA_mass}"/>
-		<inertia ixx="${MotorA_xx}" ixy="${mirror*MotorA_xy}" ixz="${MotorA_xz}" iyy="${MotorA_yy}" iyz="${mirror*MotorA_yz}" izz="${MotorA_zz}"/>
+		<origin xyz="${SteeringWheel_x} ${SteeringWheel_y} ${SteeringWheel_z}"/>
+		<mass value="${SteeringWheel_mass}"/>
+		<inertia ixx="${SteeringWheel_xx}" ixy="${SteeringWheel_xy}" ixz="${SteeringWheel_xz}" iyy="${SteeringWheel_yy}" iyz="${SteeringWheel_yz}" izz="${SteeringWheel_zz}"/>
 	</inertial>
 	<visual>
