Commit message: updated meshes and inertias for upper body

File: kyon_urdf/urdf/kyon.urdf (robot description, URDF)
Before this commit: robot kyon, 38 links, 37 joints
Links:
- link elbow_pitch_1_link: mass 0.77 -> 1.048477
- link elbow_pitch_2_link: mass 0.77 -> 1.048477
- link pelvis: mass 32.642743 -> 23.024083
- link shoulder_pitch_1_link: mass 1.8 -> 2.6591536
- link shoulder_pitch_2_link: mass 1.8 -> 2.6591536
- link shoulder_yaw_1_link: mass 1.6 -> 0.67826074
- link shoulder_yaw_2_link: mass 1.6 -> 0.67826074
- link wrist_pitch_1_link: mass 0.63 -> 0.8276976
- link wrist_pitch_2_link: mass 0.63 -> 0.8276976
- link wrist_yaw_1_link: mass 0.63 -> 0.11855953
- link wrist_yaw_2_link: mass 0.63 -> 0.11855953
Joints:
- joint elbow_pitch_1: origin xyz=0.0 0.0 0.32 rpy=-1.57079632679 0.0 0.0 -> xyz=0.0 -0.32 0.0 rpy=0.0 0.0 0.0
- joint elbow_pitch_2: origin xyz=0.0 0.0 0.32 rpy=-1.57079632679 0.0 0.0 -> xyz=0.0 -0.32 0.0 rpy=0.0 0.0 0.0
- joint shoulder_pitch_1: origin xyz=0.0 0.0 0.0735 rpy=0.0 0.0 3.14159265358 -> xyz=0.0 0.0 0.0735 rpy=-1.57079632679 0.0 -3.14159265358
- joint shoulder_pitch_2: origin xyz=0.0 0.0 0.0735 rpy=0.0 0.0 0.0 -> xyz=0.0 0.0 0.0735 rpy=-1.57079632679 0.0 0.0
- joint shoulder_yaw_1: origin xyz=0.28 0.0966072 0.203559 rpy=-0.3490656 0.0 0.0 -> xyz=0.28 0.0998258 0.203238 rpy=-0.3490656 0.0 0.0
- joint shoulder_yaw_2: origin xyz=0.28 -0.0966072 0.203559 rpy=0.3490656 0.0 0.0 -> xyz=0.28 -0.0998258 0.203238 rpy=0.3490656 0.0 0.0
- joint wrist_pitch_1: origin xyz=0.0 -0.25 -0.020502500000000003 rpy=-3.14159265359 0.0 0.0 -> xyz=0.0 -0.25 0.0 rpy=0.0 0.0 0.0
- joint wrist_pitch_2: origin xyz=0.0 -0.25 -0.020502500000000003 rpy=-3.14159265359 0.0 0.0 -> xyz=0.0 -0.25 0.0 rpy=0.0 0.0 0.0
- joint wrist_yaw_1: origin xyz=0.0 0.11586199999999999 -0.02036 rpy=-1.57079632679 0.0 0.0 -> xyz=0.0 -0.134862 0.0 rpy=1.57079632679 0.0 0.0
- joint wrist_yaw_2: origin xyz=0.0 0.11586199999999999 -0.02036 rpy=-1.57079632679 0.0 0.0 -> xyz=0.0 -0.134862 0.0 rpy=1.57079632679 0.0 0.0

File: kyon_urdf/urdf/parts/arms.urdf.xacro (robot description, xacro)
@@ -3,7 +3,7 @@
 <xacro:include filename="$(find kyon_urdf)/urdf/parts/kyon_arm.urdf.xacro"/>
 <!-- arms -->
-<xacro:kyon_arm arm_num="1"  rot="1"  parent="pelvis">
+<xacro:kyon_arm arm_num="1"  rot="-1"  parent="pelvis">
 </xacro:kyon_arm>
-<xacro:kyon_arm arm_num="2" rot="-1"  parent="pelvis">
+<xacro:kyon_arm arm_num="2" rot="1"  parent="pelvis">
 </xacro:kyon_arm>
 <xacro:if value="${PAYLOAD}">

File: kyon_urdf/urdf/parts/inertial_properties.urdf.xacro (robot description, xacro)
@@ -42,14 +42,14 @@
     <xacro:property name="MotorArm3_zz" value="${1/2 * motor_arm3_mass * cylinder_radius * cylinder_radius}"/>
     <!-- Pelvis -->
-    <xacro:property name="Pelvis_mass" value="32.642743"/>
-    <xacro:property name="Pelvis_x" value="${3.5990152e+01 * mmTom}"/>
-    <xacro:property name="Pelvis_y" value="${-3.0735925e+01 * mmTom}"/>
-    <xacro:property name="Pelvis_z" value="${3.7859444e+01 * mmTom}"/>
-    <xacro:property name="Pelvis_xx" value="${3.5499677e+05 * mm2Tom2}"/>
-    <xacro:property name="Pelvis_xy" value="${-3.9512772e+04 * mm2Tom2}"/>
-    <xacro:property name="Pelvis_xz" value="${-9.9657679e+04 * mm2Tom2}"/>
-    <xacro:property name="Pelvis_yy" value="${1.2528724e+06 * mm2Tom2}"/>
-    <xacro:property name="Pelvis_yz" value="${-5.5537486e+04 * mm2Tom2}"/>
-    <xacro:property name="Pelvis_zz" value="${1.2807784e+06 * mm2Tom2}"/>
+    <xacro:property name="Pelvis_mass" value="23.024083"/>
+    <xacro:property name="Pelvis_x" value="${4.9723680e+01 * mmTom}"/>
+    <xacro:property name="Pelvis_y" value="${2.2995169e+00 * mmTom}"/>
+    <xacro:property name="Pelvis_z" value="${5.8657543e+01 * mmTom}"/>
+    <xacro:property name="Pelvis_xx" value="${2.5825843e+05 * mm2Tom2}"/>
+    <xacro:property name="Pelvis_xy" value="${-1.5196886e+03 * mm2Tom2}"/>
+    <xacro:property name="Pelvis_xz" value="${-7.4270479e+04 * mm2Tom2}"/>
+    <xacro:property name="Pelvis_yy" value="${1.2128223e+06 * mm2Tom2}"/>
+    <xacro:property name="Pelvis_yz" value="${3.9226759e+03 * mm2Tom2}"/>
+    <xacro:property name="Pelvis_zz" value="${1.1693352e+06 * mm2Tom2}"/>
     <!-- Hip Roll -->
     <xacro:property name="HipRoll_mass" value="2.7479472"/>
@@ -118,30 +118,58 @@
 	<xacro:property name="SteeringWheel_yz" value="${0.0 * mm2Tom2}"/>
 	<xacro:property name="SteeringWheel_zz" value="${7.9333497e+03 * mm2Tom2}"/>
-    <!-- Upper Arm -->
-    <xacro:property name="UpperArm1_xx" value="${1/12 * upper_arm1_mass * (upper_arm1_width * upper_arm1_width + upper_arm1_height * upper_arm1_height)}"/>
-    <xacro:property name="UpperArm1_xy" value="0.0"/>
-    <xacro:property name="UpperArm1_xz" value="0.0"/>
-    <xacro:property name="UpperArm1_yy" value="${1/12 * upper_arm1_mass * (upper_arm1_length * upper_arm1_length + upper_arm1_height * upper_arm1_height)}"/>
-    <xacro:property name="UpperArm1_yz" value="0.0"/>
-    <xacro:property name="UpperArm1_zz" value="${1/12 * upper_arm1_mass * (upper_arm1_width * upper_arm1_width + upper_arm1_length * upper_arm1_length)}"/>
-    <xacro:property name="UpperArm2_xx" value="${1/12 * upper_arm2_mass * (upper_arm2_width * upper_arm2_width + upper_arm2_height * upper_arm2_height)}"/>
-    <xacro:property name="UpperArm2_xy" value="0.0"/>
-    <xacro:property name="UpperArm2_xz" value="0.0"/>
-    <xacro:property name="UpperArm2_yy" value="${1/12 * upper_arm2_mass * (upper_arm2_length * upper_arm2_length + upper_arm2_height * upper_arm2_height)}"/>
-    <xacro:property name="UpperArm2_yz" value="0.0"/>
-    <xacro:property name="UpperArm2_zz" value="${1/12 * upper_arm2_mass * (upper_arm2_width * upper_arm2_width + upper_arm2_length * upper_arm2_length)}"/>
-    <!-- Lower Arm -->
-    <xacro:property name="LowerArm_xx" value="${1/12 * lower_arm_mass * (lower_arm_width * lower_arm_width + lower_arm_height * lower_arm_height)}"/>
-    <xacro:property name="LowerArm_xy" value="0.0"/>
-    <xacro:property name="LowerArm_xz" value="0.0"/>
-    <xacro:property name="LowerArm_yy" value="${1/12 * lower_arm_mass * (lower_arm_length * lower_arm_length + lower_arm_height * lower_arm_height)}"/>
-    <xacro:property name="LowerArm_yz" value="0.0"/>
-    <xacro:property name="LowerArm_zz" value="${1/12 * lower_arm_mass * (lower_arm_width * lower_arm_width + lower_arm_length * lower_arm_length)}"/>
-    <!-- Ball (hollow sphere) -->
-    <xacro:property name="Ball_xx" value="${2/3 * ball_mass * ball_radius * ball_radius}"/>
-    <xacro:property name="Ball_xy" value="0.0"/>
-    <xacro:property name="Ball_xz" value="0.0"/>
-    <xacro:property name="Ball_yy" value="${2/3 * ball_mass * ball_radius * ball_radius}"/>
-    <xacro:property name="Ball_yz" value="0.0"/>
-    <xacro:property name="Ball_zz" value="${2/3 * ball_mass * ball_radius * ball_radius}"/>
+    <!-- Shoulder Yaw -->
+    <xacro:property name="ShoulderYaw_mass" value="0.67826074"/>
+    <xacro:property name="ShoulderYaw_x" value="${0.0 * mmTom}"/>
+    <xacro:property name="ShoulderYaw_y" value="${-1.3492411e-01 * mmTom}"/>
+    <xacro:property name="ShoulderYaw_z" value="${4.0858984e+01 * mmTom}"/>
+    <xacro:property name="ShoulderYaw_xx" value="${2.5001499e+03 * mm2Tom2}"/>
+    <xacro:property name="ShoulderYaw_xy" value="${-6.3655528e-01 * mm2Tom2}"/>
+    <xacro:property name="ShoulderYaw_xz" value="${1.7271059e-01 * mm2Tom2}"/>
+    <xacro:property name="ShoulderYaw_yy" value="${1.9131559e+03 * mm2Tom2}"/>
+    <xacro:property name="ShoulderYaw_yz" value="${-6.5053652e+01 * mm2Tom2}"/>
+    <xacro:property name="ShoulderYaw_zz" value="${1.9311455e+03 * mm2Tom2}"/>
+    <!-- Shoulder Pitch -->
+    <xacro:property name="ShoulderPitch_mass" value="2.6591536"/>
+    <xacro:property name="ShoulderPitch_x" value="${-8.8212748e-03 * mmTom}"/>
+    <xacro:property name="ShoulderPitch_y" value="${-1.4226587e+02 * mmTom}"/>
+    <xacro:property name="ShoulderPitch_z" value="${-4.0603042e+00 * mmTom}"/>
+    <xacro:property name="ShoulderPitch_xx" value="${5.9933923e+04 * mm2Tom2}"/>
+    <xacro:property name="ShoulderPitch_xy" value="${1.0630782e+02 * mm2Tom2}"/>
+    <xacro:property name="ShoulderPitch_xz" value="${-8.1788344e+00 * mm2Tom2}"/>
+    <xacro:property name="ShoulderPitch_yy" value="${3.2807639e+03 * mm2Tom2}"/>
+    <xacro:property name="ShoulderPitch_yz" value="${-1.0925330e+03 * mm2Tom2}"/>
+    <xacro:property name="ShoulderPitch_zz" value="${5.9801168e+04 * mm2Tom2}"/>
+   <!-- Elbow Pitch -->
+    <xacro:property name="ElbowPitch_mass" value="1.0484770"/>
+    <xacro:property name="ElbowPitch_x" value="${-3.2761312e-01 * mmTom}"/>
+    <xacro:property name="ElbowPitch_y" value="${-1.6511035e+02 * mmTom}"/>
+    <xacro:property name="ElbowPitch_z" value="${2.2799378e+01 * mmTom}"/>
+    <xacro:property name="ElbowPitch_xx" value="${1.1126010e+04 * mm2Tom2}"/>
+    <xacro:property name="ElbowPitch_xy" value="${1.7724864e+01 * mm2Tom2}"/>
+    <xacro:property name="ElbowPitch_xz" value="${6.0670899e+00 * mm2Tom2}"/>
+    <xacro:property name="ElbowPitch_yy" value="${9.5730481e+02 * mm2Tom2}"/>
+    <xacro:property name="ElbowPitch_yz" value="${-1.0167295e+03 * mm2Tom2}"/>
+    <xacro:property name="ElbowPitch_zz" value="${1.1293246e+04 * mm2Tom2}"/>
+    <!-- Wrist Pitch -->
+    <xacro:property name="WristPitch_mass" value="0.82769760"/>
+    <xacro:property name="WristPitch_x" value="${-3.5889306e-01 * mmTom}"/>
+    <xacro:property name="WristPitch_y" value="${-5.6046555e+01 * mmTom}"/>
+    <xacro:property name="WristPitch_z" value="${-1.0441123e+01 * mmTom}"/>
+    <xacro:property name="WristPitch_xx" value="${1.8979250e+03 * mm2Tom2}"/>
+    <xacro:property name="WristPitch_xy" value="${1.5812980e+01 * mm2Tom2}"/>
+    <xacro:property name="WristPitch_xz" value="${-8.8320155e+00 * mm2Tom2}"/>
+    <xacro:property name="WristPitch_yy" value="${7.2693403e+02 * mm2Tom2}"/>
+    <xacro:property name="WristPitch_yz" value="${4.4823508e+02 * mm2Tom2}"/>
+    <xacro:property name="WristPitch_zz" value="${1.8533681e+03 * mm2Tom2}"/>
+    <!-- Wrist Yaw -->
+    <xacro:property name="WristYaw_mass" value="0.11855953"/>
+    <xacro:property name="WristYaw_x" value="${0.0 * mmTom}"/>
+    <xacro:property name="WristYaw_y" value="${-1.8381849e-02 * mmTom}"/>
+    <xacro:property name="WristYaw_z" value="${-1.6592053e+01 * mmTom}"/>
+    <xacro:property name="WristYaw_xx" value="${7.0481525e+01 * mm2Tom2}"/>
+    <xacro:property name="WristYaw_xy" value="${-1.3031027e-01 * mm2Tom2}"/>
+    <xacro:property name="WristYaw_xz" value="${0.0000000e+00 * mm2Tom2}"/>
+    <xacro:property name="WristYaw_yy" value="${7.3847541e+01 * mm2Tom2}"/>
+    <xacro:property name="WristYaw_yz" value="${-2.5372645e-02 * mm2Tom2}"/>
+    <xacro:property name="WristYaw_zz" value="${1.1802904e+02 * mm2Tom2}"/>
 </robot>

File: kyon_urdf/urdf/parts/kinematics_properties.urdf.xacro (robot description, xacro)
@@ -69,6 +69,6 @@
     <!-- Arms -->
     <xacro:property name="ShoulderYaw_Ox" value="${280.00 * mmTom}"/>
-    <xacro:property name="ShoulderYaw_Oy" value="${96.6072 * mmTom}"/>
-    <xacro:property name="ShoulderYaw_Oz" value="${203.559 * mmTom}"/>
+    <xacro:property name="ShoulderYaw_Oy" value="${-99.8258 * mmTom}"/>
+    <xacro:property name="ShoulderYaw_Oz" value="${203.238 * mmTom}"/>
     <xacro:property name="ShoulderYaw_roll" value="0.3490656"/>
     <xacro:property name="ShoulderYaw_pitch" value="0.0"/>
@@ -77,23 +77,23 @@
     <xacro:property name="ShoulderPitch_Oy" value="0.0"/>
     <xacro:property name="ShoulderPitch_Oz" value="${73.5 * mmTom}"/>
-    <xacro:property name="ShoulderPitch_roll" value="0.0"/>
+    <xacro:property name="ShoulderPitch_roll" value="-${PI_2}"/>
     <xacro:property name="ShoulderPitch_pitch" value="0.0"/>
-    <xacro:property name="ShoulderPitch_yaw" value="${PI_2}"/>
+    <xacro:property name="ShoulderPitch_yaw" value="${-PI_2}"/>
     <xacro:property name="ElbowPitch_Ox" value="0.0"/>
-    <xacro:property name="ElbowPitch_Oy" value="0.0"/>
-    <xacro:property name="ElbowPitch_Oz" value="${320.00 * mmTom}"/>
-    <xacro:property name="ElbowPitch_roll" value="${-PI_2}"/>
+    <xacro:property name="ElbowPitch_Oy" value="${-320.00 * mmTom}"/>
+    <xacro:property name="ElbowPitch_Oz" value="0.0"/>
+    <xacro:property name="ElbowPitch_roll" value="0.0"/>
     <xacro:property name="ElbowPitch_pitch" value="0.0"/>
     <xacro:property name="ElbowPitch_yaw" value="0.0"/>
     <xacro:property name="WristPitch_Ox" value="0.0"/>
 	<xacro:property name="WristPitch_Oy" value="${-250.00 * mmTom}"/>
-	<xacro:property name="WristPitch_Oz" value="${-20.5025 * mmTom}"/>
-	<xacro:property name="WristPitch_roll" value="${-PI}"/>
+	<xacro:property name="WristPitch_Oz" value="0.0"/>
+	<xacro:property name="WristPitch_roll" value="0.0"/>
 	<xacro:property name="WristPitch_pitch" value="0.0"/>
 	<xacro:property name="WristPitch_yaw" value="0.0"/>
     <xacro:property name="WristYaw_Ox" value="0.0"/>
-	<xacro:property name="WristYaw_Oy" value="${115.862 * mmTom}"/>
-	<xacro:property name="WristYaw_Oz" value="${-20.360 * mmTom}"/>
-	<xacro:property name="WristYaw_roll" value="${-PI_2}"/>
+	<xacro:property name="WristYaw_Oy" value="${-134.862 * mmTom}"/>
+	<xacro:property name="WristYaw_Oz" value="0.0"/>
+	<xacro:property name="WristYaw_roll" value="${PI_2}"/>
 	<xacro:property name="WristYaw_pitch" value="0.0"/>
 	<xacro:property name="WristYaw_yaw" value="0.0"/>

File: kyon_urdf/urdf/parts/kyon_arm.urdf.xacro (robot description, xacro)
@@ -8,7 +8,7 @@
 <link name="shoulder_yaw_${arm_num}_link">
 	<inertial>
-		<origin xyz="0.0 0.0 0.0"/>
-		<mass value="${motor_arm1_mass + 0.68}"/>
-		<inertia ixx="${MotorArm1_xx}" ixy="${MotorArm1_xy}" ixz="${MotorArm1_xz}" iyy="${MotorArm1_yy}" iyz="${MotorArm1_yz}" izz="${MotorArm1_zz}"/>
+		<origin xyz="${ShoulderYaw_x} ${ShoulderYaw_y} ${ShoulderYaw_z}"/>
+		<mass value="${ShoulderYaw_mass}"/>
+		<inertia ixx="${ShoulderYaw_xx}" ixy="${ShoulderYaw_xy}" ixz="${ShoulderYaw_xz}" iyy="${ShoulderYaw_yy}" iyz="${ShoulderYaw_yz}" izz="${ShoulderYaw_zz}"/>
 	</inertial>
 	<visual>
@@ -28,7 +28,7 @@
 <link name="shoulder_pitch_${arm_num}_link">
 	<inertial>
-		<origin xyz="0.0 0.0 0.0"/>
-		<mass value="${lower_arm_mass + motor_arm2_mass}"/>
-		<inertia ixx="${LowerArm_xx}" ixy="${LowerArm_xy}" ixz="${LowerArm_xz}" iyy="${LowerArm_yy}" iyz="${LowerArm_yz}" izz="${LowerArm_zz}"/>
+		<origin xyz="${ShoulderPitch_x} ${ShoulderPitch_y} ${ShoulderPitch_z}"/>
+		<mass value="${ShoulderPitch_mass}"/>
+		<inertia ixx="${ShoulderPitch_xx}" ixy="${ShoulderPitch_xy}" ixz="${ShoulderPitch_xz}" iyy="${ShoulderPitch_yy}" iyz="${ShoulderPitch_yz}" izz="${ShoulderPitch_zz}"/>
 	</inertial>
 	<visual>
@@ -46,7 +46,7 @@
 <link name="elbow_pitch_${arm_num}_link">
 	<inertial>
-		<origin xyz="${upper_arm1_length / 2} 0.0 0.0"/>
-		<mass value="${upper_arm1_mass}"/>
-		<inertia ixx="${UpperArm1_xx}" ixy="${UpperArm1_xy}" ixz="${UpperArm1_xz}" iyy="${UpperArm1_yy}" iyz="${UpperArm1_yz}" izz="${UpperArm1_zz}"/>
+		<origin xyz="${ElbowPitch_x} ${ElbowPitch_y} ${ElbowPitch_z}"/>
+		<mass value="${ElbowPitch_mass}"/>
+		<inertia ixx="${ElbowPitch_xx}" ixy="${ElbowPitch_xy}" ixz="${ElbowPitch_xz}" iyy="${ElbowPitch_yy}" iyz="${ElbowPitch_yz}" izz="${ElbowPitch_zz}"/>
 	</inertial>
 	<visual>
@@ -63,7 +63,7 @@
 <link name="wrist_pitch_${arm_num}_link">
 	<inertial>
-		<origin xyz="0.0 0.0 0.0"/>
-		<mass value="${motor_arm3_mass}"/>
-		<inertia ixx="${MotorArm3_xx}" ixy="${MotorArm3_xy}" ixz="${MotorArm3_xz}" iyy="${MotorArm3_yy}" iyz="${MotorArm3_yz}" izz="${MotorArm3_zz}"/>
+		<origin xyz="${WristPitch_x} ${WristPitch_y} ${WristPitch_z}"/>
+		<mass value="${WristPitch_mass}"/>
+		<inertia ixx="${WristPitch_xx}" ixy="${WristPitch_xy}" ixz="${WristPitch_xz}" iyy="${WristPitch_yy}" iyz="${WristPitch_yz}" izz="${WristPitch_zz}"/>
 	</inertial>
 	<visual>
@@ -83,7 +83,7 @@
 <link name="wrist_yaw_${arm_num}_link">
 	<inertial>
-		<origin xyz="0.0 0.0 0.0"/>
-		<mass value="${motor_arm3_mass}"/>
-		<inertia ixx="${MotorArm3_xx}" ixy="${MotorArm3_xy}" ixz="${MotorArm3_xz}" iyy="${MotorArm3_yy}" iyz="${MotorArm3_yz}" izz="${MotorArm3_zz}"/>
+		<origin xyz="${WristYaw_x} ${WristYaw_y} ${WristYaw_z}"/>
+		<mass value="${WristYaw_mass}"/>
+		<inertia ixx="${WristYaw_xx}" ixy="${WristYaw_xy}" ixz="${WristYaw_xz}" iyy="${WristYaw_yy}" iyz="${WristYaw_yz}" izz="${WristYaw_zz}"/>
 	</inertial>
 	<visual>
@@ -107,5 +107,5 @@
 	<parent link="${parent}"/>
 	<child link="shoulder_yaw_${arm_num}_link"/>
-	<origin xyz="${ShoulderYaw_Ox} ${rot * ShoulderYaw_Oy} ${ShoulderYaw_Oz}" rpy="${-rot * ShoulderYaw_roll} ${ShoulderYaw_pitch} ${ShoulderYaw_yaw}"/>
+	<origin xyz="${ShoulderYaw_Ox} ${rot * ShoulderYaw_Oy} ${ShoulderYaw_Oz}" rpy="${rot * ShoulderYaw_roll} ${ShoulderYaw_pitch} ${ShoulderYaw_yaw}"/>
 	<axis xyz="0 0 1"/>
 	<limit lower="${j_shoulder_yaw_lower[arm_num-1]}" upper="${j_shoulder_yaw_upper[arm_num-1]}" effort="${motor_effort}" velocity="${motor_velocity}"/>
@@ -115,5 +115,5 @@
 	<parent link="shoulder_yaw_${arm_num}_link"/>
 	<child link="shoulder_pitch_${arm_num}_link"/>
-	<origin xyz="${ShoulderPitch_Ox} ${ShoulderPitch_Oy} ${ShoulderPitch_Oz}" rpy="${ShoulderPitch_roll} ${ShoulderPitch_pitch} ${ShoulderPitch_yaw  + rot * PI_2}"/>
+	<origin xyz="${ShoulderPitch_Ox} ${ShoulderPitch_Oy} ${ShoulderPitch_Oz}" rpy="${ShoulderPitch_roll} ${ShoulderPitch_pitch} ${ShoulderPitch_yaw + rot * PI_2}"/>
 	<axis xyz="0 1 0"/>
 	<limit lower="${j_pitch_1_lower[arm_num-1]}" upper="${j_pitch_1_upper[arm_num-1]}" effort="${motor_effort}" velocity="${motor_velocity}"/>

File: kyon_urdf/urdf/parts/wheel_leg.urdf.xacro (robot description, xacro)
@@ -32,5 +32,4 @@
 		<origin xyz="0.0 0.0 0.0"  rpy="0.0 0.0 0.0"/>
 	  	<geometry>
-	 		<!-- <cylinder radius="${cylinder_radius}" length="${cylinder_length}"/> -->
 			<mesh filename="package://kyon_urdf/meshes/mesh_wheel.stl" scale="0.001 0.001 0.001"/>
 		</geometry>
@@ -40,5 +39,4 @@
 		<origin xyz="0.0 0.0 0.0"  rpy="0.0 0.0 0.0"/>
 		<geometry>
-	 		<!-- <cylinder radius="${cylinder_radius}" length="${cylinder_length}"/> -->
 			<mesh filename="package://kyon_urdf/meshes/collision/mesh_wheel.stl" scale="0.001 0.001 0.001"/>
 		</geometry>

Commit message: capsule && generated files

File: kyon_urdf/urdf/kyon.urdf (robot description, URDF)
Before this commit: robot kyon, 38 links, 37 joints
Links:
- removed link ankle_yaw_1_link
- removed link ankle_yaw_2_link
- removed link ankle_yaw_3_link
- removed link ankle_yaw_4_link
- removed link dagana_1_clamp
- removed link dagana_2_clamp
- removed link wheel_1_link
- removed link wheel_2_link
- removed link wheel_3_link
- removed link wheel_4_link
- added link contact_1
- added link contact_2
- added link contact_3
- added link contact_4
- added link dagana_1_claw, mass 0.25739835; collision mesh filename=package://kyon_urdf/meshes/collision/mesh_dagana-clamp.stl scale=0.001 0.001 0.001; visual mesh filename=package://kyon_urdf/meshes/mesh_dagana-clamp.stl scale=0.001 0.001 0.001
- added link dagana_2_claw, mass 0.25739835; collision mesh filename=package://kyon_urdf/meshes/collision/mesh_dagana-clamp.stl scale=0.001 0.001 0.001; visual mesh filename=package://kyon_urdf/meshes/mesh_dagana-clamp.stl scale=0.001 0.001 0.001
- link dagana_1_base: mass 1.8 -> 0.96534359
- link dagana_2_base: mass 1.8 -> 0.96534359
- link knee_pitch_1_link: mass 1.4555296 -> 0.70900216; geometry collision mesh filename=package://kyon_urdf/meshes/collision/mesh_foot-leg.stl scale=-0.001 0.001 0.001; visual mesh filename=package://kyon_urdf/meshes/mesh_foot-leg.stl scale=-0.001 0.001 0.001
- link knee_pitch_2_link: mass 1.4555296 -> 0.70900216; geometry collision mesh filename=package://kyon_urdf/meshes/collision/mesh_foot-leg.stl scale=0.001 0.001 0.001; visual mesh filename=package://kyon_urdf/meshes/mesh_foot-leg.stl scale=0.001 0.001 0.001
- link knee_pitch_3_link: mass 1.4555296 -> 0.70900216; geometry collision mesh filename=package://kyon_urdf/meshes/collision/mesh_foot-leg.stl scale=-0.001 0.001 0.001; visual mesh filename=package://kyon_urdf/meshes/mesh_foot-leg.stl scale=-0.001 0.001 0.001
- link knee_pitch_4_link: mass 1.4555296 -> 0.70900216; geometry collision mesh filename=package://kyon_urdf/meshes/collision/mesh_foot-leg.stl scale=0.001 0.001 0.001; visual mesh filename=package://kyon_urdf/meshes/mesh_foot-leg.stl scale=0.001 0.001 0.001
Joints:
- removed joint ankle_yaw_1
- removed joint ankle_yaw_2
- removed joint ankle_yaw_3
- removed joint ankle_yaw_4
- removed joint imu_link
- removed joint wheel_joint_1
- removed joint wheel_joint_2
- removed joint wheel_joint_3
- removed joint wheel_joint_4
- added joint contact_1_joint: type fixed, parent knee_pitch_1_link, child contact_1, origin xyz=0.03 -0.35 0.03 rpy=-1.57 0 0.785
- added joint contact_2_joint: type fixed, parent knee_pitch_2_link, child contact_2, origin xyz=-0.03 -0.35 0.03 rpy=1.57 0 2.356
- added joint contact_3_joint: type fixed, parent knee_pitch_3_link, child contact_3, origin xyz=0.03 -0.35 0.03 rpy=-1.57 0 0.785
- added joint contact_4_joint: type fixed, parent knee_pitch_4_link, child contact_4, origin xyz=-0.03 -0.35 0.03 rpy=1.57 0 2.356
- added joint imu_joint: type fixed, parent pelvis, child imu_link
- joint dagana_1_clamp_joint: child dagana_1_clamp -> dagana_1_claw
- joint dagana_2_clamp_joint: child dagana_2_clamp -> dagana_2_claw
- joint shoulder_pitch_1: axis 0 1 0 -> 0 0 1
- joint shoulder_pitch_2: axis 0 1 0 -> 0 0 1
