Commit message: re-generate urdf, srdf for fix directions in arm joints

File: kyon_urdf/urdf/kyon.urdf (robot description, URDF)
Before this commit: robot kyon, 34 links, 33 joints
Links:
- link dagana_1_base: geometry collision mesh filename=package://kyon_urdf/meshes/collision/mesh_dagana-base-base-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 scale=0.001 0.001 0.001; collision mesh filename=package://kyon_urdf/meshes/collision/mesh_dagana-base-simpl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 scale=0.001 0.001 0.001
- link dagana_1_claw: geometry collision mesh filename=package://kyon_urdf/meshes/collision/mesh_dagana-clamp-base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 scale=0.001 0.001 0.001; collision mesh filename=package://kyon_urdf/meshes/collision/mesh_dagana-clamp-simp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 scale=0.001 0.001 0.001
- link dagana_2_base: geometry collision mesh filename=package://kyon_urdf/meshes/collision/mesh_dagana-base-base-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 scale=0.001 0.001 0.001; collision mesh filename=package://kyon_urdf/meshes/collision/mesh_dagana-base-simpl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 scale=0.001 0.001 0.001
- link dagana_2_claw: geometry collision mesh filename=package://kyon_urdf/meshes/collision/mesh_dagana-clamp-base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 scale=0.001 0.001 0.001; collision mesh filename=package://kyon_urdf/meshes/collision/mesh_dagana-clamp-simp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 scale=0.001 0.001 0.001
- link pelvis: geometry collision mesh filename=package://kyon_urdf/meshes/collision/mesh_pelvis.stl scale=0.001 0.001 0.001; visual mesh filename=package://kyon_urdf/meshes/mesh_pelvis_no_lidar.stl scale=0.001 0.001 0.001
Joints:
- joint contact_1_joint: origin xyz=0.03 -0.35 0.03 rpy=-1.57 0 0.785 -> xyz=0.0 -0.3 0.054 rpy=-1.57 0 0.785
- joint contact_2_joint: origin xyz=-0.03 -0.35 0.03 rpy=1.57 0 2.356 -> xyz=-0.0 -0.3 0.054 rpy=1.57 0 2.356
- joint contact_3_joint: origin xyz=0.03 -0.35 0.03 rpy=-1.57 0 0.785 -> xyz=0.0 -0.3 0.054 rpy=-1.57 0 0.785
- joint contact_4_joint: origin xyz=-0.03 -0.35 0.03 rpy=1.57 0 2.356 -> xyz=-0.0 -0.3 0.054 rpy=1.57 0 2.356
- joint elbow_pitch_1: axis 0 0 1 -> 0 0 -1
- joint elbow_pitch_2: axis 0 0 1 -> 0 0 -1
- joint imu_joint: origin (none) -> xyz=-0.256190 0 0.103 rpy=3.14159265359 0 0
- joint shoulder_yaw_1: axis 0 0 1 -> 0 0 -1
- joint shoulder_yaw_2: axis 0 0 1 -> 0 0 -1
- joint wrist_pitch_1: axis 0 0 1 -> 0 0 -1
- joint wrist_pitch_2: axis 0 0 1 -> 0 0 -1
