Commit message: fix capsules

File: kyon_urdf/urdf/kyon_capsule.urdf (robot description, URDF)
Before this commit: robot kyon, 34 links, 33 joints
Joints:
- joint reference: origin (none) -> xyz=0.0 0.0 0.6 rpy=0 0 0

Commit message: fix ub signs in capsule urdf

File: kyon_urdf/urdf/kyon_capsule.urdf (robot description, URDF)
Before this commit: robot kyon, 34 links, 33 joints
Joints:
- joint elbow_pitch_1: axis 0.0 0.0 1.0 -> 0.0 0.0 -1.0
- joint elbow_pitch_2: axis 0.0 0.0 1.0 -> 0.0 0.0 -1.0
- joint shoulder_yaw_1: axis 0.0 0.0 1.0 -> 0.0 0.0 -1.0
- joint shoulder_yaw_2: axis 0.0 0.0 1.0 -> 0.0 0.0 -1.0
- joint wrist_pitch_1: axis 0.0 0.0 1.0 -> 0.0 0.0 -1.0
- joint wrist_pitch_2: axis 0.0 0.0 1.0 -> 0.0 0.0 -1.0

Commit message: wheel capsule

File: kyon_urdf/urdf/kyon_capsule.urdf (robot description, URDF)
Before this commit: robot kyon, 34 links, 33 joints
Joints:
- joint elbow_pitch_1: axis 0.0 0.0 1.0 -> 0.0 0.0 -1.0
- joint elbow_pitch_2: axis 0.0 0.0 1.0 -> 0.0 0.0 -1.0
- joint reference: origin (none) -> xyz=0.0 0.0 0.6 rpy=0 0 0
- joint shoulder_yaw_1: axis 0.0 0.0 1.0 -> 0.0 0.0 -1.0
- joint shoulder_yaw_2: axis 0.0 0.0 1.0 -> 0.0 0.0 -1.0
- joint wrist_pitch_1: axis 0.0 0.0 1.0 -> 0.0 0.0 -1.0
- joint wrist_pitch_2: axis 0.0 0.0 1.0 -> 0.0 0.0 -1.0
