Commit message: fixed capsule model

File: kyon_urdf/urdf/kyon_wheels_capsule.urdf (robot description, URDF)
Before this commit: robot kyon, 42 links, 41 joints
Links:
- link ankle_yaw_1_link: geometry collision cylinder length=0.24025318703748175 radius=0.058406; collision sphere radius=0.058406
- link ankle_yaw_2_link: geometry collision cylinder length=0.24025318703748175 radius=0.058406; collision sphere radius=0.058406
- link ankle_yaw_3_link: geometry collision cylinder length=0.24025318703748175 radius=0.058406; collision sphere radius=0.058406
- link ankle_yaw_4_link: geometry collision cylinder length=0.24025318703748175 radius=0.058406; collision sphere radius=0.058406
- link dagana_1_base: geometry collision cylinder length=0.05560094231679104 radius=0.0463682; collision mesh filename=package://kyon_urdf/meshes/collision/mesh_dagana-base-base-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 scale=0.001 0.001 0.001
- link dagana_1_claw: geometry collision cylinder length=0.06837212339526175 radius=0.0356173; collision mesh filename=package://kyon_urdf/meshes/collision/mesh_dagana-clamp-simp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 scale=0.001 0.001 0.001
- link dagana_2_base: geometry collision cylinder length=0.05560094231679104 radius=0.0463682; collision mesh filename=package://kyon_urdf/meshes/collision/mesh_dagana-base-base-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 scale=0.001 0.001 0.001
- link dagana_2_claw: geometry collision cylinder length=0.06837212339526175 radius=0.0356173; collision mesh filename=package://kyon_urdf/meshes/collision/mesh_dagana-clamp-simp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 scale=0.001 0.001 0.001
- link elbow_pitch_1_link: geometry collision cylinder length=0.23685382242345215 radius=0.0581584; collision sphere radius=0.0581584
- link elbow_pitch_2_link: geometry collision cylinder length=0.23685382242345215 radius=0.0581584; collision sphere radius=0.0581584
- link hip_pitch_1_link: geometry collision cylinder length=0.3004661110170414 radius=0.110589; collision sphere radius=0.110589
- link hip_pitch_2_link: geometry collision cylinder length=0.3004661110170414 radius=0.110589; collision sphere radius=0.110589
- link hip_pitch_3_link: geometry collision cylinder length=0.3004661110170414 radius=0.110589; collision sphere radius=0.110589
- link hip_pitch_4_link: geometry collision cylinder length=0.3004661110170414 radius=0.110589; collision sphere radius=0.110589
- link hip_roll_1_link: geometry collision cylinder length=0.14024696973705675 radius=0.0763481; collision sphere radius=0.0763481
- link hip_roll_2_link: geometry collision cylinder length=0.14024696973705536 radius=0.0763481; collision sphere radius=0.0763481
- link hip_roll_3_link: geometry collision cylinder length=0.14024696973705675 radius=0.0763481; collision sphere radius=0.0763481
- link hip_roll_4_link: geometry collision cylinder length=0.14024696973705536 radius=0.0763481; collision sphere radius=0.0763481
- link knee_pitch_1_link: geometry collision cylinder length=0.007315665155126021 radius=0.0660721; collision sphere radius=0.0660721
- link knee_pitch_2_link: geometry collision cylinder length=0.007315665155126021 radius=0.0660721; collision sphere radius=0.0660721
- link knee_pitch_3_link: geometry collision cylinder length=0.007315665155126021 radius=0.0660721; collision sphere radius=0.0660721
- link knee_pitch_4_link: geometry collision cylinder length=0.007315665155126021 radius=0.0660721; collision sphere radius=0.0660721
- link pelvis: geometry collision cylinder length=0.7715265904067888 radius=0.180153; collision sphere radius=0.180153
- link shoulder_pitch_1_link: geometry collision cylinder length=0.33021118992969195 radius=0.0630638; collision sphere radius=0.0630638
- link shoulder_pitch_2_link: geometry collision cylinder length=0.33021118992969195 radius=0.0630638; collision sphere radius=0.0630638
- link shoulder_yaw_1_link: geometry collision cylinder length=0.06680404009166925 radius=0.0700029; collision sphere radius=0.0700029
- link shoulder_yaw_2_link: geometry collision cylinder length=0.06680404009166925 radius=0.0700029; collision sphere radius=0.0700029
- link wheel_1: geometry collision cylinder length=0.019845524355384083 radius=0.109681; collision sphere radius=0.109681
- link wheel_2: geometry collision cylinder length=0.019845524355384083 radius=0.109681; collision sphere radius=0.109681
- link wheel_3: geometry collision cylinder length=0.019845524355384083 radius=0.109681; collision sphere radius=0.109681
- link wheel_4: geometry collision cylinder length=0.019845524355384083 radius=0.109681; collision sphere radius=0.109681
- link wrist_pitch_1_link: geometry collision cylinder length=0.07557658310998112 radius=0.0522867; collision sphere radius=0.0522867
- link wrist_pitch_2_link: geometry collision cylinder length=0.07557658310998112 radius=0.0522867; collision sphere radius=0.0522867
- link wrist_yaw_1_link: geometry collision cylinder length=0.00015248374464368804 radius=0.0436334; collision sphere radius=0.0436334
- link wrist_yaw_2_link: geometry collision cylinder length=0.00015248374464368804 radius=0.0436334; collision sphere radius=0.0436334
