Commit message: Signed-off-by: Andrea Patrizi <andreapatrizi1b6e6@gmail.com>

File: kyon_urdf/urdf/kyon_base.urdf.xacro (robot description, xacro)
@@ -9,4 +9,9 @@
 <xacro:include filename="${KYON_ROOT}/urdf/parts/limits.urdf.xacro" />
 <link name="base_link"/>
+<joint name="base_joint" type="fixed">
+    <parent link="base_link"/>
+    <child link="pelvis"/>
+    <origin xyz="0 0 0" rpy="0 0 0" />
+</joint>
 <link name="pelvis">
 	<inertial>
@@ -30,9 +35,4 @@
 	</collision>
 </link>
-<joint name="base_joint" type="fixed">
-    <parent link="pelvis"/>
-    <child link="base_link"/>
-    <origin xyz="0 0 0" rpy="0 0 0" />
-</joint>
 <xacro:if value="${ADD_SENSORS}">
     <xacro:include filename="${REALSENSE_GAZEBO_DESCRIPTION_ROOT}/urdf/_d435i.urdf.xacro" />

File: kyon_urdf/urdf/parts/kyon_leg.urdf.xacro (robot description, xacro)
@@ -142,5 +142,5 @@
                 <origin xyz="0.0 0.0 0.0" rpy="0.0 0.0 0.0" />
                 <geometry>
-                    <mesh filename="package://kyon_urdf/meshes/mesh_wheel23.stl"
+                    <mesh filename="${KYON_ROOT}/meshes/mesh_wheel23.stl"
                         scale="0.001 0.001 ${mirror*0.001}" />
                 </geometry>
@@ -150,5 +150,5 @@
                 <origin xyz="0 0 0" rpy="0 0 0" />
                 <geometry>
-                    <mesh filename="package://kyon_urdf/meshes/collision/mesh_wheel23.stl"
+                    <mesh filename="${KYON_ROOT}/meshes/collision/mesh_wheel23.stl"
                         scale="0.001 0.001 ${mirror*0.001}" />
                 </geometry>

Commit message: mujoco config files

File: kyon_urdf/urdf/kyon_base.urdf.xacro (robot description, xacro)
@@ -35,4 +35,9 @@
     <origin xyz="0 0 0" rpy="0 0 0" />
 </joint>
+<link name="imu_link"/>
+<joint name="imu_link" type="fixed">
+    <parent link="pelvis"/>
+    <child link="imu_link"/>
+</joint>
 <xacro:if value="${ADD_SENSORS}">
     <xacro:include filename="$(find realsense_gazebo_description)/urdf/_d435i.urdf.xacro" />
