Commit message: added upper body and pelvis mesh (no inertial information yet)

File: kyon_urdf/urdf/kyon_base.urdf.xacro (robot description, xacro)
@@ -18,6 +18,6 @@
 		<origin xyz="0.0 0 0.0"  rpy="0.0 0.0 0.0"/>
 		<geometry>
-	 		<box size="${pelvis_length} ${pelvis_width} ${pelvis_height}"/>
-	 		<!--mesh filename="package://kyon_urdf/meshes/mesh_pelvis.stl" scale="0.001 0.001 0.001"/-->
+	 		<!--box size="${pelvis_length} ${pelvis_width} ${pelvis_height}"/-->
+	 		<mesh filename="package://kyon_urdf/meshes/mesh_pelvis.stl" scale="0.001 0.001 0.001"/>
 		</geometry>
 	</visual>
@@ -25,6 +25,6 @@
 		<origin xyz="0.0 0 0.0"  rpy="0.0 0.0 0.0"/>
 		<geometry>
-	  		<box size="${pelvis_length} ${pelvis_width} ${pelvis_height}"/>
-	  		<!--mesh filename="package://kyon_urdf/meshes/mesh_pelvis.stl" scale="0.001 0.001 0.001"/-->
+	  		<!--box size="${pelvis_length} ${pelvis_width} ${pelvis_height}"/-->
+	  		<mesh filename="package://kyon_urdf/meshes/collision/mesh_pelvis.stl" scale="0.001 0.001 0.001"/>
 		</geometry>
 	</collision>

File: kyon_urdf/urdf/kyon_r0p10.urdf (robot description, URDF)
Before this commit: robot kyon, 42 links, 41 joints
Links:
- removed link elbow_pitch_1
- removed link elbow_pitch_2
- removed link shoulder_pitch_1
- removed link shoulder_pitch_2
- removed link shoulder_yaw_1
- removed link shoulder_yaw_2
- added link elbow_pitch_motor_1, mass 0.8; collision cylinder length=0.1 radius=0.07; visual cylinder length=0.1 radius=0.07
- added link elbow_pitch_motor_2, mass 0.8; collision cylinder length=0.1 radius=0.07; visual cylinder length=0.1 radius=0.07
- added link lower_arm_1, mass 1.0; collision box size=0.32 0.1 0.1; visual box size=0.32 0.1 0.1
- added link lower_arm_2, mass 1.0; collision box size=0.32 0.1 0.1; visual box size=0.32 0.1 0.1
- added link shoulder_pitch_motor_1, mass 0.8; collision cylinder length=0.1 radius=0.07; visual cylinder length=0.1 radius=0.07
- added link shoulder_pitch_motor_2, mass 0.8; collision cylinder length=0.1 radius=0.07; visual cylinder length=0.1 radius=0.07
- added link shoulder_yaw_motor_1, mass 1.6; collision cylinder length=0.1 radius=0.07; visual cylinder length=0.1 radius=0.07
- added link shoulder_yaw_motor_2, mass 1.6; collision cylinder length=0.1 radius=0.07; visual cylinder length=0.1 radius=0.07
- added link upper_arm1_1, mass 0.77; collision box size=0.3 0.05 0.05; visual box size=0.3 0.05 0.05
- added link upper_arm1_2, mass 0.77; collision box size=0.3 0.05 0.05; visual box size=0.3 0.05 0.05
- link pelvis: geometry collision box size=0.8 0.45 0.2; visual box size=0.8 0.45 0.2
Joints:
- added joint elbow_pitch_stator_1: type fixed, parent lower_arm_1, child elbow_pitch_motor_1, origin xyz=0.32 0.0 0.0 rpy=0.0 0.0 0.0
- added joint elbow_pitch_stator_2: type fixed, parent lower_arm_2, child elbow_pitch_motor_2, origin xyz=0.32 0.0 0.0 rpy=0.0 0.0 0.0
- added joint shoulder_pitch_stator_1: type fixed, parent shoulder_yaw_motor_1, child shoulder_pitch_motor_1, origin xyz=0.0 0.0 0.05 rpy=-1.57079632679 0.0 0.0
- added joint shoulder_pitch_stator_2: type fixed, parent shoulder_yaw_motor_2, child shoulder_pitch_motor_2, origin xyz=0.0 0.0 0.05 rpy=-1.57079632679 0.0 0.0
- joint elbow_pitch_1: child elbow_pitch_1 -> upper_arm1_1; origin xyz=0.0 0.0 0.32 rpy=-1.57079632679 0.0 0.0 -> xyz=0.0 0.0 0.0 rpy=0.0 0.0 0.0; parent shoulder_pitch_1 -> elbow_pitch_motor_1
- joint elbow_pitch_2: child elbow_pitch_2 -> upper_arm1_2; origin xyz=0.0 0.0 0.32 rpy=-1.57079632679 0.0 0.0 -> xyz=0.0 0.0 0.0 rpy=0.0 0.0 0.0; parent shoulder_pitch_2 -> elbow_pitch_motor_2
- joint hip_pitch_stator_1: origin xyz=0.0 0.12000000000000001 0.0 rpy=-1.57079632679 0.0 0.0 -> xyz=0.0 0.07 0.0 rpy=-1.57079632679 0.0 0.0
- joint hip_pitch_stator_2: origin xyz=0.0 -0.12000000000000001 0.0 rpy=-1.57079632679 0.0 0.0 -> xyz=0.0 -0.07 0.0 rpy=-1.57079632679 0.0 0.0
- joint hip_pitch_stator_3: origin xyz=0.0 0.12000000000000001 0.0 rpy=-1.57079632679 0.0 0.0 -> xyz=0.0 0.07 0.0 rpy=-1.57079632679 0.0 0.0
- joint hip_pitch_stator_4: origin xyz=0.0 -0.12000000000000001 0.0 rpy=-1.57079632679 0.0 0.0 -> xyz=0.0 -0.07 0.0 rpy=-1.57079632679 0.0 0.0
- joint hip_roll_1: origin xyz=0.41 0.0775 0.0 rpy=0.0 1.57079632679 0.0 -> xyz=0.4 0.225 0.0 rpy=0.0 1.57079632679 0.0
- joint hip_roll_2: origin xyz=0.41 -0.0775 0.0 rpy=0.0 1.57079632679 0.0 -> xyz=0.4 -0.225 0.0 rpy=0.0 1.57079632679 0.0
- joint hip_roll_3: origin xyz=-0.41 0.0775 0.0 rpy=0.0 1.57079632679 0.0 -> xyz=-0.4 0.225 0.0 rpy=0.0 1.57079632679 0.0
- joint hip_roll_4: origin xyz=-0.41 -0.0775 0.0 rpy=0.0 1.57079632679 0.0 -> xyz=-0.4 -0.225 0.0 rpy=0.0 1.57079632679 0.0
- joint shoulder_pitch_1: axis 0 1 0 -> 0 0 1; child shoulder_pitch_1 -> lower_arm_1; origin xyz=0.0 0.0 0.0735 rpy=0.0 0.0 3.14159265358 -> xyz=0.0 0.0 0.0 rpy=0.0 0.0 -1.57079632679; parent shoulder_yaw_1 -> shoulder_pitch_motor_1
- joint shoulder_pitch_2: axis 0 1 0 -> 0 0 1; child shoulder_pitch_2 -> lower_arm_2; origin xyz=0.0 0.0 0.0735 rpy=0.0 0.0 0.0 -> xyz=0.0 0.0 0.0 rpy=0.0 0.0 -1.57079632679; parent shoulder_yaw_2 -> shoulder_pitch_motor_2
- joint shoulder_yaw_1: child shoulder_yaw_1 -> shoulder_yaw_motor_1; origin xyz=0.27 0.10299599999999999 0.18721700000000002 rpy=-0.3490656 0.0 0.0 -> xyz=0.30000000000000004 0.175 0.1 rpy=-0.0 0.2 0.0
- joint shoulder_yaw_2: child shoulder_yaw_2 -> shoulder_yaw_motor_2; origin xyz=0.27 -0.10299599999999999 0.18721700000000002 rpy=0.3490656 0.0 0.0 -> xyz=0.30000000000000004 -0.175 0.1 rpy=0.0 0.2 0.0
- joint wrist_pitch_stator_1: origin xyz=0.0 -0.25 0.0 rpy=0.0 0.0 -1.57079632679 -> xyz=0.3 0.0 0.0 rpy=0.0 0.0 0.0; parent elbow_pitch_1 -> upper_arm1_1
- joint wrist_pitch_stator_2: origin xyz=0.0 -0.25 0.0 rpy=0.0 0.0 -1.57079632679 -> xyz=0.3 0.0 0.0 rpy=0.0 0.0 0.0; parent elbow_pitch_2 -> upper_arm1_2

File: kyon_urdf/urdf/kyon_r0p30.urdf (robot description, URDF)
Before this commit: robot kyon, 42 links, 41 joints
Links:
- removed link elbow_pitch_1
- removed link elbow_pitch_2
- removed link shoulder_pitch_1
- removed link shoulder_pitch_2
- removed link shoulder_yaw_1
- removed link shoulder_yaw_2
- added link elbow_pitch_motor_1, mass 0.8; collision cylinder length=0.1 radius=0.07; visual cylinder length=0.1 radius=0.07
- added link elbow_pitch_motor_2, mass 0.8; collision cylinder length=0.1 radius=0.07; visual cylinder length=0.1 radius=0.07
- added link lower_arm_1, mass 1.0; collision box size=0.32 0.1 0.1; visual box size=0.32 0.1 0.1
- added link lower_arm_2, mass 1.0; collision box size=0.32 0.1 0.1; visual box size=0.32 0.1 0.1
- added link shoulder_pitch_motor_1, mass 0.8; collision cylinder length=0.1 radius=0.07; visual cylinder length=0.1 radius=0.07
- added link shoulder_pitch_motor_2, mass 0.8; collision cylinder length=0.1 radius=0.07; visual cylinder length=0.1 radius=0.07
- added link shoulder_yaw_motor_1, mass 1.6; collision cylinder length=0.1 radius=0.07; visual cylinder length=0.1 radius=0.07
- added link shoulder_yaw_motor_2, mass 1.6; collision cylinder length=0.1 radius=0.07; visual cylinder length=0.1 radius=0.07
- added link upper_arm1_1, mass 0.77; collision box size=0.3 0.05 0.05; visual box size=0.3 0.05 0.05
- added link upper_arm1_2, mass 0.77; collision box size=0.3 0.05 0.05; visual box size=0.3 0.05 0.05
- link pelvis: geometry collision box size=0.8 0.45 0.2; visual box size=0.8 0.45 0.2
Joints:
- added joint elbow_pitch_stator_1: type fixed, parent lower_arm_1, child elbow_pitch_motor_1, origin xyz=0.32 0.0 0.0 rpy=0.0 0.0 0.0
- added joint elbow_pitch_stator_2: type fixed, parent lower_arm_2, child elbow_pitch_motor_2, origin xyz=0.32 0.0 0.0 rpy=0.0 0.0 0.0
- added joint shoulder_pitch_stator_1: type fixed, parent shoulder_yaw_motor_1, child shoulder_pitch_motor_1, origin xyz=0.0 0.0 0.05 rpy=-1.57079632679 0.0 0.0
- added joint shoulder_pitch_stator_2: type fixed, parent shoulder_yaw_motor_2, child shoulder_pitch_motor_2, origin xyz=0.0 0.0 0.05 rpy=-1.57079632679 0.0 0.0
- joint elbow_pitch_1: child elbow_pitch_1 -> upper_arm1_1; origin xyz=0.0 0.0 0.32 rpy=-1.57079632679 0.0 0.0 -> xyz=0.0 0.0 0.0 rpy=0.0 0.0 0.0; parent shoulder_pitch_1 -> elbow_pitch_motor_1
- joint elbow_pitch_2: child elbow_pitch_2 -> upper_arm1_2; origin xyz=0.0 0.0 0.32 rpy=-1.57079632679 0.0 0.0 -> xyz=0.0 0.0 0.0 rpy=0.0 0.0 0.0; parent shoulder_pitch_2 -> elbow_pitch_motor_2
- joint hip_pitch_stator_1: origin xyz=0.0 0.12000000000000001 0.0 rpy=-1.57079632679 0.0 0.0 -> xyz=0.0 0.07 0.0 rpy=-1.57079632679 0.0 0.0
- joint hip_pitch_stator_2: origin xyz=0.0 -0.12000000000000001 0.0 rpy=-1.57079632679 0.0 0.0 -> xyz=0.0 -0.07 0.0 rpy=-1.57079632679 0.0 0.0
- joint hip_pitch_stator_3: origin xyz=0.0 0.12000000000000001 0.0 rpy=-1.57079632679 0.0 0.0 -> xyz=0.0 0.07 0.0 rpy=-1.57079632679 0.0 0.0
- joint hip_pitch_stator_4: origin xyz=0.0 -0.12000000000000001 0.0 rpy=-1.57079632679 0.0 0.0 -> xyz=0.0 -0.07 0.0 rpy=-1.57079632679 0.0 0.0
- joint hip_roll_1: origin xyz=0.41 0.0775 0.0 rpy=0.0 1.57079632679 0.0 -> xyz=0.4 0.225 0.0 rpy=0.0 1.57079632679 0.0
- joint hip_roll_2: origin xyz=0.41 -0.0775 0.0 rpy=0.0 1.57079632679 0.0 -> xyz=0.4 -0.225 0.0 rpy=0.0 1.57079632679 0.0
- joint hip_roll_3: origin xyz=-0.41 0.0775 0.0 rpy=0.0 1.57079632679 0.0 -> xyz=-0.4 0.225 0.0 rpy=0.0 1.57079632679 0.0
- joint hip_roll_4: origin xyz=-0.41 -0.0775 0.0 rpy=0.0 1.57079632679 0.0 -> xyz=-0.4 -0.225 0.0 rpy=0.0 1.57079632679 0.0
- joint shoulder_pitch_1: axis 0 1 0 -> 0 0 1; child shoulder_pitch_1 -> lower_arm_1; origin xyz=0.0 0.0 0.0735 rpy=0.0 0.0 3.14159265358 -> xyz=0.0 0.0 0.0 rpy=0.0 0.0 -1.57079632679; parent shoulder_yaw_1 -> shoulder_pitch_motor_1
- joint shoulder_pitch_2: axis 0 1 0 -> 0 0 1; child shoulder_pitch_2 -> lower_arm_2; origin xyz=0.0 0.0 0.0735 rpy=0.0 0.0 0.0 -> xyz=0.0 0.0 0.0 rpy=0.0 0.0 -1.57079632679; parent shoulder_yaw_2 -> shoulder_pitch_motor_2
- joint shoulder_yaw_1: child shoulder_yaw_1 -> shoulder_yaw_motor_1; origin xyz=0.27 0.10299599999999999 0.18721700000000002 rpy=-0.3490656 0.0 0.0 -> xyz=0.30000000000000004 0.175 0.1 rpy=-0.0 0.6 0.0
- joint shoulder_yaw_2: child shoulder_yaw_2 -> shoulder_yaw_motor_2; origin xyz=0.27 -0.10299599999999999 0.18721700000000002 rpy=0.3490656 0.0 0.0 -> xyz=0.30000000000000004 -0.175 0.1 rpy=0.0 0.6 0.0
- joint wrist_pitch_stator_1: origin xyz=0.0 -0.25 0.0 rpy=0.0 0.0 -1.57079632679 -> xyz=0.3 0.0 0.0 rpy=0.0 0.0 0.0; parent elbow_pitch_1 -> upper_arm1_1
- joint wrist_pitch_stator_2: origin xyz=0.0 -0.25 0.0 rpy=0.0 0.0 -1.57079632679 -> xyz=0.3 0.0 0.0 rpy=0.0 0.0 0.0; parent elbow_pitch_2 -> upper_arm1_2

File: kyon_urdf/urdf/kyon_r20p00.urdf (robot description, URDF)
Before this commit: robot kyon, 42 links, 41 joints
Links:
- removed link ball_arm_1
- removed link ball_arm_2
- added link dagana_1_bottom_link, mass 4.6117745e-01; collision mesh filename=package://dagana_urdf/meshes/dg0002-ch.stl scale=0.001 0.001 0.001; visual mesh filename=package://dagana_urdf/meshes/dg0002.stl scale=0.001 0.001 0.001
- added link dagana_1_tcp
- added link dagana_1_top_link, mass 1.7432400; collision mesh filename=package://dagana_urdf/meshes/dg0001-ch.stl scale=0.001 0.001 0.001; visual mesh filename=package://dagana_urdf/meshes/dg0001-simplified.stl scale=0.001 0.001 0.001
- added link dagana_2_bottom_link, mass 4.6117745e-01; collision mesh filename=package://dagana_urdf/meshes/dg0002-ch.stl scale=0.001 0.001 0.001; visual mesh filename=package://dagana_urdf/meshes/dg0002.stl scale=0.001 0.001 0.001
- added link dagana_2_tcp
- added link dagana_2_top_link, mass 1.7432400; collision mesh filename=package://dagana_urdf/meshes/dg0001-ch.stl scale=0.001 0.001 0.001; visual mesh filename=package://dagana_urdf/meshes/dg0001-simplified.stl scale=0.001 0.001 0.001
Joints:
- removed joint hand_joint_1
- removed joint hand_joint_2
- added joint dagana_1_claw_joint: type fixed, parent dagana_1_top_link, child dagana_1_bottom_link, origin xyz=0.0 -0.028 0.05025 rpy=1.57079632679 0 3.14159265359, axis -1 0 0, limit lower=0 upper=1 effort=1000 velocity=2.0
- added joint dagana_1_mount_joint: type fixed, parent wrist_1, child dagana_1_top_link, origin xyz=0 0 0 rpy=0 0 0
- added joint dagana_1_tcp_joint: type fixed, parent dagana_1_top_link, child dagana_1_tcp, origin xyz=0 -0.05 0.15 rpy=0 0 0
- added joint dagana_2_claw_joint: type fixed, parent dagana_2_top_link, child dagana_2_bottom_link, origin xyz=0.0 -0.028 0.05025 rpy=1.57079632679 0 3.14159265359, axis -1 0 0, limit lower=0 upper=1 effort=1000 velocity=2.0
- added joint dagana_2_mount_joint: type fixed, parent wrist_2, child dagana_2_top_link, origin xyz=0 0 0 rpy=0 0 0
- added joint dagana_2_tcp_joint: type fixed, parent dagana_2_top_link, child dagana_2_tcp, origin xyz=0 -0.05 0.15 rpy=0 0 0

File: kyon_urdf/urdf/kyon_r20p10.urdf (robot description, URDF)
Before this commit: robot kyon, 42 links, 41 joints
Links:
- removed link ball_arm_1
- removed link ball_arm_2
- added link dagana_1_bottom_link, mass 4.6117745e-01; collision mesh filename=package://dagana_urdf/meshes/dg0002-ch.stl scale=0.001 0.001 0.001; visual mesh filename=package://dagana_urdf/meshes/dg0002.stl scale=0.001 0.001 0.001
- added link dagana_1_tcp
- added link dagana_1_top_link, mass 1.7432400; collision mesh filename=package://dagana_urdf/meshes/dg0001-ch.stl scale=0.001 0.001 0.001; visual mesh filename=package://dagana_urdf/meshes/dg0001-simplified.stl scale=0.001 0.001 0.001
- added link dagana_2_bottom_link, mass 4.6117745e-01; collision mesh filename=package://dagana_urdf/meshes/dg0002-ch.stl scale=0.001 0.001 0.001; visual mesh filename=package://dagana_urdf/meshes/dg0002.stl scale=0.001 0.001 0.001
- added link dagana_2_tcp
- added link dagana_2_top_link, mass 1.7432400; collision mesh filename=package://dagana_urdf/meshes/dg0001-ch.stl scale=0.001 0.001 0.001; visual mesh filename=package://dagana_urdf/meshes/dg0001-simplified.stl scale=0.001 0.001 0.001
Joints:
- removed joint hand_joint_1
- removed joint hand_joint_2
- added joint dagana_1_claw_joint: type fixed, parent dagana_1_top_link, child dagana_1_bottom_link, origin xyz=0.0 -0.028 0.05025 rpy=1.57079632679 0 3.14159265359, axis -1 0 0, limit lower=0 upper=1 effort=1000 velocity=2.0
- added joint dagana_1_mount_joint: type fixed, parent wrist_1, child dagana_1_top_link, origin xyz=0 0 0 rpy=0 0 0
- added joint dagana_1_tcp_joint: type fixed, parent dagana_1_top_link, child dagana_1_tcp, origin xyz=0 -0.05 0.15 rpy=0 0 0
- added joint dagana_2_claw_joint: type fixed, parent dagana_2_top_link, child dagana_2_bottom_link, origin xyz=0.0 -0.028 0.05025 rpy=1.57079632679 0 3.14159265359, axis -1 0 0, limit lower=0 upper=1 effort=1000 velocity=2.0
- added joint dagana_2_mount_joint: type fixed, parent wrist_2, child dagana_2_top_link, origin xyz=0 0 0 rpy=0 0 0
- added joint dagana_2_tcp_joint: type fixed, parent dagana_2_top_link, child dagana_2_tcp, origin xyz=0 -0.05 0.15 rpy=0 0 0
- joint shoulder_yaw_1: origin xyz=0.27 0.10299599999999999 0.18721700000000002 rpy=-0.3490656 0.0 0.0 -> xyz=0.32 0.10299599999999999 0.18721700000000002 rpy=-0.3490656 0.0 0.0
- joint shoulder_yaw_2: origin xyz=0.27 -0.10299599999999999 0.18721700000000002 rpy=0.3490656 0.0 0.0 -> xyz=0.32 -0.10299599999999999 0.18721700000000002 rpy=0.3490656 0.0 0.0

File: kyon_urdf/urdf/kyon_r20p20.urdf (robot description, URDF)
Before this commit: robot kyon, 42 links, 41 joints
Links:
- removed link ball_arm_1
- removed link ball_arm_2
- added link dagana_1_bottom_link, mass 4.6117745e-01; collision mesh filename=package://dagana_urdf/meshes/dg0002-ch.stl scale=0.001 0.001 0.001; visual mesh filename=package://dagana_urdf/meshes/dg0002.stl scale=0.001 0.001 0.001
- added link dagana_1_tcp
- added link dagana_1_top_link, mass 1.7432400; collision mesh filename=package://dagana_urdf/meshes/dg0001-ch.stl scale=0.001 0.001 0.001; visual mesh filename=package://dagana_urdf/meshes/dg0001-simplified.stl scale=0.001 0.001 0.001
- added link dagana_2_bottom_link, mass 4.6117745e-01; collision mesh filename=package://dagana_urdf/meshes/dg0002-ch.stl scale=0.001 0.001 0.001; visual mesh filename=package://dagana_urdf/meshes/dg0002.stl scale=0.001 0.001 0.001
- added link dagana_2_tcp
- added link dagana_2_top_link, mass 1.7432400; collision mesh filename=package://dagana_urdf/meshes/dg0001-ch.stl scale=0.001 0.001 0.001; visual mesh filename=package://dagana_urdf/meshes/dg0001-simplified.stl scale=0.001 0.001 0.001
Joints:
- removed joint hand_joint_1
- removed joint hand_joint_2
- added joint dagana_1_claw_joint: type fixed, parent dagana_1_top_link, child dagana_1_bottom_link, origin xyz=0.0 -0.028 0.05025 rpy=1.57079632679 0 3.14159265359, axis -1 0 0, limit lower=0 upper=1 effort=1000 velocity=2.0
- added joint dagana_1_mount_joint: type fixed, parent wrist_1, child dagana_1_top_link, origin xyz=0 0 0 rpy=0 0 0
- added joint dagana_1_tcp_joint: type fixed, parent dagana_1_top_link, child dagana_1_tcp, origin xyz=0 -0.05 0.15 rpy=0 0 0
- added joint dagana_2_claw_joint: type fixed, parent dagana_2_top_link, child dagana_2_bottom_link, origin xyz=0.0 -0.028 0.05025 rpy=1.57079632679 0 3.14159265359, axis -1 0 0, limit lower=0 upper=1 effort=1000 velocity=2.0
- added joint dagana_2_mount_joint: type fixed, parent wrist_2, child dagana_2_top_link, origin xyz=0 0 0 rpy=0 0 0
- added joint dagana_2_tcp_joint: type fixed, parent dagana_2_top_link, child dagana_2_tcp, origin xyz=0 -0.05 0.15 rpy=0 0 0
- joint shoulder_yaw_1: origin xyz=0.27 0.10299599999999999 0.18721700000000002 rpy=-0.3490656 0.0 0.0 -> xyz=0.27 0.10299599999999999 0.18721700000000002 rpy=-0.3490656 0.4 0.0
- joint shoulder_yaw_2: origin xyz=0.27 -0.10299599999999999 0.18721700000000002 rpy=0.3490656 0.0 0.0 -> xyz=0.27 -0.10299599999999999 0.18721700000000002 rpy=0.3490656 0.4 0.0

File: kyon_urdf/urdf/parts/kinematics_properties.urdf.xacro (robot description, xacro)
@@ -1,4 +1,5 @@
 <?xml version="1.0"?>
 <robot  xmlns:xacro="http://ros.org/wiki/xacro">
+    <xacro:property name="mTomm" value="0.001"/>
     <xacro:property name="kin_yaml_file" value="$(find kyon_urdf)/urdf/config/kinematics_properties.yaml" />
     <xacro:property name="kin_props" value="${xacro.load_yaml(kin_yaml_file)}"/>
@@ -34,5 +35,5 @@
     <!-- Origin -->
     <xacro:property name="HipPitch_Ox" value="0.0"/>
-    <xacro:property name="HipPitch_Oy" value="${-cylinder_radius}"/>
+    <xacro:property name="HipPitch_Oy" value="${-cylinder_radius - cylinder_length / 2}"/>
     <xacro:property name="HipPitch_Oz" value="0.0"/>
     <xacro:property name="HipPitch_roll" value="${-PI_2}"/>
@@ -66,29 +67,20 @@
     <xacro:property name="Ankle_yaw" value="0.0"/>
     <!-- Arms -->
-    <xacro:property name="ShoulderYaw_Ox" value="${pelvis_length / 2}"/>
-    <xacro:property name="ShoulderYaw_Oy" value="${pelvis_width / 2}"/>
-    <xacro:property name="ShoulderYaw_Oz" value="${pelvis_height / 2}"/>
-    <xacro:property name="ShoulderYaw_roll" value="0.0"/>
+    <xacro:property name="ShoulderYaw_Ox" value="${320.00 * mTomm}"/>
+    <xacro:property name="ShoulderYaw_Oy" value="${102.996 * mTomm}"/>
+    <xacro:property name="ShoulderYaw_Oz" value="${187.217 * mTomm}"/>
+    <xacro:property name="ShoulderYaw_roll" value="0.3490656"/>
     <xacro:property name="ShoulderYaw_pitch" value="0.0"/>
     <xacro:property name="ShoulderYaw_yaw" value="0.0"/>
-    <xacro:property name="ShoulderYaw_OffsetX" value="0.1"/>
-    <xacro:property name="ShoulderYaw_OffsetY" value="0.05"/>
-    <xacro:property name="ShoulderYaw_OffsetZ" value="0.0"/>
     <xacro:property name="ShoulderPitch_Ox" value="0.0"/>
     <xacro:property name="ShoulderPitch_Oy" value="0.0"/>
-    <xacro:property name="ShoulderPitch_Oz" value="${cylinder_length / 2}"/>
-    <xacro:property name="ShoulderPitch_roll" value="${-PI_2}"/>
+    <xacro:property name="ShoulderPitch_Oz" value="${73.5 * mTomm}"/>
+    <xacro:property name="ShoulderPitch_roll" value="0.0"/>
     <xacro:property name="ShoulderPitch_pitch" value="0.0"/>
-    <xacro:property name="ShoulderPitch_yaw" value="0.0"/>
-    <xacro:property name="LowerArm_Ox" value="0.0"/>
-    <xacro:property name="LowerArm_Oy" value="0.0"/>
-    <xacro:property name="LowerArm_Oz" value="0.0"/>
-    <xacro:property name="LowerArm_roll" value="0.0"/>
-    <xacro:property name="LowerArm_pitch" value="0.0"/>
-    <xacro:property name="LowerArm_yaw" value="${-PI_2}"/>
-    <xacro:property name="ElbowPitch_Ox" value="${lower_arm_length}"/>
+    <xacro:property name="ShoulderPitch_yaw" value="${PI_2}"/>>
+    <xacro:property name="ElbowPitch_Ox" value="0.0"/>
     <xacro:property name="ElbowPitch_Oy" value="0.0"/>
-    <xacro:property name="ElbowPitch_Oz" value="0.0"/>
-    <xacro:property name="ElbowPitch_roll" value="0.0"/>
+    <xacro:property name="ElbowPitch_Oz" value="${320.00 * mTomm}"/>
+    <xacro:property name="ElbowPitch_roll" value="${-PI_2}"/>
     <xacro:property name="ElbowPitch_pitch" value="0.0"/>
     <xacro:property name="ElbowPitch_yaw" value="0.0"/>
@@ -99,10 +91,10 @@
     <xacro:property name="UpperArm1_pitch" value="0.0"/>
     <xacro:property name="UpperArm1_yaw" value="0.0"/>
-    <xacro:property name="WristPitch_Ox" value="${upper_arm1_length}"/>
-	<xacro:property name="WristPitch_Oy" value="0.0"/>
+    <xacro:property name="WristPitch_Ox" value="0.0"/>
+	<xacro:property name="WristPitch_Oy" value="${-250.00 * mTomm}"/>
 	<xacro:property name="WristPitch_Oz" value="0.0"/>
 	<xacro:property name="WristPitch_roll" value="0.0"/>
 	<xacro:property name="WristPitch_pitch" value="0.0"/>
-	<xacro:property name="WristPitch_yaw" value="0.0"/>
+	<xacro:property name="WristPitch_yaw" value="${-PI_2}"/>
 	<xacro:property name="UpperArm2_Ox" value="0.0"/>
     <xacro:property name="UpperArm2_Oy" value="0.0"/>
