Commit message: added upper body and pelvis mesh (no inertial information yet)

File: kyon_urdf/urdf/parts/kyon_arm.urdf.xacro (robot description, xacro)
@@ -5,5 +5,5 @@
 <!-- LINKS -->
 <!-- shoulder yaw -->
-<link name="shoulder_yaw_motor_${arm_num}">
+<link name="shoulder_yaw_${arm_num}">
 	<inertial>
 		<origin xyz="0.0 0.0 0.0"/>
@@ -14,5 +14,6 @@
 		<origin xyz="0.0 0.0 0.0"  rpy="0.0 0.0 0.0"/>
 		<geometry>
-			<cylinder radius="${cylinder_radius}" length="${cylinder_length}"/>
+			<!--cylinder radius="${cylinder_radius}" length="${cylinder_length}"/-->
+			<mesh filename="package://kyon_urdf/meshes/mesh_sh-yaw.stl" scale="0.001 0.001 0.001"/>
 		</geometry>
 		<material name="dark_grey"/>
@@ -21,68 +22,32 @@
 		<origin xyz="0.0 0.0 0.0"  rpy="0.0 0.0 0.0"/>
 		<geometry>
-			<cylinder radius="${cylinder_radius}" length="${cylinder_length}"/>
+			<!--cylinder radius="${cylinder_radius}" length="${cylinder_length}"/-->
+			<mesh filename="package://kyon_urdf/meshes/collision/mesh_sh-yaw.stl" scale="0.001 0.001 0.001"/>
 		</geometry>
 	</collision>
 </link>
-<link name="shoulder_pitch_motor_${arm_num}">
+<link name="shoulder_pitch_${arm_num}">
 	<inertial>
 		<origin xyz="0.0 0.0 0.0"/>
-		<mass value="${motor_arm2_mass}"/>
-		<inertia ixx="${MotorArm2_xx}" ixy="${MotorArm2_xy}" ixz="${MotorArm2_xz}" iyy="${MotorArm2_yy}" iyz="${MotorArm2_yz}" izz="${MotorArm2_zz}"/>
+		<mass value="${lower_arm_mass + motor_arm2_mass}"/>
+		<inertia ixx="${LowerArm_xx}" ixy="${LowerArm_xy}" ixz="${LowerArm_xz}" iyy="${LowerArm_yy}" iyz="${LowerArm_yz}" izz="${LowerArm_zz}"/>
 	</inertial>
 	<visual>
-		<origin xyz="0.0 0.0 0.0"  rpy="0.0 0.0 0.0"/>
+		<!--origin xyz="${lower_arm_length / 2} 0.0 0.0"  rpy="0.0 0.0 0.0"/-->
 	  	<geometry>
-	 		<cylinder radius="${cylinder_radius}" length="${cylinder_length}"/>
+			<!--box size="${lower_arm_length} ${lower_arm_width} ${lower_arm_height}"/-->
+	 		<mesh filename="package://kyon_urdf/meshes/mesh_sh-pitch.stl" scale="0.001 0.001 0.001"/>
 	  	</geometry>
   		<material name="dark_grey"/>
 	</visual>
 	<collision>
-		<origin xyz="0.0 0.0 0.0"  rpy="0.0 0.0 0.0"/>
-		<geometry>
-			<cylinder radius="${cylinder_radius}" length="${cylinder_length}"/>
+		<!--origin xyz="${lower_arm_length / 2} 0.0 0.0"  rpy="0.0 0.0 0.0"/-->
+	  	<geometry>
+			<!--box size="${lower_arm_length} ${lower_arm_width} ${lower_arm_height}"/-->
+			<mesh filename="package://kyon_urdf/meshes/collision/mesh_sh-pitch.stl" scale="0.001 0.001 0.001"/>
 		</geometry>
 	</collision>
 </link>
-<link name="lower_arm_${arm_num}">
-	<inertial>
-		<origin xyz="${lower_arm_length / 2} 0.0 0.0"/>
-		<mass value="${lower_arm_mass}"/>
-		<inertia ixx="${LowerArm_xx}" ixy="${LowerArm_xy}" ixz="${LowerArm_xz}" iyy="${LowerArm_yy}" iyz="${LowerArm_yz}" izz="${LowerArm_zz}"/>
-	</inertial>
-	<visual>
-		<origin xyz="${lower_arm_length / 2} 0.0 0.0"  rpy="0.0 0.0 0.0"/>
-		<geometry>
-			<box size="${lower_arm_length} ${lower_arm_width} ${lower_arm_height}"/>
-		</geometry>
-	</visual>
-	<collision>
-		<origin xyz="${lower_arm_length / 2} 0.0 0.0"  rpy="0.0 0.0 0.0"/>
-		<geometry>
-			<box size="${lower_arm_length} ${lower_arm_width} ${lower_arm_height}"/>
-		</geometry>
-	</collision>
-</link>
-<link name="elbow_pitch_motor_${arm_num}">
-	<inertial>
-		<origin xyz="0.0 0.0 0.0"/>
-		<mass value="${motor_arm2_mass}"/>
-		<inertia ixx="${MotorArm2_xx}" ixy="${MotorArm2_xy}" ixz="${MotorArm2_xz}" iyy="${MotorArm2_yy}" iyz="${MotorArm2_yz}" izz="${MotorArm2_zz}"/>
-	</inertial>
-	<visual>
-		<origin xyz="0.0 0.0 0.0"  rpy="0.0 0.0 0.0"/>
-	  	<geometry>
-	 		<cylinder radius="${cylinder_radius}" length="${cylinder_length}"/>
-	  	</geometry>
-  		<material name="dark_grey"/>
-	</visual>
-	<collision>
-		<origin xyz="0.0 0.0 0.0"  rpy="0.0 0.0 0.0"/>
-		<geometry>
-			<cylinder radius="${cylinder_radius}" length="${cylinder_length}"/>
-		</geometry>
-	</collision>
-</link>
-<link name="upper_arm1_${arm_num}">
+<link name="elbow_pitch_${arm_num}">
 	<inertial>
 		<origin xyz="${upper_arm1_length / 2} 0.0 0.0"/>
@@ -91,13 +56,15 @@
 	</inertial>
 	<visual>
-		<origin xyz="${upper_arm1_length / 2} 0.0 0.0"  rpy="0.0 0.0 0.0"/>
+		<!--origin xyz="${upper_arm1_length / 2} 0.0 0.0"  rpy="0.0 0.0 0.0"/-->
 		<geometry>
-			<box size="${upper_arm1_length} ${upper_arm1_width} ${upper_arm1_height}"/>
+			<!--box size="${upper_arm1_length} ${upper_arm1_width} ${upper_arm1_height}"/-->
+			<mesh filename="package://kyon_urdf/meshes/mesh_elbow.stl" scale="0.001 0.001 0.001"/>
 		</geometry>
 	</visual>
 	<collision>
-		<origin xyz="${lower_arm_length / 2} 0.0 0.0"  rpy="0.0 0.0 0.0"/>
+		<!--origin xyz="${lower_arm_length / 2} 0.0 0.0"  rpy="0.0 0.0 0.0"/-->
 		<geometry>
-			<box size="${upper_arm1_length} ${upper_arm1_width} ${upper_arm1_height}"/>
+			<!--box size="${upper_arm1_length} ${upper_arm1_width} ${upper_arm1_height}"/-->
+			<mesh filename="package://kyon_urdf/meshes/mesh_elbow.stl" scale="0.001 0.001 0.001"/>
 		</geometry>
 	</collision>
@@ -168,37 +135,26 @@
 <joint name="shoulder_yaw_${arm_num}" type="revolute">
 	<parent link="${parent}"/>
-	<child link="shoulder_yaw_motor_${arm_num}"/>
-	<origin xyz="${ShoulderYaw_Ox - ShoulderYaw_OffsetX} ${rot * ShoulderYaw_Oy - rot * ShoulderYaw_OffsetY} ${ShoulderYaw_Oz - ShoulderYaw_OffsetZ}" rpy="${-rot * ShoulderYaw_roll} ${ShoulderYaw_pitch} ${ShoulderYaw_yaw}"/>
+	<child link="shoulder_yaw_${arm_num}"/>
+	<origin xyz="${ShoulderYaw_Ox} ${rot * ShoulderYaw_Oy} ${ShoulderYaw_Oz}" rpy="${-rot * ShoulderYaw_roll} ${ShoulderYaw_pitch} ${ShoulderYaw_yaw}"/>
 	<axis xyz="0 0 1"/>
 	<limit lower="${j_shoulder_yaw_lower[arm_num-1]}" upper="${j_shoulder_yaw_upper[arm_num-1]}" effort="${motor_effort}" velocity="${motor_velocity}"/>
 </joint>
-<joint name="shoulder_pitch_stator_${arm_num}" type="fixed">
-	<parent link="shoulder_yaw_motor_${arm_num}"/>
-	<child link="shoulder_pitch_motor_${arm_num}"/>
-	<origin xyz="${ShoulderPitch_Ox} ${ShoulderPitch_Oy} ${ShoulderPitch_Oz}" rpy="${ShoulderPitch_roll} ${ShoulderPitch_pitch} ${ShoulderPitch_yaw}"/>
-</joint>
 <!-- arm pitch 1 -->
 <joint name="shoulder_pitch_${arm_num}" type="revolute">
-	<parent link="shoulder_pitch_motor_${arm_num}"/>
-	<child link="lower_arm_${arm_num}"/>
-	<origin xyz="${LowerArm_Ox} ${LowerArm_Oy} ${LowerArm_Oz}" rpy="${LowerArm_roll} ${LowerArm_pitch} ${LowerArm_yaw}"/>
+	<parent link="shoulder_yaw_${arm_num}"/>
+	<child link="shoulder_pitch_${arm_num}"/>
+	<origin xyz="${ShoulderPitch_Ox} ${ShoulderPitch_Oy} ${ShoulderPitch_Oz}" rpy="${ShoulderPitch_roll} ${ShoulderPitch_pitch} ${ShoulderPitch_yaw  + rot * PI_2}"/>
+	<axis xyz="0 1 0"/>
+	<limit lower="${j_pitch_1_lower[arm_num-1]}" upper="${j_pitch_1_upper[arm_num-1]}" effort="${motor_effort}" velocity="${motor_velocity}"/>
+</joint>
+<joint name="elbow_pitch_${arm_num}" type="revolute">
+	<parent link="shoulder_pitch_${arm_num}"/>
+	<child link="elbow_pitch_${arm_num}"/>
+	<origin xyz="${ElbowPitch_Ox} ${ElbowPitch_Oy} ${ElbowPitch_Oz}" rpy="${ElbowPitch_roll} ${ElbowPitch_pitch} ${ElbowPitch_yaw}"/>
 	<axis xyz="0 0 1"/>
 	<limit lower="${j_pitch_1_lower[arm_num-1]}" upper="${j_pitch_1_upper[arm_num-1]}" effort="${motor_effort}" velocity="${motor_velocity}"/>
 </joint>
-<joint name="elbow_pitch_stator_${arm_num}" type="fixed">
-	<parent link="lower_arm_${arm_num}"/>
-	<child link="elbow_pitch_motor_${arm_num}"/>
-	<origin xyz="${ElbowPitch_Ox} ${ElbowPitch_Oy} ${ElbowPitch_Oz}" rpy="${ElbowPitch_roll} ${ElbowPitch_pitch} ${ElbowPitch_yaw}"/>
-</joint>
-<!-- arm pitch 2 -->
-<joint name="elbow_pitch_${arm_num}" type="revolute">
-	<parent link="elbow_pitch_motor_${arm_num}"/>
-	<child link="upper_arm1_${arm_num}"/>
-	<origin xyz="${UpperArm1_Ox} ${UpperArm1_Oy} ${UpperArm1_Oz}" rpy="${UpperArm1_roll} ${UpperArm1_pitch} ${UpperArm1_yaw}"/>
-	<axis xyz="0 0 1"/>
-	<limit lower="${j_pitch_2_lower[arm_num-1]}" upper="${j_pitch_2_upper[arm_num-1]}" effort="${motor_effort}" velocity="${motor_velocity}"/>
-</joint>
 <joint name="wrist_pitch_stator_${arm_num}" type="fixed">
-	<parent link="upper_arm1_${arm_num}"/>
+	<parent link="elbow_pitch_${arm_num}"/>
 	<child link="wrist_pitch_motor_${arm_num}"/>
 	<origin xyz="${WristPitch_Ox} ${WristPitch_Oy} ${WristPitch_Oz}" rpy="${WristPitch_roll} ${WristPitch_pitch} ${WristPitch_yaw}"/>

Commit message: bugfix: joint name != link name

File: kyon_urdf/urdf/kyon_base.urdf.xacro (robot description, xacro)
@@ -34,5 +34,5 @@
 </joint>
 <link name="imu_link"/>
-<joint name="imu_link" type="fixed">
+<joint name="imu_joint" type="fixed">
     <parent link="pelvis"/>
     <child link="imu_link"/>

Commit message: Change default world + remove lidar from pelvis mesh

File: kyon_urdf/urdf/kyon_base.urdf.xacro (robot description, xacro)
@@ -18,5 +18,5 @@
 		<origin xyz="0.0 0 0.0"  rpy="0.0 0.0 0.0"/>
 		<geometry>
-	 		<mesh filename="package://kyon_urdf/meshes/mesh_pelvis.stl" scale="0.001 0.001 0.001"/>
+	 		<mesh filename="package://kyon_urdf/meshes/mesh_pelvis_no_lidar.stl" scale="0.001 0.001 0.001"/>
 		</geometry>
 	</visual>
@@ -47,5 +47,5 @@
         align_depth="true"
         unite_imu_method="false"
-        visualize="true"
+        visualize="false"
         accel_fps="300"
         gyro_fps="300"
@@ -68,5 +68,5 @@
         align_depth="true"
         unite_imu_method="false"
-        visualize="true"
+        visualize="false"
         accel_fps="300"
         gyro_fps="300"
@@ -110,5 +110,5 @@
         align_depth="true"
         unite_imu_method="false"
-        visualize="true"
+        visualize="false"
         accel_fps="300"
         gyro_fps="300"
@@ -131,5 +131,5 @@
         align_depth="true"
         unite_imu_method="false"
-        visualize="true"
+        visualize="false"
         accel_fps="300"
         gyro_fps="300"
@@ -167,8 +167,8 @@
     </xacro:sensor_d435i> -->
     <!-- Velodyne -->
-    <!-- <xacro:include filename="$(find velodyne_description)/urdf/VLP-16.urdf.xacro"/>
+    <xacro:include filename="$(find velodyne_description)/urdf/VLP-16.urdf.xacro"/>
     <xacro:VLP-16 parent="pelvis" name="velodyne" topic="/velodyne_points" hz="10" samples="440">
-        <origin xyz="0.36 0 0.11" rpy="0 0 0" />
-    </xacro:VLP-16> -->
+        <origin xyz="0.43 0 0.118" rpy="0 0 0.5220063" />
+    </xacro:VLP-16>
 </xacro:if>
 <xacro:if value="${ADD_UPPER_BODY}">

Commit message: moved imu link in correct position

File: kyon_urdf/urdf/kyon_base.urdf.xacro (robot description, xacro)
@@ -35,4 +35,5 @@
 <link name="imu_link"/>
 <joint name="imu_joint" type="fixed">
+	<origin xyz="-0.256190 0 0.103" rpy="${PI} 0 0"/>
     <parent link="pelvis"/>
     <child link="imu_link"/>

Commit message: merge --squash dev/fix_arm_joints_axis

File: kyon_urdf/urdf/kyon_base.urdf.xacro (robot description, xacro)
@@ -18,5 +18,5 @@
 		<origin xyz="0.0 0 0.0"  rpy="0.0 0.0 0.0"/>
 		<geometry>
-	 		<mesh filename="package://kyon_urdf/meshes/mesh_pelvis.stl" scale="0.001 0.001 0.001"/>
+	 		<mesh filename="package://kyon_urdf/meshes/mesh_pelvis_no_lidar.stl" scale="0.001 0.001 0.001"/>
 		</geometry>
 	</visual>
@@ -35,4 +35,5 @@
 <link name="imu_link"/>
 <joint name="imu_joint" type="fixed">
+	<origin xyz="-0.256190 0 0.103" rpy="${PI} 0 0"/>
     <parent link="pelvis"/>
     <child link="imu_link"/>
@@ -47,5 +48,5 @@
         align_depth="true"
         unite_imu_method="false"
-        visualize="true"
+        visualize="false"
         accel_fps="300"
         gyro_fps="300"
@@ -68,5 +69,5 @@
         align_depth="true"
         unite_imu_method="false"
-        visualize="true"
+        visualize="false"
         accel_fps="300"
         gyro_fps="300"
@@ -110,5 +111,5 @@
         align_depth="true"
         unite_imu_method="false"
-        visualize="true"
+        visualize="false"
         accel_fps="300"
         gyro_fps="300"
@@ -131,5 +132,5 @@
         align_depth="true"
         unite_imu_method="false"
-        visualize="true"
+        visualize="false"
         accel_fps="300"
         gyro_fps="300"
@@ -167,8 +168,8 @@
     </xacro:sensor_d435i> -->
     <!-- Velodyne -->
-    <!-- <xacro:include filename="$(find velodyne_description)/urdf/VLP-16.urdf.xacro"/>
+    <xacro:include filename="$(find velodyne_description)/urdf/VLP-16.urdf.xacro"/>
     <xacro:VLP-16 parent="pelvis" name="velodyne" topic="/velodyne_points" hz="10" samples="440">
-        <origin xyz="0.36 0 0.11" rpy="0 0 0" />
-    </xacro:VLP-16> -->
+        <origin xyz="0.43 0 0.118" rpy="0 0 0.5220063" />
+    </xacro:VLP-16>
 </xacro:if>
 <xacro:if value="${ADD_UPPER_BODY}">

Commit message: cameras' mount frames

File: kyon_urdf/urdf/kyon_base.urdf.xacro (robot description, xacro)
@@ -59,8 +59,33 @@
     <child link="imu_link"/>
 </joint>
+<!-- CAMERA BASE FRAMES -->
+<link name="up_front_camera_mount_link"/>
+<joint name="up_front_camera_mount_link" type="fixed">
+    <parent link="pelvis"/>
+    <child link="up_front_camera_mount_link"/>
+    <origin xyz="0.526174 0 0.0674608" rpy="0 -0.1745327 0"/>
+</joint>
+<link name="down_front_camera_mount_link"/>
+<joint name="down_front_camera_mount_link" type="fixed">
+    <parent link="pelvis"/>
+    <child link="down_front_camera_mount_link"/>
+    <origin xyz="0.509601 0 0.00343992" rpy="0 0.9250251 0"/>
+</joint>
+<link name="left_camera_mount_link"/>
+<joint name="left_camera_mount_link" type="fixed">
+    <parent link="pelvis"/>
+    <child link="left_camera_mount_link"/>
+    <origin xyz="0 0.150100 0.109486" rpy="0 0.3490656 1.5707963"/>
+</joint>
+<link name="right_camera_mount_link"/>
+<joint name="right_camera_mount_link" type="fixed">
+    <parent link="pelvis"/>
+    <child link="right_camera_mount_link"/>
+    <origin xyz="0 -0.150100 0.109486" rpy="0 0.3490656 -1.5707963"/>
+</joint>
 <xacro:if value="${ADD_CAMERAS}">
     <xacro:include filename="$(find realsense_gazebo_description)/urdf/_d435i.urdf.xacro" />
     <!-- LEFT D435 CAMERA -->
-    <xacro:sensor_d435i parent="pelvis"
+    <xacro:sensor_d435i parent="left_camera_mount_link"
         name="D435_left"
         topics_ns="D435_left"
@@ -80,8 +105,7 @@
         color_height="720"
         color_fps="1">
-        <origin xyz="0 0.150100 0.109486" rpy="0 0.3490656 1.5707963"/>
     </xacro:sensor_d435i>
     <!-- RIGHT D435 CAMERA -->
-    <xacro:sensor_d435i parent="pelvis"
+    <xacro:sensor_d435i parent="right_camera_mount_link"
         name="D435_right"
         topics_ns="D435_right"
@@ -101,8 +125,7 @@
         color_height="720"
         color_fps="1">
-        <origin xyz="0 -0.150100 0.109486" rpy="0 0.3490656 -1.5707963"/>
     </xacro:sensor_d435i>
     <!-- FRONT1 D435 CAMERA -->
-    <xacro:sensor_d435i parent="pelvis"
+    <xacro:sensor_d435i parent="up_front_camera_mount_link"
         name="D435_front1"
         topics_ns="D435_front1"
@@ -122,8 +145,7 @@
         color_height="720"
         color_fps="30">
-        <origin xyz="0.526174 0 0.0674608" rpy="0 -0.1745327 0"/>
     </xacro:sensor_d435i>
     <!-- FRONT2 D435 CAMERA -->
-    <xacro:sensor_d435i parent="pelvis"
+    <xacro:sensor_d435i parent="down_front_camera_mount_link"
         name="D435_front2"
         topics_ns="D435_front2"
@@ -143,5 +165,4 @@
         color_height="720"
         color_fps="30">
-        <origin xyz="0.509601 0 0.00343992" rpy="0 0.9250251 0"/>
     </xacro:sensor_d435i>
 </xacro:if>

Commit message: renamed camra mounts

File: kyon_urdf/urdf/kyon_base.urdf.xacro (robot description, xacro)
@@ -60,18 +60,18 @@
 </joint>
 <!-- CAMERA BASE FRAMES -->
-<link name="up_front_camera_mount_link"/>
-<joint name="up_front_camera_mount_link" type="fixed">
-    <parent link="pelvis"/>
-    <child link="up_front_camera_mount_link"/>
+<link name="zed_front_up_mount_link"/>
+<joint name="zed_front_up_mount_joint" type="fixed">
+    <parent link="pelvis"/>
+    <child link="zed_front_up_mount_link"/>
     <origin xyz="0.526174 0 0.0674608" rpy="0 -0.1745327 0"/>
 </joint>
-<link name="down_front_camera_mount_link"/>
-<joint name="down_front_camera_mount_link" type="fixed">
-    <parent link="pelvis"/>
-    <child link="down_front_camera_mount_link"/>
+<link name="zed_front_down_mount_link"/>
+<joint name="zed_front_down_mount_joint" type="fixed">
+    <parent link="pelvis"/>
+    <child link="zed_front_down_mount_link"/>
     <origin xyz="0.509601 0 0.00343992" rpy="0 0.9250251 0"/>
 </joint>
 <link name="left_camera_mount_link"/>
-<joint name="left_camera_mount_link" type="fixed">
+<joint name="left_camera_mount_joint" type="fixed">
     <parent link="pelvis"/>
     <child link="left_camera_mount_link"/>
@@ -79,5 +79,5 @@
 </joint>
 <link name="right_camera_mount_link"/>
-<joint name="right_camera_mount_link" type="fixed">
+<joint name="right_camera_mount_joint" type="fixed">
     <parent link="pelvis"/>
     <child link="right_camera_mount_link"/>

Commit message: fix camera link name and origin tags

File: kyon_urdf/urdf/kyon_base.urdf.xacro (robot description, xacro)
@@ -105,4 +105,5 @@
         color_height="720"
         color_fps="1">
+        <origin xyz="0 0 0" rpy="0 0 0"/>
     </xacro:sensor_d435i>
     <!-- RIGHT D435 CAMERA -->
@@ -125,7 +126,8 @@
         color_height="720"
         color_fps="1">
+        <origin xyz="0 0 0" rpy="0 0 0"/>
     </xacro:sensor_d435i>
     <!-- FRONT1 D435 CAMERA -->
-    <xacro:sensor_d435i parent="up_front_camera_mount_link"
+    <xacro:sensor_d435i parent="zed_front_up_mount_link"
         name="D435_front1"
         topics_ns="D435_front1"
@@ -145,7 +147,8 @@
         color_height="720"
         color_fps="30">
+        <origin xyz="0 0 0" rpy="0 0 0"/>
     </xacro:sensor_d435i>
     <!-- FRONT2 D435 CAMERA -->
-    <xacro:sensor_d435i parent="down_front_camera_mount_link"
+    <xacro:sensor_d435i parent="zed_front_down_mount_link"
         name="D435_front2"
         topics_ns="D435_front2"
@@ -165,4 +168,5 @@
         color_height="720"
         color_fps="30">
+        <origin xyz="0 0 0" rpy="0 0 0"/>
     </xacro:sensor_d435i>
 </xacro:if>

Commit message: add hesai lidar frame

File: kyon_urdf/urdf/kyon_base.urdf.xacro (robot description, xacro)
@@ -172,4 +172,10 @@
 </xacro:if>
 <!-- Velodyne -->
+<link name="hesai_lidar"/>
+<joint name="hesai_lidar_joints" type="fixed">
+    <origin xyz="0.43 0 0.118" rpy="0 0 0.5220063" />
+    <parent link="pelvis"/>
+	<child link="hesai_lidar"/>
+</joint>
 <xacro:if value="${ADD_VELODYNE}">
     <xacro:include filename="$(find velodyne_description)/urdf/VLP-16.urdf.xacro"/>

Commit message: modify camera parameters for elevation_mapping_cupy

File: kyon_urdf/urdf/kyon_base.urdf.xacro (robot description, xacro)
@@ -64,5 +64,5 @@
     <parent link="pelvis"/>
     <child link="zed_front_up_mount_link"/>
-    <origin xyz="0.526174 0 0.0674608" rpy="0 -0.1745327 0"/>
+    <origin xyz="-0.509601 0 0.00343992" rpy="0 2.0250251 -${PI}"/>
 </joint>
 <link name="zed_front_down_mount_link"/>
@@ -94,15 +94,15 @@
         unite_imu_method="false"
         visualize="false"
-        accel_fps="300"
-        gyro_fps="300"
-        depth_width="1280"
-        depth_height="720"
-        depth_fps="10"
-        infra_width="1280"
-        infra_height="720"
-        infra_fps="10"
-        color_width="1280"
-        color_height="720"
-        color_fps="1">
+        accel_fps="30"
+        gyro_fps="30"
+        depth_width="320"
+        depth_height="162"
+        depth_fps="30"
+        infra_width="320"
+        infra_height="162"
+        infra_fps="30"
+        color_width="320"
+        color_height="162"
+        color_fps="30">
         <origin xyz="0 0 0" rpy="0 0 0"/>
     </xacro:sensor_d435i>
@@ -115,15 +115,15 @@
         unite_imu_method="false"
         visualize="false"
-        accel_fps="300"
-        gyro_fps="300"
-        depth_width="1280"
-        depth_height="720"
-        depth_fps="10"
-        infra_width="1280"
-        infra_height="720"
-        infra_fps="10"
-        color_width="1280"
-        color_height="720"
-        color_fps="1">
+        accel_fps="30"
+        gyro_fps="30"
+        depth_width="320"
+        depth_height="162"
+        depth_fps="30"
+        infra_width="848"
+        infra_height="480"
+        infra_fps="30"
+        color_width="848"
+        color_height="480"
+        color_fps="30">
         <origin xyz="0 0 0" rpy="0 0 0"/>
     </xacro:sensor_d435i>
@@ -136,14 +136,14 @@
         unite_imu_method="false"
         visualize="false"
-        accel_fps="300"
-        gyro_fps="300"
-        depth_width="1280"
-        depth_height="720"
-        depth_fps="90"
-        infra_width="1280"
-        infra_height="720"
-        infra_fps="90"
-        color_width="1280"
-        color_height="720"
+        accel_fps="30"
+        gyro_fps="30"
+        depth_width="320"
+        depth_height="162"
+        depth_fps="30"
+        infra_width="320"
+        infra_height="162"
+        infra_fps="30"
+        color_width="320"
+        color_height="162"
         color_fps="30">
         <origin xyz="0 0 0" rpy="0 0 0"/>
@@ -157,14 +157,14 @@
         unite_imu_method="false"
         visualize="false"
-        accel_fps="300"
-        gyro_fps="300"
-        depth_width="1280"
-        depth_height="720"
-        depth_fps="90"
-        infra_width="1280"
-        infra_height="720"
-        infra_fps="90"
-        color_width="1280"
-        color_height="720"
+        accel_fps="30"
+        gyro_fps="30"
+        depth_width="320"
+        depth_height="162"
+        depth_fps="30"
+        infra_width="320"
+        infra_height="162"
+        infra_fps="30"
+        color_width="320"
+        color_height="162"
         color_fps="30">
         <origin xyz="0 0 0" rpy="0 0 0"/>
