Commit message: default to continuous joints for wheels

File: kyon_urdf/urdf/kyon_leg_wheel.urdf (robot description, URDF)
Before this commit: robot kyon, 7 links, 6 joints
Joints:
- joint wheel_joint_2: type revolute -> continuous

File: kyon_urdf/urdf/parts/steering_wheel.urdf.xacro (robot description, xacro)
@@ -84,5 +84,5 @@
     <limit lower="${ankle_yaw_lower[leg_num-1]}" upper="${ankle_yaw_upper[leg_num-1]}" effort="${motorA_effort}" velocity="${motorA_velocity}"/>
 </joint>
-<joint name="wheel_joint_${leg_num}" type="revolute">
+<joint name="wheel_joint_${leg_num}" type="continuous">
     <parent link="ankle_yaw_${leg_num}_link"/>
     <child link="wheel_${leg_num}"/>
