Commit message: first version with minimal collisions

File: kyon_isaac/urdf/kyon_minimal.urdf (robot description, URDF)
Before this commit: robot kyon, 33 links, 32 joints
Links:
- link dagana_1_base: geometry collision box size=0.09 0.03 0.09; collision box size=0.095 0.08 0.06
- link dagana_1_claw: geometry collision box size=0.09 0.03 0.09; visual mesh filename=/workspace/iit-kyon-ros-pkg/kyon_isaac/urdf/meshes/mesh_dag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 scale=0.001 0.001 0.001
- link dagana_2_base: geometry collision box size=0.09 0.03 0.09; collision box size=0.095 0.08 0.06
- link dagana_2_claw: geometry collision box size=0.09 0.03 0.09; visual mesh filename=/workspace/iit-kyon-ros-pkg/kyon_isaac/urdf/meshes/mesh_dag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 scale=0.001 0.001 0.001
- link elbow_pitch_1_link: geometry collision box size=0.08 0.14 0.05; visual mesh filename=/workspace/iit-kyon-ros-pkg/kyon_isaac/urdf/meshes/mesh_elb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 scale=0.001 0.001 0.001
- link elbow_pitch_2_link: geometry collision box size=0.08 0.14 0.05; visual mesh filename=/workspace/iit-kyon-ros-pkg/kyon_isaac/urdf/meshes/mesh_elb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 scale=0.001 0.001 0.001
- link hip_roll_1_link: geometry visual mesh filename=/workspace/iit-kyon-ros-pkg/kyon_isaac/urdf/meshes/mesh_hip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 scale=0.001 -0.001 0.001
- link hip_roll_2_link: geometry visual mesh filename=/workspace/iit-kyon-ros-pkg/kyon_isaac/urdf/meshes/mesh_hip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 scale=0.001 0.001 0.001
- link hip_roll_3_link: geometry visual mesh filename=/workspace/iit-kyon-ros-pkg/kyon_isaac/urdf/meshes/mesh_hip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 scale=0.001 -0.001 0.001
- link hip_roll_4_link: geometry visual mesh filename=/workspace/iit-kyon-ros-pkg/kyon_isaac/urdf/meshes/mesh_hip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 scale=0.001 0.001 0.001
- link pelvis: geometry collision cylinder length=0.5 radius=0.17; visual mesh filename=/workspace/iit-kyon-ros-pkg/kyon_isaac/urdf/meshes/mesh_pel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 scale=0.001 0.001 0.001
- link shoulder_pitch_1_link: geometry collision box size=0.08 0.19 0.05; collision cylinder length=0.12 radius=0.055
- link shoulder_pitch_2_link: geometry collision box size=0.08 0.19 0.05; collision cylinder length=0.12 radius=0.055
- link shoulder_yaw_1_link: geometry collision cylinder length=0.16 radius=0.07; visual mesh filename=/workspace/iit-kyon-ros-pkg/kyon_isaac/urdf/meshes/mesh_sh_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 scale=0.001 0.001 0.001
- link shoulder_yaw_2_link: geometry collision cylinder length=0.16 radius=0.07; visual mesh filename=/workspace/iit-kyon-ros-pkg/kyon_isaac/urdf/meshes/mesh_sh_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 scale=0.001 0.001 0.001
- link wrist_pitch_1_link: geometry collision cylinder length=0.1 radius=0.04; visual mesh filename=/workspace/iit-kyon-ros-pkg/kyon_isaac/urdf/meshes/mesh_wri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 scale=0.001 0.001 0.001
- link wrist_pitch_2_link: geometry collision cylinder length=0.1 radius=0.04; visual mesh filename=/workspace/iit-kyon-ros-pkg/kyon_isaac/urdf/meshes/mesh_wri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 scale=0.001 0.001 0.001
- link wrist_yaw_1_link: geometry collision cylinder length=0.1 radius=0.04; visual mesh filename=/workspace/iit-kyon-ros-pkg/kyon_isaac/urdf/meshes/mesh_wri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 scale=0.001 0.001 0.001
- link wrist_yaw_2_link: geometry collision cylinder length=0.1 radius=0.04; visual mesh filename=/workspace/iit-kyon-ros-pkg/kyon_isaac/urdf/meshes/mesh_wri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 scale=0.001 0.001 0.001

Commit message: update pelvis and hip pitch collisions

File: kyon_isaac/urdf/kyon_minimal.urdf (robot description, URDF)
Before this commit: robot kyon, 33 links, 32 joints
Links:
- link hip_pitch_1_link: geometry collision box size=0.11 0.3 0.08; collision cylinder length=0.06 radius=0.052
- link hip_pitch_2_link: geometry collision box size=0.11 0.3 0.08; collision cylinder length=0.06 radius=0.052
- link hip_pitch_3_link: geometry collision box size=0.11 0.3 0.08; collision cylinder length=0.06 radius=0.052
- link hip_pitch_4_link: geometry collision box size=0.11 0.3 0.08; collision cylinder length=0.06 radius=0.052
- link pelvis: geometry collision cylinder length=0.50 radius=0.15; visual mesh filename=/workspace/iit-kyon-ros-pkg/kyon_isaac/urdf/meshes/mesh_pel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 scale=0.001 0.001 0.001
