Commit message: meshes for visual, dummy boxes for collision

File: kyon_isaac/urdf/kyon.urdf (robot description, URDF)
Before this commit: robot kyon, 32 links, 31 joints
Links:
- added link base_link
- link dagana_1_base: geometry collision box size=0.894 0.1615 0.356; visual mesh filename=/home/idadiotis/forest_ws/src/iit-kyon-ros-pkg/kyon_urdf/me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 scale=0.001 0.001 0.001
- link dagana_1_claw: geometry collision box size=0.894 0.1615 0.356; visual mesh filename=/home/idadiotis/forest_ws/src/iit-kyon-ros-pkg/kyon_urdf/me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 scale=0.001 0.001 0.001
- link dagana_2_base: geometry collision box size=0.894 0.1615 0.356; visual mesh filename=/home/idadiotis/forest_ws/src/iit-kyon-ros-pkg/kyon_urdf/me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 scale=0.001 0.001 0.001
- link dagana_2_claw: geometry collision box size=0.894 0.1615 0.356; visual mesh filename=/home/idadiotis/forest_ws/src/iit-kyon-ros-pkg/kyon_urdf/me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 scale=0.001 0.001 0.001
- link elbow_pitch_1_link: geometry collision box size=0.894 0.1615 0.356; visual mesh filename=/home/idadiotis/forest_ws/src/iit-kyon-ros-pkg/kyon_urdf/me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 scale=0.001 0.001 0.001
- link elbow_pitch_2_link: geometry collision box size=0.894 0.1615 0.356; visual mesh filename=/home/idadiotis/forest_ws/src/iit-kyon-ros-pkg/kyon_urdf/me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 scale=0.001 0.001 0.001
- link hip_pitch_1_link: geometry collision box size=0.894 0.1615 0.356; visual mesh filename=/home/idadiotis/forest_ws/src/iit-kyon-ros-pkg/kyon_urdf/me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 scale=0.001 0.001 0.001
- link hip_pitch_2_link: geometry collision box size=0.894 0.1615 0.356; visual mesh filename=/home/idadiotis/forest_ws/src/iit-kyon-ros-pkg/kyon_urdf/me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 scale=0.001 0.001 0.001
- link hip_pitch_3_link: geometry collision box size=0.894 0.1615 0.356; visual mesh filename=/home/idadiotis/forest_ws/src/iit-kyon-ros-pkg/kyon_urdf/me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 scale=0.001 0.001 0.001
- link hip_pitch_4_link: geometry collision box size=0.894 0.1615 0.356; visual mesh filename=/home/idadiotis/forest_ws/src/iit-kyon-ros-pkg/kyon_urdf/me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 scale=0.001 0.001 0.001
- link hip_roll_1_link: geometry collision box size=0.894 0.1615 0.356; visual mesh filename=/home/idadiotis/forest_ws/src/iit-kyon-ros-pkg/kyon_urdf/me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 scale=0.001 -0.001 0.001
- link hip_roll_2_link: geometry collision box size=0.894 0.1615 0.356; visual mesh filename=/home/idadiotis/forest_ws/src/iit-kyon-ros-pkg/kyon_urdf/me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 scale=0.001 0.001 0.001
- link hip_roll_3_link: geometry collision box size=0.894 0.1615 0.356; visual mesh filename=/home/idadiotis/forest_ws/src/iit-kyon-ros-pkg/kyon_urdf/me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 scale=0.001 -0.001 0.001
- link hip_roll_4_link: geometry collision box size=0.894 0.1615 0.356; visual mesh filename=/home/idadiotis/forest_ws/src/iit-kyon-ros-pkg/kyon_urdf/me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 scale=0.001 0.001 0.001
- link knee_pitch_1_link: geometry collision box size=0.894 0.1615 0.356; visual mesh filename=/home/idadiotis/forest_ws/src/iit-kyon-ros-pkg/kyon_urdf/me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 scale=-0.001 0.001 0.001
- link knee_pitch_2_link: geometry collision box size=0.894 0.1615 0.356; visual mesh filename=/home/idadiotis/forest_ws/src/iit-kyon-ros-pkg/kyon_urdf/me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 scale=0.001 0.001 0.001
- link knee_pitch_3_link: geometry collision box size=0.894 0.1615 0.356; visual mesh filename=/home/idadiotis/forest_ws/src/iit-kyon-ros-pkg/kyon_urdf/me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 scale=-0.001 0.001 0.001
- link knee_pitch_4_link: geometry collision box size=0.894 0.1615 0.356; visual mesh filename=/home/idadiotis/forest_ws/src/iit-kyon-ros-pkg/kyon_urdf/me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 scale=0.001 0.001 0.001
- link pelvis: geometry collision box size=0.894 0.1615 0.356; visual mesh filename=/home/idadiotis/forest_ws/src/iit-kyon-ros-pkg/kyon_urdf/me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 scale=0.001 0.001 0.001
- link shoulder_pitch_1_link: geometry collision box size=0.894 0.1615 0.356; visual mesh filename=/home/idadiotis/forest_ws/src/iit-kyon-ros-pkg/kyon_urdf/me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 scale=0.001 0.001 0.001
- link shoulder_pitch_2_link: geometry collision box size=0.894 0.1615 0.356; visual mesh filename=/home/idadiotis/forest_ws/src/iit-kyon-ros-pkg/kyon_urdf/me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 scale=0.001 0.001 0.001
- link shoulder_yaw_1_link: geometry collision box size=0.894 0.1615 0.356; visual mesh filename=/home/idadiotis/forest_ws/src/iit-kyon-ros-pkg/kyon_urdf/me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 scale=0.001 0.001 0.001
- link shoulder_yaw_2_link: geometry collision box size=0.894 0.1615 0.356; visual mesh filename=/home/idadiotis/forest_ws/src/iit-kyon-ros-pkg/kyon_urdf/me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 scale=0.001 0.001 0.001
- link wrist_pitch_1_link: geometry collision box size=0.894 0.1615 0.356; visual mesh filename=/home/idadiotis/forest_ws/src/iit-kyon-ros-pkg/kyon_urdf/me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 scale=0.001 0.001 0.001
- link wrist_pitch_2_link: geometry collision box size=0.894 0.1615 0.356; visual mesh filename=/home/idadiotis/forest_ws/src/iit-kyon-ros-pkg/kyon_urdf/me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 scale=0.001 0.001 0.001
- link wrist_yaw_1_link: geometry collision box size=0.894 0.1615 0.356; visual mesh filename=/home/idadiotis/forest_ws/src/iit-kyon-ros-pkg/kyon_urdf/me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 scale=0.001 0.001 0.001
- link wrist_yaw_2_link: geometry collision box size=0.894 0.1615 0.356; visual mesh filename=/home/idadiotis/forest_ws/src/iit-kyon-ros-pkg/kyon_urdf/me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 scale=0.001 0.001 0.001
Joints:
- added joint base_joint: type fixed, parent pelvis, child base_link, origin xyz=0 0 0 rpy=0 0 0
- joint hip_roll_1: parent pelvis -> base_link
- joint hip_roll_2: parent pelvis -> base_link
- joint hip_roll_3: parent pelvis -> base_link
- joint hip_roll_4: parent pelvis -> base_link
- joint imu_joint: parent pelvis -> base_link
- joint shoulder_yaw_1: parent pelvis -> base_link
- joint shoulder_yaw_2: parent pelvis -> base_link

Commit message: fix wrong path for visuals

File: kyon_isaac/urdf/kyon.urdf (robot description, URDF)
Before this commit: robot kyon, 33 links, 32 joints
Links:
- link dagana_1_base: geometry collision box size=0.894 0.1615 0.356; visual mesh filename=/workspace/iit-kyon-ros-pkg/kyon_isaac/meshes/mesh_dagana_b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 scale=0.001 0.001 0.001
- link dagana_1_claw: geometry collision box size=0.894 0.1615 0.356; visual mesh filename=/workspace/iit-kyon-ros-pkg/kyon_isaac/meshes/mesh_dagana_c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 scale=0.001 0.001 0.001
- link dagana_2_base: geometry collision box size=0.894 0.1615 0.356; visual mesh filename=/workspace/iit-kyon-ros-pkg/kyon_isaac/meshes/mesh_dagana_b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 scale=0.001 0.001 0.001
- link dagana_2_claw: geometry collision box size=0.894 0.1615 0.356; visual mesh filename=/workspace/iit-kyon-ros-pkg/kyon_isaac/meshes/mesh_dagana_c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 scale=0.001 0.001 0.001
- link elbow_pitch_1_link: geometry collision box size=0.894 0.1615 0.356; visual mesh filename=/workspace/iit-kyon-ros-pkg/kyon_isaac/meshes/mesh_elbow.stl scale=0.001 0.001 0.001
- link elbow_pitch_2_link: geometry collision box size=0.894 0.1615 0.356; visual mesh filename=/workspace/iit-kyon-ros-pkg/kyon_isaac/meshes/mesh_elbow.stl scale=0.001 0.001 0.001
- link hip_pitch_1_link: geometry collision box size=0.894 0.1615 0.356; visual mesh filename=/workspace/iit-kyon-ros-pkg/kyon_isaac/meshes/mesh_hip_pitc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 scale=0.001 0.001 0.001
- link hip_pitch_2_link: geometry collision box size=0.894 0.1615 0.356; visual mesh filename=/workspace/iit-kyon-ros-pkg/kyon_isaac/meshes/mesh_hip_pitc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 scale=0.001 0.001 0.001
- link hip_pitch_3_link: geometry collision box size=0.894 0.1615 0.356; visual mesh filename=/workspace/iit-kyon-ros-pkg/kyon_isaac/meshes/mesh_hip_pitc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 scale=0.001 0.001 0.001
- link hip_pitch_4_link: geometry collision box size=0.894 0.1615 0.356; visual mesh filename=/workspace/iit-kyon-ros-pkg/kyon_isaac/meshes/mesh_hip_pitc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 scale=0.001 0.001 0.001
- link hip_roll_1_link: geometry collision box size=0.894 0.1615 0.356; visual mesh filename=/workspace/iit-kyon-ros-pkg/kyon_isaac/meshes/mesh_hip_roll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 scale=0.001 -0.001 0.001
- link hip_roll_2_link: geometry collision box size=0.894 0.1615 0.356; visual mesh filename=/workspace/iit-kyon-ros-pkg/kyon_isaac/meshes/mesh_hip_roll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 scale=0.001 0.001 0.001
- link hip_roll_3_link: geometry collision box size=0.894 0.1615 0.356; visual mesh filename=/workspace/iit-kyon-ros-pkg/kyon_isaac/meshes/mesh_hip_roll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 scale=0.001 -0.001 0.001
- link hip_roll_4_link: geometry collision box size=0.894 0.1615 0.356; visual mesh filename=/workspace/iit-kyon-ros-pkg/kyon_isaac/meshes/mesh_hip_roll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 scale=0.001 0.001 0.001
- link knee_pitch_1_link: geometry collision box size=0.894 0.1615 0.356; visual mesh filename=/workspace/iit-kyon-ros-pkg/kyon_isaac/meshes/mesh_foot_leg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 scale=-0.001 0.001 0.001
- link knee_pitch_2_link: geometry collision box size=0.894 0.1615 0.356; visual mesh filename=/workspace/iit-kyon-ros-pkg/kyon_isaac/meshes/mesh_foot_leg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 scale=0.001 0.001 0.001
- link knee_pitch_3_link: geometry collision box size=0.894 0.1615 0.356; visual mesh filename=/workspace/iit-kyon-ros-pkg/kyon_isaac/meshes/mesh_foot_leg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 scale=-0.001 0.001 0.001
- link knee_pitch_4_link: geometry collision box size=0.894 0.1615 0.356; visual mesh filename=/workspace/iit-kyon-ros-pkg/kyon_isaac/meshes/mesh_foot_leg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 scale=0.001 0.001 0.001
- link pelvis: geometry collision box size=0.894 0.1615 0.356; visual mesh filename=/workspace/iit-kyon-ros-pkg/kyon_isaac/meshes/mesh_pelvis.s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 scale=0.001 0.001 0.001
- link shoulder_pitch_1_link: geometry collision box size=0.894 0.1615 0.356; visual mesh filename=/workspace/iit-kyon-ros-pkg/kyon_isaac/meshes/mesh_sh_pitch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 scale=0.001 0.001 0.001
- link shoulder_pitch_2_link: geometry collision box size=0.894 0.1615 0.356; visual mesh filename=/workspace/iit-kyon-ros-pkg/kyon_isaac/meshes/mesh_sh_pitch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 scale=0.001 0.001 0.001
- link shoulder_yaw_1_link: geometry collision box size=0.894 0.1615 0.356; visual mesh filename=/workspace/iit-kyon-ros-pkg/kyon_isaac/meshes/mesh_sh_yaw.s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 scale=0.001 0.001 0.001
- link shoulder_yaw_2_link: geometry collision box size=0.894 0.1615 0.356; visual mesh filename=/workspace/iit-kyon-ros-pkg/kyon_isaac/meshes/mesh_sh_yaw.s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 scale=0.001 0.001 0.001
- link wrist_pitch_1_link: geometry collision box size=0.894 0.1615 0.356; visual mesh filename=/workspace/iit-kyon-ros-pkg/kyon_isaac/meshes/mesh_wrist_pi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 scale=0.001 0.001 0.001
- link wrist_pitch_2_link: geometry collision box size=0.894 0.1615 0.356; visual mesh filename=/workspace/iit-kyon-ros-pkg/kyon_isaac/meshes/mesh_wrist_pi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 scale=0.001 0.001 0.001
- link wrist_yaw_1_link: geometry collision box size=0.894 0.1615 0.356; visual mesh filename=/workspace/iit-kyon-ros-pkg/kyon_isaac/meshes/mesh_wrist_ya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 scale=0.001 0.001 0.001
- link wrist_yaw_2_link: geometry collision box size=0.894 0.1615 0.356; visual mesh filename=/workspace/iit-kyon-ros-pkg/kyon_isaac/meshes/mesh_wrist_ya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 scale=0.001 0.001 0.001

Commit message: again fix wrong path

File: kyon_isaac/urdf/kyon.urdf (robot description, URDF)
Before this commit: robot kyon, 33 links, 32 joints
Links:
- link dagana_1_base: geometry collision box size=0.894 0.1615 0.356; visual mesh filename=/workspace/iit-kyon-ros-pkg/kyon_isaac/urdf/meshes/mesh_dag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 scale=0.001 0.001 0.001
- link dagana_1_claw: geometry collision box size=0.894 0.1615 0.356; visual mesh filename=/workspace/iit-kyon-ros-pkg/kyon_isaac/urdf/meshes/mesh_dag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 scale=0.001 0.001 0.001
- link dagana_2_base: geometry collision box size=0.894 0.1615 0.356; visual mesh filename=/workspace/iit-kyon-ros-pkg/kyon_isaac/urdf/meshes/mesh_dag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 scale=0.001 0.001 0.001
- link dagana_2_claw: geometry collision box size=0.894 0.1615 0.356; visual mesh filename=/workspace/iit-kyon-ros-pkg/kyon_isaac/urdf/meshes/mesh_dag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 scale=0.001 0.001 0.001
- link elbow_pitch_1_link: geometry collision box size=0.894 0.1615 0.356; visual mesh filename=/workspace/iit-kyon-ros-pkg/kyon_isaac/urdf/meshes/mesh_elb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 scale=0.001 0.001 0.001
- link elbow_pitch_2_link: geometry collision box size=0.894 0.1615 0.356; visual mesh filename=/workspace/iit-kyon-ros-pkg/kyon_isaac/urdf/meshes/mesh_elb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 scale=0.001 0.001 0.001
- link hip_pitch_1_link: geometry collision box size=0.894 0.1615 0.356; visual mesh filename=/workspace/iit-kyon-ros-pkg/kyon_isaac/urdf/meshes/mesh_hip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 scale=0.001 0.001 0.001
- link hip_pitch_2_link: geometry collision box size=0.894 0.1615 0.356; visual mesh filename=/workspace/iit-kyon-ros-pkg/kyon_isaac/urdf/meshes/mesh_hip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 scale=0.001 0.001 0.001
- link hip_pitch_3_link: geometry collision box size=0.894 0.1615 0.356; visual mesh filename=/workspace/iit-kyon-ros-pkg/kyon_isaac/urdf/meshes/mesh_hip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 scale=0.001 0.001 0.001
- link hip_pitch_4_link: geometry collision box size=0.894 0.1615 0.356; visual mesh filename=/workspace/iit-kyon-ros-pkg/kyon_isaac/urdf/meshes/mesh_hip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 scale=0.001 0.001 0.001
- link hip_roll_1_link: geometry collision box size=0.894 0.1615 0.356; visual mesh filename=/workspace/iit-kyon-ros-pkg/kyon_isaac/urdf/meshes/mesh_hip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 scale=0.001 -0.001 0.001
- link hip_roll_2_link: geometry collision box size=0.894 0.1615 0.356; visual mesh filename=/workspace/iit-kyon-ros-pkg/kyon_isaac/urdf/meshes/mesh_hip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 scale=0.001 0.001 0.001
- link hip_roll_3_link: geometry collision box size=0.894 0.1615 0.356; visual mesh filename=/workspace/iit-kyon-ros-pkg/kyon_isaac/urdf/meshes/mesh_hip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 scale=0.001 -0.001 0.001
- link hip_roll_4_link: geometry collision box size=0.894 0.1615 0.356; visual mesh filename=/workspace/iit-kyon-ros-pkg/kyon_isaac/urdf/meshes/mesh_hip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 scale=0.001 0.001 0.001
- link knee_pitch_1_link: geometry collision box size=0.894 0.1615 0.356; visual mesh filename=/workspace/iit-kyon-ros-pkg/kyon_isaac/urdf/meshes/mesh_foo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 scale=-0.001 0.001 0.001
- link knee_pitch_2_link: geometry collision box size=0.894 0.1615 0.356; visual mesh filename=/workspace/iit-kyon-ros-pkg/kyon_isaac/urdf/meshes/mesh_foo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 scale=0.001 0.001 0.001
- link knee_pitch_3_link: geometry collision box size=0.894 0.1615 0.356; visual mesh filename=/workspace/iit-kyon-ros-pkg/kyon_isaac/urdf/meshes/mesh_foo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 scale=-0.001 0.001 0.001
- link knee_pitch_4_link: geometry collision box size=0.894 0.1615 0.356; visual mesh filename=/workspace/iit-kyon-ros-pkg/kyon_isaac/urdf/meshes/mesh_foo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 scale=0.001 0.001 0.001
- link pelvis: geometry collision box size=0.894 0.1615 0.356; visual mesh filename=/workspace/iit-kyon-ros-pkg/kyon_isaac/urdf/meshes/mesh_pel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 scale=0.001 0.001 0.001
- link shoulder_pitch_1_link: geometry collision box size=0.894 0.1615 0.356; visual mesh filename=/workspace/iit-kyon-ros-pkg/kyon_isaac/urdf/meshes/mesh_sh_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 scale=0.001 0.001 0.001
- link shoulder_pitch_2_link: geometry collision box size=0.894 0.1615 0.356; visual mesh filename=/workspace/iit-kyon-ros-pkg/kyon_isaac/urdf/meshes/mesh_sh_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 scale=0.001 0.001 0.001
- link shoulder_yaw_1_link: geometry collision box size=0.894 0.1615 0.356; visual mesh filename=/workspace/iit-kyon-ros-pkg/kyon_isaac/urdf/meshes/mesh_sh_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 scale=0.001 0.001 0.001
- link shoulder_yaw_2_link: geometry collision box size=0.894 0.1615 0.356; visual mesh filename=/workspace/iit-kyon-ros-pkg/kyon_isaac/urdf/meshes/mesh_sh_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 scale=0.001 0.001 0.001
- link wrist_pitch_1_link: geometry collision box size=0.894 0.1615 0.356; visual mesh filename=/workspace/iit-kyon-ros-pkg/kyon_isaac/urdf/meshes/mesh_wri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 scale=0.001 0.001 0.001
- link wrist_pitch_2_link: geometry collision box size=0.894 0.1615 0.356; visual mesh filename=/workspace/iit-kyon-ros-pkg/kyon_isaac/urdf/meshes/mesh_wri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 scale=0.001 0.001 0.001
- link wrist_yaw_1_link: geometry collision box size=0.894 0.1615 0.356; visual mesh filename=/workspace/iit-kyon-ros-pkg/kyon_isaac/urdf/meshes/mesh_wri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 scale=0.001 0.001 0.001
- link wrist_yaw_2_link: geometry collision box size=0.894 0.1615 0.356; visual mesh filename=/workspace/iit-kyon-ros-pkg/kyon_isaac/urdf/meshes/mesh_wri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 scale=0.001 0.001 0.001

Commit message: simplify upper body collision (wip)

File: kyon_isaac/urdf/kyon.urdf (robot description, URDF)
Before this commit: robot kyon, 33 links, 32 joints
Links:
- link dagana_1_base: geometry collision box size=0.095 0.08 0.06; collision box size=0.11 0.03 0.09
- link dagana_1_claw: geometry collision box size=0.11 0.03 0.09; visual mesh filename=/workspace/iit-kyon-ros-pkg/kyon_isaac/urdf/meshes/mesh_dag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 scale=0.001 0.001 0.001
- link elbow_pitch_1_link: geometry collision box size=0.08 0.14 0.05; visual mesh filename=/workspace/iit-kyon-ros-pkg/kyon_isaac/urdf/meshes/mesh_elb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 scale=0.001 0.001 0.001
- link hip_pitch_1_link: geometry collision box size=0.13 0.4 0.08; collision cylinder length=0.17 radius=0.065
- link hip_pitch_2_link: geometry collision box size=0.13 0.4 0.08; collision cylinder length=0.17 radius=0.065
- link hip_pitch_3_link: geometry collision box size=0.13 0.4 0.08; collision cylinder length=0.17 radius=0.065
- link hip_pitch_4_link: geometry collision box size=0.13 0.4 0.08; collision cylinder length=0.17 radius=0.065
- link hip_roll_1_link: geometry visual mesh filename=/workspace/iit-kyon-ros-pkg/kyon_isaac/urdf/meshes/mesh_hip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 scale=0.001 -0.001 0.001
- link hip_roll_2_link: geometry visual mesh filename=/workspace/iit-kyon-ros-pkg/kyon_isaac/urdf/meshes/mesh_hip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 scale=0.001 0.001 0.001
- link hip_roll_3_link: geometry visual mesh filename=/workspace/iit-kyon-ros-pkg/kyon_isaac/urdf/meshes/mesh_hip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 scale=0.001 -0.001 0.001
- link hip_roll_4_link: geometry visual mesh filename=/workspace/iit-kyon-ros-pkg/kyon_isaac/urdf/meshes/mesh_hip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 scale=0.001 0.001 0.001
- link knee_pitch_1_link: geometry collision box size=0.05 0.33 0.04; collision sphere radius=0.03
- link knee_pitch_2_link: geometry collision box size=0.05 0.33 0.04; collision sphere radius=0.03
- link knee_pitch_3_link: geometry collision box size=0.05 0.33 0.04; collision sphere radius=0.03
- link knee_pitch_4_link: geometry collision box size=0.05 0.33 0.04; collision sphere radius=0.03
- link pelvis: geometry collision box size=1.0 0.1615 0.30; visual mesh filename=/workspace/iit-kyon-ros-pkg/kyon_isaac/urdf/meshes/mesh_pel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 scale=0.001 0.001 0.001
- link shoulder_pitch_1_link: geometry collision box size=0.08 0.19 0.05; collision cylinder length=0.12 radius=0.055
- link shoulder_yaw_1_link: geometry collision cylinder length=0.16 radius=0.07; visual mesh filename=/workspace/iit-kyon-ros-pkg/kyon_isaac/urdf/meshes/mesh_sh_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 scale=0.001 0.001 0.001
- link wrist_pitch_1_link: geometry collision cylinder length=0.1 radius=0.04; visual mesh filename=/workspace/iit-kyon-ros-pkg/kyon_isaac/urdf/meshes/mesh_wri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 scale=0.001 0.001 0.001
- link wrist_yaw_1_link: geometry collision cylinder length=0.1 radius=0.04; visual mesh filename=/workspace/iit-kyon-ros-pkg/kyon_isaac/urdf/meshes/mesh_wri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 scale=0.001 0.001 0.001
Joints:
- joint hip_roll_1: parent base_link -> pelvis
