Commit message: update urdf with detailed collision

File: kyon_isaac/urdf/kyon.urdf (robot description, URDF)
Before this commit: robot kyon, 33 links, 32 joints
Links:
- removed link base_link
- link dagana_1_base: geometry collision mesh filename=/workspace/iit-kyon-ros-pkg/kyon_isaac/urdf/meshes/collisio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 scale=0.001 0.001 0.001; visual mesh filename=/workspace/iit-kyon-ros-pkg/kyon_isaac/urdf/meshes/mesh_dag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 scale=0.001 0.001 0.001
- link dagana_1_claw: geometry collision mesh filename=/workspace/iit-kyon-ros-pkg/kyon_isaac/urdf/meshes/collisio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 scale=0.001 0.001 0.001; visual mesh filename=/workspace/iit-kyon-ros-pkg/kyon_isaac/urdf/meshes/mesh_dag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 scale=0.001 0.001 0.001
- link dagana_2_base: geometry collision mesh filename=/workspace/iit-kyon-ros-pkg/kyon_isaac/urdf/meshes/collisio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 scale=0.001 0.001 0.001; visual mesh filename=/workspace/iit-kyon-ros-pkg/kyon_isaac/urdf/meshes/mesh_dag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 scale=0.001 0.001 0.001
- link dagana_2_claw: geometry collision mesh filename=/workspace/iit-kyon-ros-pkg/kyon_isaac/urdf/meshes/collisio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 scale=0.001 0.001 0.001; visual mesh filename=/workspace/iit-kyon-ros-pkg/kyon_isaac/urdf/meshes/mesh_dag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 scale=0.001 0.001 0.001
- link elbow_pitch_1_link: geometry collision mesh filename=/workspace/iit-kyon-ros-pkg/kyon_isaac/urdf/meshes/mesh_elb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 scale=0.001 0.001 0.001; visual mesh filename=/workspace/iit-kyon-ros-pkg/kyon_isaac/urdf/meshes/mesh_elb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 scale=0.001 0.001 0.001
- link elbow_pitch_2_link: geometry collision mesh filename=/workspace/iit-kyon-ros-pkg/kyon_isaac/urdf/meshes/mesh_elb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 scale=0.001 0.001 0.001; visual mesh filename=/workspace/iit-kyon-ros-pkg/kyon_isaac/urdf/meshes/mesh_elb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 scale=0.001 0.001 0.001
- link hip_pitch_1_link: geometry collision mesh filename=/workspace/iit-kyon-ros-pkg/kyon_isaac/urdf/meshes/collisio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 scale=0.001 0.001 0.001; visual mesh filename=/workspace/iit-kyon-ros-pkg/kyon_isaac/urdf/meshes/mesh_hip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 scale=0.001 0.001 0.001
- link hip_pitch_2_link: geometry collision mesh filename=/workspace/iit-kyon-ros-pkg/kyon_isaac/urdf/meshes/collisio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 scale=0.001 0.001 0.001; visual mesh filename=/workspace/iit-kyon-ros-pkg/kyon_isaac/urdf/meshes/mesh_hip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 scale=0.001 0.001 0.001
- link hip_pitch_3_link: geometry collision mesh filename=/workspace/iit-kyon-ros-pkg/kyon_isaac/urdf/meshes/collisio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 scale=0.001 0.001 0.001; visual mesh filename=/workspace/iit-kyon-ros-pkg/kyon_isaac/urdf/meshes/mesh_hip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 scale=0.001 0.001 0.001
- link hip_pitch_4_link: geometry collision mesh filename=/workspace/iit-kyon-ros-pkg/kyon_isaac/urdf/meshes/collisio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 scale=0.001 0.001 0.001; visual mesh filename=/workspace/iit-kyon-ros-pkg/kyon_isaac/urdf/meshes/mesh_hip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 scale=0.001 0.001 0.001
- link hip_roll_1_link: geometry collision mesh filename=/workspace/iit-kyon-ros-pkg/kyon_isaac/urdf/meshes/collisio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 scale=0.001 -0.001 0.001; visual mesh filename=/workspace/iit-kyon-ros-pkg/kyon_isaac/urdf/meshes/mesh_hip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 scale=0.001 -0.001 0.001
- link hip_roll_2_link: geometry collision mesh filename=/workspace/iit-kyon-ros-pkg/kyon_isaac/urdf/meshes/collisio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 scale=0.001 0.001 0.001; visual mesh filename=/workspace/iit-kyon-ros-pkg/kyon_isaac/urdf/meshes/mesh_hip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 scale=0.001 0.001 0.001
- link hip_roll_3_link: geometry collision mesh filename=/workspace/iit-kyon-ros-pkg/kyon_isaac/urdf/meshes/collisio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 scale=0.001 -0.001 0.001; visual mesh filename=/workspace/iit-kyon-ros-pkg/kyon_isaac/urdf/meshes/mesh_hip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 scale=0.001 -0.001 0.001
- link hip_roll_4_link: geometry collision mesh filename=/workspace/iit-kyon-ros-pkg/kyon_isaac/urdf/meshes/collisio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 scale=0.001 0.001 0.001; visual mesh filename=/workspace/iit-kyon-ros-pkg/kyon_isaac/urdf/meshes/mesh_hip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 scale=0.001 0.001 0.001
- link knee_pitch_1_link: geometry collision mesh filename=/workspace/iit-kyon-ros-pkg/kyon_isaac/urdf/meshes/collisio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 scale=-0.001 0.001 0.001; visual mesh filename=/workspace/iit-kyon-ros-pkg/kyon_isaac/urdf/meshes/mesh_foo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 scale=-0.001 0.001 0.001
- link knee_pitch_2_link: geometry collision mesh filename=/workspace/iit-kyon-ros-pkg/kyon_isaac/urdf/meshes/collisio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 scale=0.001 0.001 0.001; visual mesh filename=/workspace/iit-kyon-ros-pkg/kyon_isaac/urdf/meshes/mesh_foo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 scale=0.001 0.001 0.001
- link knee_pitch_3_link: geometry collision mesh filename=/workspace/iit-kyon-ros-pkg/kyon_isaac/urdf/meshes/collisio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 scale=-0.001 0.001 0.001; visual mesh filename=/workspace/iit-kyon-ros-pkg/kyon_isaac/urdf/meshes/mesh_foo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 scale=-0.001 0.001 0.001
- link knee_pitch_4_link: geometry collision mesh filename=/workspace/iit-kyon-ros-pkg/kyon_isaac/urdf/meshes/collisio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 scale=0.001 0.001 0.001; visual mesh filename=/workspace/iit-kyon-ros-pkg/kyon_isaac/urdf/meshes/mesh_foo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 scale=0.001 0.001 0.001
- link pelvis: geometry collision mesh filename=/workspace/iit-kyon-ros-pkg/kyon_isaac/urdf/meshes/collisio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 scale=0.001 0.001 0.001; visual mesh filename=/workspace/iit-kyon-ros-pkg/kyon_isaac/urdf/meshes/mesh_pel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 scale=0.001 0.001 0.001
- link shoulder_pitch_1_link: geometry collision mesh filename=/workspace/iit-kyon-ros-pkg/kyon_isaac/urdf/meshes/collisio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 scale=0.001 0.001 0.001; visual mesh filename=/workspace/iit-kyon-ros-pkg/kyon_isaac/urdf/meshes/mesh_sh_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 scale=0.001 0.001 0.001
- link shoulder_pitch_2_link: geometry collision mesh filename=/workspace/iit-kyon-ros-pkg/kyon_isaac/urdf/meshes/collisio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 scale=0.001 0.001 0.001; visual mesh filename=/workspace/iit-kyon-ros-pkg/kyon_isaac/urdf/meshes/mesh_sh_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 scale=0.001 0.001 0.001
- link shoulder_yaw_1_link: geometry collision mesh filename=/workspace/iit-kyon-ros-pkg/kyon_isaac/urdf/meshes/collisio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 scale=0.001 0.001 0.001; visual mesh filename=/workspace/iit-kyon-ros-pkg/kyon_isaac/urdf/meshes/mesh_sh_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 scale=0.001 0.001 0.001
- link shoulder_yaw_2_link: geometry collision mesh filename=/workspace/iit-kyon-ros-pkg/kyon_isaac/urdf/meshes/collisio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 scale=0.001 0.001 0.001; visual mesh filename=/workspace/iit-kyon-ros-pkg/kyon_isaac/urdf/meshes/mesh_sh_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 scale=0.001 0.001 0.001
- link wrist_pitch_1_link: geometry collision mesh filename=/workspace/iit-kyon-ros-pkg/kyon_isaac/urdf/meshes/collisio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 scale=0.001 0.001 0.001; visual mesh filename=/workspace/iit-kyon-ros-pkg/kyon_isaac/urdf/meshes/mesh_wri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 scale=0.001 0.001 0.001
- link wrist_pitch_2_link: geometry collision mesh filename=/workspace/iit-kyon-ros-pkg/kyon_isaac/urdf/meshes/collisio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 scale=0.001 0.001 0.001; visual mesh filename=/workspace/iit-kyon-ros-pkg/kyon_isaac/urdf/meshes/mesh_wri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 scale=0.001 0.001 0.001
- link wrist_yaw_1_link: geometry collision mesh filename=/workspace/iit-kyon-ros-pkg/kyon_isaac/urdf/meshes/collisio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 scale=0.001 0.001 0.001; visual mesh filename=/workspace/iit-kyon-ros-pkg/kyon_isaac/urdf/meshes/mesh_wri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 scale=0.001 0.001 0.001
- link wrist_yaw_2_link: geometry collision mesh filename=/workspace/iit-kyon-ros-pkg/kyon_isaac/urdf/meshes/collisio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 scale=0.001 0.001 0.001; visual mesh filename=/workspace/iit-kyon-ros-pkg/kyon_isaac/urdf/meshes/mesh_wri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 scale=0.001 0.001 0.001
Joints:
- removed joint base_joint
- joint hip_roll_2: parent base_link -> pelvis
- joint hip_roll_3: parent base_link -> pelvis
- joint hip_roll_4: parent base_link -> pelvis
- joint imu_joint: parent base_link -> pelvis
- joint shoulder_yaw_1: parent base_link -> pelvis
- joint shoulder_yaw_2: parent base_link -> pelvis

Commit message: update urdf for isaac and usd for xacro consistency

File: kyon_isaac/urdf/kyon.urdf (robot description, URDF)
Before this commit: robot kyon, 32 links, 31 joints
Joints:
- joint contact_1_joint: origin xyz=0.03 -0.35 0.03 rpy=-1.57 0 0.785 -> xyz=0.0 -0.3 0.054 rpy=-1.57 0 0.785
- joint contact_2_joint: origin xyz=-0.03 -0.35 0.03 rpy=1.57 0 2.356 -> xyz=-0.0 -0.3 0.054 rpy=1.57 0 2.356
- joint contact_3_joint: origin xyz=0.03 -0.35 0.03 rpy=-1.57 0 0.785 -> xyz=0.0 -0.3 0.054 rpy=-1.57 0 0.785
- joint contact_4_joint: origin xyz=-0.03 -0.35 0.03 rpy=1.57 0 2.356 -> xyz=-0.0 -0.3 0.054 rpy=1.57 0 2.356
- joint elbow_pitch_1: axis 0 0 1 -> 0 0 -1
- joint elbow_pitch_2: axis 0 0 1 -> 0 0 -1
- joint imu_joint: origin (none) -> xyz=-0.256190 0 0.103 rpy=3.14159265359 0 0
- joint shoulder_yaw_1: axis 0 0 1 -> 0 0 -1
- joint shoulder_yaw_2: axis 0 0 1 -> 0 0 -1
- joint wrist_pitch_1: axis 0 0 1 -> 0 0 -1
- joint wrist_pitch_2: axis 0 0 1 -> 0 0 -1

File: kyon_isaac/urdf/kyon_minimal.urdf (robot description, URDF)
Before this commit: robot kyon, 33 links, 32 joints
Joints:
- joint contact_1_joint: origin xyz=0.03 -0.35 0.03 rpy=-1.57 0 0.785 -> xyz=0.0 -0.3 0.054 rpy=-1.57 0 0.785
- joint contact_2_joint: origin xyz=-0.03 -0.35 0.03 rpy=1.57 0 2.356 -> xyz=-0.0 -0.3 0.054 rpy=1.57 0 2.356
- joint contact_3_joint: origin xyz=0.03 -0.35 0.03 rpy=-1.57 0 0.785 -> xyz=0.0 -0.3 0.054 rpy=-1.57 0 0.785
- joint contact_4_joint: origin xyz=-0.03 -0.35 0.03 rpy=1.57 0 2.356 -> xyz=-0.0 -0.3 0.054 rpy=1.57 0 2.356
- joint elbow_pitch_1: axis 0 0 1 -> 0 0 -1
- joint elbow_pitch_2: axis 0 0 1 -> 0 0 -1
- joint imu_joint: origin (none) -> xyz=-0.256190 0 0.103 rpy=3.14159265359 0 0
- joint shoulder_yaw_1: axis 0 0 1 -> 0 0 -1
- joint shoulder_yaw_2: axis 0 0 1 -> 0 0 -1
- joint wrist_pitch_1: axis 0 0 1 -> 0 0 -1
- joint wrist_pitch_2: axis 0 0 1 -> 0 0 -1
