Commit message: addedo wheels

File: kyon_srdf/srdf/kyon.srdf.xacro (robot description, xacro)
@@ -12,16 +12,32 @@
     </group>
     <xacro:if value="${ADD_LEGS}">
-        <group name="front_left_leg">
-            <chain base_link="pelvis" tip_link="ball_1" />
-        </group>
-        <group name="front_right_leg">
-            <chain base_link="pelvis" tip_link="ball_2" />
-        </group>
-        <group name="rear_right_leg">
-            <chain base_link="pelvis" tip_link="ball_4" />
-        </group>
-        <group name="rear_left_leg">
-            <chain base_link="pelvis" tip_link="ball_3" />
-        </group>
+    	<xacro:if value="${ADD_WHEELS}">
+			<group name="front_left_leg">
+		        <chain base_link="pelvis" tip_link="wheel_1" />
+		    </group>
+		    <group name="front_right_leg">
+		        <chain base_link="pelvis" tip_link="wheel_2" />
+		    </group>
+		    <group name="rear_right_leg">
+		        <chain base_link="pelvis" tip_link="wheel_4" />
+		    </group>
+		    <group name="rear_left_leg">
+		        <chain base_link="pelvis" tip_link="wheel_3" />
+		    </group>
+		</xacro:if>
+		<xacro:unless value="${ADD_WHEELS}">
+		    <group name="front_left_leg">
+		        <chain base_link="pelvis" tip_link="ball_1" />
+		    </group>
+		    <group name="front_right_leg">
+		        <chain base_link="pelvis" tip_link="ball_2" />
+		    </group>
+		    <group name="rear_right_leg">
+		        <chain base_link="pelvis" tip_link="ball_4" />
+		    </group>
+		    <group name="rear_left_leg">
+		        <chain base_link="pelvis" tip_link="ball_3" />
+		    </group>
+		</xacro:unless>
     </xacro:if>
     <xacro:if value="${ADD_UPPER_BODY}">

File: kyon_urdf/urdf/config/kyon.urdf.xacro (robot description, xacro)
@@ -7,4 +7,5 @@
 <xacro:arg name="upper_body" default="true"/>
 <xacro:arg name="dagana" default="false"/>
+<xacro:arg name="wheels" default="false"/>
 <xacro:arg name="floating_joint" default="true"/>
 <xacro:arg name="sensors" default="true"/>
@@ -16,4 +17,5 @@
 <xacro:property name="ADD_SENSORS" value="$(arg sensors)" />
 <xacro:property name="ADD_DAGANA" value="$(arg dagana)"/>
+<xacro:property name="ADD_WHEELS" value="$(arg wheels)"/>
 <xacro:property name="ADD_FLOATING_BASE" value="$(arg floating_joint)" />
 <xacro:property name="ADD_VIRTUAL_FRAME" value="false" />

File: kyon_urdf/urdf/parts/inertial_properties.urdf.xacro (robot description, xacro)
@@ -88,3 +88,15 @@
     <xacro:property name="Ball_yz" value="0.0"/>
     <xacro:property name="Ball_zz" value="${2/3 * ball_mass * ball_radius * ball_radius}"/>
+    <xacro:property name="Wheel23_mass" value="1.8569388e+00"/>
+    <!-- Center of Mass -->
+	<xacro:property name="Wheel23_x" value="${0.0 * mmTom}"/>
+	<xacro:property name="Wheel23_y" value="${0.0 * mmTom}"/>
+	<xacro:property name="Wheel23_z" value="${-1.5403767e-01 * mmTom}"/>
+	<!-- Inertia -->
+	<xacro:property name="Wheel23_xx" value="${8.6373591e+03 * mm2Tom2}"/>
+	<xacro:property name="Wheel23_yy" value="${8.6373644e+03 * mm2Tom2}"/>
+	<xacro:property name="Wheel23_zz" value="${1.6376551e+04 * mm2Tom2}"/>
+	<xacro:property name="Wheel23_xy" value="${0.0 * mm2Tom2}"/>
+	<xacro:property name="Wheel23_xz" value="${0.0 * mm2Tom2}"/>
+	<xacro:property name="Wheel23_yz" value="${0.0 * mm2Tom2}"/>
 </robot>

File: kyon_urdf/urdf/parts/kinematics_properties.urdf.xacro (robot description, xacro)
@@ -117,3 +117,9 @@
     <xacro:property name="EndEffector_pitch" value="${PI_2}"/>
     <xacro:property name="EndEffector_yaw" value="0.0"/>
+    <xacro:property name="Wheel23_Ox" value="0.0"/>
+    <xacro:property name="Wheel23_Oy" value="0.0"/>
+    <xacro:property name="Wheel23_Oz" value="${ball_radius}"/>
+    <xacro:property name="Wheel23_roll" value="0.0"/>
+    <xacro:property name="Wheel23_pitch" value="0.0"/>
+    <xacro:property name="Wheel23_yaw" value="0.0"/>
 </robot>

File: kyon_urdf/urdf/parts/kyon_leg.urdf.xacro (robot description, xacro)
@@ -124,4 +124,37 @@
 	</collision>
 </link>
+<xacro:if value="${ADD_WHEELS}">
+	<joint name="wheel_joint_${leg_num}" type="continuous">
+            <parent link="ball_${leg_num}" />
+            <child link="wheel_${leg_num}" />
+            <origin xyz="${Wheel23_Ox} ${Wheel23_Oy} ${-mirror*Wheel23_Oz}" rpy="${Wheel23_roll} ${Wheel23_pitch} ${Wheel23_yaw}" />
+            <axis xyz="0 0 ${mirror}"/>
+            <limit effort="${motor_effort}" velocity="${motor_velocity}" />  <!-- 23 Nm, 1
+            rad/s-->
+        </joint>
+        <link name="wheel_${leg_num}">
+            <inertial>
+                <origin xyz="${Wheel23_x} ${Wheel23_y} ${mirror*Wheel23_z}" />
+                <mass value="${Wheel23_mass}" />
+                <inertia ixx="${Wheel23_xx}" ixy="${Wheel23_xy}" ixz="${mirror*Wheel23_xz}" iyy="${Wheel23_yy}" iyz="${mirror*Wheel23_yz}" izz="${Wheel23_zz}" />
+            </inertial>
+            <visual>
+                <origin xyz="0.0 0.0 0.0" rpy="0.0 0.0 0.0" />
+                <geometry>
+                    <mesh filename="package://centauro_urdf/meshes/v2/mesh_wheel23.stl"
+                        scale="0.001 0.001 ${mirror*0.001}" />
+                </geometry>
+                <material name="black" />
+            </visual>
+            <collision>
+                <origin xyz="0 0 0" rpy="0 0 0" />
+                <geometry>
+                    <mesh filename="package://centauro_urdf/meshes/v2/collision/mesh_wheel23.stl"
+                        scale="0.001 0.001 ${mirror*0.001}" />
+                </geometry>
+                <material name="black" />
+            </collision>
+        </link>
+</xacro:if>
 <!-- joints -->
 <joint name="hip_roll_${leg_num}" type="revolute">

Commit message: now using optional find package, optional package root explicitly as argument
Signed-off-by: Andrea Patrizi <andreapatrizi1b6e6@gmail.com>

File: kyon_srdf/srdf/kyon.srdf.xacro (robot description, xacro)
@@ -6,5 +6,7 @@
 <robot xmlns:xacro="http://ros.org/wiki/xacro" name="kyon">
     <!-- ************ MODEL CONFIGURATION ************ -->
-    <xacro:arg name="config" default="$(find kyon_urdf)/urdf/config/kyon.urdf.xacro"/>
+    <xacro:arg name="kyon_root" default="$(find kyon_urdf)" />
+    <xacro:property name="KYON_ROOT" value="$(arg kyon_root)" />
+    <xacro:arg name="config" default="${KYON_ROOT}/urdf/config/kyon.urdf.xacro"/>
     <xacro:include filename="$(arg config)"/>
     <group name="base">

File: kyon_urdf/urdf/kyon.urdf.xacro (robot description, xacro)
@@ -1,9 +1,24 @@
 <?xml version="1.0"?>
 <robot xmlns:xacro="http://ros.org/wiki/xacro" name="kyon">
-<xacro:arg name="config" default="$(find kyon_urdf)/urdf/config/kyon.urdf.xacro"/>
+<!-- This argument and property should be in the top level xacro and
+will be propagated to all its downstream childs -->
+<xacro:arg name="kyon_root" default="$(find kyon_urdf)" />
+<xacro:property name="KYON_ROOT" value="$(arg kyon_root)" />
+<xacro:arg name="config" default="${KYON_ROOT}/urdf/config/kyon.urdf.xacro"/>
 <!-- ************ MODEL CONFIGURATION ************ -->
 <xacro:include filename="$(arg config)"/>
+<!-- here the properties from the config are set -->
+<xacro:if value="${ADD_DAGANA}">
+	<xacro:arg name="dagana_root" default="$(find dagana_urdf)" />
+	<xacro:property name="DAGANA_ROOT" value="$(arg dagana_root)" />
+</xacro:if>
+<xacro:if value="${ADD_SENSORS}">
+	<xacro:arg name="realsense_gazebo_description_root" default="$(find realsense_gazebo_description)" />
+	<xacro:property name="REALSENSE_GAZEBO_DESCRIPTION_ROOT" value="$(arg realsense_gazebo_description_root)" />
+	<xacro:arg name="velodyne_description_root" default="$(find velodyne_description)" />
+	<xacro:property name="VELODYNE_DESCRIPTION_ROOT" value="$(arg velodyne_description_root)" />
+</xacro:if>
 <!-- ************ CETC-SAT plain model ************ -->
-<xacro:include filename="$(find kyon_urdf)/urdf/kyon_base.urdf.xacro"/>
+<xacro:include filename="${KYON_ROOT}/urdf/kyon_base.urdf.xacro"/>
 <!-- ************ Control frames ************ -->
 <!--xacro:include filename="$(find pholus_urdf)/urdf/control_frames.urdf.xacro"/-->

File: kyon_urdf/urdf/kyon_base.urdf.xacro (robot description, xacro)
@@ -3,9 +3,9 @@
 <xacro:arg name="bilevel_codes" default="false" /> <!-- if true, load codes vars from externally provided files-->
 <xacro:arg name="sample_idx" default = "0"/>
-<xacro:include filename="$(find kyon_urdf)/urdf/utils.urdf.xacro" />
-<xacro:include filename="$(find kyon_urdf)/urdf/parts/kinematics_properties.urdf.xacro" />
+<xacro:include filename="${KYON_ROOT}/urdf/utils.urdf.xacro" />
+<xacro:include filename="${KYON_ROOT}/urdf/parts/kinematics_properties.urdf.xacro" />
 <!-- NOTE: here we need to include "kinematics_properties" first because "inertial_properties" depends on it-->
-<xacro:include filename="$(find kyon_urdf)/urdf/parts/inertial_properties.urdf.xacro" />
-<xacro:include filename="$(find kyon_urdf)/urdf/parts/limits.urdf.xacro" />
+<xacro:include filename="${KYON_ROOT}/urdf/parts/inertial_properties.urdf.xacro" />
+<xacro:include filename="${KYON_ROOT}/urdf/parts/limits.urdf.xacro" />
 <link name="base_link"/>
 <link name="pelvis">
@@ -36,5 +36,5 @@
 </joint>
 <xacro:if value="${ADD_SENSORS}">
-    <xacro:include filename="$(find realsense_gazebo_description)/urdf/_d435i.urdf.xacro" />
+    <xacro:include filename="${REALSENSE_GAZEBO_DESCRIPTION_ROOT}/urdf/_d435i.urdf.xacro" />
     <!-- LEFT D435 CAMERA -->
     <xacro:sensor_d435i parent="pelvis"
@@ -164,5 +164,5 @@
     </xacro:sensor_d435i>
     <!-- Velodyne -->
-    <xacro:include filename="$(find velodyne_description)/urdf/VLP-16.urdf.xacro"/>
+    <xacro:include filename="${VELODYNE_DESCRIPTION_ROOT}/urdf/VLP-16.urdf.xacro"/>
     <xacro:VLP-16 parent="pelvis" name="velodyne" topic="/velodyne_points" hz="10" samples="440">
         <origin xyz="0.36 0 0.11" rpy="0 0 0" />
@@ -170,8 +170,8 @@
 </xacro:if>
 <xacro:if value="${ADD_UPPER_BODY}">
-    <xacro:include filename="$(find kyon_urdf)/urdf/parts/arms.urdf.xacro" />
+    <xacro:include filename="${KYON_ROOT}/urdf/parts/arms.urdf.xacro" />
 </xacro:if>
 <xacro:if value="${ADD_LEGS}">
-	<xacro:include filename="$(find kyon_urdf)/urdf/parts/legs.urdf.xacro" />
+	<xacro:include filename="${KYON_ROOT}/urdf/parts/legs.urdf.xacro" />
 </xacro:if>
 <xacro:if value="${PAYLOAD}">

File: kyon_urdf/urdf/kyon_robot.urdf.xacro (robot description, xacro)
@@ -1,8 +1,10 @@
 <?xml version="1.0"?>
 <robot xmlns:xacro="http://ros.org/wiki/xacro" name="kyon">
-  <xacro:include filename="$(find kyon_urdf)/urdf/kyon.urdf.xacro" />
-  <xacro:include filename="$(find kyon_urdf)/urdf/gazebo/kyon.gazebo.xacro" />
-  <xacro:include filename="$(find kyon_urdf)/urdf/gazebo/xbot.gazebo.xacro" />
-  <xacro:include filename="$(find kyon_urdf)/urdf/gazebo/materials.gazebo.xacro" />
+  <!-- Define PACKAGE_ROOT as a xacro argument with a default value -->
+  <xacro:arg name="PACKAGE_ROOT" default="$(find kyon_urdf)" />
+  <xacro:include filename="${KYON_ROOT}/urdf/kyon.urdf.xacro" />
+  <xacro:include filename="${KYON_ROOT}/urdf/gazebo/kyon.gazebo.xacro" />
+  <xacro:include filename="${KYON_ROOT}/urdf/gazebo/xbot.gazebo.xacro" />
+  <xacro:include filename="${KYON_ROOT}/urdf/gazebo/materials.gazebo.xacro" />
   <xacro:unless value="${ADD_LEGS}">
     <link name="world"/>

File: kyon_urdf/urdf/parts/arms.urdf.xacro (robot description, xacro)
@@ -1,7 +1,7 @@
 <?xml version="1.0"?>
 <robot xmlns:xacro="http://ros.org/wiki/xacro">
-<xacro:include filename="$(find kyon_urdf)/urdf/parts/kyon_arm.urdf.xacro"/>
-<xacro:include filename="$(find kyon_urdf)/urdf/parts/kyon_ball_ee.xacro"/>
-<xacro:include filename="$(find dagana_urdf)/urdf/dagana_macro.urdf.xacro"/>
+<xacro:include filename="${KYON_ROOT}/urdf/parts/kyon_arm.urdf.xacro"/>
+<xacro:include filename="${KYON_ROOT}/urdf/parts/kyon_ball_ee.xacro"/>
+<xacro:include filename="${DAGANA_ROOT}/urdf/dagana_macro.urdf.xacro"/>
 <!-- arms -->
 <xacro:kyon_arm arm_num="1"  rot="1"  parent="pelvis">

File: kyon_urdf/urdf/parts/inertial_properties.urdf.xacro (robot description, xacro)
@@ -1,5 +1,5 @@
 <?xml version="1.0"?>
 <robot  xmlns:xacro="http://ros.org/wiki/xacro">
-    <xacro:property name="inertial_yaml_file" value="$(find kyon_urdf)/urdf/config/inertial_properties.yaml" />
+    <xacro:property name="inertial_yaml_file" value="${KYON_ROOT}/urdf/config/inertial_properties.yaml" />
     <xacro:property name="inertial_props" value="${xacro.load_yaml(inertial_yaml_file)}"/>
     <xacro:property name="pelvis_mass" value="${inertial_props['pelvis_mass']}"/>

File: kyon_urdf/urdf/parts/kinematics_properties.urdf.xacro (robot description, xacro)
@@ -1,5 +1,5 @@
 <?xml version="1.0"?>
 <robot  xmlns:xacro="http://ros.org/wiki/xacro">
-    <xacro:property name="kin_yaml_file" value="$(find kyon_urdf)/urdf/config/kinematics_properties.yaml" />
+    <xacro:property name="kin_yaml_file" value="${KYON_ROOT}/urdf/config/kinematics_properties.yaml" />
     <xacro:property name="kin_props" value="${xacro.load_yaml(kin_yaml_file)}"/>
     <xacro:property name="cylinder_radius" value="${kin_props['cylinder_radius']}"/>

File: kyon_urdf/urdf/parts/legs.urdf.xacro (robot description, xacro)
@@ -1,5 +1,5 @@
 <?xml version="1.0"?>
 <robot xmlns:xacro="http://ros.org/wiki/xacro">
-<xacro:include filename="$(find kyon_urdf)/urdf/parts/kyon_leg.urdf.xacro" />
+<xacro:include filename="${KYON_ROOT}/urdf/parts/kyon_leg.urdf.xacro" />
 <xacro:kyon_leg leg_num="1" origin_x="1" origin_y="-1" mirror="-1">
 </xacro:kyon_leg>
