Commit message: fixed link names && contact_i frame && more launch and configs

File: kyon_srdf/srdf/kyon.srdf.xacro (robot description, xacro)
@@ -28,14 +28,14 @@
 		<xacro:unless value="${ADD_WHEELS}">
 		    <group name="front_left_leg">
-		        <chain base_link="pelvis" tip_link="ball_1" />
+		        <chain base_link="pelvis" tip_link="contact_1" />
 		    </group>
 		    <group name="front_right_leg">
-		        <chain base_link="pelvis" tip_link="ball_2" />
+		        <chain base_link="pelvis" tip_link="contact_2" />
 		    </group>
 		    <group name="rear_right_leg">
-		        <chain base_link="pelvis" tip_link="ball_4" />
+		        <chain base_link="pelvis" tip_link="contact_4" />
 		    </group>
 		    <group name="rear_left_leg">
-		        <chain base_link="pelvis" tip_link="ball_3" />
+		        <chain base_link="pelvis" tip_link="contact_3" />
 		    </group>
 		</xacro:unless>
@@ -44,9 +44,15 @@
     	<xacro:if value="${ADD_DAGANA}">
 			<group name="left_arm">
-				<chain base_link="pelvis" tip_link="dagana_1_bottom_link"/>
+				<chain base_link="pelvis" tip_link="dagana_1_clamp"/>
 			</group>
 			<group name="right_arm">
-				<chain base_link="pelvis" tip_link="dagana_2_bottom_link"/>
+				<chain base_link="pelvis" tip_link="dagana_2_clamp"/>
 			</group>
+            <!-- <group name="left_hand">
+				<chain base_link="dagana_1_base" tip_link="dagana_1_clamp"/>
+			</group>
+            <group name="right_hand">
+				<chain base_link="dagana_1_base" tip_link="dagana_2_clamp"/>
+			</group> -->
 		</xacro:if>
 		<xacro:unless value="${ADD_DAGANA}">
@@ -70,4 +76,8 @@
             <group name="right_arm"/>
         </xacro:if>
+        <!-- <xacro:if value="${ADD_DAGANA}">
+            <group name="left_hand"/>
+            <group name="right_hand"/>
+        </xacro:if> -->
     </group>
     <!-- Homing posture -->
@@ -78,23 +88,23 @@
             <joint name="knee_pitch_1" value="-1.4"/>
             <joint name="hip_roll_2" value="0.0"/>
-            <joint name="hip_pitch_2" value="0.7"/>
-            <joint name="knee_pitch_2" value="-1.4"/>
+            <joint name="hip_pitch_2" value="-0.7"/>
+            <joint name="knee_pitch_2" value="1.4"/>
             <joint name="hip_roll_3" value="0.0"/>
             <joint name="hip_pitch_3" value="0.7"/>
             <joint name="knee_pitch_3" value="-1.4"/>
             <joint name="hip_roll_4" value="0.0"/>
-            <joint name="hip_pitch_4" value="0.7"/>
-            <joint name="knee_pitch_4" value="-1.4"/>
+            <joint name="hip_pitch_4" value="-0.7"/>
+            <joint name="knee_pitch_4" value="1.4"/>
         </xacro:if>
         <xacro:if value="${ADD_UPPER_BODY}">
-            <joint name="shoulder_yaw_1" value="-0.05"/>
-            <joint name="shoulder_pitch_1" value="0.50"/>
-            <joint name="elbow_pitch_1" value="1.25"/>
-            <joint name="wrist_pitch_1" value="0.0"/>
+            <joint name="shoulder_yaw_1" value="0.0"/>
+            <joint name="shoulder_pitch_1" value="1.7"/>
+            <joint name="elbow_pitch_1" value="-2.50"/>
+            <joint name="wrist_pitch_1" value="0.75"/>
             <joint name="wrist_yaw_1" value="0.0"/>
-            <joint name="shoulder_yaw_2" value="0.05"/>
-            <joint name="shoulder_pitch_2" value="0.50"/>
-            <joint name="elbow_pitch_2" value="1.25"/>
-            <joint name="wrist_pitch_2" value="0.0"/>
+            <joint name="shoulder_yaw_2" value="0.0"/>
+            <joint name="shoulder_pitch_2" value="-1.70"/>
+            <joint name="elbow_pitch_2" value="2.50"/>
+            <joint name="wrist_pitch_2" value="-0.75"/>
             <joint name="wrist_yaw_2" value="0.0"/>
         </xacro:if>

File: kyon_urdf/urdf/parts/foot_leg.urdf.xacro (robot description, xacro)
@@ -3,5 +3,5 @@
 <!-- macro legs -->
 <xacro:macro name="foot_leg" params="leg_num parent origin_x origin_y mirror">
-<link name="knee_pitch_${leg_num}">
+<link name="knee_pitch_${leg_num}_link">
     <inertial>
         <origin xyz="0.0 0.0 0.0"/>
@@ -25,9 +25,15 @@
 <joint name="knee_pitch_${leg_num}" type="revolute">
     <parent link="${parent}"/>
-    <child link="knee_pitch_${leg_num}"/>
+    <child link="knee_pitch_${leg_num}_link"/>
     <origin xyz="${KneePitch_Ox} ${KneePitch_Oy} ${KneePitch_Oz}" rpy="${KneePitch_roll} ${KneePitch_pitch} ${KneePitch_yaw}"/>
     <axis xyz="0 0 1"/>
     <limit lower="${knee_pitch_lower[leg_num-1]}" upper="${knee_pitch_upper[leg_num-1]}" effort="${motor_effort}" velocity="${motor_velocity}"/>
 </joint>
+<link name="contact_${leg_num}"/>
+<joint name="contact_${leg_num}_joint" type="fixed">
+    <parent link="knee_pitch_${leg_num}_link"/>
+    <child link="contact_${leg_num}"/>
+    <origin xyz="${-mirror*0.03} -0.35 0.03" rpy="${1.57*mirror} ${0} ${0.785 if mirror == -1 else 2.356}"/>
+</joint>
 </xacro:macro>
 </robot>

File: kyon_urdf/urdf/parts/kyon_arm.urdf.xacro (robot description, xacro)
@@ -6,5 +6,5 @@
 <!-- LINKS -->
 <!-- shoulder yaw -->
-<link name="shoulder_yaw_${arm_num}">
+<link name="shoulder_yaw_${arm_num}_link">
 	<inertial>
 		<origin xyz="0.0 0.0 0.0"/>
@@ -26,5 +26,5 @@
 	</collision>
 </link>
-<link name="shoulder_pitch_${arm_num}">
+<link name="shoulder_pitch_${arm_num}_link">
 	<inertial>
 		<origin xyz="0.0 0.0 0.0"/>
@@ -44,5 +44,5 @@
 	</collision>
 </link>
-<link name="elbow_pitch_${arm_num}">
+<link name="elbow_pitch_${arm_num}_link">
 	<inertial>
 		<origin xyz="${upper_arm1_length / 2} 0.0 0.0"/>
@@ -61,5 +61,5 @@
 	</collision>
 </link>
-<link name="wrist_pitch_${arm_num}">
+<link name="wrist_pitch_${arm_num}_link">
 	<inertial>
 		<origin xyz="0.0 0.0 0.0"/>
@@ -81,5 +81,5 @@
 	</collision>
 </link>
-<link name="wrist_yaw_${arm_num}">
+<link name="wrist_yaw_${arm_num}_link">
 	<inertial>
 		<origin xyz="0.0 0.0 0.0"/>
@@ -106,5 +106,5 @@
 <joint name="shoulder_yaw_${arm_num}" type="revolute">
 	<parent link="${parent}"/>
-	<child link="shoulder_yaw_${arm_num}"/>
+	<child link="shoulder_yaw_${arm_num}_link"/>
 	<origin xyz="${ShoulderYaw_Ox} ${rot * ShoulderYaw_Oy} ${ShoulderYaw_Oz}" rpy="${-rot * ShoulderYaw_roll} ${ShoulderYaw_pitch} ${ShoulderYaw_yaw}"/>
 	<axis xyz="0 0 1"/>
@@ -113,6 +113,6 @@
 <!-- arm pitch 1 -->
 <joint name="shoulder_pitch_${arm_num}" type="revolute">
-	<parent link="shoulder_yaw_${arm_num}"/>
-	<child link="shoulder_pitch_${arm_num}"/>
+	<parent link="shoulder_yaw_${arm_num}_link"/>
+	<child link="shoulder_pitch_${arm_num}_link"/>
 	<origin xyz="${ShoulderPitch_Ox} ${ShoulderPitch_Oy} ${ShoulderPitch_Oz}" rpy="${ShoulderPitch_roll} ${ShoulderPitch_pitch} ${ShoulderPitch_yaw  + rot * PI_2}"/>
 	<axis xyz="0 1 0"/>
@@ -120,6 +120,6 @@
 </joint>
 <joint name="elbow_pitch_${arm_num}" type="revolute">
-	<parent link="shoulder_pitch_${arm_num}"/>
-	<child link="elbow_pitch_${arm_num}"/>
+	<parent link="shoulder_pitch_${arm_num}_link"/>
+	<child link="elbow_pitch_${arm_num}_link"/>
 	<origin xyz="${ElbowPitch_Ox} ${ElbowPitch_Oy} ${ElbowPitch_Oz}" rpy="${ElbowPitch_roll} ${ElbowPitch_pitch} ${ElbowPitch_yaw}"/>
 	<axis xyz="0 0 1"/>
@@ -127,6 +127,6 @@
 </joint>
 <joint name="wrist_pitch_${arm_num}" type="revolute">
-	<parent link="elbow_pitch_${arm_num}"/>
-	<child link="wrist_pitch_${arm_num}"/>
+	<parent link="elbow_pitch_${arm_num}_link"/>
+	<child link="wrist_pitch_${arm_num}_link"/>
 	<origin xyz="${WristPitch_Ox} ${WristPitch_Oy} ${WristPitch_Oz}" rpy="${WristPitch_roll} ${WristPitch_pitch} ${WristPitch_yaw}"/>
 	<axis xyz="0 0 1"/>
@@ -134,6 +134,6 @@
 </joint>
 <joint name="wrist_yaw_${arm_num}" type="revolute">
-	<parent link="wrist_pitch_${arm_num}"/>
-	<child link="wrist_yaw_${arm_num}"/>
+	<parent link="wrist_pitch_${arm_num}_link"/>
+	<child link="wrist_yaw_${arm_num}_link"/>
 	<origin xyz="${WristYaw_Ox} ${WristYaw_Oy} ${WristYaw_Oz}" rpy="${WristYaw_roll} ${WristYaw_pitch} ${WristYaw_yaw}"/>
 	<axis xyz="0 0 1"/>
@@ -141,5 +141,5 @@
 </joint>
 <xacro:if value="${ADD_DAGANA}">
-	<xacro:kyon_dagana arm_num="${arm_num}" parent="wrist_yaw_${arm_num}"/>
+	<xacro:kyon_dagana arm_num="${arm_num}" parent="wrist_yaw_${arm_num}_link"/>
 </xacro:if>
 </xacro:macro>

File: kyon_urdf/urdf/parts/kyon_dagana.urdf.xacro (robot description, xacro)
@@ -3,5 +3,5 @@
 <!-- macro legs -->
 <xacro:macro name="kyon_dagana" params="arm_num parent">
-<link name="dagana${arm_num}_base">
+<link name="dagana_${arm_num}_base">
     <inertial>
         <origin xyz="0.0 0.0 0.0"/>
@@ -23,5 +23,5 @@
     </collision>
 </link>
-<link name="dagana${arm_num}_clamp">
+<link name="dagana_${arm_num}_clamp">
     <inertial>
         <origin xyz="0.0 0.0 0.0"/>
@@ -43,12 +43,12 @@
     </collision>
 </link>
-<joint name="dagana${arm_num}_base_joint" type="fixed">
+<joint name="dagana_${arm_num}_base_joint" type="fixed">
     <parent link="${parent}"/>
-    <child link="dagana${arm_num}_base"/>
+    <child link="dagana_${arm_num}_base"/>
     <origin xyz="${DaganaBase_Ox} ${DaganaBase_Oy} ${DaganaBase_Oz}" rpy="${DaganaBase_roll} ${DaganaBase_pitch} ${DaganaBase_yaw}"/>
 </joint>
-<joint name="dagana${arm_num}_clamp_joint" type="revolute">
-    <parent link="dagana${arm_num}_base"/>
-    <child link="dagana${arm_num}_clamp"/>
+<joint name="dagana_${arm_num}_clamp_joint" type="revolute">
+    <parent link="dagana_${arm_num}_base"/>
+    <child link="dagana_${arm_num}_clamp"/>
     <origin xyz="${DaganaClamp_Ox} ${DaganaClamp_Oy} ${DaganaClamp_Oz}" rpy="${DaganaClamp_roll} ${DaganaClamp_pitch} ${DaganaClamp_yaw}"/>
     <axis xyz="0 0 1"/>

File: kyon_urdf/urdf/parts/kyon_leg.urdf.xacro (robot description, xacro)
@@ -8,5 +8,5 @@
 <xacro:macro name="kyon_leg" params="leg_num origin_x origin_y mirror">
 <!-- links -->
-<link name="hip_roll_${leg_num}">
+<link name="hip_roll_${leg_num}_link">
 	<inertial>
 		<origin xyz="0.0 0.0 0.0"/>
@@ -30,5 +30,5 @@
 	</collision>
 </link>
-<link name="hip_pitch_${leg_num}">
+<link name="hip_pitch_${leg_num}_link">
 	<inertial>
 		<origin xyz="0.0 0.0 0.0"/>
@@ -53,5 +53,5 @@
 <joint name="hip_roll_${leg_num}" type="revolute">
 	<parent link="pelvis"/>
-	<child link="hip_roll_${leg_num}"/>
+	<child link="hip_roll_${leg_num}_link"/>
 	<origin xyz="${origin_x * HipRoll_Ox} ${origin_y * HipRoll_Oy} ${HipRoll_Oz}" rpy="${HipRoll_roll} ${origin_x*HipRoll_pitch} ${HipRoll_yaw}"/>
 	<axis xyz="0 0 1"/>
@@ -59,6 +59,6 @@
 </joint>
 <joint name="hip_pitch_${leg_num}" type="revolute">
-	<parent link="hip_roll_${leg_num}"/>
-	<child link="hip_pitch_${leg_num}"/>
+	<parent link="hip_roll_${leg_num}_link"/>
+	<child link="hip_pitch_${leg_num}_link"/>
 	<origin xyz="${origin_x * HipPitch_Ox} ${origin_y * HipPitch_Oy} ${HipPitch_Oz}" rpy="${origin_y*HipPitch_roll} ${origin_x*origin_y*HipPitch_pitch} ${HipPitch_yaw}"/>
 	<axis xyz="0 0 1"/>
@@ -66,11 +66,11 @@
 </joint>
 <xacro:if value="${ADD_FEET}">
-	<xacro:foot_leg leg_num="${leg_num}" parent="hip_pitch_${leg_num}" origin_x="${origin_x}" origin_y="${origin_y}" mirror="${mirror}"/>
+	<xacro:foot_leg leg_num="${leg_num}" parent="hip_pitch_${leg_num}_link" origin_x="${origin_x}" origin_y="${origin_y}" mirror="${mirror}"/>
 </xacro:if>
 <xacro:if value="${ADD_STEERING_WHEELS}">
-	<xacro:steering_wheel leg_num="${leg_num}" parent="hip_pitch_${leg_num}" origin_x="${origin_x}" origin_y="${origin_y}" mirror="${mirror}"/>
+	<xacro:steering_wheel leg_num="${leg_num}" parent="hip_pitch_${leg_num}_link" origin_x="${origin_x}" origin_y="${origin_y}" mirror="${mirror}"/>
 </xacro:if>
 <xacro:if value="${ADD_WHEELS}">
-	<xacro:wheel_leg leg_num="${leg_num}" parent="hip_pitch_${leg_num}" origin_x="${origin_x}" origin_y="${origin_y}" mirror="${mirror}"/>
+	<xacro:wheel_leg leg_num="${leg_num}" parent="hip_pitch_${leg_num}_link" origin_x="${origin_x}" origin_y="${origin_y}" mirror="${mirror}"/>
 </xacro:if>
 </xacro:macro>

File: kyon_urdf/urdf/parts/limits.urdf.xacro (robot description, xacro)
@@ -11,6 +11,6 @@
 <xacro:property name="j_shoulder_yaw_lower" value="${[-3.312, -3.3458]}"/>
 <xacro:property name="j_shoulder_yaw_upper" value="${[3.312, 3.3458]}"/>
-<xacro:property name="j_pitch_1_lower" value="${[-2.4056, -2.3266, -2.4696, -2.3426]}"/>
-<xacro:property name="j_pitch_1_upper" value="${[2.4056, 2.3266, 2.4696, 2.3426]}"/>
+<xacro:property name="j_pitch_1_lower" value="${[-3, -3]}"/>
+<xacro:property name="j_pitch_1_upper" value="${[3, 3]}"/>
 <xacro:property name="j_pitch_2_lower" value="${[-2.4056, -2.3266, -2.4696, -2.3426]}"/>
 <xacro:property name="j_pitch_2_upper" value="${[2.4056, 2.3266, 2.4696, 2.3426]}"/>

File: kyon_urdf/urdf/parts/steering_wheel.urdf.xacro (robot description, xacro)
@@ -3,5 +3,5 @@
 <!-- macro legs -->
 <xacro:macro name="steering_wheel" params="leg_num parent origin_x origin_y mirror">
-<link name="knee_pitch_${leg_num}">
+<link name="knee_pitch_${leg_num}_link">
     <inertial>
 		<origin xyz="0.0 0.0 0.0"/>
@@ -25,5 +25,5 @@
 	</collision>
 </link>
-<link name="ankle_yaw_${leg_num}">
+<link name="ankle_yaw_${leg_num}_link">
     <inertial>
 		<origin xyz="0.0 0.0 0.0"/>
@@ -47,5 +47,5 @@
 	</collision>
 </link>
-<link name="wheel_${leg_num}">
+<link name="wheel_${leg_num}_link">
     <inertial>
 		<origin xyz="0.0 0.0 0.0"/>
@@ -71,5 +71,5 @@
 <joint name="knee_pitch_${leg_num}" type="revolute">
     <parent link="${parent}"/>
-    <child link="knee_pitch_${leg_num}"/>
+    <child link="knee_pitch_${leg_num}_link"/>
     <origin xyz="${KneePitch_Ox} ${KneePitch_Oy} ${KneePitch_Oz}" rpy="${KneePitch_roll} ${KneePitch_pitch} ${KneePitch_yaw}"/>
     <axis xyz="0 0 1"/>
@@ -77,6 +77,6 @@
 </joint>
 <joint name="ankle_yaw_${leg_num}" type="revolute">
-    <parent link="knee_pitch_${leg_num}"/>
-    <child link="ankle_yaw_${leg_num}"/>
+    <parent link="knee_pitch_${leg_num}_link"/>
+    <child link="ankle_yaw_${leg_num}_link"/>
     <origin xyz="${AnkleYaw_Ox} ${AnkleYaw_Oy} ${AnkleYaw_Oz}" rpy="${AnkleYaw_roll} ${AnkleYaw_pitch} ${AnkleYaw_yaw}"/>
     <axis xyz="0 0 1"/>
@@ -84,6 +84,6 @@
 </joint>
 <joint name="wheel_joint_${leg_num}" type="revolute">
-    <parent link="ankle_yaw_${leg_num}"/>
-    <child link="wheel_${leg_num}"/>
+    <parent link="ankle_yaw_${leg_num}_link"/>
+    <child link="wheel_${leg_num}_link"/>
     <origin xyz="${SteeringWheel_Ox} ${SteeringWheel_Oy} ${SteeringWheel_Oz}" rpy="${SteeringWheel_roll} ${SteeringWheel_pitch} ${SteeringWheel_yaw}"/>
     <axis xyz="0 0 1"/>

File: kyon_urdf/urdf/parts/wheel_leg.urdf.xacro (robot description, xacro)
@@ -3,5 +3,5 @@
 <!-- macro legs -->
 <xacro:macro name="wheel_leg" params="leg_num parent origin_x origin_y mirror">
-<link name="knee_pitch_${leg_num}">
+<link name="knee_pitch_${leg_num}_link">
     <inertial>
         <origin xyz="0.0 0.0 0.0"/>
@@ -23,5 +23,5 @@
     </collision>
 </link>
-<link name="wheel_${leg_num}">
+<link name="wheel_${leg_num}_link">
     <inertial>
 		<origin xyz="0.0 0.0 0.0"/>
@@ -47,5 +47,5 @@
 <joint name="knee_pitch_${leg_num}" type="revolute">
     <parent link="${parent}"/>
-    <child link="knee_pitch_${leg_num}"/>
+    <child link="knee_pitch_${leg_num}_link"/>
     <origin xyz="${KneePitch_Ox} ${KneePitch_Oy} ${KneePitch_Oz}" rpy="${KneePitch_roll} ${KneePitch_pitch} ${KneePitch_yaw}"/>
     <axis xyz="0 0 1"/>
@@ -54,5 +54,5 @@
 <joint name="wheel_joint_${leg_num}" type="revolute">
     <parent link="knee_pitch_${leg_num}"/>
-    <child link="wheel_${leg_num}"/>
+    <child link="wheel_${leg_num}_link"/>
     <origin xyz="${Wheel_Ox} ${Wheel_Oy} ${Wheel_Oz}" rpy="${Wheel_roll} ${Wheel_pitch} ${Wheel_yaw}"/>
     <axis xyz="0 0 1"/>

Commit message: few fix and changed colors in gazebo

File: kyon_srdf/srdf/kyon.srdf.xacro (robot description, xacro)
@@ -44,8 +44,8 @@
     	<xacro:if value="${ADD_DAGANA}">
 			<group name="left_arm">
-				<chain base_link="pelvis" tip_link="dagana_1_clamp"/>
+				<chain base_link="pelvis" tip_link="dagana_1_claw"/>
 			</group>
 			<group name="right_arm">
-				<chain base_link="pelvis" tip_link="dagana_2_clamp"/>
+				<chain base_link="pelvis" tip_link="dagana_2_claw"/>
 			</group>
             <!-- <group name="left_hand">

File: kyon_urdf/urdf/gazebo/kyon.gazebo.xacro (robot description, xacro)
@@ -50,5 +50,5 @@
             <provideFeedback>true</provideFeedback>
         </gazebo>
-        <gazebo reference="ball_1">
+        <gazebo reference="knee_pitch_1_link">
         	<kp>1000000.0</kp>
 			<kd>100.0</kd>
@@ -58,5 +58,5 @@
 			<maxContacts>1</maxContacts>
 		</gazebo>
-		<gazebo reference="ball_2">
+		<gazebo reference="knee_pitch_2_link">
         	<kp>1000000.0</kp>
 			<kd>100.0</kd>
@@ -66,5 +66,5 @@
 			<maxContacts>1</maxContacts>
 		</gazebo>
-		<gazebo reference="ball_3">
+		<gazebo reference="knee_pitch_3_link">
         	<kp>1000000.0</kp>
 			<kd>100.0</kd>
@@ -74,5 +74,5 @@
 			<maxContacts>1</maxContacts>
 		</gazebo>
-		<gazebo reference="ball_4">
+		<gazebo reference="knee_pitch_4_link">
         	<kp>1000000.0</kp>
 			<kd>100.0</kd>

File: kyon_urdf/urdf/gazebo/materials.gazebo.xacro (robot description, xacro)
@@ -2,42 +2,36 @@
 <robot xmlns:xacro="http://ros.org/wiki/xacro">
 <xacro:macro name="kyon_leg_materials" params="leg_num">
-<gazebo reference="hip_roll_${leg_num}">
-	<material>Gazebo/LightBlueLaser</material>
-</gazebo>
-<gazebo reference="hip_pitch_stator_${leg_num}">
-	<material>Gazebo/BlackTransparent</material>
-</gazebo>
-<gazebo reference="hip_pitch_${leg_num}">
-	<material>Gazebo/LightBlueLaser</material>
-</gazebo>
-<gazebo reference="knee_pitch_stator_${leg_num}">
-	<material>Gazebo/LightBlueLaser</material>
-</gazebo>
-<gazebo reference="knee_pitch_${leg_num}">
-	<material>Gazebo/LightBlueLaser</material>
-</gazebo>
-<gazebo reference="ball_joint_${leg_num}">
-	<material>Gazebo/BlackTransparent</material>
-</gazebo>
+	<gazebo reference="hip_roll_${leg_num}_link">
+		<material>Gazebo/Grey</material>
+	</gazebo>
+	<gazebo reference="hip_pitch_${leg_num}_link">
+		<material>Gazebo/SkyBlue</material>
+	</gazebo>
+	<gazebo reference="knee_pitch_${leg_num}_link">
+		<material>Gazebo/Grey</material>
+	</gazebo>
 </xacro:macro>
 <xacro:macro name="kyon_arm_materials" params="arm_num">
-<gazebo reference="shoulder_yaw_${arm_num}">
-	<material>Gazebo/BlackTransparent</material>
-</gazebo>
-<gazebo reference="shoulder_pitch_stator_${arm_num}">
-	<material>Gazebo/LightBlueLaser</material>
-</gazebo>
-<gazebo reference="shoulder_pitch_${arm_num}">
-	<material>Gazebo/LightBlueLaser</material>
-</gazebo>
-<gazebo reference="elbow_pitch_stator_${arm_num}">
-	<material>Gazebo/LightBlueLaser</material>
-</gazebo>
-<gazebo reference="elbow_pitch_${arm_num}">
-	<material>Gazebo/BlackTransparent</material>
-</gazebo>
-<gazebo reference="hand_joint_${arm_num}">
-	<material>Gazebo/LightBlueLaser</material>
-</gazebo>
+	<gazebo reference="shoulder_yaw_${arm_num}_link">
+		<material>Gazebo/Grey</material>
+	</gazebo>
+	<gazebo reference="shoulder_pitch_${arm_num}_link">
+		<material>Gazebo/SkyBlue</material>
+	</gazebo>
+	<gazebo reference="elbow_pitch_${arm_num}_link">
+		<material>Gazebo/Grey</material>
+	</gazebo>
+	<gazebo reference="wrist_pitch_${arm_num}_link">
+		<material>Gazebo/SkyBlue</material>
+	</gazebo>
+	<gazebo reference="wrist_yaw_${arm_num}_link">
+		<material>Gazebo/SkyBlue</material>
+	</gazebo>
+	<gazebo reference="dagana_${arm_num}_base">
+		<material>Gazebo/Grey</material>
+	</gazebo>
+	<gazebo reference="dagana_${arm_num}_claw">
+		<material>Gazebo/Grey</material>
+	</gazebo>
 </xacro:macro>
 <gazebo reference="pelvis">
@@ -45,18 +39,12 @@
 </gazebo>
 <xacro:if value="${ADD_LEGS}">
-<xacro:kyon_leg_materials leg_num="1"/>
-<xacro:kyon_leg_materials leg_num="2"/>
-<xacro:kyon_leg_materials leg_num="3"/>
-<xacro:kyon_leg_materials leg_num="4"/>
+	<xacro:kyon_leg_materials leg_num="1"/>
+	<xacro:kyon_leg_materials leg_num="2"/>
+	<xacro:kyon_leg_materials leg_num="3"/>
+	<xacro:kyon_leg_materials leg_num="4"/>
 </xacro:if>
 <xacro:if value="${ADD_UPPER_BODY}">
-<xacro:kyon_arm_materials arm_num="1"/>
-<xacro:kyon_arm_materials arm_num="2"/>
-<gazebo reference="ball_arm_1">
-	<material>Gazebo/BlackTransparent</material>
-</gazebo>
-<gazebo reference="ball_arm_2">
-	<material>Gazebo/BlackTransparent</material>
-</gazebo>
+	<xacro:kyon_arm_materials arm_num="1"/>
+	<xacro:kyon_arm_materials arm_num="2"/>
 </xacro:if>
 <xacro:if value="${ADD_WHEELS}"/>

File: kyon_urdf/urdf/parts/kyon_arm.urdf.xacro (robot description, xacro)
@@ -116,5 +116,5 @@
 	<child link="shoulder_pitch_${arm_num}_link"/>
 	<origin xyz="${ShoulderPitch_Ox} ${ShoulderPitch_Oy} ${ShoulderPitch_Oz}" rpy="${ShoulderPitch_roll} ${ShoulderPitch_pitch} ${ShoulderPitch_yaw + rot * PI_2}"/>
-	<axis xyz="0 1 0"/>
+	<axis xyz="0 0 1"/>
 	<limit lower="${j_pitch_1_lower[arm_num-1]}" upper="${j_pitch_1_upper[arm_num-1]}" effort="${motor_effort}" velocity="${motor_velocity}"/>
 </joint>

File: kyon_urdf/urdf/parts/wheel_leg.urdf.xacro (robot description, xacro)
@@ -25,7 +25,7 @@
 <link name="wheel_${leg_num}_link">
     <inertial>
-		<origin xyz="0.0 0.0 0.0"/>
-		<mass value="${motorA_mass}"/>
-		<inertia ixx="${MotorA_xx}" ixy="${mirror*MotorA_xy}" ixz="${MotorA_xz}" iyy="${MotorA_yy}" iyz="${mirror*MotorA_yz}" izz="${MotorA_zz}"/>
+		<origin xyz="${Wheel_x} ${Wheel_y} ${Wheel_z}"/>
+		<mass value="${Wheel_mass}"/>
+		<inertia ixx="${Wheel_xx}" ixy="${Wheel_xy}" ixz="${Wheel_xz}" iyy="${Wheel_yy}" iyz="${Wheel_yz}" izz="${Wheel_zz}"/>
 	</inertial>
 	<visual>
