Commit message: fix srdf and excluded collisions and imu joint name

File: kyon_srdf/srdf/kyon.srdf.xacro (robot description, xacro)
@@ -110,3 +110,92 @@
         </xacro:if>
     </group_state>
+    <!--DISABLE COLLISIONS: By default it is assumed that any link of the robot could potentially come into collision with any other link in the robot. This tag disables collision checking between a specified pair of links. -->
+    <disable_collisions link1="dagana_1_base" link2="dagana_1_clamp" reason="Adjacent"/>
+    <disable_collisions link1="dagana_1_base" link2="elbow_pitch_1_link" reason="Never"/>
+    <disable_collisions link1="dagana_1_base" link2="wrist_pitch_1_link" reason="Never"/>
+    <disable_collisions link1="dagana_1_base" link2="wrist_yaw_1_link" reason="Adjacent"/>
+    <disable_collisions link1="dagana_2_base" link2="dagana_2_clamp" reason="Adjacent"/>
+    <disable_collisions link1="dagana_2_base" link2="elbow_pitch_2_link" reason="Never"/>
+    <disable_collisions link1="dagana_2_base" link2="wrist_pitch_2_link" reason="Never"/>
+    <disable_collisions link1="dagana_2_base" link2="wrist_yaw_2_link" reason="Adjacent"/>
+    <disable_collisions link1="elbow_pitch_1_link" link2="hip_roll_4_link" reason="Never"/>
+    <disable_collisions link1="elbow_pitch_1_link" link2="shoulder_pitch_1_link" reason="Adjacent"/>
+    <disable_collisions link1="elbow_pitch_1_link" link2="wrist_pitch_1_link" reason="Adjacent"/>
+    <disable_collisions link1="elbow_pitch_2_link" link2="hip_roll_3_link" reason="Never"/>
+    <disable_collisions link1="elbow_pitch_2_link" link2="shoulder_pitch_2_link" reason="Adjacent"/>
+    <disable_collisions link1="elbow_pitch_2_link" link2="wrist_pitch_2_link" reason="Adjacent"/>
+    <disable_collisions link1="elbow_pitch_2_link" link2="wrist_yaw_2_link" reason="Never"/>
+    <disable_collisions link1="hip_pitch_1_link" link2="hip_pitch_3_link" reason="Never"/>
+    <disable_collisions link1="hip_pitch_1_link" link2="hip_pitch_4_link" reason="Never"/>
+    <disable_collisions link1="hip_pitch_1_link" link2="hip_roll_1_link" reason="Adjacent"/>
+    <disable_collisions link1="hip_pitch_1_link" link2="hip_roll_3_link" reason="Never"/>
+    <disable_collisions link1="hip_pitch_1_link" link2="hip_roll_4_link" reason="Never"/>
+    <disable_collisions link1="hip_pitch_1_link" link2="knee_pitch_1_link" reason="Adjacent"/>
+    <disable_collisions link1="hip_pitch_1_link" link2="pelvis" reason="Default"/>
+    <disable_collisions link1="hip_pitch_2_link" link2="hip_pitch_3_link" reason="Never"/>
+    <disable_collisions link1="hip_pitch_2_link" link2="hip_pitch_4_link" reason="Never"/>
+    <disable_collisions link1="hip_pitch_2_link" link2="hip_roll_2_link" reason="Adjacent"/>
+    <disable_collisions link1="hip_pitch_2_link" link2="hip_roll_3_link" reason="Never"/>
+    <disable_collisions link1="hip_pitch_2_link" link2="hip_roll_4_link" reason="Never"/>
+    <disable_collisions link1="hip_pitch_2_link" link2="knee_pitch_2_link" reason="Adjacent"/>
+    <disable_collisions link1="hip_pitch_2_link" link2="pelvis" reason="Default"/>
+    <disable_collisions link1="hip_pitch_3_link" link2="hip_roll_1_link" reason="Never"/>
+    <disable_collisions link1="hip_pitch_3_link" link2="hip_roll_2_link" reason="Never"/>
+    <disable_collisions link1="hip_pitch_3_link" link2="hip_roll_3_link" reason="Adjacent"/>
+    <disable_collisions link1="hip_pitch_3_link" link2="knee_pitch_3_link" reason="Adjacent"/>
+    <disable_collisions link1="hip_pitch_3_link" link2="pelvis" reason="Default"/>
+    <disable_collisions link1="hip_pitch_3_link" link2="shoulder_yaw_1_link" reason="Never"/>
+    <disable_collisions link1="hip_pitch_3_link" link2="shoulder_yaw_2_link" reason="Never"/>
+    <disable_collisions link1="hip_pitch_4_link" link2="hip_roll_1_link" reason="Never"/>
+    <disable_collisions link1="hip_pitch_4_link" link2="hip_roll_2_link" reason="Never"/>
+    <disable_collisions link1="hip_pitch_4_link" link2="hip_roll_4_link" reason="Adjacent"/>
+    <disable_collisions link1="hip_pitch_4_link" link2="knee_pitch_4_link" reason="Adjacent"/>
+    <disable_collisions link1="hip_pitch_4_link" link2="pelvis" reason="Default"/>
+    <disable_collisions link1="hip_pitch_4_link" link2="shoulder_yaw_1_link" reason="Never"/>
+    <disable_collisions link1="hip_pitch_4_link" link2="shoulder_yaw_2_link" reason="Never"/>
+    <disable_collisions link1="hip_roll_1_link" link2="hip_roll_2_link" reason="Never"/>
+    <disable_collisions link1="hip_roll_1_link" link2="hip_roll_3_link" reason="Never"/>
+    <disable_collisions link1="hip_roll_1_link" link2="hip_roll_4_link" reason="Never"/>
+    <disable_collisions link1="hip_roll_1_link" link2="knee_pitch_1_link" reason="Never"/>
+    <disable_collisions link1="hip_roll_1_link" link2="knee_pitch_2_link" reason="Never"/>
+    <disable_collisions link1="hip_roll_1_link" link2="knee_pitch_3_link" reason="Never"/>
+    <disable_collisions link1="hip_roll_1_link" link2="knee_pitch_4_link" reason="Never"/>
+    <disable_collisions link1="hip_roll_1_link" link2="pelvis" reason="Adjacent"/>
+    <disable_collisions link1="hip_roll_1_link" link2="shoulder_yaw_1_link" reason="Never"/>
+    <disable_collisions link1="hip_roll_1_link" link2="shoulder_yaw_2_link" reason="Never"/>
+    <disable_collisions link1="hip_roll_2_link" link2="hip_roll_3_link" reason="Never"/>
+    <disable_collisions link1="hip_roll_2_link" link2="hip_roll_4_link" reason="Never"/>
+    <disable_collisions link1="hip_roll_2_link" link2="knee_pitch_1_link" reason="Never"/>
+    <disable_collisions link1="hip_roll_2_link" link2="knee_pitch_2_link" reason="Never"/>
+    <disable_collisions link1="hip_roll_2_link" link2="knee_pitch_3_link" reason="Never"/>
+    <disable_collisions link1="hip_roll_2_link" link2="knee_pitch_4_link" reason="Never"/>
+    <disable_collisions link1="hip_roll_2_link" link2="pelvis" reason="Adjacent"/>
+    <disable_collisions link1="hip_roll_2_link" link2="shoulder_yaw_1_link" reason="Never"/>
+    <disable_collisions link1="hip_roll_2_link" link2="shoulder_yaw_2_link" reason="Never"/>
+    <disable_collisions link1="hip_roll_3_link" link2="hip_roll_4_link" reason="Never"/>
+    <disable_collisions link1="hip_roll_3_link" link2="knee_pitch_1_link" reason="Never"/>
+    <disable_collisions link1="hip_roll_3_link" link2="knee_pitch_2_link" reason="Never"/>
+    <disable_collisions link1="hip_roll_3_link" link2="knee_pitch_3_link" reason="Never"/>
+    <disable_collisions link1="hip_roll_3_link" link2="knee_pitch_4_link" reason="Never"/>
+    <disable_collisions link1="hip_roll_3_link" link2="pelvis" reason="Adjacent"/>
+    <disable_collisions link1="hip_roll_3_link" link2="shoulder_pitch_1_link" reason="Never"/>
+    <disable_collisions link1="hip_roll_3_link" link2="shoulder_pitch_2_link" reason="Never"/>
+    <disable_collisions link1="hip_roll_3_link" link2="shoulder_yaw_1_link" reason="Never"/>
+    <disable_collisions link1="hip_roll_3_link" link2="shoulder_yaw_2_link" reason="Never"/>
+    <disable_collisions link1="hip_roll_4_link" link2="knee_pitch_1_link" reason="Never"/>
+    <disable_collisions link1="hip_roll_4_link" link2="knee_pitch_2_link" reason="Never"/>
+    <disable_collisions link1="hip_roll_4_link" link2="knee_pitch_3_link" reason="Never"/>
+    <disable_collisions link1="hip_roll_4_link" link2="knee_pitch_4_link" reason="Never"/>
+    <disable_collisions link1="hip_roll_4_link" link2="pelvis" reason="Adjacent"/>
+    <disable_collisions link1="hip_roll_4_link" link2="shoulder_pitch_1_link" reason="Never"/>
+    <disable_collisions link1="hip_roll_4_link" link2="shoulder_pitch_2_link" reason="Never"/>
+    <disable_collisions link1="hip_roll_4_link" link2="shoulder_yaw_1_link" reason="Never"/>
+    <disable_collisions link1="hip_roll_4_link" link2="shoulder_yaw_2_link" reason="Never"/>
+    <disable_collisions link1="pelvis" link2="shoulder_yaw_1_link" reason="Adjacent"/>
+    <disable_collisions link1="pelvis" link2="shoulder_yaw_2_link" reason="Adjacent"/>
+    <disable_collisions link1="shoulder_pitch_1_link" link2="shoulder_yaw_1_link" reason="Adjacent"/>
+    <disable_collisions link1="shoulder_pitch_2_link" link2="shoulder_yaw_2_link" reason="Adjacent"/>
+    <disable_collisions link1="shoulder_yaw_1_link" link2="shoulder_yaw_2_link" reason="Never"/>
+    <disable_collisions link1="wrist_pitch_1_link" link2="wrist_yaw_1_link" reason="Adjacent"/>
+    <disable_collisions link1="wrist_pitch_2_link" link2="wrist_yaw_2_link" reason="Adjacent"/>
 </robot>

File: kyon_urdf/urdf/kyon.urdf (robot description, URDF)
Before this commit: robot kyon, 38 links, 37 joints
Links:
- removed link ankle_yaw_1
- removed link ankle_yaw_2
- removed link ankle_yaw_3
- removed link ankle_yaw_4
- removed link dagana1_base
- removed link dagana1_clamp
- removed link dagana2_base
- removed link dagana2_clamp
- removed link elbow_pitch_1
- removed link elbow_pitch_2
- removed link hip_pitch_1
- removed link hip_pitch_2
- removed link hip_pitch_3
- removed link hip_pitch_4
- removed link hip_roll_1
- removed link hip_roll_2
- removed link hip_roll_3
- removed link hip_roll_4
- removed link knee_pitch_1
- removed link knee_pitch_2
- removed link knee_pitch_3
- removed link knee_pitch_4
- removed link shoulder_pitch_1
- removed link shoulder_pitch_2
- removed link shoulder_yaw_1
- removed link shoulder_yaw_2
- removed link wheel_1
- removed link wheel_2
- removed link wheel_3
- removed link wheel_4
- removed link wrist_pitch_1
- removed link wrist_pitch_2
- removed link wrist_yaw_1
- removed link wrist_yaw_2
- added link contact_1
- added link contact_2
- added link contact_3
- added link contact_4
- added link dagana_1_base, mass 1.8; collision mesh filename=package://kyon_urdf/meshes/collision/mesh_dagana-base.stl scale=0.001 0.001 0.001; visual mesh filename=package://kyon_urdf/meshes/mesh_dagana-base.stl scale=0.001 0.001 0.001
- added link dagana_1_clamp, mass 1.8; collision mesh filename=package://kyon_urdf/meshes/collision/mesh_dagana-clamp.stl scale=0.001 0.001 0.001; visual mesh filename=package://kyon_urdf/meshes/mesh_dagana-clamp.stl scale=0.001 0.001 0.001
- added link dagana_2_base, mass 1.8; collision mesh filename=package://kyon_urdf/meshes/collision/mesh_dagana-base.stl scale=0.001 0.001 0.001; visual mesh filename=package://kyon_urdf/meshes/mesh_dagana-base.stl scale=0.001 0.001 0.001
- added link dagana_2_clamp, mass 1.8; collision mesh filename=package://kyon_urdf/meshes/collision/mesh_dagana-clamp.stl scale=0.001 0.001 0.001; visual mesh filename=package://kyon_urdf/meshes/mesh_dagana-clamp.stl scale=0.001 0.001 0.001
- added link elbow_pitch_1_link, mass 0.77; collision mesh filename=package://kyon_urdf/meshes/mesh_elbow.stl scale=0.001 0.001 0.001; visual mesh filename=package://kyon_urdf/meshes/mesh_elbow.stl scale=0.001 0.001 0.001
- added link elbow_pitch_2_link, mass 0.77; collision mesh filename=package://kyon_urdf/meshes/mesh_elbow.stl scale=0.001 0.001 0.001; visual mesh filename=package://kyon_urdf/meshes/mesh_elbow.stl scale=0.001 0.001 0.001
- added link hip_pitch_1_link, mass 1.8; collision mesh filename=package://kyon_urdf/meshes/collision/mesh_hip-pitch.stl scale=0.001 0.001 0.001; visual mesh filename=package://kyon_urdf/meshes/mesh_hip-pitch.stl scale=0.001 0.001 0.001
- added link hip_pitch_2_link, mass 1.8; collision mesh filename=package://kyon_urdf/meshes/collision/mesh_hip-pitch.stl scale=0.001 0.001 0.001; visual mesh filename=package://kyon_urdf/meshes/mesh_hip-pitch.stl scale=0.001 0.001 0.001
- added link hip_pitch_3_link, mass 1.8; collision mesh filename=package://kyon_urdf/meshes/collision/mesh_hip-pitch.stl scale=0.001 0.001 0.001; visual mesh filename=package://kyon_urdf/meshes/mesh_hip-pitch.stl scale=0.001 0.001 0.001
- added link hip_pitch_4_link, mass 1.8; collision mesh filename=package://kyon_urdf/meshes/collision/mesh_hip-pitch.stl scale=0.001 0.001 0.001; visual mesh filename=package://kyon_urdf/meshes/mesh_hip-pitch.stl scale=0.001 0.001 0.001
- added link hip_roll_1_link, mass 1.8; collision mesh filename=package://kyon_urdf/meshes/collision/mesh_hip-roll.stl scale=0.001 -0.001 0.001; visual mesh filename=package://kyon_urdf/meshes/mesh_hip-roll.stl scale=0.001 -0.001 0.001
- added link hip_roll_2_link, mass 1.8; collision mesh filename=package://kyon_urdf/meshes/collision/mesh_hip-roll.stl scale=0.001 0.001 0.001; visual mesh filename=package://kyon_urdf/meshes/mesh_hip-roll.stl scale=0.001 0.001 0.001
- added link hip_roll_3_link, mass 1.8; collision mesh filename=package://kyon_urdf/meshes/collision/mesh_hip-roll.stl scale=0.001 -0.001 0.001; visual mesh filename=package://kyon_urdf/meshes/mesh_hip-roll.stl scale=0.001 -0.001 0.001
- added link hip_roll_4_link, mass 1.8; collision mesh filename=package://kyon_urdf/meshes/collision/mesh_hip-roll.stl scale=0.001 0.001 0.001; visual mesh filename=package://kyon_urdf/meshes/mesh_hip-roll.stl scale=0.001 0.001 0.001
- added link knee_pitch_1_link, mass 1.8; collision mesh filename=package://kyon_urdf/meshes/collision/mesh_foot-leg.stl scale=-0.001 0.001 0.001; visual mesh filename=package://kyon_urdf/meshes/mesh_foot-leg.stl scale=-0.001 0.001 0.001
- added link knee_pitch_2_link, mass 1.8; collision mesh filename=package://kyon_urdf/meshes/collision/mesh_foot-leg.stl scale=0.001 0.001 0.001; visual mesh filename=package://kyon_urdf/meshes/mesh_foot-leg.stl scale=0.001 0.001 0.001
- added link knee_pitch_3_link, mass 1.8; collision mesh filename=package://kyon_urdf/meshes/collision/mesh_foot-leg.stl scale=-0.001 0.001 0.001; visual mesh filename=package://kyon_urdf/meshes/mesh_foot-leg.stl scale=-0.001 0.001 0.001
- added link knee_pitch_4_link, mass 1.8; collision mesh filename=package://kyon_urdf/meshes/collision/mesh_foot-leg.stl scale=0.001 0.001 0.001; visual mesh filename=package://kyon_urdf/meshes/mesh_foot-leg.stl scale=0.001 0.001 0.001
- added link shoulder_pitch_1_link, mass 1.8; collision mesh filename=package://kyon_urdf/meshes/collision/mesh_sh-pitch.stl scale=0.001 0.001 0.001; visual mesh filename=package://kyon_urdf/meshes/mesh_sh-pitch.stl scale=0.001 0.001 0.001
- added link shoulder_pitch_2_link, mass 1.8; collision mesh filename=package://kyon_urdf/meshes/collision/mesh_sh-pitch.stl scale=0.001 0.001 0.001; visual mesh filename=package://kyon_urdf/meshes/mesh_sh-pitch.stl scale=0.001 0.001 0.001
- added link shoulder_yaw_1_link, mass 1.6; collision mesh filename=package://kyon_urdf/meshes/collision/mesh_sh-yaw.stl scale=0.001 0.001 0.001; visual mesh filename=package://kyon_urdf/meshes/mesh_sh-yaw.stl scale=0.001 0.001 0.001
- added link shoulder_yaw_2_link, mass 1.6; collision mesh filename=package://kyon_urdf/meshes/collision/mesh_sh-yaw.stl scale=0.001 0.001 0.001; visual mesh filename=package://kyon_urdf/meshes/mesh_sh-yaw.stl scale=0.001 0.001 0.001
- added link wrist_pitch_1_link, mass 0.63; collision mesh filename=package://kyon_urdf/meshes/collision/mesh_wrist-pitch.stl scale=0.001 0.001 0.001; visual mesh filename=package://kyon_urdf/meshes/mesh_wrist-pitch.stl scale=0.001 0.001 0.001
- added link wrist_pitch_2_link, mass 0.63; collision mesh filename=package://kyon_urdf/meshes/collision/mesh_wrist-pitch.stl scale=0.001 0.001 0.001; visual mesh filename=package://kyon_urdf/meshes/mesh_wrist-pitch.stl scale=0.001 0.001 0.001
- added link wrist_yaw_1_link, mass 0.63; collision mesh filename=package://kyon_urdf/meshes/collision/mesh_wrist-yaw.stl scale=0.001 0.001 0.001; visual mesh filename=package://kyon_urdf/meshes/mesh_wrist-yaw.stl scale=0.001 0.001 0.001
- added link wrist_yaw_2_link, mass 0.63; collision mesh filename=package://kyon_urdf/meshes/collision/mesh_wrist-yaw.stl scale=0.001 0.001 0.001; visual mesh filename=package://kyon_urdf/meshes/mesh_wrist-yaw.stl scale=0.001 0.001 0.001
Joints:
- removed joint ankle_yaw_1
- removed joint ankle_yaw_2
- removed joint ankle_yaw_3
- removed joint ankle_yaw_4
- removed joint dagana1_base_joint
- removed joint dagana1_clamp_joint
- removed joint dagana2_base_joint
- removed joint dagana2_clamp_joint
- removed joint imu_link
- removed joint wheel_joint_1
- removed joint wheel_joint_2
- removed joint wheel_joint_3
- removed joint wheel_joint_4
- added joint contact_1_joint: type fixed, parent knee_pitch_1_link, child contact_1, origin xyz=0.03 -0.35 0.03 rpy=-1.57 0 0.785
- added joint contact_2_joint: type fixed, parent knee_pitch_2_link, child contact_2, origin xyz=-0.03 -0.35 0.03 rpy=1.57 0 2.356
- added joint contact_3_joint: type fixed, parent knee_pitch_3_link, child contact_3, origin xyz=0.03 -0.35 0.03 rpy=-1.57 0 0.785
- added joint contact_4_joint: type fixed, parent knee_pitch_4_link, child contact_4, origin xyz=-0.03 -0.35 0.03 rpy=1.57 0 2.356
- added joint dagana_1_base_joint: type fixed, parent wrist_yaw_1_link, child dagana_1_base, origin xyz=0.0 0.0 0.0 rpy=0.0 0.0 0.0
- added joint dagana_1_clamp_joint: type revolute, parent dagana_1_base, child dagana_1_clamp, origin xyz=0.0361625 0.016 0.044 rpy=0.0 1.57079632679 0.0, axis 0 0 1, limit lower=-3.4056 upper=3.4056 effort=132 velocity=15.5
- added joint dagana_2_base_joint: type fixed, parent wrist_yaw_2_link, child dagana_2_base, origin xyz=0.0 0.0 0.0 rpy=0.0 0.0 0.0
- added joint dagana_2_clamp_joint: type revolute, parent dagana_2_base, child dagana_2_clamp, origin xyz=0.0361625 0.016 0.044 rpy=0.0 1.57079632679 0.0, axis 0 0 1, limit lower=-3.3266 upper=3.3266 effort=132 velocity=15.5
- added joint imu_link_joint: type fixed, parent pelvis, child imu_link
- joint elbow_pitch_1: child elbow_pitch_1 -> elbow_pitch_1_link; limit lower=-2.4056 upper=2.4056 effort=132 velocity=15.5 -> lower=-3 upper=3 effort=132 velocity=15.5; parent shoulder_pitch_1 -> shoulder_pitch_1_link
- joint elbow_pitch_2: child elbow_pitch_2 -> elbow_pitch_2_link; limit lower=-2.3266 upper=2.3266 effort=132 velocity=15.5 -> lower=-3 upper=3 effort=132 velocity=15.5; parent shoulder_pitch_2 -> shoulder_pitch_2_link
- joint hip_pitch_1: child hip_pitch_1 -> hip_pitch_1_link; parent hip_roll_1 -> hip_roll_1_link
- joint hip_pitch_2: child hip_pitch_2 -> hip_pitch_2_link; parent hip_roll_2 -> hip_roll_2_link
- joint hip_pitch_3: child hip_pitch_3 -> hip_pitch_3_link; parent hip_roll_3 -> hip_roll_3_link
- joint hip_pitch_4: child hip_pitch_4 -> hip_pitch_4_link; parent hip_roll_4 -> hip_roll_4_link
- joint hip_roll_1: child hip_roll_1 -> hip_roll_1_link
- joint hip_roll_2: child hip_roll_2 -> hip_roll_2_link
- joint hip_roll_3: child hip_roll_3 -> hip_roll_3_link
- joint hip_roll_4: child hip_roll_4 -> hip_roll_4_link
- joint knee_pitch_1: child knee_pitch_1 -> knee_pitch_1_link; parent hip_pitch_1 -> hip_pitch_1_link
- joint knee_pitch_2: child knee_pitch_2 -> knee_pitch_2_link; parent hip_pitch_2 -> hip_pitch_2_link
- joint knee_pitch_3: child knee_pitch_3 -> knee_pitch_3_link; parent hip_pitch_3 -> hip_pitch_3_link
- joint knee_pitch_4: child knee_pitch_4 -> knee_pitch_4_link; parent hip_pitch_4 -> hip_pitch_4_link
- joint shoulder_pitch_1: child shoulder_pitch_1 -> shoulder_pitch_1_link; limit lower=-2.4056 upper=2.4056 effort=132 velocity=15.5 -> lower=-3 upper=3 effort=132 velocity=15.5; parent shoulder_yaw_1 -> shoulder_yaw_1_link
- joint shoulder_pitch_2: child shoulder_pitch_2 -> shoulder_pitch_2_link; limit lower=-2.3266 upper=2.3266 effort=132 velocity=15.5 -> lower=-3 upper=3 effort=132 velocity=15.5; parent shoulder_yaw_2 -> shoulder_yaw_2_link
- joint shoulder_yaw_1: child shoulder_yaw_1 -> shoulder_yaw_1_link
- joint shoulder_yaw_2: child shoulder_yaw_2 -> shoulder_yaw_2_link
- joint wrist_pitch_1: child wrist_pitch_1 -> wrist_pitch_1_link; parent elbow_pitch_1 -> elbow_pitch_1_link
- joint wrist_pitch_2: child wrist_pitch_2 -> wrist_pitch_2_link; parent elbow_pitch_2 -> elbow_pitch_2_link
- joint wrist_yaw_1: child wrist_yaw_1 -> wrist_yaw_1_link; parent wrist_pitch_1 -> wrist_pitch_1_link
- joint wrist_yaw_2: child wrist_yaw_2 -> wrist_yaw_2_link; parent wrist_pitch_2 -> wrist_pitch_2_link

File: kyon_urdf/urdf/kyon_base.urdf.xacro (robot description, xacro)
@@ -36,5 +36,5 @@
 </joint>
 <link name="imu_link"/>
-<joint name="imu_link" type="fixed">
+<joint name="imu_link_joint" type="fixed">
     <parent link="pelvis"/>
     <child link="imu_link"/>
