Commit message: renamed root

File: kyon_srdf/srdf/kyon.srdf.xacro (robot description, xacro)
@@ -7,6 +7,6 @@
     <!-- ************ MODEL CONFIGURATION ************ -->
     <xacro:arg name="kyon_root" default="$(find kyon_urdf)" />
-    <xacro:property name="KYON_ROOT" value="$(arg kyon_root)" />
-    <xacro:arg name="config" default="${KYON_ROOT}/urdf/config/kyon.urdf.xacro"/>
+    <xacro:property name="ROOT" value="$(arg kyon_root)" />
+    <xacro:arg name="config" default="${ROOT}/urdf/config/kyon.urdf.xacro"/>
     <xacro:include filename="$(arg config)"/>
     <group name="base">

File: kyon_urdf/urdf/kyon.urdf.xacro (robot description, xacro)
@@ -4,5 +4,5 @@
 will be propagated to all its downstream childs -->
 <xacro:arg name="kyon_root" default="$(find kyon_urdf)" />
-<xacro:property name="KYON_ROOT" value="$(arg kyon_root)" />
+<xacro:property name="ROOT" value="$(arg kyon_root)" />
 <!-- setting use_abs_mesh_paths should be kept to false
 for use with tools like RViz, which does not accept plain
@@ -14,8 +14,8 @@
 <xacro:if value="${USE_ABS_MESH_PATHS}">
 	<xacro:if value="${USE_LOCAL_FILESYS_FOR_MESHES}">
-	<xacro:property name="MESH_PATH" value="file://${KYON_ROOT}/meshes" />
+	<xacro:property name="MESH_PATH" value="file://${ROOT}/meshes" />
 	</xacro:if>
 	<xacro:unless value="${USE_LOCAL_FILESYS_FOR_MESHES}">
-	<xacro:property name="MESH_PATH" value="${KYON_ROOT}/meshes" />
+	<xacro:property name="MESH_PATH" value="${ROOT}/meshes" />
 	</xacro:unless>
 	</xacro:if>
@@ -23,5 +23,5 @@
 <xacro:property name="MESH_PATH" value="package://kyon_urdf/meshes" />
 </xacro:unless>
-<xacro:arg name="config" default="${KYON_ROOT}/urdf/config/kyon.urdf.xacro"/>
+<xacro:arg name="config" default="${ROOT}/urdf/config/kyon.urdf.xacro"/>
 <!-- ************ MODEL CONFIGURATION ************ -->
 <xacro:include filename="$(arg config)"/>
@@ -38,5 +38,5 @@
 </xacro:if>
 <!-- ************ CETC-SAT plain model ************ -->
-<xacro:include filename="${KYON_ROOT}/urdf/kyon_base.urdf.xacro"/>
+<xacro:include filename="${ROOT}/urdf/kyon_base.urdf.xacro"/>
 <!-- ************ Control frames ************ -->
 <!--xacro:include filename="$(find pholus_urdf)/urdf/control_frames.urdf.xacro"/-->

File: kyon_urdf/urdf/kyon_base.urdf.xacro (robot description, xacro)
@@ -3,9 +3,9 @@
 <xacro:arg name="bilevel_codes" default="false" /> <!-- if true, load codes vars from externally provided files-->
 <xacro:arg name="sample_idx" default = "0"/>
-<xacro:include filename="${KYON_ROOT}/urdf/utils.urdf.xacro" />
-<xacro:include filename="${KYON_ROOT}/urdf/parts/kinematics_properties.urdf.xacro" />
+<xacro:include filename="${ROOT}/urdf/utils.urdf.xacro" />
+<xacro:include filename="${ROOT}/urdf/parts/kinematics_properties.urdf.xacro" />
 <!-- NOTE: here we need to include "kinematics_properties" first because "inertial_properties" depends on it-->
-<xacro:include filename="${KYON_ROOT}/urdf/parts/inertial_properties.urdf.xacro" />
-<xacro:include filename="${KYON_ROOT}/urdf/parts/limits.urdf.xacro" />
+<xacro:include filename="${ROOT}/urdf/parts/inertial_properties.urdf.xacro" />
+<xacro:include filename="${ROOT}/urdf/parts/limits.urdf.xacro" />
 <link name="base_link"/>
 <joint name="base_joint" type="fixed">
@@ -170,8 +170,8 @@
 </xacro:if>
 <xacro:if value="${ADD_UPPER_BODY}">
-    <xacro:include filename="${KYON_ROOT}/urdf/parts/arms.urdf.xacro" />
+    <xacro:include filename="${ROOT}/urdf/parts/arms.urdf.xacro" />
 </xacro:if>
 <xacro:if value="${ADD_LEGS}">
-	<xacro:include filename="${KYON_ROOT}/urdf/parts/legs.urdf.xacro" />
+	<xacro:include filename="${ROOT}/urdf/parts/legs.urdf.xacro" />
 </xacro:if>
 <xacro:if value="${PAYLOAD}">

File: kyon_urdf/urdf/kyon_robot.urdf.xacro (robot description, xacro)
@@ -4,5 +4,5 @@
   will be propagated to all its downstream childs -->
   <xacro:arg name="kyon_root" default="$(find kyon_urdf)" />
-  <xacro:property name="KYON_ROOT" value="$(arg kyon_root)" />
+  <xacro:property name="ROOT" value="$(arg kyon_root)" />
   <!-- setting use_abs_mesh_paths should be kept to false
   for use with tools like RViz, which does not accept plain
@@ -11,13 +11,13 @@
   <xacro:property name="USE_ABS_MESH_PATHS" value="$(arg use_abs_mesh_paths)" />
   <xacro:if value="${USE_ABS_MESH_PATHS}">
-    <xacro:property name="MESH_PATH" value="${KYON_ROOT}/meshes" />
+    <xacro:property name="MESH_PATH" value="${ROOT}/meshes" />
   </xacro:if>
   <xacro:unless value="${USE_ABS_MESH_PATHS}">
     <xacro:property name="MESH_PATH" value="package://kyon_urdf/meshes" />
   </xacro:unless>
-  <xacro:include filename="${KYON_ROOT}/urdf/kyon.urdf.xacro" />
-  <xacro:include filename="${KYON_ROOT}/urdf/gazebo/kyon.gazebo.xacro" />
-  <xacro:include filename="${KYON_ROOT}/urdf/gazebo/xbot.gazebo.xacro" />
-  <xacro:include filename="${KYON_ROOT}/urdf/gazebo/materials.gazebo.xacro" />
+  <xacro:include filename="${ROOT}/urdf/kyon.urdf.xacro" />
+  <xacro:include filename="${ROOT}/urdf/gazebo/kyon.gazebo.xacro" />
+  <xacro:include filename="${ROOT}/urdf/gazebo/xbot.gazebo.xacro" />
+  <xacro:include filename="${ROOT}/urdf/gazebo/materials.gazebo.xacro" />
   <xacro:unless value="${ADD_LEGS}">
     <link name="world"/>

File: kyon_urdf/urdf/parts/arms.urdf.xacro (robot description, xacro)
@@ -1,6 +1,6 @@
 <?xml version="1.0"?>
 <robot xmlns:xacro="http://ros.org/wiki/xacro">
-<xacro:include filename="${KYON_ROOT}/urdf/parts/kyon_arm.urdf.xacro"/>
-<xacro:include filename="${KYON_ROOT}/urdf/parts/kyon_ball_ee.xacro"/>
+<xacro:include filename="${ROOT}/urdf/parts/kyon_arm.urdf.xacro"/>
+<xacro:include filename="${ROOT}/urdf/parts/kyon_ball_ee.xacro"/>
 <xacro:include filename="${DAGANA_ROOT}/urdf/dagana_macro.urdf.xacro"/>
 <!-- arms -->

File: kyon_urdf/urdf/parts/inertial_properties.urdf.xacro (robot description, xacro)
@@ -1,5 +1,5 @@
 <?xml version="1.0"?>
 <robot  xmlns:xacro="http://ros.org/wiki/xacro">
-    <xacro:property name="inertial_yaml_file" value="${KYON_ROOT}/urdf/config/inertial_properties.yaml" />
+    <xacro:property name="inertial_yaml_file" value="${ROOT}/urdf/config/inertial_properties.yaml" />
     <xacro:property name="inertial_props" value="${xacro.load_yaml(inertial_yaml_file)}"/>
     <xacro:property name="pelvis_mass" value="${inertial_props['pelvis_mass']}"/>

File: kyon_urdf/urdf/parts/kinematics_properties.urdf.xacro (robot description, xacro)
@@ -1,5 +1,5 @@
 <?xml version="1.0"?>
 <robot  xmlns:xacro="http://ros.org/wiki/xacro">
-    <xacro:property name="kin_yaml_file" value="${KYON_ROOT}/urdf/config/kinematics_properties.yaml" />
+    <xacro:property name="kin_yaml_file" value="${ROOT}/urdf/config/kinematics_properties.yaml" />
     <xacro:property name="kin_props" value="${xacro.load_yaml(kin_yaml_file)}"/>
     <xacro:property name="cylinder_radius" value="${kin_props['cylinder_radius']}"/>

File: kyon_urdf/urdf/parts/legs.urdf.xacro (robot description, xacro)
@@ -1,5 +1,5 @@
 <?xml version="1.0"?>
 <robot xmlns:xacro="http://ros.org/wiki/xacro">
-<xacro:include filename="${KYON_ROOT}/urdf/parts/kyon_leg.urdf.xacro" />
+<xacro:include filename="${ROOT}/urdf/parts/kyon_leg.urdf.xacro" />
 <xacro:kyon_leg leg_num="1" origin_x="1" origin_y="-1" mirror="-1">
 </xacro:kyon_leg>

Commit message: Signed-off-by: Andrea Patrizi <andreapatrizi1b6e6@gmail.com>

File: kyon_srdf/srdf/kyon.srdf.xacro (robot description, xacro)
@@ -6,6 +6,6 @@
 <robot xmlns:xacro="http://ros.org/wiki/xacro" name="kyon">
     <!-- ************ MODEL CONFIGURATION ************ -->
-    <xacro:arg name="kyon_root" default="$(find kyon_urdf)" />
-    <xacro:property name="ROOT" value="$(arg kyon_root)" />
+    <xacro:arg name="root" default="$(find kyon_urdf)" />
+    <xacro:property name="ROOT" value="$(arg root)" />
     <xacro:arg name="config" default="${ROOT}/urdf/config/kyon.urdf.xacro"/>
     <xacro:include filename="$(arg config)"/>

File: kyon_urdf/urdf/kyon.urdf.xacro (robot description, xacro)
@@ -3,6 +3,6 @@
 <!-- This argument and property should be in the top level xacro and
 will be propagated to all its downstream childs -->
-<xacro:arg name="kyon_root" default="$(find kyon_urdf)" />
-<xacro:property name="ROOT" value="$(arg kyon_root)" />
+<xacro:arg name="root" default="$(find kyon_urdf)" />
+<xacro:property name="ROOT" value="$(arg root)" />
 <!-- setting use_abs_mesh_paths should be kept to false
 for use with tools like RViz, which does not accept plain

File: kyon_urdf/urdf/kyon_robot.urdf.xacro (robot description, xacro)
@@ -3,6 +3,6 @@
   <!-- This argument and property should be in the top level xacro and
   will be propagated to all its downstream childs -->
-  <xacro:arg name="kyon_root" default="$(find kyon_urdf)" />
-  <xacro:property name="ROOT" value="$(arg kyon_root)" />
+  <xacro:arg name="root" default="$(find kyon_urdf)" />
+  <xacro:property name="ROOT" value="$(arg root)" />
   <!-- setting use_abs_mesh_paths should be kept to false
   for use with tools like RViz, which does not accept plain

Commit message: fixed launch files and few errors and tested with kyon_controller simulator.launch in all configurations

File: kyon_srdf/srdf/kyon.srdf.xacro (robot description, xacro)
@@ -14,17 +14,17 @@
     	<xacro:if value="${ADD_WHEELS}">
 			<group name="front_left_leg">
-		        <chain base_link="pelvis" tip_link="wheel_1" />
+		        <chain base_link="pelvis" tip_link="wheel_1_link" />
 		    </group>
 		    <group name="front_right_leg">
-		        <chain base_link="pelvis" tip_link="wheel_2" />
+		        <chain base_link="pelvis" tip_link="wheel_2_link" />
 		    </group>
 		    <group name="rear_right_leg">
-		        <chain base_link="pelvis" tip_link="wheel_4" />
+		        <chain base_link="pelvis" tip_link="wheel_4_link" />
 		    </group>
 		    <group name="rear_left_leg">
-		        <chain base_link="pelvis" tip_link="wheel_3" />
+		        <chain base_link="pelvis" tip_link="wheel_3_link" />
 		    </group>
 		</xacro:if>
-		<xacro:unless value="${ADD_WHEELS}">
+		<xacro:if value="${ADD_FEET}">
 		    <group name="front_left_leg">
 		        <chain base_link="pelvis" tip_link="contact_1" />
@@ -39,29 +39,27 @@
 		        <chain base_link="pelvis" tip_link="contact_3" />
 		    </group>
-		</xacro:unless>
+		</xacro:if>
+        <xacro:if value="${ADD_STEERING_WHEELS}">
+            <group name="front_left_leg">
+                <chain base_link="pelvis" tip_link="wheel_1_link"/>
+            </group>
+            <group name="front_right_leg">
+		        <chain base_link="pelvis" tip_link="wheel_2_link" />
+		    </group>
+		    <group name="rear_right_leg">
+		        <chain base_link="pelvis" tip_link="wheel_4_link" />
+		    </group>
+		    <group name="rear_left_leg">
+		        <chain base_link="pelvis" tip_link="wheel_3_link" />
+		    </group>
+        </xacro:if>
     </xacro:if>
     <xacro:if value="${ADD_UPPER_BODY}">
-    	<xacro:if value="${ADD_DAGANA}">
-			<group name="left_arm">
-				<chain base_link="pelvis" tip_link="dagana_1_claw"/>
-			</group>
-			<group name="right_arm">
-				<chain base_link="pelvis" tip_link="dagana_2_claw"/>
-			</group>
-            <!-- <group name="left_hand">
-				<chain base_link="dagana_1_base" tip_link="dagana_1_clamp"/>
-			</group>
-            <group name="right_hand">
-				<chain base_link="dagana_1_base" tip_link="dagana_2_clamp"/>
-			</group> -->
-		</xacro:if>
-		<xacro:unless value="${ADD_DAGANA}">
-			<group name="left_arm">
-				<chain base_link="pelvis" tip_link="ball_arm_1"/>
-			</group>
-			<group name="right_arm">
-				<chain base_link="pelvis" tip_link="ball_arm_2"/>
-			</group>
-		</xacro:unless>
+		<group name="left_arm">
+			<chain base_link="pelvis" tip_link="dagana_1_claw"/>
+		</group>
+		<group name="right_arm">
+			<chain base_link="pelvis" tip_link="dagana_2_claw"/>
+		</group>
     </xacro:if>
     <group name="chains">        <!--THIS HAS TO BE THE LAST GROUP IN THE FILE -->
@@ -76,8 +74,4 @@
             <group name="right_arm"/>
         </xacro:if>
-        <!-- <xacro:if value="${ADD_DAGANA}">
-            <group name="left_hand"/>
-            <group name="right_hand"/>
-        </xacro:if> -->
     </group>
     <!-- Homing posture -->
