Commit message: fixed launch files and few errors and tested with kyon_controller simulator.launch in all configurations

File: kyon_urdf/urdf/kyon.urdf (robot description, URDF)
Before this commit: robot kyon, 34 links, 33 joints
Links:
- removed link contact_1
- removed link contact_2
- removed link contact_3
- removed link contact_4
- added link D435_front1_accel_frame
- added link D435_front1_accel_optical_frame
- added link D435_front1_bottom_screw_frame
- added link D435_front1_color_frame
- added link D435_front1_color_optical_frame
- added link D435_front1_depth_frame
- added link D435_front1_depth_optical_frame
- added link D435_front1_gyro_frame
- added link D435_front1_gyro_optical_frame
- added link D435_front1_left_ir_frame
- added link D435_front1_left_ir_optical_frame
- added link D435_front1_link, mass 0.564; collision box size=0.02505 0.09 0.025; visual mesh filename=package://realsense2_description/meshes/d435.dae
- added link D435_front1_right_ir_frame
- added link D435_front1_right_ir_optical_frame
- added link D435_front2_accel_frame
- added link D435_front2_accel_optical_frame
- added link D435_front2_bottom_screw_frame
- added link D435_front2_color_frame
- added link D435_front2_color_optical_frame
- added link D435_front2_depth_frame
- added link D435_front2_depth_optical_frame
- added link D435_front2_gyro_frame
- added link D435_front2_gyro_optical_frame
- added link D435_front2_left_ir_frame
- added link D435_front2_left_ir_optical_frame
- added link D435_front2_link, mass 0.564; collision box size=0.02505 0.09 0.025; visual mesh filename=package://realsense2_description/meshes/d435.dae
- added link D435_front2_right_ir_frame
- added link D435_front2_right_ir_optical_frame
- added link D435_front3_accel_frame
- added link D435_front3_accel_optical_frame
- added link D435_front3_bottom_screw_frame
- added link D435_front3_color_frame
- added link D435_front3_color_optical_frame
- added link D435_front3_depth_frame
- added link D435_front3_depth_optical_frame
- added link D435_front3_gyro_frame
- added link D435_front3_gyro_optical_frame
- added link D435_front3_left_ir_frame
- added link D435_front3_left_ir_optical_frame
- added link D435_front3_link, mass 0.564; collision box size=0.02505 0.09 0.025; visual mesh filename=package://realsense2_description/meshes/d435.dae
- added link D435_front3_right_ir_frame
- added link D435_front3_right_ir_optical_frame
- added link D435_left_accel_frame
- added link D435_left_accel_optical_frame
- added link D435_left_bottom_screw_frame
- added link D435_left_color_frame
- added link D435_left_color_optical_frame
- added link D435_left_depth_frame
- added link D435_left_depth_optical_frame
- added link D435_left_gyro_frame
- added link D435_left_gyro_optical_frame
- added link D435_left_left_ir_frame
- added link D435_left_left_ir_optical_frame
- added link D435_left_link, mass 0.564; collision box size=0.02505 0.09 0.025; visual mesh filename=package://realsense2_description/meshes/d435.dae
- added link D435_left_right_ir_frame
- added link D435_left_right_ir_optical_frame
- added link D435_rear_accel_frame
- added link D435_rear_accel_optical_frame
- added link D435_rear_bottom_screw_frame
- added link D435_rear_color_frame
- added link D435_rear_color_optical_frame
- added link D435_rear_depth_frame
- added link D435_rear_depth_optical_frame
- added link D435_rear_gyro_frame
- added link D435_rear_gyro_optical_frame
- added link D435_rear_left_ir_frame
- added link D435_rear_left_ir_optical_frame
- added link D435_rear_link, mass 0.564; collision box size=0.02505 0.09 0.025; visual mesh filename=package://realsense2_description/meshes/d435.dae
- added link D435_rear_right_ir_frame
- added link D435_rear_right_ir_optical_frame
- added link D435_right_accel_frame
- added link D435_right_accel_optical_frame
- added link D435_right_bottom_screw_frame
- added link D435_right_color_frame
- added link D435_right_color_optical_frame
- added link D435_right_depth_frame
- added link D435_right_depth_optical_frame
- added link D435_right_gyro_frame
- added link D435_right_gyro_optical_frame
- added link D435_right_left_ir_frame
- added link D435_right_left_ir_optical_frame
- added link D435_right_link, mass 0.564; collision box size=0.02505 0.09 0.025; visual mesh filename=package://realsense2_description/meshes/d435.dae
- added link D435_right_right_ir_frame
- added link D435_right_right_ir_optical_frame
- added link velodyne, mass 0.01; collision sphere radius=0; visual mesh filename=package://velodyne_description/meshes/VLP16_scan.dae
- added link velodyne_base_link, mass 0.83; collision cylinder length=0.0717 radius=0.0516; visual mesh filename=package://velodyne_description/meshes/VLP16_base_1.dae
- added link wheel_1_link, mass 1.263839; collision mesh filename=package://kyon_urdf/meshes/collision/mesh_wheel.stl scale=0.001 0.001 0.001; visual mesh filename=package://kyon_urdf/meshes/mesh_wheel.stl scale=0.001 0.001 0.001
- added link wheel_2_link, mass 1.263839; collision mesh filename=package://kyon_urdf/meshes/collision/mesh_wheel.stl scale=0.001 0.001 0.001; visual mesh filename=package://kyon_urdf/meshes/mesh_wheel.stl scale=0.001 0.001 0.001
- added link wheel_3_link, mass 1.263839; collision mesh filename=package://kyon_urdf/meshes/collision/mesh_wheel.stl scale=0.001 0.001 0.001; visual mesh filename=package://kyon_urdf/meshes/mesh_wheel.stl scale=0.001 0.001 0.001
- added link wheel_4_link, mass 1.263839; collision mesh filename=package://kyon_urdf/meshes/collision/mesh_wheel.stl scale=0.001 0.001 0.001; visual mesh filename=package://kyon_urdf/meshes/mesh_wheel.stl scale=0.001 0.001 0.001
- link knee_pitch_1_link: mass 0.70900216 -> 1.8; geometry collision mesh filename=package://kyon_urdf/meshes/collision/mesh_fixed-wheel-leg.s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 scale=-0.001 0.001 0.001; visual mesh filename=package://kyon_urdf/meshes/mesh_fixed-wheel-leg.stl scale=-0.001 0.001 0.001
- link knee_pitch_2_link: mass 0.70900216 -> 1.8; geometry collision mesh filename=package://kyon_urdf/meshes/collision/mesh_fixed-wheel-leg.s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 scale=0.001 0.001 0.001; visual mesh filename=package://kyon_urdf/meshes/mesh_fixed-wheel-leg.stl scale=0.001 0.001 0.001
- link knee_pitch_3_link: mass 0.70900216 -> 1.8; geometry collision mesh filename=package://kyon_urdf/meshes/collision/mesh_fixed-wheel-leg.s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 scale=-0.001 0.001 0.001; visual mesh filename=package://kyon_urdf/meshes/mesh_fixed-wheel-leg.stl scale=-0.001 0.001 0.001
- link knee_pitch_4_link: mass 0.70900216 -> 1.8; geometry collision mesh filename=package://kyon_urdf/meshes/collision/mesh_fixed-wheel-leg.s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 scale=0.001 0.001 0.001; visual mesh filename=package://kyon_urdf/meshes/mesh_fixed-wheel-leg.stl scale=0.001 0.001 0.001
Joints:
- removed joint contact_1_joint
- removed joint contact_2_joint
- removed joint contact_3_joint
- removed joint contact_4_joint
- added joint D435_front1_accel_joint: type fixed, parent D435_front1_link, child D435_front1_accel_frame, origin xyz=-0.00174 0.00552 0.0176 rpy=0 0 0
- added joint D435_front1_accel_optical_joint: type fixed, parent D435_front1_accel_frame, child D435_front1_accel_optical_frame, origin xyz=0 0 0 rpy=-1.5707963267948966 0 -1.5707963267948966
- added joint D435_front1_color_joint: type fixed, parent D435_front1_depth_frame, child D435_front1_color_frame, origin xyz=0 0.015 0 rpy=0 0 0
- added joint D435_front1_color_optical_joint: type fixed, parent D435_front1_color_frame, child D435_front1_color_optical_frame, origin xyz=0 0 0 rpy=-1.5707963267948966 0 -1.5707963267948966
- added joint D435_front1_depth_joint: type fixed, parent D435_front1_link, child D435_front1_depth_frame, origin xyz=0 0 0 rpy=0 0 0
- added joint D435_front1_depth_optical_joint: type fixed, parent D435_front1_depth_frame, child D435_front1_depth_optical_frame, origin xyz=0 0 0 rpy=-1.5707963267948966 0 -1.5707963267948966
- added joint D435_front1_gyro_joint: type fixed, parent D435_front1_link, child D435_front1_gyro_frame, origin xyz=-0.00174 0.00552 0.0176 rpy=0 0 0
- added joint D435_front1_gyro_optical_joint: type fixed, parent D435_front1_gyro_frame, child D435_front1_gyro_optical_frame, origin xyz=0 0 0 rpy=-1.5707963267948966 0 -1.5707963267948966
- added joint D435_front1_joint: type fixed, parent pelvis, child D435_front1_bottom_screw_frame, origin xyz=0.40 -0.08 0 rpy=-1.57 0 0.34
- added joint D435_front1_left_ir_joint: type fixed, parent D435_front1_depth_frame, child D435_front1_left_ir_frame, origin xyz=0 0.0 0 rpy=0 0 0
- added joint D435_front1_left_ir_optical_joint: type fixed, parent D435_front1_left_ir_frame, child D435_front1_left_ir_optical_frame, origin xyz=0 0 0 rpy=-1.5707963267948966 0 -1.5707963267948966
- added joint D435_front1_link_joint: type fixed, parent D435_front1_bottom_screw_frame, child D435_front1_link, origin xyz=0 0.0175 0.0125 rpy=0 0 0
- added joint D435_front1_right_ir_joint: type fixed, parent D435_front1_depth_frame, child D435_front1_right_ir_frame, origin xyz=0 -0.05 0 rpy=0 0 0
- added joint D435_front1_right_ir_optical_joint: type fixed, parent D435_front1_right_ir_frame, child D435_front1_right_ir_optical_frame, origin xyz=0 0 0 rpy=-1.5707963267948966 0 -1.5707963267948966
- added joint D435_front2_accel_joint: type fixed, parent D435_front2_link, child D435_front2_accel_frame, origin xyz=-0.00174 0.00552 0.0176 rpy=0 0 0
- added joint D435_front2_accel_optical_joint: type fixed, parent D435_front2_accel_frame, child D435_front2_accel_optical_frame, origin xyz=0 0 0 rpy=-1.5707963267948966 0 -1.5707963267948966
- added joint D435_front2_color_joint: type fixed, parent D435_front2_depth_frame, child D435_front2_color_frame, origin xyz=0 0.015 0 rpy=0 0 0
- added joint D435_front2_color_optical_joint: type fixed, parent D435_front2_color_frame, child D435_front2_color_optical_frame, origin xyz=0 0 0 rpy=-1.5707963267948966 0 -1.5707963267948966
- added joint D435_front2_depth_joint: type fixed, parent D435_front2_link, child D435_front2_depth_frame, origin xyz=0 0 0 rpy=0 0 0
- added joint D435_front2_depth_optical_joint: type fixed, parent D435_front2_depth_frame, child D435_front2_depth_optical_frame, origin xyz=0 0 0 rpy=-1.5707963267948966 0 -1.5707963267948966
- added joint D435_front2_gyro_joint: type fixed, parent D435_front2_link, child D435_front2_gyro_frame, origin xyz=-0.00174 0.00552 0.0176 rpy=0 0 0
- added joint D435_front2_gyro_optical_joint: type fixed, parent D435_front2_gyro_frame, child D435_front2_gyro_optical_frame, origin xyz=0 0 0 rpy=-1.5707963267948966 0 -1.5707963267948966
- added joint D435_front2_joint: type fixed, parent pelvis, child D435_front2_bottom_screw_frame, origin xyz=0.40 0.08 0 rpy=-1.57 0 -0.34
- added joint D435_front2_left_ir_joint: type fixed, parent D435_front2_depth_frame, child D435_front2_left_ir_frame, origin xyz=0 0.0 0 rpy=0 0 0
- added joint D435_front2_left_ir_optical_joint: type fixed, parent D435_front2_left_ir_frame, child D435_front2_left_ir_optical_frame, origin xyz=0 0 0 rpy=-1.5707963267948966 0 -1.5707963267948966
- added joint D435_front2_link_joint: type fixed, parent D435_front2_bottom_screw_frame, child D435_front2_link, origin xyz=0 0.0175 0.0125 rpy=0 0 0
- added joint D435_front2_right_ir_joint: type fixed, parent D435_front2_depth_frame, child D435_front2_right_ir_frame, origin xyz=0 -0.05 0 rpy=0 0 0
- added joint D435_front2_right_ir_optical_joint: type fixed, parent D435_front2_right_ir_frame, child D435_front2_right_ir_optical_frame, origin xyz=0 0 0 rpy=-1.5707963267948966 0 -1.5707963267948966
- added joint D435_front3_accel_joint: type fixed, parent D435_front3_link, child D435_front3_accel_frame, origin xyz=-0.00174 0.00552 0.0176 rpy=0 0 0
- added joint D435_front3_accel_optical_joint: type fixed, parent D435_front3_accel_frame, child D435_front3_accel_optical_frame, origin xyz=0 0 0 rpy=-1.5707963267948966 0 -1.5707963267948966
- added joint D435_front3_color_joint: type fixed, parent D435_front3_depth_frame, child D435_front3_color_frame, origin xyz=0 0.015 0 rpy=0 0 0
- added joint D435_front3_color_optical_joint: type fixed, parent D435_front3_color_frame, child D435_front3_color_optical_frame, origin xyz=0 0 0 rpy=-1.5707963267948966 0 -1.5707963267948966
- added joint D435_front3_depth_joint: type fixed, parent D435_front3_link, child D435_front3_depth_frame, origin xyz=0 0 0 rpy=0 0 0
- added joint D435_front3_depth_optical_joint: type fixed, parent D435_front3_depth_frame, child D435_front3_depth_optical_frame, origin xyz=0 0 0 rpy=-1.5707963267948966 0 -1.5707963267948966
- added joint D435_front3_gyro_joint: type fixed, parent D435_front3_link, child D435_front3_gyro_frame, origin xyz=-0.00174 0.00552 0.0176 rpy=0 0 0
- added joint D435_front3_gyro_optical_joint: type fixed, parent D435_front3_gyro_frame, child D435_front3_gyro_optical_frame, origin xyz=0 0 0 rpy=-1.5707963267948966 0 -1.5707963267948966
- added joint D435_front3_joint: type fixed, parent pelvis, child D435_front3_bottom_screw_frame, origin xyz=0.37 0 -0.11 rpy=0 0.75 0
- added joint D435_front3_left_ir_joint: type fixed, parent D435_front3_depth_frame, child D435_front3_left_ir_frame, origin xyz=0 0.0 0 rpy=0 0 0
- added joint D435_front3_left_ir_optical_joint: type fixed, parent D435_front3_left_ir_frame, child D435_front3_left_ir_optical_frame, origin xyz=0 0 0 rpy=-1.5707963267948966 0 -1.5707963267948966
- added joint D435_front3_link_joint: type fixed, parent D435_front3_bottom_screw_frame, child D435_front3_link, origin xyz=0 0.0175 0.0125 rpy=0 0 0
- added joint D435_front3_right_ir_joint: type fixed, parent D435_front3_depth_frame, child D435_front3_right_ir_frame, origin xyz=0 -0.05 0 rpy=0 0 0
- added joint D435_front3_right_ir_optical_joint: type fixed, parent D435_front3_right_ir_frame, child D435_front3_right_ir_optical_frame, origin xyz=0 0 0 rpy=-1.5707963267948966 0 -1.5707963267948966
- added joint D435_left_accel_joint: type fixed, parent D435_left_link, child D435_left_accel_frame, origin xyz=-0.00174 0.00552 0.0176 rpy=0 0 0
- added joint D435_left_accel_optical_joint: type fixed, parent D435_left_accel_frame, child D435_left_accel_optical_frame, origin xyz=0 0 0 rpy=-1.5707963267948966 0 -1.5707963267948966
- added joint D435_left_color_joint: type fixed, parent D435_left_depth_frame, child D435_left_color_frame, origin xyz=0 0.015 0 rpy=0 0 0
- added joint D435_left_color_optical_joint: type fixed, parent D435_left_color_frame, child D435_left_color_optical_frame, origin xyz=0 0 0 rpy=-1.5707963267948966 0 -1.5707963267948966
- added joint D435_left_depth_joint: type fixed, parent D435_left_link, child D435_left_depth_frame, origin xyz=0 0 0 rpy=0 0 0
- added joint D435_left_depth_optical_joint: type fixed, parent D435_left_depth_frame, child D435_left_depth_optical_frame, origin xyz=0 0 0 rpy=-1.5707963267948966 0 -1.5707963267948966
- added joint D435_left_gyro_joint: type fixed, parent D435_left_link, child D435_left_gyro_frame, origin xyz=-0.00174 0.00552 0.0176 rpy=0 0 0
- added joint D435_left_gyro_optical_joint: type fixed, parent D435_left_gyro_frame, child D435_left_gyro_optical_frame, origin xyz=0 0 0 rpy=-1.5707963267948966 0 -1.5707963267948966
- added joint D435_left_joint: type fixed, parent pelvis, child D435_left_bottom_screw_frame, origin xyz=-0.175 0.22 0 rpy=0 0.35 1.57
- added joint D435_left_left_ir_joint: type fixed, parent D435_left_depth_frame, child D435_left_left_ir_frame, origin xyz=0 0.0 0 rpy=0 0 0
- added joint D435_left_left_ir_optical_joint: type fixed, parent D435_left_left_ir_frame, child D435_left_left_ir_optical_frame, origin xyz=0 0 0 rpy=-1.5707963267948966 0 -1.5707963267948966
- added joint D435_left_link_joint: type fixed, parent D435_left_bottom_screw_frame, child D435_left_link, origin xyz=0 0.0175 0.0125 rpy=0 0 0
- added joint D435_left_right_ir_joint: type fixed, parent D435_left_depth_frame, child D435_left_right_ir_frame, origin xyz=0 -0.05 0 rpy=0 0 0
- added joint D435_left_right_ir_optical_joint: type fixed, parent D435_left_right_ir_frame, child D435_left_right_ir_optical_frame, origin xyz=0 0 0 rpy=-1.5707963267948966 0 -1.5707963267948966
- added joint D435_rear_accel_joint: type fixed, parent D435_rear_link, child D435_rear_accel_frame, origin xyz=-0.00174 0.00552 0.0176 rpy=0 0 0
- added joint D435_rear_accel_optical_joint: type fixed, parent D435_rear_accel_frame, child D435_rear_accel_optical_frame, origin xyz=0 0 0 rpy=-1.5707963267948966 0 -1.5707963267948966
- added joint D435_rear_color_joint: type fixed, parent D435_rear_depth_frame, child D435_rear_color_frame, origin xyz=0 0.015 0 rpy=0 0 0
- added joint D435_rear_color_optical_joint: type fixed, parent D435_rear_color_frame, child D435_rear_color_optical_frame, origin xyz=0 0 0 rpy=-1.5707963267948966 0 -1.5707963267948966
- added joint D435_rear_depth_joint: type fixed, parent D435_rear_link, child D435_rear_depth_frame, origin xyz=0 0 0 rpy=0 0 0
- added joint D435_rear_depth_optical_joint: type fixed, parent D435_rear_depth_frame, child D435_rear_depth_optical_frame, origin xyz=0 0 0 rpy=-1.5707963267948966 0 -1.5707963267948966
- added joint D435_rear_gyro_joint: type fixed, parent D435_rear_link, child D435_rear_gyro_frame, origin xyz=-0.00174 0.00552 0.0176 rpy=0 0 0
- added joint D435_rear_gyro_optical_joint: type fixed, parent D435_rear_gyro_frame, child D435_rear_gyro_optical_frame, origin xyz=0 0 0 rpy=-1.5707963267948966 0 -1.5707963267948966
- added joint D435_rear_joint: type fixed, parent pelvis, child D435_rear_bottom_screw_frame, origin xyz=-0.39 0 0 rpy=0 0.35 3.14
- added joint D435_rear_left_ir_joint: type fixed, parent D435_rear_depth_frame, child D435_rear_left_ir_frame, origin xyz=0 0.0 0 rpy=0 0 0
- added joint D435_rear_left_ir_optical_joint: type fixed, parent D435_rear_left_ir_frame, child D435_rear_left_ir_optical_frame, origin xyz=0 0 0 rpy=-1.5707963267948966 0 -1.5707963267948966
- added joint D435_rear_link_joint: type fixed, parent D435_rear_bottom_screw_frame, child D435_rear_link, origin xyz=0 0.0175 0.0125 rpy=0 0 0
- added joint D435_rear_right_ir_joint: type fixed, parent D435_rear_depth_frame, child D435_rear_right_ir_frame, origin xyz=0 -0.05 0 rpy=0 0 0
- added joint D435_rear_right_ir_optical_joint: type fixed, parent D435_rear_right_ir_frame, child D435_rear_right_ir_optical_frame, origin xyz=0 0 0 rpy=-1.5707963267948966 0 -1.5707963267948966
- added joint D435_right_accel_joint: type fixed, parent D435_right_link, child D435_right_accel_frame, origin xyz=-0.00174 0.00552 0.0176 rpy=0 0 0
- added joint D435_right_accel_optical_joint: type fixed, parent D435_right_accel_frame, child D435_right_accel_optical_frame, origin xyz=0 0 0 rpy=-1.5707963267948966 0 -1.5707963267948966
- added joint D435_right_color_joint: type fixed, parent D435_right_depth_frame, child D435_right_color_frame, origin xyz=0 0.015 0 rpy=0 0 0
- added joint D435_right_color_optical_joint: type fixed, parent D435_right_color_frame, child D435_right_color_optical_frame, origin xyz=0 0 0 rpy=-1.5707963267948966 0 -1.5707963267948966
- added joint D435_right_depth_joint: type fixed, parent D435_right_link, child D435_right_depth_frame, origin xyz=0 0 0 rpy=0 0 0
- added joint D435_right_depth_optical_joint: type fixed, parent D435_right_depth_frame, child D435_right_depth_optical_frame, origin xyz=0 0 0 rpy=-1.5707963267948966 0 -1.5707963267948966
- added joint D435_right_gyro_joint: type fixed, parent D435_right_link, child D435_right_gyro_frame, origin xyz=-0.00174 0.00552 0.0176 rpy=0 0 0
- added joint D435_right_gyro_optical_joint: type fixed, parent D435_right_gyro_frame, child D435_right_gyro_optical_frame, origin xyz=0 0 0 rpy=-1.5707963267948966 0 -1.5707963267948966
- added joint D435_right_joint: type fixed, parent pelvis, child D435_right_bottom_screw_frame, origin xyz=-0.175 -0.22 0 rpy=0 0.35 -1.57
- added joint D435_right_left_ir_joint: type fixed, parent D435_right_depth_frame, child D435_right_left_ir_frame, origin xyz=0 0.0 0 rpy=0 0 0
- added joint D435_right_left_ir_optical_joint: type fixed, parent D435_right_left_ir_frame, child D435_right_left_ir_optical_frame, origin xyz=0 0 0 rpy=-1.5707963267948966 0 -1.5707963267948966
- added joint D435_right_link_joint: type fixed, parent D435_right_bottom_screw_frame, child D435_right_link, origin xyz=0 0.0175 0.0125 rpy=0 0 0
- added joint D435_right_right_ir_joint: type fixed, parent D435_right_depth_frame, child D435_right_right_ir_frame, origin xyz=0 -0.05 0 rpy=0 0 0
- added joint D435_right_right_ir_optical_joint: type fixed, parent D435_right_right_ir_frame, child D435_right_right_ir_optical_frame, origin xyz=0 0 0 rpy=-1.5707963267948966 0 -1.5707963267948966
- added joint velodyne_base_mount_joint: type fixed, parent pelvis, child velodyne_base_link, origin xyz=0.36 0 0.11 rpy=0 0 0
- added joint velodyne_base_scan_joint: type fixed, parent velodyne_base_link, child velodyne, origin xyz=0 0 0.0377 rpy=0 0 0
- added joint wheel_joint_1: type revolute, parent knee_pitch_1_link, child wheel_1_link, origin xyz=0.0 -0.3 0.054 rpy=0.0 0.0 0.0, axis 0 0 1, limit lower=-3.4056 upper=3.4056 effort=132 velocity=15.5
- added joint wheel_joint_2: type revolute, parent knee_pitch_2_link, child wheel_2_link, origin xyz=0.0 -0.3 0.054 rpy=0.0 0.0 0.0, axis 0 0 1, limit lower=-3.3266 upper=3.3266 effort=132 velocity=15.5
- added joint wheel_joint_3: type revolute, parent knee_pitch_3_link, child wheel_3_link, origin xyz=0.0 -0.3 0.054 rpy=0.0 0.0 0.0, axis 0 0 1, limit lower=-3.4696 upper=3.4696 effort=132 velocity=15.5
- added joint wheel_joint_4: type revolute, parent knee_pitch_4_link, child wheel_4_link, origin xyz=0.0 -0.3 0.054 rpy=0.0 0.0 0.0, axis 0 0 1, limit lower=-3.3426 upper=3.3426 effort=132 velocity=15.5

File: kyon_urdf/urdf/parts/kyon_arm.urdf.xacro (robot description, xacro)
@@ -140,7 +140,5 @@
 	<limit lower="${j_pitch_2_lower[arm_num-1]}" upper="${j_pitch_2_upper[arm_num-1]}" effort="${motor_effort}" velocity="${motor_velocity}"/>
 </joint>
-<xacro:if value="${ADD_DAGANA}">
-	<xacro:kyon_dagana arm_num="${arm_num}" parent="wrist_yaw_${arm_num}_link"/>
-</xacro:if>
+<xacro:kyon_dagana arm_num="${arm_num}" parent="wrist_yaw_${arm_num}_link"/>
 </xacro:macro>
 <!-- /macro arms -->

File: kyon_urdf/urdf/parts/wheel_leg.urdf.xacro (robot description, xacro)
@@ -51,5 +51,5 @@
 </joint>
 <joint name="wheel_joint_${leg_num}" type="revolute">
-    <parent link="knee_pitch_${leg_num}"/>
+    <parent link="knee_pitch_${leg_num}_link"/>
     <child link="wheel_${leg_num}_link"/>
     <origin xyz="${Wheel_Ox} ${Wheel_Oy} ${Wheel_Oz}" rpy="${Wheel_roll} ${Wheel_pitch} ${Wheel_yaw}"/>
