Commit message: renamed root

File: kyon_srdf/srdf/kyon.srdf.xacro (robot description, xacro)
@@ -6,7 +6,7 @@
 <robot xmlns:xacro="http://ros.org/wiki/xacro" name="kyon">
     <!-- ************ MODEL CONFIGURATION ************ -->
-    <xacro:arg name="kyon_root" default="$(find kyon_urdf)" />
-    <xacro:property name="KYON_ROOT" value="$(arg kyon_root)" />
-    <xacro:arg name="config" default="${KYON_ROOT}/urdf/config/kyon.urdf.xacro"/>
+    <xacro:arg name="root" default="$(find kyon_urdf)" />
+    <xacro:property name="ROOT" value="$(arg root)" />
+    <xacro:arg name="config" default="${ROOT}/urdf/config/kyon.urdf.xacro"/>
     <xacro:include filename="$(arg config)"/>
     <group name="base">

File: kyon_urdf/urdf/kyon.urdf.xacro (robot description, xacro)
@@ -3,6 +3,6 @@
 <!-- This argument and property should be in the top level xacro and
 will be propagated to all its downstream childs -->
-<xacro:arg name="kyon_root" default="$(find kyon_urdf)" />
-<xacro:property name="KYON_ROOT" value="$(arg kyon_root)" />
+<xacro:arg name="root" default="$(find kyon_urdf)" />
+<xacro:property name="ROOT" value="$(arg root)" />
 <!-- setting use_abs_mesh_paths should be kept to false
 for use with tools like RViz, which does not accept plain
@@ -14,8 +14,8 @@
 <xacro:if value="${USE_ABS_MESH_PATHS}">
 	<xacro:if value="${USE_LOCAL_FILESYS_FOR_MESHES}">
-	<xacro:property name="MESH_PATH" value="file://${KYON_ROOT}/meshes" />
+	<xacro:property name="MESH_PATH" value="file://${ROOT}/meshes" />
 	</xacro:if>
 	<xacro:unless value="${USE_ABS_MESH_PATHS}">
-	<xacro:property name="MESH_PATH" value="${KYON_ROOT}/meshes" />
+	<xacro:property name="MESH_PATH" value="${ROOT}/meshes" />
 	</xacro:unless>
 	</xacro:if>
@@ -23,5 +23,5 @@
 <xacro:property name="MESH_PATH" value="package://kyon_urdf/meshes" />
 </xacro:unless>
-<xacro:arg name="config" default="${KYON_ROOT}/urdf/config/kyon.urdf.xacro"/>
+<xacro:arg name="config" default="${ROOT}/urdf/config/kyon.urdf.xacro"/>
 <!-- ************ MODEL CONFIGURATION ************ -->
 <xacro:include filename="$(arg config)"/>
@@ -38,5 +38,5 @@
 </xacro:if>
 <!-- ************ CETC-SAT plain model ************ -->
-<xacro:include filename="${KYON_ROOT}/urdf/kyon_base.urdf.xacro"/>
+<xacro:include filename="${ROOT}/urdf/kyon_base.urdf.xacro"/>
 <!-- ************ Control frames ************ -->
 <!--xacro:include filename="$(find pholus_urdf)/urdf/control_frames.urdf.xacro"/-->

File: kyon_urdf/urdf/kyon_robot.urdf.xacro (robot description, xacro)
@@ -3,6 +3,6 @@
   <!-- This argument and property should be in the top level xacro and
   will be propagated to all its downstream childs -->
-  <xacro:arg name="kyon_root" default="$(find kyon_urdf)" />
-  <xacro:property name="KYON_ROOT" value="$(arg kyon_root)" />
+  <xacro:arg name="root" default="$(find kyon_urdf)" />
+  <xacro:property name="ROOT" value="$(arg root)" />
   <!-- setting use_abs_mesh_paths should be kept to false
   for use with tools like RViz, which does not accept plain
@@ -11,13 +11,13 @@
   <xacro:property name="USE_ABS_MESH_PATHS" value="$(arg use_abs_mesh_paths)" />
   <xacro:if value="${USE_ABS_MESH_PATHS}">
-    <xacro:property name="MESH_PATH" value="${KYON_ROOT}/meshes" />
+    <xacro:property name="MESH_PATH" value="${ROOT}/meshes" />
   </xacro:if>
   <xacro:unless value="${USE_ABS_MESH_PATHS}">
     <xacro:property name="MESH_PATH" value="package://kyon_urdf/meshes" />
   </xacro:unless>
-  <xacro:include filename="${KYON_ROOT}/urdf/kyon.urdf.xacro" />
-  <xacro:include filename="${KYON_ROOT}/urdf/gazebo/kyon.gazebo.xacro" />
-  <xacro:include filename="${KYON_ROOT}/urdf/gazebo/xbot.gazebo.xacro" />
-  <xacro:include filename="${KYON_ROOT}/urdf/gazebo/materials.gazebo.xacro" />
+  <xacro:include filename="${ROOT}/urdf/kyon.urdf.xacro" />
+  <xacro:include filename="${ROOT}/urdf/gazebo/kyon.gazebo.xacro" />
+  <xacro:include filename="${ROOT}/urdf/gazebo/xbot.gazebo.xacro" />
+  <xacro:include filename="${ROOT}/urdf/gazebo/materials.gazebo.xacro" />
   <xacro:unless value="${ADD_LEGS}">
     <link name="world"/>

Commit message: commit everything

File: kyon_srdf/srdf/kyon.srdf.xacro (robot description, xacro)
@@ -63,4 +63,12 @@
 		</group>
     </xacro:if>
+    <!-- <xacro:if value="${ADD_FT_SENSORS}">
+        <group name="ft_sensors">
+            <joint name="knee_pitch_1"/>
+            <joint name="knee_pitch_2"/>
+            <joint name="knee_pitch_3"/>
+            <joint name="knee_pitch_4"/>
+        </group>
+    </xacro:if> -->
     <group name="chains">        <!--THIS HAS TO BE THE LAST GROUP IN THE FILE -->
         <xacro:if value="${ADD_LEGS}">
@@ -69,4 +77,7 @@
             <group name="rear_right_leg" />
             <group name="rear_left_leg" />
+            <!-- <xacro:if value="${ADD_FT_SENSORS}">
+                <group name="ft_sensors"/>
+            </xacro:if> -->
         </xacro:if>
         <xacro:if value="${ADD_UPPER_BODY}">

File: kyon_urdf/urdf/config/kyon.urdf.xacro (robot description, xacro)
@@ -13,4 +13,5 @@
 <xacro:arg name="payload" default="false"/>
 <xacro:arg name="steering_wheels" default="false"/>
+<xacro:arg name="ft_sensors" default="true"/>
 <!-- ************SELECT PARTS*************-->
 <!-- *************************************-->
@@ -22,4 +23,5 @@
 <xacro:property name="ADD_WHEELS" value="$(arg wheels)"/>
 <xacro:property name="ADD_STEERING_WHEELS" value="$(arg steering_wheels)"/>
+<xacro:property name="ADD_FT_SENSORS" value="$(arg ft_sensors)"/>
 <xacro:property name="ADD_FLOATING_BASE" value="$(arg floating_joint)" />
 <xacro:property name="ADD_VIRTUAL_FRAME" value="false" />

File: kyon_urdf/urdf/gazebo/ft_sensors.gazebo.xacro (robot description, xacro)
@@ -22,5 +22,5 @@
                 <always_on>true</always_on>
                 <visualize>true</visualize>
-                <update_rate>0.0</update_rate>
+                <update_rate>30.0</update_rate>
                 <pose>0.0 0.0 0.0 0.0 0.0 0.0</pose>
             </sensor>

File: kyon_urdf/urdf/gazebo/kyon.gazebo.xacro (robot description, xacro)
@@ -2,4 +2,31 @@
 <robot xmlns:xacro="http://ros.org/wiki/xacro">
     <xacro:if value="${ADD_LEGS}">
+        <gazebo reference="imu_link">
+            <sensor name="imu_link" type="imu">
+                <always_on>1</always_on>
+                <update_rate>500</update_rate>
+                <visualize>true</visualize>
+                <topic>__default_topic__</topic>
+                <imu>
+                    <!--
+                <noise>
+                <type>gaussian</type>
+                <rate>
+                    <mean>0.0</mean>
+                    <stddev>2e-4</stddev>
+                    <bias_mean>0.0000075</bias_mean>
+                    <bias_stddev>0.0000008</bias_stddev>
+                </rate>
+                <accel>
+                    <mean>0.0</mean>
+                    <stddev>1.7e-2</stddev>
+                    <bias_mean>0.1</bias_mean>
+                    <bias_stddev>0.001</bias_stddev>
+                </accel>
+                </noise>
+                -->
+                </imu>
+            </sensor>
+        </gazebo>
         <gazebo reference="hip_roll_1">
             <implicitSpringDamper>1</implicitSpringDamper>
@@ -51,32 +78,32 @@
         </gazebo>
         <gazebo reference="knee_pitch_1_link">
-        	<kp>1000000.0</kp>
-			<kd>100.0</kd>
-			<mu1>1.0</mu1>
-			<mu2>1.0</mu2>
+        	<kp>10000000.0</kp>
+			<kd>1000.0</kd>
+			<mu1>1</mu1>
+			<mu2>1</mu2>
 			<maxVel>1.0</maxVel>
 			<maxContacts>1</maxContacts>
 		</gazebo>
 		<gazebo reference="knee_pitch_2_link">
-        	<kp>1000000.0</kp>
-			<kd>100.0</kd>
-			<mu1>1.0</mu1>
-			<mu2>1.0</mu2>
+        	<kp>10000000.0</kp>
+			<kd>1000.0</kd>
+			<mu1>1</mu1>
+			<mu2>1</mu2>
 			<maxVel>1.0</maxVel>
 			<maxContacts>1</maxContacts>
 		</gazebo>
 		<gazebo reference="knee_pitch_3_link">
-        	<kp>1000000.0</kp>
-			<kd>100.0</kd>
-			<mu1>1.0</mu1>
-			<mu2>1.0</mu2>
+        	<kp>10000000.0</kp>
+			<kd>1000.0</kd>
+			<mu1>1</mu1>
+			<mu2>1</mu2>
 			<maxVel>1.0</maxVel>
 			<maxContacts>1</maxContacts>
 		</gazebo>
 		<gazebo reference="knee_pitch_4_link">
-        	<kp>1000000.0</kp>
-			<kd>100.0</kd>
-			<mu1>1.0</mu1>
-			<mu2>1.0</mu2>
+        	<kp>10000000.0</kp>
+			<kd>1000.0</kd>
+			<mu1>1</mu1>
+			<mu2>1</mu2>
 			<maxVel>1.0</maxVel>
 			<maxContacts>1</maxContacts>
@@ -159,5 +186,5 @@
 	    </gazebo>
 	</xacro:if>
-	<!-- <xacro:if value="${ADD_FT_SENSORS}">
+	<xacro:if value="${ADD_FT_SENSORS}">
 		<xacro:include filename="$(find kyon_urdf)/urdf/gazebo/ft_sensors.gazebo.xacro" />
 		<xacro:kyon_ft_sensor frame_id="knee_pitch_1"/>
@@ -165,4 +192,4 @@
 		<xacro:kyon_ft_sensor frame_id="knee_pitch_3"/>
 		<xacro:kyon_ft_sensor frame_id="knee_pitch_4"/>
-	</xacro:if> -->
+	</xacro:if>
 </robot>

File: kyon_urdf/urdf/kyon.urdf (robot description, URDF)
Before this commit: robot kyon, 34 links, 33 joints
Joints:
- joint dagana_1_clamp_joint: limit lower=-3.4056 upper=3.4056 effort=132 velocity=15.5 -> lower=-3.4056 upper=3.4056 effort=25 velocity=14
- joint dagana_2_clamp_joint: limit lower=-3.3266 upper=3.3266 effort=132 velocity=15.5 -> lower=-3.3266 upper=3.3266 effort=25 velocity=14
- joint elbow_pitch_1: limit lower=-3 upper=3 effort=132 velocity=15.5 -> lower=-3 upper=3 effort=122 velocity=4.6
- joint elbow_pitch_2: limit lower=-3 upper=3 effort=132 velocity=15.5 -> lower=-3 upper=3 effort=122 velocity=4.6
- joint hip_pitch_1: limit lower=-2.4056 upper=2.4056 effort=132 velocity=15.5 -> lower=-2.4056 upper=2.4056 effort=185 velocity=7.6
- joint hip_pitch_2: limit lower=-2.3266 upper=2.3266 effort=132 velocity=15.5 -> lower=-2.3266 upper=2.3266 effort=185 velocity=7.6
- joint hip_pitch_3: limit lower=-2.4696 upper=2.4696 effort=132 velocity=15.5 -> lower=-2.4696 upper=2.4696 effort=185 velocity=7.6
- joint hip_pitch_4: limit lower=-2.3426 upper=2.3426 effort=132 velocity=15.5 -> lower=-2.3426 upper=2.3426 effort=185 velocity=7.6
- joint hip_roll_1: limit lower=-2.03 upper=2.51 effort=132 velocity=15.5 -> lower=-2.03 upper=2.51 effort=185 velocity=7.6
- joint hip_roll_2: limit lower=-2.51 upper=2.03 effort=132 velocity=15.5 -> lower=-2.51 upper=2.03 effort=185 velocity=7.6
- joint hip_roll_3: limit lower=-2.51 upper=2.03 effort=132 velocity=15.5 -> lower=-2.51 upper=2.03 effort=185 velocity=7.6
- joint hip_roll_4: limit lower=-2.03 upper=2.51 effort=132 velocity=15.5 -> lower=-2.03 upper=2.51 effort=185 velocity=7.6
- joint knee_pitch_1: limit lower=-3.4056 upper=3.4056 effort=132 velocity=15.5 -> lower=-3.4056 upper=3.4056 effort=185 velocity=7.6
- joint knee_pitch_2: limit lower=-3.3266 upper=3.3266 effort=132 velocity=15.5 -> lower=-3.3266 upper=3.3266 effort=185 velocity=7.6
- joint knee_pitch_3: limit lower=-3.4696 upper=3.4696 effort=132 velocity=15.5 -> lower=-3.4696 upper=3.4696 effort=185 velocity=7.6
- joint knee_pitch_4: limit lower=-3.3426 upper=3.3426 effort=132 velocity=15.5 -> lower=-3.3426 upper=3.3426 effort=185 velocity=7.6
- joint shoulder_pitch_1: limit lower=-3 upper=3 effort=132 velocity=15.5 -> lower=-3 upper=3 effort=122 velocity=4.6
- joint shoulder_pitch_2: limit lower=-3 upper=3 effort=132 velocity=15.5 -> lower=-3 upper=3 effort=122 velocity=4.6
- joint shoulder_yaw_1: limit lower=-3.312 upper=3.312 effort=132 velocity=15.5 -> lower=-3.312 upper=3.312 effort=146 velocity=3.8
- joint shoulder_yaw_2: limit lower=-3.3458 upper=3.3458 effort=132 velocity=15.5 -> lower=-3.3458 upper=3.3458 effort=146 velocity=3.8
- joint wrist_pitch_1: limit lower=-2.4056 upper=2.4056 effort=132 velocity=15.5 -> lower=-2.4056 upper=2.4056 effort=25 velocity=14
- joint wrist_pitch_2: limit lower=-2.3266 upper=2.3266 effort=132 velocity=15.5 -> lower=-2.3266 upper=2.3266 effort=25 velocity=14
- joint wrist_yaw_1: limit lower=-2.4056 upper=2.4056 effort=132 velocity=15.5 -> lower=-2.4056 upper=2.4056 effort=25 velocity=14
- joint wrist_yaw_2: limit lower=-2.3266 upper=2.3266 effort=132 velocity=15.5 -> lower=-2.3266 upper=2.3266 effort=25 velocity=14

File: kyon_urdf/urdf/kyon_base.urdf.xacro (robot description, xacro)
@@ -52,11 +52,11 @@
         depth_width="1280"
         depth_height="720"
-        depth_fps="90"
-        infra_width="1280"
-        infra_height="720"
-        infra_fps="90"
-        color_width="1280"
-        color_height="720"
-        color_fps="30">
+        depth_fps="10"
+        infra_width="1280"
+        infra_height="720"
+        infra_fps="10"
+        color_width="1280"
+        color_height="720"
+        color_fps="1">
         <origin xyz="0 0.150100 0.109486" rpy="0 0.3490656 1.5707963"/>
     </xacro:sensor_d435i>
@@ -73,11 +73,11 @@
         depth_width="1280"
         depth_height="720"
-        depth_fps="90"
-        infra_width="1280"
-        infra_height="720"
-        infra_fps="90"
-        color_width="1280"
-        color_height="720"
-        color_fps="30">
+        depth_fps="10"
+        infra_width="1280"
+        infra_height="720"
+        infra_fps="10"
+        color_width="1280"
+        color_height="720"
+        color_fps="1">
         <origin xyz="0 -0.150100 0.109486" rpy="0 0.3490656 -1.5707963"/>
     </xacro:sensor_d435i>

File: kyon_urdf/urdf/parts/foot_leg.urdf.xacro (robot description, xacro)
@@ -34,5 +34,5 @@
     <parent link="knee_pitch_${leg_num}_link"/>
     <child link="contact_${leg_num}"/>
-    <origin xyz="${-mirror*0.03} -0.35 0.03" rpy="${1.57*mirror} ${0} ${0.785 if mirror == -1 else 2.356}"/>
+    <origin xyz="${-mirror*0.0} -0.3 0.054" rpy="${1.57*mirror} ${0} ${0.785 if mirror == -1 else 2.356}"/>
 </joint>
 </xacro:macro>

Commit message: Signed-off-by: Andrea Patrizi <andreapatrizi1b6e6@gmail.com>

File: kyon_srdf/srdf/kyon.srdf.xacro (robot description, xacro)
@@ -88,4 +88,8 @@
             <joint name="hip_pitch_4" value="0.7"/>
             <joint name="knee_pitch_4" value="-1.4"/>
+            <joint name="wheel_joint_1" value="0"/>
+            <joint name="wheel_joint_2" value="0"/>
+            <joint name="wheel_joint_3" value="0"/>
+            <joint name="wheel_joint_4" value="0"/>
         </xacro:if>
         <xacro:if value="${ADD_UPPER_BODY}">

Commit message: added imu

File: kyon_srdf/srdf/kyon.srdf.xacro (robot description, xacro)
@@ -12,4 +12,7 @@
     <group name="base">
         <link name="pelvis"/>
+    </group>
+    <group name="imu_sensors">
+        <link name="imu_link"/>
     </group>
     <xacro:if value="${ADD_LEGS}">

File: kyon_urdf/urdf/kyon_base.urdf.xacro (robot description, xacro)
@@ -35,4 +35,10 @@
 	</collision>
 </link>
+<link name="imu_link" />
+<joint name="imu_joint" type="fixed">
+    <parent link="pelvis" />
+    <origin xyz="0.0 0.0 0.0" rpy="0.0 0.0 0.0" />
+    <child link="imu_link" />
+</joint>
 <xacro:if value="${ADD_SENSORS}">
     <xacro:include filename="${REALSENSE_GAZEBO_DESCRIPTION_ROOT}/urdf/_d435i.urdf.xacro" />

Commit message: added IMU

File: kyon_srdf/srdf/kyon.srdf.xacro (robot description, xacro)
@@ -12,4 +12,7 @@
     <group name="base">
         <link name="pelvis"/>
+    </group>
+    <group name="imu_sensors">
+        <link name="imu_link"/>
     </group>
     <xacro:if value="${ADD_LEGS}">

Commit message: renames wheel_i_link to wheel_1

File: kyon_srdf/srdf/kyon.srdf.xacro (robot description, xacro)
@@ -14,14 +14,14 @@
     	<xacro:if value="${ADD_WHEELS}">
 			<group name="front_left_leg">
-		        <chain base_link="pelvis" tip_link="wheel_1_link" />
+		        <chain base_link="pelvis" tip_link="wheel_1" />
 		    </group>
 		    <group name="front_right_leg">
-		        <chain base_link="pelvis" tip_link="wheel_2_link" />
+		        <chain base_link="pelvis" tip_link="wheel_2" />
 		    </group>
 		    <group name="rear_right_leg">
-		        <chain base_link="pelvis" tip_link="wheel_4_link" />
+		        <chain base_link="pelvis" tip_link="wheel_4" />
 		    </group>
 		    <group name="rear_left_leg">
-		        <chain base_link="pelvis" tip_link="wheel_3_link" />
+		        <chain base_link="pelvis" tip_link="wheel_3" />
 		    </group>
 		</xacro:if>
@@ -42,14 +42,14 @@
         <xacro:if value="${ADD_STEERING_WHEELS}">
             <group name="front_left_leg">
-                <chain base_link="pelvis" tip_link="wheel_1_link"/>
+                <chain base_link="pelvis" tip_link="wheel_1"/>
             </group>
             <group name="front_right_leg">
-		        <chain base_link="pelvis" tip_link="wheel_2_link" />
+		        <chain base_link="pelvis" tip_link="wheel_2" />
 		    </group>
 		    <group name="rear_right_leg">
-		        <chain base_link="pelvis" tip_link="wheel_4_link" />
+		        <chain base_link="pelvis" tip_link="wheel_4" />
 		    </group>
 		    <group name="rear_left_leg">
-		        <chain base_link="pelvis" tip_link="wheel_3_link" />
+		        <chain base_link="pelvis" tip_link="wheel_3" />
 		    </group>
         </xacro:if>

File: kyon_urdf/urdf/parts/steering_wheel.urdf.xacro (robot description, xacro)
@@ -47,5 +47,5 @@
 	</collision>
 </link>
-<link name="wheel_${leg_num}_link">
+<link name="wheel_${leg_num}">
     <inertial>
 		<origin xyz="${SteeringWheel_x} ${SteeringWheel_y} ${SteeringWheel_z}"/>
@@ -85,5 +85,5 @@
 <joint name="wheel_joint_${leg_num}" type="revolute">
     <parent link="ankle_yaw_${leg_num}_link"/>
-    <child link="wheel_${leg_num}_link"/>
+    <child link="wheel_${leg_num}"/>
     <origin xyz="${SteeringWheel_Ox} ${SteeringWheel_Oy} ${SteeringWheel_Oz}" rpy="${SteeringWheel_roll} ${SteeringWheel_pitch} ${SteeringWheel_yaw}"/>
     <axis xyz="0 0 1"/>

File: kyon_urdf/urdf/parts/wheel_leg.urdf.xacro (robot description, xacro)
@@ -23,5 +23,5 @@
     </collision>
 </link>
-<link name="wheel_${leg_num}_link">
+<link name="wheel_${leg_num}">
     <inertial>
 		<origin xyz="${Wheel_x} ${Wheel_y} ${Wheel_z}"/>
@@ -52,5 +52,5 @@
 <joint name="wheel_joint_${leg_num}" type="revolute">
     <parent link="knee_pitch_${leg_num}_link"/>
-    <child link="wheel_${leg_num}_link"/>
+    <child link="wheel_${leg_num}"/>
     <origin xyz="${Wheel_Ox} ${Wheel_Oy} ${Wheel_Oz}" rpy="${Wheel_roll} ${Wheel_pitch} ${Wheel_yaw}"/>
     <axis xyz="0 0 1"/>

Commit message: add imu to srdf

File: kyon_srdf/srdf/kyon.srdf.xacro (robot description, xacro)
@@ -63,4 +63,7 @@
 		</group>
     </xacro:if>
+    <group name="imu_sensors">
+        <link name="imu_link"/>
+    </group>
     <!-- <xacro:if value="${ADD_FT_SENSORS}">
         <group name="ft_sensors">

Commit message: change axis signs to comply with real robot

File: kyon_srdf/srdf/kyon.srdf.xacro (robot description, xacro)
@@ -107,12 +107,12 @@
         <xacro:if value="${ADD_UPPER_BODY}">
             <joint name="shoulder_yaw_1" value="0.0"/>
-            <joint name="shoulder_pitch_1" value="1.7"/>
-            <joint name="elbow_pitch_1" value="-2.50"/>
-            <joint name="wrist_pitch_1" value="0.75"/>
+            <joint name="shoulder_pitch_1" value="1.0"/>
+            <joint name="elbow_pitch_1" value="2.50"/>
+            <joint name="wrist_pitch_1" value="-0.75"/>
             <joint name="wrist_yaw_1" value="0.0"/>
             <joint name="shoulder_yaw_2" value="0.0"/>
-            <joint name="shoulder_pitch_2" value="-1.70"/>
-            <joint name="elbow_pitch_2" value="2.50"/>
-            <joint name="wrist_pitch_2" value="-0.75"/>
+            <joint name="shoulder_pitch_2" value="-1.0"/>
+            <joint name="elbow_pitch_2" value="-2.50"/>
+            <joint name="wrist_pitch_2" value="0.75"/>
             <joint name="wrist_yaw_2" value="0.0"/>
         </xacro:if>

Commit message: change axis signs to comply with real robot

File: kyon_srdf/srdf/kyon.srdf.xacro (robot description, xacro)
@@ -104,12 +104,12 @@
         <xacro:if value="${ADD_UPPER_BODY}">
             <joint name="shoulder_yaw_1" value="0.0"/>
-            <joint name="shoulder_pitch_1" value="1.7"/>
-            <joint name="elbow_pitch_1" value="-2.50"/>
-            <joint name="wrist_pitch_1" value="0.75"/>
+            <joint name="shoulder_pitch_1" value="1.0"/>
+            <joint name="elbow_pitch_1" value="2.50"/>
+            <joint name="wrist_pitch_1" value="-0.75"/>
             <joint name="wrist_yaw_1" value="0.0"/>
             <joint name="shoulder_yaw_2" value="0.0"/>
-            <joint name="shoulder_pitch_2" value="-1.70"/>
-            <joint name="elbow_pitch_2" value="2.50"/>
-            <joint name="wrist_pitch_2" value="-0.75"/>
+            <joint name="shoulder_pitch_2" value="-1.0"/>
+            <joint name="elbow_pitch_2" value="-2.50"/>
+            <joint name="wrist_pitch_2" value="0.75"/>
             <joint name="wrist_yaw_2" value="0.0"/>
         </xacro:if>

File: kyon_urdf/urdf/parts/kyon_arm.urdf.xacro (robot description, xacro)
@@ -108,5 +108,5 @@
 	<child link="shoulder_yaw_${arm_num}_link"/>
 	<origin xyz="${ShoulderYaw_Ox} ${rot * ShoulderYaw_Oy} ${ShoulderYaw_Oz}" rpy="${rot * ShoulderYaw_roll} ${ShoulderYaw_pitch} ${ShoulderYaw_yaw}"/>
-	<axis xyz="0 0 1"/>
+	<axis xyz="0 0 -1"/>
 	<limit lower="${j_shoulder_yaw_lower[arm_num-1]}" upper="${j_shoulder_yaw_upper[arm_num-1]}" effort="${motorB_effort}" velocity="${motorB_velocity}"/>
 </joint>
@@ -123,5 +123,5 @@
 	<child link="elbow_pitch_${arm_num}_link"/>
 	<origin xyz="${ElbowPitch_Ox} ${ElbowPitch_Oy} ${ElbowPitch_Oz}" rpy="${ElbowPitch_roll} ${ElbowPitch_pitch} ${ElbowPitch_yaw}"/>
-	<axis xyz="0 0 1"/>
+	<axis xyz="0 0 -1"/>
 	<limit lower="${j_pitch_1_lower[arm_num-1]}" upper="${j_pitch_1_upper[arm_num-1]}" effort="${motorC_effort}" velocity="${motorC_velocity}"/>
 </joint>
@@ -130,5 +130,5 @@
 	<child link="wrist_pitch_${arm_num}_link"/>
 	<origin xyz="${WristPitch_Ox} ${WristPitch_Oy} ${WristPitch_Oz}" rpy="${WristPitch_roll} ${WristPitch_pitch} ${WristPitch_yaw}"/>
-	<axis xyz="0 0 1"/>
+	<axis xyz="0 0 -1"/>
 	<limit lower="${j_pitch_2_lower[arm_num-1]}" upper="${j_pitch_2_upper[arm_num-1]}" effort="${motorD_effort}" velocity="${motorD_velocity}"/>
 </joint>

Commit message: added imu and few adjustments in mujoco

File: kyon_srdf/srdf/kyon.srdf.xacro (robot description, xacro)
@@ -10,4 +10,7 @@
     <group name="base">
         <link name="pelvis"/>
+    </group>
+    <group name="imu_sensors">
+        <link name="imu_link"/>
     </group>
     <xacro:if value="${ADD_LEGS}">
