Commit message: ik configs

File: kyon_srdf/srdf/kyon.srdf.xacro (robot description, xacro)
@@ -104,4 +104,32 @@
             <joint name="hip_pitch_4" value="-0.7"/>
             <joint name="knee_pitch_4" value="1.4"/>
+        </xacro:if>
+        <xacro:if value="${ADD_UPPER_BODY}">
+            <joint name="shoulder_yaw_1" value="0.0"/>
+            <joint name="shoulder_pitch_1" value="1.0"/>
+            <joint name="elbow_pitch_1" value="2.50"/>
+            <joint name="wrist_pitch_1" value="-0.75"/>
+            <joint name="wrist_yaw_1" value="0.0"/>
+            <joint name="shoulder_yaw_2" value="0.0"/>
+            <joint name="shoulder_pitch_2" value="-1.0"/>
+            <joint name="elbow_pitch_2" value="-2.50"/>
+            <joint name="wrist_pitch_2" value="0.75"/>
+            <joint name="wrist_yaw_2" value="0.0"/>
+        </xacro:if>
+    </group_state>
+    <group_state name="parked" group="chains">
+        <xacro:if value="${ADD_LEGS}">
+            <joint name="hip_roll_1" value="0.0"/>
+            <joint name="hip_pitch_1" value="1.57"/>
+            <joint name="knee_pitch_1" value="-3.1"/>
+            <joint name="hip_roll_2" value="0.0"/>
+            <joint name="hip_pitch_2" value="-1.57"/>
+            <joint name="knee_pitch_2" value="3.1"/>
+            <joint name="hip_roll_3" value="0.0"/>
+            <joint name="hip_pitch_3" value="1.57"/>
+            <joint name="knee_pitch_3" value="-3.1"/>
+            <joint name="hip_roll_4" value="0.0"/>
+            <joint name="hip_pitch_4" value="-1.57"/>
+            <joint name="knee_pitch_4" value="3.1"/>
         </xacro:if>
         <xacro:if value="${ADD_UPPER_BODY}">

Commit message: parking

File: kyon_srdf/srdf/kyon.srdf.xacro (robot description, xacro)
@@ -114,4 +114,18 @@
             <joint name="wrist_yaw_2" value="0.0"/>
         </xacro:if>
+    </group_state>
+    <group_state name="parked" group="chains">
+        <joint name="hip_roll_1" value="0.0"/>
+        <joint name="hip_pitch_1" value="1.57"/>
+        <joint name="knee_pitch_1" value="-3.10"/>
+        <joint name="hip_roll_2" value="0.0"/>
+        <joint name="hip_pitch_2" value="-1.57"/>
+        <joint name="knee_pitch_2" value="3.1"/>
+        <joint name="hip_roll_3" value="0.0"/>
+        <joint name="hip_pitch_3" value="1.57"/>
+        <joint name="knee_pitch_3" value="-3.1"/>
+        <joint name="hip_roll_4" value="0.0"/>
+        <joint name="hip_pitch_4" value="-1.57"/>
+        <joint name="knee_pitch_4" value="3.1"/>
     </group_state>
     <!--DISABLE COLLISIONS: By default it is assumed that any link of the robot could potentially come into collision with any other link in the robot. This tag disables collision checking between a specified pair of links. -->

Commit message: fix homing signs

File: kyon_srdf/srdf/kyon.srdf.xacro (robot description, xacro)
@@ -57,8 +57,8 @@
     <xacro:if value="${ADD_UPPER_BODY}">
 		<group name="left_arm">
-			<chain base_link="pelvis" tip_link="dagana_1_claw"/>
+			<chain base_link="pelvis" tip_link="wrist_yaw_1_link"/>
 		</group>
 		<group name="right_arm">
-			<chain base_link="pelvis" tip_link="dagana_2_claw"/>
+			<chain base_link="pelvis" tip_link="wrist_yaw_2_link"/>
 		</group>
     </xacro:if>
@@ -90,15 +90,15 @@
         <xacro:if value="${ADD_LEGS}">
             <joint name="hip_roll_1" value="0.0"/>
-            <joint name="hip_pitch_1" value="0.7"/>
-            <joint name="knee_pitch_1" value="-1.4"/>
+            <joint name="hip_pitch_1" value="-0.7"/>
+            <joint name="knee_pitch_1" value="1.4"/>
             <joint name="hip_roll_2" value="0.0"/>
-            <joint name="hip_pitch_2" value="-0.7"/>
-            <joint name="knee_pitch_2" value="1.4"/>
+            <joint name="hip_pitch_2" value="0.7"/>
+            <joint name="knee_pitch_2" value="-1.4"/>
             <joint name="hip_roll_3" value="0.0"/>
-            <joint name="hip_pitch_3" value="0.7"/>
-            <joint name="knee_pitch_3" value="-1.4"/>
+            <joint name="hip_pitch_3" value="-0.7"/>
+            <joint name="knee_pitch_3" value="1.4"/>
             <joint name="hip_roll_4" value="0.0"/>
-            <joint name="hip_pitch_4" value="-0.7"/>
-            <joint name="knee_pitch_4" value="1.4"/>
+            <joint name="hip_pitch_4" value="0.7"/>
+            <joint name="knee_pitch_4" value="-1.4"/>
         </xacro:if>
         <xacro:if value="${ADD_UPPER_BODY}">

Commit message: fix parking signs

File: kyon_srdf/srdf/kyon.srdf.xacro (robot description, xacro)
@@ -117,15 +117,15 @@
     <group_state name="parked" group="chains">
         <joint name="hip_roll_1" value="0.0"/>
-        <joint name="hip_pitch_1" value="1.57"/>
-        <joint name="knee_pitch_1" value="-3.10"/>
+        <joint name="hip_pitch_1" value="-1.57"/>
+        <joint name="knee_pitch_1" value="3.10"/>
         <joint name="hip_roll_2" value="0.0"/>
-        <joint name="hip_pitch_2" value="-1.57"/>
-        <joint name="knee_pitch_2" value="3.1"/>
+        <joint name="hip_pitch_2" value="1.57"/>
+        <joint name="knee_pitch_2" value="-3.1"/>
         <joint name="hip_roll_3" value="0.0"/>
-        <joint name="hip_pitch_3" value="1.57"/>
-        <joint name="knee_pitch_3" value="-3.1"/>
+        <joint name="hip_pitch_3" value="-1.57"/>
+        <joint name="knee_pitch_3" value="3.1"/>
         <joint name="hip_roll_4" value="0.0"/>
-        <joint name="hip_pitch_4" value="-1.57"/>
-        <joint name="knee_pitch_4" value="3.1"/>
+        <joint name="hip_pitch_4" value="1.57"/>
+        <joint name="knee_pitch_4" value="-3.1"/>
     </group_state>
     <!--DISABLE COLLISIONS: By default it is assumed that any link of the robot could potentially come into collision with any other link in the robot. This tag disables collision checking between a specified pair of links. -->

Commit message: corrected motor axis

File: kyon_srdf/srdf/kyon.srdf.xacro (robot description, xacro)
@@ -93,26 +93,26 @@
         <xacro:if value="${ADD_LEGS}">
             <joint name="hip_roll_1" value="0.0"/>
-            <joint name="hip_pitch_1" value="0.7"/>
-            <joint name="knee_pitch_1" value="-1.4"/>
+            <joint name="hip_pitch_1" value="-0.7"/>
+            <joint name="knee_pitch_1" value="1.4"/>
             <joint name="hip_roll_2" value="0.0"/>
-            <joint name="hip_pitch_2" value="-0.7"/>
-            <joint name="knee_pitch_2" value="1.4"/>
+            <joint name="hip_pitch_2" value="0.7"/>
+            <joint name="knee_pitch_2" value="-1.4"/>
             <joint name="hip_roll_3" value="0.0"/>
-            <joint name="hip_pitch_3" value="0.7"/>
-            <joint name="knee_pitch_3" value="-1.4"/>
+            <joint name="hip_pitch_3" value="-0.7"/>
+            <joint name="knee_pitch_3" value="1.4"/>
             <joint name="hip_roll_4" value="0.0"/>
-            <joint name="hip_pitch_4" value="-0.7"/>
-            <joint name="knee_pitch_4" value="1.4"/>
+            <joint name="hip_pitch_4" value="0.7"/>
+            <joint name="knee_pitch_4" value="-1.4"/>
         </xacro:if>
         <xacro:if value="${ADD_UPPER_BODY}">
             <joint name="shoulder_yaw_1" value="0.0"/>
-            <joint name="shoulder_pitch_1" value="1.0"/>
-            <joint name="elbow_pitch_1" value="2.50"/>
-            <joint name="wrist_pitch_1" value="-0.75"/>
+            <joint name="shoulder_pitch_1" value="1.57"/>
+            <joint name="elbow_pitch_1" value="0.0"/>
+            <joint name="wrist_pitch_1" value="0.0"/>
             <joint name="wrist_yaw_1" value="0.0"/>
             <joint name="shoulder_yaw_2" value="0.0"/>
-            <joint name="shoulder_pitch_2" value="-1.0"/>
-            <joint name="elbow_pitch_2" value="-2.50"/>
-            <joint name="wrist_pitch_2" value="0.75"/>
+            <joint name="shoulder_pitch_2" value="-1.57"/>
+            <joint name="elbow_pitch_2" value="0.0"/>
+            <joint name="wrist_pitch_2" value="0.0"/>
             <joint name="wrist_yaw_2" value="0.0"/>
         </xacro:if>

File: kyon_urdf/urdf/parts/steering_wheel.urdf.xacro (robot description, xacro)
@@ -73,5 +73,5 @@
     <child link="knee_pitch_${leg_num}_link"/>
     <origin xyz="${KneePitch_Ox} ${KneePitch_Oy} ${KneePitch_Oz}" rpy="${KneePitch_roll} ${KneePitch_pitch} ${KneePitch_yaw}"/>
-    <axis xyz="0 0 1"/>
+    <axis xyz="0 0 -1"/>
     <limit lower="${knee_pitch_lower[leg_num-1]}" upper="${knee_pitch_upper[leg_num-1]}" effort="${motorA_effort}" velocity="${motorA_velocity}"/>
 </joint>
@@ -88,5 +88,5 @@
     <origin xyz="${SteeringWheel_Ox} ${SteeringWheel_Oy} ${SteeringWheel_Oz}" rpy="${SteeringWheel_roll} ${SteeringWheel_pitch} ${SteeringWheel_yaw}"/>
     <axis xyz="0 0 1"/>
-    <limit lower="${knee_pitch_lower[leg_num-1]}" upper="${knee_pitch_upper[leg_num-1]}" effort="${motorWheel_effort}" velocity="${motorWheel_velocity}"/>
+    <limit lower="-1e9" upper="1e9" effort="${motorWheel_effort}" velocity="${motorWheel_velocity}"/>
 </joint>
 </xacro:macro>

File: kyon_urdf/urdf/parts/wheel_leg.urdf.xacro (robot description, xacro)
@@ -49,5 +49,5 @@
     <child link="knee_pitch_${leg_num}_link"/>
     <origin xyz="${KneePitch_Ox} ${KneePitch_Oy} ${KneePitch_Oz}" rpy="${KneePitch_roll} ${KneePitch_pitch} ${KneePitch_yaw}"/>
-    <axis xyz="0 0 1"/>
+    <axis xyz="0 0 -1"/>
     <limit lower="${knee_pitch_lower[leg_num-1]}" upper="${knee_pitch_upper[leg_num-1]}" effort="${motorA_effort}" velocity="${motorA_velocity}"/>
 </joint>

Commit message: naruto pose

File: kyon_srdf/srdf/kyon.srdf.xacro (robot description, xacro)
@@ -128,4 +128,16 @@
         <joint name="hip_pitch_4" value="1.57"/>
         <joint name="knee_pitch_4" value="-3.1"/>
+    </group_state>
+    <group_state name="naruto" group="chains">
+        <joint name="shoulder_yaw_1" value="0.0"/>
+        <joint name="shoulder_pitch_1" value="1.68"/>
+        <joint name="elbow_pitch_1" value="0.1"/>
+        <joint name="wrist_pitch_1" value="0.8"/>
+        <joint name="wrist_yaw_1" value="0.0"/>
+        <joint name="shoulder_yaw_2" value="0.0"/>
+        <joint name="shoulder_pitch_2" value="-1.68"/>
+        <joint name="elbow_pitch_2" value="-0.1"/>
+        <joint name="wrist_pitch_2" value="-0.8"/>
+        <joint name="wrist_yaw_2" value="0.0"/>
     </group_state>
     <!--DISABLE COLLISIONS: By default it is assumed that any link of the robot could potentially come into collision with any other link in the robot. This tag disables collision checking between a specified pair of links. -->

Commit message: add dagana option

File: kyon_srdf/srdf/kyon.srdf.xacro (robot description, xacro)
@@ -46,8 +46,18 @@
     <xacro:if value="${ADD_UPPER_BODY}">
 		<group name="left_arm">
-			<chain base_link="pelvis" tip_link="dagana_1_claw"/>
+            <xacro:if value="${ADD_DAGANA}">
+			    <chain base_link="pelvis" tip_link="dagana_1_claw"/>
+            </xacro:if>
+            <xacro:unless value="${ADD_DAGANA}">
+                <chain base_link="pelvis" tip_link="wrist_yaw_1_link"/>
+            </xacro:unless>
 		</group>
 		<group name="right_arm">
-			<chain base_link="pelvis" tip_link="dagana_2_claw"/>
+            <xacro:if value="${ADD_DAGANA}">
+			    <chain base_link="pelvis" tip_link="dagana_2_claw"/>
+            </xacro:if>
+            <xacro:unless value="${ADD_DAGANA}">
+                <chain base_link="pelvis" tip_link="wrist_yaw_2_link"/>
+            </xacro:unless>
 		</group>
     </xacro:if>

File: kyon_urdf/urdf/config/kyon.urdf.xacro (robot description, xacro)
@@ -13,8 +13,10 @@
 <xacro:arg name="d034_li_ion" default="false"/>
 <xacro:arg name="velodyne" default="false"/>
+<xacro:arg name="dagana" default="$(arg upper_body)"/>
 <!-- ************SELECT PARTS*************-->
 <!-- *************************************-->
 <xacro:property name="ADD_LEGS" value="$(arg legs)"/>
 <xacro:property name="ADD_UPPER_BODY" value="$(arg upper_body)"/>
+<xacro:property name="ADD_DAGANA" value="$(arg dagana)"/>
 <xacro:property name="ADD_CAMERAS" value="$(arg cameras)"/>
 <xacro:property name="ADD_WHEELS" value="$(arg wheels)"/>

File: kyon_urdf/urdf/parts/kyon_arm.urdf.xacro (robot description, xacro)
@@ -148,5 +148,7 @@
 	<limit lower="${j_pitch_2_lower[arm_num-1]}" upper="${j_pitch_2_upper[arm_num-1]}" effort="${motorD_effort}" velocity="${motorD_velocity}"/>
 </joint>
-<xacro:kyon_dagana arm_num="${arm_num}" parent="wrist_yaw_${arm_num}_link"/>
+<xacro:if value="${ADD_DAGANA}">
+	<xacro:kyon_dagana arm_num="${arm_num}" parent="wrist_yaw_${arm_num}_link"/>
+</xacro:if>
 </xacro:macro>
 <!-- /macro arms -->

Commit message: a homing for the up that makes sense

File: kyon_srdf/srdf/kyon.srdf.xacro (robot description, xacro)
@@ -98,12 +98,12 @@
         <xacro:if value="${ADD_UPPER_BODY}">
             <joint name="shoulder_yaw_1" value="0.0"/>
-            <joint name="shoulder_pitch_1" value="1.57"/>
-            <joint name="elbow_pitch_1" value="0.0"/>
-            <joint name="wrist_pitch_1" value="0.0"/>
+            <joint name="shoulder_pitch_1" value="1.6"/>
+            <joint name="elbow_pitch_1" value="2.5"/>
+            <joint name="wrist_pitch_1" value="0.7"/>
             <joint name="wrist_yaw_1" value="0.0"/>
             <joint name="shoulder_yaw_2" value="0.0"/>
-            <joint name="shoulder_pitch_2" value="-1.57"/>
-            <joint name="elbow_pitch_2" value="0.0"/>
-            <joint name="wrist_pitch_2" value="0.0"/>
+            <joint name="shoulder_pitch_2" value="-1.6"/>
+            <joint name="elbow_pitch_2" value="-2.5"/>
+            <joint name="wrist_pitch_2" value="-0.7"/>
             <joint name="wrist_yaw_2" value="0.0"/>
         </xacro:if>

Commit message: fixed homing ;P

File: kyon_srdf/srdf/kyon.srdf.xacro (robot description, xacro)
@@ -98,11 +98,11 @@
         <xacro:if value="${ADD_UPPER_BODY}">
             <joint name="shoulder_yaw_1" value="0.0"/>
-            <joint name="shoulder_pitch_1" value="1.6"/>
-            <joint name="elbow_pitch_1" value="2.5"/>
+            <joint name="shoulder_pitch_1" value="1.5"/>
+            <joint name="elbow_pitch_1" value="2.6"/>
             <joint name="wrist_pitch_1" value="0.7"/>
             <joint name="wrist_yaw_1" value="0.0"/>
             <joint name="shoulder_yaw_2" value="0.0"/>
-            <joint name="shoulder_pitch_2" value="-1.6"/>
-            <joint name="elbow_pitch_2" value="-2.5"/>
+            <joint name="shoulder_pitch_2" value="-1.5"/>
+            <joint name="elbow_pitch_2" value="-2.6"/>
             <joint name="wrist_pitch_2" value="-0.7"/>
             <joint name="wrist_yaw_2" value="0.0"/>

Commit message: parking signs

File: kyon_srdf/srdf/kyon.srdf.xacro (robot description, xacro)
@@ -111,15 +111,15 @@
     <group_state name="parked" group="chains">
         <joint name="hip_roll_1" value="0.0"/>
-        <joint name="hip_pitch_1" value="1.57"/>
-        <joint name="knee_pitch_1" value="-3.10"/>
+        <joint name="hip_pitch_1" value="-1.57"/>
+        <joint name="knee_pitch_1" value="3.10"/>
         <joint name="hip_roll_2" value="0.0"/>
-        <joint name="hip_pitch_2" value="-1.57"/>
-        <joint name="knee_pitch_2" value="3.1"/>
+        <joint name="hip_pitch_2" value="1.57"/>
+        <joint name="knee_pitch_2" value="-3.1"/>
         <joint name="hip_roll_3" value="0.0"/>
-        <joint name="hip_pitch_3" value="1.57"/>
-        <joint name="knee_pitch_3" value="-3.1"/>
+        <joint name="hip_pitch_3" value="-1.57"/>
+        <joint name="knee_pitch_3" value="3.1"/>
         <joint name="hip_roll_4" value="0.0"/>
-        <joint name="hip_pitch_4" value="-1.57"/>
-        <joint name="knee_pitch_4" value="3.1"/>
+        <joint name="hip_pitch_4" value="1.57"/>
+        <joint name="knee_pitch_4" value="-3.1"/>
     </group_state>
     <!--DISABLE COLLISIONS: By default it is assumed that any link of the robot could potentially come into collision with any other link in the robot. This tag disables collision checking between a specified pair of links. -->

Commit message: upd ub homing

File: kyon_srdf/srdf/kyon.srdf.xacro (robot description, xacro)
@@ -98,12 +98,12 @@
         <xacro:if value="${ADD_UPPER_BODY}">
             <joint name="shoulder_yaw_1" value="0.0"/>
-            <joint name="shoulder_pitch_1" value="1.5"/>
-            <joint name="elbow_pitch_1" value="2.6"/>
-            <joint name="wrist_pitch_1" value="0.7"/>
+            <joint name="shoulder_pitch_1" value="1.0"/>
+            <joint name="elbow_pitch_1" value="2.0"/>
+            <joint name="wrist_pitch_1" value="0.5"/>
             <joint name="wrist_yaw_1" value="0.0"/>
             <joint name="shoulder_yaw_2" value="0.0"/>
-            <joint name="shoulder_pitch_2" value="-1.5"/>
-            <joint name="elbow_pitch_2" value="-2.6"/>
-            <joint name="wrist_pitch_2" value="-0.7"/>
+            <joint name="shoulder_pitch_2" value="-1.0"/>
+            <joint name="elbow_pitch_2" value="-2.0"/>
+            <joint name="wrist_pitch_2" value="-0.5"/>
             <joint name="wrist_yaw_2" value="0.0"/>
         </xacro:if>

Commit message: amentized urdf and srdf packages

File: kyon_srdf/srdf/kyon.srdf.xacro (robot description, xacro)
@@ -6,5 +6,7 @@
 <robot xmlns:xacro="http://ros.org/wiki/xacro" name="kyon">
     <!-- ************ MODEL CONFIGURATION ************ -->
-    <xacro:arg name="config" default="$(find kyon_urdf)/urdf/config/kyon.urdf.xacro"/>
+    <xacro:arg name="root" default="$(find kyon_urdf)" />
+    <xacro:property name="ROOT" value="$(arg root)" />
+    <xacro:arg name="config" default="${ROOT}/urdf/config/kyon.urdf.xacro"/>
     <xacro:include filename="$(arg config)"/>
     <group name="base">
