Commit message: Signed-off-by: Andrea Patrizi <andreapatrizi1b6e6@gmail.com>

File: kyon_srdf/srdf/kyon.srdf.xacro (robot description, xacro)
@@ -4,7 +4,7 @@
     A URDF file must exist for this robot as well, where the joints and the links that are referenced are defined
 -->
-<robot xmlns:xacro="http://ros.org/wiki/xacro" name="kyon">
+<robot xmlns:xacro="http://ros.org/wiki/xacro" name="kyon_real">
     <!-- ************ MODEL CONFIGURATION ************ -->
-    <xacro:arg name="root" default="$(find kyon_urdf)" />
+    <xacro:arg name="root" default="${ROOT}" />
     <xacro:property name="ROOT" value="$(arg root)" />
     <xacro:arg name="config" default="${ROOT}/urdf/config/kyon.urdf.xacro"/>

File: kyon_urdf/urdf/kyon.urdf (robot description, URDF)
Before this commit: robot kyon, 96 links, 95 joints
Links:
- link ankle_yaw_1_link: geometry collision mesh filename=${MESH_PATH}/collision/mesh_ankle-yaw.stl scale=0.001 0.001 0.001; visual mesh filename=${MESH_PATH}/mesh_ankle-yaw.stl scale=0.001 0.001 0.001
- link ankle_yaw_2_link: geometry collision mesh filename=${MESH_PATH}/collision/mesh_ankle-yaw.stl scale=0.001 0.001 0.001; visual mesh filename=${MESH_PATH}/mesh_ankle-yaw.stl scale=0.001 0.001 0.001
- link ankle_yaw_3_link: geometry collision mesh filename=${MESH_PATH}/collision/mesh_ankle-yaw.stl scale=0.001 0.001 0.001; visual mesh filename=${MESH_PATH}/mesh_ankle-yaw.stl scale=0.001 0.001 0.001
- link ankle_yaw_4_link: geometry collision mesh filename=${MESH_PATH}/collision/mesh_ankle-yaw.stl scale=0.001 0.001 0.001; visual mesh filename=${MESH_PATH}/mesh_ankle-yaw.stl scale=0.001 0.001 0.001
- link dagana_1_base: geometry collision mesh filename=${MESH_PATH}/collision/mesh_dagana-base-base-simplified.stl scale=0.001 0.001 0.001; collision mesh filename=${MESH_PATH}/collision/mesh_dagana-base-simplified.stl scale=0.001 0.001 0.001
- link dagana_1_claw: geometry collision mesh filename=${MESH_PATH}/collision/mesh_dagana-clamp-base-simplified.stl scale=0.001 0.001 0.001; collision mesh filename=${MESH_PATH}/collision/mesh_dagana-clamp-simplified.stl scale=0.001 0.001 0.001
- link dagana_2_base: geometry collision mesh filename=${MESH_PATH}/collision/mesh_dagana-base-base-simplified.stl scale=0.001 0.001 0.001; collision mesh filename=${MESH_PATH}/collision/mesh_dagana-base-simplified.stl scale=0.001 0.001 0.001
- link dagana_2_claw: geometry collision mesh filename=${MESH_PATH}/collision/mesh_dagana-clamp-base-simplified.stl scale=0.001 0.001 0.001; collision mesh filename=${MESH_PATH}/collision/mesh_dagana-clamp-simplified.stl scale=0.001 0.001 0.001
- link elbow_pitch_1_link: geometry collision mesh filename=${MESH_PATH}/mesh_elbow.stl scale=0.001 0.001 0.001; visual mesh filename=${MESH_PATH}/mesh_elbow.stl scale=0.001 0.001 0.001
- link elbow_pitch_2_link: geometry collision mesh filename=${MESH_PATH}/mesh_elbow.stl scale=0.001 0.001 0.001; visual mesh filename=${MESH_PATH}/mesh_elbow.stl scale=0.001 0.001 0.001
- link hip_pitch_1_link: geometry collision mesh filename=${MESH_PATH}/collision/mesh_hip-pitch.stl scale=0.001 0.001 0.001; visual mesh filename=${MESH_PATH}/mesh_hip-pitch.stl scale=0.001 0.001 0.001
- link hip_pitch_2_link: geometry collision mesh filename=${MESH_PATH}/collision/mesh_hip-pitch.stl scale=0.001 0.001 0.001; visual mesh filename=${MESH_PATH}/mesh_hip-pitch.stl scale=0.001 0.001 0.001
- link hip_pitch_3_link: geometry collision mesh filename=${MESH_PATH}/collision/mesh_hip-pitch.stl scale=0.001 0.001 0.001; visual mesh filename=${MESH_PATH}/mesh_hip-pitch.stl scale=0.001 0.001 0.001
- link hip_pitch_4_link: geometry collision mesh filename=${MESH_PATH}/collision/mesh_hip-pitch.stl scale=0.001 0.001 0.001; visual mesh filename=${MESH_PATH}/mesh_hip-pitch.stl scale=0.001 0.001 0.001
- link hip_roll_1_link: geometry collision mesh filename=${MESH_PATH}/collision/mesh_hip-roll.stl scale=0.001 -0.001 0.001; visual mesh filename=${MESH_PATH}/mesh_hip-roll.stl scale=0.001 -0.001 0.001
- link hip_roll_2_link: geometry collision mesh filename=${MESH_PATH}/collision/mesh_hip-roll.stl scale=0.001 0.001 0.001; visual mesh filename=${MESH_PATH}/mesh_hip-roll.stl scale=0.001 0.001 0.001
- link hip_roll_3_link: geometry collision mesh filename=${MESH_PATH}/collision/mesh_hip-roll.stl scale=0.001 -0.001 0.001; visual mesh filename=${MESH_PATH}/mesh_hip-roll.stl scale=0.001 -0.001 0.001
- link hip_roll_4_link: geometry collision mesh filename=${MESH_PATH}/collision/mesh_hip-roll.stl scale=0.001 0.001 0.001; visual mesh filename=${MESH_PATH}/mesh_hip-roll.stl scale=0.001 0.001 0.001
- link knee_pitch_1_link: geometry collision mesh filename=${MESH_PATH}/collision/mesh_knee-steering.stl scale=0.001 0.001 0.001; visual mesh filename=${MESH_PATH}/mesh_knee-steering.stl scale=0.001 0.001 0.001
- link knee_pitch_2_link: geometry collision mesh filename=${MESH_PATH}/collision/mesh_knee-steering.stl scale=0.001 0.001 0.001; visual mesh filename=${MESH_PATH}/mesh_knee-steering.stl scale=0.001 0.001 0.001
- link knee_pitch_3_link: geometry collision mesh filename=${MESH_PATH}/collision/mesh_knee-steering.stl scale=0.001 0.001 0.001; visual mesh filename=${MESH_PATH}/mesh_knee-steering.stl scale=0.001 0.001 0.001
- link knee_pitch_4_link: geometry collision mesh filename=${MESH_PATH}/collision/mesh_knee-steering.stl scale=0.001 0.001 0.001; visual mesh filename=${MESH_PATH}/mesh_knee-steering.stl scale=0.001 0.001 0.001
- link pelvis: geometry collision mesh filename=${MESH_PATH}/collision/mesh_pelvis.stl scale=0.001 0.001 0.001; visual mesh filename=${MESH_PATH}/mesh_pelvis.stl scale=0.001 0.001 0.001
- link shoulder_pitch_1_link: geometry collision mesh filename=${MESH_PATH}/collision/mesh_sh-pitch.stl scale=0.001 0.001 0.001; visual mesh filename=${MESH_PATH}/mesh_sh-pitch.stl scale=0.001 0.001 0.001
- link shoulder_pitch_2_link: geometry collision mesh filename=${MESH_PATH}/collision/mesh_sh-pitch.stl scale=0.001 0.001 0.001; visual mesh filename=${MESH_PATH}/mesh_sh-pitch.stl scale=0.001 0.001 0.001
- link shoulder_yaw_1_link: geometry collision mesh filename=${MESH_PATH}/collision/mesh_sh-yaw.stl scale=0.001 0.001 0.001; visual mesh filename=${MESH_PATH}/mesh_sh-yaw.stl scale=0.001 0.001 0.001
- link shoulder_yaw_2_link: geometry collision mesh filename=${MESH_PATH}/collision/mesh_sh-yaw.stl scale=0.001 0.001 0.001; visual mesh filename=${MESH_PATH}/mesh_sh-yaw.stl scale=0.001 0.001 0.001
- link wheel_1: geometry collision mesh filename=${MESH_PATH}/collision/mesh_wheel.stl scale=0.001 0.001 0.001; visual mesh filename=${MESH_PATH}/mesh_wheel.stl scale=0.001 0.001 0.001
- link wheel_2: geometry collision mesh filename=${MESH_PATH}/collision/mesh_wheel.stl scale=0.001 0.001 0.001; visual mesh filename=${MESH_PATH}/mesh_wheel.stl scale=0.001 0.001 0.001
- link wheel_3: geometry collision mesh filename=${MESH_PATH}/collision/mesh_wheel.stl scale=0.001 0.001 0.001; visual mesh filename=${MESH_PATH}/mesh_wheel.stl scale=0.001 0.001 0.001
- link wheel_4: geometry collision mesh filename=${MESH_PATH}/collision/mesh_wheel.stl scale=0.001 0.001 0.001; visual mesh filename=${MESH_PATH}/mesh_wheel.stl scale=0.001 0.001 0.001
- link wrist_pitch_1_link: geometry collision mesh filename=${MESH_PATH}/collision/mesh_wrist-pitch.stl scale=0.001 0.001 0.001; visual mesh filename=${MESH_PATH}/mesh_wrist-pitch.stl scale=0.001 0.001 0.001
- link wrist_pitch_2_link: geometry collision mesh filename=${MESH_PATH}/collision/mesh_wrist-pitch.stl scale=0.001 0.001 0.001; visual mesh filename=${MESH_PATH}/mesh_wrist-pitch.stl scale=0.001 0.001 0.001
- link wrist_yaw_1_link: geometry collision mesh filename=${MESH_PATH}/collision/mesh_wrist-yaw.stl scale=0.001 0.001 0.001; visual mesh filename=${MESH_PATH}/mesh_wrist-yaw.stl scale=0.001 0.001 0.001
- link wrist_yaw_2_link: geometry collision mesh filename=${MESH_PATH}/collision/mesh_wrist-yaw.stl scale=0.001 0.001 0.001; visual mesh filename=${MESH_PATH}/mesh_wrist-yaw.stl scale=0.001 0.001 0.001

File: kyon_urdf/urdf/kyon.urdf.xacro (robot description, xacro)
@@ -1,9 +1,29 @@
 <?xml version="1.0"?>
-<robot xmlns:xacro="http://ros.org/wiki/xacro" name="kyon">
-<xacro:arg name="config" default="$(find kyon_urdf)/urdf/config/kyon.urdf.xacro"/>
+<robot xmlns:xacro="http://ros.org/wiki/xacro" name="kyon_real">
+<xacro:arg name="root" default="${ROOT}" />
+<xacro:property name="ROOT" value="$(arg root)" />
+<!-- setting use_abs_mesh_paths should be kept to false
+for use with tools like RViz, which does not accept plain
+abolute paths for mesh paths-->
+<xacro:arg name="use_abs_mesh_paths" default="false" />
+<xacro:arg name="use_local_filesys_for_meshes" default="false" />
+<xacro:property name="USE_ABS_MESH_PATHS" value="$(arg use_abs_mesh_paths)" />
+<xacro:property name="USE_LOCAL_FILESYS_FOR_MESHES" value="$(arg use_local_filesys_for_meshes)" />
+<xacro:if value="${USE_ABS_MESH_PATHS}">
+	<xacro:if value="${USE_LOCAL_FILESYS_FOR_MESHES}">
+	<xacro:property name="MESH_PATH" value="file://${ROOT}/meshes" />
+	</xacro:if>
+	<xacro:unless value="${USE_LOCAL_FILESYS_FOR_MESHES}">
+	<xacro:property name="MESH_PATH" value="${ROOT}/meshes" />
+	</xacro:unless>
+	</xacro:if>
+<xacro:unless value="${USE_ABS_MESH_PATHS}">
+<xacro:property name="MESH_PATH" value="package://kyon_urdf_simple/meshes" />
+</xacro:unless>
+<xacro:arg name="config" default="${ROOT}/urdf/config/kyon.urdf.xacro"/>
 <!-- ************ MODEL CONFIGURATION ************ -->
 <xacro:include filename="$(arg config)"/>
 <!-- ************ CETC-SAT plain model ************ -->
-<xacro:include filename="$(find kyon_urdf)/urdf/kyon_base.urdf.xacro"/>
+<xacro:include filename="${ROOT}/urdf/kyon_base.urdf.xacro"/>
 <!-- ************ Control frames ************ -->
 <!--xacro:include filename="$(find pholus_urdf)/urdf/control_frames.urdf.xacro"/-->

File: kyon_urdf/urdf/kyon_base.urdf.xacro (robot description, xacro)
@@ -1,11 +1,11 @@
 <?xml version="1.0"?>
-<robot xmlns:xacro="http://ros.org/wiki/xacro" name="kyon">
+<robot xmlns:xacro="http://ros.org/wiki/xacro" name="kyon_real">
 <xacro:arg name="bilevel_codes" default="false" /> <!-- if true, load codes vars from externally provided files-->
 <xacro:arg name="sample_idx" default = "0"/>
-<xacro:include filename="$(find kyon_urdf)/urdf/utils.urdf.xacro" />
-<xacro:include filename="$(find kyon_urdf)/urdf/parts/kinematics_properties.urdf.xacro" />
+<xacro:include filename="${ROOT}/urdf/utils.urdf.xacro" />
+<xacro:include filename="${ROOT}/urdf/parts/kinematics_properties.urdf.xacro" />
 <!-- NOTE: here we need to include "kinematics_properties" first because "inertial_properties" depends on it-->
-<xacro:include filename="$(find kyon_urdf)/urdf/parts/inertial_properties.urdf.xacro" />
-<xacro:include filename="$(find kyon_urdf)/urdf/parts/limits.urdf.xacro" />
+<xacro:include filename="${ROOT}/urdf/parts/inertial_properties.urdf.xacro" />
+<xacro:include filename="${ROOT}/urdf/parts/limits.urdf.xacro" />
 <link name="base_link"/>
 <link name="pelvis">
@@ -18,5 +18,5 @@
 		<origin xyz="0.0 0 0.0"  rpy="0.0 0.0 0.0"/>
 		<geometry>
-	 		<mesh filename="package://kyon_urdf/meshes/mesh_pelvis.stl" scale="0.001 0.001 0.001"/>
+	 		<mesh filename="${MESH_PATH}/mesh_pelvis.stl" scale="0.001 0.001 0.001"/>
 		</geometry>
         <material name="dark_grey"/>
@@ -25,5 +25,5 @@
 		<origin xyz="0.0 0 0.0"  rpy="0.0 0.0 0.0"/>
 		<geometry>
-	  		<mesh filename="package://kyon_urdf/meshes/collision/mesh_pelvis.stl" scale="0.001 0.001 0.001"/>
+	  		<mesh filename="${MESH_PATH}/collision/mesh_pelvis.stl" scale="0.001 0.001 0.001"/>
 		</geometry>
 	</collision>
@@ -185,8 +185,8 @@
 </xacro:if>
 <xacro:if value="${ADD_UPPER_BODY}">
-    <xacro:include filename="$(find kyon_urdf)/urdf/parts/arms.urdf.xacro" />
+    <xacro:include filename="${ROOT}/urdf/parts/arms.urdf.xacro" />
 </xacro:if>
 <xacro:if value="${ADD_LEGS}">
-	<xacro:include filename="$(find kyon_urdf)/urdf/parts/legs.urdf.xacro" />
+	<xacro:include filename="${ROOT}/urdf/parts/legs.urdf.xacro" />
 </xacro:if>
 <xacro:if value="${PAYLOAD}">

File: kyon_urdf/urdf/kyon_capsule.urdf (robot description, URDF)
Before this commit: robot kyon, 34 links, 33 joints
Links:
- link dagana_1_base: geometry collision cylinder length=0.11025894047123985 radius=0.0591263; collision sphere radius=0.0591263
- link dagana_1_claw: geometry collision cylinder length=0.10583385976657057 radius=0.0524951; collision sphere radius=0.0524951
- link dagana_2_base: geometry collision cylinder length=0.11025894047123985 radius=0.0591263; collision sphere radius=0.0591263
- link dagana_2_claw: geometry collision cylinder length=0.10583385976657057 radius=0.0524951; collision sphere radius=0.0524951
- link elbow_pitch_1_link: geometry collision cylinder length=0.23685382242349062 radius=0.0581584; collision sphere radius=0.0581584
- link elbow_pitch_2_link: geometry collision cylinder length=0.23685382242349062 radius=0.0581584; collision sphere radius=0.0581584
- link hip_pitch_1_link: geometry collision cylinder length=0.3004661110170414 radius=0.110589; collision sphere radius=0.110589
- link hip_pitch_2_link: geometry collision cylinder length=0.3004661110170414 radius=0.110589; collision sphere radius=0.110589
- link hip_pitch_3_link: geometry collision cylinder length=0.3004661110170414 radius=0.110589; collision sphere radius=0.110589
- link hip_pitch_4_link: geometry collision cylinder length=0.3004661110170414 radius=0.110589; collision sphere radius=0.110589
- link hip_roll_1_link: geometry collision cylinder length=0.14024696973705567 radius=0.0763481; collision sphere radius=0.0763481
- link hip_roll_2_link: geometry collision cylinder length=0.1402469697370549 radius=0.0763481; collision sphere radius=0.0763481
- link hip_roll_3_link: geometry collision cylinder length=0.14024696973705567 radius=0.0763481; collision sphere radius=0.0763481
- link hip_roll_4_link: geometry collision cylinder length=0.1402469697370549 radius=0.0763481; collision sphere radius=0.0763481
- link knee_pitch_1_link: geometry collision cylinder length=0.3150057312682306 radius=0.0400971; collision sphere radius=0.0400971
- link knee_pitch_2_link: geometry collision cylinder length=0.3150057312682306 radius=0.0400971; collision sphere radius=0.0400971
- link knee_pitch_3_link: geometry collision cylinder length=0.3150057312682306 radius=0.0400971; collision sphere radius=0.0400971
- link knee_pitch_4_link: geometry collision cylinder length=0.3150057312682306 radius=0.0400971; collision sphere radius=0.0400971
- link pelvis: geometry collision cylinder length=0.749376 radius=0.1724; collision sphere radius=0.1724
- link shoulder_pitch_1_link: geometry collision cylinder length=0.3306767492610326 radius=0.0630719; collision sphere radius=0.0630719
- link shoulder_pitch_2_link: geometry collision cylinder length=0.3306767492610326 radius=0.0630719; collision sphere radius=0.0630719
- link shoulder_yaw_1_link: geometry collision cylinder length=0.06680404009166907 radius=0.0700029; collision sphere radius=0.0700029
- link shoulder_yaw_2_link: geometry collision cylinder length=0.06680404009166907 radius=0.0700029; collision sphere radius=0.0700029
- link wrist_pitch_1_link: geometry collision cylinder length=0.07557658310998112 radius=0.0522867; collision sphere radius=0.0522867
- link wrist_pitch_2_link: geometry collision cylinder length=0.07557658310998112 radius=0.0522867; collision sphere radius=0.0522867
- link wrist_yaw_1_link: geometry collision cylinder length=0.00015248374465266922 radius=0.0436334; collision sphere radius=0.0436334
- link wrist_yaw_2_link: geometry collision cylinder length=0.00015248374465266922 radius=0.0436334; collision sphere radius=0.0436334

File: kyon_urdf/urdf/kyon_leg.urdf (robot description, URDF)
Before this commit: robot kyon, 6 links, 5 joints
Links:
- link hip_pitch_2_link: geometry collision mesh filename=${MESH_PATH}/collision/mesh_hip-pitch.stl scale=0.001 0.001 0.001; visual mesh filename=${MESH_PATH}/mesh_hip-pitch.stl scale=0.001 0.001 0.001
- link hip_roll_2_link: geometry collision mesh filename=${MESH_PATH}/collision/mesh_hip-roll.stl scale=0.001 0.001 0.001; visual mesh filename=${MESH_PATH}/mesh_hip-roll.stl scale=0.001 0.001 0.001
- link knee_pitch_2_link: geometry collision mesh filename=${MESH_PATH}/collision/mesh_foot-leg.stl scale=0.001 0.001 0.001; visual mesh filename=${MESH_PATH}/mesh_foot-leg.stl scale=0.001 0.001 0.001

File: kyon_urdf/urdf/kyon_leg.urdf.xacro (robot description, xacro)
@@ -1,11 +1,11 @@
 <?xml version="1.0"?>
-<robot xmlns:xacro="http://ros.org/wiki/xacro" name="kyon">
-    <xacro:include filename="$(find kyon_urdf)/urdf/config/kyon.urdf.xacro" />
-    <xacro:include filename="$(find kyon_urdf)/urdf/parts/kyon_leg.urdf.xacro" />
-    <xacro:include filename="$(find kyon_urdf)/urdf/utils.urdf.xacro" />
+<robot xmlns:xacro="http://ros.org/wiki/xacro" name="kyon_real">
+    <xacro:include filename="${ROOT}/urdf/config/kyon.urdf.xacro" />
+    <xacro:include filename="${ROOT}/urdf/parts/kyon_leg.urdf.xacro" />
+    <xacro:include filename="${ROOT}/urdf/utils.urdf.xacro" />
     <!-- NOTE: here we need to include "kinematics_properties" first because "inertial_properties" depends on it-->
-    <xacro:include filename="$(find kyon_urdf)/urdf/parts/kinematics_properties.urdf.xacro" />
-    <xacro:include filename="$(find kyon_urdf)/urdf/parts/inertial_properties.urdf.xacro" />
-    <xacro:include filename="$(find kyon_urdf)/urdf/parts/limits.urdf.xacro" />
+    <xacro:include filename="${ROOT}/urdf/parts/kinematics_properties.urdf.xacro" />
+    <xacro:include filename="${ROOT}/urdf/parts/inertial_properties.urdf.xacro" />
+    <xacro:include filename="${ROOT}/urdf/parts/limits.urdf.xacro" />
     <link name="world"/>
     <joint name="base_joint" type="fixed">

File: kyon_urdf/urdf/kyon_leg_wheel.urdf (robot description, URDF)
Before this commit: robot kyon, 7 links, 6 joints
Links:
- link hip_pitch_2_link: geometry collision mesh filename=${MESH_PATH}/collision/mesh_hip-pitch.stl scale=0.001 0.001 0.001; visual mesh filename=${MESH_PATH}/mesh_hip-pitch.stl scale=0.001 0.001 0.001
- link hip_roll_2_link: geometry collision mesh filename=${MESH_PATH}/collision/mesh_hip-roll.stl scale=0.001 0.001 0.001; visual mesh filename=${MESH_PATH}/mesh_hip-roll.stl scale=0.001 0.001 0.001
- link knee_pitch_2_link: geometry collision mesh filename=${MESH_PATH}/collision/mesh_fixed-wheel-leg.stl scale=0.001 0.001 0.001; visual mesh filename=${MESH_PATH}/mesh_fixed-wheel-leg.stl scale=0.001 0.001 0.001
- link wheel_2_link: geometry collision mesh filename=${MESH_PATH}/collision/mesh_wheel.stl scale=0.001 0.001 0.001; visual mesh filename=${MESH_PATH}/mesh_wheel.stl scale=0.001 0.001 0.001

File: kyon_urdf/urdf/kyon_robot.urdf.xacro (robot description, xacro)
@@ -1,8 +1,8 @@
 <?xml version="1.0"?>
-<robot xmlns:xacro="http://ros.org/wiki/xacro" name="kyon">
-  <xacro:include filename="$(find kyon_urdf)/urdf/kyon.urdf.xacro" />
-  <xacro:include filename="$(find kyon_urdf)/urdf/gazebo/kyon.gazebo.xacro" />
-  <xacro:include filename="$(find kyon_urdf)/urdf/gazebo/xbot.gazebo.xacro" />
-  <xacro:include filename="$(find kyon_urdf)/urdf/gazebo/materials.gazebo.xacro" />
+<robot xmlns:xacro="http://ros.org/wiki/xacro" name="kyon_real">
+  <xacro:include filename="${ROOT}/urdf/kyon.urdf.xacro" />
+  <xacro:include filename="${ROOT}/urdf/gazebo/kyon.gazebo.xacro" />
+  <xacro:include filename="${ROOT}/urdf/gazebo/xbot.gazebo.xacro" />
+  <xacro:include filename="${ROOT}/urdf/gazebo/materials.gazebo.xacro" />
   <xacro:unless value="${ADD_LEGS}">
     <link name="world"/>
