Commit message: Signed-off-by: Andrea Patrizi <andreapatrizi1b6e6@gmail.com>

File: kyon_urdf/urdf/kyon_wheels_capsule.urdf (robot description, URDF)
Before this commit: robot kyon, 42 links, 41 joints
Links:
- link ankle_yaw_1_link: geometry collision cylinder length=0.24025318703748175 radius=0.058406; collision sphere radius=0.058406
- link ankle_yaw_2_link: geometry collision cylinder length=0.24025318703748175 radius=0.058406; collision sphere radius=0.058406
- link ankle_yaw_3_link: geometry collision cylinder length=0.24025318703748175 radius=0.058406; collision sphere radius=0.058406
- link ankle_yaw_4_link: geometry collision cylinder length=0.24025318703748175 radius=0.058406; collision sphere radius=0.058406
- link dagana_1_base: geometry collision cylinder length=0.05560094231679104 radius=0.0463682; collision mesh filename=${MESH_PATH}/collision/mesh_dagana-base-base-simplified.stl scale=0.001 0.001 0.001
- link dagana_1_claw: geometry collision cylinder length=0.06837212339526175 radius=0.0356173; collision mesh filename=${MESH_PATH}/collision/mesh_dagana-clamp-simplified.stl scale=0.001 0.001 0.001
- link dagana_2_base: geometry collision cylinder length=0.05560094231679104 radius=0.0463682; collision mesh filename=${MESH_PATH}/collision/mesh_dagana-base-base-simplified.stl scale=0.001 0.001 0.001
- link dagana_2_claw: geometry collision cylinder length=0.06837212339526175 radius=0.0356173; collision mesh filename=${MESH_PATH}/collision/mesh_dagana-clamp-simplified.stl scale=0.001 0.001 0.001
- link elbow_pitch_1_link: geometry collision cylinder length=0.23685382242345215 radius=0.0581584; collision sphere radius=0.0581584
- link elbow_pitch_2_link: geometry collision cylinder length=0.23685382242345215 radius=0.0581584; collision sphere radius=0.0581584
- link hip_pitch_1_link: geometry collision cylinder length=0.3004661110170414 radius=0.110589; collision sphere radius=0.110589
- link hip_pitch_2_link: geometry collision cylinder length=0.3004661110170414 radius=0.110589; collision sphere radius=0.110589
- link hip_pitch_3_link: geometry collision cylinder length=0.3004661110170414 radius=0.110589; collision sphere radius=0.110589
- link hip_pitch_4_link: geometry collision cylinder length=0.3004661110170414 radius=0.110589; collision sphere radius=0.110589
- link hip_roll_1_link: geometry collision cylinder length=0.14024696973705675 radius=0.0763481; collision sphere radius=0.0763481
- link hip_roll_2_link: geometry collision cylinder length=0.14024696973705536 radius=0.0763481; collision sphere radius=0.0763481
- link hip_roll_3_link: geometry collision cylinder length=0.14024696973705675 radius=0.0763481; collision sphere radius=0.0763481
- link hip_roll_4_link: geometry collision cylinder length=0.14024696973705536 radius=0.0763481; collision sphere radius=0.0763481
- link knee_pitch_1_link: geometry collision cylinder length=0.007315665155126021 radius=0.0660721; collision sphere radius=0.0660721
- link knee_pitch_2_link: geometry collision cylinder length=0.007315665155126021 radius=0.0660721; collision sphere radius=0.0660721
- link knee_pitch_3_link: geometry collision cylinder length=0.007315665155126021 radius=0.0660721; collision sphere radius=0.0660721
- link knee_pitch_4_link: geometry collision cylinder length=0.007315665155126021 radius=0.0660721; collision sphere radius=0.0660721
- link pelvis: geometry collision cylinder length=0.7715265904067888 radius=0.180153; collision sphere radius=0.180153
- link shoulder_pitch_1_link: geometry collision cylinder length=0.33021118992969195 radius=0.0630638; collision sphere radius=0.0630638
- link shoulder_pitch_2_link: geometry collision cylinder length=0.33021118992969195 radius=0.0630638; collision sphere radius=0.0630638
- link shoulder_yaw_1_link: geometry collision cylinder length=0.06680404009166925 radius=0.0700029; collision sphere radius=0.0700029
- link shoulder_yaw_2_link: geometry collision cylinder length=0.06680404009166925 radius=0.0700029; collision sphere radius=0.0700029
- link wheel_1: geometry collision cylinder length=0.019845524355384083 radius=0.109681; collision sphere radius=0.109681
- link wheel_2: geometry collision cylinder length=0.019845524355384083 radius=0.109681; collision sphere radius=0.109681
- link wheel_3: geometry collision cylinder length=0.019845524355384083 radius=0.109681; collision sphere radius=0.109681
- link wheel_4: geometry collision cylinder length=0.019845524355384083 radius=0.109681; collision sphere radius=0.109681
- link wrist_pitch_1_link: geometry collision cylinder length=0.07557658310998112 radius=0.0522867; collision sphere radius=0.0522867
- link wrist_pitch_2_link: geometry collision cylinder length=0.07557658310998112 radius=0.0522867; collision sphere radius=0.0522867
- link wrist_yaw_1_link: geometry collision cylinder length=0.00015248374464368804 radius=0.0436334; collision sphere radius=0.0436334
- link wrist_yaw_2_link: geometry collision cylinder length=0.00015248374464368804 radius=0.0436334; collision sphere radius=0.0436334

File: kyon_urdf/urdf/parts/arms.urdf.xacro (robot description, xacro)
@@ -1,5 +1,5 @@
 <?xml version="1.0"?>
 <robot xmlns:xacro="http://ros.org/wiki/xacro">
-<xacro:include filename="$(find kyon_urdf)/urdf/parts/kyon_arm.urdf.xacro"/>
+<xacro:include filename="${ROOT}/urdf/parts/kyon_arm.urdf.xacro"/>
 <!-- arms -->
 <xacro:kyon_arm arm_num="1"  rot="-1"  parent="pelvis">

File: kyon_urdf/urdf/parts/foot_leg.urdf.xacro (robot description, xacro)
@@ -12,5 +12,5 @@
         <origin xyz="0.0 0.0 0.0"  rpy="0.0 0.0 0.0"/>
         <geometry>
-            <mesh filename="package://kyon_urdf/meshes/mesh_foot-leg.stl" scale="${mirror*0.001} 0.001 0.001"/>
+            <mesh filename="${MESH_PATH}/mesh_foot-leg.stl" scale="${mirror*0.001} 0.001 0.001"/>
         </geometry>
         <material name="dark_grey"/>
@@ -19,5 +19,5 @@
         <origin xyz="0.0 0.0 0.0"  rpy="0.0 0.0 0.0"/>
         <geometry>
-            <mesh filename="package://kyon_urdf/meshes/collision/mesh_foot-leg.stl" scale="${mirror*0.001} 0.001 0.001"/>
+            <mesh filename="${MESH_PATH}/collision/mesh_foot-leg.stl" scale="${mirror*0.001} 0.001 0.001"/>
         </geometry>
     </collision>

File: kyon_urdf/urdf/parts/kyon_arm.urdf.xacro (robot description, xacro)
@@ -1,5 +1,5 @@
 <?xml version="1.0"?>
 <robot xmlns:xacro="http://ros.org/wiki/xacro">
-<xacro:include filename="$(find kyon_urdf)/urdf/parts/kyon_dagana.urdf.xacro"/>
+<xacro:include filename="${ROOT}/urdf/parts/kyon_dagana.urdf.xacro"/>
 <!-- macro arms -->
 <xacro:macro name="kyon_arm" params="arm_num rot parent">
@@ -15,5 +15,5 @@
 		<origin xyz="0.0 0.0 0.0"  rpy="0.0 0.0 0.0"/>
 		<geometry>
-			<mesh filename="package://kyon_urdf/meshes/mesh_sh-yaw.stl" scale="0.001 0.001 0.001"/>
+			<mesh filename="${MESH_PATH}/mesh_sh-yaw.stl" scale="0.001 0.001 0.001"/>
 		</geometry>
 		<material name="dark_grey"/>
@@ -22,5 +22,5 @@
 		<origin xyz="0.0 0.0 0.0"  rpy="0.0 0.0 0.0"/>
 		<geometry>
-			<mesh filename="package://kyon_urdf/meshes/collision/mesh_sh-yaw.stl" scale="0.001 0.001 0.001"/>
+			<mesh filename="${MESH_PATH}/collision/mesh_sh-yaw.stl" scale="0.001 0.001 0.001"/>
 		</geometry>
 	</collision>
@@ -34,5 +34,5 @@
 	<visual>
 	  	<geometry>
-			<mesh filename="package://kyon_urdf/meshes/mesh_sh-pitch_cover.stl" scale="0.001 0.001 0.001"/>
+			<mesh filename="${MESH_PATH}/mesh_sh-pitch_cover.stl" scale="0.001 0.001 0.001"/>
 	  	</geometry>
   		<material name="dark_grey"/>
@@ -40,5 +40,5 @@
 	<visual>
 	  	<geometry>
-	 		<mesh filename="package://kyon_urdf/meshes/mesh_sh-pitch.stl" scale="0.001 0.001 0.001"/>
+	 		<mesh filename="${MESH_PATH}/mesh_sh-pitch.stl" scale="0.001 0.001 0.001"/>
 	  	</geometry>
   		<material name="kyon_orange"/>
@@ -46,5 +46,5 @@
 	<collision>
 	  	<geometry>
-			<mesh filename="package://kyon_urdf/meshes/collision/mesh_sh-pitch.stl" scale="0.001 0.001 0.001"/>
+			<mesh filename="${MESH_PATH}/collision/mesh_sh-pitch.stl" scale="0.001 0.001 0.001"/>
 		</geometry>
 		<material name="kyon_orange"/>
@@ -59,5 +59,5 @@
 	<visual>
 		<geometry>
-			<mesh filename="package://kyon_urdf/meshes/mesh_elbow.stl" scale="0.001 0.001 0.001"/>
+			<mesh filename="${MESH_PATH}/mesh_elbow.stl" scale="0.001 0.001 0.001"/>
 		</geometry>
 		<material name="dark_grey"/>
@@ -65,5 +65,5 @@
 	<collision>
 		<geometry>
-			<mesh filename="package://kyon_urdf/meshes/mesh_elbow.stl" scale="0.001 0.001 0.001"/>
+			<mesh filename="${MESH_PATH}/mesh_elbow.stl" scale="0.001 0.001 0.001"/>
 		</geometry>
 	</collision>
@@ -78,5 +78,5 @@
 		<origin xyz="0.0 0.0 0.0"  rpy="0.0 0.0 0.0"/>
 	  	<geometry>
-	 		<mesh filename="package://kyon_urdf/meshes/mesh_wrist-pitch.stl" scale="0.001 0.001 0.001"/>
+	 		<mesh filename="${MESH_PATH}/mesh_wrist-pitch.stl" scale="0.001 0.001 0.001"/>
 	  	</geometry>
   		<material name="dark_grey"/>
@@ -85,5 +85,5 @@
 		<origin xyz="0.0 0.0 0.0"  rpy="0.0 0.0 0.0"/>
 		<geometry>
-			<mesh filename="package://kyon_urdf/meshes/collision/mesh_wrist-pitch.stl" scale="0.001 0.001 0.001"/>
+			<mesh filename="${MESH_PATH}/collision/mesh_wrist-pitch.stl" scale="0.001 0.001 0.001"/>
 		</geometry>
 	</collision>
@@ -98,5 +98,5 @@
 		<origin xyz="0.0 0.0 0.0"  rpy="0.0 0.0 0.0"/>
 	  	<geometry>
-	 		<mesh filename="package://kyon_urdf/meshes/mesh_wrist-yaw.stl" scale="0.001 0.001 0.001"/>
+	 		<mesh filename="${MESH_PATH}/mesh_wrist-yaw.stl" scale="0.001 0.001 0.001"/>
 	  	</geometry>
   		<material name="dark_grey"/>
@@ -105,5 +105,5 @@
 		<origin xyz="0.0 0.0 0.0"  rpy="0.0 0.0 0.0"/>
 		<geometry>
-			<mesh filename="package://kyon_urdf/meshes/collision/mesh_wrist-yaw.stl" scale="0.001 0.001 0.001"/>
+			<mesh filename="${MESH_PATH}/collision/mesh_wrist-yaw.stl" scale="0.001 0.001 0.001"/>
 		</geometry>
 	</collision>

File: kyon_urdf/urdf/parts/kyon_dagana.urdf.xacro (robot description, xacro)
@@ -12,5 +12,5 @@
         <origin xyz="0.0 0.0 0.0"  rpy="0.0 0.0 0.0"/>
         <geometry>
-            <mesh filename="package://kyon_urdf/meshes/mesh_dagana-base.stl" scale="0.001 0.001 0.001"/>
+            <mesh filename="${MESH_PATH}/mesh_dagana-base.stl" scale="0.001 0.001 0.001"/>
         </geometry>
         <material name="dark_grey"/>
@@ -19,5 +19,5 @@
         <origin xyz="0.0 0.0 0.0"  rpy="0.0 0.0 0.0"/>
         <geometry>
-            <mesh filename="package://kyon_urdf/meshes/collision/mesh_dagana-base-simplified.stl" scale="0.001 0.001 0.001"/>
+            <mesh filename="${MESH_PATH}/collision/mesh_dagana-base-simplified.stl" scale="0.001 0.001 0.001"/>
         </geometry>
     </collision>
@@ -25,5 +25,5 @@
         <origin xyz="0.0 0.0 0.0"  rpy="0.0 0.0 0.0"/>
         <geometry>
-            <mesh filename="package://kyon_urdf/meshes/collision/mesh_dagana-base-base-simplified.stl" scale="0.001 0.001 0.001"/>
+            <mesh filename="${MESH_PATH}/collision/mesh_dagana-base-base-simplified.stl" scale="0.001 0.001 0.001"/>
         </geometry>
     </collision>
@@ -38,5 +38,5 @@
         <origin xyz="0.0 0.0 0.0"  rpy="0.0 0.0 0.0"/>
         <geometry>
-            <mesh filename="package://kyon_urdf/meshes/mesh_dagana-clamp.stl" scale="0.001 0.001 0.001"/>
+            <mesh filename="${MESH_PATH}/mesh_dagana-clamp.stl" scale="0.001 0.001 0.001"/>
         </geometry>
         <material name="dark_grey"/>
@@ -45,5 +45,5 @@
         <origin xyz="0.0 0.0 0.0"  rpy="0.0 0.0 0.0"/>
         <geometry>
-            <mesh filename="package://kyon_urdf/meshes/collision/mesh_dagana-clamp-base-simplified.stl" scale="0.001 0.001 0.001"/>
+            <mesh filename="${MESH_PATH}/collision/mesh_dagana-clamp-base-simplified.stl" scale="0.001 0.001 0.001"/>
         </geometry>
     </collision>
@@ -51,5 +51,5 @@
         <origin xyz="0.0 0.0 0.0"  rpy="0.0 0.0 0.0"/>
         <geometry>
-            <mesh filename="package://kyon_urdf/meshes/collision/mesh_dagana-clamp-simplified.stl" scale="0.001 0.001 0.001"/>
+            <mesh filename="${MESH_PATH}/collision/mesh_dagana-clamp-simplified.stl" scale="0.001 0.001 0.001"/>
         </geometry>
     </collision>

File: kyon_urdf/urdf/parts/kyon_leg.urdf.xacro (robot description, xacro)
@@ -2,7 +2,7 @@
 <robot xmlns:xacro="http://ros.org/wiki/xacro">
 <!-- include end-effectors -->
-<xacro:include filename="$(find kyon_urdf)/urdf/parts/foot_leg.urdf.xacro"/>
-<xacro:include filename="$(find kyon_urdf)/urdf/parts/steering_wheel.urdf.xacro"/>
-<xacro:include filename="$(find kyon_urdf)/urdf/parts/wheel_leg.urdf.xacro"/>
+<xacro:include filename="${ROOT}/urdf/parts/foot_leg.urdf.xacro"/>
+<xacro:include filename="${ROOT}/urdf/parts/steering_wheel.urdf.xacro"/>
+<xacro:include filename="${ROOT}/urdf/parts/wheel_leg.urdf.xacro"/>
 <!-- macro legs -->
 <xacro:macro name="kyon_leg" params="leg_num origin_x origin_y mirror">
@@ -18,5 +18,5 @@
 	  	<geometry>
 	 		<!-- <cylinder radius="${cylinder_radius}" length="${cylinder_length}"/> -->
-			<mesh filename="package://kyon_urdf/meshes/mesh_hip-roll.stl" scale="0.001 ${mirror*0.001} 0.001"/>
+			<mesh filename="${MESH_PATH}/mesh_hip-roll.stl" scale="0.001 ${mirror*0.001} 0.001"/>
 		</geometry>
   		<material name="dark_grey"/>
@@ -26,5 +26,5 @@
 		<geometry>
 	 		<!-- <cylinder radius="${cylinder_radius}" length="${cylinder_length}"/> -->
-			<mesh filename="package://kyon_urdf/meshes/collision/mesh_hip-roll.stl" scale="0.001 ${mirror*0.001} 0.001"/>
+			<mesh filename="${MESH_PATH}/collision/mesh_hip-roll.stl" scale="0.001 ${mirror*0.001} 0.001"/>
 		</geometry>
 	</collision>
@@ -39,5 +39,5 @@
 		<origin xyz="0.0 0.0 0.0"  rpy="0.0 0.0 0.0"/>
 	  	<geometry>
-	 		<mesh filename="package://kyon_urdf/meshes/mesh_hip-pitch.stl" scale="0.001 0.001 0.001"/>
+	 		<mesh filename="${MESH_PATH}/mesh_hip-pitch.stl" scale="0.001 0.001 0.001"/>
 	  	</geometry>
   		<material name="kyon_orange"/>
@@ -46,5 +46,5 @@
 		<origin xyz="0.0 0.0 0.0"  rpy="0.0 0.0 0.0"/>
 	  	<geometry>
-	 		<mesh filename="package://kyon_urdf/meshes/mesh_hip-pitch_cover.stl" scale="0.001 0.001 0.001"/>
+	 		<mesh filename="${MESH_PATH}/mesh_hip-pitch_cover.stl" scale="0.001 0.001 0.001"/>
 	  	</geometry>
   		<material name="dark_grey"/>
@@ -53,5 +53,5 @@
 		<origin xyz="0.0 0.0 0.0"  rpy="0.0 0.0 0.0"/>
 		<geometry>
-			<mesh filename="package://kyon_urdf/meshes/collision/mesh_hip-pitch.stl" scale="0.001 0.001 0.001"/>
+			<mesh filename="${MESH_PATH}/collision/mesh_hip-pitch.stl" scale="0.001 0.001 0.001"/>
 		</geometry>
 		<material name="kyon_orange"/>

File: kyon_urdf/urdf/parts/legs.urdf.xacro (robot description, xacro)
@@ -1,5 +1,5 @@
 <?xml version="1.0"?>
 <robot xmlns:xacro="http://ros.org/wiki/xacro">
-<xacro:include filename="$(find kyon_urdf)/urdf/parts/kyon_leg.urdf.xacro" />
+<xacro:include filename="${ROOT}/urdf/parts/kyon_leg.urdf.xacro" />
 <xacro:kyon_leg leg_num="1" origin_x="1" origin_y="-1" mirror="-1">
 </xacro:kyon_leg>

File: kyon_urdf/urdf/parts/steering_wheel.urdf.xacro (robot description, xacro)
@@ -13,5 +13,5 @@
 	  	<geometry>
 	 		<!-- <cylinder radius="${cylinder_radius}" length="${cylinder_length}"/> -->
-			<mesh filename="package://kyon_urdf/meshes/mesh_knee-steering.stl" scale="0.001 0.001 0.001"/>
+			<mesh filename="${MESH_PATH}/mesh_knee-steering.stl" scale="0.001 0.001 0.001"/>
 		</geometry>
   		<material name="dark_grey"/>
@@ -21,5 +21,5 @@
 		<geometry>
 	 		<!-- <cylinder radius="${cylinder_radius}" length="${cylinder_length}"/> -->
-			<mesh filename="package://kyon_urdf/meshes/collision/mesh_knee-steering.stl" scale="0.001 0.001 0.001"/>
+			<mesh filename="${MESH_PATH}/collision/mesh_knee-steering.stl" scale="0.001 0.001 0.001"/>
 		</geometry>
 	</collision>
@@ -35,5 +35,5 @@
 	  	<geometry>
 	 		<!-- <cylinder radius="${cylinder_radius}" length="${cylinder_length}"/> -->
-			<mesh filename="package://kyon_urdf/meshes/mesh_ankle-yaw.stl" scale="0.001 0.001 0.001"/>
+			<mesh filename="${MESH_PATH}/mesh_ankle-yaw.stl" scale="0.001 0.001 0.001"/>
 		</geometry>
   		<material name="dark_grey"/>
@@ -43,5 +43,5 @@
 		<geometry>
 	 		<!-- <cylinder radius="${cylinder_radius}" length="${cylinder_length}"/> -->
-			<mesh filename="package://kyon_urdf/meshes/collision/mesh_ankle-yaw.stl" scale="0.001 0.001 0.001"/>
+			<mesh filename="${MESH_PATH}/collision/mesh_ankle-yaw.stl" scale="0.001 0.001 0.001"/>
 		</geometry>
 	</collision>
@@ -57,5 +57,5 @@
 	  	<geometry>
 	 		<!-- <cylinder radius="${cylinder_radius}" length="${cylinder_length}"/> -->
-			<mesh filename="package://kyon_urdf/meshes/mesh_wheel.stl" scale="0.001 0.001 0.001"/>
+			<mesh filename="${MESH_PATH}/mesh_wheel.stl" scale="0.001 0.001 0.001"/>
 		</geometry>
   		<material name="light_grey"/>
@@ -65,5 +65,5 @@
 		<geometry>
 	 		<!-- <cylinder radius="${cylinder_radius}" length="${cylinder_length}"/> -->
-			<mesh filename="package://kyon_urdf/meshes/collision/mesh_wheel.stl" scale="0.001 0.001 0.001"/>
+			<mesh filename="${MESH_PATH}/collision/mesh_wheel.stl" scale="0.001 0.001 0.001"/>
 		</geometry>
 		<material name="light_grey"/>

File: kyon_urdf/urdf/parts/wheel_leg.urdf.xacro (robot description, xacro)
@@ -12,5 +12,5 @@
         <origin xyz="0.0 0.0 0.0"  rpy="0.0 0.0 0.0"/>
         <geometry>
-            <mesh filename="package://kyon_urdf/meshes/mesh_fixed-wheel-leg.stl" scale="${mirror*0.001} 0.001 0.001"/>
+            <mesh filename="${MESH_PATH}/mesh_fixed-wheel-leg.stl" scale="${mirror*0.001} 0.001 0.001"/>
         </geometry>
         <material name="dark_grey"/>
@@ -19,5 +19,5 @@
         <origin xyz="0.0 0.0 0.0"  rpy="0.0 0.0 0.0"/>
         <geometry>
-            <mesh filename="package://kyon_urdf/meshes/collision/mesh_fixed-wheel-leg.stl" scale="${mirror*0.001} 0.001 0.001"/>
+            <mesh filename="${MESH_PATH}/collision/mesh_fixed-wheel-leg.stl" scale="${mirror*0.001} 0.001 0.001"/>
         </geometry>
     </collision>
@@ -32,5 +32,5 @@
 		<origin xyz="0.0 0.0 0.0"  rpy="0.0 0.0 0.0"/>
 	  	<geometry>
-			<mesh filename="package://kyon_urdf/meshes/mesh_wheel.stl" scale="0.001 0.001 0.001"/>
+			<mesh filename="${MESH_PATH}/mesh_wheel.stl" scale="0.001 0.001 0.001"/>
 		</geometry>
   		<material name="dark_grey"/>
@@ -39,5 +39,5 @@
 		<origin xyz="0.0 0.0 0.0"  rpy="0.0 0.0 0.0"/>
 		<geometry>
-			<!-- <mesh filename="package://kyon_urdf/meshes/collision/mesh_wheel.stl" scale="0.001 0.001 0.001"/> -->
+			<!-- <mesh filename="${MESH_PATH}/collision/mesh_wheel.stl" scale="0.001 0.001 0.001"/> -->
             <cylinder radius="0.11" length="0.045"/>
 		</geometry>

Commit message: Signed-off-by: Andrea Patrizi <andreapatrizi1b6e6@gmail.com>

File: kyon_srdf/srdf/kyon.srdf.xacro (robot description, xacro)
@@ -6,5 +6,5 @@
 <robot xmlns:xacro="http://ros.org/wiki/xacro" name="kyon">
     <!-- ************ MODEL CONFIGURATION ************ -->
-    <xacro:arg name="root" default="$(find kyon_urdf)" />
+    <xacro:arg name="root" default="$(find kyon_urdf_simple)" />
     <xacro:property name="ROOT" value="$(arg root)" />
     <xacro:arg name="config" default="${ROOT}/urdf/config/kyon.urdf.xacro"/>

File: kyon_urdf/urdf/kyon.urdf.xacro (robot description, xacro)
@@ -3,5 +3,5 @@
 <!-- This argument and property should be in the top level xacro and
 will be propagated to all its downstream childs -->
-<xacro:arg name="root" default="$(find kyon_urdf)" />
+<xacro:arg name="root" default="$(find kyon_urdf_simple)" />
 <xacro:property name="ROOT" value="$(arg root)" />
 <!-- setting use_abs_mesh_paths should be kept to false
@@ -21,5 +21,5 @@
 	</xacro:if>
 <xacro:unless value="${USE_ABS_MESH_PATHS}">
-<xacro:property name="MESH_PATH" value="package://kyon_urdf/meshes" />
+<xacro:property name="MESH_PATH" value="package://kyon_urdf_simple/meshes" />
 </xacro:unless>
 <xacro:arg name="config" default="${ROOT}/urdf/config/kyon.urdf.xacro"/>

Commit message: added missing wheel joints from srdf

File: kyon_srdf/srdf/kyon.srdf.xacro (robot description, xacro)
@@ -97,4 +97,8 @@
             <joint name="ankle_yaw_3" value="0.0"/>
             <joint name="ankle_yaw_4" value="0.0"/>
+            <joint name="wheel_joint_1" value="0.0"/>
+            <joint name="wheel_joint_2" value="0.0"/>
+            <joint name="wheel_joint_3" value="0.0"/>
+            <joint name="wheel_joint_4" value="0.0"/>
         </xacro:if>
         <xacro:if value="${ADD_UPPER_BODY}">
