Commit message: some updates

File: kyon_srdf/srdf/kyon.srdf.xacro (robot description, xacro)
@@ -46,18 +46,8 @@
     <xacro:if value="${ADD_UPPER_BODY}">
 		<group name="left_arm">
-            <xacro:if value="${ADD_DAGANA}">
-			    <chain base_link="pelvis" tip_link="dagana_1_claw"/>
-            </xacro:if>
-            <xacro:unless value="${ADD_DAGANA}">
-                <chain base_link="pelvis" tip_link="wrist_yaw_1_link"/>
-            </xacro:unless>
-		</group>
+		    <chain base_link="pelvis" tip_link="dagana_1_claw"/>
+     		</group>
 		<group name="right_arm">
-            <xacro:if value="${ADD_DAGANA}">
-			    <chain base_link="pelvis" tip_link="dagana_2_claw"/>
-            </xacro:if>
-            <xacro:unless value="${ADD_DAGANA}">
-                <chain base_link="pelvis" tip_link="wrist_yaw_2_link"/>
-            </xacro:unless>
+		    <chain base_link="pelvis" tip_link="dagana_2_claw"/>
 		</group>
     </xacro:if>
@@ -77,14 +67,48 @@
     <group_state name="home" group="chains">
         <xacro:if value="${ADD_LEGS}">
-            <joint name="hip_roll_1" value="0.0"/>
+            <joint name="hip_roll_1" value="0.15"/>
             <joint name="hip_pitch_1" value="-0.7"/>
             <joint name="knee_pitch_1" value="1.4"/>
-            <joint name="hip_roll_2" value="0.0"/>
+            <joint name="hip_roll_2" value="-0.15"/>
             <joint name="hip_pitch_2" value="0.7"/>
             <joint name="knee_pitch_2" value="-1.4"/>
-            <joint name="hip_roll_3" value="0.0"/>
+            <joint name="hip_roll_3" value="-0.15"/>
             <joint name="hip_pitch_3" value="-0.7"/>
             <joint name="knee_pitch_3" value="1.4"/>
-            <joint name="hip_roll_4" value="0.0"/>
+            <joint name="hip_roll_4" value="0.15"/>
+            <joint name="hip_pitch_4" value="0.7"/>
+            <joint name="knee_pitch_4" value="-1.4"/>
+        </xacro:if>
+        <!-- <xacro:if value="${ADD_WHEELS}">
+            <joint name="ankle_yaw_1" value="0.0"/>
+            <joint name="ankle_yaw_2" value="0.0"/>
+            <joint name="ankle_yaw_3" value="0.0"/>
+            <joint name="ankle_yaw_4" value="0.0"/>
+        </xacro:if> -->
+        <xacro:if value="${ADD_UPPER_BODY}">
+            <joint name="shoulder_yaw_1" value="0.0"/>
+            <joint name="shoulder_pitch_1" value="1."/>
+            <joint name="elbow_pitch_1" value="2.1"/>
+            <joint name="wrist_pitch_1" value="0.7"/>
+            <joint name="wrist_yaw_1" value="0.0"/>
+            <joint name="shoulder_yaw_2" value="0.0"/>
+            <joint name="shoulder_pitch_2" value="-1."/>
+            <joint name="elbow_pitch_2" value="-2.1"/>
+            <joint name="wrist_pitch_2" value="-0.7"/>
+            <joint name="wrist_yaw_2" value="0.0"/>
+        </xacro:if>
+    </group_state>
+        <group_state name="home_isaac" group="chains">
+        <xacro:if value="${ADD_LEGS}">
+            <joint name="hip_roll_1" value="0.15"/>
+            <joint name="hip_pitch_1" value="-0.7"/>
+            <joint name="knee_pitch_1" value="1.4"/>
+            <joint name="hip_roll_2" value="-0.15"/>
+            <joint name="hip_pitch_2" value="0.7"/>
+            <joint name="knee_pitch_2" value="-1.4"/>
+            <joint name="hip_roll_3" value="-0.15"/>
+            <joint name="hip_pitch_3" value="-0.7"/>
+            <joint name="knee_pitch_3" value="1.4"/>
+            <joint name="hip_roll_4" value="0.15"/>
             <joint name="hip_pitch_4" value="0.7"/>
             <joint name="knee_pitch_4" value="-1.4"/>
@@ -98,12 +122,12 @@
         <xacro:if value="${ADD_UPPER_BODY}">
             <joint name="shoulder_yaw_1" value="0.0"/>
-            <joint name="shoulder_pitch_1" value="1.0"/>
-            <joint name="elbow_pitch_1" value="2.0"/>
-            <joint name="wrist_pitch_1" value="0.5"/>
+            <joint name="shoulder_pitch_1" value="1.5"/>
+            <joint name="elbow_pitch_1" value="2.5"/>
+            <joint name="wrist_pitch_1" value="0.7"/>
             <joint name="wrist_yaw_1" value="0.0"/>
             <joint name="shoulder_yaw_2" value="0.0"/>
-            <joint name="shoulder_pitch_2" value="-1.0"/>
-            <joint name="elbow_pitch_2" value="-2.0"/>
-            <joint name="wrist_pitch_2" value="-0.5"/>
+            <joint name="shoulder_pitch_2" value="-1.5"/>
+            <joint name="elbow_pitch_2" value="-2.5"/>
+            <joint name="wrist_pitch_2" value="-0.7"/>
             <joint name="wrist_yaw_2" value="0.0"/>
         </xacro:if>

File: kyon_urdf/urdf/config/kyon.urdf.xacro (robot description, xacro)
@@ -14,9 +14,10 @@
 <xacro:arg name="velodyne" default="false"/>
 <xacro:arg name="dagana" default="$(arg upper_body)"/>
+<xacro:arg name="add_collision" default="true"/>
+<xacro:arg name="hesai_jt128" default="false"/>
 <!-- ************SELECT PARTS*************-->
 <!-- *************************************-->
 <xacro:property name="ADD_LEGS" value="$(arg legs)"/>
 <xacro:property name="ADD_UPPER_BODY" value="$(arg upper_body)"/>
-<xacro:property name="ADD_DAGANA" value="$(arg dagana)"/>
 <xacro:property name="ADD_CAMERAS" value="$(arg cameras)"/>
 <xacro:property name="ADD_WHEELS" value="$(arg wheels)"/>
@@ -25,4 +26,5 @@
 <xacro:property name="ADD_FLOATING_BASE" value="$(arg floating_joint)"/>
 <xacro:property name="ADD_VELODYNE" value="$(arg velodyne)"/>
+<xacro:property name="ADD_HESAI_JT128" value="$(arg hesai_jt128)"/>
 <xacro:property name="ADD_VIRTUAL_FRAME" value="false" />
 <xacro:property name="PAYLOAD" value="$(arg payload)"/>

File: kyon_urdf/urdf/kyon_base.urdf.xacro (robot description, xacro)
@@ -178,17 +178,4 @@
 	<child link="hesai_lidar"/>
 </joint>
-<xacro:if value="${ADD_VELODYNE}">
-    <xacro:include filename="$(find velodyne_description)/urdf/VLP-16.urdf.xacro"/>
-    <xacro:VLP-16 parent="pelvis" name="velodyne" topic="/velodyne_points" hz="10" samples="440">
-        <origin xyz="0.43 0 0.118" rpy="0 0 0.5220063" />
-    </xacro:VLP-16>
-</xacro:if>
-<!-- Velodyne -->
-<xacro:if value="${ADD_VELODYNE}">
-    <xacro:include filename="$(find velodyne_description)/urdf/VLP-16.urdf.xacro"/>
-    <xacro:VLP-16 parent="pelvis" name="velodyne">
-        <origin xyz="0.47 0 0.11" rpy="0 0 0" />
-    </xacro:VLP-16>
-</xacro:if>
 <xacro:if value="${ADD_UPPER_BODY}">
     <xacro:include filename="$(find kyon_urdf)/urdf/parts/arms.urdf.xacro" />
@@ -218,3 +205,27 @@
 	</joint>
 </xacro:if>
+<!-- Hesai JT128 -->
+<xacro:if value="${ADD_HESAI_JT128}">
+    <link name="hesai_jt128_link">
+        <inertial>
+        <mass value="0.2"/>
+        <origin xyz="0 0 0" rpy="0 0 0"/>
+        <inertia ixx="0.001" ixy="0" ixz="0"
+                iyy="0.001" iyz="0"
+                izz="0.001"/>
+        </inertial>
+        <visual>
+            <origin xyz="0.0 0.0 0.0"  rpy="0.0 0.0 0.0"/>
+            <geometry>
+                <mesh filename="package://kyon_urdf/meshes/hesai_jt128.stl" scale="0.0001 0.0001 0.0001"/>
+            </geometry>
+            <material name="dark_grey"/>
+        </visual>
+    </link>
+    <joint name="hesai_jt128_joint" type="fixed">
+        <origin xyz="0.43 0 -0.118" rpy="${PI} 0 0" />
+        <parent link="pelvis"/>
+        <child link="hesai_jt128_link"/>
+    </joint>
+</xacro:if>
 </robot>

Commit message: some updates

File: kyon_srdf/srdf/kyon.srdf.xacro (robot description, xacro)
@@ -100,4 +100,38 @@
     </group_state>
         <group_state name="home_isaac" group="chains">
+        <xacro:if value="${ADD_LEGS}">
+            <joint name="hip_roll_1" value="0.15"/>
+            <joint name="hip_pitch_1" value="-0.7"/>
+            <joint name="knee_pitch_1" value="1.4"/>
+            <joint name="hip_roll_2" value="-0.15"/>
+            <joint name="hip_pitch_2" value="0.7"/>
+            <joint name="knee_pitch_2" value="-1.4"/>
+            <joint name="hip_roll_3" value="-0.15"/>
+            <joint name="hip_pitch_3" value="-0.7"/>
+            <joint name="knee_pitch_3" value="1.4"/>
+            <joint name="hip_roll_4" value="0.15"/>
+            <joint name="hip_pitch_4" value="0.7"/>
+            <joint name="knee_pitch_4" value="-1.4"/>
+        </xacro:if>
+        <xacro:if value="${ADD_WHEELS}">
+            <joint name="ankle_yaw_1" value="0.0"/>
+            <joint name="ankle_yaw_2" value="0.0"/>
+            <joint name="ankle_yaw_3" value="0.0"/>
+            <joint name="ankle_yaw_4" value="0.0"/>
+        </xacro:if>
+        <xacro:if value="${ADD_UPPER_BODY}">
+            <joint name="shoulder_yaw_1" value="0.0"/>
+            <joint name="shoulder_pitch_1" value="1.5"/>
+            <joint name="elbow_pitch_1" value="2.5"/>
+            <joint name="wrist_pitch_1" value="0.7"/>
+            <joint name="wrist_yaw_1" value="0.0"/>
+            <joint name="shoulder_yaw_2" value="0.0"/>
+            <joint name="shoulder_pitch_2" value="-1.5"/>
+            <joint name="elbow_pitch_2" value="-2.5"/>
+            <joint name="wrist_pitch_2" value="-0.7"/>
+            <joint name="wrist_yaw_2" value="0.0"/>
+        </xacro:if>
+    </group_state>
+    <group_state name="home_isaac" group="chains">
         <xacro:if value="${ADD_LEGS}">
             <joint name="hip_roll_1" value="0.15"/>

File: kyon_urdf/urdf/kyon.urdf (robot description, URDF)
Before this commit: robot kyon, 96 links, 95 joints
Links:
- removed link D435_front1_accel_frame
- removed link D435_front1_accel_optical_frame
- removed link D435_front1_bottom_screw_frame
- removed link D435_front1_color_frame
- removed link D435_front1_color_optical_frame
- removed link D435_front1_depth_frame
- removed link D435_front1_depth_optical_frame
- removed link D435_front1_gyro_frame
- removed link D435_front1_gyro_optical_frame
- removed link D435_front1_left_ir_frame
- removed link D435_front1_left_ir_optical_frame
- removed link D435_front1_link
- removed link D435_front1_right_ir_frame
- removed link D435_front1_right_ir_optical_frame
- removed link D435_front2_accel_frame
- removed link D435_front2_accel_optical_frame
- removed link D435_front2_bottom_screw_frame
- removed link D435_front2_color_frame
- removed link D435_front2_color_optical_frame
- removed link D435_front2_depth_frame
- removed link D435_front2_depth_optical_frame
- removed link D435_front2_gyro_frame
- removed link D435_front2_gyro_optical_frame
- removed link D435_front2_left_ir_frame
- removed link D435_front2_left_ir_optical_frame
- removed link D435_front2_link
- removed link D435_front2_right_ir_frame
- removed link D435_front2_right_ir_optical_frame
- removed link D435_left_accel_frame
- removed link D435_left_accel_optical_frame
- removed link D435_left_bottom_screw_frame
- removed link D435_left_color_frame
- removed link D435_left_color_optical_frame
- removed link D435_left_depth_frame
- removed link D435_left_depth_optical_frame
- removed link D435_left_gyro_frame
- removed link D435_left_gyro_optical_frame
- removed link D435_left_left_ir_frame
- removed link D435_left_left_ir_optical_frame
- removed link D435_left_link
- removed link D435_left_right_ir_frame
- removed link D435_left_right_ir_optical_frame
- removed link D435_right_accel_frame
- removed link D435_right_accel_optical_frame
- removed link D435_right_bottom_screw_frame
- removed link D435_right_color_frame
- removed link D435_right_color_optical_frame
- removed link D435_right_depth_frame
- removed link D435_right_depth_optical_frame
- removed link D435_right_gyro_frame
- removed link D435_right_gyro_optical_frame
- removed link D435_right_left_ir_frame
- removed link D435_right_left_ir_optical_frame
- removed link D435_right_link
- removed link D435_right_right_ir_frame
- removed link D435_right_right_ir_optical_frame
- removed link velodyne
- removed link velodyne_base_link
- added link contact_1
- added link contact_2
- added link contact_3
- added link contact_4
- added link hesai_lidar
- added link left_camera_mount_link
- added link right_camera_mount_link
- added link zed_front_down_mount_link
- added link zed_front_up_mount_link
- link dagana_1_base: geometry visual mesh filename=package://kyon_urdf/meshes/mesh_dagana-base.stl scale=0.001 0.001 0.001
- link dagana_1_claw: geometry visual mesh filename=package://kyon_urdf/meshes/mesh_dagana-clamp.stl scale=0.001 0.001 0.001
- link dagana_2_base: geometry visual mesh filename=package://kyon_urdf/meshes/mesh_dagana-base.stl scale=0.001 0.001 0.001
- link dagana_2_claw: geometry visual mesh filename=package://kyon_urdf/meshes/mesh_dagana-clamp.stl scale=0.001 0.001 0.001
Joints:
- removed joint D435_front1_accel_joint
- removed joint D435_front1_accel_optical_joint
- removed joint D435_front1_color_joint
- removed joint D435_front1_color_optical_joint
- removed joint D435_front1_depth_joint
- removed joint D435_front1_depth_optical_joint
- removed joint D435_front1_gyro_joint
- removed joint D435_front1_gyro_optical_joint
- removed joint D435_front1_joint
- removed joint D435_front1_left_ir_joint
- removed joint D435_front1_left_ir_optical_joint
- removed joint D435_front1_link_joint
- removed joint D435_front1_right_ir_joint
- removed joint D435_front1_right_ir_optical_joint
- removed joint D435_front2_accel_joint
- removed joint D435_front2_accel_optical_joint
- removed joint D435_front2_color_joint
- removed joint D435_front2_color_optical_joint
- removed joint D435_front2_depth_joint
- removed joint D435_front2_depth_optical_joint
- removed joint D435_front2_gyro_joint
- removed joint D435_front2_gyro_optical_joint
- removed joint D435_front2_joint
- removed joint D435_front2_left_ir_joint
- removed joint D435_front2_left_ir_optical_joint
- removed joint D435_front2_link_joint
- removed joint D435_front2_right_ir_joint
- removed joint D435_front2_right_ir_optical_joint
- removed joint D435_left_accel_joint
- removed joint D435_left_accel_optical_joint
- removed joint D435_left_color_joint
- removed joint D435_left_color_optical_joint
- removed joint D435_left_depth_joint
- removed joint D435_left_depth_optical_joint
- removed joint D435_left_gyro_joint
- removed joint D435_left_gyro_optical_joint
- removed joint D435_left_joint
- removed joint D435_left_left_ir_joint
- removed joint D435_left_left_ir_optical_joint
- removed joint D435_left_link_joint
- removed joint D435_left_right_ir_joint
- removed joint D435_left_right_ir_optical_joint
- removed joint D435_right_accel_joint
- removed joint D435_right_accel_optical_joint
- removed joint D435_right_color_joint
- removed joint D435_right_color_optical_joint
- removed joint D435_right_depth_joint
- removed joint D435_right_depth_optical_joint
- removed joint D435_right_gyro_joint
- removed joint D435_right_gyro_optical_joint
- removed joint D435_right_joint
- removed joint D435_right_left_ir_joint
- removed joint D435_right_left_ir_optical_joint
- removed joint D435_right_link_joint
- removed joint D435_right_right_ir_joint
- removed joint D435_right_right_ir_optical_joint
- removed joint velodyne_base_mount_joint
- removed joint velodyne_base_scan_joint
- added joint contact_joint_1: type fixed, parent ankle_yaw_1_link, child contact_1, origin xyz=0.0 0.0  -0.3275
- added joint contact_joint_2: type fixed, parent ankle_yaw_2_link, child contact_2, origin xyz=0.0 0.0  -0.3275
- added joint contact_joint_3: type fixed, parent ankle_yaw_3_link, child contact_3, origin xyz=0.0 0.0  -0.3275
- added joint contact_joint_4: type fixed, parent ankle_yaw_4_link, child contact_4, origin xyz=0.0 0.0  -0.3275
- added joint hesai_lidar_joints: type fixed, parent pelvis, child hesai_lidar, origin xyz=0.43 0 0.118 rpy=0 0 0.5220063
- added joint left_camera_mount_joint: type fixed, parent pelvis, child left_camera_mount_link, origin xyz=0 0.150100 0.109486 rpy=0 0.3490656 1.5707963
- added joint right_camera_mount_joint: type fixed, parent pelvis, child right_camera_mount_link, origin xyz=0 -0.150100 0.109486 rpy=0 0.3490656 -1.5707963
- added joint zed_front_down_mount_joint: type fixed, parent pelvis, child zed_front_down_mount_link, origin xyz=0.509601 0 0.00343992 rpy=0 0.9250251 0
- added joint zed_front_up_mount_joint: type fixed, parent pelvis, child zed_front_up_mount_link, origin xyz=0.526174 0 0.0674608 rpy=0 -0.1745327 0
- joint ankle_yaw_1: limit lower=-3.4056 upper=3.4056 effort=185 velocity=7.6 -> lower=-3.0 upper=3.0 effort=185 velocity=7.6
- joint ankle_yaw_2: limit lower=-3.3266 upper=3.3266 effort=185 velocity=7.6 -> lower=-3.0 upper=3.0 effort=185 velocity=7.6
- joint ankle_yaw_3: limit lower=-3.4696 upper=3.4696 effort=185 velocity=7.6 -> lower=-3.0 upper=3.0 effort=185 velocity=7.6
- joint ankle_yaw_4: limit lower=-3.3426 upper=3.3426 effort=185 velocity=7.6 -> lower=-3.0 upper=3.0 effort=185 velocity=7.6
- joint dagana_1_base_joint: origin xyz=0.0 0.0 0.0 rpy=0.0 0.0 0.0 -> xyz=0.0 0.0 0.0 rpy=0.0 0.0 -1.57079632679
- joint dagana_1_clamp_joint: axis 0 0 1 -> 0 0 -1; limit lower=-3.4056 upper=3.4056 effort=25 velocity=14 -> lower=0 upper=1.2 effort=25 velocity=14
- joint dagana_2_base_joint: origin xyz=0.0 0.0 0.0 rpy=0.0 0.0 0.0 -> xyz=0.0 0.0 0.0 rpy=0.0 0.0 1.57079632679
- joint dagana_2_clamp_joint: axis 0 0 1 -> 0 0 -1; limit lower=-3.3266 upper=3.3266 effort=25 velocity=14 -> lower=0 upper=1.2 effort=25 velocity=14
- joint elbow_pitch_1: limit lower=-3 upper=3 effort=122 velocity=4.6 -> lower=-2.8 upper=2.8 effort=122 velocity=4.6
- joint elbow_pitch_2: limit lower=-3 upper=3 effort=122 velocity=4.6 -> lower=-2.8 upper=2.8 effort=122 velocity=4.6
- joint hip_roll_1: limit lower=-2.03 upper=2.51 effort=185 velocity=7.6 -> lower=-0.65 upper=0.65 effort=185 velocity=7.6
- joint hip_roll_2: limit lower=-2.51 upper=2.03 effort=185 velocity=7.6 -> lower=-0.65 upper=0.65 effort=185 velocity=7.6
- joint hip_roll_3: limit lower=-2.51 upper=2.03 effort=185 velocity=7.6 -> lower=-0.65 upper=0.65 effort=185 velocity=7.6
- joint hip_roll_4: limit lower=-2.03 upper=2.51 effort=185 velocity=7.6 -> lower=-0.65 upper=0.65 effort=185 velocity=7.6
- joint knee_pitch_1: limit lower=-3.4056 upper=3.4056 effort=185 velocity=7.6 -> lower=-3.2 upper=3.2 effort=185 velocity=7.6
- joint knee_pitch_2: limit lower=-3.3266 upper=3.3266 effort=185 velocity=7.6 -> lower=-3.2 upper=3.2 effort=185 velocity=7.6
- joint knee_pitch_3: limit lower=-3.4696 upper=3.4696 effort=185 velocity=7.6 -> lower=-3.2 upper=3.2 effort=185 velocity=7.6
- joint knee_pitch_4: limit lower=-3.3426 upper=3.3426 effort=185 velocity=7.6 -> lower=-3.2 upper=3.2 effort=185 velocity=7.6
- joint reference: origin (none) -> xyz=0 0 0.6
- joint shoulder_pitch_1: limit lower=-3 upper=3 effort=122 velocity=4.6 -> lower=-2.2 upper=2.2 effort=146 velocity=3.8
- joint shoulder_pitch_2: limit lower=-3 upper=3 effort=122 velocity=4.6 -> lower=-2.2 upper=2.2 effort=146 velocity=3.8
- joint shoulder_yaw_1: limit lower=-3.312 upper=3.312 effort=146 velocity=3.8 -> lower=-3.0 upper=3.0 effort=122 velocity=4.6
- joint shoulder_yaw_2: limit lower=-3.3458 upper=3.3458 effort=146 velocity=3.8 -> lower=-3.0 upper=3.0 effort=122 velocity=4.6
- joint wheel_joint_1: limit lower=-1e9 upper=1e9 effort=100 velocity=20 -> lower=-1e9 upper=1e9 effort=100 velocity=30
- joint wheel_joint_2: limit lower=-1e9 upper=1e9 effort=100 velocity=20 -> lower=-1e9 upper=1e9 effort=100 velocity=30
- joint wheel_joint_3: limit lower=-1e9 upper=1e9 effort=100 velocity=20 -> lower=-1e9 upper=1e9 effort=100 velocity=30
- joint wheel_joint_4: limit lower=-1e9 upper=1e9 effort=100 velocity=20 -> lower=-1e9 upper=1e9 effort=100 velocity=30
- joint wrist_pitch_1: limit lower=-2.4056 upper=2.4056 effort=25 velocity=14 -> lower=-1.6 upper=1.6 effort=25 velocity=14
- joint wrist_pitch_2: limit lower=-2.3266 upper=2.3266 effort=25 velocity=14 -> lower=-1.6 upper=1.6 effort=25 velocity=14
- joint wrist_yaw_1: limit lower=-2.4056 upper=2.4056 effort=25 velocity=14 -> lower=-2.7 upper=2.7 effort=25 velocity=14
- joint wrist_yaw_2: limit lower=-2.3266 upper=2.3266 effort=25 velocity=14 -> lower=-2.7 upper=2.7 effort=25 velocity=14

File: kyon_urdf/urdf/parts/kyon_arm.urdf.xacro (robot description, xacro)
@@ -148,7 +148,5 @@
 	<limit lower="${j_wrist_yaw_lower[arm_num-1]}" upper="${j_wrist_yaw_upper[arm_num-1]}" effort="${motorD_effort}" velocity="${motorD_velocity}"/>
 </joint>
-<xacro:if value="${ADD_DAGANA}">
-	<xacro:kyon_dagana arm_num="${arm_num}" parent="wrist_yaw_${arm_num}_link"/>
-</xacro:if>
+<xacro:kyon_dagana arm_num="${arm_num}" parent="wrist_yaw_${arm_num}_link"/>
 </xacro:macro>
 <!-- /macro arms -->

File: kyon_urdf/urdf/parts/kyon_dagana.urdf.xacro (robot description, xacro)
@@ -16,5 +16,5 @@
         <material name="dark_grey"/>
     </visual>
-    <collision>
+    <!-- <collision>
         <origin xyz="0.0 0.0 0.0"  rpy="0.0 0.0 0.0"/>
         <geometry>
@@ -27,5 +27,5 @@
             <mesh filename="package://kyon_urdf/meshes/collision/mesh_dagana-base-base-simplified.stl" scale="0.001 0.001 0.001"/>
         </geometry>
-    </collision>
+    </collision> -->
 </link>
 <link name="dagana_${arm_num}_claw">
@@ -42,5 +42,5 @@
         <material name="dark_grey"/>
     </visual>
-    <collision>
+    <!-- <collision>
         <origin xyz="0.0 0.0 0.0"  rpy="0.0 0.0 0.0"/>
         <geometry>
@@ -53,5 +53,5 @@
             <mesh filename="package://kyon_urdf/meshes/collision/mesh_dagana-clamp-simplified.stl" scale="0.001 0.001 0.001"/>
         </geometry>
-    </collision>
+    </collision> -->
 </link>
 <joint name="dagana_${arm_num}_base_joint" type="fixed">

File: kyon_urdf/urdf/parts/kyon_leg.urdf.xacro (robot description, xacro)
@@ -80,10 +80,10 @@
 	<xacro:foot_leg leg_num="${leg_num}" parent="hip_pitch_${leg_num}_link" origin_x="${origin_x}" origin_y="${origin_y}" mirror="${mirror}"/>
 </xacro:unless>
+<!-- <xacro:if value="${ADD_WHEELS}"> -->
+	<!-- <xacro:steering_wheel leg_num="${leg_num}" parent="hip_pitch_${leg_num}_link" origin_x="${origin_x}" origin_y="${origin_y}" mirror="${mirror}"/> -->
+<!-- </xacro:if> -->
 <xacro:if value="${ADD_WHEELS}">
-	<xacro:steering_wheel leg_num="${leg_num}" parent="hip_pitch_${leg_num}_link" origin_x="${origin_x}" origin_y="${origin_y}" mirror="${mirror}"/>
+    <xacro:wheel_leg leg_num="${leg_num}" parent="hip_pitch_${leg_num}_link" origin_x="${origin_x}" origin_y="${origin_y}" mirror="${mirror}"/>
 </xacro:if>
-<!-- <xacro:if value="${ADD_WHEELS}">
-    <xacro:wheel_leg leg_num="${leg_num}" parent="hip_pitch_${leg_num}_link" origin_x="${origin_x}" origin_y="${origin_y}" mirror="${mirror}"/>
-</xacro:if> -->
 </xacro:macro>
 <!-- /macro legs -->
