Commit message: parking improvements

File: kyon_srdf/srdf/kyon.srdf.xacro (robot description, xacro)
@@ -168,15 +168,15 @@
     </group_state>
     <group_state name="parked" group="chains">
-        <joint name="hip_roll_1" value="0.0"/>
-        <joint name="hip_pitch_1" value="-1.57"/>
+        <joint name="hip_roll_1" value="0.06"/>
+        <joint name="hip_pitch_1" value="-1.53"/>
         <joint name="knee_pitch_1" value="3.10"/>
-        <joint name="hip_roll_2" value="0.0"/>
-        <joint name="hip_pitch_2" value="1.57"/>
+        <joint name="hip_roll_2" value="-0.06"/>
+        <joint name="hip_pitch_2" value="1.53"/>
         <joint name="knee_pitch_2" value="-3.1"/>
-        <joint name="hip_roll_3" value="0.0"/>
-        <joint name="hip_pitch_3" value="-1.57"/>
+        <joint name="hip_roll_3" value="-0.06"/>
+        <joint name="hip_pitch_3" value="-1.53"/>
         <joint name="knee_pitch_3" value="3.1"/>
-        <joint name="hip_roll_4" value="0.0"/>
-        <joint name="hip_pitch_4" value="1.57"/>
+        <joint name="hip_roll_4" value="0.06"/>
+        <joint name="hip_pitch_4" value="1.53"/>
         <joint name="knee_pitch_4" value="-3.1"/>
     </group_state>

Commit message: refined homing ub

File: kyon_srdf/srdf/kyon.srdf.xacro (robot description, xacro)
@@ -88,12 +88,12 @@
         <xacro:if value="${ADD_UPPER_BODY}">
             <joint name="shoulder_yaw_1" value="0.0"/>
-            <joint name="shoulder_pitch_1" value="1."/>
-            <joint name="elbow_pitch_1" value="2.1"/>
-            <joint name="wrist_pitch_1" value="0.7"/>
+            <joint name="shoulder_pitch_1" value="1.3"/>
+            <joint name="elbow_pitch_1" value="2.75"/>
+            <joint name="wrist_pitch_1" value="0.2"/>
             <joint name="wrist_yaw_1" value="0.0"/>
             <joint name="shoulder_yaw_2" value="0.0"/>
-            <joint name="shoulder_pitch_2" value="-1."/>
-            <joint name="elbow_pitch_2" value="-2.1"/>
-            <joint name="wrist_pitch_2" value="-0.7"/>
+            <joint name="shoulder_pitch_2" value="-1.3"/>
+            <joint name="elbow_pitch_2" value="-2.75"/>
+            <joint name="wrist_pitch_2" value="-0.2"/>
             <joint name="wrist_yaw_2" value="0.0"/>
         </xacro:if>

Commit message: first commit towards refactor

File: kyon_srdf/srdf/kyon.srdf.xacro (robot description, xacro)
@@ -44,5 +44,5 @@
 		</xacro:unless>
     </xacro:if>
-    <xacro:if value="${ADD_UPPER_BODY}">
+    <xacro:if value="${ADD_ARMS}">
 		<group name="left_arm">
 		    <chain base_link="pelvis" tip_link="dagana_1_claw"/>
@@ -59,5 +59,5 @@
             <group name="rear_left_leg" />
         </xacro:if>
-        <xacro:if value="${ADD_UPPER_BODY}">
+        <xacro:if value="${ADD_ARMS}">
             <group name="left_arm"/>
             <group name="right_arm"/>
@@ -66,4 +66,72 @@
     <!-- Homing posture -->
     <group_state name="home" group="chains">
+        <xacro:if value="${ADD_LEGS}">
+            <joint name="hip_roll_1" value="0.0"/>
+            <joint name="hip_pitch_1" value="-0.6"/>
+            <joint name="knee_pitch_1" value="1.2"/>
+            <joint name="hip_roll_2" value="-0.0"/>
+            <joint name="hip_pitch_2" value="0.6"/>
+            <joint name="knee_pitch_2" value="-1.2"/>
+            <joint name="hip_roll_3" value="-0.0"/>
+            <joint name="hip_pitch_3" value="-0.6"/>
+            <joint name="knee_pitch_3" value="1.2"/>
+            <joint name="hip_roll_4" value="0.0"/>
+            <joint name="hip_pitch_4" value="0.6"/>
+            <joint name="knee_pitch_4" value="-1.2"/>
+        </xacro:if>
+        <!-- <xacro:if value="${ADD_WHEELS}">
+            <joint name="ankle_yaw_1" value="0.0"/>
+            <joint name="ankle_yaw_2" value="0.0"/>
+            <joint name="ankle_yaw_3" value="0.0"/>
+            <joint name="ankle_yaw_4" value="0.0"/>
+        </xacro:if> -->
+        <xacro:if value="${ADD_ARMS}">
+            <joint name="shoulder_yaw_1" value="0.0"/>
+            <joint name="shoulder_pitch_1" value="1.3"/>
+            <joint name="elbow_pitch_1" value="2.75"/>
+            <joint name="wrist_pitch_1" value="0.2"/>
+            <joint name="wrist_yaw_1" value="0.0"/>
+            <joint name="shoulder_yaw_2" value="0.0"/>
+            <joint name="shoulder_pitch_2" value="-1.3"/>
+            <joint name="elbow_pitch_2" value="-2.75"/>
+            <joint name="wrist_pitch_2" value="-0.2"/>
+            <joint name="wrist_yaw_2" value="0.0"/>
+        </xacro:if>
+    </group_state>
+        <group_state name="home_isaac" group="chains">
+        <xacro:if value="${ADD_LEGS}">
+            <joint name="hip_roll_1" value="0.15"/>
+            <joint name="hip_pitch_1" value="-0.6"/>
+            <joint name="knee_pitch_1" value="1.2"/>
+            <joint name="hip_roll_2" value="-0.15"/>
+            <joint name="hip_pitch_2" value="0.6"/>
+            <joint name="knee_pitch_2" value="-1.2"/>
+            <joint name="hip_roll_3" value="-0.15"/>
+            <joint name="hip_pitch_3" value="-0.6"/>
+            <joint name="knee_pitch_3" value="1.2"/>
+            <joint name="hip_roll_4" value="0.15"/>
+            <joint name="hip_pitch_4" value="0.6"/>
+            <joint name="knee_pitch_4" value="-1.2"/>
+        </xacro:if>
+        <xacro:if value="${ADD_WHEELS}">
+            <joint name="ankle_yaw_1" value="0.0"/>
+            <joint name="ankle_yaw_2" value="0.0"/>
+            <joint name="ankle_yaw_3" value="0.0"/>
+            <joint name="ankle_yaw_4" value="0.0"/>
+        </xacro:if>
+        <xacro:if value="${ADD_ARMS}">
+            <joint name="shoulder_yaw_1" value="0.0"/>
+            <joint name="shoulder_pitch_1" value="1.5"/>
+            <joint name="elbow_pitch_1" value="2.5"/>
+            <joint name="wrist_pitch_1" value="0.7"/>
+            <joint name="wrist_yaw_1" value="0.0"/>
+            <joint name="shoulder_yaw_2" value="0.0"/>
+            <joint name="shoulder_pitch_2" value="-1.5"/>
+            <joint name="elbow_pitch_2" value="-2.5"/>
+            <joint name="wrist_pitch_2" value="-0.7"/>
+            <joint name="wrist_yaw_2" value="0.0"/>
+        </xacro:if>
+    </group_state>
+    <group_state name="home_isaac" group="chains">
         <xacro:if value="${ADD_LEGS}">
             <joint name="hip_roll_1" value="0.15"/>
@@ -80,38 +148,4 @@
             <joint name="knee_pitch_4" value="-1.4"/>
         </xacro:if>
-        <!-- <xacro:if value="${ADD_WHEELS}">
-            <joint name="ankle_yaw_1" value="0.0"/>
-            <joint name="ankle_yaw_2" value="0.0"/>
-            <joint name="ankle_yaw_3" value="0.0"/>
-            <joint name="ankle_yaw_4" value="0.0"/>
-        </xacro:if> -->
-        <xacro:if value="${ADD_UPPER_BODY}">
-            <joint name="shoulder_yaw_1" value="0.0"/>
-            <joint name="shoulder_pitch_1" value="1.3"/>
-            <joint name="elbow_pitch_1" value="2.75"/>
-            <joint name="wrist_pitch_1" value="0.2"/>
-            <joint name="wrist_yaw_1" value="0.0"/>
-            <joint name="shoulder_yaw_2" value="0.0"/>
-            <joint name="shoulder_pitch_2" value="-1.3"/>
-            <joint name="elbow_pitch_2" value="-2.75"/>
-            <joint name="wrist_pitch_2" value="-0.2"/>
-            <joint name="wrist_yaw_2" value="0.0"/>
-        </xacro:if>
-    </group_state>
-        <group_state name="home_isaac" group="chains">
-        <xacro:if value="${ADD_LEGS}">
-            <joint name="hip_roll_1" value="0.15"/>
-            <joint name="hip_pitch_1" value="-0.7"/>
-            <joint name="knee_pitch_1" value="1.4"/>
-            <joint name="hip_roll_2" value="-0.15"/>
-            <joint name="hip_pitch_2" value="0.7"/>
-            <joint name="knee_pitch_2" value="-1.4"/>
-            <joint name="hip_roll_3" value="-0.15"/>
-            <joint name="hip_pitch_3" value="-0.7"/>
-            <joint name="knee_pitch_3" value="1.4"/>
-            <joint name="hip_roll_4" value="0.15"/>
-            <joint name="hip_pitch_4" value="0.7"/>
-            <joint name="knee_pitch_4" value="-1.4"/>
-        </xacro:if>
         <xacro:if value="${ADD_WHEELS}">
             <joint name="ankle_yaw_1" value="0.0"/>
@@ -120,39 +154,5 @@
             <joint name="ankle_yaw_4" value="0.0"/>
         </xacro:if>
-        <xacro:if value="${ADD_UPPER_BODY}">
-            <joint name="shoulder_yaw_1" value="0.0"/>
-            <joint name="shoulder_pitch_1" value="1.5"/>
-            <joint name="elbow_pitch_1" value="2.5"/>
-            <joint name="wrist_pitch_1" value="0.7"/>
-            <joint name="wrist_yaw_1" value="0.0"/>
-            <joint name="shoulder_yaw_2" value="0.0"/>
-            <joint name="shoulder_pitch_2" value="-1.5"/>
-            <joint name="elbow_pitch_2" value="-2.5"/>
-            <joint name="wrist_pitch_2" value="-0.7"/>
-            <joint name="wrist_yaw_2" value="0.0"/>
-        </xacro:if>
-    </group_state>
-    <group_state name="home_isaac" group="chains">
-        <xacro:if value="${ADD_LEGS}">
-            <joint name="hip_roll_1" value="0.15"/>
-            <joint name="hip_pitch_1" value="-0.7"/>
-            <joint name="knee_pitch_1" value="1.4"/>
-            <joint name="hip_roll_2" value="-0.15"/>
-            <joint name="hip_pitch_2" value="0.7"/>
-            <joint name="knee_pitch_2" value="-1.4"/>
-            <joint name="hip_roll_3" value="-0.15"/>
-            <joint name="hip_pitch_3" value="-0.7"/>
-            <joint name="knee_pitch_3" value="1.4"/>
-            <joint name="hip_roll_4" value="0.15"/>
-            <joint name="hip_pitch_4" value="0.7"/>
-            <joint name="knee_pitch_4" value="-1.4"/>
-        </xacro:if>
-        <xacro:if value="${ADD_WHEELS}">
-            <joint name="ankle_yaw_1" value="0.0"/>
-            <joint name="ankle_yaw_2" value="0.0"/>
-            <joint name="ankle_yaw_3" value="0.0"/>
-            <joint name="ankle_yaw_4" value="0.0"/>
-        </xacro:if>
-        <xacro:if value="${ADD_UPPER_BODY}">
+        <xacro:if value="${ADD_ARMS}">
             <joint name="shoulder_yaw_1" value="0.0"/>
             <joint name="shoulder_pitch_1" value="1.5"/>

File: kyon_urdf/urdf/config/kyon.urdf.xacro (robot description, xacro)
@@ -5,5 +5,5 @@
 <!-- command line arguments -->
 <xacro:arg name="legs" default="true"/>
-<xacro:arg name="upper_body" default="true"/>
+<xacro:arg name="arms" default="true"/>
 <xacro:arg name="wheels" default="false"/>
 <xacro:arg name="floating_joint" default="true"/>
@@ -12,7 +12,5 @@
 <xacro:arg name="camera_left" default="false"/>
 <xacro:arg name="camera_right" default="false"/>
-<xacro:arg name="payload" default="false"/>
-<xacro:arg name="varta" default="false"/>
-<xacro:arg name="d034_li_ion" default="false"/>
+<xacro:arg name="battery" default="true"/>
 <xacro:arg name="velodyne" default="false"/>
 <xacro:arg name="add_collision" default="true"/>
@@ -21,5 +19,5 @@
 <!-- *************************************-->
 <xacro:property name="ADD_LEGS" value="$(arg legs)"/>
-<xacro:property name="ADD_UPPER_BODY" value="$(arg upper_body)"/>
+<xacro:property name="ADD_ARMS" value="$(arg arms)"/>
 <xacro:property name="ADD_CAMERAS" value="$(arg cameras)"/>
 <xacro:property name="ADD_FU_CAMERA" value="$(arg camera_front_up)"/>
@@ -28,6 +26,5 @@
 <xacro:property name="ADD_RIGHT_CAMERA" value="$(arg camera_right)"/>
 <xacro:property name="ADD_WHEELS" value="$(arg wheels)"/>
-<xacro:property name="ADD_VARTA" value="$(arg varta)"/>
-<xacro:property name="ADD_D034_LI_ION" value="$(arg d034_li_ion)"/>
+<xacro:property name="ADD_BATTERY" value="$(arg battery)"/>
 <xacro:property name="ADD_FLOATING_BASE" value="$(arg floating_joint)"/>
 <xacro:property name="ADD_VELODYNE" value="$(arg velodyne)"/>
@@ -35,4 +32,3 @@
 <xacro:property name="ADD_VIRTUAL_FRAME" value="false" />
 <xacro:property name="ADD_COLLISION" value="$(arg add_collision)"/>
-<xacro:property name="PAYLOAD" value="$(arg payload)"/>
 </robot>

File: kyon_urdf/urdf/gazebo/kyon.gazebo.xacro (robot description, xacro)
@@ -131,5 +131,5 @@
 		</gazebo>
     </xacro:if>
-    <xacro:if value="${ADD_UPPER_BODY}">
+    <xacro:if value="${ADD_ARMS}">
         <gazebo reference="shoulder_yaw_1">
             <implicitSpringDamper>1</implicitSpringDamper>

File: kyon_urdf/urdf/gazebo/materials.gazebo.xacro (robot description, xacro)
@@ -44,5 +44,5 @@
 	<xacro:kyon_leg_materials leg_num="4"/>
 </xacro:if>
-<xacro:if value="${ADD_UPPER_BODY}">
+<xacro:if value="${ADD_ARMS}">
 	<xacro:kyon_arm_materials arm_num="1"/>
 	<xacro:kyon_arm_materials arm_num="2"/>

File: kyon_urdf/urdf/kyon_base.urdf.xacro (robot description, xacro)
@@ -31,5 +31,5 @@
     </xacro:if>
 </link>
-<xacro:if value="${ADD_VARTA or ADD_D034_LI_ION}">
+<xacro:if value="${ADD_BATTERY}">
     <link name="battery">
         <inertial>
@@ -93,30 +93,9 @@
 	<child link="hesai_lidar"/>
 </joint>
-<xacro:if value="${ADD_UPPER_BODY}">
+<xacro:if value="${ADD_ARMS}">
     <xacro:include filename="$(find kyon_urdf)/urdf/parts/arms.urdf.xacro" />
 </xacro:if>
 <xacro:if value="${ADD_LEGS}">
 	<xacro:include filename="$(find kyon_urdf)/urdf/parts/legs.urdf.xacro" />
-</xacro:if>
-<xacro:if value="${PAYLOAD}">
-	<link name="payload_pelvis">
-		<inertial>
-		    <origin xyz="0.0 0.0 0.0"/>
-			<mass value="20"/>
-			<inertia ixx="0.13" iyy="0.13" izz="0.13" ixy="0" ixz="0" iyz="0"/>
-		</inertial>
-		<visual>
-			<origin xyz="0.0 0.0 0.0"  rpy="0.0 0.0 0.0"/>
-			<geometry>
-				<box size="0.2 0.2 0.2"/>
-			</geometry>
-			<material name="dark_grey"/>
-		</visual>
-	</link>
-	<joint name="pelvis_to_payload" type="fixed">
-		<origin xyz="-0.2 0.0 ${pelvis_height / 2 + 0.1}"/>
-		<parent link="pelvis"/>
-		<child link="payload_pelvis"/>
-	</joint>
 </xacro:if>
 <!-- Hesai JT128 -->

File: kyon_urdf/urdf/parts/arms.urdf.xacro (robot description, xacro)
@@ -7,43 +7,3 @@
 <xacro:kyon_arm arm_num="2" rot="1"  parent="pelvis">
 </xacro:kyon_arm>
-<xacro:if value="${PAYLOAD}">
-	<link name="payload_1">
-		<inertial>
-			<origin xyz="0.0 0.0 0.0"/>
-			<mass value="4"/>
-			<inertia ixx="0.0267" iyy="0.0267" izz="0.0267" ixy="0" ixz="0" iyz="0"/>
-		</inertial>
-		<visual>
-			<origin xyz="0.0 0.0 0.0"  rpy="0.0 0.0 0.0"/>
-			<geometry>
-				<box size="0.2 0.2 0.2"/>
-			</geometry>
-			<material name="dark_grey"/>
-		</visual>
-	</link>
-	<joint name="hand_to_payload_1" type="fixed">
-		<origin xyz="0 0.1 0.0" rpy="0 0 0"/>
-		<parent link="dagana_1_bottom_link"/>
-		<child link="payload_1"/>
-	</joint>
-	<link name="payload_2">
-		<inertial>
-			<origin xyz="0.0 0.0 0.0"/>
-			<mass value="4"/>
-			<inertia ixx="0.0267" iyy="0.0267" izz="0.0267" ixy="0" ixz="0" iyz="0"/>
-		</inertial>
-		<visual>
-			<origin xyz="0.0 0.0 0.0"  rpy="0.0 0.0 0.0"/>
-			<geometry>
-				<box size="0.2 0.2 0.2"/>
-			</geometry>
-			<material name="dark_grey"/>
-		</visual>
-	</link>
-	<joint name="hand_to_payload_2" type="fixed">
-		<origin xyz="0 0.1 0.0" rpy="0 0 0"/>
-		<parent link="dagana_2_bottom_link"/>
-		<child link="payload_2"/>
-	</joint>
-</xacro:if>
 </robot>

File: kyon_urdf/urdf/parts/inertial_properties.urdf.xacro (robot description, xacro)
@@ -3,9 +3,6 @@
     <xacro:property name="mm2Tom2" value="${0.001*0.001}"/>
     <!-- Battery -->
-    <xacro:if value="${ADD_VARTA}">
+    <xacro:if value="${ADD_BATTERY}">
         <xacro:property name="Battery_mass" value="9.8"/>
-    </xacro:if>
-    <xacro:if value="${ADD_D034_LI_ION}">
-        <xacro:property name="Battery_mass" value="5.8"/>
     </xacro:if>
     <xacro:property name="Battery_xx" value="${1/12 * Battery_mass * (Battery_zsize * Battery_zsize + Battery_ysize * Battery_ysize)}"/>

File: kyon_urdf/urdf/parts/kinematics_properties.urdf.xacro (robot description, xacro)
@@ -5,13 +5,8 @@
     <!-- Compound properties (i.e. based on the props parsed from the yaml) -->
     <!-- Battery -->
-    <xacro:if value="${ADD_VARTA}">
+    <xacro:if value="${ADD_BATTERY}">
         <xacro:property name="Battery_xsize" value="${329.000 * mmTom}"/>
         <xacro:property name="Battery_ysize" value="${225.000 * mmTom}"/>
         <xacro:property name="Battery_zsize" value="${79.300 * mmTom}"/>
-    </xacro:if>
-    <xacro:if value="${ADD_D034_LI_ION}">
-        <xacro:property name="Battery_xsize" value="${262.000 * mmTom}"/>
-        <xacro:property name="Battery_ysize" value="${50.000 * mmTom}"/>
-        <xacro:property name="Battery_zsize" value="${72.300 * mmTom}"/>
     </xacro:if>
     <xacro:property name="Battery_Ox" value="0.0"/>

File: kyon_urdf/urdf/parts/kyon_leg.urdf.xacro (robot description, xacro)
@@ -83,7 +83,4 @@
 	<xacro:steering_wheel leg_num="${leg_num}" parent="hip_pitch_${leg_num}_link" origin_x="${origin_x}" origin_y="${origin_y}" mirror="${mirror}"/>
 </xacro:if>
-<!-- <xacro:if value="${ADD_WHEELS}"> -->
-    <!-- <xacro:wheel_leg leg_num="${leg_num}" parent="hip_pitch_${leg_num}_link" origin_x="${origin_x}" origin_y="${origin_y}" mirror="${mirror}"/> -->
-<!-- </xacro:if> -->
 </xacro:macro>
 <!-- /macro legs -->

Commit message: homing ub not in self collision according to capsule

File: kyon_srdf/srdf/kyon.srdf.xacro (robot description, xacro)
@@ -89,11 +89,11 @@
             <joint name="shoulder_yaw_1" value="0.0"/>
             <joint name="shoulder_pitch_1" value="1.3"/>
-            <joint name="elbow_pitch_1" value="2.75"/>
-            <joint name="wrist_pitch_1" value="0.2"/>
+            <joint name="elbow_pitch_1" value="2.50"/>
+            <joint name="wrist_pitch_1" value="0.45"/>
             <joint name="wrist_yaw_1" value="0.0"/>
             <joint name="shoulder_yaw_2" value="0.0"/>
             <joint name="shoulder_pitch_2" value="-1.3"/>
-            <joint name="elbow_pitch_2" value="-2.75"/>
-            <joint name="wrist_pitch_2" value="-0.2"/>
+            <joint name="elbow_pitch_2" value="-2.50"/>
+            <joint name="wrist_pitch_2" value="-0.45"/>
             <joint name="wrist_yaw_2" value="0.0"/>
         </xacro:if>
