Commit message: fix cameras in gz

File: kyon_gazebo/urdf/kyon_sensors.urdf.xacro (robot description, xacro)
@@ -3,6 +3,4 @@
     <gazebo reference="imu_link">
         <sensor name="imu_link" type="imu">
-            <gz_frame_id>imu_link</gz_frame_id>
-            <pose relative_to='imu_link'>0 0 0 0 0 0</pose>
             <always_on>1</always_on>
             <update_rate>200</update_rate>
@@ -11,40 +9,4 @@
         </sensor>
     </gazebo>
-    <xacro:if value="${ADD_HESAI_JT128}">
-        <gazebo reference="hesai_jt128_joint">
-            <preserveFixedJoint>true</preserveFixedJoint>
-        </gazebo>
-        <gazebo reference="hesai_jt128_link">
-            <sensor name="hesai_jt128_gpu_lidar" type="gpu_lidar">
-                <gz_frame_id>hesai_jt128_link</gz_frame_id>
-                <pose>0 0 0 0 0 0</pose>
-                <topic>/hesai_jt128</topic>
-                <update_rate>20</update_rate>
-                <ray>
-                    <scan>
-                        <horizontal>
-                            <samples>1800</samples>
-                            <resolution>1</resolution>
-                            <min_angle>-3.14159265359</min_angle>
-                            <max_angle>3.14159265359</max_angle>
-                        </horizontal>
-                        <vertical>
-                            <samples>128</samples>
-                            <resolution>1</resolution>
-                            <min_angle>-1.64933614313</min_angle>
-                            <max_angle>1.64933614313</max_angle>
-                        </vertical>
-                    </scan>
-                    <range>
-                        <min>0.05</min>
-                        <max>40.0</max>
-                        <resolution>0.01</resolution>
-                    </range>
-                </ray>
-                <always_on>true</always_on>
-                <visualize>true</visualize>
-            </sensor>
-        </gazebo>
-    </xacro:if>
     <xacro:if value="${ADD_VELODYNE}">
         <gazebo reference="hesai_lidar">
@@ -65,6 +27,6 @@
                             <samples>16</samples>
                             <resolution>1</resolution>
-                            <min_angle>-${52.5*PI/180.0}</min_angle>
-                            <max_angle>${52.5*PI/180.0}</max_angle>
+                            <min_angle>-${52.5*M_PI/180.0}</min_angle>
+                            <max_angle>${52.5*M_PI/180.0}</max_angle>
                         </vertical>
                     </scan>

File: kyon_urdf/urdf/config/kyon.urdf.xacro (robot description, xacro)
@@ -8,5 +8,8 @@
 <xacro:arg name="wheels" default="false"/>
 <xacro:arg name="floating_joint" default="true"/>
-<xacro:arg name="cameras" default="false"/>
+<xacro:arg name="camera_front_up" default="false"/>
+<xacro:arg name="camera_front_down" default="false"/>
+<xacro:arg name="camera_left" default="false"/>
+<xacro:arg name="camera_right" default="false"/>
 <xacro:arg name="payload" default="false"/>
 <xacro:arg name="varta" default="false"/>
@@ -21,4 +24,8 @@
 <xacro:property name="ADD_UPPER_BODY" value="$(arg upper_body)"/>
 <xacro:property name="ADD_CAMERAS" value="$(arg cameras)"/>
+<xacro:property name="ADD_FU_CAMERA" value="$(arg camera_front_up)"/>
+<xacro:property name="ADD_FD_CAMERA" value="$(arg camera_front_down)"/>
+<xacro:property name="ADD_LEFT_CAMERA" value="$(arg camera_left)"/>
+<xacro:property name="ADD_RIGHT_CAMERA" value="$(arg camera_right)"/>
 <xacro:property name="ADD_WHEELS" value="$(arg wheels)"/>
 <xacro:property name="ADD_VARTA" value="$(arg varta)"/>

File: kyon_urdf/urdf/kyon_base.urdf.xacro (robot description, xacro)
@@ -86,91 +86,4 @@
     <origin xyz="0 -0.150100 0.109486" rpy="0 0.3490656 -1.5707963"/>
 </joint>
-<xacro:if value="${ADD_CAMERAS}">
-    <xacro:include filename="$(find realsense_gazebo_description)/urdf/_d435i.urdf.xacro" />
-    <!-- LEFT D435 CAMERA -->
-    <xacro:sensor_d435i parent="left_camera_mount_link"
-        name="D435_left"
-        topics_ns="D435_left"
-        enable_pointCloud="true"
-        align_depth="true"
-        unite_imu_method="false"
-        visualize="false"
-        accel_fps="300"
-        gyro_fps="300"
-        depth_width="1280"
-        depth_height="720"
-        depth_fps="10"
-        infra_width="1280"
-        infra_height="720"
-        infra_fps="10"
-        color_width="1280"
-        color_height="720"
-        color_fps="1">
-        <origin xyz="0 0 0" rpy="0 0 0"/>
-    </xacro:sensor_d435i>
-    <!-- RIGHT D435 CAMERA -->
-    <xacro:sensor_d435i parent="right_camera_mount_link"
-        name="D435_right"
-        topics_ns="D435_right"
-        enable_pointCloud="true"
-        align_depth="true"
-        unite_imu_method="false"
-        visualize="false"
-        accel_fps="300"
-        gyro_fps="300"
-        depth_width="1280"
-        depth_height="720"
-        depth_fps="10"
-        infra_width="1280"
-        infra_height="720"
-        infra_fps="10"
-        color_width="1280"
-        color_height="720"
-        color_fps="1">
-        <origin xyz="0 0 0" rpy="0 0 0"/>
-    </xacro:sensor_d435i>
-    <!-- FRONT1 D435 CAMERA -->
-    <xacro:sensor_d435i parent="zed_front_up_mount_link"
-        name="D435_front1"
-        topics_ns="D435_front1"
-        enable_pointCloud="true"
-        align_depth="true"
-        unite_imu_method="false"
-        visualize="false"
-        accel_fps="300"
-        gyro_fps="300"
-        depth_width="1280"
-        depth_height="720"
-        depth_fps="90"
-        infra_width="1280"
-        infra_height="720"
-        infra_fps="90"
-        color_width="1280"
-        color_height="720"
-        color_fps="30">
-        <origin xyz="0 0 0" rpy="0 0 0"/>
-    </xacro:sensor_d435i>
-    <!-- FRONT2 D435 CAMERA -->
-    <xacro:sensor_d435i parent="zed_front_down_mount_link"
-        name="D435_front2"
-        topics_ns="D435_front2"
-        enable_pointCloud="true"
-        align_depth="true"
-        unite_imu_method="false"
-        visualize="false"
-        accel_fps="300"
-        gyro_fps="300"
-        depth_width="1280"
-        depth_height="720"
-        depth_fps="90"
-        infra_width="1280"
-        infra_height="720"
-        infra_fps="90"
-        color_width="1280"
-        color_height="720"
-        color_fps="30">
-        <origin xyz="0 0 0" rpy="0 0 0"/>
-    </xacro:sensor_d435i>
-</xacro:if>
 <!-- Velodyne -->
 <link name="hesai_lidar"/>

Commit message: some updates

File: kyon_gazebo/urdf/kyon_sensors.urdf.xacro (robot description, xacro)
@@ -3,4 +3,6 @@
     <gazebo reference="imu_link">
         <sensor name="imu_link" type="imu">
+            <gz_frame_id>imu_link</gz_frame_id>
+            <pose relative_to='imu_link'>0 0 0 0 0 0</pose>
             <always_on>1</always_on>
             <update_rate>200</update_rate>
@@ -9,4 +11,40 @@
         </sensor>
     </gazebo>
+    <xacro:if value="${ADD_HESAI_JT128}">
+        <gazebo reference="hesai_jt128_joint">
+            <preserveFixedJoint>true</preserveFixedJoint>
+        </gazebo>
+        <gazebo reference="hesai_jt128_link">
+            <sensor name="hesai_jt128_gpu_lidar" type="gpu_lidar">
+                <gz_frame_id>hesai_jt128_link</gz_frame_id>
+                <pose>0 0 0 0 0 0</pose>
+                <topic>/hesai_jt128</topic>
+                <update_rate>20</update_rate>
+                <ray>
+                    <scan>
+                        <horizontal>
+                            <samples>1800</samples>
+                            <resolution>1</resolution>
+                            <min_angle>-3.14159265359</min_angle>
+                            <max_angle>3.14159265359</max_angle>
+                        </horizontal>
+                        <vertical>
+                            <samples>128</samples>
+                            <resolution>1</resolution>
+                            <min_angle>-1.64933614313</min_angle>
+                            <max_angle>1.64933614313</max_angle>
+                        </vertical>
+                    </scan>
+                    <range>
+                        <min>0.05</min>
+                        <max>40.0</max>
+                        <resolution>0.01</resolution>
+                    </range>
+                </ray>
+                <always_on>true</always_on>
+                <visualize>true</visualize>
+            </sensor>
+        </gazebo>
+    </xacro:if>
     <xacro:if value="${ADD_VELODYNE}">
         <gazebo reference="hesai_lidar">
@@ -27,6 +65,6 @@
                             <samples>16</samples>
                             <resolution>1</resolution>
-                            <min_angle>-${52.5*M_PI/180.0}</min_angle>
-                            <max_angle>${52.5*M_PI/180.0}</max_angle>
+                            <min_angle>-${52.5*PI/180.0}</min_angle>
+                            <max_angle>${52.5*PI/180.0}</max_angle>
                         </vertical>
                     </scan>

File: kyon_srdf/srdf/kyon.srdf.xacro (robot description, xacro)
@@ -46,18 +46,8 @@
     <xacro:if value="${ADD_UPPER_BODY}">
 		<group name="left_arm">
-            <xacro:if value="${ADD_DAGANA}">
-			    <chain base_link="pelvis" tip_link="dagana_1_claw"/>
-            </xacro:if>
-            <xacro:unless value="${ADD_DAGANA}">
-                <chain base_link="pelvis" tip_link="wrist_yaw_1_link"/>
-            </xacro:unless>
-		</group>
+		    <chain base_link="pelvis" tip_link="dagana_1_claw"/>
+     		</group>
 		<group name="right_arm">
-            <xacro:if value="${ADD_DAGANA}">
-			    <chain base_link="pelvis" tip_link="dagana_2_claw"/>
-            </xacro:if>
-            <xacro:unless value="${ADD_DAGANA}">
-                <chain base_link="pelvis" tip_link="wrist_yaw_2_link"/>
-            </xacro:unless>
+		    <chain base_link="pelvis" tip_link="dagana_2_claw"/>
 		</group>
     </xacro:if>
@@ -77,14 +67,48 @@
     <group_state name="home" group="chains">
         <xacro:if value="${ADD_LEGS}">
-            <joint name="hip_roll_1" value="0.0"/>
+            <joint name="hip_roll_1" value="0.15"/>
             <joint name="hip_pitch_1" value="-0.7"/>
             <joint name="knee_pitch_1" value="1.4"/>
-            <joint name="hip_roll_2" value="0.0"/>
+            <joint name="hip_roll_2" value="-0.15"/>
             <joint name="hip_pitch_2" value="0.7"/>
             <joint name="knee_pitch_2" value="-1.4"/>
-            <joint name="hip_roll_3" value="0.0"/>
+            <joint name="hip_roll_3" value="-0.15"/>
             <joint name="hip_pitch_3" value="-0.7"/>
             <joint name="knee_pitch_3" value="1.4"/>
-            <joint name="hip_roll_4" value="0.0"/>
+            <joint name="hip_roll_4" value="0.15"/>
+            <joint name="hip_pitch_4" value="0.7"/>
+            <joint name="knee_pitch_4" value="-1.4"/>
+        </xacro:if>
+        <!-- <xacro:if value="${ADD_WHEELS}">
+            <joint name="ankle_yaw_1" value="0.0"/>
+            <joint name="ankle_yaw_2" value="0.0"/>
+            <joint name="ankle_yaw_3" value="0.0"/>
+            <joint name="ankle_yaw_4" value="0.0"/>
+        </xacro:if> -->
+        <xacro:if value="${ADD_UPPER_BODY}">
+            <joint name="shoulder_yaw_1" value="0.0"/>
+            <joint name="shoulder_pitch_1" value="1."/>
+            <joint name="elbow_pitch_1" value="2.1"/>
+            <joint name="wrist_pitch_1" value="0.7"/>
+            <joint name="wrist_yaw_1" value="0.0"/>
+            <joint name="shoulder_yaw_2" value="0.0"/>
+            <joint name="shoulder_pitch_2" value="-1."/>
+            <joint name="elbow_pitch_2" value="-2.1"/>
+            <joint name="wrist_pitch_2" value="-0.7"/>
+            <joint name="wrist_yaw_2" value="0.0"/>
+        </xacro:if>
+    </group_state>
+        <group_state name="home_isaac" group="chains">
+        <xacro:if value="${ADD_LEGS}">
+            <joint name="hip_roll_1" value="0.15"/>
+            <joint name="hip_pitch_1" value="-0.7"/>
+            <joint name="knee_pitch_1" value="1.4"/>
+            <joint name="hip_roll_2" value="-0.15"/>
+            <joint name="hip_pitch_2" value="0.7"/>
+            <joint name="knee_pitch_2" value="-1.4"/>
+            <joint name="hip_roll_3" value="-0.15"/>
+            <joint name="hip_pitch_3" value="-0.7"/>
+            <joint name="knee_pitch_3" value="1.4"/>
+            <joint name="hip_roll_4" value="0.15"/>
             <joint name="hip_pitch_4" value="0.7"/>
             <joint name="knee_pitch_4" value="-1.4"/>
@@ -98,12 +122,12 @@
         <xacro:if value="${ADD_UPPER_BODY}">
             <joint name="shoulder_yaw_1" value="0.0"/>
-            <joint name="shoulder_pitch_1" value="1.0"/>
-            <joint name="elbow_pitch_1" value="2.0"/>
-            <joint name="wrist_pitch_1" value="0.5"/>
+            <joint name="shoulder_pitch_1" value="1.5"/>
+            <joint name="elbow_pitch_1" value="2.5"/>
+            <joint name="wrist_pitch_1" value="0.7"/>
             <joint name="wrist_yaw_1" value="0.0"/>
             <joint name="shoulder_yaw_2" value="0.0"/>
-            <joint name="shoulder_pitch_2" value="-1.0"/>
-            <joint name="elbow_pitch_2" value="-2.0"/>
-            <joint name="wrist_pitch_2" value="-0.5"/>
+            <joint name="shoulder_pitch_2" value="-1.5"/>
+            <joint name="elbow_pitch_2" value="-2.5"/>
+            <joint name="wrist_pitch_2" value="-0.7"/>
             <joint name="wrist_yaw_2" value="0.0"/>
         </xacro:if>

File: kyon_urdf/urdf/config/kyon.urdf.xacro (robot description, xacro)
@@ -16,11 +16,10 @@
 <xacro:arg name="d034_li_ion" default="false"/>
 <xacro:arg name="velodyne" default="false"/>
-<xacro:arg name="dagana" default="$(arg upper_body)"/>
 <xacro:arg name="add_collision" default="true"/>
+<xacro:arg name="hesai_jt128" default="false"/>
 <!-- ************SELECT PARTS*************-->
 <!-- *************************************-->
 <xacro:property name="ADD_LEGS" value="$(arg legs)"/>
 <xacro:property name="ADD_UPPER_BODY" value="$(arg upper_body)"/>
-<xacro:property name="ADD_DAGANA" value="$(arg dagana)"/>
 <xacro:property name="ADD_CAMERAS" value="$(arg cameras)"/>
 <xacro:property name="ADD_FU_CAMERA" value="$(arg camera_front_up)"/>
@@ -33,4 +32,5 @@
 <xacro:property name="ADD_FLOATING_BASE" value="$(arg floating_joint)"/>
 <xacro:property name="ADD_VELODYNE" value="$(arg velodyne)"/>
+<xacro:property name="ADD_HESAI_JT128" value="$(arg hesai_jt128)"/>
 <xacro:property name="ADD_VIRTUAL_FRAME" value="false" />
 <xacro:property name="ADD_COLLISION" value="$(arg add_collision)"/>

File: kyon_urdf/urdf/kyon_base.urdf.xacro (robot description, xacro)
@@ -93,17 +93,4 @@
 	<child link="hesai_lidar"/>
 </joint>
-<xacro:if value="${ADD_VELODYNE}">
-    <xacro:include filename="$(find velodyne_description)/urdf/VLP-16.urdf.xacro"/>
-    <xacro:VLP-16 parent="pelvis" name="velodyne" topic="/velodyne_points" hz="10" samples="440">
-        <origin xyz="0.43 0 0.118" rpy="0 0 0.5220063" />
-    </xacro:VLP-16>
-</xacro:if>
-<!-- Velodyne -->
-<xacro:if value="${ADD_VELODYNE}">
-    <xacro:include filename="$(find velodyne_description)/urdf/VLP-16.urdf.xacro"/>
-    <xacro:VLP-16 parent="pelvis" name="velodyne">
-        <origin xyz="0.47 0 0.11" rpy="0 0 0" />
-    </xacro:VLP-16>
-</xacro:if>
 <xacro:if value="${ADD_UPPER_BODY}">
     <xacro:include filename="$(find kyon_urdf)/urdf/parts/arms.urdf.xacro" />
@@ -133,3 +120,27 @@
 	</joint>
 </xacro:if>
+<!-- Hesai JT128 -->
+<xacro:if value="${ADD_HESAI_JT128}">
+    <link name="hesai_jt128_link">
+        <inertial>
+        <mass value="0.2"/>
+        <origin xyz="0 0 0" rpy="0 0 0"/>
+        <inertia ixx="0.001" ixy="0" ixz="0"
+                iyy="0.001" iyz="0"
+                izz="0.001"/>
+        </inertial>
+        <visual>
+            <origin xyz="0.0 0.0 0.0"  rpy="0.0 0.0 0.0"/>
+            <geometry>
+                <mesh filename="package://kyon_urdf/meshes/hesai_jt128.stl" scale="0.0001 0.0001 0.0001"/>
+            </geometry>
+            <material name="dark_grey"/>
+        </visual>
+    </link>
+    <joint name="hesai_jt128_joint" type="fixed">
+        <origin xyz="0.43 0 -0.118" rpy="${PI} 0 0" />
+        <parent link="pelvis"/>
+        <child link="hesai_jt128_link"/>
+    </joint>
+</xacro:if>
 </robot>

Commit message: added second hesai_jt128

File: kyon_gazebo/urdf/kyon_sensors.urdf.xacro (robot description, xacro)
@@ -12,12 +12,46 @@
     </gazebo>
     <xacro:if value="${ADD_HESAI_JT128}">
-        <gazebo reference="hesai_jt128_joint">
+        <gazebo reference="hesai_jt128_front_joint">
             <preserveFixedJoint>true</preserveFixedJoint>
         </gazebo>
-        <gazebo reference="hesai_jt128_link">
-            <sensor name="hesai_jt128_gpu_lidar" type="gpu_lidar">
-                <gz_frame_id>hesai_jt128_link</gz_frame_id>
+        <gazebo reference="hesai_jt128_front_link">
+            <sensor name="hesai_jt128_gpu_lidar_front" type="gpu_lidar">
+                <gz_frame_id>hesai_jt128_front_link</gz_frame_id>
                 <pose>0 0 0 0 0 0</pose>
-                <topic>/hesai_jt128</topic>
+                <topic>/hesai_jt128_front</topic>
+                <update_rate>20</update_rate>
+                <ray>
+                    <scan>
+                        <horizontal>
+                            <samples>1800</samples>
+                            <resolution>1</resolution>
+                            <min_angle>-3.14159265359</min_angle>
+                            <max_angle>3.14159265359</max_angle>
+                        </horizontal>
+                        <vertical>
+                            <samples>128</samples>
+                            <resolution>1</resolution>
+                            <min_angle>-1.64933614313</min_angle>
+                            <max_angle>1.64933614313</max_angle>
+                        </vertical>
+                    </scan>
+                    <range>
+                        <min>0.05</min>
+                        <max>40.0</max>
+                        <resolution>0.01</resolution>
+                    </range>
+                </ray>
+                <always_on>true</always_on>
+                <visualize>true</visualize>
+            </sensor>
+        </gazebo>
+        <gazebo reference="hesai_jt128_back_joint">
+            <preserveFixedJoint>true</preserveFixedJoint>
+        </gazebo>
+        <gazebo reference="hesai_jt128_back_link">
+            <sensor name="hesai_jt128_gpu_lidar_back" type="gpu_lidar">
+                <gz_frame_id>hesai_jt128_back_link</gz_frame_id>
+                <pose>0 0 0 0 0 0</pose>
+                <topic>/hesai_jt128_back</topic>
                 <update_rate>20</update_rate>
                 <ray>

File: kyon_urdf/urdf/kyon_base.urdf.xacro (robot description, xacro)
@@ -122,5 +122,5 @@
 <!-- Hesai JT128 -->
 <xacro:if value="${ADD_HESAI_JT128}">
-    <link name="hesai_jt128_link">
+    <link name="hesai_jt128_front_link">
         <inertial>
         <mass value="0.2"/>
@@ -138,8 +138,29 @@
         </visual>
     </link>
-    <joint name="hesai_jt128_joint" type="fixed">
+    <joint name="hesai_jt128_front_joint" type="fixed">
         <origin xyz="0.43 0 -0.118" rpy="${PI} 0 0" />
         <parent link="pelvis"/>
-        <child link="hesai_jt128_link"/>
+        <child link="hesai_jt128_front_link"/>
+    </joint>
+    <link name="hesai_jt128_back_link">
+        <inertial>
+        <mass value="0.2"/>
+        <origin xyz="0 0 0" rpy="0 0 0"/>
+        <inertia ixx="0.001" ixy="0" ixz="0"
+                iyy="0.001" iyz="0"
+                izz="0.001"/>
+        </inertial>
+        <visual>
+            <origin xyz="0.0 0.0 0.0"  rpy="0.0 0.0 0.0"/>
+            <geometry>
+                <mesh filename="package://kyon_urdf/meshes/hesai_jt128.stl" scale="0.0001 0.0001 0.0001"/>
+            </geometry>
+            <material name="dark_grey"/>
+        </visual>
+    </link>
+    <joint name="hesai_jt128_back_joint" type="fixed">
+        <origin xyz="-0.43 0 -0.118" rpy="${PI} 0 0" />
+        <parent link="pelvis"/>
+        <child link="hesai_jt128_back_link"/>
     </joint>
 </xacro:if>

File: kyon_urdf/urdf/kyon_spheres.urdf (robot description, URDF)
Before this commit: robot kyon, 40 links, 39 joints
Links:
- removed link hesai_jt128_link
- added link hesai_jt128_back_link, mass 0.2; collision sphere radius=0.05; visual mesh filename=package://hesai_jt128_gz_sim_plugin/meshes/hesai_jt128.stl scale=0.0001 0.0001 0.0001
- added link hesai_jt128_front_link, mass 0.2; collision sphere radius=0.05; visual mesh filename=package://hesai_jt128_gz_sim_plugin/meshes/hesai_jt128.stl scale=0.0001 0.0001 0.0001
Joints:
- removed joint hesai_jt128_joint
- added joint hesai_jt128_back_joint: type fixed, parent pelvis, child hesai_jt128_back_link, origin xyz=-0.43 0 -0.118 rpy=3.14159265359 0 0
- added joint hesai_jt128_front_joint: type fixed, parent pelvis, child hesai_jt128_front_link, origin xyz=0.43 0 -0.118 rpy=3.14159265359 0 0
