Commit message: changed few variable names

File: kyon_gazebo/urdf/kyon_sensors.urdf.xacro (robot description, xacro)
@@ -81,5 +81,5 @@
         </gazebo>
     </xacro:if>
-    <xacro:if value="${ADD_VELODYNE}">
+    <xacro:if value="${ADD_LIDAR}">
         <gazebo reference="hesai_lidar">
             <sensor name='gpu_lidar' type='gpu_lidar'>

File: kyon_srdf/srdf/kyon.srdf.xacro (robot description, xacro)
@@ -68,15 +68,15 @@
         <xacro:if value="${ADD_LEGS}">
             <joint name="hip_roll_1" value="0.0"/>
-            <joint name="hip_pitch_1" value="-0.6"/>
-            <joint name="knee_pitch_1" value="1.2"/>
+            <joint name="hip_pitch_1" value="-0.7"/>
+            <joint name="knee_pitch_1" value="1.4"/>
             <joint name="hip_roll_2" value="-0.0"/>
-            <joint name="hip_pitch_2" value="0.6"/>
-            <joint name="knee_pitch_2" value="-1.2"/>
+            <joint name="hip_pitch_2" value="0.7"/>
+            <joint name="knee_pitch_2" value="-1.4"/>
             <joint name="hip_roll_3" value="-0.0"/>
-            <joint name="hip_pitch_3" value="-0.6"/>
-            <joint name="knee_pitch_3" value="1.2"/>
+            <joint name="hip_pitch_3" value="-0.7"/>
+            <joint name="knee_pitch_3" value="1.4"/>
             <joint name="hip_roll_4" value="0.0"/>
-            <joint name="hip_pitch_4" value="0.6"/>
-            <joint name="knee_pitch_4" value="-1.2"/>
+            <joint name="hip_pitch_4" value="0.7"/>
+            <joint name="knee_pitch_4" value="-1.4"/>
         </xacro:if>
         <!-- <xacro:if value="${ADD_WHEELS}">
@@ -99,18 +99,18 @@
         </xacro:if>
     </group_state>
-        <group_state name="home_isaac" group="chains">
+    <group_state name="home_isaac" group="chains">
         <xacro:if value="${ADD_LEGS}">
             <joint name="hip_roll_1" value="0.15"/>
-            <joint name="hip_pitch_1" value="-0.6"/>
-            <joint name="knee_pitch_1" value="1.2"/>
+            <joint name="hip_pitch_1" value="-0.7"/>
+            <joint name="knee_pitch_1" value="1.4"/>
             <joint name="hip_roll_2" value="-0.15"/>
-            <joint name="hip_pitch_2" value="0.6"/>
-            <joint name="knee_pitch_2" value="-1.2"/>
+            <joint name="hip_pitch_2" value="0.7"/>
+            <joint name="knee_pitch_2" value="-1.4"/>
             <joint name="hip_roll_3" value="-0.15"/>
-            <joint name="hip_pitch_3" value="-0.6"/>
-            <joint name="knee_pitch_3" value="1.2"/>
+            <joint name="hip_pitch_3" value="-0.7"/>
+            <joint name="knee_pitch_3" value="1.4"/>
             <joint name="hip_roll_4" value="0.15"/>
-            <joint name="hip_pitch_4" value="0.6"/>
-            <joint name="knee_pitch_4" value="-1.2"/>
+            <joint name="hip_pitch_4" value="0.7"/>
+            <joint name="knee_pitch_4" value="-1.4"/>
         </xacro:if>
         <xacro:if value="${ADD_WHEELS}">

File: kyon_urdf/urdf/config/kyon.urdf.xacro (robot description, xacro)
@@ -10,8 +10,6 @@
 <xacro:arg name="camera_front_up" default="false"/>
 <xacro:arg name="camera_front_down" default="false"/>
-<xacro:arg name="camera_left" default="false"/>
-<xacro:arg name="camera_right" default="false"/>
 <xacro:arg name="battery" default="true"/>
-<xacro:arg name="velodyne" default="false"/>
+<xacro:arg name="lidar" default="false"/>
 <xacro:arg name="add_collision" default="true"/>
 <xacro:arg name="hesai_jt128" default="false"/>
@@ -28,11 +26,8 @@
 <xacro:property name="ADD_FU_CAMERA" value="$(arg camera_front_up)"/>
 <xacro:property name="ADD_FD_CAMERA" value="$(arg camera_front_down)"/>
-<xacro:property name="ADD_FD_ZED_MODEL" value="$(arg add_zed_model_front_down)"/>
-<xacro:property name="ADD_LEFT_CAMERA" value="$(arg camera_left)"/>
-<xacro:property name="ADD_RIGHT_CAMERA" value="$(arg camera_right)"/>
 <xacro:property name="ADD_WHEELS" value="$(arg wheels)"/>
 <xacro:property name="ADD_BATTERY" value="$(arg battery)"/>
 <xacro:property name="ADD_FLOATING_BASE" value="$(arg floating_joint)"/>
-<xacro:property name="ADD_VELODYNE" value="$(arg velodyne)"/>
+<xacro:property name="ADD_LIDAR" value="$(arg lidar)"/>
 <xacro:property name="ADD_HESAI_JT128" value="$(arg hesai_jt128)"/>
 <xacro:property name="ADD_VIRTUAL_FRAME" value="false" />

File: kyon_urdf/urdf/kyon_base.urdf.xacro (robot description, xacro)
@@ -74,17 +74,5 @@
     <origin xyz="0.509601 0 0.00343992" rpy="0 0.9250251 0"/>
 </joint>
-<link name="left_camera_mount_link"/>
-<joint name="left_camera_mount_joint" type="fixed">
-    <parent link="pelvis"/>
-    <child link="left_camera_mount_link"/>
-    <origin xyz="0 0.150100 0.109486" rpy="0 0.3490656 1.5707963"/>
-</joint>
-<link name="right_camera_mount_link"/>
-<joint name="right_camera_mount_joint" type="fixed">
-    <parent link="pelvis"/>
-    <child link="right_camera_mount_link"/>
-    <origin xyz="0 -0.150100 0.109486" rpy="0 0.3490656 -1.5707963"/>
-</joint>
-<!-- Velodyne -->
+<!-- lidar -->
 <link name="hesai_lidar"/>
 <joint name="hesai_lidar_joints" type="fixed">

Commit message: worlds/gz/sensors tweaks

File: kyon_gazebo/urdf/kyon_sensors.urdf.xacro (robot description, xacro)
@@ -147,9 +147,11 @@
             <sensor name="zed_front_down" type="rgbd_camera">
                 <gz_frame_id>zed_front_down_mount_link</gz_frame_id>
+                <!-- Left-lens offset, matching _LEFT_EYE_OFFSET in kyon_isaac rough_vision_env_cfg.py -->
+                <pose relative_to="zed_front_down_mount_link">0.015 0.025 0.015 0 0 0</pose>
                 <camera>
-                    <horizontal_fov>1.83</horizontal_fov>
+                    <horizontal_fov>1.8403</horizontal_fov>
                     <image>
-                        <width>320</width>
-                        <height>240</height>
+                        <width>96</width>
+                        <height>60</height>
                     </image>
                     <clip>
@@ -161,5 +163,5 @@
                     <clip>
                         <near>0.1</near>
-                        <far>5.0</far>
+                        <far>20.0</far>
                     </clip>
                 </depth_camera>

File: kyon_urdf/urdf/kyon_base.urdf.xacro (robot description, xacro)
@@ -57,5 +57,8 @@
 <link name="imu_link"/>
 <joint name="imu_joint" type="fixed">
-	<origin xyz="-0.256190 0 0.103" rpy="${PI} 0 0"/>
+	<!-- rpy zeroed: the gazebo IMU already publishes pelvis-aligned data, so the toolkit
+	     applying rpy=pi as base_T_imu inverted projected_gravity. Restore for real hw. -->
+	<origin xyz="-0.256190 0 0.103" rpy="0 0 0"/>
+	<!-- <origin xyz="-0.256190 0 0.103" rpy="${PI} 0 0"/> -->
     <parent link="pelvis"/>
     <child link="imu_link"/>

Commit message: gazebo: remove additional fake link not matching real robot urdf

File: kyon_gazebo/urdf/kyon_sensors.urdf.xacro (robot description, xacro)
@@ -115,16 +115,10 @@
     </xacro:if>
     <!-- Hesai QT128: 1800 x 264 rows of 0.4 deg, sim_hesai_adapter picks one per ring
-         (config/sim_hesai_adapter.yaml must match) -->
+         (config/sim_hesai_adapter.yaml must match). No TF frame of its own: the real robot has none. -->
     <xacro:if value="$(arg hesai_qt128)">
-        <link name="hesai_qt128"/>
-        <joint name="hesai_qt128_joint" type="fixed">
-            <parent link="$(arg hesai_qt128_parent)"/>
-            <child link="hesai_qt128"/>
-            <origin xyz="$(arg hesai_qt128_x) $(arg hesai_qt128_y) $(arg hesai_qt128_z)"
-                    rpy="$(arg hesai_qt128_roll) $(arg hesai_qt128_pitch) $(arg hesai_qt128_yaw)"/>
-        </joint>
-        <gazebo reference="hesai_qt128">
+        <gazebo reference="$(arg hesai_qt128_parent)">
             <sensor name="hesai_qt128" type="gpu_lidar">
-                <gz_frame_id>hesai_qt128</gz_frame_id>
+                <gz_frame_id>hesai_lidar</gz_frame_id>
+                <pose relative_to="$(arg hesai_qt128_parent)">$(arg hesai_qt128_x) $(arg hesai_qt128_y) $(arg hesai_qt128_z) $(arg hesai_qt128_roll) $(arg hesai_qt128_pitch) $(arg hesai_qt128_yaw)</pose>
                 <topic>/hesai_qt128</topic>
                 <update_rate>10</update_rate>
