Commit message: gazebo: add qt128 adapter to match gz and real sensor

File: kyon_gazebo/urdf/kyon_gazebo.urdf.xacro (robot description, xacro)
@@ -1,4 +1,16 @@
 <?xml version="1.0"?>
 <robot xmlns:xacro="http://ros.org/wiki/xacro" name="kyon">
+<!-- Hesai QT128 on hesai_qt128_parent; default pose: lio_mapping's calibrated extrinsic (imu_link) -->
+<xacro:arg name="hesai_qt128" default="false"/>
+<xacro:arg name="hesai_qt128_parent" default="imu_link"/>
+<xacro:arg name="hesai_qt128_x" default="0.6862"/>
+<xacro:arg name="hesai_qt128_y" default="0.0"/>
+<xacro:arg name="hesai_qt128_z" default="-0.015"/>
+<xacro:arg name="hesai_qt128_roll" default="3.141592653589793"/>
+<xacro:arg name="hesai_qt128_pitch" default="0.0"/>
+<xacro:arg name="hesai_qt128_yaw" default="-2.0928021889929584"/>
+<!-- World pose of the root link (pelvis) as nav_msgs/Odometry -->
+<xacro:arg name="ground_truth" default="false"/>
+<xacro:arg name="ground_truth_topic" default="/sim/ground_truth"/>
 <xacro:include filename="$(find kyon_urdf)/urdf/kyon_robot.urdf.xacro" />
 <xacro:include filename="$(find kyon_gazebo)/urdf/kyon_sensors.urdf.xacro" />

File: kyon_gazebo/urdf/kyon_sensors.urdf.xacro (robot description, xacro)
@@ -114,4 +114,62 @@
         </gazebo>
     </xacro:if>
+    <!-- Hesai QT128: 1800 x 264 rows of 0.4 deg, sim_hesai_adapter picks one per ring
+         (config/sim_hesai_adapter.yaml must match) -->
+    <xacro:if value="$(arg hesai_qt128)">
+        <link name="hesai_qt128"/>
+        <joint name="hesai_qt128_joint" type="fixed">
+            <parent link="$(arg hesai_qt128_parent)"/>
+            <child link="hesai_qt128"/>
+            <origin xyz="$(arg hesai_qt128_x) $(arg hesai_qt128_y) $(arg hesai_qt128_z)"
+                    rpy="$(arg hesai_qt128_roll) $(arg hesai_qt128_pitch) $(arg hesai_qt128_yaw)"/>
+        </joint>
+        <gazebo reference="hesai_qt128">
+            <sensor name="hesai_qt128" type="gpu_lidar">
+                <gz_frame_id>hesai_qt128</gz_frame_id>
+                <topic>/hesai_qt128</topic>
+                <update_rate>10</update_rate>
+                <always_on>true</always_on>
+                <visualize>false</visualize>
+                <lidar>
+                    <scan>
+                        <!-- One column per 0.2 deg over [-pi, pi) -->
+                        <horizontal>
+                            <samples>1800</samples>
+                            <resolution>1</resolution>
+                            <min_angle>${-PI}</min_angle>
+                            <max_angle>${PI - 2*PI/1800}</max_angle>
+                        </horizontal>
+                        <vertical>
+                            <samples>264</samples>
+                            <resolution>1</resolution>
+                            <min_angle>${-52.8*PI/180.0}</min_angle>
+                            <max_angle>${52.4*PI/180.0}</max_angle>
+                        </vertical>
+                    </scan>
+                    <range>
+                        <min>0.05</min>
+                        <max>50.0</max>
+                        <resolution>0.01</resolution>
+                    </range>
+                    <noise>
+                        <type>gaussian</type>
+                        <mean>0.0</mean>
+                        <stddev>0.01</stddev>
+                    </noise>
+                </lidar>
+            </sensor>
+        </gazebo>
+    </xacro:if>
+    <xacro:if value="$(arg ground_truth)">
+        <gazebo>
+            <plugin filename="gz-sim-odometry-publisher-system" name="gz::sim::systems::OdometryPublisher">
+                <odom_frame>sim_world</odom_frame>
+                <robot_base_frame>pelvis</robot_base_frame>
+                <odom_topic>$(arg ground_truth_topic)</odom_topic>
+                <dimensions>3</dimensions>
+                <odom_publish_frequency>200</odom_publish_frequency>
+            </plugin>
+        </gazebo>
+    </xacro:if>
     <xacro:if value="${ADD_FU_CAMERA}">
         <gazebo reference="zed_front_up_mount_link">
