Commit message: added force/torque sensors to knee
Signed-off-by: FrancescoRuscelli <francescoruscelli24@gmail.com>

File: kyon_urdf/urdf/config/kyon.urdf.xacro (robot description, xacro)
@@ -11,4 +11,5 @@
 <xacro:arg name="sensors" default="true"/>
 <xacro:arg name="payload" default="false"/>
+<xacro:arg name="ft_sensors" default="false"/>
 <!-- ************SELECT PARTS*************-->
 <!-- *************************************-->
@@ -18,4 +19,5 @@
 <xacro:property name="ADD_DAGANA" value="$(arg dagana)"/>
 <xacro:property name="ADD_WHEELS" value="$(arg wheels)"/>
+<xacro:property name="ADD_FT_SENSORS" value="$(arg ft_sensors)"/>
 <xacro:property name="ADD_FLOATING_BASE" value="$(arg floating_joint)" />
 <xacro:property name="ADD_VIRTUAL_FRAME" value="false" />

File: kyon_urdf/urdf/gazebo/kyon.gazebo.xacro (robot description, xacro)
@@ -229,3 +229,10 @@
         </gazebo>
     </xacro:if>
+	<xacro:if value="${ADD_FT_SENSORS}">
+		<xacro:include filename="$(find kyon_urdf)/urdf/gazebo/ft_sensors.gazebo.xacro" />
+		<xacro:kyon_ft_sensor frame_id="knee_pitch_1"/>
+		<xacro:kyon_ft_sensor frame_id="knee_pitch_2"/>
+		<xacro:kyon_ft_sensor frame_id="knee_pitch_3"/>
+		<xacro:kyon_ft_sensor frame_id="knee_pitch_4"/>
+	</xacro:if>
 </robot>
