Commit message: new macros for modular legs (missing wheel configuration)

File: kyon_urdf/urdf/config/kyon.urdf.xacro (robot description, xacro)
@@ -7,4 +7,5 @@
 <xacro:arg name="upper_body" default="true"/>
 <xacro:arg name="dagana" default="false"/>
+<xacro:arg name="feet" default="true"/>
 <xacro:arg name="wheels" default="false"/>
 <xacro:arg name="floating_joint" default="true"/>
@@ -12,4 +13,5 @@
 <xacro:arg name="payload" default="false"/>
 <xacro:arg name="ft_sensors" default="false"/>
+<xacro:arg name="steering_wheels" default="false"/>
 <!-- ************SELECT PARTS*************-->
 <!-- *************************************-->
@@ -18,5 +20,7 @@
 <xacro:property name="ADD_SENSORS" value="$(arg sensors)" />
 <xacro:property name="ADD_DAGANA" value="$(arg dagana)"/>
+<xacro:property name="ADD_FEET" value="$(arg feet)"/>
 <xacro:property name="ADD_WHEELS" value="$(arg wheels)"/>
+<xacro:property name="ADD_STEERING_WHEELS" value="$(arg steering_wheels)"/>
 <xacro:property name="ADD_FT_SENSORS" value="$(arg ft_sensors)"/>
 <xacro:property name="ADD_FLOATING_BASE" value="$(arg floating_joint)" />

File: kyon_urdf/urdf/kyon.urdf (robot description, URDF)
Before this commit: robot kyon, 42 links, 41 joints
Links:
- removed link ball_1
- removed link ball_2
- removed link ball_3
- removed link ball_4
- removed link hip_pitch_motor_1
- removed link hip_pitch_motor_2
- removed link hip_pitch_motor_3
- removed link hip_pitch_motor_4
- removed link hip_roll_motor_1
- removed link hip_roll_motor_2
- removed link hip_roll_motor_3
- removed link hip_roll_motor_4
- removed link knee_pitch_motor_1
- removed link knee_pitch_motor_2
- removed link knee_pitch_motor_3
- removed link knee_pitch_motor_4
- removed link lower_leg_1
- removed link lower_leg_2
- removed link lower_leg_3
- removed link lower_leg_4
- removed link upper_leg_1
- removed link upper_leg_2
- removed link upper_leg_3
- removed link upper_leg_4
- added link hip_pitch_1, mass 1.8; collision mesh filename=package://kyon_urdf/meshes/collision/mesh_hip-pitch.stl scale=0.001 0.001 0.001; visual mesh filename=package://kyon_urdf/meshes/mesh_hip-pitch.stl scale=0.001 0.001 0.001
- added link hip_pitch_2, mass 1.8; collision mesh filename=package://kyon_urdf/meshes/collision/mesh_hip-pitch.stl scale=0.001 0.001 0.001; visual mesh filename=package://kyon_urdf/meshes/mesh_hip-pitch.stl scale=0.001 0.001 0.001
- added link hip_pitch_3, mass 1.8; collision mesh filename=package://kyon_urdf/meshes/collision/mesh_hip-pitch.stl scale=0.001 0.001 0.001; visual mesh filename=package://kyon_urdf/meshes/mesh_hip-pitch.stl scale=0.001 0.001 0.001
- added link hip_pitch_4, mass 1.8; collision mesh filename=package://kyon_urdf/meshes/collision/mesh_hip-pitch.stl scale=0.001 0.001 0.001; visual mesh filename=package://kyon_urdf/meshes/mesh_hip-pitch.stl scale=0.001 0.001 0.001
- added link hip_roll_1, mass 1.8; collision mesh filename=package://kyon_urdf/meshes/collision/mesh_hip-roll.stl scale=0.001 -0.001 0.001; visual mesh filename=package://kyon_urdf/meshes/mesh_hip-roll.stl scale=0.001 -0.001 0.001
- added link hip_roll_2, mass 1.8; collision mesh filename=package://kyon_urdf/meshes/collision/mesh_hip-roll.stl scale=0.001 0.001 0.001; visual mesh filename=package://kyon_urdf/meshes/mesh_hip-roll.stl scale=0.001 0.001 0.001
- added link hip_roll_3, mass 1.8; collision mesh filename=package://kyon_urdf/meshes/collision/mesh_hip-roll.stl scale=0.001 -0.001 0.001; visual mesh filename=package://kyon_urdf/meshes/mesh_hip-roll.stl scale=0.001 -0.001 0.001
- added link hip_roll_4, mass 1.8; collision mesh filename=package://kyon_urdf/meshes/collision/mesh_hip-roll.stl scale=0.001 0.001 0.001; visual mesh filename=package://kyon_urdf/meshes/mesh_hip-roll.stl scale=0.001 0.001 0.001
- added link knee_pitch_1, mass 1.8; collision mesh filename=package://kyon_urdf/meshes/collision/mesh_foot-leg.stl scale=-0.001 0.001 0.001; visual mesh filename=package://kyon_urdf/meshes/mesh_foot-leg.stl scale=-0.001 0.001 0.001
- added link knee_pitch_2, mass 1.8; collision mesh filename=package://kyon_urdf/meshes/collision/mesh_foot-leg.stl scale=0.001 0.001 0.001; visual mesh filename=package://kyon_urdf/meshes/mesh_foot-leg.stl scale=0.001 0.001 0.001
- added link knee_pitch_3, mass 1.8; collision mesh filename=package://kyon_urdf/meshes/collision/mesh_foot-leg.stl scale=-0.001 0.001 0.001; visual mesh filename=package://kyon_urdf/meshes/mesh_foot-leg.stl scale=-0.001 0.001 0.001
- added link knee_pitch_4, mass 1.8; collision mesh filename=package://kyon_urdf/meshes/collision/mesh_foot-leg.stl scale=0.001 0.001 0.001; visual mesh filename=package://kyon_urdf/meshes/mesh_foot-leg.stl scale=0.001 0.001 0.001
Joints:
- removed joint ball_joint_1
- removed joint ball_joint_2
- removed joint ball_joint_3
- removed joint ball_joint_4
- removed joint hip_pitch_stator_1
- removed joint hip_pitch_stator_2
- removed joint hip_pitch_stator_3
- removed joint hip_pitch_stator_4
- removed joint knee_pitch_stator_1
- removed joint knee_pitch_stator_2
- removed joint knee_pitch_stator_3
- removed joint knee_pitch_stator_4
- joint hip_pitch_1: child upper_leg_1 -> hip_pitch_1; origin xyz=0.0 -0.0 0.0 rpy=0.0 0.0 0.0 -> xyz=0.0 0.05086 0.0 rpy=-1.57079632679 1.57079632679 0.0; parent hip_pitch_motor_1 -> hip_roll_1
- joint hip_pitch_2: child upper_leg_2 -> hip_pitch_2; origin xyz=0.0 0.0 0.0 rpy=0.0 0.0 0.0 -> xyz=0.0 -0.05086 0.0 rpy=1.57079632679 -1.57079632679 0.0; parent hip_pitch_motor_2 -> hip_roll_2
- joint hip_pitch_3: child upper_leg_3 -> hip_pitch_3; origin xyz=0.0 -0.0 0.0 rpy=0.0 0.0 0.0 -> xyz=-0.0 0.05086 0.0 rpy=-1.57079632679 -1.57079632679 0.0; parent hip_pitch_motor_3 -> hip_roll_3
- joint hip_pitch_4: child upper_leg_4 -> hip_pitch_4; origin xyz=0.0 0.0 0.0 rpy=0.0 0.0 0.0 -> xyz=-0.0 -0.05086 0.0 rpy=1.57079632679 1.57079632679 0.0; parent hip_pitch_motor_4 -> hip_roll_4
- joint hip_roll_1: child hip_roll_motor_1 -> hip_roll_1; origin xyz=0.41 0.0775 0.0 rpy=0.0 1.57079632679 0.0 -> xyz=0.40936 0.0775 0.0 rpy=0.0 1.57079632679 0.0
- joint hip_roll_2: child hip_roll_motor_2 -> hip_roll_2; origin xyz=0.41 -0.0775 0.0 rpy=0.0 1.57079632679 0.0 -> xyz=0.40936 -0.0775 0.0 rpy=0.0 1.57079632679 0.0
- joint hip_roll_3: child hip_roll_motor_3 -> hip_roll_3; origin xyz=-0.41 0.0775 0.0 rpy=0.0 1.57079632679 0.0 -> xyz=-0.40936 0.0775 0.0 rpy=0.0 -1.57079632679 0.0
- joint hip_roll_4: child hip_roll_motor_4 -> hip_roll_4; origin xyz=-0.41 -0.0775 0.0 rpy=0.0 1.57079632679 0.0 -> xyz=-0.40936 -0.0775 0.0 rpy=0.0 -1.57079632679 0.0
- joint knee_pitch_1: child lower_leg_1 -> knee_pitch_1; origin xyz=0.35 0.0 0.0 rpy=0.0 0.0 0.0 -> xyz=0.0 -0.34600000000000003 0.16671000000000002 rpy=0.0 0.0 0.0; parent upper_leg_1 -> hip_pitch_1
- joint knee_pitch_2: child lower_leg_2 -> knee_pitch_2; origin xyz=0.35 0.0 0.0 rpy=0.0 0.0 0.0 -> xyz=0.0 -0.34600000000000003 0.16671000000000002 rpy=0.0 0.0 0.0; parent upper_leg_2 -> hip_pitch_2
- joint knee_pitch_3: child lower_leg_3 -> knee_pitch_3; origin xyz=0.35 0.0 0.0 rpy=0.0 0.0 0.0 -> xyz=0.0 -0.34600000000000003 0.16671000000000002 rpy=0.0 0.0 0.0; parent upper_leg_3 -> hip_pitch_3
- joint knee_pitch_4: child lower_leg_4 -> knee_pitch_4; origin xyz=0.35 0.0 0.0 rpy=0.0 0.0 0.0 -> xyz=0.0 -0.34600000000000003 0.16671000000000002 rpy=0.0 0.0 0.0; parent upper_leg_4 -> hip_pitch_4

File: kyon_urdf/urdf/parts/kinematics_properties.urdf.xacro (robot description, xacro)
@@ -27,6 +27,6 @@
     <!-- Compound properties (i.e. based on the props parsed from the yaml) -->
     <!-- Origin -->
-    <xacro:property name="HipRoll_Ox" value="${pelvis_length / 2}"/>
-    <xacro:property name="HipRoll_Oy" value="${-pelvis_width / 2}"/>
+    <xacro:property name="HipRoll_Ox" value="${409.360 * mTomm}"/>
+    <xacro:property name="HipRoll_Oy" value="${77.500 * mTomm}"/>
     <xacro:property name="HipRoll_Oz" value="0.0"/>
     <xacro:property name="HipRoll_roll" value="0.0"/>
@@ -35,37 +35,31 @@
     <!-- Origin -->
     <xacro:property name="HipPitch_Ox" value="0.0"/>
-    <xacro:property name="HipPitch_Oy" value="${-cylinder_radius - cylinder_length / 2}"/>
+    <xacro:property name="HipPitch_Oy" value="${50.860 * mmTom}"/>
     <xacro:property name="HipPitch_Oz" value="0.0"/>
     <xacro:property name="HipPitch_roll" value="${-PI_2}"/>
-    <xacro:property name="HipPitch_pitch" value="0.0"/>
+    <xacro:property name="HipPitch_pitch" value="${PI_2}"/>
     <xacro:property name="HipPitch_yaw" value="0.0"/>
-    <xacro:property name="UpperLeg_Ox" value="0.0"/>
-    <xacro:property name="UpperLeg_Oy" value="0.0"/>
-    <xacro:property name="UpperLeg_Oz" value="0.0"/>
-    <xacro:property name="UpperLeg_roll" value="0.0"/>
-    <xacro:property name="UpperLeg_pitch" value="0.0"/>
-    <xacro:property name="UpperLeg_yaw" value="0.0"/>
     <!-- Origin -->
     <xacro:property name="KneePitch_Ox" value="0.0"/>
-    <xacro:property name="KneePitch_Oy" value="0.0"/>
-    <xacro:property name="KneePitch_Oz" value="0.0"/>
+    <xacro:property name="KneePitch_Oy" value="${-346.000 * mmTom}"/>
+    <xacro:property name="KneePitch_Oz" value="${166.710 * mmTom}"/>
     <xacro:property name="KneePitch_roll" value="0.0"/>
     <xacro:property name="KneePitch_pitch" value="0.0"/>
     <xacro:property name="KneePitch_yaw" value="0.0"/>
-    <xacro:property name="LowerLeg_Ox" value="${upper_leg_length}"/>
-    <xacro:property name="LowerLeg_Oy" value="0.0"/>
-    <xacro:property name="LowerLeg_Oz" value="0.0"/>
-    <xacro:property name="LowerLeg_roll" value="0.0"/>
-    <xacro:property name="LowerLeg_pitch" value="0.0"/>
-    <xacro:property name="LowerLeg_yaw" value="0.0"/>
+    <xacro:property name="AnkleYaw_Ox" value="0.0"/>
+    <xacro:property name="AnkleYaw_Oy" value="${-10.000 * mmTom}"/>
+    <xacro:property name="AnkleYaw_Oz" value="${67.000 * mmTom}"/>
+    <xacro:property name="AnkleYaw_roll" value="-${PI_2}"/>
+    <xacro:property name="AnkleYaw_pitch" value="0.0"/>
+    <xacro:property name="AnkleYaw_yaw" value="0.0"/>
     <!-- Origin -->
-    <xacro:property name="Ankle_Ox" value="${lower_leg_length}"/>
-    <xacro:property name="Ankle_Oy" value="0.0"/>
-    <xacro:property name="Ankle_Oz" value="0.0"/>
-    <xacro:property name="Ankle_roll" value="0.0"/>
-    <xacro:property name="Ankle_pitch" value="0.0"/>
-    <xacro:property name="Ankle_yaw" value="0.0"/>
+    <xacro:property name="Wheel_Ox" value="0.0"/>
+    <xacro:property name="Wheel_Oy" value="0.0"/>
+    <xacro:property name="Wheel_Oz" value="${-290.000 * mmTom}"/>
+    <xacro:property name="Wheel_roll" value="${PI_2}"/>
+    <xacro:property name="Wheel_pitch" value="0.0"/>
+    <xacro:property name="Wheel_yaw" value="0.0"/>
     <!-- Arms -->
-    <xacro:property name="ShoulderYaw_Ox" value="${320.00 * mTomm}"/>
+    <xacro:property name="ShoulderYaw_Ox" value="${270.00 * mTomm}"/>
     <xacro:property name="ShoulderYaw_Oy" value="${102.996 * mTomm}"/>
     <xacro:property name="ShoulderYaw_Oz" value="${187.217 * mTomm}"/>
@@ -78,5 +72,5 @@
     <xacro:property name="ShoulderPitch_roll" value="0.0"/>
     <xacro:property name="ShoulderPitch_pitch" value="0.0"/>
-    <xacro:property name="ShoulderPitch_yaw" value="${PI_2}"/>>
+    <xacro:property name="ShoulderPitch_yaw" value="${PI_2}"/>
     <xacro:property name="ElbowPitch_Ox" value="0.0"/>
     <xacro:property name="ElbowPitch_Oy" value="0.0"/>

File: kyon_urdf/urdf/parts/kyon_leg.urdf.xacro (robot description, xacro)
@@ -1,8 +1,33 @@
 <?xml version="1.0"?>
 <robot xmlns:xacro="http://ros.org/wiki/xacro">
+<!-- include end-effectors -->
+<xacro:include filename="$(find kyon_urdf)/urdf/parts/foot_leg.urdf.xacro" />
+<xacro:include filename="$(find kyon_urdf)/urdf/parts/steering_wheel.urdf.xacro" />
 <!-- macro legs -->
 <xacro:macro name="kyon_leg" params="leg_num origin_x origin_y mirror">
 <!-- links -->
-<link name="hip_roll_motor_${leg_num}">
+<link name="hip_roll_${leg_num}">
+	<inertial>
+		<origin xyz="0.0 0.0 0.0"/>
+		<mass value="${motorA_mass}"/>
+		<inertia ixx="${MotorA_xx}" ixy="${mirror*MotorA_xy}" ixz="${MotorA_xz}" iyy="${MotorA_yy}" iyz="${mirror*MotorA_yz}" izz="${MotorA_zz}"/>
+	</inertial>
+	<visual>
+		<origin xyz="0.0 0.0 0.0"  rpy="0.0 0.0 0.0"/>
+	  	<geometry>
+	 		<!-- <cylinder radius="${cylinder_radius}" length="${cylinder_length}"/> -->
+			<mesh filename="package://kyon_urdf/meshes/mesh_hip-roll.stl" scale="0.001 ${mirror*0.001} 0.001"/>
+		</geometry>
+  		<material name="dark_grey"/>
+	</visual>
+	<collision>
+		<origin xyz="0.0 0.0 0.0"  rpy="0.0 0.0 0.0"/>
+		<geometry>
+	 		<!-- <cylinder radius="${cylinder_radius}" length="${cylinder_length}"/> -->
+			<mesh filename="package://kyon_urdf/meshes/collision/mesh_hip-roll.stl" scale="0.001 ${mirror*0.001} 0.001"/>
+		</geometry>
+	</collision>
+</link>
+<link name="hip_pitch_${leg_num}">
 	<inertial>
 		<origin xyz="0.0 0.0 0.0"/>
@@ -13,5 +38,5 @@
 		<origin xyz="0.0 0.0 0.0"  rpy="0.0 0.0 0.0"/>
 	  	<geometry>
-	 		<cylinder radius="${cylinder_radius}" length="${cylinder_length}"/>
+	 		<mesh filename="package://kyon_urdf/meshes/mesh_hip-pitch.stl" scale="0.001 0.001 0.001"/>
 	  	</geometry>
   		<material name="dark_grey"/>
@@ -20,179 +45,29 @@
 		<origin xyz="0.0 0.0 0.0"  rpy="0.0 0.0 0.0"/>
 		<geometry>
-			<cylinder radius="${cylinder_radius}" length="${cylinder_length}"/>
+			<mesh filename="package://kyon_urdf/meshes/collision/mesh_hip-pitch.stl" scale="0.001 0.001 0.001"/>
 		</geometry>
 	</collision>
 </link>
-<link name="hip_pitch_motor_${leg_num}">
-	<inertial>
-		<origin xyz="0.0 0.0 0.0"/>
-		<mass value="${motorA_mass}"/>
-		<inertia ixx="${MotorA_xx}" ixy="${MotorA_xy}" ixz="${MotorA_xz}" iyy="${MotorA_yy}" iyz="${MotorA_yz}" izz="${MotorA_zz}"/>
-	</inertial>
-	<visual>
-		<origin xyz="0.0 0.0 0.0"  rpy="0.0 0.0 0.0"/>
-	  	<geometry>
-	 		<cylinder radius="${cylinder_radius}" length="${cylinder_length}"/>
-	  	</geometry>
-  		<material name="dark_grey"/>
-	</visual>
-	<collision>
-		<origin xyz="0.0 0.0 0.0"  rpy="0.0 0.0 0.0"/>
-		<geometry>
-			<cylinder radius="${cylinder_radius}" length="${cylinder_length}"/>
-		</geometry>
-	</collision>
-</link>
-<link name="knee_pitch_motor_${leg_num}">
-	<inertial>
-		<origin xyz="0.0 0.0 0.0"/>
-		<mass value="${motorA_mass}"/>
-		<inertia ixx="${MotorA_xx}" ixy="${MotorA_xy}" ixz="${MotorA_xz}" iyy="${MotorA_yy}" iyz="${MotorA_yz}" izz="${MotorA_zz}"/>
-	</inertial>
-	<visual>
-		<origin xyz="0.0 0.0 0.0"  rpy="0.0 0.0 0.0"/>
-	  	<geometry>
-	 		<cylinder radius="${cylinder_radius}" length="${cylinder_length}"/>
-	  	</geometry>
-  		<material name="dark_grey"/>
-	</visual>
-	<collision>
-		<origin xyz="0.0 0.0 0.0"  rpy="0.0 0.0 0.0"/>
-		<geometry>
-			<cylinder radius="${cylinder_radius}" length="${cylinder_length}"/>
-		</geometry>
-	</collision>
-</link>
-<link name="upper_leg_${leg_num}">
-	<inertial>
-		<origin xyz="${upper_leg_length / 2} 0.0 0.0"/>
-		<mass value="${upper_leg_mass}"/>
-		<inertia ixx="${UpperLeg_xx}" ixy="${UpperLeg_xy}" ixz="${UpperLeg_xz}" iyy="${UpperLeg_yy}" iyz="${UpperLeg_yz}" izz="${UpperLeg_zz}"/>
-	</inertial>
-	<origin xyz="0.0 0.0 0.0" rpy="0.0 0.0 0.0"/>
-	<visual>
-		<origin xyz="${upper_leg_length / 2} 0.0 0.0"  rpy="0.0 0.0 0.0"/>
-	  	<geometry>
-	 		<box size="${upper_leg_length} ${upper_leg_width} ${upper_leg_height}"/>
-	  	</geometry>
-  		<material name="dark_grey"/>
-	</visual>
-	<collision>
-		<origin xyz="${upper_leg_length / 2} 0.0 0.0"  rpy="0.0 0.0 0.0"/>
-		<geometry>
-			<box size="${upper_leg_length} ${upper_leg_width} ${upper_leg_height}"/>
-		</geometry>
-	</collision>
-</link>
-<link name="lower_leg_${leg_num}">
-	<inertial>
-		<origin xyz="${lower_leg_length / 2} 0.0 0.0"/>
-		<mass value="${lower_leg_mass}"/>
-		<inertia ixx="${LowerLeg_xx}" ixy="${LowerLeg_xy}" ixz="${LowerLeg_xz}" iyy="${LowerLeg_yy}" iyz="${LowerLeg_yz}" izz="${LowerLeg_zz}"/>
-	</inertial>
-	<visual>
-		<origin xyz="${lower_leg_length / 2} 0.0 0.0"  rpy="0.0 0.0 0.0"/>
-	  	<geometry>
-	 		<box size="${lower_leg_length} ${lower_leg_width} ${lower_leg_height}"/>
-	  	</geometry>
-  		<material name="dark_grey"/>
-	</visual>
-	<collision>
-		<origin xyz="${lower_leg_length / 2} 0.0 0.0"  rpy="0.0 0.0 0.0"/>
-		<geometry>
-	 		<box size="${lower_leg_length} ${lower_leg_width} ${lower_leg_height}"/>
-		</geometry>
-	</collision>
-</link>
-<link name="ball_${leg_num}">
-	<inertial>
-		<origin xyz="0.0 0.0 0.0"/>
-		<mass value="${ball_mass}"/>
-		<inertia ixx="${Ball_xx}" ixy="${Ball_xy}" ixz="${Ball_xz}" iyy="${Ball_yy}" iyz="${Ball_yz}" izz="${Ball_zz}"/>
-	</inertial>
-	<visual>
-		<origin xyz="0.0 0.0 0.0" rpy="0.0 0.0 0.0"/>
-		<geometry>
-			<sphere radius="${ball_radius}"/>
-		</geometry>
-	</visual>
-	<collision>
-		<origin xyz="0.0 0.0 0.0" rpy="0.0 0.0 0.0"/>
-		<geometry>
-			<sphere radius="${ball_radius}"/>
-		</geometry>
-	</collision>
-</link>
-<xacro:if value="${ADD_WHEELS}">
-	<joint name="wheel_joint_${leg_num}" type="revolute">
-            <parent link="ball_${leg_num}" />
-            <child link="wheel_${leg_num}" />
-            <origin xyz="${Wheel23_Ox} ${Wheel23_Oy} ${-mirror*Wheel23_Oz}" rpy="${Wheel23_roll} ${Wheel23_pitch} ${Wheel23_yaw}" />
-            <axis xyz="0 0 ${mirror}"/>
-            <limit lower="-1e6" upper="1e6" effort="${motor_effort}" velocity="30." />
-            <!--limit effort="${motor_effort}" velocity="${motor_velocity}" /-->
-        </joint>
-        <link name="wheel_${leg_num}">
-            <inertial>
-                <origin xyz="${Wheel23_x} ${Wheel23_y} ${mirror*Wheel23_z}" />
-                <mass value="${Wheel23_mass}" />
-                <inertia ixx="${Wheel23_xx}" ixy="${Wheel23_xy}" ixz="${mirror*Wheel23_xz}" iyy="${Wheel23_yy}" iyz="${mirror*Wheel23_yz}" izz="${Wheel23_zz}" />
-            </inertial>
-            <visual>
-                <origin xyz="0.0 0.0 0.0" rpy="0.0 0.0 0.0" />
-                <geometry>
-                    <mesh filename="package://kyon_urdf/meshes/mesh_wheel23.stl"
-                        scale="0.001 0.001 ${mirror*0.001}" />
-                </geometry>
-                <material name="black" />
-            </visual>
-            <collision>
-                <origin xyz="0 0 0" rpy="0 0 0" />
-                <geometry>
-                    <!--mesh filename="package://kyon_urdf/meshes/collision/mesh_wheel23.stl"
-                        scale="0.001 0.001 ${mirror*0.001}" /-->
-                    <sphere radius="0.125"/>
-                </geometry>
-                <material name="black" />
-            </collision>
-        </link>
-</xacro:if>
 <!-- joints -->
 <joint name="hip_roll_${leg_num}" type="revolute">
 	<parent link="pelvis"/>
-	<child link="hip_roll_motor_${leg_num}"/>
-	<origin xyz="${origin_x * HipRoll_Ox} ${origin_y * HipRoll_Oy} ${HipRoll_Oz}" rpy="${HipRoll_roll} ${HipRoll_pitch} ${HipRoll_yaw}"/>
+	<child link="hip_roll_${leg_num}"/>
+	<origin xyz="${origin_x * HipRoll_Ox} ${origin_y * HipRoll_Oy} ${HipRoll_Oz}" rpy="${HipRoll_roll} ${origin_x*HipRoll_pitch} ${HipRoll_yaw}"/>
 	<axis xyz="0 0 1"/>
-    <limit lower="${hip_roll_lower[leg_num-1]}" upper="${hip_roll_upper[leg_num-1]}" effort="${motor_effort}" velocity="${motor_velocity}"/> <!-- 200 Nm, 1 rad/s-->
-</joint>
-<joint name="hip_pitch_stator_${leg_num}" type="fixed">
-	<parent link="hip_roll_motor_${leg_num}"/>
-	<child link="hip_pitch_motor_${leg_num}"/>
-	<origin xyz="${HipPitch_Ox} ${mirror * (HipPitch_Oy)} ${HipPitch_Oz}" rpy="${HipPitch_roll} ${HipPitch_pitch} ${HipPitch_yaw}"/>
-</joint>
-<joint name="knee_pitch_stator_${leg_num}" type="fixed">
-	<parent link="hip_pitch_motor_${leg_num}"/>
-	<child link="knee_pitch_motor_${leg_num}"/>
-	<origin xyz="${KneePitch_Ox} ${KneePitch_Oy} ${KneePitch_Oz}" rpy="${KneePitch_roll} ${KneePitch_pitch} ${KneePitch_yaw}"/>
+    <limit lower="${hip_roll_lower[leg_num-1]}" upper="${hip_roll_upper[leg_num-1]}" effort="${motor_effort}" velocity="${motor_velocity}"/>
 </joint>
 <joint name="hip_pitch_${leg_num}" type="revolute">
-	<parent link="hip_pitch_motor_${leg_num}"/>
-	<child link="upper_leg_${leg_num}"/>
-	<origin xyz="${UpperLeg_Ox} ${mirror*(UpperLeg_Oy)} ${UpperLeg_Oz}" rpy="${UpperLeg_roll} ${UpperLeg_pitch} ${UpperLeg_yaw}"/>
+	<parent link="hip_roll_${leg_num}"/>
+	<child link="hip_pitch_${leg_num}"/>
+	<origin xyz="${origin_x * HipPitch_Ox} ${origin_y * HipPitch_Oy} ${HipPitch_Oz}" rpy="${origin_y*HipPitch_roll} ${origin_x*origin_y*HipPitch_pitch} ${HipPitch_yaw}"/>
 	<axis xyz="0 0 1"/>
-   <limit lower="${hip_pitch_lower[leg_num-1]}" upper="${hip_pitch_upper[leg_num-1]}" effort="${motor_effort}" velocity="${motor_velocity}"/> <!-- 200 Nm, 1 rad/s-->
+	<limit lower="${hip_pitch_lower[leg_num-1]}" upper="${hip_pitch_upper[leg_num-1]}" effort="${motor_effort}" velocity="${motor_velocity}"/>
 </joint>
-<joint name="knee_pitch_${leg_num}" type="revolute">
-	<parent link="upper_leg_${leg_num}"/>
-	<child link="lower_leg_${leg_num}"/>
-	<origin xyz="${LowerLeg_Ox} ${LowerLeg_Oy} ${LowerLeg_Oz}" rpy="${LowerLeg_roll} ${LowerLeg_pitch} ${LowerLeg_yaw}"/>
-	<axis xyz="0 0 1"/>
-   <limit lower="${knee_pitch_lower[leg_num-1]}" upper="${knee_pitch_upper[leg_num-1]}" effort="${motor_effort}" velocity="${motor_velocity}"/> <!-- 200 Nm, 1 rad/s-->
-</joint>
-<joint name="ball_joint_${leg_num}" type="fixed">
-	<parent link="lower_leg_${leg_num}"/>
-	<child link="ball_${leg_num}"/>
-	<origin xyz="${Ankle_Ox} ${Ankle_Oy} ${Ankle_Oz}" rpy="${Ankle_roll} ${Ankle_pitch} ${Ankle_yaw}"/>
-</joint>
+<xacro:if value="${ADD_FEET}">
+	<xacro:foot_leg leg_num="${leg_num}" parent="hip_pitch_${leg_num}" origin_x="${origin_x}" origin_y="${origin_y}" mirror="${mirror}"/>
+</xacro:if>
+<xacro:if value="${ADD_STEERING_WHEELS}">
+	<xacro:steering_wheel leg_num="${leg_num}" parent="hip_pitch_${leg_num}" origin_x="${origin_x}" origin_y="${origin_y}" mirror="${mirror}"/>
+</xacro:if>
 </xacro:macro>
 <!-- /macro legs -->

File: kyon_urdf/urdf/parts/legs.urdf.xacro (robot description, xacro)
@@ -2,11 +2,11 @@
 <robot xmlns:xacro="http://ros.org/wiki/xacro">
 <xacro:include filename="$(find kyon_urdf)/urdf/parts/kyon_leg.urdf.xacro" />
-<xacro:kyon_leg leg_num="1" origin_x="1" origin_y="-1" mirror="-1">
+<xacro:kyon_leg leg_num="1" origin_x="1" origin_y="1" mirror="-1">
 </xacro:kyon_leg>
-<xacro:kyon_leg leg_num="2" origin_x="1" origin_y="1" mirror="1">
+<xacro:kyon_leg leg_num="2" origin_x="1" origin_y="-1" mirror="1">
 </xacro:kyon_leg>
-<xacro:kyon_leg leg_num="3" origin_x="-1" origin_y="-1" mirror="-1">
+<xacro:kyon_leg leg_num="3" origin_x="-1" origin_y="1" mirror="-1">
 </xacro:kyon_leg>
-<xacro:kyon_leg leg_num="4" origin_x="-1" origin_y="1" mirror="1">
+<xacro:kyon_leg leg_num="4" origin_x="-1" origin_y="-1" mirror="1">
 </xacro:kyon_leg>
 </robot>
