Commit message: updated wheel leg inertial properties

File: kyon_urdf/urdf/config/kyon.urdf.xacro (robot description, xacro)
@@ -10,5 +10,5 @@
 <xacro:arg name="wheels" default="false"/>
 <xacro:arg name="floating_joint" default="true"/>
-<xacro:arg name="sensors" default="true"/>
+<xacro:arg name="sensors" default="false"/>
 <xacro:arg name="payload" default="false"/>
 <xacro:arg name="ft_sensors" default="false"/>

File: kyon_urdf/urdf/kyon.urdf (robot description, URDF)
Before this commit: robot kyon, 120 links, 119 joints
Links:
- removed link D435_front1_accel_frame
- removed link D435_front1_accel_optical_frame
- removed link D435_front1_bottom_screw_frame
- removed link D435_front1_color_frame
- removed link D435_front1_color_optical_frame
- removed link D435_front1_depth_frame
- removed link D435_front1_depth_optical_frame
- removed link D435_front1_gyro_frame
- removed link D435_front1_gyro_optical_frame
- removed link D435_front1_left_ir_frame
- removed link D435_front1_left_ir_optical_frame
- removed link D435_front1_link
- removed link D435_front1_right_ir_frame
- removed link D435_front1_right_ir_optical_frame
- removed link D435_front2_accel_frame
- removed link D435_front2_accel_optical_frame
- removed link D435_front2_bottom_screw_frame
- removed link D435_front2_color_frame
- removed link D435_front2_color_optical_frame
- removed link D435_front2_depth_frame
- removed link D435_front2_depth_optical_frame
- removed link D435_front2_gyro_frame
- removed link D435_front2_gyro_optical_frame
- removed link D435_front2_left_ir_frame
- removed link D435_front2_left_ir_optical_frame
- removed link D435_front2_link
- removed link D435_front2_right_ir_frame
- removed link D435_front2_right_ir_optical_frame
- removed link D435_front3_accel_frame
- removed link D435_front3_accel_optical_frame
- removed link D435_front3_bottom_screw_frame
- removed link D435_front3_color_frame
- removed link D435_front3_color_optical_frame
- removed link D435_front3_depth_frame
- removed link D435_front3_depth_optical_frame
- removed link D435_front3_gyro_frame
- removed link D435_front3_gyro_optical_frame
- removed link D435_front3_left_ir_frame
- removed link D435_front3_left_ir_optical_frame
- removed link D435_front3_link
- removed link D435_front3_right_ir_frame
- removed link D435_front3_right_ir_optical_frame
- removed link D435_left_accel_frame
- removed link D435_left_accel_optical_frame
- removed link D435_left_bottom_screw_frame
- removed link D435_left_color_frame
- removed link D435_left_color_optical_frame
- removed link D435_left_depth_frame
- removed link D435_left_depth_optical_frame
- removed link D435_left_gyro_frame
- removed link D435_left_gyro_optical_frame
- removed link D435_left_left_ir_frame
- removed link D435_left_left_ir_optical_frame
- removed link D435_left_link
- removed link D435_left_right_ir_frame
- removed link D435_left_right_ir_optical_frame
- removed link D435_rear_accel_frame
- removed link D435_rear_accel_optical_frame
- removed link D435_rear_bottom_screw_frame
- removed link D435_rear_color_frame
- removed link D435_rear_color_optical_frame
- removed link D435_rear_depth_frame
- removed link D435_rear_depth_optical_frame
- removed link D435_rear_gyro_frame
- removed link D435_rear_gyro_optical_frame
- removed link D435_rear_left_ir_frame
- removed link D435_rear_left_ir_optical_frame
- removed link D435_rear_link
- removed link D435_rear_right_ir_frame
- removed link D435_rear_right_ir_optical_frame
- removed link D435_right_accel_frame
- removed link D435_right_accel_optical_frame
- removed link D435_right_bottom_screw_frame
- removed link D435_right_color_frame
- removed link D435_right_color_optical_frame
- removed link D435_right_depth_frame
- removed link D435_right_depth_optical_frame
- removed link D435_right_gyro_frame
- removed link D435_right_gyro_optical_frame
- removed link D435_right_left_ir_frame
- removed link D435_right_left_ir_optical_frame
- removed link D435_right_link
- removed link D435_right_right_ir_frame
- removed link D435_right_right_ir_optical_frame
- removed link velodyne
- removed link velodyne_base_link
- removed link wheel_1_link
- removed link wheel_2_link
- removed link wheel_3_link
- removed link wheel_4_link
- added link contact_1
- added link contact_2
- added link contact_3
- added link contact_4
- link knee_pitch_1_link: mass 1.8 -> 0.70900216; geometry collision mesh filename=package://kyon_urdf/meshes/collision/mesh_foot-leg.stl scale=-0.001 0.001 0.001; visual mesh filename=package://kyon_urdf/meshes/mesh_foot-leg.stl scale=-0.001 0.001 0.001
- link knee_pitch_2_link: mass 1.8 -> 0.70900216; geometry collision mesh filename=package://kyon_urdf/meshes/collision/mesh_foot-leg.stl scale=0.001 0.001 0.001; visual mesh filename=package://kyon_urdf/meshes/mesh_foot-leg.stl scale=0.001 0.001 0.001
- link knee_pitch_3_link: mass 1.8 -> 0.70900216; geometry collision mesh filename=package://kyon_urdf/meshes/collision/mesh_foot-leg.stl scale=-0.001 0.001 0.001; visual mesh filename=package://kyon_urdf/meshes/mesh_foot-leg.stl scale=-0.001 0.001 0.001
- link knee_pitch_4_link: mass 1.8 -> 0.70900216; geometry collision mesh filename=package://kyon_urdf/meshes/collision/mesh_foot-leg.stl scale=0.001 0.001 0.001; visual mesh filename=package://kyon_urdf/meshes/mesh_foot-leg.stl scale=0.001 0.001 0.001
Joints:
- removed joint D435_front1_accel_joint
- removed joint D435_front1_accel_optical_joint
- removed joint D435_front1_color_joint
- removed joint D435_front1_color_optical_joint
- removed joint D435_front1_depth_joint
- removed joint D435_front1_depth_optical_joint
- removed joint D435_front1_gyro_joint
- removed joint D435_front1_gyro_optical_joint
- removed joint D435_front1_joint
- removed joint D435_front1_left_ir_joint
- removed joint D435_front1_left_ir_optical_joint
- removed joint D435_front1_link_joint
- removed joint D435_front1_right_ir_joint
- removed joint D435_front1_right_ir_optical_joint
- removed joint D435_front2_accel_joint
- removed joint D435_front2_accel_optical_joint
- removed joint D435_front2_color_joint
- removed joint D435_front2_color_optical_joint
- removed joint D435_front2_depth_joint
- removed joint D435_front2_depth_optical_joint
- removed joint D435_front2_gyro_joint
- removed joint D435_front2_gyro_optical_joint
- removed joint D435_front2_joint
- removed joint D435_front2_left_ir_joint
- removed joint D435_front2_left_ir_optical_joint
- removed joint D435_front2_link_joint
- removed joint D435_front2_right_ir_joint
- removed joint D435_front2_right_ir_optical_joint
- removed joint D435_front3_accel_joint
- removed joint D435_front3_accel_optical_joint
- removed joint D435_front3_color_joint
- removed joint D435_front3_color_optical_joint
- removed joint D435_front3_depth_joint
- removed joint D435_front3_depth_optical_joint
- removed joint D435_front3_gyro_joint
- removed joint D435_front3_gyro_optical_joint
- removed joint D435_front3_joint
- removed joint D435_front3_left_ir_joint
- removed joint D435_front3_left_ir_optical_joint
- removed joint D435_front3_link_joint
- removed joint D435_front3_right_ir_joint
- removed joint D435_front3_right_ir_optical_joint
- removed joint D435_left_accel_joint
- removed joint D435_left_accel_optical_joint
- removed joint D435_left_color_joint
- removed joint D435_left_color_optical_joint
- removed joint D435_left_depth_joint
- removed joint D435_left_depth_optical_joint
- removed joint D435_left_gyro_joint
- removed joint D435_left_gyro_optical_joint
- removed joint D435_left_joint
- removed joint D435_left_left_ir_joint
- removed joint D435_left_left_ir_optical_joint
- removed joint D435_left_link_joint
- removed joint D435_left_right_ir_joint
- removed joint D435_left_right_ir_optical_joint
- removed joint D435_rear_accel_joint
- removed joint D435_rear_accel_optical_joint
- removed joint D435_rear_color_joint
- removed joint D435_rear_color_optical_joint
- removed joint D435_rear_depth_joint
- removed joint D435_rear_depth_optical_joint
- removed joint D435_rear_gyro_joint
- removed joint D435_rear_gyro_optical_joint
- removed joint D435_rear_joint
- removed joint D435_rear_left_ir_joint
- removed joint D435_rear_left_ir_optical_joint
- removed joint D435_rear_link_joint
- removed joint D435_rear_right_ir_joint
- removed joint D435_rear_right_ir_optical_joint
- removed joint D435_right_accel_joint
- removed joint D435_right_accel_optical_joint
- removed joint D435_right_color_joint
- removed joint D435_right_color_optical_joint
- removed joint D435_right_depth_joint
- removed joint D435_right_depth_optical_joint
- removed joint D435_right_gyro_joint
- removed joint D435_right_gyro_optical_joint
- removed joint D435_right_joint
- removed joint D435_right_left_ir_joint
- removed joint D435_right_left_ir_optical_joint
- removed joint D435_right_link_joint
- removed joint D435_right_right_ir_joint
- removed joint D435_right_right_ir_optical_joint
- removed joint velodyne_base_mount_joint
- removed joint velodyne_base_scan_joint
- removed joint wheel_joint_1
- removed joint wheel_joint_2
- removed joint wheel_joint_3
- removed joint wheel_joint_4
- added joint contact_1_joint: type fixed, parent knee_pitch_1_link, child contact_1, origin xyz=0.03 -0.35 0.03 rpy=-1.57 0 0.785
- added joint contact_2_joint: type fixed, parent knee_pitch_2_link, child contact_2, origin xyz=-0.03 -0.35 0.03 rpy=1.57 0 2.356
- added joint contact_3_joint: type fixed, parent knee_pitch_3_link, child contact_3, origin xyz=0.03 -0.35 0.03 rpy=-1.57 0 0.785
- added joint contact_4_joint: type fixed, parent knee_pitch_4_link, child contact_4, origin xyz=-0.03 -0.35 0.03 rpy=1.57 0 2.356

File: kyon_urdf/urdf/parts/inertial_properties.urdf.xacro (robot description, xacro)
@@ -56,14 +56,14 @@
     <xacro:property name="KneePitchSteeringWheel_yz" value="${5.5514749e+02 * mm2Tom2}"/>
     <xacro:property name="KneePitchSteeringWheel_zz" value="${2.0709191e+03 * mm2Tom2}"/>
-    <xacro:property name="KneePitchWheel_mass" value="0.70900216"/>
-    <xacro:property name="KneePitchWheel_xx" value="${5.1193011e-03 * mmTom}"/>
-    <xacro:property name="KneePitchWheel_y" value="${-1.0291595e+02 * mmTom}"/>
-    <xacro:property name="KneePitchWheel_z" value="${-1.2895495e+00 * mmTom}"/>
-    <xacro:property name="KneePitchWheel_xx" value="${1.2517512e+04 * mm2Tom2}"/>
-    <xacro:property name="KneePitchWheel_xy" value="${-5.4385779e-01 * mm2Tom2}"/>
-    <xacro:property name="KneePitchWheel_xz" value="${1.4538899e-01 * mm2Tom2}"/>
-    <xacro:property name="KneePitchWheel_yy" value="${8.0474409e+02 * mm2Tom2}"/>
-    <xacro:property name="KneePitchWheel_yz" value="${1.7446290e+03 * mm2Tom2}"/>
-    <xacro:property name="KneePitchWheel_zz" value="${1.2307020e+04 * mm2Tom2}"/>
+    <xacro:property name="KneePitchWheel_mass" value="1.5016388"/>
+    <xacro:property name="KneePitchWheel_x" value="${-1.7834738e-01 * mmTom}"/>
+    <xacro:property name="KneePitchWheel_y" value="${-2.5371445e+02 * mmTom}"/>
+    <xacro:property name="KneePitchWheel_z" value="${4.1781751e+01 * mmTom}"/>
+    <xacro:property name="KneePitchWheel_xx" value="${1.1851050e+04 * mm2Tom2}"/>
+    <xacro:property name="KneePitchWheel_xy" value="${5.3594921e+02 * mm2Tom2}"/>
+    <xacro:property name="KneePitchWheel_xz" value="${-1.9109120e+03 * mm2Tom2}"/>
+    <xacro:property name="KneePitchWheel_yy" value="${-2.2822244e+03 * mm2Tom2}"/>
+    <xacro:property name="KneePitchWheel_yz" value="${1.4122439e+03 * mm2Tom2}"/>
+    <xacro:property name="KneePitchWheel_zz" value="${1.2166274e+04 * mm2Tom2}"/>
     <!-- Ankle Yaw -->
     <xacro:property name="AnkleYaw_mass" value="1.4941965"/>

File: kyon_urdf/urdf/parts/wheel_leg.urdf.xacro (robot description, xacro)
@@ -5,5 +5,5 @@
 <link name="knee_pitch_${leg_num}_link">
     <inertial>
-        <origin xyz="0.0 0.0 0.0"/>
+        <origin xyz="${KneePitchWheel_x} ${KneePitchWheel_y} ${KneePitchWheel_z}"/>
         <mass value="${KneePitchWheel_mass}"/>
         <inertia ixx="${KneePitchWheel_xx}" ixy="${mirror*KneePitchWheel_xy}" ixz="${mirror*KneePitchWheel_xz}" iyy="${KneePitchWheel_yy}" iyz="${KneePitchWheel_yz}" izz="${KneePitchWheel_zz}"/>

Commit message: updated cameras

File: kyon_urdf/urdf/config/kyon.urdf.xacro (robot description, xacro)
@@ -6,5 +6,5 @@
 <xacro:arg name="legs" default="true"/>
 <xacro:arg name="upper_body" default="true"/>
-<xacro:arg name="dagana" default="false"/>
+<xacro:arg name="dagana" default="true"/>
 <xacro:arg name="feet" default="true"/>
 <xacro:arg name="wheels" default="false"/>
@@ -12,5 +12,4 @@
 <xacro:arg name="sensors" default="true"/>
 <xacro:arg name="payload" default="false"/>
-<xacro:arg name="ft_sensors" default="false"/>
 <xacro:arg name="steering_wheels" default="false"/>
 <!-- ************SELECT PARTS*************-->
@@ -23,5 +22,4 @@
 <xacro:property name="ADD_WHEELS" value="$(arg wheels)"/>
 <xacro:property name="ADD_STEERING_WHEELS" value="$(arg steering_wheels)"/>
-<xacro:property name="ADD_FT_SENSORS" value="$(arg ft_sensors)"/>
 <xacro:property name="ADD_FLOATING_BASE" value="$(arg floating_joint)" />
 <xacro:property name="ADD_VIRTUAL_FRAME" value="false" />

File: kyon_urdf/urdf/gazebo/kyon.gazebo.xacro (robot description, xacro)
@@ -159,5 +159,5 @@
 	    </gazebo>
 	</xacro:if>
-	<xacro:if value="${ADD_FT_SENSORS}">
+	<!-- <xacro:if value="${ADD_FT_SENSORS}">
 		<xacro:include filename="$(find kyon_urdf)/urdf/gazebo/ft_sensors.gazebo.xacro" />
 		<xacro:kyon_ft_sensor frame_id="knee_pitch_1"/>
@@ -165,4 +165,4 @@
 		<xacro:kyon_ft_sensor frame_id="knee_pitch_3"/>
 		<xacro:kyon_ft_sensor frame_id="knee_pitch_4"/>
-	</xacro:if>
+	</xacro:if> -->
 </robot>

File: kyon_urdf/urdf/kyon_base.urdf.xacro (robot description, xacro)
@@ -59,5 +59,5 @@
         color_height="720"
         color_fps="30">
-        <origin xyz="-0.175 0.22 0" rpy="0 0.35 1.57"/>
+        <origin xyz="0 0.150100 0.109486" rpy="0 0.3490656 1.5707963"/>
     </xacro:sensor_d435i>
     <!-- RIGHT D435 CAMERA -->
@@ -80,8 +80,8 @@
         color_height="720"
         color_fps="30">
-        <origin xyz="-0.175 -0.22 0" rpy="0 0.35 -1.57"/>
+        <origin xyz="0 -0.150100 0.109486" rpy="0 0.3490656 -1.5707963"/>
     </xacro:sensor_d435i>
     <!-- REAR D435 CAMERA -->
-    <xacro:sensor_d435i parent="pelvis"
+    <!-- <xacro:sensor_d435i parent="pelvis"
         name="D435_rear"
         topics_ns="D435_rear"
@@ -102,5 +102,5 @@
         color_fps="30">
         <origin xyz="-0.39 0 0" rpy="0 0.35 3.14"/>
-    </xacro:sensor_d435i>
+    </xacro:sensor_d435i> -->
     <!-- FRONT1 D435 CAMERA -->
     <xacro:sensor_d435i parent="pelvis"
@@ -122,5 +122,5 @@
         color_height="720"
         color_fps="30">
-        <origin xyz="0.40 -0.08 0" rpy="-1.57 0 0.34"/>
+        <origin xyz="0.526174 0 0.0674608" rpy="0 -0.1745327 0"/>
     </xacro:sensor_d435i>
     <!-- FRONT2 D435 CAMERA -->
@@ -143,8 +143,8 @@
         color_height="720"
         color_fps="30">
-        <origin xyz="0.40 0.08 0" rpy="-1.57 0 -0.34"/>
+        <origin xyz="0.509601 0 0.00343992" rpy="0 0.9250251 0"/>
     </xacro:sensor_d435i>
     <!-- FRONT3 (down) D435 CAMERA -->
-    <xacro:sensor_d435i parent="pelvis"
+    <!-- <xacro:sensor_d435i parent="pelvis"
         name="D435_front3"
         topics_ns="D435_front3"
@@ -165,10 +165,10 @@
         color_fps="30">
         <origin xyz="0.37 0 -0.11" rpy="0 0.75 0"/>
-    </xacro:sensor_d435i>
+    </xacro:sensor_d435i> -->
     <!-- Velodyne -->
-    <xacro:include filename="$(find velodyne_description)/urdf/VLP-16.urdf.xacro"/>
+    <!-- <xacro:include filename="$(find velodyne_description)/urdf/VLP-16.urdf.xacro"/>
     <xacro:VLP-16 parent="pelvis" name="velodyne" topic="/velodyne_points" hz="10" samples="440">
         <origin xyz="0.36 0 0.11" rpy="0 0 0" />
-    </xacro:VLP-16>
+    </xacro:VLP-16> -->
 </xacro:if>
 <xacro:if value="${ADD_UPPER_BODY}">

Commit message: updated cameras

File: kyon_urdf/urdf/config/kyon.urdf.xacro (robot description, xacro)
@@ -6,5 +6,5 @@
 <xacro:arg name="legs" default="true"/>
 <xacro:arg name="upper_body" default="true"/>
-<xacro:arg name="dagana" default="false"/>
+<xacro:arg name="dagana" default="true"/>
 <xacro:arg name="feet" default="true"/>
 <xacro:arg name="wheels" default="false"/>
@@ -12,5 +12,4 @@
 <xacro:arg name="sensors" default="false"/>
 <xacro:arg name="payload" default="false"/>
-<xacro:arg name="ft_sensors" default="false"/>
 <xacro:arg name="steering_wheels" default="false"/>
 <!-- ************SELECT PARTS*************-->
@@ -23,5 +22,4 @@
 <xacro:property name="ADD_WHEELS" value="$(arg wheels)"/>
 <xacro:property name="ADD_STEERING_WHEELS" value="$(arg steering_wheels)"/>
-<xacro:property name="ADD_FT_SENSORS" value="$(arg ft_sensors)"/>
 <xacro:property name="ADD_FLOATING_BASE" value="$(arg floating_joint)" />
 <xacro:property name="ADD_VIRTUAL_FRAME" value="false" />
