Commit message: migrated kyon_urdf to ros2
added velodyne

modified plugins in kyon_urdf/urdf/gazebo to be compatible with
new Gazebo

File: kyon_urdf/urdf/config/kyon.urdf.xacro (robot description, xacro)
@@ -14,4 +14,11 @@
 <xacro:arg name="steering_wheels" default="false"/>
 <xacro:arg name="ft_sensors" default="true"/>
+<xacro:arg name="velodyne" default="false"/>
+<xacro:if value="$(arg feet)">
+    <xacro:if value="$(arg wheels)">
+        <xacro:property name="error_flag" value="${xacro.error('Arguments feet and wheels are both true. \n If you meant to use wheels, please set feet:=false.\n')}"/>
+        ${error_flag}
+    </xacro:if>
+</xacro:if>
 <!-- ************SELECT PARTS*************-->
 <!-- *************************************-->
@@ -24,4 +31,5 @@
 <xacro:property name="ADD_STEERING_WHEELS" value="$(arg steering_wheels)"/>
 <xacro:property name="ADD_FT_SENSORS" value="$(arg ft_sensors)"/>
+<xacro:property name="ADD_VELODYNE" value="$(arg velodyne)"/>
 <xacro:property name="ADD_FLOATING_BASE" value="$(arg floating_joint)" />
 <xacro:property name="ADD_VIRTUAL_FRAME" value="false" />

File: kyon_urdf/urdf/gazebo/ft_sensors.gazebo.xacro (robot description, xacro)
@@ -6,14 +6,17 @@
         Note that this sign convention is opposite of the reaction forces
         of the Joint on the Links" -->
-        <gazebo>
-            <plugin name="ft_sensor" filename="libgazebo_ros_ft_sensor.so">
+        <!-- <gazebo> -->
+            <!-- <plugin filename="gz-sim-forcetorque-system" name="gz::sim::systems::ForceTorque"> -->
+                <!-- <updateRate>0.0</updateRate> 0.0 is as fast as possible -->
+                <!-- <topicName>ft_sensors/${frame_id}</topicName> -->
+                <!-- <jointName>${frame_id}</jointName> -->
+            <!-- </plugin> -->
+        <!-- </gazebo> -->
+        <gazebo reference="${frame_id}">
+            <provideFeedback>true</provideFeedback>
+            <sensor type="force_torque" name="${frame_id}_fts">
                 <updateRate>0.0</updateRate> <!-- 0.0 is as fast as possible -->
                 <topicName>ft_sensors/${frame_id}</topicName>
                 <jointName>${frame_id}</jointName>
-            </plugin>
-        </gazebo>
-        <gazebo reference="${frame_id}">
-            <provideFeedback>true</provideFeedback>
-            <sensor type="force_torque" name="${frame_id}_fts">
                 <force_torque>
                     <frame>sensor</frame>

File: kyon_urdf/urdf/gazebo/kyon.gazebo.xacro (robot description, xacro)
@@ -193,3 +193,40 @@
 		<xacro:kyon_ft_sensor frame_id="knee_pitch_4"/>
 	</xacro:if>
+    <xacro:if value="${ADD_VELODYNE}">
+        <gazebo reference="velodyne">
+            <sensor name="VLP16_lidar_front_gpu_lidar" type="gpu_lidar">
+                <gz_frame_id>velodyne</gz_frame_id>
+                <topic>/VLP16_lidar_front</topic>
+                <update_rate>10</update_rate>
+                <ray>
+                  <scan>
+                    <horizontal>
+                      <samples>440</samples>
+                      <resolution>1</resolution>
+                      <min_angle>-1.04</min_angle>
+                      <max_angle>3.66</max_angle>
+                    </horizontal>
+                    <!-- <vertical>
+                      <samples>16</samples>
+                      <resolution>1</resolution>
+                      <min_angle>-0.2617993877991494</min_angle>
+                      <max_angle>0.2617993877991494</max_angle>
+                    </vertical> -->
+                  </scan>
+                  <range>
+                    <min>0.9</min>
+                    <max>130.0</max>
+                    <resolution>0.01</resolution>
+                  </range>
+                  <noise>
+                    <type>gaussian</type>
+                    <mean>0.0</mean>
+                    <stddev>0.008</stddev>
+                  </noise>
+                </ray>
+                <always_on>1</always_on>
+                <visualize>true</visualize>
+              </sensor>
+        </gazebo>
+    </xacro:if>
 </robot>

File: kyon_urdf/urdf/gazebo/xbot.gazebo.xacro (robot description, xacro)
@@ -2,5 +2,5 @@
 <robot xmlns:xacro="http://ros.org/wiki/xacro">
 <gazebo>
-    <plugin name="xbot2_link_state_sensor" filename="libxbot2_gz_link_state_sensor.so">
+    <!-- <plugin name="xbot2_link_state_sensor" filename="libxbot2_gz_link_state_sensor.so">
         <links>
             <link name="pelvis"/>
@@ -8,39 +8,37 @@
     </plugin>
     <plugin name="xbot2_ft_driver" filename="libxbot2_gz_ft_server.so"/>
-    <plugin name="xbot2_imu_driver" filename="libxbot2_gz_imu_server.so"/>
-    <plugin name="xbot2_joint_driver" filename="libxbot2_gz_joint_server.so">
-        <pid>
-            <gain name="lowpwr_mot" p="100"  d="1"/>
-            <gain name="small_mot"  p="500"  d="5"/>
-            <gain name="medium_mot" p="1000" d="10"/>
-            <gain name="big_mot"    p="1500" d="20"/>
-            <gain name="wheel"      p="0"    d="10"/>
-            <pid name="shoulder_yaw_1" profile="medium_mot"/>
-            <pid name="shoulder_pitch_1" profile="medium_mot"/>
-            <pid name="elbow_pitch_1" profile="small_mot"/>
-            <pid name="wrist_pitch_1" profile="small_mot"/>
-            <pid name="wrist_yaw_1" profile="small_mot"/>
-            <pid name="shoulder_yaw_2" profile="medium_mot"/>
-            <pid name="shoulder_pitch_2" profile="medium_mot"/>
-            <pid name="elbow_pitch_2" profile="small_mot"/>
-            <pid name="wrist_pitch_2" profile="small_mot"/>
-            <pid name="wrist_yaw_2" profile="small_mot"/>
-            <pid name="hip_roll_1"     profile="big_mot"/>
-            <pid name="hip_pitch_1"  profile="big_mot"/>
-            <pid name="knee_pitch_1"   profile="big_mot"/>
-            <pid name="wheel_joint_1" profile="wheel"/>
-            <pid name="hip_roll_2"     profile="big_mot"/>
-            <pid name="hip_pitch_2"  profile="big_mot"/>
-            <pid name="knee_pitch_2"   profile="big_mot"/>
-            <pid name="wheel_joint_2" profile="wheel"/>
-            <pid name="hip_roll_3"     profile="big_mot"/>
-            <pid name="hip_pitch_3"  profile="big_mot"/>
-            <pid name="knee_pitch_3"   profile="big_mot"/>
-            <pid name="wheel_joint_3" profile="wheel"/>
-            <pid name="hip_roll_4"     profile="big_mot"/>
-            <pid name="hip_pitch_4"  profile="big_mot"/>
-            <pid name="knee_pitch_4"   profile="big_mot"/>
-            <pid name="wheel_joint_4" profile="wheel"/>
-        </pid>
+    <plugin name="xbot2_imu_driver" filename="libxbot2_gz_imu_server.so"/> -->
+    <plugin name="gz::sim::systems::GzJointServer" filename="libxbot2_gz_joint_server.so">
+            <profile name="lowpwr_mot" p="100"  d="1"/>
+            <profile name="small_mot"  p="500"  d="5"/>
+            <profile name="medium_mot" p="1000" d="10"/>
+            <profile name="big_mot"    p="1500" d="20"/>
+            <profile name="wheel"      p="0"    d="10"/>
+            <pid name="shoulder_yaw_1"      profile="medium_mot"/>
+            <pid name="shoulder_pitch_1"    profile="medium_mot"/>
+            <pid name="elbow_pitch_1"       profile="small_mot"/>
+            <pid name="wrist_pitch_1"       profile="small_mot"/>
+            <pid name="wrist_yaw_1"         profile="small_mot"/>
+            <pid name="shoulder_yaw_2"      profile="medium_mot"/>
+            <pid name="shoulder_pitch_2"    profile="medium_mot"/>
+            <pid name="elbow_pitch_2"       profile="small_mot"/>
+            <pid name="wrist_pitch_2"       profile="small_mot"/>
+            <pid name="wrist_yaw_2"         profile="small_mot"/>
+            <pid name="hip_roll_1"          profile="big_mot"/>
+            <pid name="hip_pitch_1"         profile="big_mot"/>
+            <pid name="knee_pitch_1"        profile="big_mot"/>
+            <pid name="wheel_joint_1"       profile="wheel"/>
+            <pid name="hip_roll_2"          profile="big_mot"/>
+            <pid name="hip_pitch_2"         profile="big_mot"/>
+            <pid name="knee_pitch_2"        profile="big_mot"/>
+            <pid name="wheel_joint_2"       profile="wheel"/>
+            <pid name="hip_roll_3"          profile="big_mot"/>
+            <pid name="hip_pitch_3"         profile="big_mot"/>
+            <pid name="knee_pitch_3"        profile="big_mot"/>
+            <pid name="wheel_joint_3"       profile="wheel"/>
+            <pid name="hip_roll_4"          profile="big_mot"/>
+            <pid name="hip_pitch_4"         profile="big_mot"/>
+            <pid name="knee_pitch_4"        profile="big_mot"/>
+            <pid name="wheel_joint_4"       profile="wheel"/>
     </plugin>
 </gazebo>

File: kyon_urdf/urdf/kyon_base.urdf.xacro (robot description, xacro)
@@ -172,4 +172,11 @@
     </xacro:VLP-16> -->
 </xacro:if>
+<!-- Velodyne -->
+<xacro:if value="${ADD_VELODYNE}">
+    <xacro:include filename="$(find velodyne_description)/urdf/VLP-16.urdf.xacro"/>
+    <xacro:VLP-16 parent="pelvis" name="velodyne">
+        <origin xyz="0.47 0 0.11" rpy="0 0 0" />
+    </xacro:VLP-16>
+</xacro:if>
 <xacro:if value="${ADD_UPPER_BODY}">
     <xacro:include filename="$(find kyon_urdf)/urdf/parts/arms.urdf.xacro" />

Commit message: updates

File: kyon_urdf/urdf/config/kyon.urdf.xacro (robot description, xacro)
@@ -6,5 +6,4 @@
 <xacro:arg name="legs" default="true"/>
 <xacro:arg name="upper_body" default="true"/>
-<xacro:arg name="dagana" default="true"/>
 <xacro:arg name="feet" default="true"/>
 <xacro:arg name="wheels" default="false"/>
@@ -19,5 +18,4 @@
 <xacro:property name="ADD_UPPER_BODY" value="$(arg upper_body)" />
 <xacro:property name="ADD_SENSORS" value="$(arg sensors)" />
-<xacro:property name="ADD_DAGANA" value="$(arg dagana)"/>
 <xacro:property name="ADD_FEET" value="$(arg feet)"/>
 <xacro:property name="ADD_WHEELS" value="$(arg wheels)"/>

Commit message: footonly simplified collision (wip, only leg)

File: kyon_urdf/urdf/config/kyon.urdf.xacro (robot description, xacro)
@@ -8,4 +8,5 @@
 <xacro:arg name="dagana" default="true"/>
 <xacro:arg name="feet" default="true"/>
+<xacro:arg name="footonly_collision" default="false"/>
 <xacro:arg name="wheels" default="false"/>
 <xacro:arg name="floating_joint" default="true"/>
@@ -35,3 +36,4 @@
 <xacro:property name="ADD_VIRTUAL_FRAME" value="false" />
 <xacro:property name="PAYLOAD" value="$(arg payload)"/>
+<xacro:property name="FOOTONLY_COLLISION" value="$(arg footonly_collision)"/>
 </robot>

File: kyon_urdf/urdf/parts/foot_leg.urdf.xacro (robot description, xacro)
@@ -1,39 +1,60 @@
 <?xml version="1.0"?>
 <robot xmlns:xacro="http://ros.org/wiki/xacro">
-<!-- macro legs -->
-<xacro:macro name="foot_leg" params="leg_num parent origin_x origin_y mirror">
-<link name="knee_pitch_${leg_num}_link">
-    <inertial>
-        <origin xyz="${KneePitch_x} ${KneePitch_y} ${KneePitch_z}"/>
-        <mass value="${KneePitch_mass}"/>
-        <inertia ixx="${KneePitch_xx}" ixy="${mirror*KneePitch_xy}" ixz="${mirror*KneePitch_xz}" iyy="${KneePitch_yy}" iyz="${KneePitch_yz}" izz="${KneePitch_zz}"/>
-    </inertial>
-    <visual>
-        <origin xyz="0.0 0.0 0.0"  rpy="0.0 0.0 0.0"/>
-        <geometry>
-            <mesh filename="package://kyon_urdf/meshes/mesh_foot-leg.stl" scale="${mirror*0.001} 0.001 0.001"/>
-        </geometry>
-        <material name="dark_grey"/>
-    </visual>
-    <collision>
-        <origin xyz="0.0 0.0 0.0"  rpy="0.0 0.0 0.0"/>
-        <geometry>
-            <mesh filename="package://kyon_urdf/meshes/collision/mesh_foot-leg.stl" scale="${mirror*0.001} 0.001 0.001"/>
-        </geometry>
-    </collision>
-</link>
-<joint name="knee_pitch_${leg_num}" type="revolute">
-    <parent link="${parent}"/>
-    <child link="knee_pitch_${leg_num}_link"/>
-    <origin xyz="${KneePitch_Ox} ${KneePitch_Oy} ${KneePitch_Oz}" rpy="${KneePitch_roll} ${KneePitch_pitch} ${KneePitch_yaw}"/>
-    <axis xyz="0 0 1"/>
-    <limit lower="${knee_pitch_lower[leg_num-1]}" upper="${knee_pitch_upper[leg_num-1]}" effort="${motorA_effort}" velocity="${motorA_velocity}"/>
-</joint>
-<link name="contact_${leg_num}"/>
-<joint name="contact_${leg_num}_joint" type="fixed">
-    <parent link="knee_pitch_${leg_num}_link"/>
-    <child link="contact_${leg_num}"/>
-    <origin xyz="${-mirror*0.0} -0.3 0.054" rpy="${1.57*mirror} ${0} ${0.785 if mirror == -1 else 2.356}"/>
-</joint>
-</xacro:macro>
+    <!-- macro legs -->
+    <xacro:macro name="foot_leg" params="leg_num parent origin_x origin_y mirror footonly_collision=false">
+        <link name="knee_pitch_${leg_num}_link">
+            <inertial>
+                <origin xyz="${KneePitch_x} ${KneePitch_y} ${KneePitch_z}" />
+                <mass value="${KneePitch_mass}" />
+                <inertia ixx="${KneePitch_xx}" ixy="${mirror*KneePitch_xy}"
+                    ixz="${mirror*KneePitch_xz}" iyy="${KneePitch_yy}" iyz="${KneePitch_yz}"
+                    izz="${KneePitch_zz}" />
+            </inertial>
+            <visual>
+                <origin xyz="0.0 0.0 0.0" rpy="0.0 0.0 0.0" />
+                <geometry>
+                    <mesh filename="package://kyon_urdf/meshes/mesh_foot-leg.stl"
+                        scale="${mirror*0.001} 0.001 0.001" />
+                </geometry>
+                <material name="dark_grey" />
+            </visual>
+            <xacro:unless value="${footonly_collision}">
+                <collision>
+                    <origin xyz="0.0 0.0 0.0" rpy="0.0 0.0 0.0" />
+                    <geometry>
+                        <mesh filename="package://kyon_urdf/meshes/collision/mesh_foot-leg.stl"
+                            scale="${mirror*0.001} 0.001 0.001" />
+                    </geometry>
+                </collision>
+            </xacro:unless>
+        </link>
+        <joint name="knee_pitch_${leg_num}" type="revolute">
+            <parent link="${parent}" />
+            <child link="knee_pitch_${leg_num}_link" />
+            <origin xyz="${KneePitch_Ox} ${KneePitch_Oy} ${KneePitch_Oz}"
+                rpy="${KneePitch_roll} ${KneePitch_pitch} ${KneePitch_yaw}" />
+            <axis xyz="0 0 1" />
+            <limit lower="${knee_pitch_lower[leg_num-1]}" upper="${knee_pitch_upper[leg_num-1]}"
+                effort="${motorA_effort}" velocity="${motorA_velocity}" />
+        </joint>
+        <link name="contact_${leg_num}">
+            <xacro:if value="${footonly_collision}">
+                <collision name="contact_${leg_num}">
+                    <origin xyz="0.0 0.0 0.0" rpy="0.0 0.0 0.0" />
+                    <geometry>
+                        <sphere radius="0.03" />
+                    </geometry>
+                    <material>
+                        <color rgba="0 1.0 1.0 1.0" />
+                    </material>
+                </collision>
+            </xacro:if>
+        </link>
+        <joint name="contact_${leg_num}_joint" type="fixed">
+            <parent link="knee_pitch_${leg_num}_link" />
+            <child link="contact_${leg_num}" />
+            <origin xyz="${-mirror*0.0} -0.31 0.022"
+                rpy="${1.57*mirror} ${0} ${0.785 if mirror == -1 else 2.356}" />
+        </joint>
+    </xacro:macro>
 </robot>

File: kyon_urdf/urdf/parts/kyon_leg.urdf.xacro (robot description, xacro)
@@ -6,5 +6,5 @@
 <xacro:include filename="$(find kyon_urdf)/urdf/parts/wheel_leg.urdf.xacro"/>
 <!-- macro legs -->
-<xacro:macro name="kyon_leg" params="leg_num origin_x origin_y mirror">
+<xacro:macro name="kyon_leg" params="leg_num origin_x origin_y mirror footonly_collision=false">
 <!-- links -->
 <link name="hip_roll_${leg_num}_link">
@@ -22,4 +22,5 @@
   		<material name="dark_grey"/>
 	</visual>
+	<xacro:unless value="${footonly_collision}">
 	<collision>
 		<origin xyz="0.0 0.0 0.0"  rpy="0.0 0.0 0.0"/>
@@ -29,4 +30,5 @@
 		</geometry>
 	</collision>
+	</xacro:unless>
 </link>
 <link name="hip_pitch_${leg_num}_link">
@@ -43,4 +45,5 @@
   		<material name="dark_grey"/>
 	</visual>
+	<xacro:unless value="${footonly_collision}">
 	<collision>
 		<origin xyz="0.0 0.0 0.0"  rpy="0.0 0.0 0.0"/>
@@ -49,4 +52,5 @@
 		</geometry>
 	</collision>
+	</xacro:unless>
 </link>
 <!-- joints -->
@@ -66,5 +70,7 @@
 </joint>
 <xacro:if value="${ADD_FEET}">
-	<xacro:foot_leg leg_num="${leg_num}" parent="hip_pitch_${leg_num}_link" origin_x="${origin_x}" origin_y="${origin_y}" mirror="${mirror}"/>
+	<xacro:foot_leg leg_num="${leg_num}" parent="hip_pitch_${leg_num}_link"
+			origin_x="${origin_x}" origin_y="${origin_y}" mirror="${mirror}"
+			footonly_collision="${footonly_collision}"/>
 </xacro:if>
 <xacro:if value="${ADD_STEERING_WHEELS}">

File: kyon_urdf/urdf/parts/legs.urdf.xacro (robot description, xacro)
@@ -2,11 +2,11 @@
 <robot xmlns:xacro="http://ros.org/wiki/xacro">
 <xacro:include filename="$(find kyon_urdf)/urdf/parts/kyon_leg.urdf.xacro" />
-<xacro:kyon_leg leg_num="1" origin_x="1" origin_y="-1" mirror="-1">
+<xacro:kyon_leg leg_num="1" origin_x="1" origin_y="-1" mirror="-1" footonly_collision="${FOOTONLY_COLLISION}">
 </xacro:kyon_leg>
-<xacro:kyon_leg leg_num="2" origin_x="1" origin_y="1" mirror="1">
+<xacro:kyon_leg leg_num="2" origin_x="1" origin_y="1" mirror="1" footonly_collision="${FOOTONLY_COLLISION}">
 </xacro:kyon_leg>
-<xacro:kyon_leg leg_num="3" origin_x="-1" origin_y="-1" mirror="-1">
+<xacro:kyon_leg leg_num="3" origin_x="-1" origin_y="-1" mirror="-1" footonly_collision="${FOOTONLY_COLLISION}">
 </xacro:kyon_leg>
-<xacro:kyon_leg leg_num="4" origin_x="-1" origin_y="1" mirror="1">
+<xacro:kyon_leg leg_num="4" origin_x="-1" origin_y="1" mirror="1" footonly_collision="${FOOTONLY_COLLISION}">
 </xacro:kyon_leg>
 </robot>

Commit message: added foot contact collision

File: kyon_urdf/urdf/config/kyon.urdf.xacro (robot description, xacro)
@@ -14,4 +14,5 @@
 <xacro:arg name="velodyne" default="false"/>
 <xacro:arg name="dagana" default="$(arg upper_body)"/>
+<xacro:arg name="foot_contact_collision" default="true"/>
 <!-- ************SELECT PARTS*************-->
 <!-- *************************************-->
@@ -27,3 +28,4 @@
 <xacro:property name="ADD_VIRTUAL_FRAME" value="false" />
 <xacro:property name="PAYLOAD" value="$(arg payload)"/>
+<xacro:property name="FOOT_CONTACT_COLLISION" value="$(arg foot_contact_collision)"/>
 </robot>

File: kyon_urdf/urdf/parts/foot_leg.urdf.xacro (robot description, xacro)
@@ -30,9 +30,21 @@
     <limit lower="${knee_pitch_lower[leg_num-1]}" upper="${knee_pitch_upper[leg_num-1]}" effort="${motorA_effort}" velocity="${motorA_velocity}"/>
 </joint>
-<link name="contact_${leg_num}"/>
+<link name="contact_${leg_num}">
+    <xacro:if value="${FOOT_CONTACT_COLLISION}">
+        <collision name="contact_${leg_num}">
+            <origin xyz="0.0 0.0 0.0" rpy="0.0 0.0 0.0" />
+            <geometry>
+                <sphere radius="0.039" />
+            </geometry>
+            <material>
+                <color rgba="0 1.0 1.0 1.0" />
+            </material>
+        </collision>
+    </xacro:if>
+</link>
 <joint name="contact_${leg_num}_joint" type="fixed">
     <parent link="knee_pitch_${leg_num}_link"/>
     <child link="contact_${leg_num}"/>
-    <origin xyz="${-mirror*0.0} -0.3 0.054" rpy="${1.57*mirror} ${0} ${0.785 if mirror == -1 else 2.356}"/>
+    <origin xyz="${-mirror*0.0} -0.305 0.054" rpy="${1.57*mirror} ${0} ${0.785 if mirror == -1 else 2.356}"/>
 </joint>
 </xacro:macro>

Commit message: make mjlab happy

File: kyon_urdf/urdf/config/kyon.urdf.xacro (robot description, xacro)
@@ -28,4 +28,5 @@
 <xacro:property name="ADD_HESAI_JT128" value="$(arg hesai_jt128)"/>
 <xacro:property name="ADD_VIRTUAL_FRAME" value="false" />
+<xacro:property name="ADD_COLLISION" value="$(arg add_collision)"/>
 <xacro:property name="PAYLOAD" value="$(arg payload)"/>
 </robot>

File: kyon_urdf/urdf/kyon_base.urdf.xacro (robot description, xacro)
@@ -22,4 +22,5 @@
         <material name="dark_grey"/>
 	</visual>
+    <xacro:if value="${ADD_COLLISION}">
 	<collision>
 		<origin xyz="0.0 0 0.0"  rpy="0.0 0.0 0.0"/>
@@ -28,4 +29,5 @@
 		</geometry>
 	</collision>
+    </xacro:if>
 </link>
 <xacro:if value="${ADD_VARTA or ADD_D034_LI_ION}">

Commit message: make mjlab happy

File: kyon_urdf/urdf/config/kyon.urdf.xacro (robot description, xacro)
@@ -14,4 +14,5 @@
 <xacro:arg name="velodyne" default="false"/>
 <xacro:arg name="dagana" default="$(arg upper_body)"/>
+<xacro:arg name="add_collision" default="true"/>
 <!-- ************SELECT PARTS*************-->
 <!-- *************************************-->
@@ -26,4 +27,5 @@
 <xacro:property name="ADD_VELODYNE" value="$(arg velodyne)"/>
 <xacro:property name="ADD_VIRTUAL_FRAME" value="false" />
+<xacro:property name="ADD_COLLISION" value="$(arg add_collision)"/>
 <xacro:property name="PAYLOAD" value="$(arg payload)"/>
 </robot>

File: kyon_urdf/urdf/kyon_base.urdf.xacro (robot description, xacro)
@@ -22,4 +22,5 @@
         <material name="dark_grey"/>
 	</visual>
+    <xacro:if value="${ADD_COLLISION}">
 	<collision>
 		<origin xyz="0.0 0 0.0"  rpy="0.0 0.0 0.0"/>
@@ -28,4 +29,5 @@
 		</geometry>
 	</collision>
+    </xacro:if>
 </link>
 <xacro:if value="${ADD_VARTA or ADD_D034_LI_ION}">

File: kyon_urdf/urdf/parts/foot_leg.urdf.xacro (robot description, xacro)
@@ -16,4 +16,5 @@
         <material name="dark_grey"/>
     </visual>
+    <xacro:if value="${ADD_COLLISION}">
     <collision>
         <origin xyz="0.0 0.0 0.0"  rpy="0.0 0.0 0.0"/>
@@ -22,4 +23,5 @@
         </geometry>
     </collision>
+    </xacro:if>
 </link>
 <joint name="knee_pitch_${leg_num}" type="revolute">
@@ -30,5 +32,19 @@
     <limit lower="${knee_pitch_lower[leg_num-1]}" upper="${knee_pitch_upper[leg_num-1]}" effort="${motorA_effort}" velocity="${motorA_velocity}"/>
 </joint>
-<link name="contact_${leg_num}"/>
+<link name="contact_${leg_num}">
+    <visual>
+        <origin xyz="0 0 0" rpy="0 0 0"/>
+        <geometry>
+            <sphere radius="0.03"/>
+        </geometry>
+        <material name="white"/>
+    </visual>
+    <collision name="contact_${leg_num}">
+        <origin xyz="0 0 0" rpy="0 0 0"/>
+        <geometry>
+            <sphere radius="0.03"/>
+        </geometry>
+    </collision>
+</link>
 <joint name="contact_${leg_num}_joint" type="fixed">
     <parent link="knee_pitch_${leg_num}_link"/>

File: kyon_urdf/urdf/parts/kyon_leg.urdf.xacro (robot description, xacro)
@@ -22,4 +22,5 @@
   		<material name="dark_grey"/>
 	</visual>
+	<xacro:if value="${ADD_COLLISION}">
 	<collision>
 		<origin xyz="0.0 0.0 0.0"  rpy="0.0 0.0 0.0"/>
@@ -29,4 +30,5 @@
 		</geometry>
 	</collision>
+	</xacro:if>
 </link>
 <link name="hip_pitch_${leg_num}_link">
@@ -50,4 +52,5 @@
   		<material name="dark_grey"/>
 	</visual>
+	<xacro:if value="${ADD_COLLISION}">
 	<collision>
 		<origin xyz="0.0 0.0 0.0"  rpy="0.0 0.0 0.0"/>
@@ -57,4 +60,5 @@
 		<material name="kyon_orange"/>
 	</collision>
+	</xacro:if>
 </link>
 <!-- joints -->
