Commit message: fix cameras in gz

File: kyon_urdf/urdf/config/kyon.urdf.xacro (robot description, xacro)
@@ -8,5 +8,8 @@
 <xacro:arg name="wheels" default="false"/>
 <xacro:arg name="floating_joint" default="true"/>
-<xacro:arg name="cameras" default="false"/>
+<xacro:arg name="camera_front_up" default="false"/>
+<xacro:arg name="camera_front_down" default="false"/>
+<xacro:arg name="camera_left" default="false"/>
+<xacro:arg name="camera_right" default="false"/>
 <xacro:arg name="payload" default="false"/>
 <xacro:arg name="varta" default="false"/>
@@ -21,4 +24,8 @@
 <xacro:property name="ADD_DAGANA" value="$(arg dagana)"/>
 <xacro:property name="ADD_CAMERAS" value="$(arg cameras)"/>
+<xacro:property name="ADD_FU_CAMERA" value="$(arg camera_front_up)"/>
+<xacro:property name="ADD_FD_CAMERA" value="$(arg camera_front_down)"/>
+<xacro:property name="ADD_LEFT_CAMERA" value="$(arg camera_left)"/>
+<xacro:property name="ADD_RIGHT_CAMERA" value="$(arg camera_right)"/>
 <xacro:property name="ADD_WHEELS" value="$(arg wheels)"/>
 <xacro:property name="ADD_VARTA" value="$(arg varta)"/>

File: kyon_urdf/urdf/gazebo/kyon.gazebo.xacro (robot description, xacro)
@@ -2,31 +2,4 @@
 <robot xmlns:xacro="http://ros.org/wiki/xacro">
     <xacro:if value="${ADD_LEGS}">
-        <gazebo reference="imu_link">
-            <sensor name="imu_link" type="imu">
-                <always_on>1</always_on>
-                <update_rate>500</update_rate>
-                <visualize>true</visualize>
-                <topic>__default_topic__</topic>
-                <imu>
-                    <!--
-                <noise>
-                <type>gaussian</type>
-                <rate>
-                    <mean>0.0</mean>
-                    <stddev>2e-4</stddev>
-                    <bias_mean>0.0000075</bias_mean>
-                    <bias_stddev>0.0000008</bias_stddev>
-                </rate>
-                <accel>
-                    <mean>0.0</mean>
-                    <stddev>1.7e-2</stddev>
-                    <bias_mean>0.1</bias_mean>
-                    <bias_stddev>0.001</bias_stddev>
-                </accel>
-                </noise>
-                -->
-                </imu>
-            </sensor>
-        </gazebo>
         <gazebo reference="hip_roll_1">
             <implicitSpringDamper>1</implicitSpringDamper>

File: kyon_urdf/urdf/kyon_base.urdf.xacro (robot description, xacro)
@@ -86,91 +86,4 @@
     <origin xyz="0 -0.150100 0.109486" rpy="0 0.3490656 -1.5707963"/>
 </joint>
-<xacro:if value="${ADD_CAMERAS}">
-    <xacro:include filename="$(find realsense_gazebo_description)/urdf/_d435i.urdf.xacro" />
-    <!-- LEFT D435 CAMERA -->
-    <xacro:sensor_d435i parent="left_camera_mount_link"
-        name="D435_left"
-        topics_ns="D435_left"
-        enable_pointCloud="true"
-        align_depth="true"
-        unite_imu_method="false"
-        visualize="false"
-        accel_fps="300"
-        gyro_fps="300"
-        depth_width="1280"
-        depth_height="720"
-        depth_fps="10"
-        infra_width="1280"
-        infra_height="720"
-        infra_fps="10"
-        color_width="1280"
-        color_height="720"
-        color_fps="1">
-        <origin xyz="0 0 0" rpy="0 0 0"/>
-    </xacro:sensor_d435i>
-    <!-- RIGHT D435 CAMERA -->
-    <xacro:sensor_d435i parent="right_camera_mount_link"
-        name="D435_right"
-        topics_ns="D435_right"
-        enable_pointCloud="true"
-        align_depth="true"
-        unite_imu_method="false"
-        visualize="false"
-        accel_fps="300"
-        gyro_fps="300"
-        depth_width="1280"
-        depth_height="720"
-        depth_fps="10"
-        infra_width="1280"
-        infra_height="720"
-        infra_fps="10"
-        color_width="1280"
-        color_height="720"
-        color_fps="1">
-        <origin xyz="0 0 0" rpy="0 0 0"/>
-    </xacro:sensor_d435i>
-    <!-- FRONT1 D435 CAMERA -->
-    <xacro:sensor_d435i parent="zed_front_up_mount_link"
-        name="D435_front1"
-        topics_ns="D435_front1"
-        enable_pointCloud="true"
-        align_depth="true"
-        unite_imu_method="false"
-        visualize="false"
-        accel_fps="300"
-        gyro_fps="300"
-        depth_width="1280"
-        depth_height="720"
-        depth_fps="90"
-        infra_width="1280"
-        infra_height="720"
-        infra_fps="90"
-        color_width="1280"
-        color_height="720"
-        color_fps="30">
-        <origin xyz="0 0 0" rpy="0 0 0"/>
-    </xacro:sensor_d435i>
-    <!-- FRONT2 D435 CAMERA -->
-    <xacro:sensor_d435i parent="zed_front_down_mount_link"
-        name="D435_front2"
-        topics_ns="D435_front2"
-        enable_pointCloud="true"
-        align_depth="true"
-        unite_imu_method="false"
-        visualize="false"
-        accel_fps="300"
-        gyro_fps="300"
-        depth_width="1280"
-        depth_height="720"
-        depth_fps="90"
-        infra_width="1280"
-        infra_height="720"
-        infra_fps="90"
-        color_width="1280"
-        color_height="720"
-        color_fps="30">
-        <origin xyz="0 0 0" rpy="0 0 0"/>
-    </xacro:sensor_d435i>
-</xacro:if>
 <!-- Velodyne -->
 <link name="hesai_lidar"/>

Commit message: added fixed joint and boxy dagana

File: kyon_urdf/urdf/config/kyon.urdf.xacro (robot description, xacro)
@@ -16,4 +16,8 @@
 <xacro:arg name="add_collision" default="true"/>
 <xacro:arg name="hesai_jt128" default="false"/>
+<xacro:arg name="add_fixed_base_joint" default="false"/>
+<xacro:arg name="fixed_base_x" default="0.0"/>
+<xacro:arg name="fixed_base_y" default="0.0"/>
+<xacro:arg name="fixed_base_z" default="0.0"/>
 <!-- ************SELECT PARTS*************-->
 <!-- *************************************-->
@@ -32,3 +36,7 @@
 <xacro:property name="ADD_VIRTUAL_FRAME" value="false" />
 <xacro:property name="ADD_COLLISION" value="$(arg add_collision)"/>
+<xacro:property name="ADD_FIXED_BASE" value="$(arg add_fixed_base_joint)"/>
+<xacro:property name="FIXED_BASE_X" value="$(arg fixed_base_x)"/>
+<xacro:property name="FIXED_BASE_Y" value="$(arg fixed_base_y)"/>
+<xacro:property name="FIXED_BASE_Z" value="$(arg fixed_base_z)"/>
 </robot>

File: kyon_urdf/urdf/kyon.urdf.xacro (robot description, xacro)
@@ -16,3 +16,11 @@
 	</joint>
 </xacro:if>
+<xacro:if value="${ADD_FIXED_BASE}">
+	<link name="world"/>
+	<joint name="reference" type="fixed">
+		<parent link="world"/>
+		<child link="pelvis"/>
+		<origin xyz="${FIXED_BASE_X} ${FIXED_BASE_Y} ${FIXED_BASE_Z}"/>
+	</joint>
+</xacro:if>
 </robot>

File: kyon_urdf/urdf/parts/kyon_dagana.urdf.xacro (robot description, xacro)
@@ -12,7 +12,38 @@
         <origin xyz="0.0 0.0 0.0"  rpy="0.0 0.0 0.0"/>
         <geometry>
-            <mesh filename="package://kyon_urdf/meshes/mesh_dagana-base.stl" scale="0.001 0.001 0.001"/>
+            <mesh filename="package://kyon_urdf/meshes/mesh_dagana-base-boxy.stl" scale="0.001 0.001 0.001"/>
         </geometry>
         <material name="dark_grey"/>
+    </visual>
+    <visual>
+        <origin xyz="0 -0.0145 0.181" rpy="0 1.5707 0" />
+        <geometry>
+            <cylinder radius="0.01" length="0.0279"/>
+        </geometry>
+    </visual>
+    <visual>
+        <origin xyz="0.0 0.0007432 0.0405" rpy="0 0 0" />
+        <geometry>
+            <box size="0.0879  0.0844864 0.081"/>
+        </geometry>
+    </visual>
+    <collision>
+        <origin xyz="0.0 0.0 0.0"  rpy="0.0 0.0 0.0"/>
+        <geometry>
+            <mesh filename="package://kyon_urdf/meshes/mesh_dagana-base-boxy.stl" scale="0.001 0.001 0.001"/>
+        </geometry>
+        <material name="dark_grey"/>
+    </collision>
+    <collision>
+        <origin xyz="0 -0.0145 0.181" rpy="0 1.5707 0" />
+        <geometry>
+            <cylinder radius="0.01" length="0.0279"/>
+        </geometry>
+    </collision>
+    <visual>
+        <origin xyz="0.0 0.0007432 0.0405" rpy="0 0 0" />
+        <geometry>
+            <box size="0.0879  0.0844864 0.081"/>
+        </geometry>
     </visual>
     <!-- <collision>
@@ -38,8 +69,27 @@
         <origin xyz="0.0 0.0 0.0"  rpy="0.0 0.0 0.0"/>
         <geometry>
-            <mesh filename="package://kyon_urdf/meshes/mesh_dagana-clamp.stl" scale="0.001 0.001 0.001"/>
+            <mesh filename="package://kyon_urdf/meshes/mesh_dagana-clamp-boxy.stl" scale="0.001 0.001 0.001"/>
         </geometry>
         <material name="dark_grey"/>
     </visual>
+    <visual>
+        <origin xyz="-0.137 0.0 -0.0362125" rpy="0 0 0" />
+        <geometry>
+            <cylinder radius="0.01" length="0.0279"/>
+        </geometry>
+    </visual>
+    <collision>
+        <origin xyz="0.0 0.0 0.0"  rpy="0.0 0.0 0.0"/>
+        <geometry>
+            <mesh filename="package://kyon_urdf/meshes/mesh_dagana-clamp-boxy.stl" scale="0.001 0.001 0.001"/>
+        </geometry>
+        <material name="dark_grey"/>
+    </collision>
+    <collision>
+        <origin xyz="-0.137 0.0 -0.0362125" rpy="0 0 0" />
+        <geometry>
+            <cylinder radius="0.01" length="0.0279"/>
+        </geometry>
+    </collision>
     <!-- <collision>
         <origin xyz="0.0 0.0 0.0"  rpy="0.0 0.0 0.0"/>

Commit message: added fixed joint and boxy dagana

File: kyon_urdf/urdf/config/kyon.urdf.xacro (robot description, xacro)
@@ -18,4 +18,8 @@
 <xacro:arg name="add_collision" default="true"/>
 <xacro:arg name="hesai_jt128" default="false"/>
+<xacro:arg name="add_fixed_base_joint" default="false"/>
+<xacro:arg name="fixed_base_x" default="0.0"/>
+<xacro:arg name="fixed_base_y" default="0.0"/>
+<xacro:arg name="fixed_base_z" default="0.0"/>
 <!-- ************SELECT PARTS*************-->
 <!-- *************************************-->
@@ -36,3 +40,7 @@
 <xacro:property name="ADD_COLLISION" value="$(arg add_collision)"/>
 <xacro:property name="PAYLOAD" value="$(arg payload)"/>
+<xacro:property name="ADD_FIXED_BASE" value="$(arg add_fixed_base_joint)"/>
+<xacro:property name="FIXED_BASE_X" value="$(arg fixed_base_x)"/>
+<xacro:property name="FIXED_BASE_Y" value="$(arg fixed_base_y)"/>
+<xacro:property name="FIXED_BASE_Z" value="$(arg fixed_base_z)"/>
 </robot>

File: kyon_urdf/urdf/kyon.urdf.xacro (robot description, xacro)
@@ -16,3 +16,11 @@
 	</joint>
 </xacro:if>
+<xacro:if value="${ADD_FIXED_BASE}">
+	<link name="world"/>
+	<joint name="reference" type="fixed">
+		<parent link="world"/>
+		<child link="pelvis"/>
+		<origin xyz="${FIXED_BASE_X} ${FIXED_BASE_Y} ${FIXED_BASE_Z}"/>
+	</joint>
+</xacro:if>
 </robot>
