Commit message: Optional lowres meshes

File: kyon_urdf/urdf/config/kyon.urdf.xacro (robot description, xacro)
@@ -22,4 +22,5 @@
 <xacro:arg name="fixed_base_y" default="0.0"/>
 <xacro:arg name="fixed_base_z" default="0.0"/>
+<xacro:arg name="visual_mesh_subfolder" default="visual_lowres"/> <!-- pass an empty string to get the original high resolution meshes -->
 <!-- ************SELECT PARTS*************-->
 <!-- *************************************-->
@@ -29,4 +30,5 @@
 <xacro:property name="ADD_FU_CAMERA" value="$(arg camera_front_up)"/>
 <xacro:property name="ADD_FD_CAMERA" value="$(arg camera_front_down)"/>
+<xacro:property name="ADD_FD_ZED_MODEL" value="$(arg add_zed_model_front_down)"/>
 <xacro:property name="ADD_LEFT_CAMERA" value="$(arg camera_left)"/>
 <xacro:property name="ADD_RIGHT_CAMERA" value="$(arg camera_right)"/>
@@ -40,4 +42,5 @@
 <xacro:property name="ADD_COLLISION" value="$(arg add_collision)"/>
 <xacro:property name="PAYLOAD" value="$(arg payload)"/>
+<xacro:property name="VISUAL_MESH_SUBFOLDER" value="$(arg visual_mesh_subfolder)"/>
 <xacro:property name="ADD_FIXED_BASE" value="$(arg add_fixed_base_joint)"/>
 <xacro:property name="FIXED_BASE_X" value="$(arg fixed_base_x)"/>

File: kyon_urdf/urdf/parts/kyon_leg.urdf.xacro (robot description, xacro)
@@ -18,5 +18,5 @@
 	  	<geometry>
 	 		<!-- <cylinder radius="${cylinder_radius}" length="${cylinder_length}"/> -->
-			<mesh filename="package://kyon_urdf/meshes/mesh_hip-roll.stl" scale="0.001 ${mirror*0.001} 0.001"/>
+			<mesh filename="package://kyon_urdf/meshes/${VISUAL_MESH_SUBFOLDER}/mesh_hip-roll.stl" scale="0.001 ${mirror*0.001} 0.001"/>
 		</geometry>
   		<material name="dark_grey"/>
@@ -41,5 +41,5 @@
 		<origin xyz="0.0 0.0 0.0"  rpy="0.0 0.0 0.0"/>
 	  	<geometry>
-	 		<mesh filename="package://kyon_urdf/meshes/mesh_hip-pitch.stl" scale="0.001 0.001 0.001"/>
+	 		<mesh filename="package://kyon_urdf/meshes/${VISUAL_MESH_SUBFOLDER}/mesh_hip-pitch.stl" scale="0.001 0.001 0.001"/>
 	  	</geometry>
   		<material name="kyon_orange"/>
@@ -48,5 +48,5 @@
 		<origin xyz="0.0 0.0 0.0"  rpy="0.0 0.0 0.0"/>
 	  	<geometry>
-	 		<mesh filename="package://kyon_urdf/meshes/mesh_hip-pitch_cover.stl" scale="0.001 0.001 0.001"/>
+	 		<mesh filename="package://kyon_urdf/meshes/${VISUAL_MESH_SUBFOLDER}/mesh_hip-pitch_cover.stl" scale="0.001 0.001 0.001"/>
 	  	</geometry>
   		<material name="dark_grey"/>

Commit message: Optional lowres meshes

File: kyon_urdf/urdf/config/kyon.urdf.xacro (robot description, xacro)
@@ -20,4 +20,5 @@
 <xacro:arg name="fixed_base_y" default="0.0"/>
 <xacro:arg name="fixed_base_z" default="0.0"/>
+<xacro:arg name="visual_mesh_subfolder" default="visual_lowres"/> <!-- pass an empty string to get the original high resolution meshes -->
 <!-- ************SELECT PARTS*************-->
 <!-- *************************************-->
@@ -27,4 +28,5 @@
 <xacro:property name="ADD_FU_CAMERA" value="$(arg camera_front_up)"/>
 <xacro:property name="ADD_FD_CAMERA" value="$(arg camera_front_down)"/>
+<xacro:property name="ADD_FD_ZED_MODEL" value="$(arg add_zed_model_front_down)"/>
 <xacro:property name="ADD_LEFT_CAMERA" value="$(arg camera_left)"/>
 <xacro:property name="ADD_RIGHT_CAMERA" value="$(arg camera_right)"/>
@@ -36,4 +38,6 @@
 <xacro:property name="ADD_VIRTUAL_FRAME" value="false" />
 <xacro:property name="ADD_COLLISION" value="$(arg add_collision)"/>
+<xacro:property name="PAYLOAD" value="$(arg payload)"/>
+<xacro:property name="VISUAL_MESH_SUBFOLDER" value="$(arg visual_mesh_subfolder)"/>
 <xacro:property name="ADD_FIXED_BASE" value="$(arg add_fixed_base_joint)"/>
 <xacro:property name="FIXED_BASE_X" value="$(arg fixed_base_x)"/>

File: kyon_urdf/urdf/kyon_base.urdf.xacro (robot description, xacro)
@@ -18,5 +18,5 @@
 		<origin xyz="0.0 0 0.0"  rpy="0.0 0.0 0.0"/>
 		<geometry>
-	 		<mesh filename="package://kyon_urdf/meshes/mesh_pelvis.stl" scale="0.001 0.001 0.001"/>
+	 		<mesh filename="package://kyon_urdf/meshes/${VISUAL_MESH_SUBFOLDER}/mesh_pelvis.stl" scale="0.001 0.001 0.001"/>
 		</geometry>
         <material name="dark_grey"/>

File: kyon_urdf/urdf/parts/foot_leg.urdf.xacro (robot description, xacro)
@@ -12,5 +12,5 @@
         <origin xyz="0.0 0.0 0.0"  rpy="0.0 0.0 0.0"/>
         <geometry>
-            <mesh filename="package://kyon_urdf/meshes/mesh_foot-leg.stl" scale="${mirror*0.001} 0.001 0.001"/>
+            <mesh filename="package://kyon_urdf/meshes/${VISUAL_MESH_SUBFOLDER}/mesh_foot-leg.stl" scale="${mirror*0.001} 0.001 0.001"/>
         </geometry>
         <material name="dark_grey"/>

File: kyon_urdf/urdf/parts/kyon_arm.urdf.xacro (robot description, xacro)
@@ -15,5 +15,5 @@
 		<origin xyz="0.0 0.0 0.0"  rpy="0.0 0.0 0.0"/>
 		<geometry>
-			<mesh filename="package://kyon_urdf/meshes/mesh_sh-yaw.stl" scale="0.001 0.001 0.001"/>
+			<mesh filename="package://kyon_urdf/meshes/${VISUAL_MESH_SUBFOLDER}/mesh_sh-yaw.stl" scale="0.001 0.001 0.001"/>
 		</geometry>
 		<material name="dark_grey"/>
@@ -34,5 +34,5 @@
 	<visual>
 	  	<geometry>
-			<mesh filename="package://kyon_urdf/meshes/mesh_sh-pitch_cover.stl" scale="0.001 0.001 0.001"/>
+			<mesh filename="package://kyon_urdf/meshes/${VISUAL_MESH_SUBFOLDER}/mesh_sh-pitch_cover.stl" scale="0.001 0.001 0.001"/>
 	  	</geometry>
   		<material name="dark_grey"/>
@@ -40,5 +40,5 @@
 	<visual>
 	  	<geometry>
-	 		<mesh filename="package://kyon_urdf/meshes/mesh_sh-pitch.stl" scale="0.001 0.001 0.001"/>
+	 		<mesh filename="package://kyon_urdf/meshes/${VISUAL_MESH_SUBFOLDER}/mesh_sh-pitch.stl" scale="0.001 0.001 0.001"/>
 	  	</geometry>
   		<material name="kyon_orange"/>
@@ -59,5 +59,5 @@
 	<visual>
 		<geometry>
-			<mesh filename="package://kyon_urdf/meshes/mesh_elbow.stl" scale="0.001 0.001 0.001"/>
+			<mesh filename="package://kyon_urdf/meshes/${VISUAL_MESH_SUBFOLDER}/mesh_elbow.stl" scale="0.001 0.001 0.001"/>
 		</geometry>
 		<material name="dark_grey"/>
@@ -65,5 +65,5 @@
 	<collision>
 		<geometry>
-			<mesh filename="package://kyon_urdf/meshes/mesh_elbow.stl" scale="0.001 0.001 0.001"/>
+			<mesh filename="package://kyon_urdf/meshes/${VISUAL_MESH_SUBFOLDER}/mesh_elbow.stl" scale="0.001 0.001 0.001"/>
 		</geometry>
 	</collision>
@@ -78,5 +78,5 @@
 		<origin xyz="0.0 0.0 0.0"  rpy="0.0 0.0 0.0"/>
 	  	<geometry>
-	 		<mesh filename="package://kyon_urdf/meshes/mesh_wrist-pitch.stl" scale="0.001 0.001 0.001"/>
+	 		<mesh filename="package://kyon_urdf/meshes/${VISUAL_MESH_SUBFOLDER}/mesh_wrist-pitch.stl" scale="0.001 0.001 0.001"/>
 	  	</geometry>
   		<material name="dark_grey"/>
@@ -98,5 +98,5 @@
 		<origin xyz="0.0 0.0 0.0"  rpy="0.0 0.0 0.0"/>
 	  	<geometry>
-	 		<mesh filename="package://kyon_urdf/meshes/mesh_wrist-yaw.stl" scale="0.001 0.001 0.001"/>
+	 		<mesh filename="package://kyon_urdf/meshes/${VISUAL_MESH_SUBFOLDER}/mesh_wrist-yaw.stl" scale="0.001 0.001 0.001"/>
 	  	</geometry>
   		<material name="dark_grey"/>

File: kyon_urdf/urdf/parts/kyon_dagana.urdf.xacro (robot description, xacro)
@@ -12,5 +12,5 @@
         <origin xyz="0.0 0.0 0.0"  rpy="0.0 0.0 0.0"/>
         <geometry>
-            <mesh filename="package://kyon_urdf/meshes/mesh_dagana-base-boxy.stl" scale="0.001 0.001 0.001"/>
+            <mesh filename="package://kyon_urdf/meshes/${VISUAL_MESH_SUBFOLDER}/mesh_dagana-base-boxy.stl" scale="0.001 0.001 0.001"/>
         </geometry>
         <material name="dark_grey"/>
@@ -31,5 +31,5 @@
         <origin xyz="0.0 0.0 0.0"  rpy="0.0 0.0 0.0"/>
         <geometry>
-            <mesh filename="package://kyon_urdf/meshes/mesh_dagana-base-boxy.stl" scale="0.001 0.001 0.001"/>
+            <mesh filename="package://kyon_urdf/meshes/${VISUAL_MESH_SUBFOLDER}/mesh_dagana-base-boxy.stl" scale="0.001 0.001 0.001"/>
         </geometry>
         <material name="dark_grey"/>
@@ -69,5 +69,5 @@
         <origin xyz="0.0 0.0 0.0"  rpy="0.0 0.0 0.0"/>
         <geometry>
-            <mesh filename="package://kyon_urdf/meshes/mesh_dagana-clamp-boxy.stl" scale="0.001 0.001 0.001"/>
+            <mesh filename="package://kyon_urdf/meshes/${VISUAL_MESH_SUBFOLDER}/mesh_dagana-clamp-boxy.stl" scale="0.001 0.001 0.001"/>
         </geometry>
         <material name="dark_grey"/>
@@ -82,5 +82,5 @@
         <origin xyz="0.0 0.0 0.0"  rpy="0.0 0.0 0.0"/>
         <geometry>
-            <mesh filename="package://kyon_urdf/meshes/mesh_dagana-clamp-boxy.stl" scale="0.001 0.001 0.001"/>
+            <mesh filename="package://kyon_urdf/meshes/${VISUAL_MESH_SUBFOLDER}/mesh_dagana-clamp-boxy.stl" scale="0.001 0.001 0.001"/>
         </geometry>
         <material name="dark_grey"/>

File: kyon_urdf/urdf/parts/kyon_leg.urdf.xacro (robot description, xacro)
@@ -18,5 +18,5 @@
 	  	<geometry>
 	 		<!-- <cylinder radius="${cylinder_radius}" length="${cylinder_length}"/> -->
-			<mesh filename="package://kyon_urdf/meshes/mesh_hip-roll.stl" scale="0.001 ${mirror*0.001} 0.001"/>
+			<mesh filename="package://kyon_urdf/meshes/${VISUAL_MESH_SUBFOLDER}/mesh_hip-roll.stl" scale="0.001 ${mirror*0.001} 0.001"/>
 		</geometry>
   		<material name="dark_grey"/>
@@ -41,5 +41,5 @@
 		<origin xyz="0.0 0.0 0.0"  rpy="0.0 0.0 0.0"/>
 	  	<geometry>
-	 		<mesh filename="package://kyon_urdf/meshes/mesh_hip-pitch.stl" scale="0.001 0.001 0.001"/>
+	 		<mesh filename="package://kyon_urdf/meshes/${VISUAL_MESH_SUBFOLDER}/mesh_hip-pitch.stl" scale="0.001 0.001 0.001"/>
 	  	</geometry>
   		<material name="kyon_orange"/>
@@ -48,5 +48,5 @@
 		<origin xyz="0.0 0.0 0.0"  rpy="0.0 0.0 0.0"/>
 	  	<geometry>
-	 		<mesh filename="package://kyon_urdf/meshes/mesh_hip-pitch_cover.stl" scale="0.001 0.001 0.001"/>
+	 		<mesh filename="package://kyon_urdf/meshes/${VISUAL_MESH_SUBFOLDER}/mesh_hip-pitch_cover.stl" scale="0.001 0.001 0.001"/>
 	  	</geometry>
   		<material name="dark_grey"/>

File: kyon_urdf/urdf/parts/steering_wheel.urdf.xacro (robot description, xacro)
@@ -13,5 +13,5 @@
 	  	<geometry>
 	 		<!-- <cylinder radius="${cylinder_radius}" length="${cylinder_length}"/> -->
-			<mesh filename="package://kyon_urdf/meshes/mesh_knee-steering.stl" scale="0.001 0.001 0.001"/>
+			<mesh filename="package://kyon_urdf/meshes/${VISUAL_MESH_SUBFOLDER}/mesh_knee-steering.stl" scale="0.001 0.001 0.001"/>
 		</geometry>
   		<material name="dark_grey"/>
@@ -35,5 +35,5 @@
 	  	<geometry>
 	 		<!-- <cylinder radius="${cylinder_radius}" length="${cylinder_length}"/> -->
-			<mesh filename="package://kyon_urdf/meshes/mesh_ankle-yaw.stl" scale="0.001 0.001 0.001"/>
+			<mesh filename="package://kyon_urdf/meshes/${VISUAL_MESH_SUBFOLDER}/mesh_ankle-yaw.stl" scale="0.001 0.001 0.001"/>
 		</geometry>
   		<material name="dark_grey"/>
@@ -57,5 +57,5 @@
 	  	<geometry>
 	 		<!-- <cylinder radius="${cylinder_radius}" length="${cylinder_length}"/> -->
-			<mesh filename="package://kyon_urdf/meshes/mesh_wheel.stl" scale="0.001 0.001 0.001"/>
+			<mesh filename="package://kyon_urdf/meshes/${VISUAL_MESH_SUBFOLDER}/mesh_wheel.stl" scale="0.001 0.001 0.001"/>
 		</geometry>
   		<material name="light_grey"/>

File: kyon_urdf/urdf/parts/wheel_leg.urdf.xacro (robot description, xacro)
@@ -12,5 +12,5 @@
         <origin xyz="0.0 0.0 0.0"  rpy="0.0 0.0 0.0"/>
         <geometry>
-            <mesh filename="package://kyon_urdf/meshes/mesh_fixed-wheel-leg.stl" scale="${mirror*0.001} 0.001 0.001"/>
+            <mesh filename="package://kyon_urdf/meshes/${VISUAL_MESH_SUBFOLDER}/mesh_fixed-wheel-leg.stl" scale="${mirror*0.001} 0.001 0.001"/>
         </geometry>
         <material name="dark_grey"/>
@@ -32,5 +32,5 @@
 		<origin xyz="0.0 0.0 0.0"  rpy="0.0 0.0 0.0"/>
 	  	<geometry>
-			<mesh filename="package://kyon_urdf/meshes/mesh_wheel.stl" scale="0.001 0.001 0.001"/>
+			<mesh filename="package://kyon_urdf/meshes/${VISUAL_MESH_SUBFOLDER}/mesh_wheel.stl" scale="0.001 0.001 0.001"/>
 		</geometry>
   		<material name="dark_grey"/>

Commit message: referencing zed description to kyon xacro

File: kyon_urdf/urdf/config/kyon.urdf.xacro (robot description, xacro)
@@ -22,5 +22,4 @@
 <xacro:property name="ADD_LEGS" value="$(arg legs)"/>
 <xacro:property name="ADD_UPPER_BODY" value="$(arg upper_body)"/>
-<xacro:property name="ADD_CAMERAS" value="$(arg cameras)"/>
 <xacro:property name="ADD_FU_CAMERA" value="$(arg camera_front_up)"/>
 <xacro:property name="ADD_FD_CAMERA" value="$(arg camera_front_down)"/>

File: kyon_urdf/urdf/kyon.urdf.xacro (robot description, xacro)
@@ -6,4 +6,26 @@
 <!-- ************ CETC-SAT plain model ************ -->
 <xacro:include filename="$(find kyon_urdf)/urdf/kyon_base.urdf.xacro"/>
+<!-- ************ Optional ZED Mini cameras ************ -->
+<xacro:include filename="$(find zed_description)/urdf/zed_macro.urdf.xacro"/>
+<xacro:if value="${ADD_FU_CAMERA}">
+	<xacro:zed_camera name="zed_front_up" model="zedm">
+		<origin xyz="0 0 0" rpy="0 0 0"/>
+	</xacro:zed_camera>
+	<joint name="zed_front_up_camera_mount_joint" type="fixed">
+		<parent link="zed_front_up_mount_link"/>
+		<child link="zed_front_up_camera_link"/>
+		<origin xyz="0 0 0" rpy="0 0 0"/>
+	</joint>
+</xacro:if>
+<xacro:if value="${ADD_FD_CAMERA}">
+	<xacro:zed_camera name="zed_front_down" model="zedm">
+		<origin xyz="0 0 0" rpy="0 0 0"/>
+	</xacro:zed_camera>
+	<joint name="zed_front_down_camera_mount_joint" type="fixed">
+		<parent link="zed_front_down_mount_link"/>
+		<child link="zed_front_down_camera_link"/>
+		<origin xyz="0 0 0" rpy="0 0 0"/>
+	</joint>
+</xacro:if>
 <!-- ************ Control frames ************ -->
 <!--xacro:include filename="$(find pholus_urdf)/urdf/control_frames.urdf.xacro"/-->
