Commit message: feat(kyon): add selectable collision representations
- add tuned primitive collisions and simplified convex meshes\n- retain analytic wheel cylinders and continuous wheel joints\n- document the collision-model switch and geometry choices

File: kyon_urdf/urdf/config/kyon.urdf.xacro (robot description, xacro)
@@ -17,4 +17,5 @@
 <xacro:arg name="velodyne" default="false"/>
 <xacro:arg name="add_collision" default="true"/>
+<xacro:arg name="primitive_collisions" default="false"/>
 <xacro:arg name="hesai_jt128" default="false"/>
 <!-- ************SELECT PARTS*************-->
@@ -35,4 +36,5 @@
 <xacro:property name="ADD_VIRTUAL_FRAME" value="false" />
 <xacro:property name="ADD_COLLISION" value="$(arg add_collision)"/>
+<xacro:property name="USE_PRIMITIVE_COLLISIONS" value="$(arg primitive_collisions)"/>
 <xacro:property name="PAYLOAD" value="$(arg payload)"/>
 </robot>

File: kyon_urdf/urdf/kyon_base.urdf.xacro (robot description, xacro)
@@ -24,7 +24,10 @@
     <xacro:if value="${ADD_COLLISION}">
 	<collision>
-		<origin xyz="0.0 0 0.0"  rpy="0.0 0.0 0.0"/>
+		<!-- This remains the sole mesh in primitive-collision mode. Its
+		     100-triangle convex hull converts reliably, while an enclosing box
+		     creates false pelvis/shoulder collisions in the nominal posture. -->
+		<origin xyz="0 0 0" rpy="0 0 0"/>
 		<geometry>
-	  		<mesh filename="package://kyon_urdf/meshes/collision/mesh_pelvis.stl" scale="0.001 0.001 0.001"/>
+			<mesh filename="package://kyon_urdf/meshes/collision_simplified/mesh_pelvis.stl" scale="0.001 0.001 0.001"/>
 		</geometry>
 	</collision>

File: kyon_urdf/urdf/parts/foot_leg.urdf.xacro (robot description, xacro)
@@ -18,7 +18,17 @@
     <xacro:if value="${ADD_COLLISION}">
     <collision>
-        <origin xyz="0.0 0.0 0.0"  rpy="0.0 0.0 0.0"/>
+        <xacro:if value="${USE_PRIMITIVE_COLLISIONS}">
+            <origin xyz="0 -0.154688 0.021831" rpy="0 0 0"/>
+        </xacro:if>
+        <xacro:unless value="${USE_PRIMITIVE_COLLISIONS}">
+            <origin xyz="0 0 0" rpy="0 0 0"/>
+        </xacro:unless>
         <geometry>
-            <mesh filename="package://kyon_urdf/meshes/collision/mesh_foot-leg.stl" scale="${mirror*0.001} 0.001 0.001"/>
+            <xacro:if value="${USE_PRIMITIVE_COLLISIONS}">
+                <box size="0.079951 0.377576 0.043661"/>
+            </xacro:if>
+            <xacro:unless value="${USE_PRIMITIVE_COLLISIONS}">
+                <mesh filename="package://kyon_urdf/meshes/collision_simplified/mesh_foot-leg.stl" scale="${mirror*0.001} 0.001 0.001"/>
+            </xacro:unless>
         </geometry>
     </collision>

File: kyon_urdf/urdf/parts/kyon_arm.urdf.xacro (robot description, xacro)
@@ -19,10 +19,22 @@
 		<material name="dark_grey"/>
 	</visual>
-	<collision>
-		<origin xyz="0.0 0.0 0.0"  rpy="0.0 0.0 0.0"/>
-		<geometry>
-			<mesh filename="package://kyon_urdf/meshes/collision/mesh_sh-yaw.stl" scale="0.001 0.001 0.001"/>
-		</geometry>
-	</collision>
+	<xacro:if value="${ADD_COLLISION}">
+	<collision>
+		<xacro:if value="${USE_PRIMITIVE_COLLISIONS}">
+			<origin xyz="0 0 0.0465" rpy="0 0 0"/>
+		</xacro:if>
+		<xacro:unless value="${USE_PRIMITIVE_COLLISIONS}">
+			<origin xyz="0 0 0" rpy="0 0 0"/>
+		</xacro:unless>
+		<geometry>
+			<xacro:if value="${USE_PRIMITIVE_COLLISIONS}">
+				<box size="0.112 0.124 0.166"/>
+			</xacro:if>
+			<xacro:unless value="${USE_PRIMITIVE_COLLISIONS}">
+				<mesh filename="package://kyon_urdf/meshes/collision_simplified/mesh_sh-yaw.stl" scale="0.001 0.001 0.001"/>
+			</xacro:unless>
+		</geometry>
+	</collision>
+	</xacro:if>
 </link>
 <link name="shoulder_pitch_${arm_num}_link">
@@ -44,10 +56,20 @@
   		<material name="kyon_orange"/>
 	</visual>
-	<collision>
-	  	<geometry>
-			<mesh filename="package://kyon_urdf/meshes/collision/mesh_sh-pitch.stl" scale="0.001 0.001 0.001"/>
+	<xacro:if value="${ADD_COLLISION}">
+	<collision>
+		<xacro:if value="${USE_PRIMITIVE_COLLISIONS}">
+			<origin xyz="0.000013 -0.159507 -0.0155" rpy="0 0 0"/>
+		</xacro:if>
+	  	<geometry>
+			<xacro:if value="${USE_PRIMITIVE_COLLISIONS}">
+				<box size="0.111975 0.430987 0.089"/>
+			</xacro:if>
+			<xacro:unless value="${USE_PRIMITIVE_COLLISIONS}">
+				<mesh filename="package://kyon_urdf/meshes/collision_simplified/mesh_sh-pitch.stl" scale="0.001 0.001 0.001"/>
+			</xacro:unless>
 		</geometry>
 		<material name="kyon_orange"/>
 	</collision>
+	</xacro:if>
 </link>
 <link name="elbow_pitch_${arm_num}_link">
@@ -63,9 +85,19 @@
 		<material name="dark_grey"/>
 	</visual>
-	<collision>
-		<geometry>
-			<mesh filename="package://kyon_urdf/meshes/mesh_elbow.stl" scale="0.001 0.001 0.001"/>
-		</geometry>
-	</collision>
+	<xacro:if value="${ADD_COLLISION}">
+	<collision>
+		<xacro:if value="${USE_PRIMITIVE_COLLISIONS}">
+			<origin xyz="0 -0.1175 0.02936" rpy="0 0 0"/>
+		</xacro:if>
+		<geometry>
+			<xacro:if value="${USE_PRIMITIVE_COLLISIONS}">
+				<box size="0.11 0.345 0.058"/>
+			</xacro:if>
+			<xacro:unless value="${USE_PRIMITIVE_COLLISIONS}">
+				<mesh filename="package://kyon_urdf/meshes/collision_simplified/mesh_elbow.stl" scale="0.001 0.001 0.001"/>
+			</xacro:unless>
+		</geometry>
+	</collision>
+	</xacro:if>
 </link>
 <link name="wrist_pitch_${arm_num}_link">
@@ -82,10 +114,22 @@
   		<material name="dark_grey"/>
 	</visual>
-	<collision>
-		<origin xyz="0.0 0.0 0.0"  rpy="0.0 0.0 0.0"/>
-		<geometry>
-			<mesh filename="package://kyon_urdf/meshes/collision/mesh_wrist-pitch.stl" scale="0.001 0.001 0.001"/>
-		</geometry>
-	</collision>
+	<xacro:if value="${ADD_COLLISION}">
+	<collision>
+		<xacro:if value="${USE_PRIMITIVE_COLLISIONS}">
+			<origin xyz="0 -0.026 -0.011524" rpy="0 0 0"/>
+		</xacro:if>
+		<xacro:unless value="${USE_PRIMITIVE_COLLISIONS}">
+			<origin xyz="0 0 0" rpy="0 0 0"/>
+		</xacro:unless>
+		<geometry>
+			<xacro:if value="${USE_PRIMITIVE_COLLISIONS}">
+				<box size="0.08 0.132 0.104943"/>
+			</xacro:if>
+			<xacro:unless value="${USE_PRIMITIVE_COLLISIONS}">
+				<mesh filename="package://kyon_urdf/meshes/collision_simplified/mesh_wrist-pitch.stl" scale="0.001 0.001 0.001"/>
+			</xacro:unless>
+		</geometry>
+	</collision>
+	</xacro:if>
 </link>
 <link name="wrist_yaw_${arm_num}_link">
@@ -102,10 +146,22 @@
   		<material name="dark_grey"/>
 	</visual>
-	<collision>
-		<origin xyz="0.0 0.0 0.0"  rpy="0.0 0.0 0.0"/>
-		<geometry>
-			<mesh filename="package://kyon_urdf/meshes/collision/mesh_wrist-yaw.stl" scale="0.001 0.001 0.001"/>
-		</geometry>
-	</collision>
+	<xacro:if value="${ADD_COLLISION}">
+	<collision>
+		<xacro:if value="${USE_PRIMITIVE_COLLISIONS}">
+			<origin xyz="0 0 -0.02125" rpy="0 0 0"/>
+		</xacro:if>
+		<xacro:unless value="${USE_PRIMITIVE_COLLISIONS}">
+			<origin xyz="0 0 0" rpy="0 0 0"/>
+		</xacro:unless>
+		<geometry>
+			<xacro:if value="${USE_PRIMITIVE_COLLISIONS}">
+				<box size="0.079994 0.08 0.0425"/>
+			</xacro:if>
+			<xacro:unless value="${USE_PRIMITIVE_COLLISIONS}">
+				<mesh filename="package://kyon_urdf/meshes/collision_simplified/mesh_wrist-yaw.stl" scale="0.001 0.001 0.001"/>
+			</xacro:unless>
+		</geometry>
+	</collision>
+	</xacro:if>
 </link>
 <!-- /LINKS -->

File: kyon_urdf/urdf/parts/kyon_leg.urdf.xacro (robot description, xacro)
@@ -23,11 +23,12 @@
 	</visual>
 	<xacro:if value="${ADD_COLLISION}">
+	<xacro:unless value="${USE_PRIMITIVE_COLLISIONS}">
 	<collision>
-		<origin xyz="0.0 0.0 0.0"  rpy="0.0 0.0 0.0"/>
+		<origin xyz="0 0 0" rpy="0 0 0"/>
 		<geometry>
-	 		<!-- <cylinder radius="${cylinder_radius}" length="${cylinder_length}"/> -->
-			<mesh filename="package://kyon_urdf/meshes/collision/mesh_hip-roll.stl" scale="0.001 ${mirror*0.001} 0.001"/>
+			<mesh filename="package://kyon_urdf/meshes/collision_simplified/mesh_hip-roll.stl" scale="0.001 ${mirror*0.001} 0.001"/>
 		</geometry>
 	</collision>
+	</xacro:unless>
 	</xacro:if>
 </link>
@@ -54,7 +55,17 @@
 	<xacro:if value="${ADD_COLLISION}">
 	<collision>
-		<origin xyz="0.0 0.0 0.0"  rpy="0.0 0.0 0.0"/>
+		<xacro:if value="${USE_PRIMITIVE_COLLISIONS}">
+			<origin xyz="0 -0.165 0.19736" rpy="0 0 0"/>
+		</xacro:if>
+		<xacro:unless value="${USE_PRIMITIVE_COLLISIONS}">
+			<origin xyz="0 0 0" rpy="0 0 0"/>
+		</xacro:unless>
 		<geometry>
-			<mesh filename="package://kyon_urdf/meshes/collision/mesh_hip-pitch.stl" scale="0.001 0.001 0.001"/>
+			<xacro:if value="${USE_PRIMITIVE_COLLISIONS}">
+				<box size="0.138 0.468 0.094"/>
+			</xacro:if>
+			<xacro:unless value="${USE_PRIMITIVE_COLLISIONS}">
+				<mesh filename="package://kyon_urdf/meshes/collision_simplified/mesh_hip-pitch.stl" scale="0.001 0.001 0.001"/>
+			</xacro:unless>
 		</geometry>
 		<material name="kyon_orange"/>

File: kyon_urdf/urdf/parts/steering_wheel.urdf.xacro (robot description, xacro)
@@ -17,11 +17,22 @@
   		<material name="dark_grey"/>
 	</visual>
+	<xacro:if value="${ADD_COLLISION}">
 	<collision>
-		<origin xyz="0.0 0.0 0.0"  rpy="0.0 0.0 0.0"/>
+		<xacro:if value="${USE_PRIMITIVE_COLLISIONS}">
+			<origin xyz="0 0.005 0.055995" rpy="0 0 0"/>
+		</xacro:if>
+		<xacro:unless value="${USE_PRIMITIVE_COLLISIONS}">
+			<origin xyz="0 0 0" rpy="0 0 0"/>
+		</xacro:unless>
 		<geometry>
-	 		<!-- <cylinder radius="${cylinder_radius}" length="${cylinder_length}"/> -->
-			<mesh filename="package://kyon_urdf/meshes/collision/mesh_knee-steering.stl" scale="0.001 0.001 0.001"/>
+			<xacro:if value="${USE_PRIMITIVE_COLLISIONS}">
+				<box size="0.073333 0.076667 0.10"/>
+			</xacro:if>
+			<xacro:unless value="${USE_PRIMITIVE_COLLISIONS}">
+				<mesh filename="package://kyon_urdf/meshes/collision_simplified/mesh_knee-steering.stl" scale="0.001 0.001 0.001"/>
+			</xacro:unless>
 		</geometry>
 	</collision>
+	</xacro:if>
 </link>
 <link name="ankle_yaw_${leg_num}_link">
@@ -39,11 +50,22 @@
   		<material name="dark_grey"/>
 	</visual>
+	<xacro:if value="${ADD_COLLISION}">
 	<collision>
-		<origin xyz="0.0 0.0 0.0"  rpy="0.0 0.0 0.0"/>
+		<xacro:if value="${USE_PRIMITIVE_COLLISIONS}">
+			<origin xyz="0 -0.0025 -0.035" rpy="0 0 0"/>
+		</xacro:if>
+		<xacro:unless value="${USE_PRIMITIVE_COLLISIONS}">
+			<origin xyz="0 0 0" rpy="0 0 0"/>
+		</xacro:unless>
 		<geometry>
-	 		<!-- <cylinder radius="${cylinder_radius}" length="${cylinder_length}"/> -->
-			<mesh filename="package://kyon_urdf/meshes/collision/mesh_ankle-yaw.stl" scale="0.001 0.001 0.001"/>
+			<xacro:if value="${USE_PRIMITIVE_COLLISIONS}">
+				<box size="0.073333 0.076667 0.14"/>
+			</xacro:if>
+			<xacro:unless value="${USE_PRIMITIVE_COLLISIONS}">
+				<mesh filename="package://kyon_urdf/meshes/collision_simplified/mesh_ankle-yaw.stl" scale="0.001 0.001 0.001"/>
+			</xacro:unless>
 		</geometry>
 	</collision>
+	</xacro:if>
 </link>
 <link name="wheel_${leg_num}">
@@ -61,12 +83,13 @@
   		<material name="light_grey"/>
 	</visual>
+	<xacro:if value="${ADD_COLLISION}">
 	<collision>
-		<origin xyz="0.0 0.0 0.0"  rpy="0.0 0.0 0.0"/>
+		<origin xyz="0 0 0.005" rpy="0 0 0"/>
 		<geometry>
-	 		<!-- <cylinder radius="${cylinder_radius}" length="${cylinder_length}"/> -->
-			<mesh filename="package://kyon_urdf/meshes/collision/mesh_wheel.stl" scale="0.001 0.001 0.001"/>
+			<cylinder radius="0.107" length="0.0596"/>
 		</geometry>
 		<material name="light_grey"/>
 	</collision>
+	</xacro:if>
 </link>
 <joint name="knee_pitch_${leg_num}" type="revolute">
@@ -84,10 +107,10 @@
     <limit lower="${ankle_yaw_lower[leg_num-1]}" upper="${ankle_yaw_upper[leg_num-1]}" effort="${motorA_effort}" velocity="${motorA_velocity}"/>
 </joint>
-<joint name="wheel_joint_${leg_num}" type="revolute">
+<joint name="wheel_joint_${leg_num}" type="continuous">
     <parent link="ankle_yaw_${leg_num}_link"/>
     <child link="wheel_${leg_num}"/>
     <origin xyz="${SteeringWheel_Ox} ${SteeringWheel_Oy} ${SteeringWheel_Oz}" rpy="${SteeringWheel_roll} ${SteeringWheel_pitch} ${SteeringWheel_yaw}"/>
     <axis xyz="0 0 1"/>
-    <limit lower="-1e9" upper="1e9" effort="${motorWheel_effort}" velocity="${motorWheel_velocity}"/>
+    <limit effort="${motorWheel_effort}" velocity="${motorWheel_velocity}"/>
 </joint>
 <joint name="contact_joint_${leg_num}" type="fixed">

File: kyon_urdf/urdf/parts/wheel_leg.urdf.xacro (robot description, xacro)
@@ -16,10 +16,22 @@
         <material name="dark_grey"/>
     </visual>
+    <xacro:if value="${ADD_COLLISION}">
     <collision>
-        <origin xyz="0.0 0.0 0.0"  rpy="0.0 0.0 0.0"/>
+        <xacro:if value="${USE_PRIMITIVE_COLLISIONS}">
+            <origin xyz="0 -0.15925 0.02785" rpy="0 0 0"/>
+        </xacro:if>
+        <xacro:unless value="${USE_PRIMITIVE_COLLISIONS}">
+            <origin xyz="0 0 0" rpy="0 0 0"/>
+        </xacro:unless>
         <geometry>
-            <mesh filename="package://kyon_urdf/meshes/collision/mesh_fixed-wheel-leg.stl" scale="${mirror*0.001} 0.001 0.001"/>
+            <xacro:if value="${USE_PRIMITIVE_COLLISIONS}">
+                <box size="0.111997 0.3935 0.0607"/>
+            </xacro:if>
+            <xacro:unless value="${USE_PRIMITIVE_COLLISIONS}">
+                <mesh filename="package://kyon_urdf/meshes/collision_simplified/mesh_fixed-wheel-leg.stl" scale="${mirror*0.001} 0.001 0.001"/>
+            </xacro:unless>
         </geometry>
     </collision>
+    </xacro:if>
 </link>
 <link name="wheel_${leg_num}">
@@ -36,11 +48,12 @@
   		<material name="dark_grey"/>
 	</visual>
+	<xacro:if value="${ADD_COLLISION}">
 	<collision>
-		<origin xyz="0.0 0.0 0.0"  rpy="0.0 0.0 0.0"/>
+		<origin xyz="0 0 0.005" rpy="0 0 0"/>
 		<geometry>
-			<!-- <mesh filename="package://kyon_urdf/meshes/collision/mesh_wheel.stl" scale="0.001 0.001 0.001"/> -->
-            <cylinder radius="0.11" length="0.045"/>
+			<cylinder radius="0.107" length="0.0596"/>
 		</geometry>
 	</collision>
+	</xacro:if>
 </link>
 <link name="contact_${leg_num}"/>

Commit message: feet?

File: kyon_urdf/urdf/config/kyon.urdf.xacro (robot description, xacro)
@@ -7,4 +7,5 @@
 <xacro:arg name="upper_body" default="true"/>
 <xacro:arg name="wheels" default="false"/>
+<xacro:arg name="feet" default="false"/>
 <xacro:arg name="floating_joint" default="true"/>
 <xacro:arg name="camera_front_up" default="false"/>
@@ -34,4 +35,6 @@
 <xacro:property name="ADD_RIGHT_CAMERA" value="$(arg camera_right)"/>
 <xacro:property name="ADD_WHEELS" value="$(arg wheels)"/>
+<!-- Flat feet instead of the contact spheres: the wheeled leg with a foot plate in place of the wheel -->
+<xacro:property name="ADD_FEET" value="$(arg feet)"/>
 <xacro:property name="ADD_VARTA" value="$(arg varta)"/>
 <xacro:property name="ADD_D034_LI_ION" value="$(arg d034_li_ion)"/>

File: kyon_urdf/urdf/parts/kyon_leg.urdf.xacro (robot description, xacro)
@@ -3,4 +3,5 @@
 <!-- include end-effectors -->
 <xacro:include filename="$(find kyon_urdf)/urdf/parts/foot_leg.urdf.xacro"/>
+<xacro:include filename="$(find kyon_urdf)/urdf/parts/foot_plate_leg.urdf.xacro"/>
 <xacro:include filename="$(find kyon_urdf)/urdf/parts/steering_wheel.urdf.xacro"/>
 <xacro:include filename="$(find kyon_urdf)/urdf/parts/wheel_leg.urdf.xacro"/>
@@ -78,5 +79,10 @@
 </joint>
 <xacro:unless value="${ADD_WHEELS}">
-	<xacro:foot_leg leg_num="${leg_num}" parent="hip_pitch_${leg_num}_link" origin_x="${origin_x}" origin_y="${origin_y}" mirror="${mirror}"/>
+	<xacro:if value="${ADD_FEET}">
+		<xacro:foot_plate_leg leg_num="${leg_num}" parent="hip_pitch_${leg_num}_link" origin_x="${origin_x}" origin_y="${origin_y}" mirror="${mirror}"/>
+	</xacro:if>
+	<xacro:unless value="${ADD_FEET}">
+		<xacro:foot_leg leg_num="${leg_num}" parent="hip_pitch_${leg_num}_link" origin_x="${origin_x}" origin_y="${origin_y}" mirror="${mirror}"/>
+	</xacro:unless>
 </xacro:unless>
 <xacro:if value="${ADD_WHEELS}">

File: kyon_urdf/urdf/parts/limits.urdf.xacro (robot description, xacro)
@@ -10,4 +10,6 @@
 <xacro:property name="ankle_yaw_lower" value="${[-3.0, -3.0, -3.0, -3.0]}"/>
 <xacro:property name="ankle_yaw_upper" value="${[ 3.0,  3.0,  3.0,  3.0]}"/>
+<xacro:property name="ankle_pitch_lower" value="${[-1.3, -1.3, -1.3, -1.3]}"/>
+<xacro:property name="ankle_pitch_upper" value="${[ 1.3,  1.3,  1.3,  1.3]}"/>
 <!-- Arms -->
 <xacro:property name="j_shoulder_yaw_lower" value="${[-3.0, -3.0]}"/>
